File: schematic/cells/sheets/gate_trigger_input.kicad_sch (KiCad schematic)
At the start: 11 parts, among them J1208 PORT_LOAD, J1209 PORT_LOAD, J1210 PORT_LOAD, J1211 PORT_LOAD, U1206 LM393BIDR, U1207 SN74HC14DR

Commit message: Close master schematic integration gates
Audit locked panel coverage, netlist parity, sensitive islands and all active units; terminate spare cells, refresh evidence, and record rail budget overshoot and draft exports.
Connections:
- net +5V: now also U1206.6 (-)
- net AGND: now also U1206.5 (+), U1207.11, U1207.13, U1207.3, U1207.5, U1207.9
- no-connect marks 17 -> 10
Changed lines of the file:
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@@
     ))
   )
-  (no_connect (at 347.98 48.26))
-  (no_connect (at 347.98 53.34))
+  (global_label "AGND" (shape passive) (at 347.98 48.26 0) (effects (font (size 1.27 1.27)) (justify right)))
+  (global_label "+5V" (shape passive) (at 347.98 53.34 0) (effects (font (size 1.27 1.27)) (justify right)))
   (no_connect (at 363.22 50.8))
   (symbol (lib_id "zudo-osc-hole-field:LM393BIDR") (at 50.8 76.2 0) (unit 3)
@@
     ))
   )
-  (no_connect (at 144.78 76.2))
+  (global_label "AGND" (shape passive) (at 144.78 76.2 0) (effects (font (size 1.27 1.27)) (justify right)))
   (no_connect (at 160.02 76.2))
   (symbol (lib_id "zudo-osc-hole-field:SN74HC14DR") (at 203.2 76.2 0) (unit 3)
@@
     ))
   )
-  (no_connect (at 195.58 76.2))
+  (global_label "AGND" (shape passive) (at 195.58 76.2 0) (effects (font (size 1.27 1.27)) (justify right)))
   (no_connect (at 210.82 76.2))
   (symbol (lib_id "zudo-osc-hole-field:SN74HC14DR") (at 254 76.2 0) (unit 4)
@@
   )
   (no_connect (at 261.62 76.2))
-  (no_connect (at 246.38 76.2))
+  (global_label "AGND" (shape passive) (at 246.38 76.2 0) (effects (font (size 1.27 1.27)) (justify right)))
   (symbol (lib_id "zudo-osc-hole-field:SN74HC14DR") (at 304.8 76.2 0) (unit 5)
     (exclude_from_sim no) (in_bom yes) (on_board yes) (dnp no)
@@
   )
   (no_connect (at 312.42 76.2))
-  (no_connect (at 297.18 76.2))
+  (global_label "AGND" (shape passive) (at 297.18 76.2 0) (effects (font (size 1.27 1.27)) (justify right)))
   (symbol (lib_id "zudo-osc-hole-field:SN74HC14DR") (at 355.6 76.2 0) (unit 6)
     (exclude_from_sim no) (in_bom yes) (on_board yes) (dnp no)
@@
   )
   (no_connect (at 363.22 76.2))
-  (no_connect (at 347.98 76.2))
+  (global_label "AGND" (shape passive) (at 347.98 76.2 0) (effects (font (size 1.27 1.27)) (justify right)))
   (symbol (lib_id "zudo-osc-hole-field:SN74HC14DR") (at 50.8 101.6 0) (unit 7)
     (exclude_from_sim no) (in_bom yes) (on_board yes) (dnp no)
