File: schematic/cells/sheets/slew_island.kicad_sch (KiCad schematic)
At the start: 9 parts, among them U1901 OPA4197IPWR, U1909 OPA4197IPWR

Commit message: Close master schematic integration gates
Audit locked panel coverage, netlist parity, sensitive islands and all active units; terminate spare cells, refresh evidence, and record rail budget overshoot and draft exports.
Connections:
- net AGND: now also U1901.10 (+), U1901.12 (+), U1901.5 (+), U1909.10 (+), U1909.12 (+), U1909.5 (+)
- net slew_island_C_H1_SLEW___POST_SPARE_3: now reaches U1909.8
- net slew_island_C_H1_SLEW___POST_SPARE_3: now also U1909.9 (-)
- net slew_island_C_H1_SLEW___PRE_SPARE_3: now reaches U1901.8
- net slew_island_C_H1_SLEW___PRE_SPARE_3: now also U1901.9 (-)
- net slew_island_C_H1_SLEW___PRE_SPARE_4: now reaches U1901.13 (-)
- net slew_island_C_H1_SLEW___PRE_SPARE_4: now also U1901.14
- net slew_island_C_H1_SLEW___PRE_SPARE_2: now reaches U1901.6 (-)
- net slew_island_C_H1_SLEW___PRE_SPARE_2: now also U1901.7
- net slew_island_C_H1_SLEW___POST_SPARE_4: now reaches U1909.13 (-)
- net slew_island_C_H1_SLEW___POST_SPARE_4: now also U1909.14
- net slew_island_C_H1_SLEW___POST_SPARE_2: now reaches U1909.6 (-)
- net slew_island_C_H1_SLEW___POST_SPARE_2: now also U1909.7
- no-connect marks 20 -> 2
Changed lines of the file:
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@@
     ))
   )
-  (no_connect (at 93.98 48.26))
-  (no_connect (at 93.98 53.34))
-  (no_connect (at 109.22 50.8))
+  (global_label "AGND" (shape passive) (at 93.98 48.26 0) (effects (font (size 1.27 1.27)) (justify right)))
+  (label "slew_island_C_H1_SLEW___PRE_SPARE_2" (at 93.98 53.34 0) (effects (font (size 1.27 1.27)) (justify right)))
+  (label "slew_island_C_H1_SLEW___PRE_SPARE_2" (at 109.22 50.8 180) (effects (font (size 1.27 1.27)) (justify left)))
   (symbol (lib_id "zudo-osc-hole-field:OPA4197IPWR") (at 152.4 50.8 0) (unit 3)
     (exclude_from_sim no) (in_bom yes) (on_board yes) (dnp no)
@@
     ))
   )
-  (no_connect (at 160.02 50.8))
-  (no_connect (at 144.78 53.34))
-  (no_connect (at 144.78 48.26))
+  (label "slew_island_C_H1_SLEW___PRE_SPARE_3" (at 160.02 50.8 180) (effects (font (size 1.27 1.27)) (justify left)))
+  (label "slew_island_C_H1_SLEW___PRE_SPARE_3" (at 144.78 53.34 0) (effects (font (size 1.27 1.27)) (justify right)))
+  (global_label "AGND" (shape passive) (at 144.78 48.26 0) (effects (font (size 1.27 1.27)) (justify right)))
   (symbol (lib_id "zudo-osc-hole-field:OPA4197IPWR") (at 203.2 50.8 0) (unit 4)
     (exclude_from_sim no) (in_bom yes) (on_board yes) (dnp no)
@@
     ))
   )
-  (no_connect (at 195.58 48.26))
-  (no_connect (at 195.58 53.34))
-  (no_connect (at 210.82 50.8))
+  (global_label "AGND" (shape passive) (at 195.58 48.26 0) (effects (font (size 1.27 1.27)) (justify right)))
+  (label "slew_island_C_H1_SLEW___PRE_SPARE_4" (at 195.58 53.34 0) (effects (font (size 1.27 1.27)) (justify right)))
+  (label "slew_island_C_H1_SLEW___PRE_SPARE_4" (at 210.82 50.8 180) (effects (font (size 1.27 1.27)) (justify left)))
   (symbol (lib_id "zudo-osc-hole-field:OPA4197IPWR") (at 254 50.8 0) (unit 5)
     (exclude_from_sim no) (in_bom yes) (on_board yes) (dnp no)
@@
     ))
   )
-  (no_connect (at 347.98 73.66))
-  (no_connect (at 347.98 78.74))
-  (no_connect (at 363.22 76.2))
+  (global_label "AGND" (shape passive) (at 347.98 73.66 0) (effects (font (size 1.27 1.27)) (justify right)))
+  (label "slew_island_C_H1_SLEW___POST_SPARE_2" (at 347.98 78.74 0) (effects (font (size 1.27 1.27)) (justify right)))
+  (label "slew_island_C_H1_SLEW___POST_SPARE_2" (at 363.22 76.2 180) (effects (font (size 1.27 1.27)) (justify left)))
   (symbol (lib_id "zudo-osc-hole-field:OPA4197IPWR") (at 50.8 101.6 0) (unit 3)
     (exclude_from_sim no) (in_bom yes) (on_board yes) (dnp no)
@@
     ))
   )
-  (no_connect (at 58.42 101.6))
-  (no_connect (at 43.18 104.14))
-  (no_connect (at 43.18 99.06))
+  (label "slew_island_C_H1_SLEW___POST_SPARE_3" (at 58.42 101.6 180) (effects (font (size 1.27 1.27)) (justify left)))
+  (label "slew_island_C_H1_SLEW___POST_SPARE_3" (at 43.18 104.14 0) (effects (font (size 1.27 1.27)) (justify right)))
+  (global_label "AGND" (shape passive) (at 43.18 99.06 0) (effects (font (size 1.27 1.27)) (justify right)))
   (symbol (lib_id "zudo-osc-hole-field:OPA4197IPWR") (at 101.6 101.6 0) (unit 4)
     (exclude_from_sim no) (in_bom yes) (on_board yes) (dnp no)
@@
     ))
   )
-  (no_connect (at 93.98 99.06))
-  (no_connect (at 93.98 104.14))
-  (no_connect (at 109.22 101.6))
+  (global_label "AGND" (shape passive) (at 93.98 99.06 0) (effects (font (size 1.27 1.27)) (justify right)))
+  (label "slew_island_C_H1_SLEW___POST_SPARE_4" (at 93.98 104.14 0) (effects (font (size 1.27 1.27)) (justify right)))
+  (label "slew_island_C_H1_SLEW___POST_SPARE_4" (at 109.22 101.6 180) (effects (font (size 1.27 1.27)) (justify left)))
   (symbol (lib_id "zudo-osc-hole-field:OPA4197IPWR") (at 152.4 101.6 0) (unit 5)
     (exclude_from_sim no) (in_bom yes) (on_board yes) (dnp no)
