File: schematic/sheets/noise.kicad_sch (KiCad schematic)
At the start: 56 parts, among them J1109 WQP518MA, J1110 WQP518MA, J1209 WQP518MA, J1210 WQP518MA, U6101 NOISE2, U6102 OPA4196IDR, U6103 OPA4196IDR, U6104 OPA4196IDR, U6105 OPA4196IDR

Commit message: Refine source I/O regions and preserve whole package boundaries
Parts:
- C6101, C6102, C6103, C6104, C6105, C6106, C6107, C6108, C6109, R6101, R6102, R6103, R6104, R6105, R6106, R6107, R6108, R6109, R6110, R6111, R6114, R6115, R6118, R6119, R6122, R6123, RV6101, RV6102, RV6103, RV6104, U6101, U6102, U6103: BoardRegion (none) -> core
- C6110: BoardRegion (none) -> core; Decouples (none) -> SOURCE; Island NOISE_ANALOG -> NOISE_DIGITAL
- C6111, C6112: BoardRegion (none) -> core; Decouples (none) -> PACK_OPA4196IDR_0; Island NOISE_ANALOG -> IO_CORE:${SHEETNAME}
- C6113, C6114: BoardRegion (none) -> core; Decouples (none) -> PACK_OPA4196IDR_1; Island NOISE_ANALOG -> IO_CORE:${SHEETNAME}
- C6115, C6116: BoardRegion (none) -> core; Decouples (none) -> PACK_OPA4196IDR_2; Island NOISE_ANALOG -> IO_CORE:${SHEETNAME}
- C6117, C6118: BoardRegion (none) -> jack; Decouples (none) -> PACK_OPA4196IDR_3; Island NOISE_ANALOG -> IO_JACK:${SHEETNAME}
- J1109, J1110, J1209, J1210: BoardRegion (none) -> jack; Island (none) -> IO_JACK:${SHEETNAME}
- R6112, R6113, R6116, R6117, R6120, R6121, R6124, R6125, U6105: BoardRegion (none) -> jack; Island NOISE_ANALOG -> IO_JACK:${SHEETNAME}
- U6102, U6103, U6104: BoardRegion (none) -> core; Island NOISE_ANALOG -> IO_CORE:${SHEETNAME}
- U6103: BoardRegion (none) -> core; LogicalCellKey general_output_J_N1_WHITE_WHITE__A.1 -> PINK_LEVEL.1; Role general_output:A -> noise:PINK_LEVEL
- U6103: BoardRegion (none) -> core; LogicalCellKey PINK_LEVEL.1 -> BLUE_LEVEL.1; Role noise:PINK_LEVEL -> noise:BLUE_LEVEL
- U6104: BoardRegion (none) -> core; Island NOISE_ANALOG -> IO_CORE:${SHEETNAME}; LogicalCellKey BROWN_LEVEL.1 -> (none); Role noise:BROWN_LEVEL -> noise:unused grounded follower
- U6104: BoardRegion (none) -> core; LogicalCellKey general_output_J_N1_WHITE_PINK__A.1 -> BROWN_LEVEL.1; Role general_output:A -> noise:BROWN_LEVEL
- U6104: BoardRegion (none) -> core; Island NOISE_ANALOG -> IO_CORE:${SHEETNAME}; LogicalCellKey BLUE_LEVEL.1 -> (none); Role noise:BLUE_LEVEL -> noise:unused grounded follower
- U6104: BoardRegion (none) -> core; Island NOISE_ANALOG -> IO_CORE:${SHEETNAME}; LogicalCellKey general_output_J_N1_WHITE_BLUE__A.1 -> (none); Role general_output:A -> noise:unused grounded follower
- U6105: BoardRegion (none) -> jack; Island NOISE_ANALOG -> IO_JACK:${SHEETNAME}; LogicalCellKey general_output_J_N1_WHITE_BROWN__A.1 -> general_output_J_N1_WHITE_WHITE__A.1
- U6105: BoardRegion (none) -> jack; Island NOISE_ANALOG -> IO_JACK:${SHEETNAME}; LogicalCellKey (none) -> general_output_J_N1_WHITE_BROWN__A.1; Role noise:unused grounded follower -> general_output:A
- U6105: BoardRegion (none) -> jack; Island NOISE_ANALOG -> IO_JACK:${SHEETNAME}; LogicalCellKey (none) -> general_output_J_N1_WHITE_PINK__A.1; Role noise:unused grounded follower -> general_output:A
- U6105: BoardRegion (none) -> jack; Island NOISE_ANALOG -> IO_JACK:${SHEETNAME}; LogicalCellKey (none) -> general_output_J_N1_WHITE_BLUE__A.1; Role noise:unused grounded follower -> general_output:A
Connections:
- net PACK_OPA4196IDR_3_UNUSED1 is gone; now on net Cdbc5aa_DRIVE: U6105.6 (-), U6105.7
- net PACK_OPA4196IDR_3_UNUSED2 is gone; now on net Ce44f9a_DRIVE: U6105.8, U6105.9 (-)
- net PACK_OPA4196IDR_3_UNUSED3 is gone; now on net Cde1183_DRIVE: U6105.13 (-), U6105.14
- net AGND: now also U6103.10 (+), U6104.10 (+), U6104.3 (+); no longer U6105.10 (+), U6105.12 (+), U6105.5 (+)
- net BLUE_LEVEL: now also U6103.14, U6105.10 (+); no longer U6104.10 (+), U6104.7
- net BLUE_LEVEL_SUM: now also U6103.13 (-); no longer U6104.6 (-)
- net BROWN_LEVEL: now also U6104.1, U6105.12 (+); no longer U6104.14, U6105.3 (+)
- net BROWN_LEVEL_SUM: now also U6104.2 (-); no longer U6104.13 (-)
- net Cbe877b_DRIVE: now also U6105.1, U6105.2 (-); no longer U6103.8, U6103.9 (-)
- net Cdbc5aa_DRIVE: no longer U6104.1, U6104.2 (-)
- net Cde1183_DRIVE: no longer U6105.1, U6105.2 (-)
- net Ce44f9a_DRIVE: no longer U6104.8, U6104.9 (-)
- net PINK_LEVEL: now also U6103.8, U6105.5 (+); no longer U6103.14, U6104.3 (+)
- net PINK_LEVEL_SUM: now also U6103.9 (-); no longer U6103.13 (-)
- net WHITE_LEVEL: now also U6105.3 (+); no longer U6103.10 (+)
- new net PACK_OPA4196IDR_2_IO_UNUSED2: U6104.6 (-), U6104.7
- new net PACK_OPA4196IDR_2_IO_UNUSED3: U6104.8, U6104.9 (-)
- new net PACK_OPA4196IDR_2_IO_UNUSED4: U6104.13 (-), U6104.14
