File: schematic/sheets/filter.kicad_sch (KiCad schematic)
At the start: 258 parts, among them J601 WQP518MA, J602 WQP518MA, J603 WQP518MA, J604 WQP518MA, J605 WQP518MA, J606 WQP518MA, J607 WQP518MA, J608 WQP518MA, Q2101 BCM847BS,115, Q2102 MMBT3906,215, Q2103 MMBT3906,215, Q2104 MMBT3906,215, Q2105 MMBT3906,215, Q2106 MMBT3906,215, U2101 REF5050AIDR, U2102 ADG5412FBRUZ, U2103 ADG5412FBRUZ, U2104 ADG5412FBRUZ, U2105 ADG5412FBRUZ, U2106 LM13700M/NOPB, U2107 LM13700M/NOPB, U2108 OPA4197IPWR, U2109 OPA4197IPWR, U2110 OPA4196IDR, U2111 OPA4196IDR, U2112 OPA4196IDR, U2113 OPA4196IDR, U2114 OPA4196IDR, U2115 OPA4196IDR, U2116 OPA4196IDR, U2117 OPA4196IDR, U2118 OPA4196IDR, U2119 OPA4196IDR

Commit message: Refine source I/O regions and preserve whole package boundaries
Parts:
- C2101, C2102, C2103, C2104, C2105, C2106, C2107, C2108, C2109, C2110, C2111, C2112, C2113, C2114, C2115, D2105, D2106, D2107, D2108, D2109, D2110, D2111, D2112, D2113, D2114, D2115, D2116, D2117, D2118, D2119, D2120, D2121, D2122, D2123, D2124, Q2101, Q2102, Q2103, Q2104, Q2105, Q2106, R2101, R2102, R2103, R2104, R2121, R2122, R2123, R2124, R2125, R2126, R2127, R2128, R2129, R2130, R2131, R2132, R2133, R2134, R2135, R2136, R2137, R2138, R2139, R2140, R2141, R2142, R2143, R2144, R2145, R2146, R2147, R2148, R2149, R2150, R2151, R2152, R2153, R2154, R2155, R2156, R2157, R2158, R2159, R2160, R2161, R2162, R2163, R2164, R2165, R2166, R2167, R2168, R2169, R2170, R2171, R2172, R2173, R2174, R2175, R2176, R2177, R2178, R2179, R2180, R2181, R2182, R2183, R2184, R2185, R2186, R2187, R2188, R2189, R2190, R2191, R2192, R2193, R2194, R2195, R2196, R2197, R2198, R2199, RB2101, RB2102, RB2103, RB2104, RB2105, RV2107, RV2108, RV2109, RV2110, RV2111, RV2112, RV2113, U2101, U2106, U2107, U2108, U2109: BoardRegion (none) -> core
- C2116: BoardRegion (none) -> core; Decouples (none) -> CORE_reference_generator_J_F1_IN_LOCAL__U
- C2117, C2118: BoardRegion (none) -> jack; Decouples (none) -> CORE_input_fault_switch_J_F1_IN_IN__U; Island FILTER_CORE:${SHEETNAME} -> IO_JACK:${SHEETNAME}
- C2119, C2120: BoardRegion (none) -> jack; Decouples (none) -> CORE_input_fault_switch_J_F1_IN_FREQ__U; Island FILTER_CORE:${SHEETNAME} -> IO_JACK:${SHEETNAME}
- C2121, C2122: BoardRegion (none) -> jack; Decouples (none) -> CORE_input_fault_switch_J_F1_IN_RES__U; Island FILTER_CORE:${SHEETNAME} -> IO_JACK:${SHEETNAME}
- C2123, C2124: BoardRegion (none) -> jack; Decouples (none) -> CORE_input_fault_switch_J_F1_IN_GAIN__U; Island FILTER_CORE:${SHEETNAME} -> IO_JACK:${SHEETNAME}
- C2125, C2126: BoardRegion (none) -> core; Decouples (none) -> CORE_OTA_INTEGRATORS
- C2127, C2128: BoardRegion (none) -> core; Decouples (none) -> CORE_OTA_GAIN_RESONANCE
- C2129, C2130: BoardRegion (none) -> core; Decouples (none) -> CORE_PACK_OPA4197IPWR_0; Island FILTER_CORE:${SHEETNAME} -> IO_CORE:${SHEETNAME}
- C2131, C2132: BoardRegion (none) -> core; Decouples (none) -> CORE_PACK_OPA4197IPWR_1; Island FILTER_CORE:${SHEETNAME} -> IO_CORE:${SHEETNAME}
- C2133, C2134: BoardRegion (none) -> core; Decouples (none) -> CORE_PACK_OPA4196IDR_0; Island FILTER_CORE:${SHEETNAME} -> IO_CORE:${SHEETNAME}
- C2135, C2136: BoardRegion (none) -> core; Decouples (none) -> CORE_PACK_OPA4196IDR_1; Island FILTER_CORE:${SHEETNAME} -> IO_CORE:${SHEETNAME}
- C2137, C2138: BoardRegion (none) -> core; Decouples (none) -> CORE_PACK_OPA4196IDR_2; Island FILTER_CORE:${SHEETNAME} -> IO_CORE:${SHEETNAME}
- C2139, C2140: BoardRegion (none) -> core; Decouples (none) -> CORE_PACK_OPA4196IDR_3; Island FILTER_CORE:${SHEETNAME} -> IO_CORE:${SHEETNAME}
- C2141, C2142: BoardRegion (none) -> core; Decouples (none) -> CORE_PACK_OPA4196IDR_4; Island FILTER_CORE:${SHEETNAME} -> IO_CORE:${SHEETNAME}
- C2143, C2144: BoardRegion (none) -> core; Decouples (none) -> CORE_PACK_OPA4196IDR_5; Island FILTER_CORE:${SHEETNAME} -> IO_CORE:${SHEETNAME}
- C2145, C2146: BoardRegion (none) -> core; Decouples (none) -> CORE_PACK_OPA4196IDR_6; Island FILTER_CORE:${SHEETNAME} -> IO_CORE:${SHEETNAME}
- C2147, C2148: BoardRegion (none) -> jack; Decouples (none) -> CORE_PACK_OPA4196IDR_7; Island FILTER_CORE:${SHEETNAME} -> IO_JACK:${SHEETNAME}
- C2149, C2150: BoardRegion (none) -> jack; Decouples (none) -> CORE_PACK_OPA4196IDR_8; Island FILTER_CORE:${SHEETNAME} -> IO_JACK:${SHEETNAME}
- C2151, C2152: BoardRegion (none) -> jack; Decouples (none) -> LED_PACK_OPA4196IDR_0; Island FILTER_LEDS:${SHEETNAME} -> IO_JACK:${SHEETNAME}
- D2101, D2102, D2103, D2104, R2105, R2106, R2107, R2108, R2109, R2110, R2111, R2112, R2113, R2114, R2115, R2116, R2117, R2118, R2119, R2120, RB2106, RB2107, RB2108, RB2109, RB2110, RB2111, RB2112, RB2113, U2102, U2103, U2104, U2105, U2117, U2118: BoardRegion (none) -> jack; Island FILTER_CORE:${SHEETNAME} -> IO_JACK:${SHEETNAME}
- D2125, D2126, D2127, D2128, D2130, D2131, D2132, D2133, D2135, D2136, D2137, D2138, D2140, D2141, D2142, D2143, D601, D602, D603, D604, RB2114, RB2115, RB2116, RB2117, U2119: BoardRegion (none) -> jack
- J601, J602, J603, J604, J605, J606, J607, J608: BoardRegion (none) -> jack; Island (none) -> IO_JACK:${SHEETNAME}
- RV601, RV602, RV603, RV604, RV605, RV606: BoardRegion (none) -> control; Island (none) -> IO_CONTROL:${SHEETNAME}
- U2108, U2109, U2110, U2111, U2112, U2113, U2114, U2115, U2116: BoardRegion (none) -> core; Island FILTER_CORE:${SHEETNAME} -> IO_CORE:${SHEETNAME}
- U2110: BoardRegion (none) -> core; LogicalCellKey high_impedance_input_J_F1_IN_RES__A.1 -> dc_control_source_C_F1_FREQ_FREQ__A.1; Role high_impedance_input:A -> dc_control_source:A
- U2110: BoardRegion (none) -> core; LogicalCellKey high_impedance_input_J_F1_IN_FREQ__A.1 -> bipolar_attenuverter_C_F1_FREQ__FREQ__A.1; Role high_impedance_input:A -> bipolar_attenuverter:A
- U2110: BoardRegion (none) -> core; LogicalCellKey high_impedance_input_J_F1_IN_IN__A.1 -> remote_buffer_J_F1_IN_FREQ__A.1; Role high_impedance_input:A -> remote_buffer:A
- U2110: BoardRegion (none) -> core; LogicalCellKey high_impedance_input_J_F1_IN_GAIN__A.1 -> remote_buffer_J_F1_IN_RES__A.1; Role high_impedance_input:A -> remote_buffer:A
- U2111: BoardRegion (none) -> core; LogicalCellKey remote_buffer_J_F1_IN_RES__A.1 -> bipolar_attenuverter_C_F1_GAIN__GAIN__A.1; Role remote_buffer:A -> bipolar_attenuverter:A
- U2111: BoardRegion (none) -> core; LogicalCellKey dc_control_source_C_F1_FREQ_FREQ__A.1 -> remote_buffer_J_F1_IN_GAIN__A.1; Role dc_control_source:A -> remote_buffer:A
- U2111: BoardRegion (none) -> core; LogicalCellKey bipolar_attenuverter_C_F1_FREQ__FREQ__A.1 -> dc_control_source_C_F1_RES_RES__A.1; Role bipolar_attenuverter:A -> dc_control_source:A
- U2111: BoardRegion (none) -> core; LogicalCellKey remote_buffer_J_F1_IN_FREQ__A.1 -> bipolar_attenuverter_C_F1_RES__RES__A.1; Role remote_buffer:A -> bipolar_attenuverter:A
- U2112: BoardRegion (none) -> core; LogicalCellKey bipolar_attenuverter_C_F1_GAIN__GAIN__A.1 -> BP_BUFFER.1; Role bipolar_attenuverter:A -> filter:BP_BUFFER; Sensitive (none) -> BP_INT
- U2112: BoardRegion (none) -> core; LogicalCellKey dc_control_source_C_F1_RES_RES__A.1 -> FREQ_SUM.1; Role dc_control_source:A -> filter:FREQ_SUM
- U2112: BoardRegion (none) -> core; LogicalCellKey remote_buffer_J_F1_IN_GAIN__A.1 -> HP_SUM.1; Role remote_buffer:A -> filter:HP_SUM
- U2112: BoardRegion (none) -> core; LogicalCellKey bipolar_attenuverter_C_F1_RES__RES__A.1 -> dc_control_source_C_F1_GAIN_GAIN__A.1; Role bipolar_attenuverter:A -> dc_control_source:A
- U2113: BoardRegion (none) -> core; LogicalCellKey HP_SUM.1 -> RES_CONTROL_INVERT.1; Role filter:HP_SUM -> filter:RES_CONTROL_INVERT
- U2113: BoardRegion (none) -> core; LogicalCellKey FREQ_SUM.1 -> RES_CONTROL_SUM.1; Role filter:FREQ_SUM -> filter:RES_CONTROL_SUM
- U2113: BoardRegion (none) -> core; LogicalCellKey BP_BUFFER.1 -> RES_CONTROL_BUFFER.1; Role filter:BP_BUFFER -> filter:RES_CONTROL_BUFFER; Sensitive BP_INT -> (none)
- U2113: BoardRegion (none) -> core; LogicalCellKey dc_control_source_C_F1_GAIN_GAIN__A.1 -> LP_BUFFER.1; Role dc_control_source:A -> filter:LP_BUFFER; Sensitive (none) -> LP_INT
- U2114: BoardRegion (none) -> core; LogicalCellKey RES_CONTROL_INVERT.1 -> DRY_CONTROL_SUM.1; Role filter:RES_CONTROL_INVERT -> filter:DRY_CONTROL_SUM
- U2114: BoardRegion (none) -> core; LogicalCellKey LP_BUFFER.1 -> RES_EMITTER_TARGET.1; Role filter:LP_BUFFER -> filter:RES_EMITTER_TARGET; Sensitive LP_INT -> (none)
- U2114: BoardRegion (none) -> core; LogicalCellKey RES_CONTROL_SUM.1 -> RES_CURRENT_SERVO.1; Role filter:RES_CONTROL_SUM -> filter:RES_CURRENT_SERVO
- U2114: BoardRegion (none) -> core; LogicalCellKey RES_CONTROL_BUFFER.1 -> DRY_CONTROL_INVERT.1; Role filter:RES_CONTROL_BUFFER -> filter:DRY_CONTROL_INVERT
- U2115: BoardRegion (none) -> core; LogicalCellKey RES_EMITTER_TARGET.1 -> DRY_CONTROL_BUFFER.1; Role filter:RES_EMITTER_TARGET -> filter:DRY_CONTROL_BUFFER
- U2115: BoardRegion (none) -> core; LogicalCellKey RES_CURRENT_SERVO.1 -> DRY_EMITTER_TARGET.1; Role filter:RES_CURRENT_SERVO -> filter:DRY_EMITTER_TARGET
- U2115: BoardRegion (none) -> core; LogicalCellKey DRY_CONTROL_SUM.1 -> DRY_CURRENT_SERVO.1; Role filter:DRY_CONTROL_SUM -> filter:DRY_CURRENT_SERVO
- U2115: BoardRegion (none) -> core; LogicalCellKey DRY_CONTROL_INVERT.1 -> RESONANCE_TIA.1; Role filter:DRY_CONTROL_INVERT -> filter:RESONANCE_TIA
- U2116: BoardRegion (none) -> core; LogicalCellKey DRY_CONTROL_BUFFER.1 -> DRY_TIA.1; Role filter:DRY_CONTROL_BUFFER -> filter:DRY_TIA
- U2116: BoardRegion (none) -> core; Island FILTER_CORE:${SHEETNAME} -> IO_CORE:${SHEETNAME}; LogicalCellKey RESONANCE_TIA.1 -> (none); Role filter:RESONANCE_TIA -> filter:unused grounded follower
- U2116: BoardRegion (none) -> core; Island FILTER_CORE:${SHEETNAME} -> IO_CORE:${SHEETNAME}; LogicalCellKey DRY_CURRENT_SERVO.1 -> (none); Role filter:DRY_CURRENT_SERVO -> filter:unused grounded follower
- U2116: BoardRegion (none) -> core; Island FILTER_CORE:${SHEETNAME} -> IO_CORE:${SHEETNAME}; LogicalCellKey DRY_EMITTER_TARGET.1 -> (none); Role filter:DRY_EMITTER_TARGET -> filter:unused grounded follower
- U2117: BoardRegion (none) -> jack; Island FILTER_CORE:${SHEETNAME} -> IO_JACK:${SHEETNAME}; LogicalCellKey general_output_J_F1_IN_BP__A.1 -> high_impedance_input_J_F1_IN_RES__A.1; Role general_output:A -> high_impedance_input:A
- U2117: BoardRegion (none) -> jack; Island FILTER_CORE:${SHEETNAME} -> IO_JACK:${SHEETNAME}; LogicalCellKey DRY_TIA.1 -> high_impedance_input_J_F1_IN_IN__A.1; Role filter:DRY_TIA -> high_impedance_input:A
- U2117: BoardRegion (none) -> jack; Island FILTER_CORE:${SHEETNAME} -> IO_JACK:${SHEETNAME}; LogicalCellKey general_output_J_F1_IN_HP__A.1 -> high_impedance_input_J_F1_IN_GAIN__A.1; Role general_output:A -> high_impedance_input:A
- U2117: BoardRegion (none) -> jack; Island FILTER_CORE:${SHEETNAME} -> IO_JACK:${SHEETNAME}; LogicalCellKey general_output_J_F1_IN_LP__A.1 -> high_impedance_input_J_F1_IN_FREQ__A.1; Role general_output:A -> high_impedance_input:A
- U2118: BoardRegion (none) -> jack; Island FILTER_CORE:${SHEETNAME} -> IO_JACK:${SHEETNAME}; LogicalCellKey (none) -> general_output_J_F1_IN_BP__A.1; Role filter:unused grounded follower -> general_output:A
- U2118: BoardRegion (none) -> jack; Island FILTER_CORE:${SHEETNAME} -> IO_JACK:${SHEETNAME}; LogicalCellKey (none) -> general_output_J_F1_IN_HP__A.1; Role filter:unused grounded follower -> general_output:A
- U2118: BoardRegion (none) -> jack; Island FILTER_CORE:${SHEETNAME} -> IO_JACK:${SHEETNAME}; LogicalCellKey (none) -> general_output_J_F1_IN_OUT__A.1; Role filter:unused grounded follower -> general_output:A
- U2118: BoardRegion (none) -> jack; Island FILTER_CORE:${SHEETNAME} -> IO_JACK:${SHEETNAME}; LogicalCellKey general_output_J_F1_IN_OUT__A.1 -> general_output_J_F1_IN_LP__A.1
- U2119: BoardRegion (none) -> jack; Island FILTER_LEDS:${SHEETNAME} -> IO_JACK:${SHEETNAME}
Connections:
- net PACK_OPA4196IDR_8_UNUSED1 is gone; now on net C29cc99_DRIVE: U2118.6 (-), U2118.7
- net PACK_OPA4196IDR_8_UNUSED2 is gone; now on net C2b02f4_DRIVE: U2118.8, U2118.9 (-)
- net PACK_OPA4196IDR_8_UNUSED3 is gone; now on net C56c9d6_DRIVE: U2118.13 (-), U2118.14
- net AGND: now also U2112.5 (+), U2113.10 (+), U2114.12 (+), U2116.10 (+), U2116.3 (+), U2116.5 (+); no longer U2114.5 (+), U2115.10 (+), U2117.3 (+), U2118.10 (+), U2118.12 (+), U2118.5 (+)
- net BP_CORE: now also U2112.13 (-), U2112.14, U2118.5 (+); no longer U2113.13 (-), U2113.14, U2117.10 (+)
- net BP_INT: now also U2112.12 (+); no longer U2113.12 (+)
- net C11c270_DRIVE: now also U2111.8; no longer U2112.8
- net C11c270_FB: now also U2111.9 (-); no longer U2112.9 (-)
- net C14689f_W_SENSE: now also U2110.10 (+); no longer U2111.10 (+)
- net C29cc99_DRIVE: no longer U2117.8, U2117.9 (-)
- net C2b02f4_DRIVE: no longer U2117.13 (-), U2117.14
- net C2b474d_SUM: now also U2110.6 (-); no longer U2111.6 (-)
- net C2b474d_W_SENSE: now also U2110.5 (+); no longer U2111.5 (+)
- net C56c9d6_DRIVE: no longer U2118.1, U2118.2 (-)
- net C5d31c8_DRIVE: now also U2118.1, U2118.2 (-); no longer U2117.6 (-), U2117.7
- net C72459f_SENSE: now also U2117.12 (+); no longer U2110.12 (+)
- net C7fa4f0_SENSE: now also U2117.3 (+); no longer U2110.3 (+)
- net C8c344f_W_SENSE: now also U2111.5 (+); no longer U2112.5 (+)
- net C908572_SENSE: now also U2117.5 (+); no longer U2110.5 (+)
- net C945bba_SENSE: now also U2117.10 (+); no longer U2110.10 (+)
- net Ca72ec0_W_SENSE: now also U2112.3 (+); no longer U2113.3 (+)
- net Cb3b460_SUM: now also U2111.13 (-); no longer U2112.13 (-)
- net Cb3b460_W_SENSE: now also U2111.12 (+); no longer U2112.12 (+)
- net Cb5b1dc_SUM: now also U2111.2 (-); no longer U2112.2 (-)
- net Cb5b1dc_W_SENSE: now also U2111.3 (+); no longer U2112.3 (+)
- net Cef1e35_DRIVE: now also U2110.1; no longer U2111.1
- net Cef1e35_FB: now also U2110.2 (-); no longer U2111.2 (-)
- net Cf75ecf_DRIVE: now also U2110.14; no longer U2111.14
- net Cf75ecf_FB: now also U2110.13 (-); no longer U2111.13 (-)
- net DRY_BASE_DRIVE: now also U2115.8; no longer U2116.8
- net DRY_COMMAND: now also U2115.1, U2115.2 (-); no longer U2116.1, U2116.2 (-)
- net DRY_CONTROL_CLAMP: now also U2115.3 (+); no longer U2116.3 (+)
- net DRY_CONTROL_INV: now also U2114.13 (-); no longer U2115.13 (-)
- net DRY_CONTROL_NEG: now also U2114.8; no longer U2115.8
- net DRY_CONTROL_RAW: now also U2114.14; no longer U2115.14
- net DRY_CONTROL_SUM: now also U2114.9 (-); no longer U2115.9 (-)
- net DRY_CORE: now also U2116.1, U2118.12 (+); no longer U2117.1, U2118.3 (+)
- net DRY_EMITTER: now also U2115.9 (-); no longer U2116.9 (-)
- net DRY_INT: now also U2116.2 (-); no longer U2117.2 (-)
- net DRY_TARGET: now also U2115.10 (+), U2115.7; no longer U2116.10 (+), U2116.7
- net DRY_TARGET_SUM: now also U2115.6 (-); no longer U2116.6 (-)
- net FREQ_BUFFER: now also U2110.3 (+), U2117.6 (-), U2117.7; no longer U2110.6 (-), U2110.7, U2111.3 (+)
- net FREQ_DEPTH: now also U2110.7; no longer U2111.7
- net FREQ_MANUAL: now also U2110.8, U2110.9 (-); no longer U2111.8, U2111.9 (-)
- net FREQ_NEG: now also U2112.7; no longer U2113.7
- net FREQ_SUM: now also U2112.6 (-); no longer U2113.6 (-)
- net GAIN_BUFFER: now also U2111.10 (+), U2117.13 (-), U2117.14; no longer U2110.13 (-), U2110.14, U2112.10 (+)
- net GAIN_DEPTH: now also U2111.14; no longer U2112.14
- net GAIN_MANUAL: now also U2112.1, U2112.2 (-); no longer U2113.1, U2113.2 (-)
- net HP_CORE: now also U2112.8, U2118.10 (+); no longer U2113.8, U2117.12 (+)
- net HP_PLUS: now also U2112.10 (+); no longer U2113.10 (+)
- net HP_SUM: now also U2112.9 (-); no longer U2113.9 (-)
- net IN_BUFFER: now also U2117.1, U2117.2 (-); no longer U2110.1, U2110.2 (-)
- net LP_CORE: now also U2113.1, U2113.2 (-), U2118.3 (+); no longer U2114.1, U2114.2 (-), U2117.5 (+)
- net LP_INT: now also U2113.3 (+); no longer U2114.3 (+)
- net REF25: now also U2114.3 (+), U2115.5 (+); no longer U2115.3 (+), U2116.5 (+)
- net RES_BASE_DRIVE: now also U2114.7; no longer U2115.7
- net RES_BUFFER: now also U2110.12 (+), U2117.8, U2117.9 (-); no longer U2110.8, U2110.9 (-), U2111.12 (+)
- net RES_COMMAND: now also U2113.13 (-), U2113.14; no longer U2114.13 (-), U2114.14
- net RES_CONTROL_CLAMP: now also U2113.12 (+); no longer U2114.12 (+)
- net RES_CONTROL_INV: now also U2113.9 (-); no longer U2114.9 (-)
- net RES_CONTROL_NEG: now also U2113.7; no longer U2114.7
- net RES_CONTROL_RAW: now also U2113.8; no longer U2114.8
- net RES_CONTROL_SUM: now also U2113.6 (-); no longer U2114.6 (-)
- net RES_DEPTH: now also U2111.1; no longer U2112.1
- net RES_EMITTER: now also U2114.6 (-); no longer U2115.6 (-)
- net RES_INT: now also U2115.13 (-); no longer U2116.13 (-)
- net RES_MANUAL: now also U2111.6 (-), U2111.7; no longer U2112.6 (-), U2112.7
- net RES_NEG: now also U2115.14; no longer U2116.14
- net RES_TARGET: now also U2114.1, U2114.5 (+); no longer U2115.1, U2115.5 (+)
- net RES_TARGET_SUM: now also U2114.2 (-); no longer U2115.2 (-)
- net PACK_OPA4197IPWR_1_UNUSED1 renamed CORE_PACK_OPA4197IPWR_1_IO_UNUSED2
- net PACK_OPA4197IPWR_1_UNUSED2 renamed CORE_PACK_OPA4197IPWR_1_IO_UNUSED3
- net PACK_OPA4197IPWR_1_UNUSED3 renamed CORE_PACK_OPA4197IPWR_1_IO_UNUSED4
- new net CORE_PACK_OPA4196IDR_6_IO_UNUSED2: U2116.6 (-), U2116.7
- new net CORE_PACK_OPA4196IDR_6_IO_UNUSED3: U2116.8, U2116.9 (-)
- new net CORE_PACK_OPA4196IDR_6_IO_UNUSED4: U2116.13 (-), U2116.14

Commit message: Select exact compact indicator LEDs and audit fixed centres
Parts:
- D601, D602, D603, D604: value KT-0603W -> APHHS1005QWF/D; footprint zudo-osc-hole-field:LED0603-R-RD_WHITE -> zudo-osc-hole-field:LED0402-Kingbright-White; symbol zudo-osc-hole-field:0603Whitelight_C2290 -> zudo-osc-hole-field:Kingbright_White_0402; LCSC C2290 -> (none); MPN KT-0603W -> APHHS1005QWF/D; Manufacturer KENTO -> Kingbright
- RB2114, RB2115, RB2116, RB2117: value 4990 Ω -> 5600 Ω
Connections:
- net C9fcdd2_LED_A: now also D603.2 (A); no longer D603.1 (A)
- net C9fcdd2_LED_K: now also D603.1 (K); no longer D603.2 (K)
- net Cb3d4a2_LED_A: now also D601.2 (A); no longer D601.1 (A)
- net Cb3d4a2_LED_K: now also D601.1 (K); no longer D601.2 (K)
- net Cb6d8fd_LED_A: now also D602.2 (A); no longer D602.1 (A)
- net Cb6d8fd_LED_K: now also D602.1 (K); no longer D602.2 (K)
- net Cfc4b03_LED_A: now also D604.2 (A); no longer D604.1 (A)
- net Cfc4b03_LED_K: now also D604.1 (K); no longer D604.2 (K)
Other:
- moved on the sheet: D601, D602, D603, D604
