File: schematic/sheets/mix4_vca.kicad_sch (KiCad schematic)
At the start: 214 parts, among them J1101 WQP518MA, J1102 WQP518MA, J1103 WQP518MA, J1104 WQP518MA, J1105 WQP518MA, J1106 WQP518MA, Q8301 MMBT3906,215, U8301 REF5050AIDR, U8302 ADG5412FBRUZ, U8303 ADG5412FBRUZ, U8304 ADG5412FBRUZ, U8305 ADG5412FBRUZ, U8306 ADG5412FBRUZ, U8307 LM13700M/NOPB, U8308 OPA4197IPWR, U8309 OPA4196IDR, U8310 OPA4196IDR, U8311 OPA4196IDR, U8312 OPA4196IDR, U8313 OPA4196IDR, U8314 OPA4196IDR, U8315 LM393BIDR, U8316 LM393BIDR, U8317 OPA4196IDR, U8318 OPA4196IDR, U8319 OPA4196IDR

Commit message: Select exact compact indicator LEDs and audit fixed centres
Parts:
- D1101, D1102, D1103, D1104, D1105, D1106: value KT-0603W -> APHHS1005QWF/D; footprint zudo-osc-hole-field:LED0603-R-RD_WHITE -> zudo-osc-hole-field:LED0402-Kingbright-White; symbol zudo-osc-hole-field:0603Whitelight_C2290 -> zudo-osc-hole-field:Kingbright_White_0402; LCSC C2290 -> (none); MPN KT-0603W -> APHHS1005QWF/D; Manufacturer KENTO -> Kingbright
- D11061: value KT-0603R -> APG1005SEC/E-T; footprint zudo-osc-hole-field:LED0603-RD -> zudo-osc-hole-field:LED0402-Kingbright-Red; symbol zudo-osc-hole-field:KT-0603R -> zudo-osc-hole-field:Kingbright_Red_0402; LCSC C2286 -> (none); MPN KT-0603R -> APG1005SEC/E-T; Manufacturer KENTO -> Kingbright
- R8383, R8384, R8385, R8386, R8387, R8388: value 4990 Ω -> 5600 Ω
Connections:
- net C2169e5_LED_A: now also D1103.2 (A); no longer D1103.1 (A)
- net C2169e5_LED_K: now also D1103.1 (K); no longer D1103.2 (K)
- net C320656_LED_A: now also D1105.2 (A); no longer D1105.1 (A)
- net C320656_LED_K: now also D1105.1 (K); no longer D1105.2 (K)
- net C412fd1_LED_A: now also D1101.2 (A); no longer D1101.1 (A)
- net C412fd1_LED_K: now also D1101.1 (K); no longer D1101.2 (K)
- net C93bba0_LED_A: now also D1102.2 (A); no longer D1102.1 (A)
- net C93bba0_LED_K: now also D1102.1 (K); no longer D1102.2 (K)
- net Cd59875_LED_A: now also D1106.2 (A); no longer D1106.1 (A)
- net Cd59875_LED_K: now also D1106.1 (K); no longer D1106.2 (K)
- net Cf876de_LED_A: now also D1104.2 (A); no longer D1104.1 (A)
- net Cf876de_LED_K: now also D1104.1 (K); no longer D1104.2 (K)
Other:
- moved on the sheet: D1101, D1102, D1103, D1104, D1105, D1106
