File: schematic/sheets/wavefolder.kicad_sch (KiCad schematic)
At the start: 170 parts, among them J1007 WQP518MA, J1008 WQP518MA, J907 WQP518MA, J908 WQP518MA, Q5101 MMBT3906,215, U5101 REF5050AIDR, U5102 ADG5412FBRUZ, U5103 ADG5412FBRUZ, U5104 ADG5412FBRUZ, U5105 LM13700M/NOPB, U5106 OPA4197IPWR, U5107 OPA4196IDR, U5108 OPA4196IDR, U5109 OPA4196IDR, U5110 OPA4196IDR, U5111 OPA4196IDR, U5112 OPA4196IDR, U5113 OPA4196IDR

Commit message: Refine source I/O regions and preserve whole package boundaries
Parts:
- C5101, C5102, C5103, C5104, C5105, C5106, C5107, C5108, C5109, C5110, C5111, C5112, C5113, C5114, C5115, C5116, C5117, C5118, D5104, D5105, D5106, D5107, D5108, D5109, D5110, D5111, D5112, D5113, Q5101, R5101, R5102, R5103, R5104, R5117, R5118, R5119, R5120, R5121, R5122, R5123, R5124, R5125, R5126, R5127, R5128, R5129, R5130, R5131, R5132, R5133, R5134, R5135, R5136, R5137, R5138, R5139, R5140, R5141, R5142, R5143, R5144, R5145, R5146, R5147, R5148, R5149, R5150, R5151, R5152, R5153, R5154, R5155, R5156, R5157, R5158, R5159, R5160, R5161, R5162, R5163, R5164, R5165, R5166, R5167, R5168, R5169, R5170, RV5104, RV5105, U5101, U5105, U5106: BoardRegion (none) -> core
- C5119: BoardRegion (none) -> core; Decouples (none) -> CORE_reference_generator_J_W2_IN_LOCAL__U
- C5120, C5121: BoardRegion (none) -> jack; Decouples (none) -> CORE_input_fault_switch_J_W2_IN_IN__U; Island FOLDER_CORE:${SHEETNAME} -> IO_JACK:${SHEETNAME}
- C5122, C5123: BoardRegion (none) -> jack; Decouples (none) -> CORE_input_fault_switch_J_W2_IN_FOLD__U; Island FOLDER_CORE:${SHEETNAME} -> IO_JACK:${SHEETNAME}
- C5124, C5125: BoardRegion (none) -> jack; Decouples (none) -> CORE_input_fault_switch_J_W2_IN_BIAS__U; Island FOLDER_CORE:${SHEETNAME} -> IO_JACK:${SHEETNAME}
- C5126, C5127: BoardRegion (none) -> core; Decouples (none) -> CORE_OTA
- C5128, C5129: BoardRegion (none) -> core; Decouples (none) -> CORE_PACK_OPA4197IPWR_0; Island FOLDER_CORE:${SHEETNAME} -> IO_CORE:${SHEETNAME}
- C5130, C5131: BoardRegion (none) -> core; Decouples (none) -> CORE_PACK_OPA4196IDR_0; Island FOLDER_CORE:${SHEETNAME} -> IO_CORE:${SHEETNAME}
- C5132, C5133: BoardRegion (none) -> core; Decouples (none) -> CORE_PACK_OPA4196IDR_1; Island FOLDER_CORE:${SHEETNAME} -> IO_CORE:${SHEETNAME}
- C5134, C5135: BoardRegion (none) -> core; Decouples (none) -> CORE_PACK_OPA4196IDR_2; Island FOLDER_CORE:${SHEETNAME} -> IO_CORE:${SHEETNAME}
- C5136, C5137: BoardRegion (none) -> core; Decouples (none) -> CORE_PACK_OPA4196IDR_3; Island FOLDER_CORE:${SHEETNAME} -> IO_CORE:${SHEETNAME}
- C5138, C5139: BoardRegion (none) -> core; Decouples (none) -> CORE_PACK_OPA4196IDR_4; Island FOLDER_CORE:${SHEETNAME} -> IO_CORE:${SHEETNAME}
- C5140, C5141: BoardRegion (none) -> jack; Decouples (none) -> CORE_PACK_OPA4196IDR_5; Island FOLDER_CORE:${SHEETNAME} -> IO_JACK:${SHEETNAME}
- C5142, C5143: BoardRegion (none) -> jack; Decouples (none) -> LED_PACK_OPA4196IDR_0; Island FOLDER_LEDS:${SHEETNAME} -> IO_JACK:${SHEETNAME}
- D1007, D5114, D5115, D5116, D5117, D5119, D5120, D5121, D5122, D5124, D5125, D5126, D5127, D907, D908, R5173, R5174, R5175, U5113: BoardRegion (none) -> jack
- D5101, D5102, D5103, R5105, R5106, R5107, R5108, R5109, R5110, R5111, R5112, R5113, R5114, R5115, R5116, R5171, R5172, U5102, U5103, U5104, U5112: BoardRegion (none) -> jack; Island FOLDER_CORE:${SHEETNAME} -> IO_JACK:${SHEETNAME}
- J1007, J1008, J907, J908: BoardRegion (none) -> jack; Island (none) -> IO_JACK:${SHEETNAME}
- RV1007, RV1008, RV907, RV908: BoardRegion (none) -> control; Island (none) -> IO_CONTROL:${SHEETNAME}
- U5106, U5107, U5108, U5109, U5110, U5111: BoardRegion (none) -> core; Island FOLDER_CORE:${SHEETNAME} -> IO_CORE:${SHEETNAME}
- U5107: BoardRegion (none) -> core; LogicalCellKey high_impedance_input_J_W2_IN_FOLD__A.1 -> dc_control_source_C_W2_BIAS_BIAS__A.1; Role high_impedance_input:A -> dc_control_source:A
- U5107: BoardRegion (none) -> core; LogicalCellKey high_impedance_input_J_W2_IN_BIAS__A.1 -> remote_buffer_J_W2_IN_FOLD__A.1; Role high_impedance_input:A -> remote_buffer:A
- U5107: BoardRegion (none) -> core; LogicalCellKey dc_control_source_C_W2_FOLD_FOLD__A.1 -> bipolar_attenuverter_C_W2_FOLD__FOLD__A.1; Role dc_control_source:A -> bipolar_attenuverter:A
- U5107: BoardRegion (none) -> core; LogicalCellKey high_impedance_input_J_W2_IN_IN__A.1 -> dc_control_source_C_W2_FOLD_FOLD__A.1; Role high_impedance_input:A -> dc_control_source:A
- U5108: BoardRegion (none) -> core; LogicalCellKey bipolar_attenuverter_C_W2_FOLD__FOLD__A.1 -> CONTROL_BUFFER.1; Role bipolar_attenuverter:A -> wavefolder:CONTROL_BUFFER
- U5108: BoardRegion (none) -> core; LogicalCellKey remote_buffer_J_W2_IN_FOLD__A.1 -> CONTROL_INVERT.1; Role remote_buffer:A -> wavefolder:CONTROL_INVERT
- U5108: BoardRegion (none) -> core; LogicalCellKey dc_control_source_C_W2_BIAS_BIAS__A.1 -> CONTROL_SUM.1; Role dc_control_source:A -> wavefolder:CONTROL_SUM
- U5108: BoardRegion (none) -> core; LogicalCellKey CONTROL_SUM.1 -> EMITTER_TARGET.1; Role wavefolder:CONTROL_SUM -> wavefolder:EMITTER_TARGET
- U5109: BoardRegion (none) -> core; LogicalCellKey CONTROL_INVERT.1 -> CURRENT_SERVO.1; Role wavefolder:CONTROL_INVERT -> wavefolder:CURRENT_SERVO
- U5109: BoardRegion (none) -> core; LogicalCellKey EMITTER_TARGET.1 -> DRIVE_SUM.1; Role wavefolder:EMITTER_TARGET -> wavefolder:DRIVE_SUM; Sensitive (none) -> FOLDER_SUM
- U5109: BoardRegion (none) -> core; LogicalCellKey CURRENT_SERVO.1 -> DRIVE_INVERT.1; Role wavefolder:CURRENT_SERVO -> wavefolder:DRIVE_INVERT
- U5109: BoardRegion (none) -> core; LogicalCellKey CONTROL_BUFFER.1 -> PRE_GAIN.1; Role wavefolder:CONTROL_BUFFER -> wavefolder:PRE_GAIN; Sensitive (none) -> PRE_GAIN_SUM
- U5110: BoardRegion (none) -> core; LogicalCellKey DRIVE_INVERT.1 -> F3.1; Role wavefolder:DRIVE_INVERT -> wavefolder:F3; Sensitive (none) -> F3_CLIP,F3_SUM
- U5110: BoardRegion (none) -> core; LogicalCellKey F1.1 -> F4.1; Role wavefolder:F1 -> wavefolder:F4; Sensitive F1_CLIP,F1_SUM -> F4_CLIP,F4_SUM
- U5110: BoardRegion (none) -> core; LogicalCellKey PRE_GAIN.1 -> F1.1; Role wavefolder:PRE_GAIN -> wavefolder:F1; Sensitive PRE_GAIN_SUM -> F1_CLIP,F1_SUM
- U5110: BoardRegion (none) -> core; LogicalCellKey DRIVE_SUM.1 -> F2.1; Role wavefolder:DRIVE_SUM -> wavefolder:F2; Sensitive FOLDER_SUM -> F2_CLIP,F2_SUM
- U5111: BoardRegion (none) -> core; LogicalCellKey F3.1 -> AC_BUFFER.1; Role wavefolder:F3 -> wavefolder:AC_BUFFER; Sensitive F3_CLIP,F3_SUM -> AC_NODE
- U5111: BoardRegion (none) -> core; LogicalCellKey F4.1 -> remote_buffer_J_W2_IN_LEVEL__A.1; Role wavefolder:F4 -> remote_buffer:A; Sensitive F4_CLIP,F4_SUM -> (none)
- U5111: BoardRegion (none) -> core; LogicalCellKey F2.1 -> OUTPUT_SCALE.1; Role wavefolder:F2 -> wavefolder:OUTPUT_SCALE; Sensitive F2_CLIP,F2_SUM -> (none)
- U5111: BoardRegion (none) -> core; LogicalCellKey OUTPUT_SCALE.1 -> level_attenuator_C_W2_LEVEL_LEVEL__A.1; Role wavefolder:OUTPUT_SCALE -> level_attenuator:A
- U5112: BoardRegion (none) -> jack; Island FOLDER_CORE:${SHEETNAME} -> IO_JACK:${SHEETNAME}; LogicalCellKey remote_buffer_J_W2_IN_LEVEL__A.1 -> high_impedance_input_J_W2_IN_FOLD__A.1; Role remote_buffer:A -> high_impedance_input:A
- U5112: BoardRegion (none) -> jack; Island FOLDER_CORE:${SHEETNAME} -> IO_JACK:${SHEETNAME}; LogicalCellKey level_attenuator_C_W2_LEVEL_LEVEL__A.1 -> high_impedance_input_J_W2_IN_BIAS__A.1; Role level_attenuator:A -> high_impedance_input:A
- U5112: BoardRegion (none) -> jack; Island FOLDER_CORE:${SHEETNAME} -> IO_JACK:${SHEETNAME}; LogicalCellKey AC_BUFFER.1 -> high_impedance_input_J_W2_IN_IN__A.1; Role wavefolder:AC_BUFFER -> high_impedance_input:A; Sensitive AC_NODE -> (none)
- U5113: BoardRegion (none) -> jack; Island FOLDER_LEDS:${SHEETNAME} -> IO_JACK:${SHEETNAME}
Connections:
- net AC_BUFFER: now also U5111.10 (+), U5111.6 (-), U5111.7; no longer U5112.1, U5112.2 (-), U5112.5 (+)
- net AC_NODE: now also U5111.5 (+); no longer U5112.3 (+)
- net AGND: now also U5108.3 (+), U5108.5 (+), U5109.10 (+), U5109.12 (+), U5109.5 (+); no longer U5108.12 (+), U5109.3 (+), U5110.10 (+), U5110.3 (+), U5110.5 (+)
- net BASE_DRIVE: now also U5109.1; no longer U5109.14
- net BIAS_BUFFER: now also U5112.8, U5112.9 (-); no longer U5107.8, U5107.9 (-)
- net BIAS_MANUAL: now also U5107.6 (-), U5107.7; no longer U5108.1, U5108.2 (-)
- net C01cf3e_DRIVE: now also U5111.8; no longer U5112.7
- net C01cf3e_FB: now also U5111.9 (-); no longer U5112.6 (-)
- net C4c1698_W_SENSE: now also U5107.5 (+); no longer U5108.3 (+)
- net C554ad0_SENSE: now also U5112.10 (+); no longer U5107.10 (+)
- net C629978_W_SENSE: now also U5111.12 (+); no longer U5112.10 (+)
- net C74d1de_SENSE: now also U5112.5 (+); no longer U5107.5 (+)
- net C75db46_W_SENSE: now also U5107.3 (+); no longer U5107.12 (+)
- net C8df94f_SENSE: now also U5112.3 (+); no longer U5107.3 (+)
- net C9cfd7a_DRIVE: now also U5107.8; no longer U5108.7
- net C9cfd7a_FB: now also U5107.9 (-); no longer U5108.6 (-)
- net COMMAND: now also U5108.8, U5108.9 (-); no longer U5109.6 (-), U5109.7
- net CONTROL_CLAMP: now also U5108.10 (+); no longer U5109.5 (+)
- net CONTROL_INV: now also U5108.6 (-); no longer U5109.2 (-)
- net CONTROL_NEG: now also U5108.1; no longer U5108.14
- net CONTROL_RAW: now also U5108.7; no longer U5109.1
- net CONTROL_SUM: now also U5108.2 (-); no longer U5108.13 (-)
- net Cb36f8a_SUM: now also U5107.13 (-); no longer U5108.9 (-)
- net Cb36f8a_W_SENSE: now also U5107.12 (+); no longer U5108.10 (+)
- net DRIVE_INV_SUM: now also U5109.13 (-); no longer U5110.9 (-)
- net EMITTER: now also U5109.2 (-); no longer U5109.13 (-)
- net F1_CLIP: now also U5110.3 (+); no longer U5110.12 (+)
- net F1_OUT: now also U5110.1; no longer U5110.14
- net F1_SUM: now also U5110.2 (-); no longer U5110.13 (-)
- net F2_CLIP: now also U5110.5 (+); no longer U5111.3 (+)
- net F2_OUT: now also U5110.7; no longer U5111.1
- net F2_SUM: now also U5110.6 (-); no longer U5111.2 (-)
- net F3_CLIP: now also U5110.10 (+); no longer U5111.5 (+)
- net F3_OUT: now also U5110.8; no longer U5111.7
- net F3_SUM: now also U5110.9 (-); no longer U5111.6 (-)
- net F4_CLIP: now also U5110.12 (+); no longer U5111.10 (+)
- net F4_OUT: now also U5110.14, U5111.3 (+); no longer U5111.12 (+), U5111.8
- net F4_SUM: now also U5110.13 (-); no longer U5111.9 (-)
- net FOLDER_DRIVE: now also U5109.14; no longer U5110.8
- net FOLDER_NEG: now also U5109.8; no longer U5110.7
- net FOLDER_SUM: now also U5109.9 (-); no longer U5110.6 (-)
- net FOLD_BUFFER: now also U5107.10 (+), U5112.6 (-), U5112.7; no longer U5107.6 (-), U5107.7, U5108.5 (+)
- net FOLD_DEPTH: now also U5107.14; no longer U5108.8
- net FOLD_MANUAL: now also U5107.1, U5107.2 (-); no longer U5107.13 (-), U5107.14
- net IN_BUFFER: now also U5112.1, U5112.2 (-); no longer U5107.1, U5107.2 (-)
- net LEVEL_OUT: now also U5111.13 (-), U5111.14; no longer U5112.8, U5112.9 (-)
- net OUTPUT_FB: now also U5111.2 (-); no longer U5111.13 (-)
- net PRE_AC: now also U5111.1; no longer U5111.14
- net PRE_GAIN: now also U5109.7; no longer U5110.1
- net PRE_GAIN_SUM: now also U5109.6 (-); no longer U5110.2 (-)
- net REF25: now also U5108.12 (+); no longer U5109.10 (+)
- net TARGET: now also U5108.14, U5109.3 (+); no longer U5109.12 (+), U5109.8
- net TARGET_SUM: now also U5108.13 (-); no longer U5109.9 (-)
- net PACK_OPA4196IDR_0_UNUSED3 renamed LED_PACK_OPA4196IDR_0_IO_UNUSED4
- net PACK_OPA4197IPWR_0_UNUSED3 renamed CORE_PACK_OPA4197IPWR_0_IO_UNUSED4

Commit message: Select exact compact indicator LEDs and audit fixed centres
Parts:
- D1007, D907, D908: value KT-0603W -> APHHS1005QWF/D; footprint zudo-osc-hole-field:LED0603-R-RD_WHITE -> zudo-osc-hole-field:LED0402-Kingbright-White; symbol zudo-osc-hole-field:0603Whitelight_C2290 -> zudo-osc-hole-field:Kingbright_White_0402; LCSC C2290 -> (none); MPN KT-0603W -> APHHS1005QWF/D; Manufacturer KENTO -> Kingbright
- R5173, R5174, R5175: value 4990 Ω -> 5600 Ω
Connections:
- net C029db8_LED_A: now also D908.2 (A); no longer D908.1 (A)
- net C029db8_LED_K: now also D908.1 (K); no longer D908.2 (K)
- net C20383d_LED_A: now also D907.2 (A); no longer D907.1 (A)
- net C20383d_LED_K: now also D907.1 (K); no longer D907.2 (K)
- net Cb68133_LED_A: now also D1007.2 (A); no longer D1007.1 (A)
- net Cb68133_LED_K: now also D1007.1 (K); no longer D1007.2 (K)
Other:
- moved on the sheet: D1007, D907, D908
