File: boards/osc-jack/sheets/envelope_E6_J.kicad_sch (KiCad schematic)
At the start: 66 parts, among them J1801 WQP518MA, J1802 WQP518MA, J1803 WQP518MA, J1804 WQP518MA, J1805 WQP518MA, J1806 WQP518MA, J1807 WQP518MA, U4602 ADG5412FBRUZ, U4603 ADG5412FBRUZ, U4604 ADG5412FBRUZ, U4646 OPA4196IDR, U4647 OPA4196IDR, U4648 OPA4196IDR

Commit message: Reserve clear jack-board geometry and align projected schematic fields
Parts:
- C4615: Island IO_JACK:${SHEETNAME} -> (none); Role envelope:C_DEC_CORE_input_fault_switch_J_E1_SIG_SIG__U_0 -> (none)
- C4616: Island IO_JACK:${SHEETNAME} -> (none); Role envelope:C_DEC_CORE_input_fault_switch_J_E1_SIG_SIG__U_1 -> (none)
- C4617: Island IO_JACK:${SHEETNAME} -> (none); Role envelope:C_DEC_CORE_input_fault_switch_J_E1_SIG_RISE__U_0 -> (none)
- C4618: Island IO_JACK:${SHEETNAME} -> (none); Role envelope:C_DEC_CORE_input_fault_switch_J_E1_SIG_RISE__U_1 -> (none)
- C4619: Island IO_JACK:${SHEETNAME} -> (none); Role envelope:C_DEC_CORE_input_fault_switch_J_E1_SIG_FALL__U_0 -> (none)
- C4620: Island IO_JACK:${SHEETNAME} -> (none); Role envelope:C_DEC_CORE_input_fault_switch_J_E1_SIG_FALL__U_1 -> (none)
- C4672: Island IO_JACK:${SHEETNAME} -> (none); Role envelope:C_DEC_CORE_PACK_OPA4196IDR_4_0 -> (none)
- C4673: Island IO_JACK:${SHEETNAME} -> (none); Role envelope:C_DEC_CORE_PACK_OPA4196IDR_4_1 -> (none)
- C4674: Island IO_JACK:${SHEETNAME} -> (none); Role envelope:C_DEC_LED_PACK_OPA4196IDR_0_0 -> (none)
- C4675: Island IO_JACK:${SHEETNAME} -> (none); Role envelope:C_DEC_LED_PACK_OPA4196IDR_0_1 -> (none)
- C4676: Island IO_JACK:${SHEETNAME} -> (none); Role envelope:C_DEC_LED_PACK_OPA4196IDR_1_0 -> (none)
- C4677: Island IO_JACK:${SHEETNAME} -> (none); Role envelope:C_DEC_LED_PACK_OPA4196IDR_1_1 -> (none)
- D1801, D1802, D1803: Island IO_JACK:${SHEETNAME} -> (none); Role magnitude_indicator:LED -> (none)
- D4601, D4602, D4603: Island IO_JACK:${SHEETNAME} -> (none); Role high_impedance_input:D -> (none)
- D4607, D4612, D4617: Island IO_JACK:${SHEETNAME} -> (none); Role magnitude_indicator:D1 -> (none)
- D4608, D4613, D4618: Island IO_JACK:${SHEETNAME} -> (none); Role magnitude_indicator:D2 -> (none)
- D4609, D4614, D4619: Island IO_JACK:${SHEETNAME} -> (none); Role magnitude_indicator:D3 -> (none)
- D4610, D4615, D4620: Island IO_JACK:${SHEETNAME} -> (none); Role magnitude_indicator:D4 -> (none)
- J1801: Island IO_JACK:${SHEETNAME} -> (none); Role envelope:J_SIG -> (none)
- J1802: Island IO_JACK:${SHEETNAME} -> (none); Role envelope:J_RISE -> (none)
- J1803: Island IO_JACK:${SHEETNAME} -> (none); Role envelope:J_FALL -> (none)
- J1804: Island IO_JACK:${SHEETNAME} -> (none); Role envelope:J_ENV -> (none)
- J1805: Island IO_JACK:${SHEETNAME} -> (none); Role envelope:J_BIP -> (none)
- J1806: Island IO_JACK:${SHEETNAME} -> (none); Role envelope:J_EOC -> (none)
- J1807: Island IO_JACK:${SHEETNAME} -> (none); Role envelope:J_STG -> (none)
- R4605, R4609, R4613: Island IO_JACK:${SHEETNAME} -> (none); Role input_fault_switch:R_EN -> (none)
- R4606, R4610, R4614: Island IO_JACK:${SHEETNAME} -> (none); Role input_fault_switch:R_DRIVE -> (none)
- R4607, R4611, R4615: Island IO_JACK:${SHEETNAME} -> (none); Role high_impedance_input:R_PD -> (none)
- R4608, R4612, R4616: Island IO_JACK:${SHEETNAME} -> (none); Role high_impedance_input:R_LIMIT -> (none)
- RB4605, RB4607, RB4609, RB4611: Island IO_JACK:${SHEETNAME} -> (none); Role general_output:R_ISO_A -> (none)
- RB4606, RB4608, RB4610, RB4612: Island IO_JACK:${SHEETNAME} -> (none); Role general_output:R_ISO_B -> (none)
- RB4613, RB4614, RB4615: Island IO_JACK:${SHEETNAME} -> (none); Role magnitude_indicator:R_SENSE -> (none)
- U4602, U4603, U4604: Island IO_JACK:${SHEETNAME} -> (none); Role input_fault_switch:U -> (none)
- U4646: Island IO_JACK:${SHEETNAME} -> (none); LogicalCellKey high_impedance_input_J_E1_SIG_FALL__A.1 -> (none); Role high_impedance_input:A -> (none)
- U4646: Island IO_JACK:${SHEETNAME} -> (none); LogicalCellKey high_impedance_input_J_E1_SIG_RISE__A.1 -> (none); Role high_impedance_input:A -> (none)
- U4646: Island IO_JACK:${SHEETNAME} -> (none); LogicalCellKey high_impedance_input_J_E1_SIG_SIG__A.1 -> (none); Role high_impedance_input:A -> (none)
- U4646: Island IO_JACK:${SHEETNAME} -> (none); LogicalCellKey general_output_J_E1_SIG_ENV__A.1 -> (none); Role general_output:A -> (none)
- U4646, U4647, U4648: Island IO_JACK:${SHEETNAME} -> (none); Role envelope:package supply -> (none)
- U4647: Island IO_JACK:${SHEETNAME} -> (none); LogicalCellKey general_output_J_E1_SIG_EOC__A.1 -> (none); Role general_output:A -> (none)
- U4647: Island IO_JACK:${SHEETNAME} -> (none); LogicalCellKey general_output_J_E1_SIG_STG__A.1 -> (none); Role general_output:A -> (none)
- U4647: Island IO_JACK:${SHEETNAME} -> (none); LogicalCellKey general_output_J_E1_SIG_BIP__A.1 -> (none); Role general_output:A -> (none)
- U4647: Island IO_JACK:${SHEETNAME} -> (none); LogicalCellKey magnitude_indicator_L_E1_SIG_mag_SIG__A.1 -> (none); Role magnitude_indicator:A -> (none)
- U4648: Island IO_JACK:${SHEETNAME} -> (none); LogicalCellKey magnitude_indicator_L_E1_RISE_mag_RISE__A.1 -> (none); Role magnitude_indicator:A -> (none)
- U4648: Island IO_JACK:${SHEETNAME} -> (none); LogicalCellKey magnitude_indicator_L_E1_FALL_mag_FALL__A.1 -> (none); Role magnitude_indicator:A -> (none)
- U4648: Island IO_JACK:${SHEETNAME} -> (none); Role envelope:unused grounded follower -> (none)
