File: boards/osc-jack/sheets/filter_F1_J.kicad_sch (KiCad schematic)
At the start: 81 parts, among them J601 WQP518MA, J602 WQP518MA, J603 WQP518MA, J604 WQP518MA, J605 WQP518MA, J606 WQP518MA, J607 WQP518MA, J608 WQP518MA, U2102 ADG5412FBRUZ, U2103 ADG5412FBRUZ, U2104 ADG5412FBRUZ, U2105 ADG5412FBRUZ, U2117 OPA4196IDR, U2118 OPA4196IDR, U2119 OPA4196IDR

Commit message: Reserve clear jack-board geometry and align projected schematic fields
Parts:
- C2117: Island IO_JACK:${SHEETNAME} -> (none); Role filter:C_DEC_input_fault_switch_J_F1_IN_IN__U_0 -> (none)
- C2118: Island IO_JACK:${SHEETNAME} -> (none); Role filter:C_DEC_input_fault_switch_J_F1_IN_IN__U_1 -> (none)
- C2119: Island IO_JACK:${SHEETNAME} -> (none); Role filter:C_DEC_input_fault_switch_J_F1_IN_FREQ__U_0 -> (none)
- C2120: Island IO_JACK:${SHEETNAME} -> (none); Role filter:C_DEC_input_fault_switch_J_F1_IN_FREQ__U_1 -> (none)
- C2121: Island IO_JACK:${SHEETNAME} -> (none); Role filter:C_DEC_input_fault_switch_J_F1_IN_RES__U_0 -> (none)
- C2122: Island IO_JACK:${SHEETNAME} -> (none); Role filter:C_DEC_input_fault_switch_J_F1_IN_RES__U_1 -> (none)
- C2123: Island IO_JACK:${SHEETNAME} -> (none); Role filter:C_DEC_input_fault_switch_J_F1_IN_GAIN__U_0 -> (none)
- C2124: Island IO_JACK:${SHEETNAME} -> (none); Role filter:C_DEC_input_fault_switch_J_F1_IN_GAIN__U_1 -> (none)
- C2147: Island IO_JACK:${SHEETNAME} -> (none); Role filter:C_DEC_PACK_OPA4196IDR_7_0 -> (none)
- C2148: Island IO_JACK:${SHEETNAME} -> (none); Role filter:C_DEC_PACK_OPA4196IDR_7_1 -> (none)
- C2149: Island IO_JACK:${SHEETNAME} -> (none); Role filter:C_DEC_PACK_OPA4196IDR_8_0 -> (none)
- C2150: Island IO_JACK:${SHEETNAME} -> (none); Role filter:C_DEC_PACK_OPA4196IDR_8_1 -> (none)
- C2151: Island IO_JACK:${SHEETNAME} -> (none); Role filter:C_DEC_PACK_OPA4196IDR_0_0 -> (none)
- C2152: Island IO_JACK:${SHEETNAME} -> (none); Role filter:C_DEC_PACK_OPA4196IDR_0_1 -> (none)
- D2101, D2102, D2103, D2104: Island IO_JACK:${SHEETNAME} -> (none); Role high_impedance_input:D -> (none)
- D2125, D2130, D2135, D2140: Island FILTER_LEDS:${SHEETNAME} -> (none); Role magnitude_indicator:D1 -> (none)
- D2126, D2131, D2136, D2141: Island FILTER_LEDS:${SHEETNAME} -> (none); Role magnitude_indicator:D2 -> (none)
- D2127, D2132, D2137, D2142: Island FILTER_LEDS:${SHEETNAME} -> (none); Role magnitude_indicator:D3 -> (none)
- D2128, D2133, D2138, D2143: Island FILTER_LEDS:${SHEETNAME} -> (none); Role magnitude_indicator:D4 -> (none)
- D601, D602, D603, D604: Island FILTER_LEDS:${SHEETNAME} -> (none); Role magnitude_indicator:LED -> (none)
- J601: Island IO_JACK:${SHEETNAME} -> (none); Role filter:J_IN -> (none)
- J602: Island IO_JACK:${SHEETNAME} -> (none); Role filter:J_FREQ -> (none)
- J603: Island IO_JACK:${SHEETNAME} -> (none); Role filter:J_RES -> (none)
- J604: Island IO_JACK:${SHEETNAME} -> (none); Role filter:J_GAIN -> (none)
- J605: Island IO_JACK:${SHEETNAME} -> (none); Role filter:J_LP -> (none)
- J606: Island IO_JACK:${SHEETNAME} -> (none); Role filter:J_BP -> (none)
- J607: Island IO_JACK:${SHEETNAME} -> (none); Role filter:J_HP -> (none)
- J608: Island IO_JACK:${SHEETNAME} -> (none); Role filter:J_OUT -> (none)
- R2105, R2109, R2113, R2117: Island IO_JACK:${SHEETNAME} -> (none); Role input_fault_switch:R_EN -> (none)
- R2106, R2110, R2114, R2118: Island IO_JACK:${SHEETNAME} -> (none); Role input_fault_switch:R_DRIVE -> (none)
- R2107, R2111, R2115, R2119: Island IO_JACK:${SHEETNAME} -> (none); Role high_impedance_input:R_PD -> (none)
- R2108, R2112, R2116, R2120: Island IO_JACK:${SHEETNAME} -> (none); Role high_impedance_input:R_LIMIT -> (none)
- RB2106, RB2108, RB2110, RB2112: Island IO_JACK:${SHEETNAME} -> (none); Role general_output:R_ISO_A -> (none)
- RB2107, RB2109, RB2111, RB2113: Island IO_JACK:${SHEETNAME} -> (none); Role general_output:R_ISO_B -> (none)
- RB2114, RB2115, RB2116, RB2117: Island FILTER_LEDS:${SHEETNAME} -> (none); Role magnitude_indicator:R_SENSE -> (none)
- U2102, U2103, U2104, U2105: Island IO_JACK:${SHEETNAME} -> (none); Role input_fault_switch:U -> (none)
- U2117: Island IO_JACK:${SHEETNAME} -> (none); LogicalCellKey high_impedance_input_J_F1_IN_FREQ__A.1 -> (none); Role high_impedance_input:A -> (none)
- U2117: Island IO_JACK:${SHEETNAME} -> (none); LogicalCellKey high_impedance_input_J_F1_IN_RES__A.1 -> (none); Role high_impedance_input:A -> (none)
- U2117, U2118, U2119: Island IO_JACK:${SHEETNAME} -> (none); Role filter:package supply -> (none)
- U2117: Island IO_JACK:${SHEETNAME} -> (none); LogicalCellKey high_impedance_input_J_F1_IN_IN__A.1 -> (none); Role high_impedance_input:A -> (none)
- U2117: Island IO_JACK:${SHEETNAME} -> (none); LogicalCellKey high_impedance_input_J_F1_IN_GAIN__A.1 -> (none); Role high_impedance_input:A -> (none)
- U2118: Island IO_JACK:${SHEETNAME} -> (none); LogicalCellKey general_output_J_F1_IN_BP__A.1 -> (none); Role general_output:A -> (none)
- U2118: Island IO_JACK:${SHEETNAME} -> (none); LogicalCellKey general_output_J_F1_IN_OUT__A.1 -> (none); Role general_output:A -> (none)
- U2118: Island IO_JACK:${SHEETNAME} -> (none); LogicalCellKey general_output_J_F1_IN_HP__A.1 -> (none); Role general_output:A -> (none)
- U2118: Island IO_JACK:${SHEETNAME} -> (none); LogicalCellKey general_output_J_F1_IN_LP__A.1 -> (none); Role general_output:A -> (none)
- U2119: Island FILTER_LEDS:${SHEETNAME} -> (none); LogicalCellKey magnitude_indicator_L_F1_FREQ_mag_FREQ__A.1 -> (none); Role magnitude_indicator:A -> (none)
- U2119: Island FILTER_LEDS:${SHEETNAME} -> (none); LogicalCellKey magnitude_indicator_L_F1_IN_mag_IN__A.1 -> (none); Role magnitude_indicator:A -> (none)
- U2119: Island FILTER_LEDS:${SHEETNAME} -> (none); LogicalCellKey magnitude_indicator_L_F1_RES_mag_RES__A.1 -> (none); Role magnitude_indicator:A -> (none)
- U2119: Island FILTER_LEDS:${SHEETNAME} -> (none); LogicalCellKey magnitude_indicator_L_F1_GAIN_mag_GAIN__A.1 -> (none); Role magnitude_indicator:A -> (none)
