File: boards/osc-jack/sheets/filter_F3_J.kicad_sch (KiCad schematic)
At the start: 81 parts, among them J801 WQP518MA, J802 WQP518MA, J803 WQP518MA, J804 WQP518MA, J805 WQP518MA, J806 WQP518MA, J807 WQP518MA, J808 WQP518MA, U2302 ADG5412FBRUZ, U2303 ADG5412FBRUZ, U2304 ADG5412FBRUZ, U2305 ADG5412FBRUZ, U2317 OPA4196IDR, U2318 OPA4196IDR, U2319 OPA4196IDR

Commit message: Reserve clear jack-board geometry and align projected schematic fields
Parts:
- C2317: Island IO_JACK:${SHEETNAME} -> (none); Role filter:C_DEC_input_fault_switch_J_F1_IN_IN__U_0 -> (none)
- C2318: Island IO_JACK:${SHEETNAME} -> (none); Role filter:C_DEC_input_fault_switch_J_F1_IN_IN__U_1 -> (none)
- C2319: Island IO_JACK:${SHEETNAME} -> (none); Role filter:C_DEC_input_fault_switch_J_F1_IN_FREQ__U_0 -> (none)
- C2320: Island IO_JACK:${SHEETNAME} -> (none); Role filter:C_DEC_input_fault_switch_J_F1_IN_FREQ__U_1 -> (none)
- C2321: Island IO_JACK:${SHEETNAME} -> (none); Role filter:C_DEC_input_fault_switch_J_F1_IN_RES__U_0 -> (none)
- C2322: Island IO_JACK:${SHEETNAME} -> (none); Role filter:C_DEC_input_fault_switch_J_F1_IN_RES__U_1 -> (none)
- C2323: Island IO_JACK:${SHEETNAME} -> (none); Role filter:C_DEC_input_fault_switch_J_F1_IN_GAIN__U_0 -> (none)
- C2324: Island IO_JACK:${SHEETNAME} -> (none); Role filter:C_DEC_input_fault_switch_J_F1_IN_GAIN__U_1 -> (none)
- C2347: Island IO_JACK:${SHEETNAME} -> (none); Role filter:C_DEC_PACK_OPA4196IDR_7_0 -> (none)
- C2348: Island IO_JACK:${SHEETNAME} -> (none); Role filter:C_DEC_PACK_OPA4196IDR_7_1 -> (none)
- C2349: Island IO_JACK:${SHEETNAME} -> (none); Role filter:C_DEC_PACK_OPA4196IDR_8_0 -> (none)
- C2350: Island IO_JACK:${SHEETNAME} -> (none); Role filter:C_DEC_PACK_OPA4196IDR_8_1 -> (none)
- C2351: Island IO_JACK:${SHEETNAME} -> (none); Role filter:C_DEC_PACK_OPA4196IDR_0_0 -> (none)
- C2352: Island IO_JACK:${SHEETNAME} -> (none); Role filter:C_DEC_PACK_OPA4196IDR_0_1 -> (none)
- D2301, D2302, D2303, D2304: Island IO_JACK:${SHEETNAME} -> (none); Role high_impedance_input:D -> (none)
- D2325, D2330, D2335, D2340: Island FILTER_LEDS:${SHEETNAME} -> (none); Role magnitude_indicator:D1 -> (none)
- D2326, D2331, D2336, D2341: Island FILTER_LEDS:${SHEETNAME} -> (none); Role magnitude_indicator:D2 -> (none)
- D2327, D2332, D2337, D2342: Island FILTER_LEDS:${SHEETNAME} -> (none); Role magnitude_indicator:D3 -> (none)
- D2328, D2333, D2338, D2343: Island FILTER_LEDS:${SHEETNAME} -> (none); Role magnitude_indicator:D4 -> (none)
- D801, D802, D803, D804: Island FILTER_LEDS:${SHEETNAME} -> (none); Role magnitude_indicator:LED -> (none)
- J801: Island IO_JACK:${SHEETNAME} -> (none); Role filter:J_IN -> (none)
- J802: Island IO_JACK:${SHEETNAME} -> (none); Role filter:J_FREQ -> (none)
- J803: Island IO_JACK:${SHEETNAME} -> (none); Role filter:J_RES -> (none)
- J804: Island IO_JACK:${SHEETNAME} -> (none); Role filter:J_GAIN -> (none)
- J805: Island IO_JACK:${SHEETNAME} -> (none); Role filter:J_LP -> (none)
- J806: Island IO_JACK:${SHEETNAME} -> (none); Role filter:J_BP -> (none)
- J807: Island IO_JACK:${SHEETNAME} -> (none); Role filter:J_HP -> (none)
- J808: Island IO_JACK:${SHEETNAME} -> (none); Role filter:J_OUT -> (none)
- R2305, R2309, R2313, R2317: Island IO_JACK:${SHEETNAME} -> (none); Role input_fault_switch:R_EN -> (none)
- R2306, R2310, R2314, R2318: Island IO_JACK:${SHEETNAME} -> (none); Role input_fault_switch:R_DRIVE -> (none)
- R2307, R2311, R2315, R2319: Island IO_JACK:${SHEETNAME} -> (none); Role high_impedance_input:R_PD -> (none)
- R2308, R2312, R2316, R2320: Island IO_JACK:${SHEETNAME} -> (none); Role high_impedance_input:R_LIMIT -> (none)
- RB2306, RB2308, RB2310, RB2312: Island IO_JACK:${SHEETNAME} -> (none); Role general_output:R_ISO_A -> (none)
- RB2307, RB2309, RB2311, RB2313: Island IO_JACK:${SHEETNAME} -> (none); Role general_output:R_ISO_B -> (none)
- RB2314, RB2315, RB2316, RB2317: Island FILTER_LEDS:${SHEETNAME} -> (none); Role magnitude_indicator:R_SENSE -> (none)
- U2302, U2303, U2304, U2305: Island IO_JACK:${SHEETNAME} -> (none); Role input_fault_switch:U -> (none)
- U2317: Island IO_JACK:${SHEETNAME} -> (none); LogicalCellKey high_impedance_input_J_F1_IN_FREQ__A.1 -> (none); Role high_impedance_input:A -> (none)
- U2317: Island IO_JACK:${SHEETNAME} -> (none); LogicalCellKey high_impedance_input_J_F1_IN_IN__A.1 -> (none); Role high_impedance_input:A -> (none)
- U2317, U2318, U2319: Island IO_JACK:${SHEETNAME} -> (none); Role filter:package supply -> (none)
- U2317: Island IO_JACK:${SHEETNAME} -> (none); LogicalCellKey high_impedance_input_J_F1_IN_GAIN__A.1 -> (none); Role high_impedance_input:A -> (none)
- U2317: Island IO_JACK:${SHEETNAME} -> (none); LogicalCellKey high_impedance_input_J_F1_IN_RES__A.1 -> (none); Role high_impedance_input:A -> (none)
- U2318: Island IO_JACK:${SHEETNAME} -> (none); LogicalCellKey general_output_J_F1_IN_OUT__A.1 -> (none); Role general_output:A -> (none)
- U2318: Island IO_JACK:${SHEETNAME} -> (none); LogicalCellKey general_output_J_F1_IN_HP__A.1 -> (none); Role general_output:A -> (none)
- U2318: Island IO_JACK:${SHEETNAME} -> (none); LogicalCellKey general_output_J_F1_IN_BP__A.1 -> (none); Role general_output:A -> (none)
- U2318: Island IO_JACK:${SHEETNAME} -> (none); LogicalCellKey general_output_J_F1_IN_LP__A.1 -> (none); Role general_output:A -> (none)
- U2319: Island FILTER_LEDS:${SHEETNAME} -> (none); LogicalCellKey magnitude_indicator_L_F1_RES_mag_RES__A.1 -> (none); Role magnitude_indicator:A -> (none)
- U2319: Island FILTER_LEDS:${SHEETNAME} -> (none); LogicalCellKey magnitude_indicator_L_F1_GAIN_mag_GAIN__A.1 -> (none); Role magnitude_indicator:A -> (none)
- U2319: Island FILTER_LEDS:${SHEETNAME} -> (none); LogicalCellKey magnitude_indicator_L_F1_FREQ_mag_FREQ__A.1 -> (none); Role magnitude_indicator:A -> (none)
- U2319: Island FILTER_LEDS:${SHEETNAME} -> (none); LogicalCellKey magnitude_indicator_L_F1_IN_mag_IN__A.1 -> (none); Role magnitude_indicator:A -> (none)
