File: boards/osc-jack/sheets/mix4_vca_M4A_J.kicad_sch (KiCad schematic)
At the start: 106 parts, among them J1101 WQP518MA, J1102 WQP518MA, J1103 WQP518MA, J1104 WQP518MA, J1105 WQP518MA, J1106 WQP518MA, U8302 ADG5412FBRUZ, U8303 ADG5412FBRUZ, U8304 ADG5412FBRUZ, U8305 ADG5412FBRUZ, U8306 ADG5412FBRUZ, U8314 OPA4196IDR, U8315 LM393BIDR, U8316 LM393BIDR, U8317 OPA4196IDR, U8318 OPA4196IDR, U8319 OPA4196IDR

Commit message: Reserve clear jack-board geometry and align projected schematic fields
Parts:
- C8316: Island IO_JACK:${SHEETNAME} -> (none); Role mix4_vca:C_DEC_input_fault_switch_J_M4A_1_1__U_0 -> (none)
- C8317, C8351: Island IO_JACK:${SHEETNAME} -> (none); Role mix4_vca:C_DEC_input_fault_switch_J_M4A_1_1__U_1 -> (none)
- C8318: Island IO_JACK:${SHEETNAME} -> (none); Role mix4_vca:C_DEC_input_fault_switch_J_M4A_1_2__U_0 -> (none)
- C8319: Island IO_JACK:${SHEETNAME} -> (none); Role mix4_vca:C_DEC_input_fault_switch_J_M4A_1_2__U_1 -> (none)
- C8320: Island IO_JACK:${SHEETNAME} -> (none); Role mix4_vca:C_DEC_input_fault_switch_J_M4A_1_3__U_0 -> (none)
- C8321: Island IO_JACK:${SHEETNAME} -> (none); Role mix4_vca:C_DEC_input_fault_switch_J_M4A_1_3__U_1 -> (none)
- C8322: Island IO_JACK:${SHEETNAME} -> (none); Role mix4_vca:C_DEC_input_fault_switch_J_M4A_1_4__U_0 -> (none)
- C8323: Island IO_JACK:${SHEETNAME} -> (none); Role mix4_vca:C_DEC_input_fault_switch_J_M4A_1_4__U_1 -> (none)
- C8324: Island IO_JACK:${SHEETNAME} -> (none); Role mix4_vca:C_DEC_input_fault_switch_J_M4A_1_ATTEN__U_0 -> (none)
- C8325: Island IO_JACK:${SHEETNAME} -> (none); Role mix4_vca:C_DEC_input_fault_switch_J_M4A_1_ATTEN__U_1 -> (none)
- C8328: Island IO_JACK:${SHEETNAME} -> (none); Role mix4_vca:C_DEC_PACK_OPA4197IPWR_0_0 -> (none)
- C8329: Island IO_JACK:${SHEETNAME} -> (none); Role mix4_vca:C_DEC_PACK_OPA4197IPWR_0_1 -> (none)
- C8330, C8346: Island IO_JACK:${SHEETNAME} -> (none); Role mix4_vca:C_DEC_PACK_OPA4196IDR_0_0 -> (none)
- C8331, C8347: Island IO_JACK:${SHEETNAME} -> (none); Role mix4_vca:C_DEC_PACK_OPA4196IDR_0_1 -> (none)
- C8344: Island IO_JACK:${SHEETNAME} -> (none); Role mix4_vca:C_DEC_clip_detector_L_M4A_SUM_clip_SUM__UN_0 -> (none)
- C8345: Island IO_JACK:${SHEETNAME} -> (none); Role mix4_vca:C_DEC_clip_detector_L_M4A_SUM_clip_SUM__UN_1 -> (none)
- C8348: Island IO_JACK:${SHEETNAME} -> (none); Role mix4_vca:C_DEC_PACK_OPA4196IDR_1_0 -> (none)
- C8349: Island IO_JACK:${SHEETNAME} -> (none); Role mix4_vca:C_DEC_PACK_OPA4196IDR_1_1 -> (none)
- C8350: Island IO_JACK:${SHEETNAME} -> (none); Role mix4_vca:C_DEC_reference_generator_J_M4A_1_LOCAL__U_0 -> (none)
- D1101, D1102, D1103, D1104, D1105, D1106: Island IO_JACK:${SHEETNAME} -> (none); Role magnitude_indicator:LED -> (none)
- D11061: Island IO_JACK:${SHEETNAME} -> (none); Role clip_detector:LED -> (none)
- D8308, D8309, D8310, D8311, D8312: Island IO_JACK:${SHEETNAME} -> (none); Role high_impedance_input:D -> (none)
- D8315, D8319, D8323, D8327, D8331, D8335: Island IO_JACK:${SHEETNAME} -> (none); Role magnitude_indicator:D1 -> (none)
- D8316, D8320, D8324, D8328, D8332, D8336: Island IO_JACK:${SHEETNAME} -> (none); Role magnitude_indicator:D2 -> (none)
- D8317, D8321, D8325, D8329, D8333, D8337: Island IO_JACK:${SHEETNAME} -> (none); Role magnitude_indicator:D3 -> (none)
- D8318, D8322, D8326, D8330, D8334, D8338: Island IO_JACK:${SHEETNAME} -> (none); Role magnitude_indicator:D4 -> (none)
- J1101: Island IO_JACK:${SHEETNAME} -> (none); Role mix4_vca:J_1 -> (none)
- J1102: Island IO_JACK:${SHEETNAME} -> (none); Role mix4_vca:J_2 -> (none)
- J1103: Island IO_JACK:${SHEETNAME} -> (none); Role mix4_vca:J_3 -> (none)
- J1104: Island IO_JACK:${SHEETNAME} -> (none); Role mix4_vca:J_4 -> (none)
- J1105: Island IO_JACK:${SHEETNAME} -> (none); Role mix4_vca:J_ATTEN -> (none)
- J1106: Island IO_JACK:${SHEETNAME} -> (none); Role mix4_vca:J_SUM -> (none)
- R8305, R8315, R8325, R8335, R8350: Island IO_JACK:${SHEETNAME} -> (none); Role input_fault_switch:R_EN -> (none)
- R8306, R8316, R8326, R8336, R8351: Island IO_JACK:${SHEETNAME} -> (none); Role input_fault_switch:R_DRIVE -> (none)
- R8307, R8317, R8327, R8337, R8352: Island IO_JACK:${SHEETNAME} -> (none); Role high_impedance_input:R_PD -> (none)
- R8308, R8318, R8328, R8338, R8353: Island IO_JACK:${SHEETNAME} -> (none); Role high_impedance_input:R_LIMIT -> (none)
- R8381: Island IO_JACK:${SHEETNAME} -> (none); Role general_output:R_ISO_A -> (none)
- R8382: Island IO_JACK:${SHEETNAME} -> (none); Role general_output:R_ISO_B -> (none)
- R8383, R8384, R8385, R8386, R8387, R8388: Island IO_JACK:${SHEETNAME} -> (none); Role magnitude_indicator:R_SENSE -> (none)
- R8389: Island IO_JACK:${SHEETNAME} -> (none); Role clip_detector:R_TOP -> (none)
- R8390: Island IO_JACK:${SHEETNAME} -> (none); Role clip_detector:R_BOT -> (none)
- R8391: Island IO_JACK:${SHEETNAME} -> (none); Role clip_detector:R_LED -> (none)
- U8302, U8303, U8304, U8305, U8306: Island IO_JACK:${SHEETNAME} -> (none); Role input_fault_switch:U -> (none)
- U8314: Island IO_JACK:${SHEETNAME} -> (none); LogicalCellKey high_impedance_input_J_M4A_1_3__A.1 -> (none); Role high_impedance_input:A -> (none)
- U8314: Island IO_JACK:${SHEETNAME} -> (none); LogicalCellKey high_impedance_input_J_M4A_1_2__A.1 -> (none); Role high_impedance_input:A -> (none)
- U8314: Island IO_JACK:${SHEETNAME} -> (none); LogicalCellKey high_impedance_input_J_M4A_1_4__A.1 -> (none); Role high_impedance_input:A -> (none)
- U8314, U8317, U8318, U8319: Island IO_JACK:${SHEETNAME} -> (none); Role mix4_vca:package supply -> (none)
- U8314: Island IO_JACK:${SHEETNAME} -> (none); LogicalCellKey high_impedance_input_J_M4A_1_1__A.1 -> (none); Role high_impedance_input:A -> (none)
- U8315: Island IO_JACK:${SHEETNAME} -> (none); Role clip_detector:UP -> (none)
- U8316: Island IO_JACK:${SHEETNAME} -> (none); Role clip_detector:UN -> (none)
- U8317: Island IO_JACK:${SHEETNAME} -> (none); LogicalCellKey general_output_J_M4A_1_SUM__A.1 -> (none); Role general_output:A -> (none)
- U8317: Island IO_JACK:${SHEETNAME} -> (none); LogicalCellKey high_impedance_input_J_M4A_1_ATTEN__A.1 -> (none); Role high_impedance_input:A -> (none)
- U8317: Island IO_JACK:${SHEETNAME} -> (none); LogicalCellKey magnitude_indicator_L_M4A_1_mag_1__A.1 -> (none); Role magnitude_indicator:A -> (none)
- U8317: Island IO_JACK:${SHEETNAME} -> (none); LogicalCellKey magnitude_indicator_L_M4A_2_mag_2__A.1 -> (none); Role magnitude_indicator:A -> (none)
- U8318: Island IO_JACK:${SHEETNAME} -> (none); LogicalCellKey magnitude_indicator_L_M4A_ATTEN_mag_ATTEN__A.1 -> (none); Role magnitude_indicator:A -> (none)
- U8318: Island IO_JACK:${SHEETNAME} -> (none); LogicalCellKey magnitude_indicator_L_M4A_3_mag_3__A.1 -> (none); Role magnitude_indicator:A -> (none)
- U8318: Island IO_JACK:${SHEETNAME} -> (none); LogicalCellKey magnitude_indicator_L_M4A_4_mag_4__A.1 -> (none); Role magnitude_indicator:A -> (none)
- U8318: Island IO_JACK:${SHEETNAME} -> (none); LogicalCellKey magnitude_indicator_L_M4A_SUM_mag_SUM__A.1 -> (none); Role magnitude_indicator:A -> (none)
- U8319: Island IO_JACK:${SHEETNAME} -> (none); Role mix4_vca:unused grounded follower -> (none)
- U8319: Island IO_JACK:${SHEETNAME} -> (none); LogicalCellKey clip_detector_L_M4A_SUM_clip_SUM__A.1 -> (none); Role clip_detector:A -> (none)
