File: boards/osc-jack/sheets/mix4_vca_M4B_J.kicad_sch (KiCad schematic)
At the start: 106 parts, among them J1201 WQP518MA, J1202 WQP518MA, J1203 WQP518MA, J1204 WQP518MA, J1205 WQP518MA, J1206 WQP518MA, U8402 ADG5412FBRUZ, U8403 ADG5412FBRUZ, U8404 ADG5412FBRUZ, U8405 ADG5412FBRUZ, U8406 ADG5412FBRUZ, U8414 OPA4196IDR, U8415 LM393BIDR, U8416 LM393BIDR, U8417 OPA4196IDR, U8418 OPA4196IDR, U8419 OPA4196IDR

Commit message: Reserve clear jack-board geometry and align projected schematic fields
Parts:
- C8416: Island IO_JACK:${SHEETNAME} -> (none); Role mix4_vca:C_DEC_input_fault_switch_J_M4A_1_1__U_0 -> (none)
- C8417, C8451: Island IO_JACK:${SHEETNAME} -> (none); Role mix4_vca:C_DEC_input_fault_switch_J_M4A_1_1__U_1 -> (none)
- C8418: Island IO_JACK:${SHEETNAME} -> (none); Role mix4_vca:C_DEC_input_fault_switch_J_M4A_1_2__U_0 -> (none)
- C8419: Island IO_JACK:${SHEETNAME} -> (none); Role mix4_vca:C_DEC_input_fault_switch_J_M4A_1_2__U_1 -> (none)
- C8420: Island IO_JACK:${SHEETNAME} -> (none); Role mix4_vca:C_DEC_input_fault_switch_J_M4A_1_3__U_0 -> (none)
- C8421: Island IO_JACK:${SHEETNAME} -> (none); Role mix4_vca:C_DEC_input_fault_switch_J_M4A_1_3__U_1 -> (none)
- C8422: Island IO_JACK:${SHEETNAME} -> (none); Role mix4_vca:C_DEC_input_fault_switch_J_M4A_1_4__U_0 -> (none)
- C8423: Island IO_JACK:${SHEETNAME} -> (none); Role mix4_vca:C_DEC_input_fault_switch_J_M4A_1_4__U_1 -> (none)
- C8424: Island IO_JACK:${SHEETNAME} -> (none); Role mix4_vca:C_DEC_input_fault_switch_J_M4A_1_ATTEN__U_0 -> (none)
- C8425: Island IO_JACK:${SHEETNAME} -> (none); Role mix4_vca:C_DEC_input_fault_switch_J_M4A_1_ATTEN__U_1 -> (none)
- C8428: Island IO_JACK:${SHEETNAME} -> (none); Role mix4_vca:C_DEC_PACK_OPA4197IPWR_0_0 -> (none)
- C8429: Island IO_JACK:${SHEETNAME} -> (none); Role mix4_vca:C_DEC_PACK_OPA4197IPWR_0_1 -> (none)
- C8430, C8446: Island IO_JACK:${SHEETNAME} -> (none); Role mix4_vca:C_DEC_PACK_OPA4196IDR_0_0 -> (none)
- C8431, C8447: Island IO_JACK:${SHEETNAME} -> (none); Role mix4_vca:C_DEC_PACK_OPA4196IDR_0_1 -> (none)
- C8444: Island IO_JACK:${SHEETNAME} -> (none); Role mix4_vca:C_DEC_clip_detector_L_M4A_SUM_clip_SUM__UN_0 -> (none)
- C8445: Island IO_JACK:${SHEETNAME} -> (none); Role mix4_vca:C_DEC_clip_detector_L_M4A_SUM_clip_SUM__UN_1 -> (none)
- C8448: Island IO_JACK:${SHEETNAME} -> (none); Role mix4_vca:C_DEC_PACK_OPA4196IDR_1_0 -> (none)
- C8449: Island IO_JACK:${SHEETNAME} -> (none); Role mix4_vca:C_DEC_PACK_OPA4196IDR_1_1 -> (none)
- C8450: Island IO_JACK:${SHEETNAME} -> (none); Role mix4_vca:C_DEC_reference_generator_J_M4A_1_LOCAL__U_0 -> (none)
- D1201, D1202, D1203, D1204, D1205, D1206: Island IO_JACK:${SHEETNAME} -> (none); Role magnitude_indicator:LED -> (none)
- D12061: Island IO_JACK:${SHEETNAME} -> (none); Role clip_detector:LED -> (none)
- D8408, D8409, D8410, D8411, D8412: Island IO_JACK:${SHEETNAME} -> (none); Role high_impedance_input:D -> (none)
- D8415, D8419, D8423, D8427, D8431, D8435: Island IO_JACK:${SHEETNAME} -> (none); Role magnitude_indicator:D1 -> (none)
- D8416, D8420, D8424, D8428, D8432, D8436: Island IO_JACK:${SHEETNAME} -> (none); Role magnitude_indicator:D2 -> (none)
- D8417, D8421, D8425, D8429, D8433, D8437: Island IO_JACK:${SHEETNAME} -> (none); Role magnitude_indicator:D3 -> (none)
- D8418, D8422, D8426, D8430, D8434, D8438: Island IO_JACK:${SHEETNAME} -> (none); Role magnitude_indicator:D4 -> (none)
- J1201: Island IO_JACK:${SHEETNAME} -> (none); Role mix4_vca:J_1 -> (none)
- J1202: Island IO_JACK:${SHEETNAME} -> (none); Role mix4_vca:J_2 -> (none)
- J1203: Island IO_JACK:${SHEETNAME} -> (none); Role mix4_vca:J_3 -> (none)
- J1204: Island IO_JACK:${SHEETNAME} -> (none); Role mix4_vca:J_4 -> (none)
- J1205: Island IO_JACK:${SHEETNAME} -> (none); Role mix4_vca:J_ATTEN -> (none)
- J1206: Island IO_JACK:${SHEETNAME} -> (none); Role mix4_vca:J_SUM -> (none)
- R8405, R8415, R8425, R8435, R8450: Island IO_JACK:${SHEETNAME} -> (none); Role input_fault_switch:R_EN -> (none)
- R8406, R8416, R8426, R8436, R8451: Island IO_JACK:${SHEETNAME} -> (none); Role input_fault_switch:R_DRIVE -> (none)
- R8407, R8417, R8427, R8437, R8452: Island IO_JACK:${SHEETNAME} -> (none); Role high_impedance_input:R_PD -> (none)
- R8408, R8418, R8428, R8438, R8453: Island IO_JACK:${SHEETNAME} -> (none); Role high_impedance_input:R_LIMIT -> (none)
- R8481: Island IO_JACK:${SHEETNAME} -> (none); Role general_output:R_ISO_A -> (none)
- R8482: Island IO_JACK:${SHEETNAME} -> (none); Role general_output:R_ISO_B -> (none)
- R8483, R8484, R8485, R8486, R8487, R8488: Island IO_JACK:${SHEETNAME} -> (none); Role magnitude_indicator:R_SENSE -> (none)
- R8489: Island IO_JACK:${SHEETNAME} -> (none); Role clip_detector:R_TOP -> (none)
- R8490: Island IO_JACK:${SHEETNAME} -> (none); Role clip_detector:R_BOT -> (none)
- R8491: Island IO_JACK:${SHEETNAME} -> (none); Role clip_detector:R_LED -> (none)
- U8402, U8403, U8404, U8405, U8406: Island IO_JACK:${SHEETNAME} -> (none); Role input_fault_switch:U -> (none)
- U8414: Island IO_JACK:${SHEETNAME} -> (none); LogicalCellKey high_impedance_input_J_M4A_1_4__A.1 -> (none); Role high_impedance_input:A -> (none)
- U8414: Island IO_JACK:${SHEETNAME} -> (none); LogicalCellKey high_impedance_input_J_M4A_1_3__A.1 -> (none); Role high_impedance_input:A -> (none)
- U8414: Island IO_JACK:${SHEETNAME} -> (none); LogicalCellKey high_impedance_input_J_M4A_1_1__A.1 -> (none); Role high_impedance_input:A -> (none)
- U8414, U8417, U8418, U8419: Island IO_JACK:${SHEETNAME} -> (none); Role mix4_vca:package supply -> (none)
- U8414: Island IO_JACK:${SHEETNAME} -> (none); LogicalCellKey high_impedance_input_J_M4A_1_2__A.1 -> (none); Role high_impedance_input:A -> (none)
- U8415: Island IO_JACK:${SHEETNAME} -> (none); Role clip_detector:UP -> (none)
- U8416: Island IO_JACK:${SHEETNAME} -> (none); Role clip_detector:UN -> (none)
- U8417: Island IO_JACK:${SHEETNAME} -> (none); LogicalCellKey high_impedance_input_J_M4A_1_ATTEN__A.1 -> (none); Role high_impedance_input:A -> (none)
- U8417: Island IO_JACK:${SHEETNAME} -> (none); LogicalCellKey general_output_J_M4A_1_SUM__A.1 -> (none); Role general_output:A -> (none)
- U8417: Island IO_JACK:${SHEETNAME} -> (none); LogicalCellKey magnitude_indicator_L_M4A_2_mag_2__A.1 -> (none); Role magnitude_indicator:A -> (none)
- U8417: Island IO_JACK:${SHEETNAME} -> (none); LogicalCellKey magnitude_indicator_L_M4A_1_mag_1__A.1 -> (none); Role magnitude_indicator:A -> (none)
- U8418: Island IO_JACK:${SHEETNAME} -> (none); LogicalCellKey magnitude_indicator_L_M4A_ATTEN_mag_ATTEN__A.1 -> (none); Role magnitude_indicator:A -> (none)
- U8418: Island IO_JACK:${SHEETNAME} -> (none); LogicalCellKey magnitude_indicator_L_M4A_3_mag_3__A.1 -> (none); Role magnitude_indicator:A -> (none)
- U8418: Island IO_JACK:${SHEETNAME} -> (none); LogicalCellKey magnitude_indicator_L_M4A_4_mag_4__A.1 -> (none); Role magnitude_indicator:A -> (none)
- U8418: Island IO_JACK:${SHEETNAME} -> (none); LogicalCellKey magnitude_indicator_L_M4A_SUM_mag_SUM__A.1 -> (none); Role magnitude_indicator:A -> (none)
- U8419: Island IO_JACK:${SHEETNAME} -> (none); Role mix4_vca:unused grounded follower -> (none)
- U8419: Island IO_JACK:${SHEETNAME} -> (none); LogicalCellKey clip_detector_L_M4A_SUM_clip_SUM__A.1 -> (none); Role clip_detector:A -> (none)
