File: boards/osc-jack/sheets/mix5_M5A_J.kicad_sch (KiCad schematic)
At the start: 106 parts, among them J901 WQP518MA, J902 WQP518MA, J903 WQP518MA, J904 WQP518MA, J905 WQP518MA, J906 WQP518MA, U8102 ADG5412FBRUZ, U8103 ADG5412FBRUZ, U8104 ADG5412FBRUZ, U8105 ADG5412FBRUZ, U8106 ADG5412FBRUZ, U8112 OPA4196IDR, U8113 LM393BIDR, U8114 LM393BIDR, U8115 OPA4196IDR, U8116 OPA4196IDR, U8117 OPA4196IDR

Commit message: Reserve clear jack-board geometry and align projected schematic fields
Parts:
- C8115: Island IO_JACK:${SHEETNAME} -> (none); Role mix5:C_DEC_input_fault_switch_J_M5A_1_1__U_0 -> (none)
- C8116, C8146: Island IO_JACK:${SHEETNAME} -> (none); Role mix5:C_DEC_input_fault_switch_J_M5A_1_1__U_1 -> (none)
- C8117: Island IO_JACK:${SHEETNAME} -> (none); Role mix5:C_DEC_input_fault_switch_J_M5A_1_2__U_0 -> (none)
- C8118: Island IO_JACK:${SHEETNAME} -> (none); Role mix5:C_DEC_input_fault_switch_J_M5A_1_2__U_1 -> (none)
- C8119: Island IO_JACK:${SHEETNAME} -> (none); Role mix5:C_DEC_input_fault_switch_J_M5A_1_3__U_0 -> (none)
- C8120: Island IO_JACK:${SHEETNAME} -> (none); Role mix5:C_DEC_input_fault_switch_J_M5A_1_3__U_1 -> (none)
- C8121: Island IO_JACK:${SHEETNAME} -> (none); Role mix5:C_DEC_input_fault_switch_J_M5A_1_4__U_0 -> (none)
- C8122: Island IO_JACK:${SHEETNAME} -> (none); Role mix5:C_DEC_input_fault_switch_J_M5A_1_4__U_1 -> (none)
- C8123: Island IO_JACK:${SHEETNAME} -> (none); Role mix5:C_DEC_input_fault_switch_J_M5A_1_5__U_0 -> (none)
- C8124: Island IO_JACK:${SHEETNAME} -> (none); Role mix5:C_DEC_input_fault_switch_J_M5A_1_5__U_1 -> (none)
- C8125: Island IO_JACK:${SHEETNAME} -> (none); Role mix5:C_DEC_PACK_OPA4197IPWR_0_0 -> (none)
- C8126: Island IO_JACK:${SHEETNAME} -> (none); Role mix5:C_DEC_PACK_OPA4197IPWR_0_1 -> (none)
- C8127, C8141: Island IO_JACK:${SHEETNAME} -> (none); Role mix5:C_DEC_PACK_OPA4196IDR_0_0 -> (none)
- C8128, C8142: Island IO_JACK:${SHEETNAME} -> (none); Role mix5:C_DEC_PACK_OPA4196IDR_0_1 -> (none)
- C8139: Island IO_JACK:${SHEETNAME} -> (none); Role mix5:C_DEC_clip_detector_L_M5A_SUM_clip_SUM__UN_0 -> (none)
- C8140: Island IO_JACK:${SHEETNAME} -> (none); Role mix5:C_DEC_clip_detector_L_M5A_SUM_clip_SUM__UN_1 -> (none)
- C8143: Island IO_JACK:${SHEETNAME} -> (none); Role mix5:C_DEC_PACK_OPA4196IDR_1_0 -> (none)
- C8144: Island IO_JACK:${SHEETNAME} -> (none); Role mix5:C_DEC_PACK_OPA4196IDR_1_1 -> (none)
- C8145: Island IO_JACK:${SHEETNAME} -> (none); Role mix5:C_DEC_reference_generator_J_M5A_1_LOCAL__U_0 -> (none)
- D8108, D8109, D8110, D8111, D8112: Island IO_JACK:${SHEETNAME} -> (none); Role high_impedance_input:D -> (none)
- D8113, D8117, D8121, D8125, D8129, D8133: Island IO_JACK:${SHEETNAME} -> (none); Role magnitude_indicator:D1 -> (none)
- D8114, D8118, D8122, D8126, D8130, D8134: Island IO_JACK:${SHEETNAME} -> (none); Role magnitude_indicator:D2 -> (none)
- D8115, D8119, D8123, D8127, D8131, D8135: Island IO_JACK:${SHEETNAME} -> (none); Role magnitude_indicator:D3 -> (none)
- D8116, D8120, D8124, D8128, D8132, D8136: Island IO_JACK:${SHEETNAME} -> (none); Role magnitude_indicator:D4 -> (none)
- D901, D902, D903, D904, D905, D906: Island IO_JACK:${SHEETNAME} -> (none); Role magnitude_indicator:LED -> (none)
- D9061: Island IO_JACK:${SHEETNAME} -> (none); Role clip_detector:LED -> (none)
- J901: Island IO_JACK:${SHEETNAME} -> (none); Role mix5:J_1 -> (none)
- J902: Island IO_JACK:${SHEETNAME} -> (none); Role mix5:J_2 -> (none)
- J903: Island IO_JACK:${SHEETNAME} -> (none); Role mix5:J_3 -> (none)
- J904: Island IO_JACK:${SHEETNAME} -> (none); Role mix5:J_4 -> (none)
- J905: Island IO_JACK:${SHEETNAME} -> (none); Role mix5:J_5 -> (none)
- J906: Island IO_JACK:${SHEETNAME} -> (none); Role mix5:J_SUM -> (none)
- R8105, R8115, R8125, R8135, R8145: Island IO_JACK:${SHEETNAME} -> (none); Role input_fault_switch:R_EN -> (none)
- R8106, R8116, R8126, R8136, R8146: Island IO_JACK:${SHEETNAME} -> (none); Role input_fault_switch:R_DRIVE -> (none)
- R8107, R8117, R8127, R8137, R8147: Island IO_JACK:${SHEETNAME} -> (none); Role high_impedance_input:R_PD -> (none)
- R8108, R8118, R8128, R8138, R8148: Island IO_JACK:${SHEETNAME} -> (none); Role high_impedance_input:R_LIMIT -> (none)
- R8167: Island IO_JACK:${SHEETNAME} -> (none); Role general_output:R_ISO_A -> (none)
- R8168: Island IO_JACK:${SHEETNAME} -> (none); Role general_output:R_ISO_B -> (none)
- R8169, R8170, R8171, R8172, R8173, R8174: Island IO_JACK:${SHEETNAME} -> (none); Role magnitude_indicator:R_SENSE -> (none)
- R8175: Island IO_JACK:${SHEETNAME} -> (none); Role clip_detector:R_TOP -> (none)
- R8176: Island IO_JACK:${SHEETNAME} -> (none); Role clip_detector:R_BOT -> (none)
- R8177: Island IO_JACK:${SHEETNAME} -> (none); Role clip_detector:R_LED -> (none)
- U8102, U8103, U8104, U8105, U8106: Island IO_JACK:${SHEETNAME} -> (none); Role input_fault_switch:U -> (none)
- U8112: Island IO_JACK:${SHEETNAME} -> (none); LogicalCellKey high_impedance_input_J_M5A_1_2__A.1 -> (none); Role high_impedance_input:A -> (none)
- U8112: Island IO_JACK:${SHEETNAME} -> (none); LogicalCellKey high_impedance_input_J_M5A_1_4__A.1 -> (none); Role high_impedance_input:A -> (none)
- U8112: Island IO_JACK:${SHEETNAME} -> (none); LogicalCellKey high_impedance_input_J_M5A_1_3__A.1 -> (none); Role high_impedance_input:A -> (none)
- U8112: Island IO_JACK:${SHEETNAME} -> (none); LogicalCellKey high_impedance_input_J_M5A_1_1__A.1 -> (none); Role high_impedance_input:A -> (none)
- U8112, U8115, U8116, U8117: Island IO_JACK:${SHEETNAME} -> (none); Role mix5:package supply -> (none)
- U8113: Island IO_JACK:${SHEETNAME} -> (none); Role clip_detector:UP -> (none)
- U8114: Island IO_JACK:${SHEETNAME} -> (none); Role clip_detector:UN -> (none)
- U8115: Island IO_JACK:${SHEETNAME} -> (none); LogicalCellKey magnitude_indicator_L_M5A_2_mag_2__A.1 -> (none); Role magnitude_indicator:A -> (none)
- U8115: Island IO_JACK:${SHEETNAME} -> (none); LogicalCellKey magnitude_indicator_L_M5A_1_mag_1__A.1 -> (none); Role magnitude_indicator:A -> (none)
- U8115: Island IO_JACK:${SHEETNAME} -> (none); LogicalCellKey general_output_J_M5A_1_SUM__A.1 -> (none); Role general_output:A -> (none)
- U8115: Island IO_JACK:${SHEETNAME} -> (none); LogicalCellKey high_impedance_input_J_M5A_1_5__A.1 -> (none); Role high_impedance_input:A -> (none)
- U8116: Island IO_JACK:${SHEETNAME} -> (none); LogicalCellKey magnitude_indicator_L_M5A_SUM_mag_SUM__A.1 -> (none); Role magnitude_indicator:A -> (none)
- U8116: Island IO_JACK:${SHEETNAME} -> (none); LogicalCellKey magnitude_indicator_L_M5A_5_mag_5__A.1 -> (none); Role magnitude_indicator:A -> (none)
- U8116: Island IO_JACK:${SHEETNAME} -> (none); LogicalCellKey magnitude_indicator_L_M5A_3_mag_3__A.1 -> (none); Role magnitude_indicator:A -> (none)
- U8116: Island IO_JACK:${SHEETNAME} -> (none); LogicalCellKey magnitude_indicator_L_M5A_4_mag_4__A.1 -> (none); Role magnitude_indicator:A -> (none)
- U8117: Island IO_JACK:${SHEETNAME} -> (none); Role mix5:unused grounded follower -> (none)
- U8117: Island IO_JACK:${SHEETNAME} -> (none); LogicalCellKey clip_detector_L_M5A_SUM_clip_SUM__A.1 -> (none); Role clip_detector:A -> (none)
