File: boards/osc-jack/sheets/mult_B2_J.kicad_sch (KiCad schematic)
At the start: 36 parts, among them J309 WQP518MA, J310 WQP518MA, J409 WQP518MA, J410 WQP518MA, U3201 ADG5412FBRUZ, U3202 OPA4197IPWR, U3203 OPA4196IDR

Commit message: Reserve clear jack-board geometry and align projected schematic fields
Parts:
- C3201, C3202, C3203: Island IO_JACK:${SHEETNAME} -> (none); Role precision_output:C_FAST -> (none)
- C3204: Island IO_JACK:${SHEETNAME} -> (none); Role mult:C_DEC_input_fault_switch_J_B1_IN_IN__U_0 -> (none)
- C3205: Island IO_JACK:${SHEETNAME} -> (none); Role mult:C_DEC_input_fault_switch_J_B1_IN_IN__U_1 -> (none)
- C3206: Island IO_JACK:${SHEETNAME} -> (none); Role mult:C_DEC_PACK_OPA4197IPWR_0_0 -> (none)
- C3207: Island IO_JACK:${SHEETNAME} -> (none); Role mult:C_DEC_PACK_OPA4197IPWR_0_1 -> (none)
- C3208: Island IO_JACK:${SHEETNAME} -> (none); Role mult:C_DEC_PACK_OPA4196IDR_0_0 -> (none)
- C3209: Island IO_JACK:${SHEETNAME} -> (none); Role mult:C_DEC_PACK_OPA4196IDR_0_1 -> (none)
- D309: Island IO_JACK:${SHEETNAME} -> (none); Role magnitude_indicator:LED -> (none)
- D3201: Island IO_JACK:${SHEETNAME} -> (none); Role high_impedance_input:D -> (none)
- D3202: Island IO_JACK:${SHEETNAME} -> (none); Role magnitude_indicator:D1 -> (none)
- D3203: Island IO_JACK:${SHEETNAME} -> (none); Role magnitude_indicator:D2 -> (none)
- D3204: Island IO_JACK:${SHEETNAME} -> (none); Role magnitude_indicator:D3 -> (none)
- D3205: Island IO_JACK:${SHEETNAME} -> (none); Role magnitude_indicator:D4 -> (none)
- J309: Island IO_JACK:${SHEETNAME} -> (none); Role mult:J_IN -> (none)
- J310: Island IO_JACK:${SHEETNAME} -> (none); Role mult:J_OUT_2 -> (none)
- J409: Island IO_JACK:${SHEETNAME} -> (none); Role mult:J_OUT_1 -> (none)
- J410: Island IO_JACK:${SHEETNAME} -> (none); Role mult:J_OUT_3 -> (none)
- R3201: Island IO_JACK:${SHEETNAME} -> (none); Role input_fault_switch:R_EN -> (none)
- R3202: Island IO_JACK:${SHEETNAME} -> (none); Role input_fault_switch:R_DRIVE -> (none)
- R3203: Island IO_JACK:${SHEETNAME} -> (none); Role high_impedance_input:R_PD -> (none)
- R3204: Island IO_JACK:${SHEETNAME} -> (none); Role high_impedance_input:R_LIMIT -> (none)
- R3205, R3208, R3211: Island IO_JACK:${SHEETNAME} -> (none); Role precision_output:R_ISO_A -> (none)
- R3206, R3209, R3212: Island IO_JACK:${SHEETNAME} -> (none); Role precision_output:R_ISO_B -> (none)
- R3207, R3210, R3213: Island IO_JACK:${SHEETNAME} -> (none); Role precision_output:R_FB -> (none)
- R3214: Island IO_JACK:${SHEETNAME} -> (none); Role magnitude_indicator:R_SENSE -> (none)
- U3201: Island IO_JACK:${SHEETNAME} -> (none); Role input_fault_switch:U -> (none)
- U3202: Island IO_JACK:${SHEETNAME} -> (none); LogicalCellKey precision_output_J_B1_IN_OUT_2__A.1 -> (none); Role precision_output:A -> (none)
- U3202: Island IO_JACK:${SHEETNAME} -> (none); LogicalCellKey precision_output_J_B1_IN_OUT_1__A.1 -> (none); Role precision_output:A -> (none)
- U3202, U3203: Island IO_JACK:${SHEETNAME} -> (none); Role mult:package supply -> (none)
- U3202: Island IO_JACK:${SHEETNAME} -> (none); LogicalCellKey precision_output_J_B1_IN_OUT_3__A.1 -> (none); Role precision_output:A -> (none)
- U3202: Island IO_JACK:${SHEETNAME} -> (none); LogicalCellKey high_impedance_input_J_B1_IN_IN__A.1 -> (none); Role high_impedance_input:A -> (none)
- U3203: Island IO_JACK:${SHEETNAME} -> (none); Role mult:unused grounded follower -> (none)
- U3203: Island IO_JACK:${SHEETNAME} -> (none); LogicalCellKey magnitude_indicator_L_B1_IN_mag_IN__A.1 -> (none); Role magnitude_indicator:A -> (none)
