File: boards/osc-jack/sheets/offset_A04_J.kicad_sch (KiCad schematic)
At the start: 59 parts, among them J1608 WQP518MA, J1609 WQP518MA, J1610 WQP518MA, U7402 ADG5412FBRUZ, U7403 ADG5412FBRUZ, U7406 OPA4197IPWR, U7407 LM393BIDR, U7408 LM393BIDR, U7409 OPA4196IDR

Commit message: Reserve clear jack-board geometry and align projected schematic fields
Parts:
- C7406: Island IO_JACK:${SHEETNAME} -> (none); Role precision_output:C_FAST -> (none)
- C7408: Island IO_JACK:${SHEETNAME} -> (none); Role offset:C_DEC_input_fault_switch_J_A01_IN_IN__U_0 -> (none)
- C7409: Island IO_JACK:${SHEETNAME} -> (none); Role offset:C_DEC_input_fault_switch_J_A01_IN_IN__U_1 -> (none)
- C7410: Island IO_JACK:${SHEETNAME} -> (none); Role offset:C_DEC_input_fault_switch_J_A01_IN_OFFSET__U_0 -> (none)
- C7411: Island IO_JACK:${SHEETNAME} -> (none); Role offset:C_DEC_input_fault_switch_J_A01_IN_OFFSET__U_1 -> (none)
- C7412: Island IO_JACK:${SHEETNAME} -> (none); Role offset:C_DEC_PACK_OPA4197IPWR_0_0 -> (none)
- C7413: Island IO_JACK:${SHEETNAME} -> (none); Role offset:C_DEC_PACK_OPA4197IPWR_0_1 -> (none)
- C7414: Island IO_JACK:${SHEETNAME} -> (none); Role offset:C_DEC_PACK_OPA4197IPWR_1_0 -> (none)
- C7415: Island IO_JACK:${SHEETNAME} -> (none); Role offset:C_DEC_PACK_OPA4197IPWR_1_1 -> (none)
- C7420: Island IO_JACK:${SHEETNAME} -> (none); Role offset:C_DEC_clip_detector_L_A01_OUT_clip_OUT__UN_0 -> (none)
- C7421: Island IO_JACK:${SHEETNAME} -> (none); Role offset:C_DEC_clip_detector_L_A01_OUT_clip_OUT__UN_1 -> (none)
- C7422: Island IO_JACK:${SHEETNAME} -> (none); Role offset:C_DEC_PACK_OPA4196IDR_0_0 -> (none)
- C7423: Island IO_JACK:${SHEETNAME} -> (none); Role offset:C_DEC_PACK_OPA4196IDR_0_1 -> (none)
- D1608, D1609, D1610: Island IO_JACK:${SHEETNAME} -> (none); Role magnitude_indicator:LED -> (none)
- D16101: Island IO_JACK:${SHEETNAME} -> (none); Role clip_detector:LED -> (none)
- D7401, D7402: Island IO_JACK:${SHEETNAME} -> (none); Role high_impedance_input:D -> (none)
- D7403, D7408, D7413: Island IO_JACK:${SHEETNAME} -> (none); Role magnitude_indicator:D1 -> (none)
- D7404, D7409, D7414: Island IO_JACK:${SHEETNAME} -> (none); Role magnitude_indicator:D2 -> (none)
- D7405, D7410, D7415: Island IO_JACK:${SHEETNAME} -> (none); Role magnitude_indicator:D3 -> (none)
- D7406, D7411, D7416: Island IO_JACK:${SHEETNAME} -> (none); Role magnitude_indicator:D4 -> (none)
- J1608: Island IO_JACK:${SHEETNAME} -> (none); Role offset:J_IN -> (none)
- J1609: Island IO_JACK:${SHEETNAME} -> (none); Role offset:J_OFFSET -> (none)
- J1610: Island IO_JACK:${SHEETNAME} -> (none); Role offset:J_OUT -> (none)
- R7405, R7409: Island IO_JACK:${SHEETNAME} -> (none); Role input_fault_switch:R_EN -> (none)
- R7406, R7410: Island IO_JACK:${SHEETNAME} -> (none); Role input_fault_switch:R_DRIVE -> (none)
- R7407, R7411: Island IO_JACK:${SHEETNAME} -> (none); Role high_impedance_input:R_PD -> (none)
- R7408, R7412: Island IO_JACK:${SHEETNAME} -> (none); Role high_impedance_input:R_LIMIT -> (none)
- R7425: Island IO_JACK:${SHEETNAME} -> (none); Role offset:R_RESTORE_IN -> (none)
- R7426: Island IO_JACK:${SHEETNAME} -> (none); Role offset:R_RESTORE_FB -> (none)
- R7427: Island IO_JACK:${SHEETNAME} -> (none); Role precision_output:R_ISO_A -> (none)
- R7428: Island IO_JACK:${SHEETNAME} -> (none); Role precision_output:R_ISO_B -> (none)
- R7429: Island IO_JACK:${SHEETNAME} -> (none); Role precision_output:R_FB -> (none)
- R7430, R7431, R7432: Island IO_JACK:${SHEETNAME} -> (none); Role magnitude_indicator:R_SENSE -> (none)
- R7433: Island IO_JACK:${SHEETNAME} -> (none); Role clip_detector:R_TOP -> (none)
- R7434: Island IO_JACK:${SHEETNAME} -> (none); Role clip_detector:R_BOT -> (none)
- R7435: Island IO_JACK:${SHEETNAME} -> (none); Role clip_detector:R_LED -> (none)
- U7402, U7403: Island IO_JACK:${SHEETNAME} -> (none); Role input_fault_switch:U -> (none)
- U7406: Island IO_JACK:${SHEETNAME} -> (none); LogicalCellKey precision_output_J_A01_IN_OUT__A.1 -> (none); Role precision_output:A -> (none)
- U7406, U7409: Island IO_JACK:${SHEETNAME} -> (none); Role offset:package supply -> (none)
- U7406: Island IO_JACK:${SHEETNAME} -> (none); LogicalCellKey high_impedance_input_J_A01_IN_OFFSET__A.1 -> (none); Role high_impedance_input:A -> (none)
- U7406: Island IO_JACK:${SHEETNAME} -> (none); LogicalCellKey RESTORE.1 -> (none); Role offset:RESTORE -> (none)
- U7406: Island IO_JACK:${SHEETNAME} -> (none); LogicalCellKey high_impedance_input_J_A01_IN_IN__A.1 -> (none); Role high_impedance_input:A -> (none)
- U7407: Island IO_JACK:${SHEETNAME} -> (none); Role clip_detector:UP -> (none)
- U7408: Island IO_JACK:${SHEETNAME} -> (none); Role clip_detector:UN -> (none)
- U7409: Island IO_JACK:${SHEETNAME} -> (none); LogicalCellKey clip_detector_L_A01_OUT_clip_OUT__A.1 -> (none); Role clip_detector:A -> (none)
- U7409: Island IO_JACK:${SHEETNAME} -> (none); LogicalCellKey magnitude_indicator_L_A01_IN_mag_IN__A.1 -> (none); Role magnitude_indicator:A -> (none)
- U7409: Island IO_JACK:${SHEETNAME} -> (none); LogicalCellKey magnitude_indicator_L_A01_OFFSET_mag_OFFSET__A.1 -> (none); Role magnitude_indicator:A -> (none)
- U7409: Island IO_JACK:${SHEETNAME} -> (none); LogicalCellKey magnitude_indicator_L_A01_OUT_mag_OUT__A.1 -> (none); Role magnitude_indicator:A -> (none)
