File: boards/osc-jack/sheets/offset_A06_J.kicad_sch (KiCad schematic)
At the start: 59 parts, among them J1808 WQP518MA, J1809 WQP518MA, J1810 WQP518MA, U7602 ADG5412FBRUZ, U7603 ADG5412FBRUZ, U7606 OPA4197IPWR, U7607 LM393BIDR, U7608 LM393BIDR, U7609 OPA4196IDR

Commit message: Reserve clear jack-board geometry and align projected schematic fields
Parts:
- C7606: Island IO_JACK:${SHEETNAME} -> (none); Role precision_output:C_FAST -> (none)
- C7608: Island IO_JACK:${SHEETNAME} -> (none); Role offset:C_DEC_input_fault_switch_J_A01_IN_IN__U_0 -> (none)
- C7609: Island IO_JACK:${SHEETNAME} -> (none); Role offset:C_DEC_input_fault_switch_J_A01_IN_IN__U_1 -> (none)
- C7610: Island IO_JACK:${SHEETNAME} -> (none); Role offset:C_DEC_input_fault_switch_J_A01_IN_OFFSET__U_0 -> (none)
- C7611: Island IO_JACK:${SHEETNAME} -> (none); Role offset:C_DEC_input_fault_switch_J_A01_IN_OFFSET__U_1 -> (none)
- C7612: Island IO_JACK:${SHEETNAME} -> (none); Role offset:C_DEC_PACK_OPA4197IPWR_0_0 -> (none)
- C7613: Island IO_JACK:${SHEETNAME} -> (none); Role offset:C_DEC_PACK_OPA4197IPWR_0_1 -> (none)
- C7614: Island IO_JACK:${SHEETNAME} -> (none); Role offset:C_DEC_PACK_OPA4197IPWR_1_0 -> (none)
- C7615: Island IO_JACK:${SHEETNAME} -> (none); Role offset:C_DEC_PACK_OPA4197IPWR_1_1 -> (none)
- C7620: Island IO_JACK:${SHEETNAME} -> (none); Role offset:C_DEC_clip_detector_L_A01_OUT_clip_OUT__UN_0 -> (none)
- C7621: Island IO_JACK:${SHEETNAME} -> (none); Role offset:C_DEC_clip_detector_L_A01_OUT_clip_OUT__UN_1 -> (none)
- C7622: Island IO_JACK:${SHEETNAME} -> (none); Role offset:C_DEC_PACK_OPA4196IDR_0_0 -> (none)
- C7623: Island IO_JACK:${SHEETNAME} -> (none); Role offset:C_DEC_PACK_OPA4196IDR_0_1 -> (none)
- D1808, D1809, D1810: Island IO_JACK:${SHEETNAME} -> (none); Role magnitude_indicator:LED -> (none)
- D18101: Island IO_JACK:${SHEETNAME} -> (none); Role clip_detector:LED -> (none)
- D7601, D7602: Island IO_JACK:${SHEETNAME} -> (none); Role high_impedance_input:D -> (none)
- D7603, D7608, D7613: Island IO_JACK:${SHEETNAME} -> (none); Role magnitude_indicator:D1 -> (none)
- D7604, D7609, D7614: Island IO_JACK:${SHEETNAME} -> (none); Role magnitude_indicator:D2 -> (none)
- D7605, D7610, D7615: Island IO_JACK:${SHEETNAME} -> (none); Role magnitude_indicator:D3 -> (none)
- D7606, D7611, D7616: Island IO_JACK:${SHEETNAME} -> (none); Role magnitude_indicator:D4 -> (none)
- J1808: Island IO_JACK:${SHEETNAME} -> (none); Role offset:J_IN -> (none)
- J1809: Island IO_JACK:${SHEETNAME} -> (none); Role offset:J_OFFSET -> (none)
- J1810: Island IO_JACK:${SHEETNAME} -> (none); Role offset:J_OUT -> (none)
- R7605, R7609: Island IO_JACK:${SHEETNAME} -> (none); Role input_fault_switch:R_EN -> (none)
- R7606, R7610: Island IO_JACK:${SHEETNAME} -> (none); Role input_fault_switch:R_DRIVE -> (none)
- R7607, R7611: Island IO_JACK:${SHEETNAME} -> (none); Role high_impedance_input:R_PD -> (none)
- R7608, R7612: Island IO_JACK:${SHEETNAME} -> (none); Role high_impedance_input:R_LIMIT -> (none)
- R7625: Island IO_JACK:${SHEETNAME} -> (none); Role offset:R_RESTORE_IN -> (none)
- R7626: Island IO_JACK:${SHEETNAME} -> (none); Role offset:R_RESTORE_FB -> (none)
- R7627: Island IO_JACK:${SHEETNAME} -> (none); Role precision_output:R_ISO_A -> (none)
- R7628: Island IO_JACK:${SHEETNAME} -> (none); Role precision_output:R_ISO_B -> (none)
- R7629: Island IO_JACK:${SHEETNAME} -> (none); Role precision_output:R_FB -> (none)
- R7630, R7631, R7632: Island IO_JACK:${SHEETNAME} -> (none); Role magnitude_indicator:R_SENSE -> (none)
- R7633: Island IO_JACK:${SHEETNAME} -> (none); Role clip_detector:R_TOP -> (none)
- R7634: Island IO_JACK:${SHEETNAME} -> (none); Role clip_detector:R_BOT -> (none)
- R7635: Island IO_JACK:${SHEETNAME} -> (none); Role clip_detector:R_LED -> (none)
- U7602, U7603: Island IO_JACK:${SHEETNAME} -> (none); Role input_fault_switch:U -> (none)
- U7606: Island IO_JACK:${SHEETNAME} -> (none); LogicalCellKey precision_output_J_A01_IN_OUT__A.1 -> (none); Role precision_output:A -> (none)
- U7606: Island IO_JACK:${SHEETNAME} -> (none); LogicalCellKey RESTORE.1 -> (none); Role offset:RESTORE -> (none)
- U7606: Island IO_JACK:${SHEETNAME} -> (none); LogicalCellKey high_impedance_input_J_A01_IN_OFFSET__A.1 -> (none); Role high_impedance_input:A -> (none)
- U7606, U7609: Island IO_JACK:${SHEETNAME} -> (none); Role offset:package supply -> (none)
- U7606: Island IO_JACK:${SHEETNAME} -> (none); LogicalCellKey high_impedance_input_J_A01_IN_IN__A.1 -> (none); Role high_impedance_input:A -> (none)
- U7607: Island IO_JACK:${SHEETNAME} -> (none); Role clip_detector:UP -> (none)
- U7608: Island IO_JACK:${SHEETNAME} -> (none); Role clip_detector:UN -> (none)
- U7609: Island IO_JACK:${SHEETNAME} -> (none); LogicalCellKey magnitude_indicator_L_A01_OFFSET_mag_OFFSET__A.1 -> (none); Role magnitude_indicator:A -> (none)
- U7609: Island IO_JACK:${SHEETNAME} -> (none); LogicalCellKey magnitude_indicator_L_A01_IN_mag_IN__A.1 -> (none); Role magnitude_indicator:A -> (none)
- U7609: Island IO_JACK:${SHEETNAME} -> (none); LogicalCellKey clip_detector_L_A01_OUT_clip_OUT__A.1 -> (none); Role clip_detector:A -> (none)
- U7609: Island IO_JACK:${SHEETNAME} -> (none); LogicalCellKey magnitude_indicator_L_A01_OUT_mag_OUT__A.1 -> (none); Role magnitude_indicator:A -> (none)
