File: boards/osc-jack/sheets/oscillator_O1_J.kicad_sch (KiCad schematic)
At the start: 57 parts, among them J101 WQP518MA, J102 WQP518MA, J103 WQP518MA, J104 WQP518MA, J105 WQP518MA, J106 WQP518MA, J107 WQP518MA, J108 WQP518MA, U1101 ADG5412FBRUZ, U1102 ADG5412FBRUZ, U1103 ADG5412FBRUZ, U1104 ADG5412FBRUZ, U1116 OPA4196IDR, U1117 OPA4196IDR, U1118 OPA4197IPWR

Commit message: Reserve clear jack-board geometry and align projected schematic fields
Parts:
- C1121, C1152: Island IO_JACK:${SHEETNAME} -> (none); Role oscillator:C_DEC_input_fault_switch_J_O1_1V_1V__U_0 -> (none)
- C1122, C1153: Island IO_JACK:${SHEETNAME} -> (none); Role oscillator:C_DEC_input_fault_switch_J_O1_1V_1V__U_1 -> (none)
- C1123: Island IO_JACK:${SHEETNAME} -> (none); Role oscillator:C_DEC_input_fault_switch_J_O1_1V_FM__U_0 -> (none)
- C1124: Island IO_JACK:${SHEETNAME} -> (none); Role oscillator:C_DEC_input_fault_switch_J_O1_1V_FM__U_1 -> (none)
- C1125: Island IO_JACK:${SHEETNAME} -> (none); Role oscillator:C_DEC_input_fault_switch_J_O1_1V_PWM__U_0 -> (none)
- C1126: Island IO_JACK:${SHEETNAME} -> (none); Role oscillator:C_DEC_input_fault_switch_J_O1_1V_PWM__U_1 -> (none)
- C1127: Island IO_JACK:${SHEETNAME} -> (none); Role oscillator:C_DEC_input_fault_switch_J_O1_1V_SYNC__U_0 -> (none)
- C1128: Island IO_JACK:${SHEETNAME} -> (none); Role oscillator:C_DEC_input_fault_switch_J_O1_1V_SYNC__U_1 -> (none)
- C1140: Island IO_JACK:${SHEETNAME} -> (none); Role oscillator:C_DEC_PACK_OPA4196IDR_0_0 -> (none)
- C1141: Island IO_JACK:${SHEETNAME} -> (none); Role oscillator:C_DEC_PACK_OPA4196IDR_0_1 -> (none)
- C1150: Island IO_JACK:${SHEETNAME} -> (none); Role oscillator:C_DEC_PACK_OPA4196IDR_5_0 -> (none)
- C1151: Island IO_JACK:${SHEETNAME} -> (none); Role oscillator:C_DEC_PACK_OPA4196IDR_5_1 -> (none)
- DO1101, DO1102, DO1103, DO1104: Island IO_JACK:${SHEETNAME} -> (none); Role high_impedance_input:D -> (none)
- J101: Island IO_JACK:${SHEETNAME} -> (none); Role oscillator:J_1V -> (none)
- J102: Island IO_JACK:${SHEETNAME} -> (none); Role oscillator:J_FM -> (none)
- J103: Island IO_JACK:${SHEETNAME} -> (none); Role oscillator:J_PWM -> (none)
- J104: Island IO_JACK:${SHEETNAME} -> (none); Role oscillator:J_SYNC -> (none)
- J105: Island IO_JACK:${SHEETNAME} -> (none); Role oscillator:J_SIN -> (none)
- J106: Island IO_JACK:${SHEETNAME} -> (none); Role oscillator:J_TRI -> (none)
- J107: Island IO_JACK:${SHEETNAME} -> (none); Role oscillator:J_SAW -> (none)
- J108: Island IO_JACK:${SHEETNAME} -> (none); Role oscillator:J_PUL -> (none)
- R1101, R1105, R1109, R1113: Island IO_JACK:${SHEETNAME} -> (none); Role input_fault_switch:R_EN -> (none)
- R1102, R1106, R1110, R1114: Island IO_JACK:${SHEETNAME} -> (none); Role input_fault_switch:R_DRIVE -> (none)
- R1103, R1107, R1111, R1115: Island IO_JACK:${SHEETNAME} -> (none); Role high_impedance_input:R_PD -> (none)
- R1104, R1108, R1112, R1116: Island IO_JACK:${SHEETNAME} -> (none); Role high_impedance_input:R_LIMIT -> (none)
- RB1102, RB1104, RB1106, RB1108: Island IO_JACK:${SHEETNAME} -> (none); Role general_output:R_ISO_A -> (none)
- RB1103, RB1105, RB1107, RB1109: Island IO_JACK:${SHEETNAME} -> (none); Role general_output:R_ISO_B -> (none)
- U1101, U1102, U1103, U1104: Island IO_JACK:${SHEETNAME} -> (none); Role input_fault_switch:U -> (none)
- U1116: Island IO_JACK:${SHEETNAME} -> (none); LogicalCellKey high_impedance_input_J_O1_1V_FM__A.1 -> (none); Role high_impedance_input:A -> (none)
- U1116: Island IO_JACK:${SHEETNAME} -> (none); LogicalCellKey general_output_J_O1_1V_SIN__A.1 -> (none); Role general_output:A -> (none)
- U1116: Island IO_JACK:${SHEETNAME} -> (none); LogicalCellKey high_impedance_input_J_O1_1V_PWM__A.1 -> (none); Role high_impedance_input:A -> (none)
- U1116, U1117, U1118: Island IO_JACK:${SHEETNAME} -> (none); Role oscillator:package supply -> (none)
- U1116: Island IO_JACK:${SHEETNAME} -> (none); LogicalCellKey high_impedance_input_J_O1_1V_SYNC__A.1 -> (none); Role high_impedance_input:A -> (none)
- U1117: Island IO_JACK:${SHEETNAME} -> (none); LogicalCellKey general_output_J_O1_1V_PUL__A.1 -> (none); Role general_output:A -> (none)
- U1117: Island IO_JACK:${SHEETNAME} -> (none); LogicalCellKey general_output_J_O1_1V_SAW__A.1 -> (none); Role general_output:A -> (none)
- U1117: Island IO_JACK:${SHEETNAME} -> (none); LogicalCellKey general_output_J_O1_1V_TRI__A.1 -> (none); Role general_output:A -> (none)
- U1117, U1118: Island IO_JACK:${SHEETNAME} -> (none); Role oscillator:unused grounded follower -> (none)
- U1118: Island IO_JACK:${SHEETNAME} -> (none); LogicalCellKey high_impedance_input_J_O1_1V_1V__A.1 -> (none); Role high_impedance_input:A -> (none)
