File: boards/osc-core/sheets/board_interfaces_K.kicad_sch (KiCad schematic)
At the start: 24 parts, among them J900002 BM08B-GHS-TBT(LF)(SN), J900004 BM08B-GHS-TBT(LF)(SN), J900006 BM08B-GHS-TBT(LF)(SN), J900008 BM08B-GHS-TBT(LF)(SN), J900010 BM08B-GHS-TBT(LF)(SN), J900012 BM08B-GHS-TBT(LF)(SN), J900014 BM08B-GHS-TBT(LF)(SN), J900016 BM08B-GHS-TBT(LF)(SN), J900018 BM08B-GHS-TBT(LF)(SN), J900020 BM08B-GHS-TBT(LF)(SN), J900022 BM08B-GHS-TBT(LF)(SN), J900024 BM08B-GHS-TBT(LF)(SN), J900026 BM08B-GHS-TBT(LF)(SN), J900028 BM08B-GHS-TBT(LF)(SN), J900030 BM08B-GHS-TBT(LF)(SN), J900032 BM08B-GHS-TBT(LF)(SN), J900034 BM08B-GHS-TBT(LF)(SN), J900036 BM08B-GHS-TBT(LF)(SN), J900038 BM08B-GHS-TBT(LF)(SN), J900040 BM08B-GHS-TBT(LF)(SN), J900042 BM08B-GHS-TBT(LF)(SN), J900044 BM08B-GHS-TBT(LF)(SN), J900046 BM08B-GHS-TBT(LF)(SN), J900048 BM08B-GHS-TBT(LF)(SN)

Commit message: Split jack partition into two boards with local bypass clusters
Parts:
- J900020: FootprintOriginMm 176.0,39.95 -> 23.0,81.95
- J900022: FootprintOriginMm 193.0,39.95 -> 40.0,81.95
- J900024: FootprintOriginMm 210.0,39.95 -> 57.0,81.95
- J900026: FootprintOriginMm 227.0,39.95 -> 74.0,81.95
- J900028: FootprintOriginMm 244.0,39.95 -> 91.0,81.95
- J900030: FootprintOriginMm 261.0,39.95 -> 108.0,81.95
- J900032: FootprintOriginMm 278.0,39.95 -> 125.0,81.95
- J900034: FootprintOriginMm 295.0,39.95 -> 142.0,81.95
- J900036: FootprintOriginMm 23.0,81.95 -> 159.0,81.95
- J900038: FootprintOriginMm 40.0,81.95 -> 23.0,123.95
- J900040: FootprintOriginMm 57.0,81.95 -> 40.0,123.95
- J900042: FootprintOriginMm 74.0,81.95 -> 57.0,123.95
- J900044: FootprintOriginMm 91.0,81.95 -> 74.0,123.95
- J900046: FootprintOriginMm 108.0,81.95 -> 91.0,123.95
- J900048: FootprintOriginMm 125.0,81.95 -> 108.0,123.95
Connections:
- net X05736A904C0279F1CE63 is gone; now on net X0ACA9FAE16CB353A0CB1: J900008.3
- net X1C4D2385F806310840A0 is gone; now on net X81CA071E9915CC31EAEA: J900002.1
- net X1E1299B7B09613B0B0D3 is gone; now on net X7985B0752A3E34339F44: J900006.5
- net X34E6E1A14D764B3D5363 is gone; now on net XA3808316751BA419D842: J900004.3
- net X47A1F716E3FE17CD7494 is gone; now on net X94210EAC11BB98036631: J900006.1
- net X4B8C26BB8E9C320C2F28 is gone; now on net XE81DCCD63340C32994FE: J900004.1
- net X5742FC5A6BE2F0A1E4D2 is gone; now on net X7C5F17AED66F7138F3A8: J900004.5
- net X5BDE0CC9A020C6F2E113 is gone; now on net X97E728989B7553A387AE: J900002.5
- net X6C227D1A4FFD615CE3B4 is gone; now on net X5A748C9F10BC16D9ED6F: J900010.3
- net X73B2519EBEC246C65607 is gone; now on net XB9D2A914247B25F8994C: J900006.7
- net X8C35A836AF988046FF6E is gone; now on net XA182BFDAEE78E0F2784C: J900012.3
- net X90CB51F278945C8C5062 is gone; now on net XFA9179FF4E8D01632C80: J900010.7
- net X965884E569C2BD8409A5 is gone; now on net XBF3BE4FDE28392550991: J900012.5
- net XA504C9B1F853C30BEAC2 is gone; now on net XFBD81EB4423EDA37C16F: J900006.3
- net XB84D06156CC830BD8E3A is gone; now on net X9D4DAF35CDBF61FFC354: J900002.3
- net XB94B6FA28DE6E550608C is gone; now on net X878F2A279999CCD4A075: J900012.1
- net XBA90FAD9780242414663 is gone; now on net X64750EAD045B08CFF878: J900008.5
- net XC6A7664726BAFEE0BCFA is gone; now on net X235805FBDE65FEABD919: J900012.7
- net XCD7957368B0652402848 is gone; now on net X2E63525FBBE899E17DBA: J900008.7
- net XD2D99513A5A51F131C78 is gone; now on net X632AF8DD6216ED26A96D: J900002.7
- net XD724017984C2562351FC is gone; now on net X7183CCEDEAABA18363B5: J900004.7
- net XE2B9B937D5CAF54AD63F is gone; now on net X419C4916FF5B54E2AC89: J900008.1
- net XED9D669DEDB8C275FBBC is gone; now on net X2F7F192BBAEF5BD8A311: J900010.5
- net XF19CF8B5CE37D561D88A is gone; now on net X8BDF2BAD2449627A6AD6: J900010.1
- net X0ACA9FAE16CB353A0CB1: no longer J900044.3
- net X235805FBDE65FEABD919: no longer J900048.7
- net X2E63525FBBE899E17DBA: no longer J900044.7
- net X2F7F192BBAEF5BD8A311: no longer J900046.5
- net X419C4916FF5B54E2AC89: no longer J900044.1
- net X5A748C9F10BC16D9ED6F: no longer J900046.3
- net X632AF8DD6216ED26A96D: no longer J900038.7
- net X64750EAD045B08CFF878: no longer J900044.5
- net X7183CCEDEAABA18363B5: no longer J900040.7
- net X7985B0752A3E34339F44: no longer J900042.5
- net X7C5F17AED66F7138F3A8: no longer J900040.5
- net X81CA071E9915CC31EAEA: no longer J900038.1
- net X878F2A279999CCD4A075: no longer J900048.1
- net X8BDF2BAD2449627A6AD6: no longer J900046.1
- net X94210EAC11BB98036631: no longer J900042.1
- net X97E728989B7553A387AE: no longer J900038.5
- net X9D4DAF35CDBF61FFC354: no longer J900038.3
- net XA182BFDAEE78E0F2784C: no longer J900048.3
- net XA3808316751BA419D842: no longer J900040.3
- net XB9D2A914247B25F8994C: no longer J900042.7
- net XBF3BE4FDE28392550991: no longer J900048.5
- net XE81DCCD63340C32994FE: no longer J900040.1
- net XFA9179FF4E8D01632C80: no longer J900046.7
- net XFBD81EB4423EDA37C16F: no longer J900042.3
- net X058BE71DAF00A5A01CA2 renamed X0615A446E46FA664032B
- net X069AA41BCE4A36C26FB2 renamed X2FE4AF262FF60AFC8887
- net X10852B4E217E1D395843 renamed XEC4C271577BFE8DBACB5
- net X12779E488E24F1864CD0 renamed X9DEA3D05C0252C14732B
- net X15A31970A06D461453EF renamed X947D4B49DF13D9BCAFA3
- net X21865D5691F958DB8F2D renamed X90A3CD82F6E195F644DD
- net X265FED80190F5E11B071 renamed X0F97D3A17222BB79FD54
- net X2D597327EED2D1A7509E renamed X7DC561B7FAF374EE5AB0
- net X346DD33A417B8C52D3FF renamed X47C2211BADF82245E208
- net X3F3C53CC94BD95AE5C54 renamed X722B62B5E67741B855CA
- net X43FA9082F43CAA3CD5CC renamed X8513A9265CE9B8AA4E49
- net X45AEDA7EA8DE3AE9B3ED renamed XC8DFE86BD3A7EAD286C6
- net X45C9091F706AFD0A887F renamed X931E79E5D5D06724201E
- net X498DE6D8563260D00A21 renamed X557F548F7D9FAD9BFC62
- net X59FBA17EF0ED74FF9324 renamed X1D5083C1689CCBDCC7AF
- net X6012073DA8F01B869B3F renamed XFC9D33C023228B9841B7
- net X6989F0D5C243DDFAAD15 renamed X272ADBD100FF77E2EEEE
- net X71B9E05195347FA9C8C2 renamed XBA3E9C437B4E486D623D
- net X7233565AE71A94755195 renamed XE696508C2D9B11400F0C
- net X78BDC6ABACC4E8D7872D renamed X3245E446D0AC7D6BACBF
- net X7A60CDBDD22898ADD05B renamed X283762E52614D8D51C1A
- net X862B85B7365A480D1EC4 renamed X3710249F479E7DA6DFCE
- net X88D1A44E36A22B77BEFF renamed XB8780C34DCDC50D9A9BA
- net X8A939B676B6F87E5F9A3 renamed XB9D8E425159DDB4164F8
- net X95E38523BB35DF833AE9 renamed X1350D6DDB5A475CC1BA8
- net X9B24D85652D0E6A4A818 renamed X00444C74247F40210707
- net X9D53207805B8DB8B6983 renamed X19B1E1FF84711BE7F475
- net X9F61A7055EEEA35F62E7 renamed X245C8A88BDE6BBB78DF6
- net XA0019CBD381390FABFAF renamed X008537AA7400D5A1B933
- net XA485A04AF81D21F345C4 renamed X47CDB73EF89C07E59C0F
- net XA83717DFE85A1843AF54 renamed X22EF82418C7C113D22A9
- net XA92686FC9F41649DE2A6 renamed XD9E610B68315B208DD4E
- net XAFB594C53DCECA3A3AD4 renamed XA1376930C555476901BB
- net XB1755A15F87901219DD1 renamed XFCBF7CEE1BED9441283A
- net XB52CB89C2AC1B41F5B1A renamed XB9C83C62FAFA64A9376E
- net XB66E196D7399A865DFDB renamed X555CDD0061680F23773B
- net XB7C2F315B2A72C7196F7 renamed X50214D29D17C9AFAE6DD
- net XBED713F0F20C2BEF6433 renamed XC8F08969780264FD50DA
- net XC0EE167C419B9155F9DB renamed XCDB392101F7276A507EC
- net XC504154F084880E31BD0 renamed XD1DF082127875B2EF3E6
- net XC960027B02DECF254F85 renamed XDFE73EDB3AA45015AAD2
- net XCD1B35E26F74529DDE12 renamed XF56F4DA8E29974FB0CE5
- net XD2CD8F2DD019093785A4 renamed XF3BE3F5F807C19D144CA
- net XE63A0B74B293D479E1AC renamed X5CD5EA02032391EA4821
- net XEE83BB852CD6F6752923 renamed X51F6671C66B653F81BC5
- net XF69333997B8E2F92DE05 renamed X0EF916B0CB53D9F46426
- net XFBFE7BE3D8ED3A77CE22 renamed X4070539D709C19A0AF65
- net XFD6D3BC4F6CA8CDDDA78 renamed X6BD40278C60E8AC692D2
- new net X09F11B5FD91688775527: J900042.1
- new net X0A690587C80EFD567FF7: J900044.7
- new net X1A3A22F4B289D6F62B00: J900046.7
- new net X20E5F5A8A70133CE0A4F: J900048.7
- new net X2E6E3A5B3A1EDB8DE440: J900038.3
- new net X4ACF6BCBD80FF39F4684: J900040.5
- new net X5929B9536D17079BD5A9: J900044.3
- new net X5BE49425103F808B4B93: J900044.5
- new net X6354D048E3F28D8D058A: J900042.5
- new net X6A4E9EB656E3E839FC9F: J900048.5
- new net X7753A9CB9C4C99AFEC62: J900046.3
- new net X7CC5966245686CF4EF46: J900046.1
- new net X80AB923B405609CBD8D4: J900042.3
- new net X873FBDA9321D775F6874: J900040.3
- new net X966F4C38FA03A1A25AF4: J900038.7
- new net X9D2B06F1BC5228248BF8: J900038.5
- new net XAC8E39F8B82E205A502C: J900044.1
- new net XD28ED4C8ADBB50D65408: J900040.1
- new net XDD3424A56BA0C1838507: J900042.7
- new net XDE7AB824E0E60E115AB7: J900040.7
- new net XDFB625F8D33B870AA8A2: J900038.1
- new net XE5186E13C39FD41C302C: J900048.1
- new net XE779E0163B1C90616ED0: J900046.5
- new net XF785BFE6DF6F90409592: J900048.3
