File: boards/osc-core/sheets/filter_F2_K.kicad_sch (KiCad schematic)
At the start: 171 parts, among them Q2201 BCM847BS,115, Q2202 MMBT3906,215, Q2203 MMBT3906,215, Q2204 MMBT3906,215, Q2205 MMBT3906,215, Q2206 MMBT3906,215, U2201 REF5050AIDR, U2206 LM13700M/NOPB, U2207 LM13700M/NOPB, U2208 OPA4197IPWR, U2209 OPA4197IPWR, U2210 OPA4196IDR, U2211 OPA4196IDR, U2212 OPA4196IDR, U2213 OPA4196IDR, U2214 OPA4196IDR, U2215 OPA4196IDR, U2216 OPA4196IDR

Commit message: Split jack partition into two boards with local bypass clusters
Parts:
- C2201: FootprintOriginMm 43.64,143.21 -> 28.64,143.46
- C2202: FootprintOriginMm 47.39,143.21 -> 32.39,143.46
- C2203: FootprintOriginMm 51.14,143.21 -> 99.89,143.46
- C2204: FootprintOriginMm 103.64,143.46 -> 202.89,143.71
- C2205: FootprintOriginMm 107.39,143.46 -> 206.64,143.71
- C2206: FootprintOriginMm 111.14,143.46 -> 210.39,143.71
- C2207: FootprintOriginMm 114.89,143.46 -> 214.14,143.71
- C2208: FootprintOriginMm 118.64,143.46 -> 217.89,143.71
- C2209: FootprintOriginMm 122.39,143.46 -> 221.64,143.71
- C2210: FootprintOriginMm 270.64,144.21 -> 225.39,143.71
- C2211: FootprintOriginMm 282.89,144.21 -> 229.14,143.71
- C2212: FootprintOriginMm 286.64,144.21 -> 232.89,143.71
- C2213: FootprintOriginMm 294.14,144.21 -> 257.64,143.71
- C2214: FootprintOriginMm 297.89,144.21 -> 261.39,143.71
- C2215: FootprintOriginMm 301.64,144.21 -> 265.14,143.71
- C2216: FootprintOriginMm 9.89,144.46 -> 58.64,144.21
- C2225: FootprintOriginMm 13.64,144.46 -> 67.39,144.21
- C2226: FootprintOriginMm 17.39,144.46 -> 71.14,144.21
- C2227: FootprintOriginMm 305.39,144.46 -> 81.14,144.21
- C2228: FootprintOriginMm 309.14,144.46 -> 84.89,144.21
- C2229: FootprintOriginMm 208.64,144.71 -> 88.64,144.21
- C2230: FootprintOriginMm 216.14,144.71 -> 132.89,144.21
- C2231: FootprintOriginMm 255.64,144.71 -> 136.64,144.21
- C2232: FootprintOriginMm 259.39,144.71 -> 140.39,144.21
- C2233: FootprintOriginMm 263.14,144.71 -> 144.14,144.21
- C2234: FootprintOriginMm 266.89,144.96 -> 165.39,144.21
- C2235: FootprintOriginMm 126.14,145.21 -> 268.89,144.21
- C2236: FootprintOriginMm 129.89,145.21 -> 272.64,144.21
- C2237: FootprintOriginMm 133.64,145.21 -> 276.39,144.21
- C2238: FootprintOriginMm 137.39,145.21 -> 280.14,144.21
- C2239: FootprintOriginMm 141.14,145.21 -> 283.89,144.21
- C2240: FootprintOriginMm 148.64,145.21 -> 147.89,144.46
- C2241: FootprintOriginMm 152.39,145.21 -> 151.64,144.46
- C2242: FootprintOriginMm 156.14,145.21 -> 155.39,144.46
- C2243: FootprintOriginMm 159.89,145.21 -> 159.14,144.46
- C2244: FootprintOriginMm 163.64,145.21 -> 287.64,144.46
- C2245: FootprintOriginMm 167.39,145.21 -> 6.14,144.71
- C2246: FootprintOriginMm 171.14,145.21 -> 13.64,144.71
- D2205: FootprintOriginMm 230.43,41.56 -> 228.93,46.06
- D2206: FootprintOriginMm 215.1,131.5 -> 216.35,130.5
- D2207: FootprintOriginMm 242.43,46.06 -> 241.93,46.06
- D2208: FootprintOriginMm 220.6,131.5 -> 226.6,130.5
- D2209: FootprintOriginMm 264.35,131.5 -> 232.1,130.5
- D2210: FootprintOriginMm 269.85,131.5 -> 237.6,130.5
- D2211: FootprintOriginMm 283.1,132.0 -> 270.35,130.5
- D2212: FootprintOriginMm 295.85,132.0 -> 275.85,130.5
- D2213: FootprintOriginMm 243.6,132.25 -> 65.1,131.0
- D2214: FootprintOriginMm 249.1,132.25 -> 141.1,131.0
- D2215: FootprintOriginMm 26.35,132.5 -> 146.6,131.0
- D2216: FootprintOriginMm 31.85,132.5 -> 152.1,131.0
- D2217: FootprintOriginMm 37.35,132.5 -> 171.35,131.0
- D2218: FootprintOriginMm 42.85,132.5 -> 281.35,131.0
- D2219: FootprintOriginMm 48.35,132.5 -> 286.85,131.0
- D2220: FootprintOriginMm 53.85,132.5 -> 292.35,131.0
- D2221: FootprintOriginMm 59.35,132.5 -> 16.6,131.25
- D2222: FootprintOriginMm 64.85,132.5 -> 76.35,131.25
- D2223: FootprintOriginMm 70.35,132.5 -> 90.6,131.25
- D2224: FootprintOriginMm 75.85,132.5 -> 96.1,131.25
- Q2201: FootprintOriginMm 273.6,84.28 -> 56.6,81.28
- Q2202: FootprintOriginMm 6.43,127.81 -> 141.18,127.56
- Q2203: FootprintOriginMm 16.43,127.81 -> 145.43,127.56
- Q2204: FootprintOriginMm 20.68,127.81 -> 149.68,127.56
- Q2205: FootprintOriginMm 24.93,127.81 -> 153.93,127.56
- Q2206: FootprintOriginMm 217.68,128.06 -> 172.18,127.56
- R2201: FootprintOriginMm 224.39,183.16 -> 126.14,180.16
- R2202: FootprintOriginMm 239.39,183.16 -> 129.89,180.16
- R2203: FootprintOriginMm 6.14,183.41 -> 133.64,180.16
- R2204: FootprintOriginMm 46.64,183.41 -> 152.64,180.16
- R2221: FootprintOriginMm 59.89,183.41 -> 257.39,180.16
- R2222: FootprintOriginMm 63.64,183.41 -> 261.14,180.16
- R2223: FootprintOriginMm 67.39,183.41 -> 137.39,180.41
- R2224: FootprintOriginMm 76.89,183.41 -> 141.14,180.41
- R2225: FootprintOriginMm 80.64,183.41 -> 144.89,180.41
- R2226: FootprintOriginMm 84.39,183.41 -> 148.64,180.41
- R2227: FootprintOriginMm 228.14,183.41 -> 9.89,180.66
- R2228: FootprintOriginMm 231.89,183.41 -> 111.14,180.66
- R2229: FootprintOriginMm 235.64,183.41 -> 171.39,180.66
- R2230: FootprintOriginMm 304.39,183.41 -> 216.14,180.66
- R2231: FootprintOriginMm 308.14,183.41 -> 231.14,180.66
- R2232: FootprintOriginMm 17.39,183.66 -> 234.89,180.66
- R2233: FootprintOriginMm 25.89,183.66 -> 270.64,180.66
- R2234: FootprintOriginMm 29.64,183.66 -> 29.64,180.91
- R2235: FootprintOriginMm 33.39,183.66 -> 33.39,180.91
- R2236: FootprintOriginMm 42.89,183.66 -> 42.89,180.91
- R2237: FootprintOriginMm 249.89,183.66 -> 46.64,180.91
- R2238: FootprintOriginMm 264.89,183.66 -> 50.39,180.91
- R2239: FootprintOriginMm 281.89,183.66 -> 69.89,180.91
- R2240: FootprintOriginMm 21.14,183.91 -> 84.39,180.91
- R2241: FootprintOriginMm 37.14,183.91 -> 93.89,180.91
- R2242: FootprintOriginMm 54.14,183.91 -> 97.64,180.91
- R2243: FootprintOriginMm 71.14,183.91 -> 101.39,180.91
- R2244: FootprintOriginMm 88.14,183.91 -> 105.14,180.91
- R2245: FootprintOriginMm 91.89,183.91 -> 114.89,180.91
- R2246: FootprintOriginMm 95.64,183.91 -> 156.39,180.91
- R2247: FootprintOriginMm 99.39,183.91 -> 160.14,180.91
- R2248: FootprintOriginMm 107.39,183.91 -> 163.89,180.91
- R2249: FootprintOriginMm 111.14,183.91 -> 167.64,180.91
- R2250: FootprintOriginMm 257.39,184.66 -> 175.14,180.91
- R2251: FootprintOriginMm 261.14,184.66 -> 178.89,180.91
- R2252: FootprintOriginMm 268.64,184.66 -> 182.64,180.91
- R2253: FootprintOriginMm 272.39,184.66 -> 186.39,180.91
- R2254: FootprintOriginMm 276.14,184.66 -> 223.64,180.91
- R2255: FootprintOriginMm 285.64,184.66 -> 227.39,180.91
- R2256: FootprintOriginMm 289.39,184.66 -> 238.64,180.91
- R2257: FootprintOriginMm 9.89,184.91 -> 6.14,181.16
- R2258: FootprintOriginMm 13.64,184.91 -> 205.14,181.16
- R2259: FootprintOriginMm 141.39,184.91 -> 302.64,181.16
- R2260: FootprintOriginMm 145.14,184.91 -> 306.39,181.16
- R2261: FootprintOriginMm 148.89,184.91 -> 310.14,181.16
- R2262: FootprintOriginMm 158.39,184.91 -> 242.39,181.41
- R2263: FootprintOriginMm 162.14,184.91 -> 249.89,181.41
- R2264: FootprintOriginMm 165.89,184.91 -> 264.89,181.41
- R2265: FootprintOriginMm 175.39,184.91 -> 274.39,181.41
- R2266: FootprintOriginMm 179.14,184.91 -> 278.14,181.41
- R2267: FootprintOriginMm 182.89,184.91 -> 281.89,181.41
- R2268: FootprintOriginMm 192.39,184.91 -> 285.64,181.41
- R2269: FootprintOriginMm 243.14,184.91 -> 289.39,181.41
- R2270: FootprintOriginMm 293.14,184.91 -> 293.14,181.41
- R2271: FootprintOriginMm 296.89,184.91 -> 296.89,181.41
- R2272: FootprintOriginMm 199.89,185.16 -> 13.64,181.66
- R2273: FootprintOriginMm 253.64,185.16 -> 17.39,181.66
- R2274: FootprintOriginMm 114.89,185.41 -> 25.89,181.66
- R2275: FootprintOriginMm 124.39,185.41 -> 190.14,181.91
- R2276: FootprintOriginMm 128.14,185.41 -> 193.89,181.91
- R2277: FootprintOriginMm 131.89,185.41 -> 197.64,181.91
- R2278: FootprintOriginMm 196.14,185.41 -> 208.89,181.91
- R2279: FootprintOriginMm 209.39,185.41 -> 219.89,181.91
- R2280: FootprintOriginMm 213.14,185.41 -> 246.14,181.91
- R2281: FootprintOriginMm 216.89,185.41 -> 59.89,182.41
- R2282: FootprintOriginMm 220.64,185.41 -> 63.64,182.41
- R2283: FootprintOriginMm 224.39,185.41 -> 76.89,182.41
- R2284: FootprintOriginMm 239.39,185.41 -> 80.64,182.41
- R2285: FootprintOriginMm 6.14,185.66 -> 124.39,182.41
- R2286: FootprintOriginMm 46.64,185.66 -> 128.14,182.41
- R2287: FootprintOriginMm 50.39,185.66 -> 131.89,182.41
- R2288: FootprintOriginMm 57.89,185.66 -> 253.64,182.41
- R2289: FootprintOriginMm 61.64,185.66 -> 257.39,182.41
- R2290: FootprintOriginMm 65.39,185.66 -> 261.14,182.41
- R2291: FootprintOriginMm 74.89,185.66 -> 141.39,182.66
- R2292: FootprintOriginMm 78.64,185.66 -> 145.14,182.66
- R2293: FootprintOriginMm 82.39,185.66 -> 148.89,182.66
- R2294: FootprintOriginMm 228.14,185.66 -> 9.89,182.91
- R2295: FootprintOriginMm 231.89,185.66 -> 108.89,182.91
- R2296: FootprintOriginMm 235.64,185.66 -> 201.39,182.91
- R2297: FootprintOriginMm 300.64,185.66 -> 212.64,182.91
- R2298: FootprintOriginMm 304.39,185.66 -> 231.14,182.91
- R2299: FootprintOriginMm 308.14,185.66 -> 234.89,182.91
- RB2201: FootprintOriginMm 294.64,221.66 -> 214.89,217.41
- RB2202: FootprintOriginMm 311.64,221.66 -> 231.89,217.41
- RB2203: FootprintOriginMm 21.14,221.91 -> 246.89,217.41
- RB2204: FootprintOriginMm 24.89,221.91 -> 263.39,217.41
- RB2205: FootprintOriginMm 28.64,221.91 -> 267.14,217.41
- RV2207: FootprintOriginMm 102.7,41.8 -> 85.7,41.8
- RV2208: FootprintOriginMm 119.7,41.8 -> 102.7,41.8
- RV2209: FootprintOriginMm 136.7,41.8 -> 119.7,41.8
- RV2210: FootprintOriginMm 153.7,41.8 -> 136.7,41.8
- RV2211: FootprintOriginMm 170.7,41.8 -> 221.7,41.8
- RV2212: FootprintOriginMm 187.7,41.8 -> 37.95,46.3
- RV2213: FootprintOriginMm 204.7,41.8 -> 45.7,51.8
- U2201: FootprintOriginMm 102.45,112.3 -> 201.95,112.3
- U2208: FootprintOriginMm 41.35,103.88 -> 8.35,102.88
- U2209: FootprintOriginMm 59.85,103.88 -> 16.6,102.88
