File: boards/osc-core/sheets/filter_F2_K.kicad_sch (KiCad schematic)
At the start: 171 parts, among them Q2201 BCM847BS,115, Q2202 MMBT3906,215, Q2203 MMBT3906,215, Q2204 MMBT3906,215, Q2205 MMBT3906,215, Q2206 MMBT3906,215, U2201 REF5050AIDR, U2206 LM13700M/NOPB, U2207 LM13700M/NOPB, U2208 OPA4197IPWR, U2209 OPA4197IPWR, U2210 OPA4196IDR, U2211 OPA4196IDR, U2212 OPA4196IDR, U2213 OPA4196IDR, U2214 OPA4196IDR, U2215 OPA4196IDR, U2216 OPA4196IDR

Commit message: WIP: locality placement source for the core board (#43)
Core packages are placed by the jack locality placer, anchored on the
core GH headers and pulled toward each module's own headers; IC/bypass
clusters stay rigid. Regenerated sources follow. Draft only.

Co-Authored-By: Claude Opus 5.5 <noreply@anthropic.com>
Parts:
- C2201: FootprintOriginMm 28.64,143.46 -> 78.89,98.96
- C2202: FootprintOriginMm 32.39,143.46 -> 107.39,100.96
- C2203: BoardSide B.Cu -> F.Cu; FootprintOriginMm 99.89,143.46 -> 96.14,155.46; KiCadOrientationDeg 180 -> 0
- C2204: BoardSide B.Cu -> F.Cu; FootprintOriginMm 202.89,143.71 -> 97.89,114.71; KiCadOrientationDeg 180 -> 0
- C2205: FootprintOriginMm 206.64,143.71 -> 76.89,103.96
- C2206: BoardSide B.Cu -> F.Cu; FootprintOriginMm 210.39,143.71 -> 89.89,114.71; KiCadOrientationDeg 180 -> 0
- C2207: FootprintOriginMm 214.14,143.71 -> 93.89,109.96
- C2208: FootprintOriginMm 217.89,143.71 -> 71.46,105.89; KiCadOrientationDeg 180 -> 90
- C2209: BoardSide B.Cu -> F.Cu; FootprintOriginMm 221.64,143.71 -> 82.89,153.46; KiCadOrientationDeg 180 -> 0
- C2210: FootprintOriginMm 225.39,143.71 -> 77.71,115.39; KiCadOrientationDeg 180 -> 90
- C2211: FootprintOriginMm 229.14,143.71 -> 78.89,101.46
- C2212: BoardSide B.Cu -> F.Cu; FootprintOriginMm 232.89,143.71 -> 75.39,107.96; KiCadOrientationDeg 180 -> 0
- C2213: BoardSide B.Cu -> F.Cu; FootprintOriginMm 257.64,143.71 -> 79.14,105.46; KiCadOrientationDeg 180 -> 0
- C2214: BoardSide B.Cu -> F.Cu; FootprintOriginMm 261.39,143.71 -> 82.64,116.96; KiCadOrientationDeg 180 -> 0
- C2215: FootprintOriginMm 265.14,143.71 -> 97.64,109.96
- C2216: BoardSide B.Cu -> F.Cu; FootprintOriginMm 58.64,144.21 -> 106.71000000000001,130.745; KiCadOrientationDeg 180 -> 90
- C2225: BoardSide B.Cu -> F.Cu; FootprintOriginMm 67.39,144.21 -> 88.48,149.445; KiCadOrientationDeg 180 -> 270
- C2226: BoardSide B.Cu -> F.Cu; FootprintOriginMm 71.14,144.21 -> 78.46,149.445; KiCadOrientationDeg 180 -> 270
- C2227: FootprintOriginMm 81.14,144.21 -> 88.71,157.04500000000002; KiCadOrientationDeg 180 -> 90
- C2228: FootprintOriginMm 84.89,144.21 -> 98.73,157.04500000000002; KiCadOrientationDeg 180 -> 90
- C2229: FootprintOriginMm 88.64,144.21 -> 103.78,126.17999999999999; KiCadOrientationDeg 180 -> 90
- C2230: FootprintOriginMm 132.89,144.21 -> 93.46000000000001,126.17999999999999; KiCadOrientationDeg 180 -> 90
- C2231: FootprintOriginMm 136.64,144.21 -> 105.56,123.03; KiCadOrientationDeg 180 -> 0
- C2232: FootprintOriginMm 140.39,144.21 -> 105.56,112.71000000000001; KiCadOrientationDeg 180 -> 0
- C2233: FootprintOriginMm 144.14,144.21 -> 98.73,134.5; KiCadOrientationDeg 180 -> 90
- C2234: FootprintOriginMm 165.39,144.21 -> 88.71,134.5; KiCadOrientationDeg 180 -> 90
- C2235: FootprintOriginMm 268.89,144.21 -> 88.71,145.63; KiCadOrientationDeg 180 -> 270
- C2236: FootprintOriginMm 272.64,144.21 -> 98.73,145.63; KiCadOrientationDeg 180 -> 270
- C2237: BoardSide B.Cu -> F.Cu; FootprintOriginMm 276.39,144.21 -> 88.71,135.89999999999998; KiCadOrientationDeg 180 -> 270
- C2238: BoardSide B.Cu -> F.Cu; FootprintOriginMm 280.14,144.21 -> 98.73,135.89999999999998; KiCadOrientationDeg 180 -> 270
- C2239: BoardSide B.Cu -> F.Cu; FootprintOriginMm 283.89,144.21 -> 98.73,144.23000000000002; KiCadOrientationDeg 180 -> 90
- C2240: BoardSide B.Cu -> F.Cu; FootprintOriginMm 147.89,144.46 -> 88.71,144.23000000000002; KiCadOrientationDeg 180 -> 90
- C2241: BoardSide B.Cu -> F.Cu; FootprintOriginMm 151.64,144.46 -> 88.48,132.23000000000002; KiCadOrientationDeg 180 -> 90
- C2242: BoardSide B.Cu -> F.Cu; FootprintOriginMm 155.39,144.46 -> 78.46,132.23000000000002; KiCadOrientationDeg 180 -> 90
- C2243: FootprintOriginMm 159.14,144.46 -> 100.48,118.0; KiCadOrientationDeg 180 -> 90
- C2244: FootprintOriginMm 287.64,144.46 -> 90.46,118.0; KiCadOrientationDeg 180 -> 90
- C2245: FootprintOriginMm 6.14,144.71 -> 90.23,123.25; KiCadOrientationDeg 180 -> 90
- C2246: FootprintOriginMm 13.64,144.71 -> 80.21,123.25; KiCadOrientationDeg 180 -> 90
- D2205: FootprintOriginMm 228.93,46.06 -> 87.81,138.43; KiCadOrientationDeg 180 -> 90
- D2206: BoardSide B.Cu -> F.Cu; FootprintOriginMm 216.35,130.5 -> 85.36,114.25; KiCadOrientationDeg 180 -> 0
- D2207: BoardSide B.Cu -> F.Cu; FootprintOriginMm 241.93,46.06 -> 94.43,128.06; KiCadOrientationDeg 180 -> 0
- D2208: BoardSide B.Cu -> F.Cu; FootprintOriginMm 226.6,130.5 -> 84.61,156.25; KiCadOrientationDeg 180 -> 0
- D2209: FootprintOriginMm 232.1,130.5 -> 85.1,109.75
- D2210: FootprintOriginMm 237.6,130.5 -> 78.85,112.0
- D2211: BoardSide B.Cu -> F.Cu; FootprintOriginMm 270.35,130.5 -> 98.86,112.0; KiCadOrientationDeg 180 -> 0
- D2212: FootprintOriginMm 275.85,130.5 -> 94.6,107.25
- D2213: BoardSide B.Cu -> F.Cu; FootprintOriginMm 65.1,131.0 -> 79.25,115.61; KiCadOrientationDeg 180 -> 270
- D2214: BoardSide B.Cu -> F.Cu; FootprintOriginMm 141.1,131.0 -> 89.11,111.25; KiCadOrientationDeg 180 -> 0
- D2215: BoardSide B.Cu -> F.Cu; FootprintOriginMm 146.6,131.0 -> 95.75,159.61; KiCadOrientationDeg 180 -> 270
- D2216: FootprintOriginMm 152.1,131.0 -> 100.1,107.25
- D2217: FootprintOriginMm 171.35,131.0 -> 89.1,106.5
- D2218: BoardSide B.Cu -> F.Cu; FootprintOriginMm 281.35,131.0 -> 84.61,159.25; KiCadOrientationDeg 180 -> 0
- D2219: BoardSide B.Cu -> F.Cu; FootprintOriginMm 286.85,131.0 -> 103.0,111.11; KiCadOrientationDeg 180 -> 270
- D2220: BoardSide B.Cu -> F.Cu; FootprintOriginMm 292.35,131.0 -> 93.75,109.36; KiCadOrientationDeg 180 -> 270
- D2221: FootprintOriginMm 16.6,131.25 -> 79.6,109.0
- D2222: BoardSide B.Cu -> F.Cu; FootprintOriginMm 76.35,131.25 -> 83.61,111.25; KiCadOrientationDeg 180 -> 0
- D2223: BoardSide B.Cu -> F.Cu; FootprintOriginMm 90.6,131.25 -> 98.11,109.0; KiCadOrientationDeg 180 -> 0
- D2224: FootprintOriginMm 96.1,131.25 -> 104.5,106.35; KiCadOrientationDeg 180 -> 90
- Q2201: FootprintOriginMm 56.6,81.28 -> 83.6,113.03
- Q2202: BoardSide B.Cu -> F.Cu; FootprintOriginMm 141.18,127.56 -> 100.93,101.81; KiCadOrientationDeg 180 -> 0
- Q2203: FootprintOriginMm 145.43,127.56 -> 84.56,106.18; KiCadOrientationDeg 180 -> 90
- Q2204: BoardSide B.Cu -> F.Cu; FootprintOriginMm 149.68,127.56 -> 99.43,161.56; KiCadOrientationDeg 180 -> 0
- Q2205: BoardSide B.Cu -> F.Cu; FootprintOriginMm 153.93,127.56 -> 93.93,114.06; KiCadOrientationDeg 180 -> 0
- Q2206: FootprintOriginMm 172.18,127.56 -> 90.06,110.18; KiCadOrientationDeg 180 -> 90
- R2201: FootprintOriginMm 126.14,180.16 -> 98.91,138.14; KiCadOrientationDeg 180 -> 90
- R2202: FootprintOriginMm 129.89,180.16 -> 93.89,104.66
- R2203: BoardSide B.Cu -> F.Cu; FootprintOriginMm 133.64,180.16 -> 98.91,139.64; KiCadOrientationDeg 180 -> 270
- R2204: FootprintOriginMm 152.64,180.16 -> 104.41,99.64; KiCadOrientationDeg 180 -> 90
- R2221: BoardSide B.Cu -> F.Cu; FootprintOriginMm 257.39,180.16 -> 88.66,139.64; KiCadOrientationDeg 180 -> 270
- R2222: BoardSide B.Cu -> F.Cu; FootprintOriginMm 261.14,180.16 -> 98.39,126.66; KiCadOrientationDeg 180 -> 0
- R2223: FootprintOriginMm 137.39,180.41 -> 101.16,147.39; KiCadOrientationDeg 180 -> 90
- R2224: FootprintOriginMm 141.14,180.41 -> 82.64,99.66
- R2225: BoardSide B.Cu -> F.Cu; FootprintOriginMm 144.89,180.41 -> 87.39,126.91; KiCadOrientationDeg 180 -> 0
- R2226: FootprintOriginMm 148.64,180.41 -> 97.64,104.66
- R2227: FootprintOriginMm 9.89,180.66 -> 100.66,121.64; KiCadOrientationDeg 180 -> 90
- R2228: FootprintOriginMm 111.14,180.66 -> 93.89,97.91
- R2229: FootprintOriginMm 171.39,180.66 -> 98.91,149.39; KiCadOrientationDeg 180 -> 90
- R2230: BoardSide B.Cu -> F.Cu; FootprintOriginMm 216.14,180.66 -> 102.14,126.66; KiCadOrientationDeg 180 -> 0
- R2231: FootprintOriginMm 231.14,180.66 -> 108.14,146.66
- R2232: BoardSide B.Cu -> F.Cu; FootprintOriginMm 234.89,180.66 -> 72.41,108.89; KiCadOrientationDeg 180 -> 270
- R2233: FootprintOriginMm 270.64,180.66 -> 98.91,153.14; KiCadOrientationDeg 180 -> 90
- R2234: BoardSide B.Cu -> F.Cu; FootprintOriginMm 29.64,180.91 -> 90.39,108.66; KiCadOrientationDeg 180 -> 0
- R2235: FootprintOriginMm 33.39,180.91 -> 109.39,123.91
- R2236: BoardSide B.Cu -> F.Cu; FootprintOriginMm 42.89,180.91 -> 96.89,101.91; KiCadOrientationDeg 180 -> 0
- R2237: FootprintOriginMm 46.64,180.91 -> 90.41,114.14; KiCadOrientationDeg 180 -> 90
- R2238: FootprintOriginMm 50.39,180.91 -> 82.41,116.89; KiCadOrientationDeg 180 -> 90
- R2239: BoardSide B.Cu -> F.Cu; FootprintOriginMm 69.89,180.91 -> 98.39,152.41; KiCadOrientationDeg 180 -> 0
- R2240: BoardSide B.Cu -> F.Cu; FootprintOriginMm 84.39,180.91 -> 90.89,101.91; KiCadOrientationDeg 180 -> 0
- R2241: FootprintOriginMm 93.89,180.91 -> 101.16,155.89; KiCadOrientationDeg 180 -> 90
- R2242: BoardSide B.Cu -> F.Cu; FootprintOriginMm 97.64,180.91 -> 86.64,108.66; KiCadOrientationDeg 180 -> 0
- R2243: BoardSide B.Cu -> F.Cu; FootprintOriginMm 101.39,180.91 -> 93.89,117.16; KiCadOrientationDeg 180 -> 0
- R2244: FootprintOriginMm 105.14,180.91 -> 97.64,97.91
- R2245: FootprintOriginMm 114.89,180.91 -> 90.14,103.91
- R2246: FootprintOriginMm 156.39,180.91 -> 80.64,106.41
- R2247: BoardSide B.Cu -> F.Cu; FootprintOriginMm 160.14,180.91 -> 106.39,110.16; KiCadOrientationDeg 180 -> 0
- R2248: FootprintOriginMm 163.89,180.91 -> 100.66,103.89; KiCadOrientationDeg 180 -> 90
- R2249: BoardSide B.Cu -> F.Cu; FootprintOriginMm 167.64,180.91 -> 79.66,110.89; KiCadOrientationDeg 180 -> 270
- R2250: FootprintOriginMm 175.14,180.91 -> 107.89,105.66
- R2251: FootprintOriginMm 178.89,180.91 -> 93.89,102.41
- R2252: FootprintOriginMm 182.64,180.91 -> 100.66,114.14; KiCadOrientationDeg 180 -> 90
- R2253: BoardSide B.Cu -> F.Cu; FootprintOriginMm 186.39,180.91 -> 82.89,108.66; KiCadOrientationDeg 180 -> 0
- R2254: FootprintOriginMm 223.64,180.91 -> 76.89,106.41
- R2255: BoardSide B.Cu -> F.Cu; FootprintOriginMm 227.39,180.91 -> 105.41,165.14; KiCadOrientationDeg 180 -> 270
- R2256: BoardSide B.Cu -> F.Cu; FootprintOriginMm 238.64,180.91 -> 97.64,117.16; KiCadOrientationDeg 180 -> 0
- R2257: FootprintOriginMm 6.14,181.16 -> 101.39,98.16
- R2258: BoardSide B.Cu -> F.Cu; FootprintOriginMm 205.14,181.16 -> 90.14,117.16; KiCadOrientationDeg 180 -> 0
- R2259: BoardSide B.Cu -> F.Cu; FootprintOriginMm 302.64,181.16 -> 89.66,153.14; KiCadOrientationDeg 180 -> 270
- R2260: BoardSide B.Cu -> F.Cu; FootprintOriginMm 306.39,181.16 -> 97.14,106.41; KiCadOrientationDeg 180 -> 0
- R2261: FootprintOriginMm 310.14,181.16 -> 87.39,113.41
- R2262: FootprintOriginMm 242.39,181.41 -> 93.89,112.41
- R2263: BoardSide B.Cu -> F.Cu; FootprintOriginMm 249.89,181.41 -> 82.16,103.39; KiCadOrientationDeg 180 -> 270
- R2264: BoardSide B.Cu -> F.Cu; FootprintOriginMm 264.89,181.41 -> 90.39,106.41; KiCadOrientationDeg 180 -> 0
- R2265: FootprintOriginMm 274.39,181.41 -> 73.14,102.91
- R2266: FootprintOriginMm 278.14,181.41 -> 85.64,156.41
- R2267: FootprintOriginMm 281.89,181.41 -> 68.39,105.16
- R2268: FootprintOriginMm 285.64,181.41 -> 97.64,102.41
- R2269: BoardSide B.Cu -> F.Cu; FootprintOriginMm 289.39,181.41 -> 93.91,100.89; KiCadOrientationDeg 180 -> 270
- R2270: FootprintOriginMm 293.14,181.41 -> 97.64,112.41
- R2271: FootprintOriginMm 296.89,181.41 -> 111.14,100.91
- R2272: FootprintOriginMm 13.64,181.66 -> 86.39,102.91
- R2273: BoardSide B.Cu -> F.Cu; FootprintOriginMm 17.39,181.66 -> 75.39,105.66; KiCadOrientationDeg 180 -> 0
- R2274: BoardSide B.Cu -> F.Cu; FootprintOriginMm 25.89,181.66 -> 102.14,152.41; KiCadOrientationDeg 180 -> 0
- R2275: BoardSide B.Cu -> F.Cu; FootprintOriginMm 190.14,181.91 -> 120.14,169.66; KiCadOrientationDeg 180 -> 0
- R2276: BoardSide B.Cu -> F.Cu; FootprintOriginMm 193.89,181.91 -> 102.64,107.16; KiCadOrientationDeg 180 -> 0
- R2277: FootprintOriginMm 197.64,181.91 -> 107.39,98.66
- R2278: BoardSide B.Cu -> F.Cu; FootprintOriginMm 208.89,181.91 -> 101.39,117.16; KiCadOrientationDeg 180 -> 0
- R2279: FootprintOriginMm 219.89,181.91 -> 84.39,97.41
- R2280: BoardSide B.Cu -> F.Cu; FootprintOriginMm 246.14,181.91 -> 86.64,106.41; KiCadOrientationDeg 180 -> 0
- R2281: FootprintOriginMm 59.89,182.41 -> 90.14,101.66
- R2282: FootprintOriginMm 63.64,182.41 -> 80.64,104.16
- R2283: BoardSide B.Cu -> F.Cu; FootprintOriginMm 76.89,182.41 -> 109.41,109.64; KiCadOrientationDeg 180 -> 270
- R2284: FootprintOriginMm 80.64,182.41 -> 103.64,102.66
- R2285: BoardSide B.Cu -> F.Cu; FootprintOriginMm 124.39,182.41 -> 106.39,107.91; KiCadOrientationDeg 180 -> 0
- R2286: BoardSide B.Cu -> F.Cu; FootprintOriginMm 128.14,182.41 -> 76.64,110.41; KiCadOrientationDeg 180 -> 0
- R2287: BoardSide B.Cu -> F.Cu; FootprintOriginMm 131.89,182.41 -> 72.89,111.91; KiCadOrientationDeg 180 -> 0
- R2288: BoardSide B.Cu -> F.Cu; FootprintOriginMm 253.64,182.41 -> 86.39,117.16; KiCadOrientationDeg 180 -> 0
- R2289: BoardSide B.Cu -> F.Cu; FootprintOriginMm 257.39,182.41 -> 93.91,104.64; KiCadOrientationDeg 180 -> 270
- R2290: FootprintOriginMm 261.14,182.41 -> 111.64,105.41
- R2291: FootprintOriginMm 141.39,182.66 -> 107.89,103.41
- R2292: BoardSide B.Cu -> F.Cu; FootprintOriginMm 145.14,182.66 -> 82.89,106.41; KiCadOrientationDeg 180 -> 0
- R2293: BoardSide B.Cu -> F.Cu; FootprintOriginMm 148.89,182.66 -> 79.14,107.91; KiCadOrientationDeg 180 -> 0
- R2294: FootprintOriginMm 9.89,182.91 -> 93.89,100.16
- R2295: BoardSide B.Cu -> F.Cu; FootprintOriginMm 108.89,182.91 -> 100.89,104.91; KiCadOrientationDeg 180 -> 0
- R2296: BoardSide B.Cu -> F.Cu; FootprintOriginMm 201.39,182.91 -> 96.89,104.16; KiCadOrientationDeg 180 -> 0
- R2297: FootprintOriginMm 212.64,182.91 -> 82.64,101.91
- R2298: BoardSide B.Cu -> F.Cu; FootprintOriginMm 231.14,182.91 -> 90.89,104.16; KiCadOrientationDeg 180 -> 0
- R2299: BoardSide B.Cu -> F.Cu; FootprintOriginMm 234.89,182.91 -> 86.64,153.41; KiCadOrientationDeg 180 -> 0
- RB2201: FootprintOriginMm 214.89,217.41 -> 97.64,100.16
- RB2202: FootprintOriginMm 231.89,217.41 -> 73.91,106.14; KiCadOrientationDeg 180 -> 90
- RB2203: FootprintOriginMm 246.89,217.41 -> 86.39,100.66
- RB2204: FootprintOriginMm 263.39,217.41 -> 101.39,100.41
- RB2205: FootprintOriginMm 267.14,217.41 -> 80.16,115.64; KiCadOrientationDeg 180 -> 90
- RV2207: BoardSide B.Cu -> F.Cu; FootprintOriginMm 85.7,41.8 -> 86.35,103.3; KiCadOrientationDeg 180 -> 0
- RV2208: FootprintOriginMm 102.7,41.8 -> 88.95,97.55
- RV2209: FootprintOriginMm 119.7,41.8 -> 102.7,133.3
- RV2210: BoardSide B.Cu -> F.Cu; FootprintOriginMm 136.7,41.8 -> 100.85,149.3; KiCadOrientationDeg 180 -> 0
- RV2211: FootprintOriginMm 221.7,41.8 -> 86.2,116.8
- RV2212: BoardSide B.Cu -> F.Cu; FootprintOriginMm 37.95,46.3 -> 93.85,152.3; KiCadOrientationDeg 180 -> 0
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
Commit message: WIP: spread core module homes and legalize module by module (#43)
The first core negotiation stalled (2501/2727 nets in conflict after 7
iterations). A RUDY map showed placement congestion: header-anchored
homes crowded ~1300 E/A packages into one corner, so modules were
scattered and 751 nets spanned 80 mm or more. Module home discs are now
spread inside the outline and notch, packages are legalized one module
at a time, and the core uses a 0.6 mm courtyard gap with a 0.5 mm IC
channel. Floorplan proxy: HPWL 162 -> 139 m, peak RUDY 1.39 -> 1.09 of
ideal four-signal-layer supply, tiles above 0.7 682 -> 160.

Co-Authored-By: Claude Opus 5.5 <noreply@anthropic.com>
Parts:
- C2201: BoardSide B.Cu -> F.Cu; FootprintOriginMm 78.89,98.96 -> 77.89,95.71; KiCadOrientationDeg 180 -> 0
- C2202: FootprintOriginMm 107.39,100.96 -> 65.96,68.89; KiCadOrientationDeg 180 -> 90
- C2203: BoardSide F.Cu -> B.Cu; FootprintOriginMm 96.14,155.46 -> 78.64,94.21; KiCadOrientationDeg 0 -> 180
- C2204: FootprintOriginMm 97.89,114.71 -> 80.14,63.71
- C2205: BoardSide B.Cu -> F.Cu; FootprintOriginMm 76.89,103.96 -> 103.39,62.21; KiCadOrientationDeg 180 -> 0
- C2206: BoardSide F.Cu -> B.Cu; FootprintOriginMm 89.89,114.71 -> 70.71,84.89; KiCadOrientationDeg 0 -> 90
- C2207: FootprintOriginMm 93.89,109.96 -> 107.96,69.89; KiCadOrientationDeg 180 -> 90
- C2208: BoardSide B.Cu -> F.Cu; FootprintOriginMm 71.46,105.89 -> 107.96,68.39; KiCadOrientationDeg 90 -> 270
- C2209: FootprintOriginMm 82.89,153.46 -> 93.64,60.96
- C2210: FootprintOriginMm 77.71,115.39 -> 101.46,93.64
- C2211: FootprintOriginMm 78.89,101.46 -> 113.71,80.39; KiCadOrientationDeg 180 -> 90
- C2212: BoardSide F.Cu -> B.Cu; FootprintOriginMm 75.39,107.96 -> 78.89,99.46; KiCadOrientationDeg 0 -> 180
- C2213: FootprintOriginMm 79.14,105.46 -> 83.14,96.96
- C2214: BoardSide F.Cu -> B.Cu; FootprintOriginMm 82.64,116.96 -> 89.14,56.21; KiCadOrientationDeg 0 -> 180
- C2215: BoardSide B.Cu -> F.Cu; FootprintOriginMm 97.64,109.96 -> 73.96,70.14; KiCadOrientationDeg 180 -> 270
- C2216: FootprintOriginMm 106.71000000000001,130.745 -> 78.995,66.46; KiCadOrientationDeg 90 -> 180
- C2225: FootprintOriginMm 88.48,149.445 -> 78.89,87.405; KiCadOrientationDeg 270 -> 180
- C2226: FootprintOriginMm 78.46,149.445 -> 90.27,87.405; KiCadOrientationDeg 270 -> 0
- C2227: BoardSide B.Cu -> F.Cu; FootprintOriginMm 88.71,157.04500000000002 -> 95.21,67.205
- C2228: BoardSide B.Cu -> F.Cu; FootprintOriginMm 98.73,157.04500000000002 -> 105.23,67.205
- C2229: FootprintOriginMm 103.78,126.17999999999999 -> 78.42999999999999,71.96000000000001; KiCadOrientationDeg 90 -> 180
- C2230: FootprintOriginMm 93.46000000000001,126.17999999999999 -> 78.42999999999999,82.28; KiCadOrientationDeg 90 -> 180
- C2231: FootprintOriginMm 105.56,123.03 -> 81.53,66.17999999999999; KiCadOrientationDeg 0 -> 90
- C2232: FootprintOriginMm 105.56,112.71000000000001 -> 71.21000000000001,66.17999999999999; KiCadOrientationDeg 0 -> 90
- C2233: FootprintOriginMm 98.73,134.5 -> 94.23,76.5
- C2234: FootprintOriginMm 88.71,134.5 -> 84.21,76.5
- C2235: FootprintOriginMm 88.71,145.63 -> 94.23,65.25; KiCadOrientationDeg 270 -> 90
- C2236: FootprintOriginMm 98.73,145.63 -> 84.21,65.25; KiCadOrientationDeg 270 -> 90
- C2237: FootprintOriginMm 88.71,135.89999999999998 -> 84.21,71.4
- C2238: FootprintOriginMm 98.73,135.89999999999998 -> 94.23,71.4
- C2239: BoardSide F.Cu -> B.Cu; FootprintOriginMm 98.73,144.23000000000002 -> 95.21,80.63000000000001; KiCadOrientationDeg 90 -> 270
- C2240: BoardSide F.Cu -> B.Cu; FootprintOriginMm 88.71,144.23000000000002 -> 105.23,80.63000000000001; KiCadOrientationDeg 90 -> 270
- C2241: BoardSide F.Cu -> B.Cu; FootprintOriginMm 88.48,132.23000000000002 -> 95.21,69.38000000000001; KiCadOrientationDeg 90 -> 270
- C2242: BoardSide F.Cu -> B.Cu; FootprintOriginMm 78.46,132.23000000000002 -> 105.23,69.38000000000001; KiCadOrientationDeg 90 -> 270
- C2243: FootprintOriginMm 100.48,118.0 -> 94.43,96.27; KiCadOrientationDeg 90 -> 270
- C2244: FootprintOriginMm 90.46,118.0 -> 94.43,84.89
- C2245: FootprintOriginMm 90.23,123.25 -> 82.75,83.21; KiCadOrientationDeg 90 -> 180
- C2246: FootprintOriginMm 80.21,123.25 -> 82.75,93.23; KiCadOrientationDeg 90 -> 180
- D2205: FootprintOriginMm 87.81,138.43 -> 82.43,60.81; KiCadOrientationDeg 90 -> 180
- D2206: BoardSide F.Cu -> B.Cu; FootprintOriginMm 85.36,114.25 -> 96.35,57.0; KiCadOrientationDeg 0 -> 180
- D2207: BoardSide F.Cu -> B.Cu; FootprintOriginMm 94.43,128.06 -> 75.43,88.06; KiCadOrientationDeg 0 -> 180
- D2208: BoardSide F.Cu -> B.Cu; FootprintOriginMm 84.61,156.25 -> 81.6,57.0; KiCadOrientationDeg 0 -> 180
- D2209: BoardSide B.Cu -> F.Cu; FootprintOriginMm 85.1,109.75 -> 92.11,94.25; KiCadOrientationDeg 180 -> 0
- D2210: BoardSide B.Cu -> F.Cu; FootprintOriginMm 78.85,112.0 -> 98.61,91.75; KiCadOrientationDeg 180 -> 0
- D2211: BoardSide F.Cu -> B.Cu; FootprintOriginMm 98.86,112.0 -> 106.5,64.1; KiCadOrientationDeg 0 -> 90
- D2212: BoardSide B.Cu -> F.Cu; FootprintOriginMm 94.6,107.25 -> 106.5,73.36; KiCadOrientationDeg 180 -> 270
- D2213: BoardSide F.Cu -> B.Cu; FootprintOriginMm 79.25,115.61 -> 71.5,89.6; KiCadOrientationDeg 270 -> 90
- D2214: FootprintOriginMm 89.11,111.25 -> 98.61,62.0
- D2215: FootprintOriginMm 95.75,159.61 -> 81.86,60.75; KiCadOrientationDeg 270 -> 0
- D2216: FootprintOriginMm 100.1,107.25 -> 67.6,80.75
- D2217: FootprintOriginMm 89.1,106.5 -> 110.75,81.1; KiCadOrientationDeg 180 -> 90
- D2218: FootprintOriginMm 84.61,159.25 -> 77.11,90.25
- D2219: BoardSide F.Cu -> B.Cu; FootprintOriginMm 103.0,111.11 -> 97.25,97.85; KiCadOrientationDeg 270 -> 90
- D2220: BoardSide F.Cu -> B.Cu; FootprintOriginMm 93.75,109.36 -> 111.5,75.35; KiCadOrientationDeg 270 -> 90
- D2221: FootprintOriginMm 79.6,109.0 -> 73.1,61.25
- D2222: BoardSide F.Cu -> B.Cu; FootprintOriginMm 83.61,111.25 -> 89.1,99.5; KiCadOrientationDeg 0 -> 180
- D2223: FootprintOriginMm 98.11,109.0 -> 71.0,73.36; KiCadOrientationDeg 0 -> 270
- D2224: FootprintOriginMm 104.5,106.35 -> 66.5,76.1
- Q2201: FootprintOriginMm 83.6,113.03 -> 101.85,61.53
- Q2202: BoardSide F.Cu -> B.Cu; FootprintOriginMm 100.93,101.81 -> 64.68,84.56; KiCadOrientationDeg 0 -> 180
- Q2203: BoardSide B.Cu -> F.Cu; FootprintOriginMm 84.56,106.18 -> 103.56,89.43; KiCadOrientationDeg 90 -> 270
- Q2204: FootprintOriginMm 99.43,161.56 -> 74.68,64.81
- Q2205: BoardSide F.Cu -> B.Cu; FootprintOriginMm 93.93,114.06 -> 106.81,88.18; KiCadOrientationDeg 0 -> 90
- Q2206: BoardSide B.Cu -> F.Cu; FootprintOriginMm 90.06,110.18 -> 89.43,60.31; KiCadOrientationDeg 90 -> 0
- R2201: FootprintOriginMm 98.91,138.14 -> 83.41,70.39
- R2202: BoardSide B.Cu -> F.Cu; FootprintOriginMm 93.89,104.66 -> 74.89,87.16; KiCadOrientationDeg 180 -> 0
- R2203: BoardSide F.Cu -> B.Cu; FootprintOriginMm 98.91,139.64 -> 73.14,73.16; KiCadOrientationDeg 270 -> 180
- R2204: BoardSide B.Cu -> F.Cu; FootprintOriginMm 104.41,99.64 -> 68.16,74.14; KiCadOrientationDeg 90 -> 270
- R2221: BoardSide F.Cu -> B.Cu; FootprintOriginMm 88.66,139.64 -> 73.14,81.66; KiCadOrientationDeg 270 -> 180
- R2222: FootprintOriginMm 98.39,126.66 -> 94.39,88.91
- R2223: FootprintOriginMm 101.16,147.39 -> 106.16,76.39
- R2224: FootprintOriginMm 82.64,99.66 -> 113.16,70.64; KiCadOrientationDeg 180 -> 90
- R2225: BoardSide F.Cu -> B.Cu; FootprintOriginMm 87.39,126.91 -> 86.89,94.16; KiCadOrientationDeg 0 -> 180
- R2226: BoardSide B.Cu -> F.Cu; FootprintOriginMm 97.64,104.66 -> 104.66,85.14; KiCadOrientationDeg 180 -> 270
- R2227: BoardSide B.Cu -> F.Cu; FootprintOriginMm 100.66,121.64 -> 99.66,85.14; KiCadOrientationDeg 90 -> 270
- R2228: FootprintOriginMm 93.89,97.91 -> 71.41,94.64; KiCadOrientationDeg 180 -> 90
- R2229: BoardSide B.Cu -> F.Cu; FootprintOriginMm 98.91,149.39 -> 77.89,84.41; KiCadOrientationDeg 90 -> 0
- R2230: FootprintOriginMm 102.14,126.66 -> 89.14,63.66
- R2231: BoardSide B.Cu -> F.Cu; FootprintOriginMm 108.14,146.66 -> 83.41,64.89; KiCadOrientationDeg 180 -> 270
- R2232: FootprintOriginMm 72.41,108.89 -> 93.39,55.91; KiCadOrientationDeg 270 -> 0
- R2233: BoardSide B.Cu -> F.Cu; FootprintOriginMm 98.91,153.14 -> 90.41,90.64; KiCadOrientationDeg 90 -> 270
- R2234: BoardSide F.Cu -> B.Cu; FootprintOriginMm 90.39,108.66 -> 77.66,58.39; KiCadOrientationDeg 0 -> 90
- R2235: BoardSide B.Cu -> F.Cu; FootprintOriginMm 109.39,123.91 -> 93.14,63.66; KiCadOrientationDeg 180 -> 0
- R2236: BoardSide F.Cu -> B.Cu; FootprintOriginMm 96.89,101.91 -> 78.64,54.16; KiCadOrientationDeg 0 -> 180
- R2237: FootprintOriginMm 90.41,114.14 -> 106.89,73.16; KiCadOrientationDeg 90 -> 180
- R2238: FootprintOriginMm 82.41,116.89 -> 89.14,58.91; KiCadOrientationDeg 90 -> 180
- R2239: FootprintOriginMm 98.39,152.41 -> 85.91,62.89; KiCadOrientationDeg 0 -> 270
- R2240: BoardSide F.Cu -> B.Cu; FootprintOriginMm 90.89,101.91 -> 89.14,51.16; KiCadOrientationDeg 0 -> 180
- R2241: BoardSide B.Cu -> F.Cu; FootprintOriginMm 101.16,155.89 -> 93.64,91.41; KiCadOrientationDeg 90 -> 0
- R2242: BoardSide F.Cu -> B.Cu; FootprintOriginMm 86.64,108.66 -> 82.89,98.41; KiCadOrientationDeg 0 -> 180
- R2243: FootprintOriginMm 93.89,117.16 -> 98.39,88.91
- R2244: BoardSide B.Cu -> F.Cu; FootprintOriginMm 97.64,97.91 -> 107.16,87.89; KiCadOrientationDeg 180 -> 270
- R2245: FootprintOriginMm 90.14,103.91 -> 74.64,93.91
- R2246: FootprintOriginMm 80.64,106.41 -> 68.16,84.39; KiCadOrientationDeg 180 -> 90
- R2247: BoardSide F.Cu -> B.Cu; FootprintOriginMm 106.39,110.16 -> 78.89,96.91; KiCadOrientationDeg 0 -> 180
- R2248: FootprintOriginMm 100.66,103.89 -> 104.89,92.91; KiCadOrientationDeg 90 -> 180
- R2249: BoardSide F.Cu -> B.Cu; FootprintOriginMm 79.66,110.89 -> 68.66,68.39; KiCadOrientationDeg 270 -> 90
- R2250: FootprintOriginMm 107.89,105.66 -> 110.66,70.64; KiCadOrientationDeg 180 -> 90
- R2251: BoardSide B.Cu -> F.Cu; FootprintOriginMm 93.89,102.41 -> 85.91,58.89; KiCadOrientationDeg 180 -> 270
- R2252: FootprintOriginMm 100.66,114.14 -> 78.14,61.66; KiCadOrientationDeg 90 -> 180
- R2253: BoardSide F.Cu -> B.Cu; FootprintOriginMm 82.89,108.66 -> 101.89,58.41; KiCadOrientationDeg 0 -> 180
- R2254: FootprintOriginMm 76.89,106.41 -> 93.41,100.39; KiCadOrientationDeg 180 -> 90
- R2255: BoardSide F.Cu -> B.Cu; FootprintOriginMm 105.41,165.14 -> 66.64,72.16; KiCadOrientationDeg 270 -> 180
- R2256: BoardSide F.Cu -> B.Cu; FootprintOriginMm 97.64,117.16 -> 107.91,80.39; KiCadOrientationDeg 0 -> 90
- R2257: BoardSide B.Cu -> F.Cu; FootprintOriginMm 101.39,98.16 -> 72.91,90.39; KiCadOrientationDeg 180 -> 270
- R2258: FootprintOriginMm 90.14,117.16 -> 102.16,85.14; KiCadOrientationDeg 0 -> 270
- R2259: BoardSide F.Cu -> B.Cu; FootprintOriginMm 89.66,153.14 -> 92.41,58.14; KiCadOrientationDeg 270 -> 90
- R2260: BoardSide F.Cu -> B.Cu; FootprintOriginMm 97.14,106.41 -> 100.89,96.91; KiCadOrientationDeg 0 -> 180
- R2261: FootprintOriginMm 87.39,113.41 -> 85.91,58.14; KiCadOrientationDeg 180 -> 90
- R2262: BoardSide B.Cu -> F.Cu; FootprintOriginMm 93.89,112.41 -> 74.16,74.14; KiCadOrientationDeg 180 -> 270
- R2263: BoardSide F.Cu -> B.Cu; FootprintOriginMm 82.16,103.39 -> 63.66,77.14; KiCadOrientationDeg 270 -> 90
- R2264: BoardSide F.Cu -> B.Cu; FootprintOriginMm 90.39,106.41 -> 110.41,86.14; KiCadOrientationDeg 0 -> 90
- R2265: FootprintOriginMm 73.14,102.91 -> 89.14,102.41
- R2266: FootprintOriginMm 85.64,156.41 -> 90.89,96.41
- R2267: FootprintOriginMm 68.39,105.16 -> 100.89,99.41
- R2268: BoardSide B.Cu -> F.Cu; FootprintOriginMm 97.64,102.41 -> 96.89,94.66; KiCadOrientationDeg 180 -> 0
- R2269: FootprintOriginMm 93.91,100.89 -> 87.14,99.41; KiCadOrientationDeg 270 -> 0
- R2270: FootprintOriginMm 97.64,112.41 -> 108.66,76.39; KiCadOrientationDeg 180 -> 90
- R2271: FootprintOriginMm 111.14,100.91 -> 114.41,76.39; KiCadOrientationDeg 180 -> 90
- R2272: FootprintOriginMm 86.39,102.91 -> 109.41,65.89; KiCadOrientationDeg 180 -> 90
- R2273: BoardSide F.Cu -> B.Cu; FootprintOriginMm 75.39,105.66 -> 111.91,66.64; KiCadOrientationDeg 0 -> 90
- R2274: BoardSide F.Cu -> B.Cu; FootprintOriginMm 102.14,152.41 -> 75.64,91.41; KiCadOrientationDeg 0 -> 180
- R2275: FootprintOriginMm 120.14,169.66 -> 100.89,94.66
- R2276: BoardSide F.Cu -> B.Cu; FootprintOriginMm 102.64,107.16 -> 92.41,54.14; KiCadOrientationDeg 0 -> 90
- R2277: FootprintOriginMm 107.39,98.66 -> 109.41,61.89; KiCadOrientationDeg 180 -> 90
- R2278: BoardSide F.Cu -> B.Cu; FootprintOriginMm 101.39,117.16 -> 86.89,96.66; KiCadOrientationDeg 0 -> 180
- R2279: FootprintOriginMm 84.39,97.41 -> 112.91,86.14; KiCadOrientationDeg 180 -> 90
- R2280: BoardSide F.Cu -> B.Cu; FootprintOriginMm 86.64,106.41 -> 85.91,54.14; KiCadOrientationDeg 0 -> 90
- R2281: BoardSide B.Cu -> F.Cu; FootprintOriginMm 90.14,101.66 -> 93.64,58.41; KiCadOrientationDeg 180 -> 0
- R2282: FootprintOriginMm 80.64,104.16 -> 89.14,53.66
- R2283: FootprintOriginMm 109.41,109.64 -> 77.89,93.16; KiCadOrientationDeg 270 -> 0
- R2284: FootprintOriginMm 103.64,102.66 -> 68.66,88.89; KiCadOrientationDeg 180 -> 90
- R2285: FootprintOriginMm 106.39,107.91 -> 87.14,96.91
- R2286: BoardSide F.Cu -> B.Cu; FootprintOriginMm 76.64,110.41 -> 74.39,58.41; KiCadOrientationDeg 0 -> 180
- R2287: BoardSide F.Cu -> B.Cu; FootprintOriginMm 72.89,111.91 -> 95.64,54.16; KiCadOrientationDeg 0 -> 180
- R2288: BoardSide F.Cu -> B.Cu; FootprintOriginMm 86.39,117.16 -> 69.41,77.14; KiCadOrientationDeg 0 -> 90
- R2289: BoardSide F.Cu -> B.Cu; FootprintOriginMm 93.91,104.64 -> 105.89,60.16; KiCadOrientationDeg 270 -> 180
- R2290: BoardSide B.Cu -> F.Cu; FootprintOriginMm 111.64,105.41 -> 109.41,74.14; KiCadOrientationDeg 180 -> 270
- R2291: FootprintOriginMm 107.89,103.41 -> 82.64,54.16
- R2292: FootprintOriginMm 82.89,106.41 -> 97.64,59.16
- R2293: FootprintOriginMm 79.14,107.91 -> 70.91,85.14; KiCadOrientationDeg 0 -> 270
- R2294: BoardSide B.Cu -> F.Cu; FootprintOriginMm 93.89,100.16 -> 71.16,68.39; KiCadOrientationDeg 180 -> 270
- R2295: FootprintOriginMm 100.89,104.91 -> 91.14,97.16
- R2296: BoardSide F.Cu -> B.Cu; FootprintOriginMm 96.89,104.16 -> 74.64,96.41; KiCadOrientationDeg 0 -> 180
- R2297: FootprintOriginMm 82.64,101.91 -> 104.89,95.41
- R2298: FootprintOriginMm 90.89,104.16 -> 95.14,97.16
- R2299: BoardSide F.Cu -> B.Cu; FootprintOriginMm 86.64,153.41 -> 82.89,95.91; KiCadOrientationDeg 0 -> 180
- RB2201: FootprintOriginMm 97.64,100.16 -> 68.66,64.39; KiCadOrientationDeg 180 -> 90
- RB2202: BoardSide B.Cu -> F.Cu; FootprintOriginMm 73.91,106.14 -> 89.39,56.91; KiCadOrientationDeg 90 -> 0
- RB2203: BoardSide B.Cu -> F.Cu; FootprintOriginMm 86.39,100.66 -> 76.89,61.16; KiCadOrientationDeg 180 -> 0
- RB2204: FootprintOriginMm 101.39,100.41 -> 84.39,100.91
- RB2205: FootprintOriginMm 80.16,115.64 -> 69.91,72.39
- RV2207: FootprintOriginMm 86.35,103.3 -> 81.85,57.05
- RV2208: FootprintOriginMm 88.95,97.55 -> 102.2,55.05
- RV2209: BoardSide B.Cu -> F.Cu; FootprintOriginMm 102.7,133.3 -> 95.6,85.55; KiCadOrientationDeg 180 -> 0
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
Commit message: WIP: same-footprint swap pass for the core placement (#43)
Ported span-penalized slot swaps (nets over 60 mm pay a quadratic
penalty), limited to same-footprint slots within 25 mm of each package's
net median. Floorplan proxy: HPWL 139 -> 105 m, median span 28.8 mm,
RUDY p99 0.78 with 68 tiles above 0.7 (JL with swaps: p99 0.81, 42).

Co-Authored-By: Claude Opus 5.5 <noreply@anthropic.com>
Parts:
- C2201: FootprintOriginMm 77.89,95.71 -> 107.96,68.39; KiCadOrientationDeg 0 -> 270
- C2203: BoardSide B.Cu -> F.Cu; FootprintOriginMm 78.64,94.21 -> 90.64,108.96; KiCadOrientationDeg 180 -> 0
- C2204: FootprintOriginMm 80.14,63.71 -> 77.89,95.71
- C2205: BoardSide F.Cu -> B.Cu; FootprintOriginMm 103.39,62.21 -> 113.71,80.39; KiCadOrientationDeg 0 -> 90
- C2206: FootprintOriginMm 70.71,84.89 -> 101.46,93.64
- C2207: FootprintOriginMm 107.96,69.89 -> 89.14,56.21; KiCadOrientationDeg 90 -> 180
- C2208: BoardSide F.Cu -> B.Cu; FootprintOriginMm 107.96,68.39 -> 78.89,99.46; KiCadOrientationDeg 270 -> 180
- C2210: BoardSide B.Cu -> F.Cu; FootprintOriginMm 101.46,93.64 -> 80.14,63.71; KiCadOrientationDeg 90 -> 0
- C2211: FootprintOriginMm 113.71,80.39 -> 107.96,69.89
- C2212: FootprintOriginMm 78.89,99.46 -> 70.71,84.89; KiCadOrientationDeg 180 -> 90
- C2213: BoardSide F.Cu -> B.Cu; FootprintOriginMm 83.14,96.96 -> 78.64,94.21; KiCadOrientationDeg 0 -> 180
- C2214: BoardSide B.Cu -> F.Cu; FootprintOriginMm 89.14,56.21 -> 103.39,62.21; KiCadOrientationDeg 180 -> 0
- D2205: FootprintOriginMm 82.43,60.81 -> 106.81,88.18; KiCadOrientationDeg 180 -> 90
- D2206: FootprintOriginMm 96.35,57.0 -> 81.6,57.0
- D2207: BoardSide B.Cu -> F.Cu; FootprintOriginMm 75.43,88.06 -> 103.56,89.43; KiCadOrientationDeg 180 -> 270
- D2208: BoardSide B.Cu -> F.Cu; FootprintOriginMm 81.6,57.0 -> 81.86,60.75; KiCadOrientationDeg 180 -> 0
- D2209: BoardSide F.Cu -> B.Cu; FootprintOriginMm 92.11,94.25 -> 97.25,97.85; KiCadOrientationDeg 0 -> 90
- D2211: FootprintOriginMm 106.5,64.1 -> 110.75,81.1
- D2212: BoardSide F.Cu -> B.Cu; FootprintOriginMm 106.5,73.36 -> 111.5,75.35; KiCadOrientationDeg 270 -> 90
- D2213: BoardSide B.Cu -> F.Cu; FootprintOriginMm 71.5,89.6 -> 106.5,73.36; KiCadOrientationDeg 90 -> 270
- D2214: BoardSide F.Cu -> B.Cu; FootprintOriginMm 98.61,62.0 -> 106.5,64.1; KiCadOrientationDeg 0 -> 90
- D2215: FootprintOriginMm 81.86,60.75 -> 98.61,62.0
- D2216: FootprintOriginMm 67.6,80.75 -> 96.35,57.0
- D2217: FootprintOriginMm 110.75,81.1 -> 89.1,99.5; KiCadOrientationDeg 90 -> 180
- D2218: FootprintOriginMm 77.11,90.25 -> 92.11,94.25
- D2219: BoardSide B.Cu -> F.Cu; FootprintOriginMm 97.25,97.85 -> 77.11,90.25; KiCadOrientationDeg 90 -> 0
- D2220: FootprintOriginMm 111.5,75.35 -> 71.5,89.6
- D2221: FootprintOriginMm 73.1,61.25 -> 67.6,80.75
- D2222: FootprintOriginMm 89.1,99.5 -> 66.5,76.1; KiCadOrientationDeg 180 -> 90
- D2224: FootprintOriginMm 66.5,76.1 -> 73.1,61.25; KiCadOrientationDeg 90 -> 180
- Q2202: BoardSide B.Cu -> F.Cu; FootprintOriginMm 64.68,84.56 -> 74.68,64.81; KiCadOrientationDeg 180 -> 0
- Q2203: BoardSide F.Cu -> B.Cu; FootprintOriginMm 103.56,89.43 -> 75.43,88.06; KiCadOrientationDeg 270 -> 180
- Q2204: BoardSide F.Cu -> B.Cu; FootprintOriginMm 74.68,64.81 -> 64.68,84.56; KiCadOrientationDeg 0 -> 180
- Q2205: BoardSide B.Cu -> F.Cu; FootprintOriginMm 106.81,88.18 -> 89.43,60.31; KiCadOrientationDeg 90 -> 0
- Q2206: BoardSide F.Cu -> B.Cu; FootprintOriginMm 89.43,60.31 -> 82.43,60.81; KiCadOrientationDeg 0 -> 180
- R2201: FootprintOriginMm 83.41,70.39 -> 73.14,81.66; KiCadOrientationDeg 90 -> 180
- R2202: FootprintOriginMm 74.89,87.16 -> 77.89,84.41
- R2203: FootprintOriginMm 73.14,73.16 -> 74.64,96.41
- R2204: BoardSide F.Cu -> B.Cu; FootprintOriginMm 68.16,74.14 -> 74.64,93.91; KiCadOrientationDeg 270 -> 180
- R2221: FootprintOriginMm 73.14,81.66 -> 94.64,137.16
- R2222: BoardSide F.Cu -> B.Cu; FootprintOriginMm 94.39,88.91 -> 90.64,136.91; KiCadOrientationDeg 0 -> 180
- R2223: FootprintOriginMm 106.16,76.39 -> 112.14,138.66; KiCadOrientationDeg 90 -> 180
- R2224: FootprintOriginMm 113.16,70.64 -> 110.41,86.14
- R2225: FootprintOriginMm 86.89,94.16 -> 63.66,77.14; KiCadOrientationDeg 180 -> 90
- R2226: BoardSide F.Cu -> B.Cu; FootprintOriginMm 104.66,85.14 -> 82.89,95.91; KiCadOrientationDeg 270 -> 180
- R2227: BoardSide F.Cu -> B.Cu; FootprintOriginMm 99.66,85.14 -> 117.41,134.14; KiCadOrientationDeg 270 -> 90
- R2228: FootprintOriginMm 71.41,94.64 -> 112.91,86.14
- R2229: BoardSide F.Cu -> B.Cu; FootprintOriginMm 77.89,84.41 -> 103.14,109.91; KiCadOrientationDeg 0 -> 180
- R2230: BoardSide F.Cu -> B.Cu; FootprintOriginMm 89.14,63.66 -> 106.41,110.14; KiCadOrientationDeg 0 -> 90
- R2231: BoardSide F.Cu -> B.Cu; FootprintOriginMm 83.41,64.89 -> 100.16,152.64; KiCadOrientationDeg 270 -> 90
- R2232: FootprintOriginMm 93.39,55.91 -> 87.14,96.91
- R2233: BoardSide F.Cu -> B.Cu; FootprintOriginMm 90.41,90.64 -> 89.14,51.16; KiCadOrientationDeg 270 -> 180
- R2234: FootprintOriginMm 77.66,58.39 -> 89.14,53.66; KiCadOrientationDeg 90 -> 180
- R2235: BoardSide F.Cu -> B.Cu; FootprintOriginMm 93.14,63.66 -> 87.39,134.16; KiCadOrientationDeg 0 -> 180
- R2236: FootprintOriginMm 78.64,54.16 -> 78.89,96.91
- R2237: BoardSide B.Cu -> F.Cu; FootprintOriginMm 106.89,73.16 -> 98.64,128.91; KiCadOrientationDeg 180 -> 0
- R2238: BoardSide B.Cu -> F.Cu; FootprintOriginMm 89.14,58.91 -> 94.64,129.16; KiCadOrientationDeg 180 -> 0
- R2239: BoardSide F.Cu -> B.Cu; FootprintOriginMm 85.91,62.89 -> 99.41,156.64; KiCadOrientationDeg 270 -> 90
- R2240: BoardSide B.Cu -> F.Cu; FootprintOriginMm 89.14,51.16 -> 91.14,97.16; KiCadOrientationDeg 180 -> 0
- R2241: BoardSide F.Cu -> B.Cu; FootprintOriginMm 93.64,91.41 -> 85.91,58.14; KiCadOrientationDeg 0 -> 90
- R2242: BoardSide B.Cu -> F.Cu; FootprintOriginMm 82.89,98.41 -> 85.91,58.89; KiCadOrientationDeg 180 -> 270
- R2243: BoardSide F.Cu -> B.Cu; FootprintOriginMm 98.39,88.91 -> 91.39,134.41; KiCadOrientationDeg 0 -> 180
- R2245: FootprintOriginMm 74.64,93.91 -> 69.41,77.14; KiCadOrientationDeg 180 -> 90
- R2246: BoardSide B.Cu -> F.Cu; FootprintOriginMm 68.16,84.39 -> 74.16,74.14; KiCadOrientationDeg 90 -> 270
- R2247: FootprintOriginMm 78.89,96.91 -> 73.14,73.16
- R2248: FootprintOriginMm 104.89,92.91 -> 69.91,72.39; KiCadOrientationDeg 180 -> 90
- R2249: BoardSide B.Cu -> F.Cu; FootprintOriginMm 68.66,68.39 -> 71.16,68.39; KiCadOrientationDeg 90 -> 270
- R2250: FootprintOriginMm 110.66,70.64 -> 77.66,58.39
- R2251: BoardSide F.Cu -> B.Cu; FootprintOriginMm 85.91,58.89 -> 78.14,61.66; KiCadOrientationDeg 270 -> 180
- R2252: FootprintOriginMm 78.14,61.66 -> 109.41,61.89; KiCadOrientationDeg 180 -> 90
- R2253: BoardSide B.Cu -> F.Cu; FootprintOriginMm 101.89,58.41 -> 93.14,63.66; KiCadOrientationDeg 180 -> 0
- R2254: BoardSide B.Cu -> F.Cu; FootprintOriginMm 93.41,100.39 -> 74.89,87.16; KiCadOrientationDeg 90 -> 0
- R2255: FootprintOriginMm 66.64,72.16 -> 68.66,88.89; KiCadOrientationDeg 180 -> 90
- R2256: FootprintOriginMm 107.91,80.39 -> 68.66,64.39
- R2257: BoardSide F.Cu -> B.Cu; FootprintOriginMm 72.91,90.39 -> 68.66,68.39; KiCadOrientationDeg 270 -> 90
- R2258: BoardSide F.Cu -> B.Cu; FootprintOriginMm 102.16,85.14 -> 85.91,54.14; KiCadOrientationDeg 270 -> 90
- R2259: FootprintOriginMm 92.41,58.14 -> 82.64,54.16; KiCadOrientationDeg 90 -> 180
- R2260: BoardSide B.Cu -> F.Cu; FootprintOriginMm 100.89,96.91 -> 90.41,90.64; KiCadOrientationDeg 180 -> 270
- R2261: FootprintOriginMm 85.91,58.14 -> 78.64,54.16; KiCadOrientationDeg 90 -> 180
- R2262: FootprintOriginMm 74.16,74.14 -> 68.16,74.14
- R2263: FootprintOriginMm 63.66,77.14 -> 68.16,84.39
- R2264: FootprintOriginMm 110.41,86.14 -> 86.89,94.16; KiCadOrientationDeg 90 -> 180
- R2265: FootprintOriginMm 89.14,102.41 -> 86.89,96.66
- R2266: BoardSide B.Cu -> F.Cu; FootprintOriginMm 90.89,96.41 -> 70.91,85.14; KiCadOrientationDeg 180 -> 270
- R2267: FootprintOriginMm 100.89,99.41 -> 71.41,94.64; KiCadOrientationDeg 180 -> 90
- R2268: FootprintOriginMm 96.89,94.66 -> 72.91,90.39; KiCadOrientationDeg 0 -> 270
- R2269: FootprintOriginMm 87.14,99.41 -> 77.89,93.16
- R2270: FootprintOriginMm 108.66,76.39 -> 92.41,54.14
- R2271: FootprintOriginMm 114.41,76.39 -> 95.64,54.16; KiCadOrientationDeg 90 -> 180
- R2272: FootprintOriginMm 109.41,65.89 -> 108.66,76.39
- R2273: BoardSide B.Cu -> F.Cu; FootprintOriginMm 111.91,66.64 -> 109.41,74.14; KiCadOrientationDeg 90 -> 270
- R2274: FootprintOriginMm 75.64,91.41 -> 74.39,58.41
- R2275: FootprintOriginMm 100.89,94.66 -> 76.89,61.16
- R2276: BoardSide B.Cu -> F.Cu; FootprintOriginMm 92.41,54.14 -> 97.64,59.16; KiCadOrientationDeg 90 -> 0
- R2277: FootprintOriginMm 109.41,61.89 -> 101.89,58.41; KiCadOrientationDeg 90 -> 180
- R2278: FootprintOriginMm 86.89,96.66 -> 113.16,70.64; KiCadOrientationDeg 180 -> 90
- R2279: FootprintOriginMm 112.91,86.14 -> 114.41,76.39
- R2280: BoardSide B.Cu -> F.Cu; FootprintOriginMm 85.91,54.14 -> 89.39,56.91; KiCadOrientationDeg 90 -> 0
- R2281: FootprintOriginMm 93.64,58.41 -> 93.39,55.91
- R2282: BoardSide B.Cu -> F.Cu; FootprintOriginMm 89.14,53.66 -> 99.66,85.14; KiCadOrientationDeg 180 -> 270
- R2283: FootprintOriginMm 77.89,93.16 -> 102.16,85.14; KiCadOrientationDeg 0 -> 270
- R2284: BoardSide B.Cu -> F.Cu; FootprintOriginMm 68.66,88.89 -> 104.66,85.14; KiCadOrientationDeg 90 -> 270
- R2285: BoardSide F.Cu -> B.Cu; FootprintOriginMm 87.14,96.91 -> 107.91,80.39; KiCadOrientationDeg 0 -> 90
- R2286: FootprintOriginMm 74.39,58.41 -> 106.16,76.39; KiCadOrientationDeg 180 -> 90
- R2287: FootprintOriginMm 95.64,54.16 -> 106.89,73.16
- R2288: BoardSide B.Cu -> F.Cu; FootprintOriginMm 69.41,77.14 -> 85.91,62.89; KiCadOrientationDeg 90 -> 270
- R2289: FootprintOriginMm 105.89,60.16 -> 92.41,58.14; KiCadOrientationDeg 180 -> 90
- R2290: FootprintOriginMm 109.41,74.14 -> 93.64,58.41; KiCadOrientationDeg 270 -> 0
- R2291: BoardSide B.Cu -> F.Cu; FootprintOriginMm 82.64,54.16 -> 89.14,63.66; KiCadOrientationDeg 180 -> 0
- R2292: BoardSide F.Cu -> B.Cu; FootprintOriginMm 97.64,59.16 -> 89.14,58.91; KiCadOrientationDeg 0 -> 180
- R2293: BoardSide F.Cu -> B.Cu; FootprintOriginMm 70.91,85.14 -> 105.89,60.16; KiCadOrientationDeg 270 -> 180
- R2294: BoardSide F.Cu -> B.Cu; FootprintOriginMm 71.16,68.39 -> 109.41,65.89; KiCadOrientationDeg 270 -> 90
- R2295: BoardSide F.Cu -> B.Cu; FootprintOriginMm 91.14,97.16 -> 111.91,66.64; KiCadOrientationDeg 0 -> 90
- R2296: FootprintOriginMm 74.64,96.41 -> 110.66,70.64; KiCadOrientationDeg 180 -> 90
- R2297: BoardSide B.Cu -> F.Cu; FootprintOriginMm 104.89,95.41 -> 93.64,91.41; KiCadOrientationDeg 180 -> 0
- R2298: FootprintOriginMm 95.14,97.16 -> 94.39,88.91
- R2299: FootprintOriginMm 82.89,95.91 -> 75.64,91.41
- RB2201: FootprintOriginMm 68.66,64.39 -> 83.41,70.39
- RB2202: FootprintOriginMm 89.39,56.91 -> 83.41,64.89; KiCadOrientationDeg 0 -> 270
- RB2203: FootprintOriginMm 76.89,61.16 -> 98.39,88.91
- RB2204: FootprintOriginMm 84.39,100.91 -> 90.89,96.41
- RB2205: FootprintOriginMm 69.91,72.39 -> 66.64,72.16; KiCadOrientationDeg 90 -> 180
- RV2211: FootprintOriginMm 102.35,88.45 -> 109.1,93.2
- RV2213: FootprintOriginMm 109.1,93.2 -> 102.35,88.45
