File: boards/osc-core/sheets/mix5_M5A_K.kicad_sch (KiCad schematic)
At the start: 76 parts, among them U8101 REF5050AIDR, U8107 OPA4197IPWR, U8108 OPA4196IDR, U8109 OPA4196IDR, U8110 OPA4196IDR, U8111 OPA4196IDR

Commit message: Split jack partition into two boards with local bypass clusters
Parts:
- C8101: FootprintOriginMm 238.64,160.46 -> 252.64,161.21
- C8102: FootprintOriginMm 242.39,160.46 -> 55.14,161.71
- C8103: FootprintOriginMm 17.64,160.71 -> 66.14,161.71
- C8104: FootprintOriginMm 21.39,160.71 -> 69.89,161.71
- C8105: FootprintOriginMm 28.89,160.71 -> 77.39,161.71
- C8106: FootprintOriginMm 32.64,160.71 -> 81.14,161.71
- C8107: FootprintOriginMm 36.39,160.71 -> 84.89,161.71
- C8108: FootprintOriginMm 40.14,160.71 -> 122.39,161.71
- C8109: FootprintOriginMm 43.89,160.71 -> 126.14,161.71
- C8110: FootprintOriginMm 99.89,160.96 -> 129.89,161.71
- C8111: FootprintOriginMm 103.64,160.96 -> 133.64,161.71
- C8112: FootprintOriginMm 107.39,160.96 -> 137.39,161.71
- C8113: FootprintOriginMm 111.14,160.96 -> 156.14,161.71
- C8114: FootprintOriginMm 114.89,160.96 -> 260.14,161.71
- C8129: FootprintOriginMm 118.64,160.96 -> 263.89,161.71
- C8130: FootprintOriginMm 267.39,161.71 -> 267.64,161.71
- C8131: FootprintOriginMm 279.89,161.71 -> 271.39,161.71
- C8132: FootprintOriginMm 283.64,161.71 -> 275.14,161.71
- C8133: FootprintOriginMm 291.14,161.71 -> 141.14,161.96
- C8134: FootprintOriginMm 294.89,161.71 -> 144.89,161.96
- C8135: FootprintOriginMm 298.64,161.71 -> 148.64,161.96
- C8136: FootprintOriginMm 10.14,161.96 -> 152.39,161.96
- C8137: FootprintOriginMm 13.89,161.96 -> 10.14,162.21
- C8138: FootprintOriginMm 302.39,161.96 -> 206.14,162.21
- R8101: FootprintOriginMm 58.14,210.91 -> 165.64,208.16
- R8102: FootprintOriginMm 75.14,210.91 -> 184.64,208.16
- R8103: FootprintOriginMm 61.89,211.16 -> 199.64,208.16
- R8104: FootprintOriginMm 78.89,211.16 -> 294.64,208.16
- R8109: FootprintOriginMm 256.39,211.66 -> 311.64,208.16
- R8110: FootprintOriginMm 273.39,211.66 -> 17.39,208.41
- R8111: FootprintOriginMm 9.89,211.91 -> 33.89,208.41
- R8112: FootprintOriginMm 13.64,211.91 -> 50.64,208.41
- R8113: FootprintOriginMm 144.89,211.91 -> 67.64,208.41
- R8114: FootprintOriginMm 161.89,211.91 -> 84.64,208.41
- R8119: FootprintOriginMm 175.39,211.91 -> 220.39,208.41
- R8120: FootprintOriginMm 283.14,211.91 -> 237.64,208.41
- R8121: FootprintOriginMm 88.39,212.16 -> 254.64,208.41
- R8122: FootprintOriginMm 92.14,212.16 -> 271.89,208.41
- R8123: FootprintOriginMm 107.39,212.16 -> 275.64,208.41
- R8124: FootprintOriginMm 124.39,212.16 -> 285.14,208.41
- R8129: FootprintOriginMm 128.14,212.16 -> 288.89,208.41
- R8130: FootprintOriginMm 241.39,212.16 -> 305.89,208.41
- R8131: FootprintOriginMm 99.64,212.41 -> 13.64,208.66
- R8132: FootprintOriginMm 116.64,212.41 -> 46.89,208.66
- R8133: FootprintOriginMm 192.39,212.41 -> 60.14,208.66
- R8134: FootprintOriginMm 209.39,212.41 -> 77.14,208.66
- R8139: FootprintOriginMm 213.14,212.41 -> 63.89,208.91
- R8140: FootprintOriginMm 231.64,212.41 -> 80.89,208.91
- R8141: FootprintOriginMm 245.14,212.41 -> 175.14,208.91
- R8142: FootprintOriginMm 248.89,212.41 -> 178.89,208.91
- R8143: FootprintOriginMm 260.14,212.41 -> 118.64,209.41
- R8144: FootprintOriginMm 277.14,212.41 -> 241.39,209.41
- R8149: FootprintOriginMm 296.39,212.41 -> 134.64,209.66
- R8150: FootprintOriginMm 6.14,212.66 -> 9.89,209.91
- R8151: FootprintOriginMm 39.89,212.66 -> 88.39,209.91
- R8152: FootprintOriginMm 43.64,212.66 -> 92.14,209.91
- R8153: FootprintOriginMm 51.14,212.66 -> 105.39,209.91
- R8154: FootprintOriginMm 71.39,212.66 -> 109.14,209.91
- R8155: FootprintOriginMm 95.89,212.66 -> 122.39,209.91
- R8156: FootprintOriginMm 111.14,212.66 -> 126.14,209.91
- R8157: FootprintOriginMm 131.89,212.66 -> 138.39,209.91
- R8158: FootprintOriginMm 148.64,212.66 -> 156.14,209.91
- R8159: FootprintOriginMm 165.64,212.66 -> 169.39,209.91
- R8160: FootprintOriginMm 179.14,212.66 -> 188.39,209.91
- R8161: FootprintOriginMm 182.89,212.66 -> 192.14,209.91
- R8162: FootprintOriginMm 196.14,212.66 -> 195.89,209.91
- R8163: FootprintOriginMm 199.89,212.66 -> 224.14,209.91
- R8164: FootprintOriginMm 222.14,212.66 -> 258.39,209.91
- R8165: FootprintOriginMm 225.89,212.66 -> 21.14,210.16
- R8166: FootprintOriginMm 292.64,212.66 -> 24.89,210.16
- U8101: FootprintOriginMm 92.2,116.8 -> 64.45,118.55
- U8107: FootprintOriginMm 41.35,110.38 -> 16.6,109.38
- U8108: FootprintOriginMm 34.95,91.2 -> 69.95,91.2
- U8109: FootprintOriginMm 52.95,91.2 -> 86.95,91.2
- U8110: FootprintOriginMm 69.95,91.2 -> 103.95,91.2
- U8111: FootprintOriginMm 86.95,91.2 -> 120.95,91.2
