File: boards/osc-core/sheets/mix5_M5A_K.kicad_sch (KiCad schematic)
At the start: 76 parts, among them U8101 REF5050AIDR, U8107 OPA4197IPWR, U8108 OPA4196IDR, U8109 OPA4196IDR, U8110 OPA4196IDR, U8111 OPA4196IDR

Commit message: WIP: locality placement source for the core board (#43)
Core packages are placed by the jack locality placer, anchored on the
core GH headers and pulled toward each module's own headers; IC/bypass
clusters stay rigid. Regenerated sources follow. Draft only.

Co-Authored-By: Claude Opus 5.5 <noreply@anthropic.com>
Parts:
- C8101: FootprintOriginMm 252.64,161.21 -> 116.64,97.71
- C8102: FootprintOriginMm 55.14,161.71 -> 115.96,101.39; KiCadOrientationDeg 180 -> 90
- C8103: FootprintOriginMm 66.14,161.71 -> 111.89,107.71
- C8104: FootprintOriginMm 69.89,161.71 -> 108.14,132.46
- C8105: FootprintOriginMm 77.39,161.71 -> 108.14,107.96
- C8106: FootprintOriginMm 81.14,161.71 -> 121.64,131.46
- C8107: BoardSide B.Cu -> F.Cu; FootprintOriginMm 84.89,161.71 -> 106.39,112.46; KiCadOrientationDeg 180 -> 0
- C8108: FootprintOriginMm 122.39,161.71 -> 107.39,129.71
- C8109: BoardSide B.Cu -> F.Cu; FootprintOriginMm 126.14,161.71 -> 99.21,157.64; KiCadOrientationDeg 180 -> 270
- C8110: BoardSide B.Cu -> F.Cu; FootprintOriginMm 129.89,161.71 -> 108.14,133.96; KiCadOrientationDeg 180 -> 0
- C8111: FootprintOriginMm 133.64,161.71 -> 115.64,106.71
- C8112: BoardSide B.Cu -> F.Cu; FootprintOriginMm 137.39,161.71 -> 111.96,143.14; KiCadOrientationDeg 180 -> 270
- C8113: FootprintOriginMm 156.14,161.71 -> 97.14,162.46
- C8114: BoardSide B.Cu -> F.Cu; FootprintOriginMm 260.14,161.71 -> 115.14,152.945; KiCadOrientationDeg 180 -> 0
- C8129: FootprintOriginMm 263.89,161.71 -> 120.78,127.42999999999999; KiCadOrientationDeg 180 -> 90
- C8130: FootprintOriginMm 267.64,161.71 -> 110.46000000000001,127.42999999999999; KiCadOrientationDeg 180 -> 90
- C8131: FootprintOriginMm 271.39,161.71 -> 118.98,135.75; KiCadOrientationDeg 180 -> 90
- C8132: FootprintOriginMm 275.14,161.71 -> 108.96,135.75; KiCadOrientationDeg 180 -> 90
- C8133: BoardSide B.Cu -> F.Cu; FootprintOriginMm 141.14,161.96 -> 108.96,137.14999999999998; KiCadOrientationDeg 180 -> 270
- C8134: BoardSide B.Cu -> F.Cu; FootprintOriginMm 144.89,161.96 -> 118.98,137.14999999999998; KiCadOrientationDeg 180 -> 270
- C8135: FootprintOriginMm 148.64,161.96 -> 104.5,136.46
- C8136: FootprintOriginMm 152.39,161.96 -> 104.5,146.48
- C8137: BoardSide B.Cu -> F.Cu; FootprintOriginMm 10.14,162.21 -> 105.9,147.98; KiCadOrientationDeg 180 -> 0
- C8138: BoardSide B.Cu -> F.Cu; FootprintOriginMm 206.14,162.21 -> 105.9,137.96; KiCadOrientationDeg 180 -> 0
- R8101: FootprintOriginMm 165.64,208.16 -> 105.39,158.91
- R8102: BoardSide B.Cu -> F.Cu; FootprintOriginMm 184.64,208.16 -> 109.14,117.16; KiCadOrientationDeg 180 -> 0
- R8103: FootprintOriginMm 199.64,208.16 -> 111.89,112.41
- R8104: BoardSide B.Cu -> F.Cu; FootprintOriginMm 294.64,208.16 -> 112.14,103.66; KiCadOrientationDeg 180 -> 0
- R8109: BoardSide B.Cu -> F.Cu; FootprintOriginMm 311.64,208.16 -> 103.64,154.66; KiCadOrientationDeg 180 -> 0
- R8110: FootprintOriginMm 17.39,208.41 -> 109.14,161.41
- R8111: BoardSide B.Cu -> F.Cu; FootprintOriginMm 33.89,208.41 -> 105.39,117.16; KiCadOrientationDeg 180 -> 0
- R8112: BoardSide B.Cu -> F.Cu; FootprintOriginMm 50.64,208.41 -> 115.89,102.91; KiCadOrientationDeg 180 -> 0
- R8113: FootprintOriginMm 67.64,208.41 -> 115.64,111.41
- R8114: FootprintOriginMm 84.64,208.41 -> 108.91,111.64; KiCadOrientationDeg 180 -> 90
- R8119: FootprintOriginMm 220.39,208.41 -> 102.41,159.64; KiCadOrientationDeg 180 -> 90
- R8120: BoardSide B.Cu -> F.Cu; FootprintOriginMm 237.64,208.41 -> 113.89,114.91; KiCadOrientationDeg 180 -> 0
- R8121: FootprintOriginMm 254.64,208.41 -> 105.39,161.16
- R8122: BoardSide B.Cu -> F.Cu; FootprintOriginMm 271.89,208.41 -> 123.89,168.91; KiCadOrientationDeg 180 -> 0
- R8123: FootprintOriginMm 275.64,208.41 -> 115.14,162.66
- R8124: BoardSide B.Cu -> F.Cu; FootprintOriginMm 285.14,208.41 -> 117.64,114.91; KiCadOrientationDeg 180 -> 0
- R8129: BoardSide B.Cu -> F.Cu; FootprintOriginMm 288.89,208.41 -> 110.14,114.91; KiCadOrientationDeg 180 -> 0
- R8130: FootprintOriginMm 305.89,208.41 -> 118.89,162.66
- R8131: BoardSide B.Cu -> F.Cu; FootprintOriginMm 13.64,208.66 -> 113.39,159.16; KiCadOrientationDeg 180 -> 0
- R8132: FootprintOriginMm 46.89,208.66 -> 112.89,98.66
- R8133: FootprintOriginMm 60.14,208.66 -> 111.89,110.16
- R8134: BoardSide B.Cu -> F.Cu; FootprintOriginMm 77.14,208.66 -> 99.89,154.66; KiCadOrientationDeg 180 -> 0
- R8139: BoardSide B.Cu -> F.Cu; FootprintOriginMm 63.89,208.91 -> 106.39,114.91; KiCadOrientationDeg 180 -> 0
- R8140: BoardSide B.Cu -> F.Cu; FootprintOriginMm 80.89,208.91 -> 102.39,156.91; KiCadOrientationDeg 180 -> 0
- R8141: FootprintOriginMm 175.14,208.91 -> 111.39,163.91
- R8142: BoardSide B.Cu -> F.Cu; FootprintOriginMm 178.89,208.91 -> 119.64,102.91; KiCadOrientationDeg 180 -> 0
- R8143: FootprintOriginMm 118.64,209.41 -> 105.89,110.41
- R8144: FootprintOriginMm 241.39,209.41 -> 115.64,109.16
- R8149: FootprintOriginMm 134.64,209.66 -> 122.41,110.39; KiCadOrientationDeg 180 -> 90
- R8150: FootprintOriginMm 9.89,209.91 -> 107.64,163.66
- R8151: FootprintOriginMm 88.39,209.91 -> 100.16,160.89; KiCadOrientationDeg 180 -> 90
- R8152: FootprintOriginMm 92.14,209.91 -> 122.89,174.66
- R8153: BoardSide B.Cu -> F.Cu; FootprintOriginMm 105.39,209.91 -> 117.14,160.41; KiCadOrientationDeg 180 -> 0
- R8154: BoardSide B.Cu -> F.Cu; FootprintOriginMm 109.14,209.91 -> 113.89,112.66; KiCadOrientationDeg 180 -> 0
- R8155: FootprintOriginMm 122.39,209.91 -> 119.39,109.16
- R8156: FootprintOriginMm 126.14,209.91 -> 115.14,164.91
- R8157: FootprintOriginMm 138.39,209.91 -> 101.64,111.16
- R8158: BoardSide B.Cu -> F.Cu; FootprintOriginMm 156.14,209.91 -> 117.64,112.66; KiCadOrientationDeg 180 -> 0
- R8159: BoardSide B.Cu -> F.Cu; FootprintOriginMm 169.39,209.91 -> 110.14,112.66; KiCadOrientationDeg 180 -> 0
- R8160: BoardSide B.Cu -> F.Cu; FootprintOriginMm 188.39,209.91 -> 102.64,114.91; KiCadOrientationDeg 180 -> 0
- R8161: FootprintOriginMm 192.14,209.91 -> 103.89,163.41
- R8162: FootprintOriginMm 195.89,209.91 -> 122.64,163.91
- R8163: FootprintOriginMm 224.14,209.91 -> 118.89,164.91
- R8164: FootprintOriginMm 258.39,209.91 -> 128.39,173.16
- R8165: BoardSide B.Cu -> F.Cu; FootprintOriginMm 21.14,210.16 -> 109.64,166.66; KiCadOrientationDeg 180 -> 0
- R8166: BoardSide B.Cu -> F.Cu; FootprintOriginMm 24.89,210.16 -> 113.39,161.41; KiCadOrientationDeg 180 -> 0
- U8101: BoardSide B.Cu -> F.Cu; FootprintOriginMm 64.45,118.55 -> 109.45,152.31
- U8107: FootprintOriginMm 16.6,109.38 -> 115.62,128.13
- U8108: FootprintOriginMm 69.95,91.2 -> 113.97,136.45
- U8109: BoardSide B.Cu -> F.Cu; FootprintOriginMm 86.95,91.2 -> 113.97,136.45; KiCadOrientationDeg 180 -> 0
- U8110: FootprintOriginMm 103.95,91.2 -> 105.2,141.47; KiCadOrientationDeg 180 -> 270
- U8111: BoardSide B.Cu -> F.Cu; FootprintOriginMm 120.95,91.2 -> 105.2,142.97; KiCadOrientationDeg 180 -> 90

Commit message: WIP: spread core module homes and legalize module by module (#43)
The first core negotiation stalled (2501/2727 nets in conflict after 7
iterations). A RUDY map showed placement congestion: header-anchored
homes crowded ~1300 E/A packages into one corner, so modules were
scattered and 751 nets spanned 80 mm or more. Module home discs are now
spread inside the outline and notch, packages are legalized one module
at a time, and the core uses a 0.6 mm courtyard gap with a 0.5 mm IC
channel. Floorplan proxy: HPWL 162 -> 139 m, peak RUDY 1.39 -> 1.09 of
ideal four-signal-layer supply, tiles above 0.7 682 -> 160.

Co-Authored-By: Claude Opus 5.5 <noreply@anthropic.com>
Parts:
- C8101: BoardSide B.Cu -> F.Cu; FootprintOriginMm 116.64,97.71 -> 90.64,133.21; KiCadOrientationDeg 180 -> 0
- C8102: BoardSide B.Cu -> F.Cu; FootprintOriginMm 115.96,101.39 -> 94.64,106.46; KiCadOrientationDeg 90 -> 0
- C8103: BoardSide B.Cu -> F.Cu; FootprintOriginMm 111.89,107.71 -> 90.64,108.96; KiCadOrientationDeg 180 -> 0
- C8104: FootprintOriginMm 108.14,132.46 -> 88.14,114.21
- C8105: FootprintOriginMm 108.14,107.96 -> 83.39,132.21
- C8106: FootprintOriginMm 121.64,131.46 -> 91.39,129.21
- C8107: BoardSide F.Cu -> B.Cu; FootprintOriginMm 106.39,112.46 -> 110.46,125.14; KiCadOrientationDeg 0 -> 90
- C8108: FootprintOriginMm 107.39,129.71 -> 87.14,126.46
- C8109: BoardSide F.Cu -> B.Cu; FootprintOriginMm 99.21,157.64 -> 79.46,113.89; KiCadOrientationDeg 270 -> 90
- C8110: FootprintOriginMm 108.14,133.96 -> 94.64,126.46
- C8111: BoardSide B.Cu -> F.Cu; FootprintOriginMm 115.64,106.71 -> 104.71,112.14; KiCadOrientationDeg 180 -> 270
- C8112: BoardSide F.Cu -> B.Cu; FootprintOriginMm 111.96,143.14 -> 101.14,112.46; KiCadOrientationDeg 270 -> 180
- C8113: FootprintOriginMm 97.14,162.46 -> 108.46,129.89; KiCadOrientationDeg 180 -> 90
- C8114: BoardSide F.Cu -> B.Cu; FootprintOriginMm 115.14,152.945 -> 99.71000000000001,108.965; KiCadOrientationDeg 0 -> 90
- C8129: BoardSide B.Cu -> F.Cu; FootprintOriginMm 120.78,127.42999999999999 -> 89.46000000000001,115.08; KiCadOrientationDeg 90 -> 270
- C8130: BoardSide B.Cu -> F.Cu; FootprintOriginMm 110.46000000000001,127.42999999999999 -> 99.78,115.08; KiCadOrientationDeg 90 -> 270
- C8131: FootprintOriginMm 118.98,135.75 -> 95.38000000000001,125.23; KiCadOrientationDeg 90 -> 0
- C8132: FootprintOriginMm 108.96,135.75 -> 95.38000000000001,115.21; KiCadOrientationDeg 90 -> 0
- C8133: BoardSide F.Cu -> B.Cu; FootprintOriginMm 108.96,137.14999999999998 -> 83.0,115.46; KiCadOrientationDeg 270 -> 180
- C8134: BoardSide F.Cu -> B.Cu; FootprintOriginMm 118.98,137.14999999999998 -> 83.0,125.48; KiCadOrientationDeg 270 -> 180
- C8135: FootprintOriginMm 104.5,136.46 -> 106.63000000000001,123.48; KiCadOrientationDeg 180 -> 0
- C8136: FootprintOriginMm 104.5,146.48 -> 106.63000000000001,113.46; KiCadOrientationDeg 180 -> 0
- C8137: BoardSide F.Cu -> B.Cu; FootprintOriginMm 105.9,147.98 -> 99.63000000000001,136.23
- C8138: BoardSide F.Cu -> B.Cu; FootprintOriginMm 105.9,137.96 -> 99.63000000000001,126.21
- R8101: FootprintOriginMm 105.39,158.91 -> 88.14,111.66
- R8102: BoardSide F.Cu -> B.Cu; FootprintOriginMm 109.14,117.16 -> 88.14,109.16; KiCadOrientationDeg 0 -> 180
- R8103: BoardSide B.Cu -> F.Cu; FootprintOriginMm 111.89,112.41 -> 98.64,126.41; KiCadOrientationDeg 180 -> 0
- R8104: BoardSide F.Cu -> B.Cu; FootprintOriginMm 112.14,103.66 -> 94.64,137.16; KiCadOrientationDeg 0 -> 180
- R8109: BoardSide F.Cu -> B.Cu; FootprintOriginMm 103.64,154.66 -> 87.39,129.16; KiCadOrientationDeg 0 -> 180
- R8110: FootprintOriginMm 109.14,161.41 -> 91.39,131.91
- R8111: FootprintOriginMm 105.39,117.16 -> 94.64,129.16
- R8112: FootprintOriginMm 115.89,102.91 -> 102.64,130.41
- R8113: FootprintOriginMm 115.64,111.41 -> 84.91,112.14; KiCadOrientationDeg 180 -> 90
- R8114: BoardSide B.Cu -> F.Cu; FootprintOriginMm 108.91,111.64 -> 102.41,116.14; KiCadOrientationDeg 90 -> 270
- R8119: BoardSide B.Cu -> F.Cu; FootprintOriginMm 102.41,159.64 -> 86.91,116.14; KiCadOrientationDeg 90 -> 270
- R8120: BoardSide F.Cu -> B.Cu; FootprintOriginMm 113.89,114.91 -> 87.39,131.66; KiCadOrientationDeg 0 -> 180
- R8121: BoardSide B.Cu -> F.Cu; FootprintOriginMm 105.39,161.16 -> 98.64,128.91; KiCadOrientationDeg 180 -> 0
- R8122: FootprintOriginMm 123.89,168.91 -> 84.66,112.14; KiCadOrientationDeg 0 -> 270
- R8123: FootprintOriginMm 115.14,162.66 -> 103.14,109.91
- R8124: FootprintOriginMm 117.64,114.91 -> 87.91,127.14; KiCadOrientationDeg 0 -> 270
- R8129: BoardSide F.Cu -> B.Cu; FootprintOriginMm 110.14,114.91 -> 83.91,128.89; KiCadOrientationDeg 0 -> 90
- R8130: BoardSide B.Cu -> F.Cu; FootprintOriginMm 118.89,162.66 -> 101.91,127.14; KiCadOrientationDeg 180 -> 270
- R8131: FootprintOriginMm 113.39,159.16 -> 91.41,129.89; KiCadOrientationDeg 0 -> 270
- R8132: FootprintOriginMm 112.89,98.66 -> 78.91,127.14; KiCadOrientationDeg 180 -> 90
- R8133: FootprintOriginMm 111.89,110.16 -> 91.39,134.41
- R8134: BoardSide F.Cu -> B.Cu; FootprintOriginMm 99.89,154.66 -> 105.91,129.89; KiCadOrientationDeg 0 -> 90
- R8139: BoardSide F.Cu -> B.Cu; FootprintOriginMm 106.39,114.91 -> 82.41,112.14; KiCadOrientationDeg 0 -> 90
- R8140: FootprintOriginMm 102.39,156.91 -> 101.39,111.66
- R8141: BoardSide B.Cu -> F.Cu; FootprintOriginMm 111.39,163.91 -> 87.89,111.66; KiCadOrientationDeg 180 -> 0
- R8142: FootprintOriginMm 119.64,102.91 -> 81.91,116.14; KiCadOrientationDeg 0 -> 270
- R8143: BoardSide B.Cu -> F.Cu; FootprintOriginMm 105.89,110.41 -> 104.91,116.14; KiCadOrientationDeg 180 -> 270
- R8144: BoardSide B.Cu -> F.Cu; FootprintOriginMm 115.64,109.16 -> 84.41,116.14; KiCadOrientationDeg 180 -> 270
- R8149: FootprintOriginMm 122.41,110.39 -> 88.14,106.66; KiCadOrientationDeg 90 -> 180
- R8150: FootprintOriginMm 107.64,163.66 -> 94.64,105.16
- R8151: BoardSide B.Cu -> F.Cu; FootprintOriginMm 100.16,160.89 -> 94.64,109.16; KiCadOrientationDeg 90 -> 0
- R8152: FootprintOriginMm 122.89,174.66 -> 102.64,104.91
- R8153: FootprintOriginMm 117.14,160.41 -> 94.64,131.66
- R8154: FootprintOriginMm 113.89,112.66 -> 85.41,127.14; KiCadOrientationDeg 0 -> 270
- R8155: FootprintOriginMm 119.39,109.16 -> 103.14,107.41
- R8156: FootprintOriginMm 115.14,164.91 -> 87.39,134.16
- R8157: FootprintOriginMm 101.64,111.16 -> 84.14,108.91
- R8158: BoardSide F.Cu -> B.Cu; FootprintOriginMm 117.64,112.66 -> 106.41,110.14; KiCadOrientationDeg 0 -> 90
- R8159: FootprintOriginMm 110.14,112.66 -> 98.64,131.41
- R8160: BoardSide F.Cu -> B.Cu; FootprintOriginMm 102.64,114.91 -> 81.41,128.89; KiCadOrientationDeg 0 -> 90
- R8161: FootprintOriginMm 103.89,163.41 -> 98.64,105.16
- R8162: BoardSide B.Cu -> F.Cu; FootprintOriginMm 122.64,163.91 -> 104.41,127.14; KiCadOrientationDeg 180 -> 270
- R8163: BoardSide B.Cu -> F.Cu; FootprintOriginMm 118.89,164.91 -> 88.14,130.41; KiCadOrientationDeg 180 -> 0
- R8164: FootprintOriginMm 128.39,173.16 -> 90.64,136.91
- R8165: FootprintOriginMm 109.64,166.66 -> 107.41,116.14; KiCadOrientationDeg 0 -> 270
- R8166: FootprintOriginMm 113.39,161.41 -> 98.64,109.16
- U8101: BoardSide F.Cu -> B.Cu; FootprintOriginMm 109.45,152.31 -> 94.7,110.3
- U8107: BoardSide B.Cu -> F.Cu; FootprintOriginMm 115.62,128.13 -> 94.62,114.38; KiCadOrientationDeg 180 -> 0
- U8108: FootprintOriginMm 113.97,136.45 -> 94.68,120.22; KiCadOrientationDeg 180 -> 90
- U8109: BoardSide F.Cu -> B.Cu; FootprintOriginMm 113.97,136.45 -> 83.7,120.47; KiCadOrientationDeg 0 -> 270
- U8110: FootprintOriginMm 105.2,141.47 -> 105.93,118.47; KiCadOrientationDeg 270 -> 90
- U8111: BoardSide F.Cu -> B.Cu; FootprintOriginMm 105.2,142.97 -> 98.93,131.22

Commit message: WIP: same-footprint swap pass for the core placement (#43)
Ported span-penalized slot swaps (nets over 60 mm pay a quadratic
penalty), limited to same-footprint slots within 25 mm of each package's
net median. Floorplan proxy: HPWL 139 -> 105 m, median span 28.8 mm,
RUDY p99 0.78 with 68 tiles above 0.7 (JL with swaps: p99 0.81, 42).

Co-Authored-By: Claude Opus 5.5 <noreply@anthropic.com>
Parts:
- C8101: BoardSide F.Cu -> B.Cu; FootprintOriginMm 90.64,133.21 -> 39.39,136.46; KiCadOrientationDeg 0 -> 180
- C8103: FootprintOriginMm 90.64,108.96 -> 94.64,126.46
- C8104: BoardSide B.Cu -> F.Cu; FootprintOriginMm 88.14,114.21 -> 104.71,112.14; KiCadOrientationDeg 180 -> 270
- C8105: FootprintOriginMm 83.39,132.21 -> 105.46,145.64; KiCadOrientationDeg 180 -> 90
- C8106: FootprintOriginMm 91.39,129.21 -> 101.14,112.46
- C8107: FootprintOriginMm 110.46,125.14 -> 87.14,126.46; KiCadOrientationDeg 90 -> 180
- C8108: BoardSide B.Cu -> F.Cu; FootprintOriginMm 87.14,126.46 -> 83.14,96.96; KiCadOrientationDeg 180 -> 0
- C8109: BoardSide B.Cu -> F.Cu; FootprintOriginMm 79.46,113.89 -> 90.64,133.21; KiCadOrientationDeg 90 -> 0
- C8110: BoardSide F.Cu -> B.Cu; FootprintOriginMm 94.64,126.46 -> 88.14,114.21; KiCadOrientationDeg 0 -> 180
- C8111: BoardSide F.Cu -> B.Cu; FootprintOriginMm 104.71,112.14 -> 108.46,129.89; KiCadOrientationDeg 270 -> 90
- C8112: FootprintOriginMm 101.14,112.46 -> 79.46,113.89; KiCadOrientationDeg 180 -> 90
- C8113: FootprintOriginMm 108.46,129.89 -> 110.46,125.14
- R8101: BoardSide B.Cu -> F.Cu; FootprintOriginMm 88.14,111.66 -> 84.66,112.14; KiCadOrientationDeg 180 -> 270
- R8102: FootprintOriginMm 88.14,109.16 -> 84.91,112.14; KiCadOrientationDeg 180 -> 90
- R8103: BoardSide F.Cu -> B.Cu; FootprintOriginMm 98.64,126.41 -> 89.14,102.41; KiCadOrientationDeg 0 -> 180
- R8104: FootprintOriginMm 94.64,137.16 -> 93.41,100.39; KiCadOrientationDeg 180 -> 90
- R8109: BoardSide B.Cu -> F.Cu; FootprintOriginMm 87.39,129.16 -> 102.64,130.41; KiCadOrientationDeg 180 -> 0
- R8110: FootprintOriginMm 91.39,131.91 -> 105.91,129.89; KiCadOrientationDeg 180 -> 90
- R8111: BoardSide F.Cu -> B.Cu; FootprintOriginMm 94.64,129.16 -> 86.16,180.89; KiCadOrientationDeg 0 -> 90
- R8112: FootprintOriginMm 102.64,130.41 -> 87.91,127.14; KiCadOrientationDeg 0 -> 270
- R8113: BoardSide B.Cu -> F.Cu; FootprintOriginMm 84.91,112.14 -> 98.64,109.16; KiCadOrientationDeg 90 -> 0
- R8114: FootprintOriginMm 102.41,116.14 -> 94.64,109.16; KiCadOrientationDeg 270 -> 0
- R8119: FootprintOriginMm 86.91,116.14 -> 110.66,150.39
- R8120: FootprintOriginMm 87.39,131.66 -> 105.66,149.64; KiCadOrientationDeg 180 -> 90
- R8121: BoardSide F.Cu -> B.Cu; FootprintOriginMm 98.64,128.91 -> 120.39,175.66; KiCadOrientationDeg 0 -> 180
- R8122: FootprintOriginMm 84.66,112.14 -> 101.91,127.14
- R8123: FootprintOriginMm 103.14,109.91 -> 98.64,105.16
- R8124: BoardSide F.Cu -> B.Cu; FootprintOriginMm 87.91,127.14 -> 100.89,99.41; KiCadOrientationDeg 270 -> 180
- R8129: FootprintOriginMm 83.91,128.89 -> 112.39,159.66; KiCadOrientationDeg 90 -> 180
- R8130: BoardSide F.Cu -> B.Cu; FootprintOriginMm 101.91,127.14 -> 109.16,160.39; KiCadOrientationDeg 270 -> 90
- R8131: BoardSide F.Cu -> B.Cu; FootprintOriginMm 91.41,129.89 -> 62.41,172.39; KiCadOrientationDeg 270 -> 90
- R8132: FootprintOriginMm 78.91,127.14 -> 66.66,122.14
- R8133: BoardSide B.Cu -> F.Cu; FootprintOriginMm 91.39,134.41 -> 87.14,99.41; KiCadOrientationDeg 180 -> 0
- R8134: FootprintOriginMm 105.91,129.89 -> 84.39,100.91; KiCadOrientationDeg 90 -> 180
- R8139: BoardSide B.Cu -> F.Cu; FootprintOriginMm 82.41,112.14 -> 127.91,142.39; KiCadOrientationDeg 90 -> 270
- R8140: FootprintOriginMm 101.39,111.66 -> 130.41,142.39; KiCadOrientationDeg 0 -> 270
- R8141: BoardSide F.Cu -> B.Cu; FootprintOriginMm 87.89,111.66 -> 129.41,172.89; KiCadOrientationDeg 0 -> 90
- R8142: FootprintOriginMm 81.91,116.14 -> 85.41,127.14
- R8143: FootprintOriginMm 104.91,116.14 -> 86.91,116.14
- R8149: FootprintOriginMm 88.14,106.66 -> 116.14,176.66
- R8150: BoardSide B.Cu -> F.Cu; FootprintOriginMm 94.64,105.16 -> 117.89,176.41; KiCadOrientationDeg 180 -> 0
- R8151: BoardSide F.Cu -> B.Cu; FootprintOriginMm 94.64,109.16 -> 124.39,170.41; KiCadOrientationDeg 0 -> 180
- R8152: BoardSide B.Cu -> F.Cu; FootprintOriginMm 102.64,104.91 -> 107.41,116.14; KiCadOrientationDeg 180 -> 270
- R8153: BoardSide F.Cu -> B.Cu; FootprintOriginMm 94.64,131.66 -> 84.14,108.91; KiCadOrientationDeg 0 -> 180
- R8154: BoardSide F.Cu -> B.Cu; FootprintOriginMm 85.41,127.14 -> 82.41,112.14; KiCadOrientationDeg 270 -> 90
- R8155: FootprintOriginMm 103.14,107.41 -> 104.89,95.41
- R8156: BoardSide B.Cu -> F.Cu; FootprintOriginMm 87.39,134.16 -> 95.14,97.16; KiCadOrientationDeg 180 -> 0
- R8157: FootprintOriginMm 84.14,108.91 -> 100.89,96.91
- R8158: BoardSide B.Cu -> F.Cu; FootprintOriginMm 106.41,110.14 -> 100.89,94.66; KiCadOrientationDeg 90 -> 0
- R8159: BoardSide F.Cu -> B.Cu; FootprintOriginMm 98.64,131.41 -> 104.89,92.91; KiCadOrientationDeg 0 -> 180
- R8160: BoardSide B.Cu -> F.Cu; FootprintOriginMm 81.41,128.89 -> 96.89,94.66; KiCadOrientationDeg 90 -> 0
- R8161: BoardSide B.Cu -> F.Cu; FootprintOriginMm 98.64,105.16 -> 130.66,154.39; KiCadOrientationDeg 180 -> 270
- R8162: FootprintOriginMm 104.41,127.14 -> 127.39,153.66; KiCadOrientationDeg 270 -> 0
- R8163: FootprintOriginMm 88.14,130.41 -> 106.91,196.39; KiCadOrientationDeg 0 -> 270
- R8164: BoardSide B.Cu -> F.Cu; FootprintOriginMm 90.64,136.91 -> 94.64,131.66; KiCadOrientationDeg 180 -> 0
- R8165: FootprintOriginMm 107.41,116.14 -> 98.64,131.41; KiCadOrientationDeg 270 -> 0
- R8166: FootprintOriginMm 98.64,109.16 -> 98.64,126.41
