File: boards/osc-core/sheets/mix5_M5B_K.kicad_sch (KiCad schematic)
At the start: 76 parts, among them U8201 REF5050AIDR, U8207 OPA4197IPWR, U8208 OPA4196IDR, U8209 OPA4196IDR, U8210 OPA4196IDR, U8211 OPA4196IDR

Commit message: Split jack partition into two boards with local bypass clusters
Parts:
- C8201: FootprintOriginMm 306.14,161.96 -> 223.64,162.21
- C8202: FootprintOriginMm 204.89,162.21 -> 239.39,162.21
- C8203: FootprintOriginMm 208.64,162.21 -> 256.39,162.21
- C8204: FootprintOriginMm 212.39,162.21 -> 114.89,162.46
- C8205: FootprintOriginMm 252.39,162.21 -> 174.89,162.46
- C8206: FootprintOriginMm 256.14,162.21 -> 278.89,162.46
- C8207: FootprintOriginMm 259.89,162.21 -> 32.64,162.71
- C8208: FootprintOriginMm 25.14,162.46 -> 36.39,162.71
- C8209: FootprintOriginMm 263.64,162.46 -> 40.14,162.71
- C8210: FootprintOriginMm 122.39,162.71 -> 43.89,162.71
- C8211: FootprintOriginMm 126.14,162.71 -> 47.64,162.71
- C8212: FootprintOriginMm 129.89,162.71 -> 51.39,162.71
- C8213: FootprintOriginMm 133.64,162.71 -> 58.89,162.71
- C8214: FootprintOriginMm 137.39,162.71 -> 73.64,162.71
- C8229: FootprintOriginMm 141.14,162.71 -> 88.64,162.71
- C8230: FootprintOriginMm 144.89,162.71 -> 99.89,162.71
- C8231: FootprintOriginMm 148.64,162.71 -> 103.64,162.71
- C8232: FootprintOriginMm 152.39,162.71 -> 107.39,162.71
- C8233: FootprintOriginMm 156.14,162.71 -> 111.14,162.71
- C8234: FootprintOriginMm 159.89,162.71 -> 118.64,162.71
- C8235: FootprintOriginMm 163.64,162.71 -> 159.89,162.71
- C8236: FootprintOriginMm 167.39,162.71 -> 163.64,162.71
- C8237: FootprintOriginMm 171.14,162.71 -> 167.39,162.71
- C8238: FootprintOriginMm 174.89,162.71 -> 171.14,162.71
- R8201: FootprintOriginMm 300.14,212.66 -> 28.64,210.16
- R8202: FootprintOriginMm 309.64,212.66 -> 37.64,210.16
- R8203: FootprintOriginMm 17.39,212.91 -> 41.39,210.16
- R8204: FootprintOriginMm 21.14,212.91 -> 54.39,210.16
- R8209: FootprintOriginMm 24.89,212.91 -> 71.39,210.16
- R8210: FootprintOriginMm 28.64,212.91 -> 101.64,210.16
- R8211: FootprintOriginMm 32.39,212.91 -> 142.14,210.16
- R8212: FootprintOriginMm 36.14,212.91 -> 152.39,210.16
- R8213: FootprintOriginMm 47.39,212.91 -> 159.89,210.16
- R8214: FootprintOriginMm 65.64,212.91 -> 203.39,210.16
- R8219: FootprintOriginMm 82.64,212.91 -> 207.14,210.16
- R8220: FootprintOriginMm 216.89,212.91 -> 210.89,210.16
- R8221: FootprintOriginMm 235.39,212.91 -> 214.64,210.16
- R8222: FootprintOriginMm 252.64,212.91 -> 227.89,210.16
- R8223: FootprintOriginMm 263.89,212.91 -> 231.64,210.16
- R8224: FootprintOriginMm 267.64,212.91 -> 245.14,210.16
- R8229: FootprintOriginMm 286.89,212.91 -> 248.89,210.16
- R8230: FootprintOriginMm 303.89,212.91 -> 262.14,210.16
- R8231: FootprintOriginMm 54.89,213.16 -> 265.89,210.16
- R8232: FootprintOriginMm 75.14,213.16 -> 279.39,210.16
- R8233: FootprintOriginMm 58.64,213.41 -> 298.39,210.16
- R8234: FootprintOriginMm 78.89,213.41 -> 302.14,210.16
- R8239: FootprintOriginMm 256.39,213.91 -> 6.14,210.41
- R8240: FootprintOriginMm 271.39,213.91 -> 95.89,210.41
- R8241: FootprintOriginMm 9.89,214.16 -> 112.89,210.41
- R8242: FootprintOriginMm 13.64,214.16 -> 129.89,210.41
- R8243: FootprintOriginMm 141.39,214.16 -> 145.89,210.41
- R8244: FootprintOriginMm 158.39,214.16 -> 163.64,210.41
- R8249: FootprintOriginMm 175.39,214.16 -> 182.64,210.41
- R8250: FootprintOriginMm 280.89,214.16 -> 199.64,210.41
- R8251: FootprintOriginMm 86.39,214.41 -> 292.64,210.41
- R8252: FootprintOriginMm 90.14,214.41 -> 309.64,210.41
- R8253: FootprintOriginMm 107.39,214.41 -> 17.39,210.66
- R8254: FootprintOriginMm 124.39,214.41 -> 32.39,210.66
- R8255: FootprintOriginMm 128.14,214.41 -> 50.64,210.66
- R8256: FootprintOriginMm 239.14,214.41 -> 67.64,210.66
- R8257: FootprintOriginMm 99.64,214.66 -> 84.64,210.66
- R8258: FootprintOriginMm 114.89,214.66 -> 218.39,210.66
- R8259: FootprintOriginMm 192.39,214.66 -> 235.39,210.66
- R8260: FootprintOriginMm 209.39,214.66 -> 252.64,210.66
- R8261: FootprintOriginMm 213.14,214.66 -> 269.64,210.66
- R8262: FootprintOriginMm 229.64,214.66 -> 273.39,210.66
- R8263: FootprintOriginMm 242.89,214.66 -> 283.14,210.66
- R8264: FootprintOriginMm 246.64,214.66 -> 286.89,210.66
- R8265: FootprintOriginMm 260.14,214.66 -> 305.89,210.66
- R8266: FootprintOriginMm 275.14,214.66 -> 13.64,210.91
- U8201: FootprintOriginMm 8.2,118.55 -> 79.95,118.55
- U8207: FootprintOriginMm 57.85,110.38 -> 33.1,110.38
- U8208: FootprintOriginMm 103.95,91.2 -> 137.95,91.2
- U8209: FootprintOriginMm 120.95,91.2 -> 204.95,91.2
- U8210: FootprintOriginMm 137.95,91.2 -> 222.95,91.2
- U8211: FootprintOriginMm 154.95,91.2 -> 239.95,91.2
