File: boards/osc-core/sheets/mix5_M5B_K.kicad_sch (KiCad schematic)
At the start: 76 parts, among them U8201 REF5050AIDR, U8207 OPA4197IPWR, U8208 OPA4196IDR, U8209 OPA4196IDR, U8210 OPA4196IDR, U8211 OPA4196IDR

Commit message: WIP: locality placement source for the core board (#43)
Core packages are placed by the jack locality placer, anchored on the
core GH headers and pulled toward each module's own headers; IC/bypass
clusters stay rigid. Regenerated sources follow. Draft only.

Co-Authored-By: Claude Opus 5.5 <noreply@anthropic.com>
Parts:
- C8201: BoardSide B.Cu -> F.Cu; FootprintOriginMm 223.64,162.21 -> 135.21,166.89; KiCadOrientationDeg 180 -> 270
- C8202: BoardSide B.Cu -> F.Cu; FootprintOriginMm 239.39,162.21 -> 128.39,166.96; KiCadOrientationDeg 180 -> 0
- C8203: FootprintOriginMm 256.39,162.21 -> 124.64,169.96
- C8204: BoardSide B.Cu -> F.Cu; FootprintOriginMm 114.89,162.46 -> 117.14,155.46; KiCadOrientationDeg 180 -> 0
- C8205: BoardSide B.Cu -> F.Cu; FootprintOriginMm 174.89,162.46 -> 133.96,158.64; KiCadOrientationDeg 180 -> 270
- C8206: FootprintOriginMm 278.89,162.46 -> 130.46,143.39; KiCadOrientationDeg 180 -> 90
- C8207: BoardSide B.Cu -> F.Cu; FootprintOriginMm 32.64,162.71 -> 117.14,167.21; KiCadOrientationDeg 180 -> 0
- C8208: FootprintOriginMm 36.39,162.71 -> 109.14,158.96
- C8209: FootprintOriginMm 40.14,162.71 -> 136.96,161.39; KiCadOrientationDeg 180 -> 90
- C8210: BoardSide B.Cu -> F.Cu; FootprintOriginMm 43.89,162.71 -> 113.39,156.71; KiCadOrientationDeg 180 -> 0
- C8211: FootprintOriginMm 47.64,162.71 -> 117.14,171.71
- C8212: BoardSide B.Cu -> F.Cu; FootprintOriginMm 51.39,162.71 -> 117.14,157.96; KiCadOrientationDeg 180 -> 0
- C8213: FootprintOriginMm 58.89,162.71 -> 109.64,170.71
- C8214: FootprintOriginMm 73.64,162.71 -> 132.46,157.715; KiCadOrientationDeg 180 -> 90
- C8229: FootprintOriginMm 88.64,162.71 -> 127.31,154.53; KiCadOrientationDeg 180 -> 0
- C8230: FootprintOriginMm 99.89,162.71 -> 127.31,144.21; KiCadOrientationDeg 180 -> 0
- C8231: FootprintOriginMm 103.64,162.71 -> 122.23,146.0; KiCadOrientationDeg 180 -> 90
- C8232: FootprintOriginMm 107.39,162.71 -> 112.21,146.0; KiCadOrientationDeg 180 -> 90
- C8233: BoardSide B.Cu -> F.Cu; FootprintOriginMm 111.14,162.71 -> 112.21,147.39999999999998; KiCadOrientationDeg 180 -> 270
- C8234: BoardSide B.Cu -> F.Cu; FootprintOriginMm 118.64,162.71 -> 122.23,147.39999999999998; KiCadOrientationDeg 180 -> 270
- C8235: FootprintOriginMm 159.89,162.71 -> 112.21,157.13; KiCadOrientationDeg 180 -> 270
- C8236: FootprintOriginMm 163.64,162.71 -> 122.23,157.13; KiCadOrientationDeg 180 -> 270
- C8237: FootprintOriginMm 167.39,162.71 -> 111.98,152.25; KiCadOrientationDeg 180 -> 90
- C8238: FootprintOriginMm 171.14,162.71 -> 101.96,152.25; KiCadOrientationDeg 180 -> 90
- R8201: BoardSide B.Cu -> F.Cu; FootprintOriginMm 28.64,210.16 -> 120.16,161.14; KiCadOrientationDeg 180 -> 270
- R8202: FootprintOriginMm 37.64,210.16 -> 126.39,163.16
- R8203: BoardSide B.Cu -> F.Cu; FootprintOriginMm 41.39,210.16 -> 117.14,162.66; KiCadOrientationDeg 180 -> 0
- R8204: BoardSide B.Cu -> F.Cu; FootprintOriginMm 54.39,210.16 -> 127.64,169.41; KiCadOrientationDeg 180 -> 0
- R8209: FootprintOriginMm 71.39,210.16 -> 122.64,166.16
- R8210: FootprintOriginMm 101.64,210.16 -> 111.39,166.16
- R8211: BoardSide B.Cu -> F.Cu; FootprintOriginMm 142.14,210.16 -> 129.41,157.89; KiCadOrientationDeg 180 -> 270
- R8212: BoardSide B.Cu -> F.Cu; FootprintOriginMm 152.39,210.16 -> 123.89,171.16; KiCadOrientationDeg 180 -> 0
- R8213: FootprintOriginMm 159.89,210.16 -> 117.14,167.16
- R8214: FootprintOriginMm 203.39,210.16 -> 134.91,157.64; KiCadOrientationDeg 180 -> 90
- R8219: FootprintOriginMm 207.14,210.16 -> 126.39,165.41
- R8220: FootprintOriginMm 210.89,210.16 -> 129.41,163.89; KiCadOrientationDeg 180 -> 90
- R8221: FootprintOriginMm 214.64,210.16 -> 132.41,161.39; KiCadOrientationDeg 180 -> 90
- R8222: BoardSide B.Cu -> F.Cu; FootprintOriginMm 227.89,210.16 -> 120.14,171.91; KiCadOrientationDeg 180 -> 0
- R8223: BoardSide B.Cu -> F.Cu; FootprintOriginMm 231.64,210.16 -> 113.39,163.66; KiCadOrientationDeg 180 -> 0
- R8224: FootprintOriginMm 245.14,210.16 -> 107.64,165.91
- R8229: BoardSide B.Cu -> F.Cu; FootprintOriginMm 248.89,210.16 -> 132.91,154.89; KiCadOrientationDeg 180 -> 270
- R8230: FootprintOriginMm 262.14,210.16 -> 120.89,168.41
- R8231: FootprintOriginMm 265.89,210.16 -> 113.39,168.41
- R8232: FootprintOriginMm 279.39,210.16 -> 132.14,172.66
- R8233: BoardSide B.Cu -> F.Cu; FootprintOriginMm 298.39,210.16 -> 120.89,164.41; KiCadOrientationDeg 180 -> 0
- R8234: BoardSide B.Cu -> F.Cu; FootprintOriginMm 302.14,210.16 -> 117.14,164.91; KiCadOrientationDeg 180 -> 0
- R8239: BoardSide B.Cu -> F.Cu; FootprintOriginMm 6.14,210.41 -> 131.66,158.64; KiCadOrientationDeg 180 -> 270
- R8240: FootprintOriginMm 95.89,210.41 -> 137.16,157.64; KiCadOrientationDeg 180 -> 90
- R8241: FootprintOriginMm 112.89,210.41 -> 134.66,161.39; KiCadOrientationDeg 180 -> 90
- R8242: FootprintOriginMm 129.89,210.41 -> 126.64,175.41
- R8243: FootprintOriginMm 145.89,210.41 -> 117.14,169.41
- R8244: FootprintOriginMm 163.64,210.41 -> 126.39,167.66
- R8249: FootprintOriginMm 182.64,210.41 -> 109.64,168.41
- R8250: BoardSide B.Cu -> F.Cu; FootprintOriginMm 199.64,210.41 -> 103.16,159.89; KiCadOrientationDeg 180 -> 270
- R8251: FootprintOriginMm 292.64,210.41 -> 104.66,166.39; KiCadOrientationDeg 180 -> 90
- R8252: BoardSide B.Cu -> F.Cu; FootprintOriginMm 309.64,210.41 -> 132.14,168.41; KiCadOrientationDeg 180 -> 0
- R8253: BoardSide B.Cu -> F.Cu; FootprintOriginMm 17.39,210.66 -> 129.41,161.64; KiCadOrientationDeg 180 -> 270
- R8254: BoardSide B.Cu -> F.Cu; FootprintOriginMm 32.39,210.66 -> 124.64,164.41; KiCadOrientationDeg 180 -> 0
- R8255: BoardSide B.Cu -> F.Cu; FootprintOriginMm 50.64,210.66 -> 109.64,164.41; KiCadOrientationDeg 180 -> 0
- R8256: FootprintOriginMm 67.64,210.66 -> 131.66,165.14; KiCadOrientationDeg 180 -> 90
- R8257: BoardSide B.Cu -> F.Cu; FootprintOriginMm 84.64,210.66 -> 113.39,165.91; KiCadOrientationDeg 180 -> 0
- R8258: FootprintOriginMm 218.39,210.66 -> 139.39,154.66
- R8259: BoardSide B.Cu -> F.Cu; FootprintOriginMm 235.39,210.66 -> 135.16,154.89; KiCadOrientationDeg 180 -> 270
- R8260: FootprintOriginMm 252.64,210.66 -> 100.91,164.64; KiCadOrientationDeg 180 -> 90
- R8261: FootprintOriginMm 269.64,210.66 -> 129.41,167.64; KiCadOrientationDeg 180 -> 90
- R8262: FootprintOriginMm 273.39,210.66 -> 120.89,170.66
- R8263: FootprintOriginMm 283.14,210.66 -> 113.39,170.66
- R8264: BoardSide B.Cu -> F.Cu; FootprintOriginMm 286.89,210.66 -> 118.64,174.16; KiCadOrientationDeg 180 -> 0
- R8265: BoardSide B.Cu -> F.Cu; FootprintOriginMm 305.89,210.66 -> 113.39,168.16; KiCadOrientationDeg 180 -> 0
- R8266: BoardSide B.Cu -> F.Cu; FootprintOriginMm 13.64,210.91 -> 120.89,166.66; KiCadOrientationDeg 180 -> 0
- U8201: FootprintOriginMm 79.95,118.55 -> 127.45,159.05
- U8207: FootprintOriginMm 33.1,110.38 -> 126.61,149.37; KiCadOrientationDeg 180 -> 90
- U8208: FootprintOriginMm 137.95,91.2 -> 117.22,146.7
- U8209: BoardSide B.Cu -> F.Cu; FootprintOriginMm 204.95,91.2 -> 117.22,146.7; KiCadOrientationDeg 180 -> 0
- U8210: FootprintOriginMm 222.95,91.2 -> 117.22,156.43; KiCadOrientationDeg 180 -> 0
- U8211: FootprintOriginMm 239.95,91.2 -> 106.97,152.95

Commit message: WIP: spread core module homes and legalize module by module (#43)
The first core negotiation stalled (2501/2727 nets in conflict after 7
iterations). A RUDY map showed placement congestion: header-anchored
homes crowded ~1300 E/A packages into one corner, so modules were
scattered and 751 nets spanned 80 mm or more. Module home discs are now
spread inside the outline and notch, packages are legalized one module
at a time, and the core uses a 0.6 mm courtyard gap with a 0.5 mm IC
channel. Floorplan proxy: HPWL 162 -> 139 m, peak RUDY 1.39 -> 1.09 of
ideal four-signal-layer supply, tiles above 0.7 682 -> 160.

Co-Authored-By: Claude Opus 5.5 <noreply@anthropic.com>
Parts:
- C8201: FootprintOriginMm 135.21,166.89 -> 109.14,153.71; KiCadOrientationDeg 270 -> 0
- C8202: BoardSide F.Cu -> B.Cu; FootprintOriginMm 128.39,166.96 -> 105.46,145.64; KiCadOrientationDeg 0 -> 90
- C8203: FootprintOriginMm 124.64,169.96 -> 127.39,135.96
- C8204: BoardSide F.Cu -> B.Cu; FootprintOriginMm 117.14,155.46 -> 126.71,144.89; KiCadOrientationDeg 0 -> 90
- C8205: BoardSide F.Cu -> B.Cu; FootprintOriginMm 133.96,158.64 -> 113.89,135.96; KiCadOrientationDeg 270 -> 180
- C8206: FootprintOriginMm 130.46,143.39 -> 114.14,155.71; KiCadOrientationDeg 90 -> 180
- C8207: FootprintOriginMm 117.14,167.21 -> 109.71,146.39; KiCadOrientationDeg 0 -> 270
- C8208: FootprintOriginMm 109.14,158.96 -> 113.89,143.71
- C8209: BoardSide B.Cu -> F.Cu; FootprintOriginMm 136.96,161.39 -> 131.96,146.39; KiCadOrientationDeg 90 -> 270
- C8210: BoardSide F.Cu -> B.Cu; FootprintOriginMm 113.39,156.71 -> 129.46,144.89; KiCadOrientationDeg 0 -> 90
- C8211: FootprintOriginMm 117.14,171.71 -> 132.46,160.14; KiCadOrientationDeg 180 -> 90
- C8212: FootprintOriginMm 117.14,157.96 -> 126.71,146.39; KiCadOrientationDeg 0 -> 270
- C8213: BoardSide B.Cu -> F.Cu; FootprintOriginMm 109.64,170.71 -> 119.14,161.46; KiCadOrientationDeg 180 -> 0
- C8214: FootprintOriginMm 132.46,157.715 -> 109.465,144.71; KiCadOrientationDeg 90 -> 180
- C8229: FootprintOriginMm 127.31,154.53 -> 125.78,139.43; KiCadOrientationDeg 0 -> 90
- C8230: FootprintOriginMm 127.31,144.21 -> 115.46000000000001,139.43; KiCadOrientationDeg 0 -> 90
- C8231: FootprintOriginMm 122.23,146.0 -> 125.73,149.0
- C8232: FootprintOriginMm 112.21,146.0 -> 115.71,149.0
- C8233: FootprintOriginMm 112.21,147.39999999999998 -> 115.71,150.39999999999998
- C8234: FootprintOriginMm 122.23,147.39999999999998 -> 125.73,150.39999999999998
- C8235: FootprintOriginMm 112.21,157.13 -> 115.71,161.38
- C8236: FootprintOriginMm 122.23,157.13 -> 125.73,161.38
- C8237: FootprintOriginMm 111.98,152.25 -> 126.71,153.13; KiCadOrientationDeg 90 -> 270
- C8238: FootprintOriginMm 101.96,152.25 -> 136.73,153.13; KiCadOrientationDeg 90 -> 270
- R8201: FootprintOriginMm 120.16,161.14 -> 114.91,146.39
- R8202: BoardSide B.Cu -> F.Cu; FootprintOriginMm 126.39,163.16 -> 120.64,142.66; KiCadOrientationDeg 180 -> 0
- R8203: FootprintOriginMm 117.14,162.66 -> 119.14,156.41
- R8204: BoardSide F.Cu -> B.Cu; FootprintOriginMm 127.64,169.41 -> 109.16,160.39; KiCadOrientationDeg 0 -> 90
- R8209: BoardSide B.Cu -> F.Cu; FootprintOriginMm 122.64,166.16 -> 114.91,154.39; KiCadOrientationDeg 180 -> 270
- R8210: BoardSide B.Cu -> F.Cu; FootprintOriginMm 111.39,166.16 -> 113.16,150.39; KiCadOrientationDeg 180 -> 270
- R8211: BoardSide F.Cu -> B.Cu; FootprintOriginMm 129.41,157.89 -> 129.14,141.66; KiCadOrientationDeg 270 -> 180
- R8212: BoardSide F.Cu -> B.Cu; FootprintOriginMm 123.89,171.16 -> 123.91,134.14; KiCadOrientationDeg 0 -> 90
- R8213: BoardSide B.Cu -> F.Cu; FootprintOriginMm 117.14,167.16 -> 128.41,150.39; KiCadOrientationDeg 180 -> 270
- R8214: BoardSide B.Cu -> F.Cu; FootprintOriginMm 134.91,157.64 -> 127.39,153.66; KiCadOrientationDeg 90 -> 0
- R8219: FootprintOriginMm 126.39,165.41 -> 110.91,156.39; KiCadOrientationDeg 180 -> 90
- R8220: FootprintOriginMm 129.41,163.89 -> 112.14,141.16; KiCadOrientationDeg 90 -> 180
- R8221: BoardSide B.Cu -> F.Cu; FootprintOriginMm 132.41,161.39 -> 124.64,142.66; KiCadOrientationDeg 90 -> 0
- R8222: BoardSide F.Cu -> B.Cu; FootprintOriginMm 120.14,171.91 -> 117.41,134.14; KiCadOrientationDeg 0 -> 90
- R8223: FootprintOriginMm 113.39,163.66 -> 116.64,142.66
- R8224: FootprintOriginMm 107.64,165.91 -> 132.16,144.89; KiCadOrientationDeg 180 -> 90
- R8229: FootprintOriginMm 132.91,154.89 -> 112.41,146.39
- R8230: FootprintOriginMm 120.89,168.41 -> 129.14,159.41
- R8231: FootprintOriginMm 113.39,168.41 -> 112.39,159.66
- R8232: BoardSide B.Cu -> F.Cu; FootprintOriginMm 132.14,172.66 -> 115.14,160.16; KiCadOrientationDeg 180 -> 0
- R8233: FootprintOriginMm 120.89,164.41 -> 129.41,146.39; KiCadOrientationDeg 0 -> 270
- R8234: FootprintOriginMm 117.14,164.91 -> 119.14,158.91
- R8239: FootprintOriginMm 131.66,158.64 -> 120.64,140.16; KiCadOrientationDeg 270 -> 0
- R8240: FootprintOriginMm 137.16,157.64 -> 129.14,139.16; KiCadOrientationDeg 90 -> 180
- R8241: BoardSide B.Cu -> F.Cu; FootprintOriginMm 134.66,161.39 -> 112.41,154.39; KiCadOrientationDeg 90 -> 270
- R8242: BoardSide B.Cu -> F.Cu; FootprintOriginMm 126.64,175.41 -> 120.64,137.66; KiCadOrientationDeg 180 -> 0
- R8243: BoardSide B.Cu -> F.Cu; FootprintOriginMm 117.14,169.41 -> 115.14,157.66; KiCadOrientationDeg 180 -> 0
- R8244: FootprintOriginMm 126.39,167.66 -> 112.14,138.66
- R8249: FootprintOriginMm 109.64,168.41 -> 108.41,156.39; KiCadOrientationDeg 180 -> 90
- R8250: FootprintOriginMm 103.16,159.89 -> 110.66,150.39
- R8251: BoardSide B.Cu -> F.Cu; FootprintOriginMm 104.66,166.39 -> 127.91,142.39; KiCadOrientationDeg 90 -> 270
- R8252: FootprintOriginMm 132.14,168.41 -> 130.41,142.39; KiCadOrientationDeg 0 -> 270
- R8253: FootprintOriginMm 129.41,161.64 -> 113.41,142.39
- R8254: FootprintOriginMm 124.64,164.41 -> 130.91,150.39; KiCadOrientationDeg 0 -> 270
- R8255: FootprintOriginMm 109.64,164.41 -> 124.64,140.16
- R8256: BoardSide B.Cu -> F.Cu; FootprintOriginMm 131.66,165.14 -> 116.64,140.16; KiCadOrientationDeg 90 -> 0
- R8257: BoardSide F.Cu -> B.Cu; FootprintOriginMm 113.39,165.91 -> 108.91,141.39; KiCadOrientationDeg 0 -> 90
- R8258: FootprintOriginMm 139.39,154.66 -> 132.41,140.89; KiCadOrientationDeg 180 -> 90
- R8259: BoardSide F.Cu -> B.Cu; FootprintOriginMm 135.16,154.89 -> 120.64,134.91; KiCadOrientationDeg 270 -> 180
- R8260: FootprintOriginMm 100.91,164.64 -> 134.66,144.89
- R8261: FootprintOriginMm 129.41,167.64 -> 129.14,161.91; KiCadOrientationDeg 90 -> 180
- R8262: FootprintOriginMm 120.89,170.66 -> 112.39,162.16
- R8263: FootprintOriginMm 113.39,170.66 -> 105.66,149.64; KiCadOrientationDeg 180 -> 90
- R8264: FootprintOriginMm 118.64,174.16 -> 110.91,142.39; KiCadOrientationDeg 0 -> 270
- R8265: FootprintOriginMm 113.39,168.16 -> 133.41,151.14; KiCadOrientationDeg 0 -> 270
- R8266: FootprintOriginMm 120.89,166.66 -> 130.66,154.39; KiCadOrientationDeg 0 -> 270
- U8201: FootprintOriginMm 127.45,159.05 -> 110.8,149.72; KiCadOrientationDeg 180 -> 270
- U8207: FootprintOriginMm 126.61,149.37 -> 120.62,140.13; KiCadOrientationDeg 90 -> 180
- U8208, U8209: FootprintOriginMm 117.22,146.7 -> 120.72,149.7
- U8210: FootprintOriginMm 117.22,156.43 -> 120.72,160.68
- U8211: FootprintOriginMm 106.97,152.95 -> 131.72,152.43; KiCadOrientationDeg 180 -> 0

Commit message: WIP: same-footprint swap pass for the core placement (#43)
Ported span-penalized slot swaps (nets over 60 mm pay a quadratic
penalty), limited to same-footprint slots within 25 mm of each package's
net median. Floorplan proxy: HPWL 139 -> 105 m, median span 28.8 mm,
RUDY p99 0.78 with 68 tiles above 0.7 (JL with swaps: p99 0.81, 42).

Co-Authored-By: Claude Opus 5.5 <noreply@anthropic.com>
Parts:
- C8201: BoardSide F.Cu -> B.Cu; FootprintOriginMm 109.14,153.71 -> 127.39,135.96; KiCadOrientationDeg 0 -> 180
- C8202: FootprintOriginMm 105.46,145.64 -> 126.71,144.89
- C8203: FootprintOriginMm 127.39,135.96 -> 114.14,155.71
- C8204: FootprintOriginMm 126.71,144.89 -> 113.89,143.71; KiCadOrientationDeg 90 -> 180
- C8205: FootprintOriginMm 113.89,135.96 -> 129.46,144.89; KiCadOrientationDeg 180 -> 90
- C8206: BoardSide B.Cu -> F.Cu; FootprintOriginMm 114.14,155.71 -> 109.71,146.39; KiCadOrientationDeg 180 -> 270
- C8207: FootprintOriginMm 109.71,146.39 -> 126.71,146.39
- C8208: FootprintOriginMm 113.89,143.71 -> 91.39,129.21
- C8210: FootprintOriginMm 129.46,144.89 -> 113.89,135.96; KiCadOrientationDeg 90 -> 180
- C8212: FootprintOriginMm 126.71,146.39 -> 109.14,153.71; KiCadOrientationDeg 270 -> 0
- R8201: BoardSide F.Cu -> B.Cu; FootprintOriginMm 114.91,146.39 -> 120.64,134.91; KiCadOrientationDeg 270 -> 180
- R8202: FootprintOriginMm 120.64,142.66 -> 120.64,137.66
- R8203: FootprintOriginMm 119.14,156.41 -> 104.41,127.14; KiCadOrientationDeg 0 -> 270
- R8204: FootprintOriginMm 109.16,160.39 -> 123.91,134.14
- R8209: FootprintOriginMm 114.91,154.39 -> 119.14,158.91; KiCadOrientationDeg 270 -> 0
- R8210: FootprintOriginMm 113.16,150.39 -> 119.14,156.41; KiCadOrientationDeg 270 -> 0
- R8211: FootprintOriginMm 129.14,141.66 -> 144.91,161.89; KiCadOrientationDeg 180 -> 90
- R8212: BoardSide B.Cu -> F.Cu; FootprintOriginMm 123.91,134.14 -> 114.91,146.39; KiCadOrientationDeg 90 -> 270
- R8213: FootprintOriginMm 128.41,150.39 -> 116.64,140.16; KiCadOrientationDeg 270 -> 0
- R8214: FootprintOriginMm 127.39,153.66 -> 116.64,142.66
- R8219: FootprintOriginMm 110.91,156.39 -> 132.16,144.89
- R8220: BoardSide B.Cu -> F.Cu; FootprintOriginMm 112.14,141.16 -> 129.41,146.39; KiCadOrientationDeg 180 -> 270
- R8221: BoardSide F.Cu -> B.Cu; FootprintOriginMm 124.64,142.66 -> 160.39,181.66; KiCadOrientationDeg 0 -> 180
- R8222: BoardSide B.Cu -> F.Cu; FootprintOriginMm 117.41,134.14 -> 120.64,142.66; KiCadOrientationDeg 90 -> 0
- R8223: FootprintOriginMm 116.64,142.66 -> 91.41,129.89; KiCadOrientationDeg 0 -> 270
- R8224: FootprintOriginMm 132.16,144.89 -> 91.39,131.91; KiCadOrientationDeg 90 -> 180
- R8229: FootprintOriginMm 112.41,146.39 -> 128.41,150.39
- R8230: BoardSide B.Cu -> F.Cu; FootprintOriginMm 129.14,159.41 -> 130.91,150.39; KiCadOrientationDeg 180 -> 270
- R8231: BoardSide B.Cu -> F.Cu; FootprintOriginMm 112.39,159.66 -> 133.41,151.14; KiCadOrientationDeg 180 -> 270
- R8232: FootprintOriginMm 115.14,160.16 -> 120.64,140.16
- R8233: FootprintOriginMm 129.41,146.39 -> 88.14,130.41; KiCadOrientationDeg 270 -> 0
- R8234: BoardSide F.Cu -> B.Cu; FootprintOriginMm 119.14,158.91 -> 87.39,129.16; KiCadOrientationDeg 0 -> 180
- R8239: BoardSide F.Cu -> B.Cu; FootprintOriginMm 120.64,140.16 -> 148.16,148.64; KiCadOrientationDeg 0 -> 90
- R8240: FootprintOriginMm 129.14,139.16 -> 145.66,146.89; KiCadOrientationDeg 180 -> 90
- R8241: BoardSide F.Cu -> B.Cu; FootprintOriginMm 112.41,154.39 -> 144.41,181.14; KiCadOrientationDeg 270 -> 90
- R8242: FootprintOriginMm 120.64,137.66 -> 124.64,142.66
- R8243: FootprintOriginMm 115.14,157.66 -> 102.41,116.14; KiCadOrientationDeg 0 -> 270
- R8244: BoardSide B.Cu -> F.Cu; FootprintOriginMm 112.14,138.66 -> 104.91,116.14; KiCadOrientationDeg 180 -> 270
- R8249: FootprintOriginMm 108.41,156.39 -> 147.16,185.14
- R8250: BoardSide F.Cu -> B.Cu; FootprintOriginMm 110.66,150.39 -> 144.66,185.14; KiCadOrientationDeg 270 -> 90
- R8251: BoardSide F.Cu -> B.Cu; FootprintOriginMm 127.91,142.39 -> 150.64,180.66; KiCadOrientationDeg 270 -> 180
- R8252: FootprintOriginMm 130.41,142.39 -> 115.14,160.16; KiCadOrientationDeg 270 -> 0
- R8253: BoardSide F.Cu -> B.Cu; FootprintOriginMm 113.41,142.39 -> 108.41,156.39; KiCadOrientationDeg 270 -> 90
- R8254: FootprintOriginMm 130.91,150.39 -> 114.91,154.39
- R8255: BoardSide F.Cu -> B.Cu; FootprintOriginMm 124.64,140.16 -> 102.64,104.91; KiCadOrientationDeg 0 -> 180
- R8256: BoardSide F.Cu -> B.Cu; FootprintOriginMm 116.64,140.16 -> 88.14,106.66; KiCadOrientationDeg 0 -> 180
- R8257: FootprintOriginMm 108.91,141.39 -> 88.14,109.16; KiCadOrientationDeg 90 -> 180
- R8258: FootprintOriginMm 132.41,140.89 -> 94.64,105.16; KiCadOrientationDeg 90 -> 180
- R8259: FootprintOriginMm 120.64,134.91 -> 88.14,111.66
- R8260: FootprintOriginMm 134.66,144.89 -> 103.14,107.41; KiCadOrientationDeg 90 -> 180
- R8262: FootprintOriginMm 112.39,162.16 -> 129.14,159.41
- R8263: FootprintOriginMm 105.66,149.64 -> 152.16,199.89
- R8264: BoardSide F.Cu -> B.Cu; FootprintOriginMm 110.91,142.39 -> 129.14,141.66; KiCadOrientationDeg 270 -> 180
- R8265: BoardSide F.Cu -> B.Cu; FootprintOriginMm 133.41,151.14 -> 129.14,139.16; KiCadOrientationDeg 270 -> 180
- R8266: FootprintOriginMm 130.66,154.39 -> 124.64,140.16; KiCadOrientationDeg 270 -> 0
