File: boards/osc-core/sheets/octave_reference_OCTAVE_REF_K.kicad_sch (KiCad schematic)
At the start: 30 parts, among them U1601 REF5050AIDR, U1602 OPA4197IPWR, U1603 OPA4197IPWR, U1604 OPA4197IPWR

Commit message: Split jack partition into two boards with local bypass clusters
Parts:
- C1601: FootprintOriginMm 129.89,142.71 -> 165.39,141.71
- C1602: FootprintOriginMm 133.64,142.71 -> 268.89,141.71
- C1603: FootprintOriginMm 137.39,142.71 -> 272.64,141.71
- C1604: FootprintOriginMm 141.14,142.71 -> 276.39,141.71
- C1605: FootprintOriginMm 144.89,142.71 -> 280.14,141.71
- C1606: FootprintOriginMm 148.64,142.71 -> 283.89,141.71
- C1607: FootprintOriginMm 152.39,142.71 -> 9.89,141.96
- C1608: FootprintOriginMm 156.14,142.71 -> 150.39,141.96
- C1609: FootprintOriginMm 159.89,142.71 -> 154.14,141.96
- R1601: FootprintOriginMm 105.14,179.41 -> 189.89,176.41
- R1602: FootprintOriginMm 108.89,179.41 -> 224.14,176.41
- R1603: FootprintOriginMm 112.64,179.41 -> 227.89,176.41
- R1604: FootprintOriginMm 259.39,180.16 -> 238.64,176.41
- R1605: FootprintOriginMm 263.14,180.16 -> 6.14,176.66
- R1606: FootprintOriginMm 270.64,180.16 -> 208.64,176.66
- R1607: FootprintOriginMm 274.39,180.16 -> 304.64,176.66
- R1608: FootprintOriginMm 278.14,180.16 -> 308.39,176.66
- R1609: FootprintOriginMm 287.64,180.16 -> 88.64,176.91
- R1610: FootprintOriginMm 291.39,180.16 -> 242.39,176.91
- R1611: FootprintOriginMm 9.89,180.41 -> 276.39,176.91
- R1612: FootprintOriginMm 13.64,180.41 -> 280.14,176.91
- R1613: FootprintOriginMm 137.39,180.41 -> 289.64,176.91
- R1614: FootprintOriginMm 141.14,180.41 -> 293.39,176.91
- R1615: FootprintOriginMm 144.89,180.41 -> 297.14,176.91
- R1616: FootprintOriginMm 148.64,180.41 -> 300.89,176.91
- U1601: FootprintOriginMm 31.45,112.3 -> 135.95,112.3
- U1602: FootprintOriginMm 205.1,99.38 -> 153.6,101.13
- U1603: FootprintOriginMm 222.1,99.38 -> 161.85,101.13
- U1604: FootprintOriginMm 238.6,99.38 -> 178.35,101.13
