File: boards/osc-core/sheets/octave_reference_OCTAVE_REF_K.kicad_sch (KiCad schematic)
At the start: 30 parts, among them U1601 REF5050AIDR, U1602 OPA4197IPWR, U1603 OPA4197IPWR, U1604 OPA4197IPWR

Commit message: WIP: locality placement source for the core board (#43)
Core packages are placed by the jack locality placer, anchored on the
core GH headers and pulled toward each module's own headers; IC/bypass
clusters stay rigid. Regenerated sources follow. Draft only.

Co-Authored-By: Claude Opus 5.5 <noreply@anthropic.com>
Parts:
- C1601: FootprintOriginMm 165.39,141.71 -> 16.46,170.39; KiCadOrientationDeg 180 -> 90
- C1602: FootprintOriginMm 268.89,141.71 -> 17.21,182.14; KiCadOrientationDeg 180 -> 90
- C1603: BoardSide B.Cu -> F.Cu; FootprintOriginMm 272.64,141.71 -> 23.96,164.64; KiCadOrientationDeg 180 -> 270
- C1604: BoardSide B.Cu -> F.Cu; FootprintOriginMm 276.39,141.71 -> 18.96,172.14; KiCadOrientationDeg 180 -> 270
- C1605: FootprintOriginMm 280.14,141.71 -> 17.21,166.64; KiCadOrientationDeg 180 -> 90
- C1606: BoardSide B.Cu -> F.Cu; FootprintOriginMm 283.89,141.71 -> 20.71,168.39; KiCadOrientationDeg 180 -> 270
- C1607: FootprintOriginMm 9.89,141.96 -> 11.89,181.71
- C1608: BoardSide B.Cu -> F.Cu; FootprintOriginMm 150.39,141.96 -> 16.71,175.89; KiCadOrientationDeg 180 -> 270
- C1609: FootprintOriginMm 154.14,141.96 -> 13.96,170.64; KiCadOrientationDeg 180 -> 90
- R1601: FootprintOriginMm 189.89,176.41 -> 20.66,177.89; KiCadOrientationDeg 180 -> 90
- R1602: FootprintOriginMm 224.14,176.41 -> 19.66,182.14; KiCadOrientationDeg 180 -> 90
- R1603: BoardSide B.Cu -> F.Cu; FootprintOriginMm 227.89,176.41 -> 23.41,184.89; KiCadOrientationDeg 180 -> 270
- R1604: BoardSide B.Cu -> F.Cu; FootprintOriginMm 238.64,176.41 -> 19.16,175.89; KiCadOrientationDeg 180 -> 270
- R1605: FootprintOriginMm 6.14,176.66 -> 21.16,174.14; KiCadOrientationDeg 180 -> 90
- R1606: BoardSide B.Cu -> F.Cu; FootprintOriginMm 208.64,176.66 -> 27.91,169.39; KiCadOrientationDeg 180 -> 270
- R1607: BoardSide B.Cu -> F.Cu; FootprintOriginMm 304.64,176.66 -> 23.41,177.89; KiCadOrientationDeg 180 -> 270
- R1608: BoardSide B.Cu -> F.Cu; FootprintOriginMm 308.39,176.66 -> 25.66,172.14; KiCadOrientationDeg 180 -> 270
- R1609: FootprintOriginMm 88.64,176.91 -> 23.41,168.14; KiCadOrientationDeg 180 -> 90
- R1610: FootprintOriginMm 242.39,176.91 -> 28.89,152.91
- R1611: FootprintOriginMm 276.39,176.91 -> 30.16,160.64; KiCadOrientationDeg 180 -> 90
- R1612: BoardSide B.Cu -> F.Cu; FootprintOriginMm 280.14,176.91 -> 29.39,166.41; KiCadOrientationDeg 180 -> 0
- R1613: BoardSide B.Cu -> F.Cu; FootprintOriginMm 289.64,176.91 -> 26.66,160.89; KiCadOrientationDeg 180 -> 270
- R1614: FootprintOriginMm 293.39,176.91 -> 18.41,178.39; KiCadOrientationDeg 180 -> 90
- R1615: FootprintOriginMm 297.14,176.91 -> 36.39,156.16
- R1616: FootprintOriginMm 300.89,176.91 -> 21.16,170.39; KiCadOrientationDeg 180 -> 90
- RV1601: FootprintOriginMm 239.45,21.8 -> 25.95,160.05
- U1601: FootprintOriginMm 135.95,112.3 -> 11.81,176.45; KiCadOrientationDeg 180 -> 90
- U1602: BoardSide B.Cu -> F.Cu; FootprintOriginMm 153.6,101.13 -> 30.85,174.63; KiCadOrientationDeg 180 -> 0
- U1603: FootprintOriginMm 161.85,101.13 -> 30.85,169.88
- U1604: FootprintOriginMm 178.35,101.13 -> 50.35,159.63

Commit message: WIP: spread core module homes and legalize module by module (#43)
The first core negotiation stalled (2501/2727 nets in conflict after 7
iterations). A RUDY map showed placement congestion: header-anchored
homes crowded ~1300 E/A packages into one corner, so modules were
scattered and 751 nets spanned 80 mm or more. Module home discs are now
spread inside the outline and notch, packages are legalized one module
at a time, and the core uses a 0.6 mm courtyard gap with a 0.5 mm IC
channel. Floorplan proxy: HPWL 162 -> 139 m, peak RUDY 1.39 -> 1.09 of
ideal four-signal-layer supply, tiles above 0.7 682 -> 160.

Co-Authored-By: Claude Opus 5.5 <noreply@anthropic.com>
Parts:
- C1601: FootprintOriginMm 16.46,170.39 -> 32.96,202.39
- C1602: FootprintOriginMm 17.21,182.14 -> 35.46,214.39
- C1603: FootprintOriginMm 23.96,164.64 -> 33.21,211.89
- C1604: FootprintOriginMm 18.96,172.14 -> 21.46,211.89
- C1605: FootprintOriginMm 17.21,166.64 -> 37.96,210.39
- C1606: BoardSide F.Cu -> B.Cu; FootprintOriginMm 20.71,168.39 -> 16.71,210.39; KiCadOrientationDeg 270 -> 90
- C1607: BoardSide B.Cu -> F.Cu; FootprintOriginMm 11.89,181.71 -> 25.64,203.46; KiCadOrientationDeg 180 -> 0
- C1608: BoardSide F.Cu -> B.Cu; FootprintOriginMm 16.71,175.89 -> 27.14,221.71; KiCadOrientationDeg 270 -> 180
- C1609: FootprintOriginMm 13.96,170.64 -> 16.71,214.39
- R1601: BoardSide B.Cu -> F.Cu; FootprintOriginMm 20.66,177.89 -> 27.39,211.16; KiCadOrientationDeg 90 -> 0
- R1602: FootprintOriginMm 19.66,182.14 -> 32.91,210.39
- R1603: BoardSide F.Cu -> B.Cu; FootprintOriginMm 23.41,184.89 -> 21.91,210.39; KiCadOrientationDeg 270 -> 90
- R1604: BoardSide F.Cu -> B.Cu; FootprintOriginMm 19.16,175.89 -> 19.41,214.39; KiCadOrientationDeg 270 -> 90
- R1605: BoardSide B.Cu -> F.Cu; FootprintOriginMm 21.16,174.14 -> 25.64,208.66; KiCadOrientationDeg 90 -> 0
- R1606: BoardSide F.Cu -> B.Cu; FootprintOriginMm 27.91,169.39 -> 32.91,206.39; KiCadOrientationDeg 270 -> 90
- R1607: BoardSide F.Cu -> B.Cu; FootprintOriginMm 23.41,177.89 -> 21.91,206.39; KiCadOrientationDeg 270 -> 90
- R1608: BoardSide F.Cu -> B.Cu; FootprintOriginMm 25.66,172.14 -> 32.91,214.39; KiCadOrientationDeg 270 -> 90
- R1609: FootprintOriginMm 23.41,168.14 -> 21.91,214.39
- R1610: FootprintOriginMm 28.89,152.91 -> 32.91,218.39; KiCadOrientationDeg 180 -> 90
- R1611: BoardSide B.Cu -> F.Cu; FootprintOriginMm 30.16,160.64 -> 30.66,211.89; KiCadOrientationDeg 90 -> 270
- R1612: FootprintOriginMm 29.39,166.41 -> 24.16,211.89; KiCadOrientationDeg 0 -> 270
- R1613: FootprintOriginMm 26.66,160.89 -> 22.41,207.89
- R1614: FootprintOriginMm 18.41,178.39 -> 35.41,210.39
- R1615: FootprintOriginMm 36.39,156.16 -> 19.41,210.39; KiCadOrientationDeg 180 -> 90
- R1616: BoardSide B.Cu -> F.Cu; FootprintOriginMm 21.16,170.39 -> 25.64,206.16; KiCadOrientationDeg 90 -> 0
- RV1601: BoardSide B.Cu -> F.Cu; FootprintOriginMm 25.95,160.05 -> 24.85,216.3; KiCadOrientationDeg 180 -> 0
- U1601: FootprintOriginMm 11.81,176.45 -> 19.2,201.05; KiCadOrientationDeg 90 -> 180
- U1602: BoardSide F.Cu -> B.Cu; FootprintOriginMm 30.85,174.63 -> 27.35,203.63; KiCadOrientationDeg 0 -> 180
- U1603: FootprintOriginMm 30.85,169.88 -> 27.35,210.38
- U1604: FootprintOriginMm 50.35,159.63 -> 27.35,217.13

Commit message: WIP: same-footprint swap pass for the core placement (#43)
Ported span-penalized slot swaps (nets over 60 mm pay a quadratic
penalty), limited to same-footprint slots within 25 mm of each package's
net median. Floorplan proxy: HPWL 139 -> 105 m, median span 28.8 mm,
RUDY p99 0.78 with 68 tiles above 0.7 (JL with swaps: p99 0.81, 42).

Co-Authored-By: Claude Opus 5.5 <noreply@anthropic.com>
Parts:
- C1601: FootprintOriginMm 32.96,202.39 -> 11.21,161.14
- C1602: BoardSide B.Cu -> F.Cu; FootprintOriginMm 35.46,214.39 -> 25.64,203.46; KiCadOrientationDeg 90 -> 0
- C1604: BoardSide F.Cu -> B.Cu; FootprintOriginMm 21.46,211.89 -> 81.71,193.89; KiCadOrientationDeg 270 -> 90
- C1605: FootprintOriginMm 37.96,210.39 -> 87.96,213.89
- C1607: BoardSide F.Cu -> B.Cu; FootprintOriginMm 25.64,203.46 -> 35.46,214.39; KiCadOrientationDeg 0 -> 90
- R1601: BoardSide F.Cu -> B.Cu; FootprintOriginMm 27.39,211.16 -> 35.41,210.39; KiCadOrientationDeg 0 -> 90
- R1602: FootprintOriginMm 32.91,210.39 -> 32.91,206.39
- R1603: BoardSide B.Cu -> F.Cu; FootprintOriginMm 21.91,210.39 -> 30.66,211.89; KiCadOrientationDeg 90 -> 270
- R1604: FootprintOriginMm 19.41,214.39 -> 32.91,210.39
- R1605: FootprintOriginMm 25.64,208.66 -> 27.39,211.16
- R1606: BoardSide B.Cu -> F.Cu; FootprintOriginMm 32.91,206.39 -> 25.64,208.66; KiCadOrientationDeg 90 -> 0
- R1607: BoardSide B.Cu -> F.Cu; FootprintOriginMm 21.91,206.39 -> 25.64,206.16; KiCadOrientationDeg 90 -> 0
- R1608: FootprintOriginMm 32.91,214.39 -> 21.91,206.39
- R1609: BoardSide B.Cu -> F.Cu; FootprintOriginMm 21.91,214.39 -> 24.16,211.89; KiCadOrientationDeg 90 -> 270
- R1610: FootprintOriginMm 32.91,218.39 -> 21.91,210.39
- R1611: BoardSide F.Cu -> B.Cu; FootprintOriginMm 30.66,211.89 -> 21.91,214.39; KiCadOrientationDeg 270 -> 90
- R1612: BoardSide F.Cu -> B.Cu; FootprintOriginMm 24.16,211.89 -> 44.91,189.89; KiCadOrientationDeg 270 -> 90
- R1613: BoardSide F.Cu -> B.Cu; FootprintOriginMm 22.41,207.89 -> 38.89,193.41; KiCadOrientationDeg 270 -> 180
- R1614: FootprintOriginMm 35.41,210.39 -> 32.91,218.39
- R1615: FootprintOriginMm 19.41,210.39 -> 32.91,214.39
- R1616: BoardSide F.Cu -> B.Cu; FootprintOriginMm 25.64,206.16 -> 42.16,193.14; KiCadOrientationDeg 0 -> 90
- U1602: FootprintOriginMm 27.35,203.63 -> 27.35,210.38
- U1603: FootprintOriginMm 27.35,210.38 -> 27.35,203.63
