File: boards/osc-core/sheets/offset_A02_K.kicad_sch (KiCad schematic)
At the start: 29 parts, among them U7201 REF5050AIDR, U7204 OPA4197IPWR, U7205 OPA4197IPWR

Commit message: Split jack partition into two boards with local bypass clusters
Parts:
- C7201: FootprintOriginMm 252.39,159.71 -> 114.89,159.96
- C7202: FootprintOriginMm 256.14,159.71 -> 176.14,159.96
- C7203: FootprintOriginMm 259.89,159.71 -> 280.89,159.96
- C7204: FootprintOriginMm 25.14,159.96 -> 32.64,160.21
- C7205: FootprintOriginMm 263.64,159.96 -> 36.39,160.21
- C7207: FootprintOriginMm 122.39,160.21 -> 40.14,160.21
- C7216: FootprintOriginMm 126.14,160.21 -> 43.89,160.21
- C7217: FootprintOriginMm 129.89,160.21 -> 47.64,160.21
- C7218: FootprintOriginMm 133.64,160.21 -> 51.39,160.21
- C7219: FootprintOriginMm 137.39,160.21 -> 62.39,160.21
- R7201: FootprintOriginMm 220.39,208.41 -> 205.39,205.66
- R7202: FootprintOriginMm 237.64,208.41 -> 209.14,205.66
- R7203: FootprintOriginMm 254.64,208.41 -> 212.89,205.66
- R7204: FootprintOriginMm 268.14,208.41 -> 216.64,205.66
- R7213: FootprintOriginMm 271.89,208.41 -> 230.14,205.66
- R7214: FootprintOriginMm 288.89,208.41 -> 233.89,205.66
- R7215: FootprintOriginMm 305.89,208.41 -> 247.14,205.66
- R7216: FootprintOriginMm 60.14,208.66 -> 250.89,205.66
- R7217: FootprintOriginMm 77.14,208.66 -> 264.39,205.66
- R7218: FootprintOriginMm 63.89,208.91 -> 268.14,205.66
- R7219: FootprintOriginMm 80.89,208.91 -> 281.39,205.66
- R7220: FootprintOriginMm 258.39,209.41 -> 298.39,205.66
- R7221: FootprintOriginMm 275.64,209.41 -> 302.14,205.66
- R7222: FootprintOriginMm 9.89,209.66 -> 6.14,205.91
- R7223: FootprintOriginMm 13.64,209.66 -> 97.89,205.91
- R7224: FootprintOriginMm 137.39,209.66 -> 115.89,205.91
- U7201: FootprintOriginMm 245.7,116.55 -> 48.95,116.8
- U7204: FootprintOriginMm 204.6,105.88 -> 161.35,107.63
- U7205: FootprintOriginMm 221.6,105.88 -> 178.35,107.63
