File: boards/osc-core/sheets/offset_A02_K.kicad_sch (KiCad schematic)
At the start: 29 parts, among them U7201 REF5050AIDR, U7204 OPA4197IPWR, U7205 OPA4197IPWR

Commit message: WIP: locality placement source for the core board (#43)
Core packages are placed by the jack locality placer, anchored on the
core GH headers and pulled toward each module's own headers; IC/bypass
clusters stay rigid. Regenerated sources follow. Draft only.

Co-Authored-By: Claude Opus 5.5 <noreply@anthropic.com>
Parts:
- C7201: BoardSide B.Cu -> F.Cu; FootprintOriginMm 114.89,159.96 -> 158.39,162.96; KiCadOrientationDeg 180 -> 0
- C7202: BoardSide B.Cu -> F.Cu; FootprintOriginMm 176.14,159.96 -> 163.71,163.64; KiCadOrientationDeg 180 -> 270
- C7203: FootprintOriginMm 280.89,159.96 -> 206.21,124.14; KiCadOrientationDeg 180 -> 90
- C7204: BoardSide B.Cu -> F.Cu; FootprintOriginMm 32.64,160.21 -> 206.39,126.71; KiCadOrientationDeg 180 -> 0
- C7205: FootprintOriginMm 36.39,160.21 -> 158.96,162.14; KiCadOrientationDeg 180 -> 90
- C7207: BoardSide B.Cu -> F.Cu; FootprintOriginMm 40.14,160.21 -> 173.95999999999998,161.245; KiCadOrientationDeg 180 -> 90
- C7216: FootprintOriginMm 43.89,160.21 -> 219.21,159.81; KiCadOrientationDeg 180 -> 270
- C7217: FootprintOriginMm 47.64,160.21 -> 229.53,159.81; KiCadOrientationDeg 180 -> 270
- C7218: FootprintOriginMm 51.39,160.21 -> 203.43,167.46
- C7219: FootprintOriginMm 62.39,160.21 -> 203.43,177.78
- R7201: FootprintOriginMm 205.39,205.66 -> 225.16,151.14; KiCadOrientationDeg 180 -> 90
- R7202: FootprintOriginMm 209.14,205.66 -> 221.14,163.66
- R7203: BoardSide B.Cu -> F.Cu; FootprintOriginMm 212.89,205.66 -> 223.39,154.66; KiCadOrientationDeg 180 -> 0
- R7204: BoardSide B.Cu -> F.Cu; FootprintOriginMm 216.64,205.66 -> 159.91,167.14; KiCadOrientationDeg 180 -> 270
- R7213: FootprintOriginMm 230.14,205.66 -> 223.16,133.14; KiCadOrientationDeg 180 -> 90
- R7214: FootprintOriginMm 233.89,205.66 -> 199.64,167.41
- R7215: FootprintOriginMm 247.14,205.66 -> 207.39,178.41
- R7216: FootprintOriginMm 250.89,205.66 -> 158.14,179.16
- R7217: FootprintOriginMm 264.39,205.66 -> 226.14,130.41
- R7218: BoardSide B.Cu -> F.Cu; FootprintOriginMm 268.14,205.66 -> 167.14,169.41; KiCadOrientationDeg 180 -> 0
- R7219: FootprintOriginMm 281.39,205.66 -> 199.66,170.39; KiCadOrientationDeg 180 -> 90
- R7220: BoardSide B.Cu -> F.Cu; FootprintOriginMm 298.39,205.66 -> 159.16,159.89; KiCadOrientationDeg 180 -> 270
- R7221: FootprintOriginMm 302.14,205.66 -> 161.41,162.39; KiCadOrientationDeg 180 -> 90
- R7222: BoardSide B.Cu -> F.Cu; FootprintOriginMm 6.14,205.91 -> 166.66,172.39; KiCadOrientationDeg 180 -> 270
- R7223: FootprintOriginMm 97.89,205.91 -> 223.16,129.39; KiCadOrientationDeg 180 -> 90
- R7224: FootprintOriginMm 115.89,205.91 -> 229.41,128.89; KiCadOrientationDeg 180 -> 90
- U7201: BoardSide B.Cu -> F.Cu; FootprintOriginMm 48.95,116.8 -> 168.95,161.31
- U7204: FootprintOriginMm 161.35,107.63 -> 224.37,159.11; KiCadOrientationDeg 180 -> 0
- U7205: FootprintOriginMm 178.35,107.63 -> 204.13,172.62; KiCadOrientationDeg 180 -> 270

Commit message: Place and rail-route the six-layer core draft (#43)
- Core through-hole packages (NOISE2 U6101) block both faces in the
  locality legalizer; the core POWER-* reserves are the TP load lands
  themselves and no longer emit keepouts over them.
- sync projects the netlist's representative multi-unit fields on the
  core so schematic parity is clean.
- route_jack_grid.py refuses an unclean start board, runs up to 40
  signal batches and skips empty ones.
- Synced, placed and prepared osc-core board; rail plane fanout, rail
  links and rail escapes: 7355 -> 5849 native open edges with 0 DRC
  errors and 0 parity per stage. Routed draft in progress.

Co-Authored-By: Claude Opus 5.5 <noreply@anthropic.com>
Parts:
- R7216: BoardSide B.Cu -> F.Cu; FootprintOriginMm 158.14,179.16 -> 161.39,179.41; KiCadOrientationDeg 180 -> 0
Changed lines of the file:
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@@
     (property "Island" "AO_CORE:${SHEETNAME}" (at 45.72 142.24 0) (effects (font (size 1.27 1.27)) (hide yes)))
     (property "BoardRegion" "core" (at 45.72 142.24 0) (effects (font (size 1.27 1.27)) (hide yes)))
-    (property "BoardSide" "B.Cu" (at 45.72 142.24 0) (effects (font (size 1.27 1.27)) (hide yes)))
+    (property "BoardSide" "F.Cu" (at 45.72 142.24 0) (effects (font (size 1.27 1.27)) (hide yes)))
     (property "BoardAssignment" "K" (at 45.72 142.24 0) (effects (font (size 1.27 1.27)) (hide yes)))
-    (property "KiCadOrientationDeg" "180" (at 45.72 142.24 0) (effects (font (size 1.27 1.27)) (hide yes)))
-    (property "FootprintOriginMm" "158.14,179.16" (at 45.72 142.24 0) (effects (font (size 1.27 1.27)) (hide yes)))
+    (property "KiCadOrientationDeg" "0" (at 45.72 142.24 0) (effects (font (size 1.27 1.27)) (hide yes)))
+    (property "FootprintOriginMm" "161.39,179.41" (at 45.72 142.24 0) (effects (font (size 1.27 1.27)) (hide yes)))
     (property "Sensitive" "" (at 45.72 142.24 0) (effects (font (size 1.27 1.27)) (hide yes)))
     (pin "1")

Commit message: WIP: spread core module homes and legalize module by module (#43)
The first core negotiation stalled (2501/2727 nets in conflict after 7
iterations). A RUDY map showed placement congestion: header-anchored
homes crowded ~1300 E/A packages into one corner, so modules were
scattered and 751 nets spanned 80 mm or more. Module home discs are now
spread inside the outline and notch, packages are legalized one module
at a time, and the core uses a 0.6 mm courtyard gap with a 0.5 mm IC
channel. Floorplan proxy: HPWL 162 -> 139 m, peak RUDY 1.39 -> 1.09 of
ideal four-signal-layer supply, tiles above 0.7 682 -> 160.

Co-Authored-By: Claude Opus 5.5 <noreply@anthropic.com>
Parts:
- C7201: BoardSide F.Cu -> B.Cu; FootprintOriginMm 158.39,162.96 -> 204.89,135.71; KiCadOrientationDeg 0 -> 180
- C7202: BoardSide F.Cu -> B.Cu; FootprintOriginMm 163.71,163.64 -> 208.21,137.64; KiCadOrientationDeg 270 -> 90
- C7203: BoardSide B.Cu -> F.Cu; FootprintOriginMm 206.21,124.14 -> 213.14,154.71; KiCadOrientationDeg 90 -> 0
- C7204: FootprintOriginMm 206.39,126.71 -> 193.46,180.14; KiCadOrientationDeg 0 -> 270
- C7205: BoardSide B.Cu -> F.Cu; FootprintOriginMm 158.96,162.14 -> 222.46,144.14; KiCadOrientationDeg 90 -> 270
- C7207: BoardSide F.Cu -> B.Cu; FootprintOriginMm 173.95999999999998,161.245 -> 211.16500000000002,138.14000000000001
- C7216: BoardSide B.Cu -> F.Cu; FootprintOriginMm 219.21,159.81 -> 205.46,143.07999999999998
- C7217: BoardSide B.Cu -> F.Cu; FootprintOriginMm 229.53,159.81 -> 215.78,143.07999999999998
- C7218: BoardSide B.Cu -> F.Cu; FootprintOriginMm 203.43,167.46 -> 202.96,135.32999999999998; KiCadOrientationDeg 180 -> 270
- C7219: BoardSide B.Cu -> F.Cu; FootprintOriginMm 203.43,177.78 -> 213.28,135.32999999999998; KiCadOrientationDeg 180 -> 270
- R7201: BoardSide B.Cu -> F.Cu; FootprintOriginMm 225.16,151.14 -> 208.64,168.91; KiCadOrientationDeg 90 -> 0
- R7202: BoardSide B.Cu -> F.Cu; FootprintOriginMm 221.14,163.66 -> 210.64,166.41; KiCadOrientationDeg 180 -> 0
- R7203: FootprintOriginMm 223.39,154.66 -> 205.89,171.41
- R7204: BoardSide F.Cu -> B.Cu; FootprintOriginMm 159.91,167.14 -> 185.14,188.41; KiCadOrientationDeg 270 -> 180
- R7213: BoardSide B.Cu -> F.Cu; FootprintOriginMm 223.16,133.14 -> 213.91,166.14; KiCadOrientationDeg 90 -> 270
- R7214: BoardSide B.Cu -> F.Cu; FootprintOriginMm 199.64,167.41 -> 206.64,166.41; KiCadOrientationDeg 180 -> 0
- R7215: BoardSide B.Cu -> F.Cu; FootprintOriginMm 207.39,178.41 -> 202.66,172.89; KiCadOrientationDeg 180 -> 270
- R7216: FootprintOriginMm 161.39,179.41 -> 219.14,142.41
- R7217: BoardSide B.Cu -> F.Cu; FootprintOriginMm 226.14,130.41 -> 204.91,163.14; KiCadOrientationDeg 180 -> 270
- R7218: FootprintOriginMm 167.14,169.41 -> 190.14,181.91
- R7219: BoardSide B.Cu -> F.Cu; FootprintOriginMm 199.66,170.39 -> 200.16,172.89; KiCadOrientationDeg 90 -> 270
- R7220: FootprintOriginMm 159.16,159.89 -> 239.16,179.64
- R7221: BoardSide B.Cu -> F.Cu; FootprintOriginMm 161.41,162.39 -> 235.64,179.16; KiCadOrientationDeg 90 -> 0
- R7222: FootprintOriginMm 166.66,172.39 -> 219.14,144.91; KiCadOrientationDeg 270 -> 0
- R7223: BoardSide B.Cu -> F.Cu; FootprintOriginMm 223.16,129.39 -> 200.14,176.16; KiCadOrientationDeg 90 -> 0
- R7224: FootprintOriginMm 229.41,128.89 -> 209.14,151.66; KiCadOrientationDeg 90 -> 180
- U7201: BoardSide F.Cu -> B.Cu; FootprintOriginMm 168.95,161.31 -> 211.8,143.83; KiCadOrientationDeg 180 -> 270
- U7204: BoardSide B.Cu -> F.Cu; FootprintOriginMm 224.37,159.11 -> 210.62,142.38
- U7205: BoardSide B.Cu -> F.Cu; FootprintOriginMm 204.13,172.62 -> 208.12,134.63; KiCadOrientationDeg 270 -> 0

Commit message: WIP: same-footprint swap pass for the core placement (#43)
Ported span-penalized slot swaps (nets over 60 mm pay a quadratic
penalty), limited to same-footprint slots within 25 mm of each package's
net median. Floorplan proxy: HPWL 139 -> 105 m, median span 28.8 mm,
RUDY p99 0.78 with 68 tiles above 0.7 (JL with swaps: p99 0.81, 42).

Co-Authored-By: Claude Opus 5.5 <noreply@anthropic.com>
Parts:
- C7201: FootprintOriginMm 204.89,135.71 -> 168.39,184.21
- C7204: BoardSide F.Cu -> B.Cu; FootprintOriginMm 193.46,180.14 -> 204.89,135.71; KiCadOrientationDeg 270 -> 180
- C7205: BoardSide F.Cu -> B.Cu; FootprintOriginMm 222.46,144.14 -> 206.14,178.96; KiCadOrientationDeg 270 -> 180
- R7201: FootprintOriginMm 208.64,168.91 -> 219.14,142.41
- R7202: BoardSide F.Cu -> B.Cu; FootprintOriginMm 210.64,166.41 -> 218.89,135.66; KiCadOrientationDeg 0 -> 180
- R7203: FootprintOriginMm 205.89,171.41 -> 210.64,166.41
- R7204: FootprintOriginMm 185.14,188.41 -> 210.41,165.14; KiCadOrientationDeg 180 -> 90
- R7213: BoardSide F.Cu -> B.Cu; FootprintOriginMm 213.91,166.14 -> 234.39,183.91; KiCadOrientationDeg 270 -> 180
- R7214: FootprintOriginMm 206.64,166.41 -> 232.16,185.39; KiCadOrientationDeg 0 -> 270
- R7215: FootprintOriginMm 202.66,172.89 -> 237.66,199.39
- R7216: BoardSide F.Cu -> B.Cu; FootprintOriginMm 219.14,142.41 -> 213.16,171.64; KiCadOrientationDeg 0 -> 90
- R7217: BoardSide F.Cu -> B.Cu; FootprintOriginMm 204.91,163.14 -> 205.16,139.14; KiCadOrientationDeg 270 -> 90
- R7218: BoardSide F.Cu -> B.Cu; FootprintOriginMm 190.14,181.91 -> 201.16,136.14; KiCadOrientationDeg 0 -> 90
- R7219: FootprintOriginMm 200.16,172.89 -> 212.64,210.16; KiCadOrientationDeg 270 -> 0
- R7220: BoardSide F.Cu -> B.Cu; FootprintOriginMm 239.16,179.64 -> 206.66,169.89; KiCadOrientationDeg 270 -> 90
- R7221: BoardSide F.Cu -> B.Cu; FootprintOriginMm 235.64,179.16 -> 198.66,136.14; KiCadOrientationDeg 0 -> 90
- R7222: BoardSide F.Cu -> B.Cu; FootprintOriginMm 219.14,144.91 -> 200.16,132.14; KiCadOrientationDeg 0 -> 90
- R7223: BoardSide F.Cu -> B.Cu; FootprintOriginMm 200.14,176.16 -> 210.39,108.16; KiCadOrientationDeg 0 -> 180
- R7224: FootprintOriginMm 209.14,151.66 -> 210.39,110.66
