File: boards/osc-core/sheets/oscillator_O2_K.kicad_sch (KiCad schematic)
At the start: 154 parts, among them Q1201 BCM847BS,115, U1205 AS3340D, U1206 LM393BIDR, U1207 SN74HC14DR, U1208 LM393BIDR, U1209 OPA4197IPWR, U1210 OPA4197IPWR, U1211 OPA4197IPWR, U1212 OPA4196IDR, U1213 OPA4196IDR, U1214 OPA4196IDR, U1215 OPA4196IDR

Commit message: Split jack partition into two boards with local bypass clusters
Parts:
- C1201: FootprintOriginMm 13.64,136.96 -> 233.39,136.21
- C1202: FootprintOriginMm 17.39,136.96 -> 237.14,136.21
- C1203: FootprintOriginMm 310.14,136.96 -> 262.64,136.21
- C1204: FootprintOriginMm 210.64,137.21 -> 266.39,136.21
- C1205: FootprintOriginMm 214.39,137.21 -> 270.14,136.21
- C1206: FootprintOriginMm 218.14,137.21 -> 62.39,136.71
- C1207: FootprintOriginMm 256.64,137.21 -> 72.64,136.71
- C1208: FootprintOriginMm 260.39,137.21 -> 76.39,136.71
- C1209: FootprintOriginMm 264.14,137.21 -> 84.14,136.71
- C1210: FootprintOriginMm 267.89,137.46 -> 87.89,136.71
- C1211: FootprintOriginMm 128.14,137.71 -> 91.64,136.71
- C1212: FootprintOriginMm 131.89,137.71 -> 133.89,136.71
- C1213: FootprintOriginMm 135.64,137.71 -> 137.64,136.71
- C1214: FootprintOriginMm 139.39,137.71 -> 141.39,136.71
- C1215: FootprintOriginMm 143.14,137.71 -> 145.14,136.71
- C1216: FootprintOriginMm 146.89,137.71 -> 148.89,136.71
- C1217: FootprintOriginMm 150.64,137.71 -> 167.64,136.71
- C1218: FootprintOriginMm 154.39,137.71 -> 273.89,136.71
- C1219: FootprintOriginMm 158.14,137.71 -> 277.64,136.71
- C1220: FootprintOriginMm 161.89,137.71 -> 281.39,136.71
- C1229: FootprintOriginMm 165.64,137.71 -> 285.14,136.71
- C1230: FootprintOriginMm 173.14,137.71 -> 11.14,136.96
- C1231: FootprintOriginMm 176.89,137.71 -> 152.64,136.96
- C1232: FootprintOriginMm 180.64,137.71 -> 156.39,136.96
- C1233: FootprintOriginMm 184.39,137.71 -> 160.14,136.96
- C1234: FootprintOriginMm 188.14,137.71 -> 163.89,136.96
- C1235: FootprintOriginMm 191.89,137.71 -> 292.64,136.96
- C1236: FootprintOriginMm 195.64,137.71 -> 6.14,137.21
- C1237: FootprintOriginMm 199.39,137.71 -> 14.89,137.21
- C1238: FootprintOriginMm 203.14,137.71 -> 124.14,137.46
- C1239: FootprintOriginMm 206.89,137.71 -> 39.89,137.71
- C1242: FootprintOriginMm 225.64,137.71 -> 47.39,137.71
- C1243: FootprintOriginMm 229.39,137.71 -> 51.14,137.71
- C1244: FootprintOriginMm 233.14,137.71 -> 54.89,137.71
- C1245: FootprintOriginMm 236.89,137.71 -> 58.64,137.71
- C1246: FootprintOriginMm 252.89,137.71 -> 66.14,137.71
- C1247: FootprintOriginMm 277.89,137.71 -> 80.14,137.71
- C1248: FootprintOriginMm 281.64,137.71 -> 95.39,137.71
- C1249: FootprintOriginMm 293.14,137.71 -> 109.14,137.71
- DO1205: FootprintOriginMm 29.18,126.06 -> 33.43,126.81
- R1217: FootprintOriginMm 246.14,167.41 -> 204.89,167.16
- R1218: FootprintOriginMm 268.64,167.41 -> 219.89,167.16
- R1219: FootprintOriginMm 272.39,167.41 -> 238.64,167.16
- R1220: FootprintOriginMm 6.14,167.66 -> 276.89,167.16
- R1221: FootprintOriginMm 47.64,167.66 -> 32.39,167.41
- R1222: FootprintOriginMm 51.39,167.66 -> 36.14,167.41
- R1223: FootprintOriginMm 55.14,167.66 -> 39.89,167.41
- R1224: FootprintOriginMm 58.89,167.66 -> 43.64,167.41
- R1225: FootprintOriginMm 62.64,167.66 -> 47.39,167.41
- R1226: FootprintOriginMm 66.39,167.66 -> 51.14,167.41
- R1227: FootprintOriginMm 70.14,167.66 -> 58.89,167.41
- R1228: FootprintOriginMm 73.89,167.66 -> 70.14,167.41
- R1229: FootprintOriginMm 77.64,167.66 -> 85.14,167.41
- R1230: FootprintOriginMm 85.14,167.66 -> 103.64,167.41
- R1231: FootprintOriginMm 88.89,167.66 -> 107.39,167.41
- R1232: FootprintOriginMm 92.64,167.66 -> 111.14,167.41
- R1233: FootprintOriginMm 234.89,167.66 -> 118.64,167.41
- R1234: FootprintOriginMm 238.64,167.66 -> 159.89,167.41
- R1235: FootprintOriginMm 242.39,167.66 -> 163.64,167.41
- R1236: FootprintOriginMm 308.64,167.66 -> 167.39,167.41
- R1237: FootprintOriginMm 17.39,167.91 -> 171.14,167.41
- R1238: FootprintOriginMm 21.14,167.91 -> 178.64,167.41
- R1239: FootprintOriginMm 28.64,167.91 -> 182.39,167.41
- R1240: FootprintOriginMm 32.39,167.91 -> 186.14,167.41
- R1241: FootprintOriginMm 36.14,167.91 -> 189.89,167.41
- R1242: FootprintOriginMm 39.89,167.91 -> 228.64,167.41
- R1243: FootprintOriginMm 43.64,167.91 -> 232.39,167.41
- R1244: FootprintOriginMm 96.39,168.16 -> 242.39,167.41
- R1245: FootprintOriginMm 100.14,168.16 -> 6.14,167.66
- R1246: FootprintOriginMm 103.89,168.16 -> 308.89,167.66
- R1247: FootprintOriginMm 107.64,168.16 -> 88.89,167.91
- R1248: FootprintOriginMm 111.39,168.16 -> 246.14,167.91
- R1249: FootprintOriginMm 115.14,168.16 -> 280.64,167.91
- R1250: FootprintOriginMm 264.89,168.91 -> 284.39,167.91
- R1251: FootprintOriginMm 276.14,168.91 -> 288.14,167.91
- R1252: FootprintOriginMm 279.89,168.91 -> 291.89,167.91
- R1253: FootprintOriginMm 289.89,168.91 -> 295.64,167.91
- R1254: FootprintOriginMm 293.64,168.91 -> 299.39,167.91
- R1255: FootprintOriginMm 297.39,168.91 -> 303.14,167.91
- R1256: FootprintOriginMm 9.89,169.16 -> 13.64,168.16
- R1257: FootprintOriginMm 13.64,169.16 -> 17.39,168.16
- R1258: FootprintOriginMm 205.64,169.16 -> 21.14,168.16
- R1259: FootprintOriginMm 209.39,169.16 -> 24.89,168.16
- R1260: FootprintOriginMm 249.89,169.16 -> 28.64,168.16
- R1261: FootprintOriginMm 253.64,169.16 -> 92.64,168.16
- R1262: FootprintOriginMm 257.39,169.16 -> 193.64,168.41
- R1263: FootprintOriginMm 301.14,169.16 -> 197.39,168.41
- R1264: FootprintOriginMm 304.89,169.16 -> 201.14,168.41
- R1265: FootprintOriginMm 24.89,169.41 -> 208.64,168.41
- R1266: FootprintOriginMm 201.89,169.41 -> 212.39,168.41
- R1267: FootprintOriginMm 261.14,169.41 -> 216.14,168.41
- R1268: FootprintOriginMm 118.89,169.66 -> 223.64,168.41
- R1269: FootprintOriginMm 122.64,169.66 -> 249.89,168.41
- R1270: FootprintOriginMm 126.39,169.66 -> 54.89,168.91
- R1271: FootprintOriginMm 130.14,169.66 -> 62.64,168.91
- R1272: FootprintOriginMm 133.89,169.66 -> 66.39,168.91
- R1273: FootprintOriginMm 198.14,169.66 -> 73.89,168.91
- R1274: FootprintOriginMm 213.14,169.66 -> 77.64,168.91
- R1275: FootprintOriginMm 216.89,169.66 -> 81.39,168.91
- R1276: FootprintOriginMm 220.64,169.66 -> 122.39,168.91
- R1277: FootprintOriginMm 224.39,169.66 -> 126.14,168.91
- R1278: FootprintOriginMm 228.14,169.66 -> 129.89,168.91
- R1279: FootprintOriginMm 246.14,169.66 -> 133.64,168.91
- R1280: FootprintOriginMm 268.64,169.66 -> 137.39,168.91
- R1281: FootprintOriginMm 272.39,169.66 -> 156.14,168.91
- R1282: FootprintOriginMm 283.64,169.66 -> 257.39,168.91
- R1283: FootprintOriginMm 6.14,169.91 -> 261.14,168.91
- R1284: FootprintOriginMm 47.39,169.91 -> 264.89,168.91
- R1285: FootprintOriginMm 51.14,169.91 -> 268.64,168.91
- R1286: FootprintOriginMm 54.89,169.91 -> 272.39,168.91
- R1287: FootprintOriginMm 58.64,169.91 -> 141.14,169.16
- R1288: FootprintOriginMm 62.39,169.91 -> 144.89,169.16
- R1289: FootprintOriginMm 66.14,169.91 -> 148.64,169.16
- R1290: FootprintOriginMm 69.89,169.91 -> 152.39,169.16
- R1291: FootprintOriginMm 73.64,169.91 -> 9.89,169.41
- R1292: FootprintOriginMm 77.39,169.91 -> 114.89,169.41
- R1293: FootprintOriginMm 81.14,169.91 -> 174.89,169.41
- R1294: FootprintOriginMm 84.89,169.91 -> 204.89,169.41
- R1295: FootprintOriginMm 88.64,169.91 -> 219.89,169.41
- R1296: FootprintOriginMm 92.39,169.91 -> 236.14,169.41
- R1297: FootprintOriginMm 231.89,169.91 -> 253.64,169.41
- R1298: FootprintOriginMm 235.64,169.91 -> 276.14,169.41
- R1299: FootprintOriginMm 239.39,169.91 -> 32.39,169.66
- RB1201: FootprintOriginMm 141.14,219.41 -> 43.64,215.41
- RB1210: FootprintOriginMm 144.89,219.41 -> 56.39,215.41
- RB1211: FootprintOriginMm 158.14,219.41 -> 73.14,215.41
- RB1212: FootprintOriginMm 161.89,219.41 -> 103.39,215.41
- RB1213: FootprintOriginMm 175.14,219.41 -> 118.64,215.41
- RB1214: FootprintOriginMm 294.64,219.41 -> 135.64,215.41
- RB1215: FootprintOriginMm 311.64,219.41 -> 152.64,215.41
- RB1216: FootprintOriginMm 22.64,219.66 -> 169.64,215.41
- RB1217: FootprintOriginMm 26.39,219.66 -> 186.64,215.41
- RB1218: FootprintOriginMm 30.14,219.66 -> 203.64,215.41
- RB1219: FootprintOriginMm 46.89,219.66 -> 60.14,215.66
- RB1220: FootprintOriginMm 60.14,219.66 -> 76.89,215.66
- RB1221: FootprintOriginMm 77.14,219.66 -> 173.39,215.66
- RVO1206: FootprintOriginMm 202.2,121.8 -> 193.95,121.8
- RVO1207: FootprintOriginMm 207.95,121.8 -> 199.7,121.8
- RVO1208: FootprintOriginMm 213.7,121.8 -> 205.45,121.8
- RVO1209: FootprintOriginMm 229.2,121.8 -> 211.2,121.8
- RVO1210: FootprintOriginMm 234.95,121.8 -> 227.7,121.8
- RVO1211: FootprintOriginMm 240.7,121.8 -> 250.45,121.8
- U1206: FootprintOriginMm 179.2,110.3 -> 211.2,110.3
- U1208: FootprintOriginMm 195.7,110.3 -> 263.2,110.3
- U1209: FootprintOriginMm 16.6,99.38 -> 86.6,99.38
- U1210: FootprintOriginMm 24.85,99.38 -> 103.6,99.38
- U1211: FootprintOriginMm 33.1,99.38 -> 120.1,99.38
