File: boards/osc-core/sheets/oscillator_O2_K.kicad_sch (KiCad schematic)
At the start: 154 parts, among them Q1201 BCM847BS,115, U1205 AS3340D, U1206 LM393BIDR, U1207 SN74HC14DR, U1208 LM393BIDR, U1209 OPA4197IPWR, U1210 OPA4197IPWR, U1211 OPA4197IPWR, U1212 OPA4196IDR, U1213 OPA4196IDR, U1214 OPA4196IDR, U1215 OPA4196IDR

Commit message: WIP: locality placement source for the core board (#43)
Core packages are placed by the jack locality placer, anchored on the
core GH headers and pulled toward each module's own headers; IC/bypass
clusters stay rigid. Regenerated sources follow. Draft only.

Co-Authored-By: Claude Opus 5.5 <noreply@anthropic.com>
Parts:
- C1201: BoardSide B.Cu -> F.Cu; FootprintOriginMm 233.39,136.21 -> 79.14,162.96; KiCadOrientationDeg 180 -> 0
- C1202: FootprintOriginMm 237.14,136.21 -> 72.14,157.46
- C1203: BoardSide B.Cu -> F.Cu; FootprintOriginMm 262.64,136.21 -> 68.39,161.21; KiCadOrientationDeg 180 -> 0
- C1204: FootprintOriginMm 266.39,136.21 -> 86.39,161.46
- C1205: BoardSide B.Cu -> F.Cu; FootprintOriginMm 270.14,136.21 -> 108.46,169.89; KiCadOrientationDeg 180 -> 270
- C1206: BoardSide B.Cu -> F.Cu; FootprintOriginMm 62.39,136.71 -> 44.39,152.71; KiCadOrientationDeg 180 -> 0
- C1207: FootprintOriginMm 72.64,136.71 -> 115.96,175.89; KiCadOrientationDeg 180 -> 90
- C1208: FootprintOriginMm 76.39,136.71 -> 96.89,220.71
- C1209: FootprintOriginMm 84.14,136.71 -> 80.14,157.71
- C1210: BoardSide B.Cu -> F.Cu; FootprintOriginMm 87.89,136.71 -> 112.96,177.39; KiCadOrientationDeg 180 -> 270
- C1211: FootprintOriginMm 91.64,136.71 -> 118.46,177.89; KiCadOrientationDeg 180 -> 90
- C1212: FootprintOriginMm 133.89,136.71 -> 119.14,174.71
- C1213: FootprintOriginMm 137.64,136.71 -> 90.14,163.46
- C1214: BoardSide B.Cu -> F.Cu; FootprintOriginMm 141.39,136.71 -> 89.21,167.14; KiCadOrientationDeg 180 -> 270
- C1215: FootprintOriginMm 145.14,136.71 -> 66.14,155.71
- C1216: BoardSide B.Cu -> F.Cu; FootprintOriginMm 148.89,136.71 -> 79.14,160.46; KiCadOrientationDeg 180 -> 0
- C1217: BoardSide B.Cu -> F.Cu; FootprintOriginMm 167.64,136.71 -> 82.89,161.96; KiCadOrientationDeg 180 -> 0
- C1218: BoardSide B.Cu -> F.Cu; FootprintOriginMm 273.89,136.71 -> 68.39,158.71; KiCadOrientationDeg 180 -> 0
- C1219: FootprintOriginMm 277.64,136.71 -> 62.39,155.46
- C1220: BoardSide B.Cu -> F.Cu; FootprintOriginMm 281.39,136.71 -> 91.71,167.14; KiCadOrientationDeg 180 -> 270
- C1229: BoardSide B.Cu -> F.Cu; FootprintOriginMm 285.14,136.71 -> 86.73,168.595; KiCadOrientationDeg 180 -> 270
- C1230: BoardSide B.Cu -> F.Cu; FootprintOriginMm 11.14,136.96 -> 76.71,171.135; KiCadOrientationDeg 180 -> 270
- C1231: FootprintOriginMm 152.64,136.96 -> 64.915,158.21; KiCadOrientationDeg 180 -> 0
- C1232: FootprintOriginMm 156.39,136.96 -> 74.94000000000001,159.96; KiCadOrientationDeg 180 -> 0
- C1233: FootprintOriginMm 160.14,136.96 -> 86.39,163.965; KiCadOrientationDeg 180 -> 0
- C1234: BoardSide B.Cu -> F.Cu; FootprintOriginMm 163.89,136.96 -> 66.21000000000001,175.32999999999998; KiCadOrientationDeg 180 -> 270
- C1235: BoardSide B.Cu -> F.Cu; FootprintOriginMm 292.64,136.96 -> 76.53,175.32999999999998; KiCadOrientationDeg 180 -> 270
- C1236: BoardSide B.Cu -> F.Cu; FootprintOriginMm 6.14,137.21 -> 82.53,194.16000000000003; KiCadOrientationDeg 180 -> 90
- C1237: BoardSide B.Cu -> F.Cu; FootprintOriginMm 14.89,137.21 -> 72.21000000000001,194.16000000000003; KiCadOrientationDeg 180 -> 90
- C1238: BoardSide B.Cu -> F.Cu; FootprintOriginMm 124.14,137.46 -> 76.53,167.16000000000003; KiCadOrientationDeg 180 -> 90
- C1239: BoardSide B.Cu -> F.Cu; FootprintOriginMm 39.89,137.71 -> 66.21000000000001,167.16000000000003; KiCadOrientationDeg 180 -> 90
- C1242: FootprintOriginMm 47.39,137.71 -> 81.13000000000001,188.48; KiCadOrientationDeg 180 -> 0
- C1243: FootprintOriginMm 51.14,137.71 -> 81.13000000000001,178.46; KiCadOrientationDeg 180 -> 0
- C1244: FootprintOriginMm 54.89,137.71 -> 76.48,173.5; KiCadOrientationDeg 180 -> 90
- C1245: FootprintOriginMm 58.64,137.71 -> 66.46,173.5; KiCadOrientationDeg 180 -> 90
- C1246: FootprintOriginMm 66.14,137.71 -> 73.52,184.2; KiCadOrientationDeg 180 -> 0
- C1247: FootprintOriginMm 80.14,137.71 -> 62.14,184.2
- C1248: FootprintOriginMm 95.39,137.71 -> 86.73,169.75; KiCadOrientationDeg 180 -> 90
- C1249: FootprintOriginMm 109.14,137.71 -> 76.71,169.75; KiCadOrientationDeg 180 -> 90
- DO1205: BoardSide B.Cu -> F.Cu; FootprintOriginMm 33.43,126.81 -> 79.43,157.31; KiCadOrientationDeg 180 -> 0
- Q1201: BoardSide B.Cu -> F.Cu; FootprintOriginMm 6.1,14.03 -> 83.35,165.03; KiCadOrientationDeg 180 -> 0
- R1217: BoardSide B.Cu -> F.Cu; FootprintOriginMm 204.89,167.16 -> 73.16,184.64; KiCadOrientationDeg 180 -> 270
- R1218: FootprintOriginMm 219.89,167.16 -> 71.39,190.91
- R1219: FootprintOriginMm 238.64,167.16 -> 76.89,188.66
- R1220: FootprintOriginMm 276.89,167.16 -> 113.39,172.91
- R1221: FootprintOriginMm 32.39,167.41 -> 76.66,177.64; KiCadOrientationDeg 180 -> 90
- R1222: BoardSide B.Cu -> F.Cu; FootprintOriginMm 36.14,167.41 -> 64.64,158.16; KiCadOrientationDeg 180 -> 0
- R1223: FootprintOriginMm 39.89,167.41 -> 75.14,190.91
- R1224: FootprintOriginMm 43.64,167.41 -> 71.39,193.16
- R1225: FootprintOriginMm 47.39,167.41 -> 75.14,193.16
- R1226: BoardSide B.Cu -> F.Cu; FootprintOriginMm 51.14,167.41 -> 94.41,218.14; KiCadOrientationDeg 180 -> 270
- R1227: FootprintOriginMm 58.89,167.41 -> 78.89,190.91
- R1228: FootprintOriginMm 70.14,167.41 -> 97.16,166.89; KiCadOrientationDeg 180 -> 90
- R1229: FootprintOriginMm 85.14,167.41 -> 78.89,193.16
- R1230: FootprintOriginMm 103.64,167.41 -> 96.89,223.16
- R1231: BoardSide B.Cu -> F.Cu; FootprintOriginMm 107.39,167.41 -> 69.14,192.91; KiCadOrientationDeg 180 -> 0
- R1232: BoardSide B.Cu -> F.Cu; FootprintOriginMm 111.14,167.41 -> 97.39,218.16; KiCadOrientationDeg 180 -> 0
- R1233: FootprintOriginMm 118.64,167.41 -> 84.16,177.64; KiCadOrientationDeg 180 -> 90
- R1234: FootprintOriginMm 159.89,167.41 -> 42.14,144.41
- R1235: FootprintOriginMm 163.64,167.41 -> 86.66,183.39; KiCadOrientationDeg 180 -> 90
- R1236: FootprintOriginMm 167.39,167.41 -> 94.39,225.41
- R1237: FootprintOriginMm 171.14,167.41 -> 86.66,179.64; KiCadOrientationDeg 180 -> 90
- R1238: BoardSide B.Cu -> F.Cu; FootprintOriginMm 178.64,167.41 -> 45.89,146.16; KiCadOrientationDeg 180 -> 0
- R1239: FootprintOriginMm 182.39,167.41 -> 68.16,159.14; KiCadOrientationDeg 180 -> 90
- R1240: BoardSide B.Cu -> F.Cu; FootprintOriginMm 186.14,167.41 -> 66.16,171.39; KiCadOrientationDeg 180 -> 270
- R1241: BoardSide B.Cu -> F.Cu; FootprintOriginMm 189.89,167.41 -> 61.66,157.39; KiCadOrientationDeg 180 -> 270
- R1242: BoardSide B.Cu -> F.Cu; FootprintOriginMm 228.64,167.41 -> 94.16,167.14; KiCadOrientationDeg 180 -> 270
- R1243: BoardSide B.Cu -> F.Cu; FootprintOriginMm 232.39,167.41 -> 69.14,155.16; KiCadOrientationDeg 180 -> 0
- R1244: BoardSide B.Cu -> F.Cu; FootprintOriginMm 242.39,167.41 -> 97.16,170.89; KiCadOrientationDeg 180 -> 270
- R1245: FootprintOriginMm 6.14,167.66 -> 87.14,176.66
- R1246: FootprintOriginMm 308.89,167.66 -> 88.91,184.64; KiCadOrientationDeg 180 -> 90
- R1247: FootprintOriginMm 88.89,167.91 -> 100.14,167.66
- R1248: BoardSide B.Cu -> F.Cu; FootprintOriginMm 246.14,167.91 -> 96.41,167.14; KiCadOrientationDeg 180 -> 270
- R1249: BoardSide B.Cu -> F.Cu; FootprintOriginMm 280.64,167.91 -> 55.64,155.16; KiCadOrientationDeg 180 -> 0
- R1250: BoardSide B.Cu -> F.Cu; FootprintOriginMm 284.39,167.91 -> 99.41,170.89; KiCadOrientationDeg 180 -> 270
- R1251: BoardSide B.Cu -> F.Cu; FootprintOriginMm 288.14,167.91 -> 115.41,177.89; KiCadOrientationDeg 180 -> 270
- R1252: FootprintOriginMm 291.89,167.91 -> 103.89,169.41
- R1253: BoardSide B.Cu -> F.Cu; FootprintOriginMm 295.64,167.91 -> 115.66,174.14; KiCadOrientationDeg 180 -> 270
- R1254: BoardSide B.Cu -> F.Cu; FootprintOriginMm 299.39,167.91 -> 98.66,167.14; KiCadOrientationDeg 180 -> 270
- R1255: FootprintOriginMm 303.14,167.91 -> 120.66,188.14; KiCadOrientationDeg 180 -> 90
- R1256: FootprintOriginMm 13.64,168.16 -> 86.91,173.64; KiCadOrientationDeg 180 -> 90
- R1257: FootprintOriginMm 17.39,168.16 -> 82.91,199.64; KiCadOrientationDeg 180 -> 90
- R1258: BoardSide B.Cu -> F.Cu; FootprintOriginMm 21.14,168.16 -> 102.41,172.89; KiCadOrientationDeg 180 -> 270
- R1259: BoardSide B.Cu -> F.Cu; FootprintOriginMm 24.89,168.16 -> 101.66,169.14; KiCadOrientationDeg 180 -> 270
- R1260: FootprintOriginMm 28.64,168.16 -> 39.16,145.89; KiCadOrientationDeg 180 -> 90
- R1261: BoardSide B.Cu -> F.Cu; FootprintOriginMm 92.64,168.16 -> 89.16,171.39; KiCadOrientationDeg 180 -> 270
- R1262: FootprintOriginMm 193.64,168.41 -> 89.16,173.64; KiCadOrientationDeg 180 -> 90
- R1263: BoardSide B.Cu -> F.Cu; FootprintOriginMm 197.39,168.41 -> 87.39,212.16; KiCadOrientationDeg 180 -> 0
- R1264: BoardSide B.Cu -> F.Cu; FootprintOriginMm 201.14,168.41 -> 75.14,199.41; KiCadOrientationDeg 180 -> 0
- R1265: BoardSide B.Cu -> F.Cu; FootprintOriginMm 208.64,168.41 -> 55.64,152.91; KiCadOrientationDeg 180 -> 0
- R1266: BoardSide B.Cu -> F.Cu; FootprintOriginMm 212.39,168.41 -> 51.89,154.91; KiCadOrientationDeg 180 -> 0
- R1267: BoardSide B.Cu -> F.Cu; FootprintOriginMm 216.14,168.41 -> 100.91,165.39; KiCadOrientationDeg 180 -> 270
- R1268: FootprintOriginMm 223.64,168.41 -> 91.89,184.66
- R1269: BoardSide B.Cu -> F.Cu; FootprintOriginMm 249.89,168.41 -> 104.66,172.89; KiCadOrientationDeg 180 -> 270
- R1270: FootprintOriginMm 54.89,168.91 -> 94.91,214.64; KiCadOrientationDeg 180 -> 90
- R1271: FootprintOriginMm 62.64,168.91 -> 59.89,200.91
- R1272: FootprintOriginMm 66.39,168.91 -> 90.39,227.91
- R1273: BoardSide B.Cu -> F.Cu; FootprintOriginMm 73.89,168.91 -> 106.16,177.39; KiCadOrientationDeg 180 -> 270
- R1274: BoardSide B.Cu -> F.Cu; FootprintOriginMm 77.64,168.91 -> 78.89,199.41; KiCadOrientationDeg 180 -> 0
- R1275: BoardSide B.Cu -> F.Cu; FootprintOriginMm 81.39,168.91 -> 95.14,221.16; KiCadOrientationDeg 180 -> 0
- R1276: BoardSide B.Cu -> F.Cu; FootprintOriginMm 122.39,168.91 -> 103.91,169.14; KiCadOrientationDeg 180 -> 270
- R1277: FootprintOriginMm 126.14,168.91 -> 89.16,169.89; KiCadOrientationDeg 180 -> 90
- R1278: BoardSide B.Cu -> F.Cu; FootprintOriginMm 129.89,168.91 -> 82.66,197.89; KiCadOrientationDeg 180 -> 270
- R1279: FootprintOriginMm 133.64,168.91 -> 105.39,218.16
- R1280: FootprintOriginMm 137.39,168.91 -> 49.14,150.66
- R1281: BoardSide B.Cu -> F.Cu; FootprintOriginMm 156.14,168.91 -> 86.91,173.39; KiCadOrientationDeg 180 -> 270
- R1282: BoardSide B.Cu -> F.Cu; FootprintOriginMm 257.39,168.91 -> 91.39,213.66; KiCadOrientationDeg 180 -> 0
- R1283: FootprintOriginMm 261.14,168.91 -> 120.91,181.39; KiCadOrientationDeg 180 -> 90
- R1284: BoardSide B.Cu -> F.Cu; FootprintOriginMm 264.89,168.91 -> 75.14,201.66; KiCadOrientationDeg 180 -> 0
- R1285: BoardSide B.Cu -> F.Cu; FootprintOriginMm 268.64,168.91 -> 108.39,209.41; KiCadOrientationDeg 180 -> 0
- R1286: FootprintOriginMm 272.39,168.91 -> 100.64,222.66
- R1287: BoardSide B.Cu -> F.Cu; FootprintOriginMm 141.14,169.16 -> 90.16,184.64; KiCadOrientationDeg 180 -> 270
- R1288: FootprintOriginMm 144.89,169.16 -> 83.64,202.66
- R1289: FootprintOriginMm 148.64,169.16 -> 59.89,203.16
- R1290: BoardSide B.Cu -> F.Cu; FootprintOriginMm 152.39,169.16 -> 92.14,223.41; KiCadOrientationDeg 180 -> 0
- R1291: BoardSide B.Cu -> F.Cu; FootprintOriginMm 9.89,169.41 -> 55.64,150.66; KiCadOrientationDeg 180 -> 0
- R1292: BoardSide B.Cu -> F.Cu; FootprintOriginMm 114.89,169.41 -> 116.39,171.16; KiCadOrientationDeg 180 -> 0
- R1293: FootprintOriginMm 174.89,169.41 -> 121.64,177.16
- R1294: FootprintOriginMm 204.89,169.41 -> 43.14,141.41
- R1295: BoardSide B.Cu -> F.Cu; FootprintOriginMm 219.89,169.41 -> 51.89,152.66; KiCadOrientationDeg 180 -> 0
- R1296: BoardSide B.Cu -> F.Cu; FootprintOriginMm 236.14,169.41 -> 45.89,143.91; KiCadOrientationDeg 180 -> 0
- R1297: BoardSide B.Cu -> F.Cu; FootprintOriginMm 253.64,169.41 -> 103.16,165.39; KiCadOrientationDeg 180 -> 270
- R1298: FootprintOriginMm 276.14,169.41 -> 111.41,175.89; KiCadOrientationDeg 180 -> 90
- R1299: BoardSide B.Cu -> F.Cu; FootprintOriginMm 32.39,169.66 -> 48.14,154.91; KiCadOrientationDeg 180 -> 0
- RB1201: FootprintOriginMm 43.64,215.41 -> 87.64,166.66
- RB1210: BoardSide B.Cu -> F.Cu; FootprintOriginMm 56.39,215.41 -> 63.91,165.39; KiCadOrientationDeg 180 -> 270
- RB1211: FootprintOriginMm 73.14,215.41 -> 71.14,159.91
- RB1212: BoardSide B.Cu -> F.Cu; FootprintOriginMm 103.39,215.41 -> 79.64,165.41; KiCadOrientationDeg 180 -> 0
- RB1213: BoardSide B.Cu -> F.Cu; FootprintOriginMm 118.64,215.41 -> 68.39,163.66; KiCadOrientationDeg 180 -> 0
- RB1214: BoardSide B.Cu -> F.Cu; FootprintOriginMm 135.64,215.41 -> 106.91,173.64; KiCadOrientationDeg 180 -> 270
- RB1215: BoardSide B.Cu -> F.Cu; FootprintOriginMm 152.64,215.41 -> 106.16,169.14; KiCadOrientationDeg 180 -> 270
- RB1216: BoardSide B.Cu -> F.Cu; FootprintOriginMm 169.64,215.41 -> 48.14,152.66; KiCadOrientationDeg 180 -> 0
- RB1217: FootprintOriginMm 186.64,215.41 -> 46.89,148.41
- RB1218: FootprintOriginMm 203.64,215.41 -> 113.66,175.89; KiCadOrientationDeg 180 -> 90
- RB1219: BoardSide B.Cu -> F.Cu; FootprintOriginMm 60.14,215.66 -> 49.64,150.41; KiCadOrientationDeg 180 -> 0
- RB1220: BoardSide B.Cu -> F.Cu; FootprintOriginMm 76.89,215.66 -> 109.16,173.64; KiCadOrientationDeg 180 -> 270
- RB1221: FootprintOriginMm 173.39,215.66 -> 43.14,148.91
- RVO1206: FootprintOriginMm 193.95,121.8 -> 92.95,167.05
- RVO1207: FootprintOriginMm 199.7,121.8 -> 124.7,180.55
- RVO1208: BoardSide B.Cu -> F.Cu; FootprintOriginMm 205.45,121.8 -> 121.85,177.55; KiCadOrientationDeg 180 -> 0
- RVO1209: BoardSide B.Cu -> F.Cu; FootprintOriginMm 211.2,121.8 -> 112.35,172.85; KiCadOrientationDeg 180 -> 270
- RVO1210: BoardSide B.Cu -> F.Cu; FootprintOriginMm 227.7,121.8 -> 63.85,161.55; KiCadOrientationDeg 180 -> 0
- RVO1211: BoardSide B.Cu -> F.Cu; FootprintOriginMm 250.45,121.8 -> 45.1,149.55; KiCadOrientationDeg 180 -> 0
- U1205: BoardSide B.Cu -> F.Cu; FootprintOriginMm 37.95,14.09 -> 81.72,172.34; KiCadOrientationDeg 180 -> 0
- U1206: FootprintOriginMm 211.2,110.3 -> 62.31,163.22; KiCadOrientationDeg 180 -> 90
- U1207: FootprintOriginMm 254.95,23.45 -> 70.43,164.97; KiCadOrientationDeg 180 -> 90
- U1208: FootprintOriginMm 263.2,110.3 -> 80.7,162.06; KiCadOrientationDeg 180 -> 0
- U1209: BoardSide B.Cu -> F.Cu; FootprintOriginMm 86.6,99.38 -> 71.37,174.63; KiCadOrientationDeg 180 -> 0
- U1210: BoardSide B.Cu -> F.Cu; FootprintOriginMm 103.6,99.38 -> 77.37,194.86
- U1211: BoardSide B.Cu -> F.Cu; FootprintOriginMm 120.1,99.38 -> 71.37,167.86
- U1212: FootprintOriginMm 262.7,23.45 -> 80.43,183.47; KiCadOrientationDeg 180 -> 90
- U1213: FootprintOriginMm 270.45,23.45 -> 71.47,174.2
- U1214: FootprintOriginMm 278.2,23.45 -> 67.83,184.2
- U1215: FootprintOriginMm 285.95,23.45 -> 81.72,170.45

Commit message: WIP: spread core module homes and legalize module by module (#43)
The first core negotiation stalled (2501/2727 nets in conflict after 7
iterations). A RUDY map showed placement congestion: header-anchored
homes crowded ~1300 E/A packages into one corner, so modules were
scattered and 751 nets spanned 80 mm or more. Module home discs are now
spread inside the outline and notch, packages are legalized one module
at a time, and the core uses a 0.6 mm courtyard gap with a 0.5 mm IC
channel. Floorplan proxy: HPWL 162 -> 139 m, peak RUDY 1.39 -> 1.09 of
ideal four-signal-layer supply, tiles above 0.7 682 -> 160.

Co-Authored-By: Claude Opus 5.5 <noreply@anthropic.com>
Parts:
- C1201: BoardSide F.Cu -> B.Cu; FootprintOriginMm 79.14,162.96 -> 62.64,164.96; KiCadOrientationDeg 0 -> 180
- C1202: BoardSide B.Cu -> F.Cu; FootprintOriginMm 72.14,157.46 -> 66.46,165.64; KiCadOrientationDeg 180 -> 270
- C1203: FootprintOriginMm 68.39,161.21 -> 92.71,169.14; KiCadOrientationDeg 0 -> 270
- C1204: BoardSide B.Cu -> F.Cu; FootprintOriginMm 86.39,161.46 -> 67.14,155.21; KiCadOrientationDeg 180 -> 0
- C1205: BoardSide F.Cu -> B.Cu; FootprintOriginMm 108.46,169.89 -> 59.21,165.64; KiCadOrientationDeg 270 -> 90
- C1206: FootprintOriginMm 44.39,152.71 -> 90.14,147.21
- C1207: BoardSide B.Cu -> F.Cu; FootprintOriginMm 115.96,175.89 -> 62.71,161.64; KiCadOrientationDeg 90 -> 270
- C1208: BoardSide B.Cu -> F.Cu; FootprintOriginMm 96.89,220.71 -> 93.46,150.14; KiCadOrientationDeg 180 -> 270
- C1209: FootprintOriginMm 80.14,157.71 -> 91.96,175.89; KiCadOrientationDeg 180 -> 90
- C1210: BoardSide F.Cu -> B.Cu; FootprintOriginMm 112.96,177.39 -> 76.14,139.96; KiCadOrientationDeg 270 -> 180
- C1211: FootprintOriginMm 118.46,177.89 -> 80.89,138.96; KiCadOrientationDeg 90 -> 180
- C1212: FootprintOriginMm 119.14,174.71 -> 64.71,146.39; KiCadOrientationDeg 180 -> 90
- C1213: BoardSide B.Cu -> F.Cu; FootprintOriginMm 90.14,163.46 -> 94.46,165.14; KiCadOrientationDeg 180 -> 270
- C1214: BoardSide F.Cu -> B.Cu; FootprintOriginMm 89.21,167.14 -> 98.96,164.64; KiCadOrientationDeg 270 -> 90
- C1215: BoardSide B.Cu -> F.Cu; FootprintOriginMm 66.14,155.71 -> 80.14,176.21; KiCadOrientationDeg 180 -> 0
- C1216: BoardSide F.Cu -> B.Cu; FootprintOriginMm 79.14,160.46 -> 97.89,168.21; KiCadOrientationDeg 0 -> 180
- C1217: BoardSide F.Cu -> B.Cu; FootprintOriginMm 82.89,161.96 -> 83.46,180.14; KiCadOrientationDeg 0 -> 90
- C1218: BoardSide F.Cu -> B.Cu; FootprintOriginMm 68.39,158.71 -> 88.14,144.46; KiCadOrientationDeg 0 -> 180
- C1219: FootprintOriginMm 62.39,155.46 -> 92.14,146.96
- C1220: BoardSide F.Cu -> B.Cu; FootprintOriginMm 91.71,167.14 -> 76.71,180.14; KiCadOrientationDeg 270 -> 90
- C1229: FootprintOriginMm 86.73,168.595 -> 86.73,148.845
- C1230: FootprintOriginMm 76.71,171.135 -> 76.71,151.385
- C1231: BoardSide B.Cu -> F.Cu; FootprintOriginMm 64.915,158.21 -> 72.765,172.70999999999998; KiCadOrientationDeg 0 -> 180
- C1232: FootprintOriginMm 74.94000000000001,159.96 -> 64.21,156.89000000000001; KiCadOrientationDeg 0 -> 90
- C1233: FootprintOriginMm 86.39,163.965 -> 72.665,145.71
- C1234: BoardSide F.Cu -> B.Cu; FootprintOriginMm 66.21000000000001,175.32999999999998 -> 85.53,151.18; KiCadOrientationDeg 270 -> 90
- C1235: BoardSide F.Cu -> B.Cu; FootprintOriginMm 76.53,175.32999999999998 -> 75.21000000000001,151.18; KiCadOrientationDeg 270 -> 90
- C1236: BoardSide F.Cu -> B.Cu; FootprintOriginMm 82.53,194.16000000000003 -> 86.46000000000001,155.31; KiCadOrientationDeg 90 -> 270
- C1237: BoardSide F.Cu -> B.Cu; FootprintOriginMm 72.21000000000001,194.16000000000003 -> 96.78,155.31; KiCadOrientationDeg 90 -> 270
- C1238: BoardSide F.Cu -> B.Cu; FootprintOriginMm 76.53,167.16000000000003 -> 69.42999999999999,168.21; KiCadOrientationDeg 90 -> 180
- C1239: BoardSide F.Cu -> B.Cu; FootprintOriginMm 66.21000000000001,167.16000000000003 -> 69.42999999999999,178.53; KiCadOrientationDeg 90 -> 180
- C1242: BoardSide B.Cu -> F.Cu; FootprintOriginMm 81.13000000000001,188.48 -> 76.71,165.14999999999998; KiCadOrientationDeg 0 -> 270
- C1243: BoardSide B.Cu -> F.Cu; FootprintOriginMm 81.13000000000001,178.46 -> 86.73,165.14999999999998; KiCadOrientationDeg 0 -> 270
- C1244: FootprintOriginMm 76.48,173.5 -> 75.21,173.13; KiCadOrientationDeg 90 -> 270
- C1245: FootprintOriginMm 66.46,173.5 -> 85.23,173.13; KiCadOrientationDeg 90 -> 270
- C1246: FootprintOriginMm 73.52,184.2 -> 85.23,160.75; KiCadOrientationDeg 0 -> 90
- C1247: FootprintOriginMm 62.14,184.2 -> 75.21,160.75; KiCadOrientationDeg 180 -> 90
- C1248: FootprintOriginMm 86.73,169.75 -> 86.21,164.88; KiCadOrientationDeg 90 -> 270
- C1249: FootprintOriginMm 76.71,169.75 -> 96.23,164.88; KiCadOrientationDeg 90 -> 270
- DO1205: FootprintOriginMm 79.43,157.31 -> 74.93,146.56
- Q1201: FootprintOriginMm 83.35,165.03 -> 65.86,161.6; KiCadOrientationDeg 0 -> 270
- R1217: FootprintOriginMm 73.16,184.64 -> 75.14,154.91; KiCadOrientationDeg 270 -> 0
- R1218: FootprintOriginMm 71.39,190.91 -> 87.91,171.89; KiCadOrientationDeg 180 -> 90
- R1219: BoardSide B.Cu -> F.Cu; FootprintOriginMm 76.89,188.66 -> 80.14,171.16; KiCadOrientationDeg 180 -> 0
- R1220: FootprintOriginMm 113.39,172.91 -> 64.91,176.89; KiCadOrientationDeg 180 -> 90
- R1221: BoardSide B.Cu -> F.Cu; FootprintOriginMm 76.66,177.64 -> 89.41,165.14; KiCadOrientationDeg 90 -> 270
- R1222: BoardSide F.Cu -> B.Cu; FootprintOriginMm 64.64,158.16 -> 61.66,157.64; KiCadOrientationDeg 0 -> 90
- R1223: FootprintOriginMm 75.14,190.91 -> 90.41,171.89; KiCadOrientationDeg 180 -> 90
- R1224: BoardSide B.Cu -> F.Cu; FootprintOriginMm 71.39,193.16 -> 88.39,154.91; KiCadOrientationDeg 180 -> 0
- R1225: BoardSide B.Cu -> F.Cu; FootprintOriginMm 75.14,193.16 -> 84.14,171.16; KiCadOrientationDeg 180 -> 0
- R1226: BoardSide F.Cu -> B.Cu; FootprintOriginMm 94.41,218.14 -> 95.39,177.16; KiCadOrientationDeg 270 -> 180
- R1227: BoardSide B.Cu -> F.Cu; FootprintOriginMm 78.89,190.91 -> 87.66,169.14; KiCadOrientationDeg 180 -> 270
- R1228: FootprintOriginMm 97.16,166.89 -> 64.91,172.89
- R1229: FootprintOriginMm 78.89,193.16 -> 88.89,149.66
- R1230: FootprintOriginMm 96.89,223.16 -> 59.16,157.64; KiCadOrientationDeg 180 -> 90
- R1231: BoardSide F.Cu -> B.Cu; FootprintOriginMm 69.14,192.91 -> 80.14,146.66; KiCadOrientationDeg 0 -> 180
- R1232: BoardSide F.Cu -> B.Cu; FootprintOriginMm 97.39,218.16 -> 72.14,140.66; KiCadOrientationDeg 0 -> 180
- R1233: BoardSide B.Cu -> F.Cu; FootprintOriginMm 84.16,177.64 -> 76.91,171.89; KiCadOrientationDeg 90 -> 270
- R1234: BoardSide B.Cu -> F.Cu; FootprintOriginMm 42.14,144.41 -> 63.91,155.14; KiCadOrientationDeg 180 -> 270
- R1235: BoardSide B.Cu -> F.Cu; FootprintOriginMm 86.66,183.39 -> 71.14,154.91; KiCadOrientationDeg 90 -> 0
- R1236: FootprintOriginMm 94.39,225.41 -> 95.41,146.39; KiCadOrientationDeg 180 -> 90
- R1237: BoardSide B.Cu -> F.Cu; FootprintOriginMm 86.66,179.64 -> 73.39,152.41; KiCadOrientationDeg 90 -> 0
- R1238: BoardSide F.Cu -> B.Cu; FootprintOriginMm 45.89,146.16 -> 60.16,153.64; KiCadOrientationDeg 0 -> 90
- R1239: BoardSide B.Cu -> F.Cu; FootprintOriginMm 68.16,159.14 -> 91.66,154.14; KiCadOrientationDeg 90 -> 270
- R1240: FootprintOriginMm 66.16,171.39 -> 68.91,161.14
- R1241: BoardSide F.Cu -> B.Cu; FootprintOriginMm 61.66,157.39 -> 62.41,168.39; KiCadOrientationDeg 270 -> 90
- R1242: FootprintOriginMm 94.16,167.14 -> 89.91,173.14
- R1243: BoardSide F.Cu -> B.Cu; FootprintOriginMm 69.14,155.16 -> 76.14,142.66; KiCadOrientationDeg 0 -> 180
- R1244: FootprintOriginMm 97.16,170.89 -> 90.14,149.91; KiCadOrientationDeg 270 -> 0
- R1245: FootprintOriginMm 87.14,176.66 -> 84.14,146.66
- R1246: FootprintOriginMm 88.91,184.64 -> 76.91,145.89
- R1247: FootprintOriginMm 100.14,167.66 -> 60.91,161.64; KiCadOrientationDeg 180 -> 90
- R1248: FootprintOriginMm 96.41,167.14 -> 95.41,161.14
- R1249: FootprintOriginMm 55.64,155.16 -> 84.14,176.16
- R1250: BoardSide F.Cu -> B.Cu; FootprintOriginMm 99.41,170.89 -> 99.66,160.64; KiCadOrientationDeg 270 -> 90
- R1251: FootprintOriginMm 115.41,177.89 -> 88.14,144.66; KiCadOrientationDeg 270 -> 0
- R1252: FootprintOriginMm 103.89,169.41 -> 62.66,152.89; KiCadOrientationDeg 180 -> 90
- R1253: FootprintOriginMm 115.66,174.14 -> 76.14,143.16; KiCadOrientationDeg 270 -> 0
- R1254: BoardSide F.Cu -> B.Cu; FootprintOriginMm 98.66,167.14 -> 64.39,149.66; KiCadOrientationDeg 270 -> 180
- R1255: BoardSide B.Cu -> F.Cu; FootprintOriginMm 120.66,188.14 -> 80.14,142.41; KiCadOrientationDeg 90 -> 0
- R1256: FootprintOriginMm 86.91,173.64 -> 88.64,175.16; KiCadOrientationDeg 90 -> 180
- R1257: BoardSide B.Cu -> F.Cu; FootprintOriginMm 82.91,199.64 -> 88.39,152.41; KiCadOrientationDeg 90 -> 0
- R1258: FootprintOriginMm 102.41,172.89 -> 66.66,169.64
- R1259: BoardSide F.Cu -> B.Cu; FootprintOriginMm 101.66,169.14 -> 80.14,141.66; KiCadOrientationDeg 270 -> 180
- R1260: FootprintOriginMm 39.16,145.89 -> 101.66,164.64
- R1261: BoardSide F.Cu -> B.Cu; FootprintOriginMm 89.16,171.39 -> 80.14,179.41; KiCadOrientationDeg 270 -> 180
- R1262: BoardSide B.Cu -> F.Cu; FootprintOriginMm 89.16,173.64 -> 80.14,173.66; KiCadOrientationDeg 90 -> 0
- R1263: FootprintOriginMm 87.39,212.16 -> 76.14,175.41
- R1264: FootprintOriginMm 75.14,199.41 -> 91.91,165.14; KiCadOrientationDeg 0 -> 270
- R1265: FootprintOriginMm 55.64,152.91 -> 94.16,154.14; KiCadOrientationDeg 0 -> 270
- R1266: BoardSide F.Cu -> B.Cu; FootprintOriginMm 51.89,154.91 -> 99.41,156.64; KiCadOrientationDeg 0 -> 90
- R1267: BoardSide F.Cu -> B.Cu; FootprintOriginMm 100.91,165.39 -> 72.14,143.16; KiCadOrientationDeg 270 -> 180
- R1268: FootprintOriginMm 91.89,184.66 -> 88.14,147.16
- R1269: FootprintOriginMm 104.66,172.89 -> 72.14,175.41; KiCadOrientationDeg 270 -> 0
- R1270: FootprintOriginMm 94.91,214.64 -> 84.14,141.66; KiCadOrientationDeg 90 -> 180
- R1271: FootprintOriginMm 59.89,200.91 -> 92.91,171.89; KiCadOrientationDeg 180 -> 90
- R1272: FootprintOriginMm 90.39,227.91 -> 58.41,161.64; KiCadOrientationDeg 180 -> 90
- R1273: BoardSide F.Cu -> B.Cu; FootprintOriginMm 106.16,177.39 -> 86.16,180.89; KiCadOrientationDeg 270 -> 90
- R1274: FootprintOriginMm 78.89,199.41 -> 68.14,157.91
- R1275: FootprintOriginMm 95.14,221.16 -> 96.66,154.64; KiCadOrientationDeg 0 -> 270
- R1276: FootprintOriginMm 103.91,169.14 -> 64.14,158.41; KiCadOrientationDeg 270 -> 0
- R1277: BoardSide B.Cu -> F.Cu; FootprintOriginMm 89.16,169.89 -> 90.16,169.14; KiCadOrientationDeg 90 -> 270
- R1278: BoardSide F.Cu -> B.Cu; FootprintOriginMm 82.66,197.89 -> 63.41,161.64; KiCadOrientationDeg 270 -> 90
- R1279: FootprintOriginMm 105.39,218.16 -> 59.91,169.64; KiCadOrientationDeg 180 -> 90
- R1280: BoardSide B.Cu -> F.Cu; FootprintOriginMm 49.14,150.66 -> 96.14,157.91; KiCadOrientationDeg 180 -> 0
- R1281: BoardSide F.Cu -> B.Cu; FootprintOriginMm 86.91,173.39 -> 64.91,168.89; KiCadOrientationDeg 270 -> 90
- R1282: BoardSide F.Cu -> B.Cu; FootprintOriginMm 91.39,213.66 -> 68.14,144.91; KiCadOrientationDeg 0 -> 180
- R1283: FootprintOriginMm 120.91,181.39 -> 68.14,142.41; KiCadOrientationDeg 90 -> 180
- R1284: FootprintOriginMm 75.14,201.66 -> 84.14,173.66
- R1285: FootprintOriginMm 108.39,209.41 -> 64.16,169.64; KiCadOrientationDeg 0 -> 270
- R1286: FootprintOriginMm 100.64,222.66 -> 100.16,152.64; KiCadOrientationDeg 180 -> 90
- R1287: BoardSide F.Cu -> B.Cu; FootprintOriginMm 90.16,184.64 -> 97.16,160.64; KiCadOrientationDeg 270 -> 90
- R1288: FootprintOriginMm 83.64,202.66 -> 80.14,144.16
- R1289: BoardSide B.Cu -> F.Cu; FootprintOriginMm 59.89,203.16 -> 73.39,149.91; KiCadOrientationDeg 180 -> 0
- R1290: BoardSide F.Cu -> B.Cu; FootprintOriginMm 92.14,223.41 -> 102.16,160.64; KiCadOrientationDeg 0 -> 90
- R1291: BoardSide F.Cu -> B.Cu; FootprintOriginMm 55.64,150.66 -> 97.66,151.14; KiCadOrientationDeg 0 -> 90
- R1292: FootprintOriginMm 116.39,171.16 -> 61.41,165.64; KiCadOrientationDeg 0 -> 270
- R1293: FootprintOriginMm 121.64,177.16 -> 101.16,168.64; KiCadOrientationDeg 180 -> 90
- R1294: FootprintOriginMm 43.14,141.41 -> 69.64,181.16
- R1295: BoardSide F.Cu -> B.Cu; FootprintOriginMm 51.89,152.66 -> 80.14,181.91; KiCadOrientationDeg 0 -> 180
- R1296: FootprintOriginMm 45.89,143.91 -> 66.41,173.64; KiCadOrientationDeg 0 -> 270
- R1297: FootprintOriginMm 103.16,165.39 -> 80.14,144.91; KiCadOrientationDeg 270 -> 0
- R1298: BoardSide B.Cu -> F.Cu; FootprintOriginMm 111.41,175.89 -> 63.91,165.64; KiCadOrientationDeg 90 -> 270
- R1299: BoardSide F.Cu -> B.Cu; FootprintOriginMm 48.14,154.91 -> 62.41,172.39; KiCadOrientationDeg 0 -> 90
- RB1201: FootprintOriginMm 87.64,166.66 -> 92.89,149.66
- RB1210: BoardSide F.Cu -> B.Cu; FootprintOriginMm 63.91,165.39 -> 65.16,152.89; KiCadOrientationDeg 270 -> 90
- RB1211: BoardSide B.Cu -> F.Cu; FootprintOriginMm 71.14,159.91 -> 87.41,173.14; KiCadOrientationDeg 180 -> 270
- RB1212: BoardSide F.Cu -> B.Cu; FootprintOriginMm 79.64,165.41 -> 86.89,177.66; KiCadOrientationDeg 0 -> 180
- RB1213: BoardSide F.Cu -> B.Cu; FootprintOriginMm 68.39,163.66 -> 84.14,144.16; KiCadOrientationDeg 0 -> 180
- RB1214: FootprintOriginMm 106.91,173.64 -> 92.41,173.14
- RB1215: BoardSide F.Cu -> B.Cu; FootprintOriginMm 106.16,169.14 -> 92.14,144.41; KiCadOrientationDeg 270 -> 180
- RB1216: FootprintOriginMm 48.14,152.66 -> 68.91,174.14; KiCadOrientationDeg 0 -> 270
- RB1217: BoardSide B.Cu -> F.Cu; FootprintOriginMm 46.89,148.41 -> 70.64,147.41; KiCadOrientationDeg 180 -> 0
- RB1218: BoardSide B.Cu -> F.Cu; FootprintOriginMm 113.66,175.89 -> 84.14,144.91; KiCadOrientationDeg 90 -> 0
- RB1219: FootprintOriginMm 49.64,150.41 -> 95.41,169.14; KiCadOrientationDeg 0 -> 270
- RB1220: FootprintOriginMm 109.16,173.64 -> 88.14,176.41; KiCadOrientationDeg 270 -> 0
- RB1221: FootprintOriginMm 43.14,148.91 -> 76.14,183.91
- RVO1206: BoardSide B.Cu -> F.Cu; FootprintOriginMm 92.95,167.05 -> 68.6,151.55; KiCadOrientationDeg 180 -> 0
- RVO1207: FootprintOriginMm 124.7,180.55 -> 103.6,155.45; KiCadOrientationDeg 180 -> 90
- RVO1208: FootprintOriginMm 121.85,177.55 -> 63.1,150.35; KiCadOrientationDeg 0 -> 270
- RVO1209: BoardSide F.Cu -> B.Cu; FootprintOriginMm 112.35,172.85 -> 88.95,141.05; KiCadOrientationDeg 270 -> 180
- RVO1210: BoardSide F.Cu -> B.Cu; FootprintOriginMm 63.85,161.55 -> 96.35,172.7; KiCadOrientationDeg 0 -> 90
- RVO1211: FootprintOriginMm 45.1,149.55 -> 98.85,162.35; KiCadOrientationDeg 0 -> 270
- U1205: FootprintOriginMm 81.72,172.34 -> 81.72,152.59
- U1206: BoardSide B.Cu -> F.Cu; FootprintOriginMm 62.31,163.22 -> 71.56,167.7; KiCadOrientationDeg 90 -> 270
- U1207: FootprintOriginMm 70.43,164.97 -> 69.22,161.4; KiCadOrientationDeg 90 -> 180
- U1208: FootprintOriginMm 80.7,162.06 -> 70.06,150.72; KiCadOrientationDeg 0 -> 90
- U1209: BoardSide F.Cu -> B.Cu; FootprintOriginMm 71.37,174.63 -> 80.37,151.88; KiCadOrientationDeg 0 -> 180
- U1210: BoardSide F.Cu -> B.Cu; FootprintOriginMm 77.37,194.86 -> 91.62,154.61; KiCadOrientationDeg 180 -> 0
- U1211: BoardSide F.Cu -> B.Cu; FootprintOriginMm 71.37,167.86 -> 70.13,173.37; KiCadOrientationDeg 180 -> 270
- U1212: BoardSide B.Cu -> F.Cu; FootprintOriginMm 80.43,183.47 -> 81.72,164.45; KiCadOrientationDeg 90 -> 0
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
Commit message: WIP: same-footprint swap pass for the core placement (#43)
Ported span-penalized slot swaps (nets over 60 mm pay a quadratic
penalty), limited to same-footprint slots within 25 mm of each package's
net median. Floorplan proxy: HPWL 139 -> 105 m, median span 28.8 mm,
RUDY p99 0.78 with 68 tiles above 0.7 (JL with swaps: p99 0.81, 42).

Co-Authored-By: Claude Opus 5.5 <noreply@anthropic.com>
Parts:
- C1202: BoardSide F.Cu -> B.Cu; FootprintOriginMm 66.46,165.64 -> 98.96,164.64; KiCadOrientationDeg 270 -> 90
- C1203: FootprintOriginMm 92.71,169.14 -> 66.46,165.64
- C1204: BoardSide F.Cu -> B.Cu; FootprintOriginMm 67.14,155.21 -> 83.39,132.21; KiCadOrientationDeg 0 -> 180
- C1206: FootprintOriginMm 90.14,147.21 -> 62.71,161.64; KiCadOrientationDeg 0 -> 270
- C1207: BoardSide F.Cu -> B.Cu; FootprintOriginMm 62.71,161.64 -> 76.71,180.14; KiCadOrientationDeg 270 -> 90
- C1208: BoardSide F.Cu -> B.Cu; FootprintOriginMm 93.46,150.14 -> 97.89,168.21; KiCadOrientationDeg 270 -> 180
- C1209: FootprintOriginMm 91.96,175.89 -> 88.14,144.46; KiCadOrientationDeg 90 -> 180
- C1213: BoardSide F.Cu -> B.Cu; FootprintOriginMm 94.46,165.14 -> 83.46,180.14; KiCadOrientationDeg 270 -> 90
- C1214: BoardSide B.Cu -> F.Cu; FootprintOriginMm 98.96,164.64 -> 67.14,155.21; KiCadOrientationDeg 90 -> 0
- C1215: FootprintOriginMm 80.14,176.21 -> 93.46,150.14; KiCadOrientationDeg 0 -> 270
- C1216: BoardSide B.Cu -> F.Cu; FootprintOriginMm 97.89,168.21 -> 92.71,169.14; KiCadOrientationDeg 180 -> 270
- C1217: FootprintOriginMm 83.46,180.14 -> 92.14,146.96; KiCadOrientationDeg 90 -> 180
- C1218: BoardSide B.Cu -> F.Cu; FootprintOriginMm 88.14,144.46 -> 90.14,147.21; KiCadOrientationDeg 180 -> 0
- C1219: FootprintOriginMm 92.14,146.96 -> 91.96,175.89; KiCadOrientationDeg 180 -> 90
- C1220: BoardSide B.Cu -> F.Cu; FootprintOriginMm 76.71,180.14 -> 80.14,176.21; KiCadOrientationDeg 90 -> 0
- R1217: BoardSide F.Cu -> B.Cu; FootprintOriginMm 75.14,154.91 -> 47.41,189.89; KiCadOrientationDeg 0 -> 90
- R1218: FootprintOriginMm 87.91,171.89 -> 52.64,190.66; KiCadOrientationDeg 90 -> 180
- R1219: BoardSide F.Cu -> B.Cu; FootprintOriginMm 80.14,171.16 -> 45.16,217.89; KiCadOrientationDeg 0 -> 90
- R1220: FootprintOriginMm 64.91,176.89 -> 62.41,168.39
- R1221: BoardSide F.Cu -> B.Cu; FootprintOriginMm 89.41,165.14 -> 99.66,160.64; KiCadOrientationDeg 270 -> 90
- R1222: FootprintOriginMm 61.66,157.64 -> 97.16,160.64
- R1223: BoardSide B.Cu -> F.Cu; FootprintOriginMm 90.41,171.89 -> 64.16,169.64; KiCadOrientationDeg 90 -> 270
- R1224: BoardSide F.Cu -> B.Cu; FootprintOriginMm 88.39,154.91 -> 64.91,168.89; KiCadOrientationDeg 0 -> 90
- R1225: BoardSide F.Cu -> B.Cu; FootprintOriginMm 84.14,171.16 -> 47.66,217.89; KiCadOrientationDeg 0 -> 90
- R1226: BoardSide B.Cu -> F.Cu; FootprintOriginMm 95.39,177.16 -> 84.14,176.16; KiCadOrientationDeg 180 -> 0
- R1227: BoardSide F.Cu -> B.Cu; FootprintOriginMm 87.66,169.14 -> 83.91,128.89; KiCadOrientationDeg 270 -> 90
- R1228: FootprintOriginMm 64.91,172.89 -> 81.41,128.89
- R1229: FootprintOriginMm 88.89,149.66 -> 44.16,201.89; KiCadOrientationDeg 180 -> 90
- R1231: FootprintOriginMm 80.14,146.66 -> 38.89,195.91
- R1232: BoardSide B.Cu -> F.Cu; FootprintOriginMm 72.14,140.66 -> 61.41,165.64; KiCadOrientationDeg 180 -> 270
- R1233: BoardSide F.Cu -> B.Cu; FootprintOriginMm 76.91,171.89 -> 40.91,209.89; KiCadOrientationDeg 270 -> 90
- R1234: BoardSide F.Cu -> B.Cu; FootprintOriginMm 63.91,155.14 -> 80.14,179.41; KiCadOrientationDeg 270 -> 180
- R1235: FootprintOriginMm 71.14,154.91 -> 76.14,175.41
- R1236: FootprintOriginMm 95.41,146.39 -> 97.66,151.14
- R1237: BoardSide F.Cu -> B.Cu; FootprintOriginMm 73.39,152.41 -> 64.91,172.89; KiCadOrientationDeg 0 -> 90
- R1238: BoardSide B.Cu -> F.Cu; FootprintOriginMm 60.16,153.64 -> 66.41,173.64; KiCadOrientationDeg 90 -> 270
- R1239: BoardSide F.Cu -> B.Cu; FootprintOriginMm 91.66,154.14 -> 52.16,176.89; KiCadOrientationDeg 270 -> 90
- R1240: FootprintOriginMm 68.91,161.14 -> 87.89,111.66; KiCadOrientationDeg 270 -> 0
- R1241: BoardSide B.Cu -> F.Cu; FootprintOriginMm 62.41,168.39 -> 80.14,144.91; KiCadOrientationDeg 90 -> 0
- R1242: BoardSide F.Cu -> B.Cu; FootprintOriginMm 89.91,173.14 -> 80.14,144.16; KiCadOrientationDeg 270 -> 180
- R1243: BoardSide B.Cu -> F.Cu; FootprintOriginMm 76.14,142.66 -> 80.14,142.41; KiCadOrientationDeg 180 -> 0
- R1244: FootprintOriginMm 90.14,149.91 -> 90.16,169.14; KiCadOrientationDeg 0 -> 270
- R1245: FootprintOriginMm 84.14,146.66 -> 59.91,169.64; KiCadOrientationDeg 180 -> 90
- R1246: FootprintOriginMm 76.91,145.89 -> 60.16,153.64
- R1247: FootprintOriginMm 60.91,161.64 -> 87.39,131.66; KiCadOrientationDeg 90 -> 180
- R1248: BoardSide F.Cu -> B.Cu; FootprintOriginMm 95.41,161.14 -> 84.14,144.16; KiCadOrientationDeg 270 -> 180
- R1249: FootprintOriginMm 84.14,176.16 -> 84.14,144.91
- R1250: BoardSide B.Cu -> F.Cu; FootprintOriginMm 99.66,160.64 -> 96.66,154.64; KiCadOrientationDeg 90 -> 270
- R1251: BoardSide F.Cu -> B.Cu; FootprintOriginMm 88.14,144.66 -> 84.14,146.66; KiCadOrientationDeg 0 -> 180
- R1252: FootprintOriginMm 62.66,152.89 -> 64.39,149.66; KiCadOrientationDeg 90 -> 180
- R1253: BoardSide F.Cu -> B.Cu; FootprintOriginMm 76.14,143.16 -> 67.39,131.16; KiCadOrientationDeg 0 -> 180
- R1254: FootprintOriginMm 64.39,149.66 -> 68.14,144.91
- R1255: BoardSide F.Cu -> B.Cu; FootprintOriginMm 80.14,142.41 -> 78.91,127.14; KiCadOrientationDeg 0 -> 90
- R1256: BoardSide B.Cu -> F.Cu; FootprintOriginMm 88.64,175.16 -> 101.39,111.66; KiCadOrientationDeg 180 -> 0
- R1257: FootprintOriginMm 88.39,152.41 -> 73.39,152.41
- R1258: BoardSide F.Cu -> B.Cu; FootprintOriginMm 66.66,169.64 -> 69.41,189.89; KiCadOrientationDeg 270 -> 90
- R1259: BoardSide B.Cu -> F.Cu; FootprintOriginMm 80.14,141.66 -> 66.66,169.64; KiCadOrientationDeg 180 -> 270
- R1260: BoardSide B.Cu -> F.Cu; FootprintOriginMm 101.66,164.64 -> 63.91,165.64; KiCadOrientationDeg 90 -> 270
- R1261: FootprintOriginMm 80.14,179.41 -> 76.14,183.91
- R1262: BoardSide F.Cu -> B.Cu; FootprintOriginMm 80.14,173.66 -> 80.14,181.91; KiCadOrientationDeg 0 -> 180
- R1263: BoardSide F.Cu -> B.Cu; FootprintOriginMm 76.14,175.41 -> 61.66,157.64; KiCadOrientationDeg 0 -> 90
- R1264: FootprintOriginMm 91.91,165.14 -> 63.91,155.14
- R1265: FootprintOriginMm 94.16,154.14 -> 84.14,171.16; KiCadOrientationDeg 270 -> 0
- R1266: BoardSide B.Cu -> F.Cu; FootprintOriginMm 99.41,156.64 -> 80.14,173.66; KiCadOrientationDeg 90 -> 0
- R1267: FootprintOriginMm 72.14,143.16 -> 84.14,141.66
- R1268: BoardSide B.Cu -> F.Cu; FootprintOriginMm 88.14,147.16 -> 84.14,173.66; KiCadOrientationDeg 180 -> 0
- R1269: FootprintOriginMm 72.14,175.41 -> 80.14,171.16
- R1270: BoardSide B.Cu -> F.Cu; FootprintOriginMm 84.14,141.66 -> 76.91,171.89; KiCadOrientationDeg 180 -> 270
- R1271: FootprintOriginMm 92.91,171.89 -> 62.66,152.89
- R1272: BoardSide B.Cu -> F.Cu; FootprintOriginMm 58.41,161.64 -> 61.91,132.89; KiCadOrientationDeg 90 -> 270
- R1273: BoardSide B.Cu -> F.Cu; FootprintOriginMm 86.16,180.89 -> 75.14,154.91; KiCadOrientationDeg 90 -> 0
- R1274: BoardSide F.Cu -> B.Cu; FootprintOriginMm 68.14,157.91 -> 87.91,171.89; KiCadOrientationDeg 0 -> 90
- R1275: BoardSide F.Cu -> B.Cu; FootprintOriginMm 96.66,154.64 -> 90.41,171.89; KiCadOrientationDeg 270 -> 90
- R1276: BoardSide F.Cu -> B.Cu; FootprintOriginMm 64.14,158.41 -> 88.89,149.66; KiCadOrientationDeg 0 -> 180
- R1277: BoardSide F.Cu -> B.Cu; FootprintOriginMm 90.16,169.14 -> 92.89,149.66; KiCadOrientationDeg 270 -> 180
- R1278: BoardSide B.Cu -> F.Cu; FootprintOriginMm 63.41,161.64 -> 68.14,157.91; KiCadOrientationDeg 90 -> 0
- R1279: BoardSide B.Cu -> F.Cu; FootprintOriginMm 59.91,169.64 -> 71.14,154.91; KiCadOrientationDeg 90 -> 0
- R1280: BoardSide F.Cu -> B.Cu; FootprintOriginMm 96.14,157.91 -> 80.14,146.66; KiCadOrientationDeg 0 -> 180
- R1281: FootprintOriginMm 64.91,168.89 -> 80.14,141.66; KiCadOrientationDeg 90 -> 180
- R1282: FootprintOriginMm 68.14,144.91 -> 76.91,145.89; KiCadOrientationDeg 180 -> 90
- R1283: BoardSide B.Cu -> F.Cu; FootprintOriginMm 68.14,142.41 -> 70.64,147.41; KiCadOrientationDeg 180 -> 0
- R1284: BoardSide F.Cu -> B.Cu; FootprintOriginMm 84.14,173.66 -> 65.16,152.89; KiCadOrientationDeg 0 -> 90
- R1285: BoardSide F.Cu -> B.Cu; FootprintOriginMm 64.16,169.64 -> 62.14,137.41; KiCadOrientationDeg 270 -> 180
- R1286: BoardSide B.Cu -> F.Cu; FootprintOriginMm 100.16,152.64 -> 73.39,149.91; KiCadOrientationDeg 90 -> 0
- R1287: BoardSide B.Cu -> F.Cu; FootprintOriginMm 97.16,160.64 -> 90.14,149.91; KiCadOrientationDeg 90 -> 0
- R1288: BoardSide B.Cu -> F.Cu; FootprintOriginMm 80.14,144.16 -> 88.39,154.91; KiCadOrientationDeg 180 -> 0
- R1289: FootprintOriginMm 73.39,149.91 -> 95.41,161.14; KiCadOrientationDeg 0 -> 270
- R1290: BoardSide B.Cu -> F.Cu; FootprintOriginMm 102.16,160.64 -> 96.14,157.91; KiCadOrientationDeg 90 -> 0
- R1291: BoardSide B.Cu -> F.Cu; FootprintOriginMm 97.66,151.14 -> 95.41,169.14; KiCadOrientationDeg 90 -> 270
- R1292: FootprintOriginMm 61.41,165.64 -> 64.14,158.41; KiCadOrientationDeg 270 -> 0
- R1293: FootprintOriginMm 101.16,168.64 -> 57.89,137.91; KiCadOrientationDeg 90 -> 180
- R1294: FootprintOriginMm 69.64,181.16 -> 58.41,161.64; KiCadOrientationDeg 180 -> 90
- R1295: FootprintOriginMm 80.14,181.91 -> 63.41,161.64; KiCadOrientationDeg 180 -> 90
- R1296: BoardSide F.Cu -> B.Cu; FootprintOriginMm 66.41,173.64 -> 60.91,161.64; KiCadOrientationDeg 270 -> 90
- R1297: FootprintOriginMm 80.14,144.91 -> 68.91,161.14; KiCadOrientationDeg 0 -> 270
- R1298: FootprintOriginMm 63.91,165.64 -> 89.41,165.14
- R1299: BoardSide B.Cu -> F.Cu; FootprintOriginMm 62.41,172.39 -> 91.91,165.14; KiCadOrientationDeg 90 -> 270
- RB1201: FootprintOriginMm 92.89,149.66 -> 102.16,160.64; KiCadOrientationDeg 180 -> 90
- RB1210: BoardSide B.Cu -> F.Cu; FootprintOriginMm 65.16,152.89 -> 91.66,154.14; KiCadOrientationDeg 90 -> 270
- RB1211: FootprintOriginMm 87.41,173.14 -> 88.39,152.41; KiCadOrientationDeg 270 -> 0
- RB1212: BoardSide B.Cu -> F.Cu; FootprintOriginMm 86.89,177.66 -> 87.41,173.14; KiCadOrientationDeg 180 -> 270
- RB1213: BoardSide B.Cu -> F.Cu; FootprintOriginMm 84.14,144.16 -> 87.66,169.14; KiCadOrientationDeg 180 -> 270
- RB1214: BoardSide F.Cu -> B.Cu; FootprintOriginMm 92.41,173.14 -> 92.14,144.41; KiCadOrientationDeg 270 -> 180
- RB1215: FootprintOriginMm 92.14,144.41 -> 95.41,146.39; KiCadOrientationDeg 180 -> 90
- RB1216: BoardSide F.Cu -> B.Cu; FootprintOriginMm 68.91,174.14 -> 88.14,147.16; KiCadOrientationDeg 270 -> 180
- RB1217: FootprintOriginMm 70.64,147.41 -> 88.14,144.66
- RB1218: FootprintOriginMm 84.14,144.91 -> 92.41,173.14; KiCadOrientationDeg 0 -> 270
- RB1219: FootprintOriginMm 95.41,169.14 -> 89.91,173.14
- RB1220: BoardSide F.Cu -> B.Cu; FootprintOriginMm 88.14,176.41 -> 88.64,175.16; KiCadOrientationDeg 0 -> 180
- RB1221: BoardSide B.Cu -> F.Cu; FootprintOriginMm 76.14,183.91 -> 88.14,176.41; KiCadOrientationDeg 180 -> 0
- RVO1206: BoardSide F.Cu -> B.Cu; FootprintOriginMm 68.6,151.55 -> 88.95,141.05; KiCadOrientationDeg 0 -> 180
- RVO1209: BoardSide B.Cu -> F.Cu; FootprintOriginMm 88.95,141.05 -> 68.6,151.55; KiCadOrientationDeg 180 -> 0
