File: boards/osc-core/sheets/oscillator_O3_K.kicad_sch (KiCad schematic)
At the start: 154 parts, among them Q1301 BCM847BS,115, U1305 AS3340D, U1306 LM393BIDR, U1307 SN74HC14DR, U1308 LM393BIDR, U1309 OPA4197IPWR, U1310 OPA4197IPWR, U1311 OPA4197IPWR, U1312 OPA4196IDR, U1313 OPA4196IDR, U1314 OPA4196IDR, U1315 OPA4196IDR

Commit message: Split jack partition into two boards with local bypass clusters
Parts:
- C1301: FootprintOriginMm 63.14,137.96 -> 127.89,137.71
- C1302: FootprintOriginMm 66.89,137.96 -> 171.39,137.71
- C1303: FootprintOriginMm 70.64,137.96 -> 175.14,137.71
- C1304: FootprintOriginMm 74.39,137.96 -> 178.89,137.71
- C1305: FootprintOriginMm 78.14,137.96 -> 182.64,137.71
- C1306: FootprintOriginMm 81.89,137.96 -> 186.39,137.71
- C1307: FootprintOriginMm 85.64,137.96 -> 190.14,137.71
- C1308: FootprintOriginMm 89.39,137.96 -> 193.89,137.71
- C1309: FootprintOriginMm 93.14,137.96 -> 197.64,137.71
- C1310: FootprintOriginMm 100.64,137.96 -> 240.89,137.71
- C1311: FootprintOriginMm 240.64,137.96 -> 244.64,137.71
- C1312: FootprintOriginMm 244.39,137.96 -> 248.39,137.71
- C1313: FootprintOriginMm 248.14,137.96 -> 252.14,137.71
- C1314: FootprintOriginMm 21.14,138.21 -> 99.14,138.21
- C1315: FootprintOriginMm 24.89,138.21 -> 255.89,138.21
- C1316: FootprintOriginMm 28.64,138.21 -> 296.39,138.21
- C1317: FootprintOriginMm 32.39,138.21 -> 300.14,138.21
- C1318: FootprintOriginMm 36.14,138.21 -> 303.89,138.21
- C1319: FootprintOriginMm 39.89,138.21 -> 307.64,138.21
- C1320: FootprintOriginMm 47.39,138.21 -> 18.64,138.46
- C1329: FootprintOriginMm 51.14,138.21 -> 22.39,138.46
- C1330: FootprintOriginMm 108.14,138.46 -> 29.89,138.46
- C1331: FootprintOriginMm 111.89,138.46 -> 33.64,138.46
- C1332: FootprintOriginMm 115.64,138.46 -> 102.89,138.46
- C1333: FootprintOriginMm 119.39,138.46 -> 205.14,138.71
- C1334: FootprintOriginMm 123.14,138.46 -> 208.89,138.71
- C1335: FootprintOriginMm 271.64,139.21 -> 212.64,138.71
- C1336: FootprintOriginMm 285.39,139.21 -> 216.39,138.71
- C1337: FootprintOriginMm 289.14,139.21 -> 220.14,138.71
- C1338: FootprintOriginMm 296.89,139.21 -> 223.89,138.71
- C1339: FootprintOriginMm 300.64,139.21 -> 227.64,138.71
- C1342: FootprintOriginMm 9.89,139.46 -> 235.14,138.71
- C1343: FootprintOriginMm 13.64,139.46 -> 259.64,138.71
- C1344: FootprintOriginMm 17.39,139.46 -> 263.39,138.71
- C1345: FootprintOriginMm 308.14,139.46 -> 267.14,138.71
- C1346: FootprintOriginMm 210.64,139.71 -> 62.39,139.21
- C1347: FootprintOriginMm 214.39,139.71 -> 69.89,139.21
- C1348: FootprintOriginMm 218.14,139.71 -> 73.64,139.21
- C1349: FootprintOriginMm 256.64,139.71 -> 83.89,139.21
- DO1305: FootprintOriginMm 33.43,126.06 -> 111.43,126.81
- R1317: FootprintOriginMm 308.64,169.91 -> 36.14,169.66
- R1318: FootprintOriginMm 17.39,170.16 -> 39.89,169.66
- R1319: FootprintOriginMm 21.14,170.16 -> 43.64,169.66
- R1320: FootprintOriginMm 28.64,170.16 -> 47.39,169.66
- R1321: FootprintOriginMm 32.39,170.16 -> 51.14,169.66
- R1322: FootprintOriginMm 36.14,170.16 -> 58.64,169.66
- R1323: FootprintOriginMm 39.89,170.16 -> 70.14,169.66
- R1324: FootprintOriginMm 43.64,170.16 -> 85.14,169.66
- R1325: FootprintOriginMm 96.14,170.41 -> 96.39,169.66
- R1326: FootprintOriginMm 99.89,170.41 -> 100.14,169.66
- R1327: FootprintOriginMm 103.64,170.41 -> 103.89,169.66
- R1328: FootprintOriginMm 107.39,170.41 -> 107.64,169.66
- R1329: FootprintOriginMm 111.14,170.41 -> 118.64,169.66
- R1330: FootprintOriginMm 114.89,170.41 -> 159.89,169.66
- R1331: FootprintOriginMm 264.89,171.16 -> 163.64,169.66
- R1332: FootprintOriginMm 276.14,171.16 -> 167.39,169.66
- R1333: FootprintOriginMm 279.89,171.16 -> 171.14,169.66
- R1334: FootprintOriginMm 287.39,171.16 -> 178.64,169.66
- R1335: FootprintOriginMm 291.14,171.16 -> 182.39,169.66
- R1336: FootprintOriginMm 294.89,171.16 -> 186.14,169.66
- R1337: FootprintOriginMm 9.89,171.41 -> 189.89,169.66
- R1338: FootprintOriginMm 13.64,171.41 -> 227.39,169.66
- R1339: FootprintOriginMm 205.64,171.41 -> 231.14,169.66
- R1340: FootprintOriginMm 249.89,171.41 -> 239.89,169.66
- R1341: FootprintOriginMm 253.64,171.41 -> 6.14,169.91
- R1342: FootprintOriginMm 257.39,171.41 -> 306.89,169.91
- R1343: FootprintOriginMm 298.64,171.41 -> 88.89,170.16
- R1344: FootprintOriginMm 302.39,171.41 -> 243.64,170.16
- R1345: FootprintOriginMm 24.89,171.66 -> 279.89,170.16
- R1346: FootprintOriginMm 201.89,171.66 -> 283.64,170.16
- R1347: FootprintOriginMm 261.14,171.66 -> 287.39,170.16
- R1348: FootprintOriginMm 118.64,171.91 -> 291.14,170.16
- R1349: FootprintOriginMm 122.39,171.91 -> 294.89,170.16
- R1350: FootprintOriginMm 126.14,171.91 -> 298.64,170.16
- R1351: FootprintOriginMm 129.89,171.91 -> 302.39,170.16
- R1352: FootprintOriginMm 133.64,171.91 -> 13.64,170.41
- R1353: FootprintOriginMm 198.14,171.91 -> 17.39,170.41
- R1354: FootprintOriginMm 212.89,171.91 -> 21.14,170.41
- R1355: FootprintOriginMm 216.64,171.91 -> 24.89,170.41
- R1356: FootprintOriginMm 220.39,171.91 -> 28.64,170.41
- R1357: FootprintOriginMm 224.14,171.91 -> 92.64,170.41
- R1358: FootprintOriginMm 227.89,171.91 -> 193.64,170.66
- R1359: FootprintOriginMm 243.14,171.91 -> 197.39,170.66
- R1360: FootprintOriginMm 268.64,171.91 -> 201.14,170.66
- R1361: FootprintOriginMm 272.39,171.91 -> 212.89,170.66
- R1362: FootprintOriginMm 283.64,171.91 -> 223.64,170.66
- R1363: FootprintOriginMm 6.14,172.16 -> 247.39,170.66
- R1364: FootprintOriginMm 47.39,172.16 -> 54.89,171.16
- R1365: FootprintOriginMm 51.14,172.16 -> 62.39,171.16
- R1366: FootprintOriginMm 54.89,172.16 -> 66.14,171.16
- R1367: FootprintOriginMm 58.64,172.16 -> 73.89,171.16
- R1368: FootprintOriginMm 62.39,172.16 -> 77.64,171.16
- R1369: FootprintOriginMm 66.14,172.16 -> 81.39,171.16
- R1370: FootprintOriginMm 69.89,172.16 -> 122.39,171.16
- R1371: FootprintOriginMm 73.64,172.16 -> 126.14,171.16
- R1372: FootprintOriginMm 77.39,172.16 -> 129.89,171.16
- R1373: FootprintOriginMm 81.14,172.16 -> 133.64,171.16
- R1374: FootprintOriginMm 84.89,172.16 -> 137.39,171.16
- R1375: FootprintOriginMm 88.64,172.16 -> 156.14,171.16
- R1376: FootprintOriginMm 92.39,172.16 -> 257.39,171.16
- R1377: FootprintOriginMm 231.64,172.16 -> 261.14,171.16
- R1378: FootprintOriginMm 235.39,172.16 -> 264.89,171.16
- R1379: FootprintOriginMm 239.14,172.16 -> 268.64,171.16
- R1380: FootprintOriginMm 306.14,172.16 -> 272.39,171.16
- R1381: FootprintOriginMm 17.39,172.41 -> 141.14,171.41
- R1382: FootprintOriginMm 21.14,172.41 -> 144.89,171.41
- R1383: FootprintOriginMm 28.64,172.41 -> 148.64,171.41
- R1384: FootprintOriginMm 32.39,172.41 -> 152.39,171.41
- R1385: FootprintOriginMm 36.14,172.41 -> 9.89,171.66
- R1386: FootprintOriginMm 39.89,172.41 -> 111.39,171.66
- R1387: FootprintOriginMm 43.64,172.41 -> 174.89,171.66
- R1388: FootprintOriginMm 96.14,172.66 -> 204.89,171.66
- R1389: FootprintOriginMm 99.89,172.66 -> 216.64,171.66
- R1390: FootprintOriginMm 103.64,172.66 -> 234.89,171.66
- R1391: FootprintOriginMm 107.39,172.66 -> 251.14,171.66
- R1392: FootprintOriginMm 111.14,172.66 -> 276.14,171.66
- R1393: FootprintOriginMm 114.89,172.66 -> 32.39,171.91
- R1394: FootprintOriginMm 264.89,173.41 -> 36.14,171.91
- R1395: FootprintOriginMm 276.14,173.41 -> 39.89,171.91
- R1396: FootprintOriginMm 279.89,173.41 -> 43.64,171.91
- R1397: FootprintOriginMm 287.39,173.41 -> 47.39,171.91
- R1398: FootprintOriginMm 291.14,173.41 -> 51.14,171.91
- R1399: FootprintOriginMm 294.89,173.41 -> 58.64,171.91
- RB1301: FootprintOriginMm 80.89,219.66 -> 114.89,216.16
- RB1310: FootprintOriginMm 260.64,219.66 -> 235.64,216.16
- RB1311: FootprintOriginMm 264.39,219.66 -> 131.89,216.41
- RB1312: FootprintOriginMm 282.64,219.66 -> 9.89,216.66
- RB1313: FootprintOriginMm 286.39,219.66 -> 107.14,216.66
- RB1314: FootprintOriginMm 298.39,219.66 -> 122.39,216.66
- RB1315: FootprintOriginMm 302.14,219.66 -> 165.89,216.66
- RB1316: FootprintOriginMm 97.89,219.91 -> 190.39,216.66
- RB1317: FootprintOriginMm 118.39,219.91 -> 220.64,216.66
- RB1318: FootprintOriginMm 133.64,219.91 -> 252.14,216.66
- RB1319: FootprintOriginMm 148.64,219.91 -> 22.64,216.91
- RB1320: FootprintOriginMm 165.64,219.91 -> 26.39,216.91
- RB1321: FootprintOriginMm 56.39,220.16 -> 39.39,216.91
- RVO1306: FootprintOriginMm 246.45,121.8 -> 256.2,121.8
- RVO1307: FootprintOriginMm 252.2,121.8 -> 261.95,121.8
- RVO1308: FootprintOriginMm 257.95,121.8 -> 267.7,121.8
- RVO1309: FootprintOriginMm 263.7,121.8 -> 30.2,122.05
- RVO1310: FootprintOriginMm 33.7,122.05 -> 46.7,122.05
- RVO1311: FootprintOriginMm 39.45,122.05 -> 52.45,122.05
- U1306: FootprintOriginMm 212.7,110.3 -> 24.7,112.3
- U1308: FootprintOriginMm 246.7,110.3 -> 41.2,112.3
- U1309: FootprintOriginMm 51.6,99.38 -> 137.1,99.38
- U1310: FootprintOriginMm 69.6,99.38 -> 145.35,99.38
- U1311: FootprintOriginMm 86.6,99.38 -> 187.1,99.38
