File: boards/osc-core/sheets/oscillator_O3_K.kicad_sch (KiCad schematic)
At the start: 154 parts, among them Q1301 BCM847BS,115, U1305 AS3340D, U1306 LM393BIDR, U1307 SN74HC14DR, U1308 LM393BIDR, U1309 OPA4197IPWR, U1310 OPA4197IPWR, U1311 OPA4197IPWR, U1312 OPA4196IDR, U1313 OPA4196IDR, U1314 OPA4196IDR, U1315 OPA4196IDR

Commit message: WIP: locality placement source for the core board (#43)
Core packages are placed by the jack locality placer, anchored on the
core GH headers and pulled toward each module's own headers; IC/bypass
clusters stay rigid. Regenerated sources follow. Draft only.

Co-Authored-By: Claude Opus 5.5 <noreply@anthropic.com>
Parts:
- C1301: FootprintOriginMm 127.89,137.71 -> 20.96,194.39; KiCadOrientationDeg 180 -> 90
- C1302: FootprintOriginMm 171.39,137.71 -> 32.64,218.71
- C1303: BoardSide B.Cu -> F.Cu; FootprintOriginMm 175.14,137.71 -> 26.46,206.89; KiCadOrientationDeg 180 -> 270
- C1304: FootprintOriginMm 178.89,137.71 -> 42.14,221.71
- C1305: FootprintOriginMm 182.64,137.71 -> 14.96,201.89; KiCadOrientationDeg 180 -> 90
- C1306: BoardSide B.Cu -> F.Cu; FootprintOriginMm 186.39,137.71 -> 39.14,223.21; KiCadOrientationDeg 180 -> 0
- C1307: FootprintOriginMm 190.14,137.71 -> 16.64,187.46
- C1308: BoardSide B.Cu -> F.Cu; FootprintOriginMm 193.89,137.71 -> 42.89,223.71; KiCadOrientationDeg 180 -> 0
- C1309: FootprintOriginMm 197.64,137.71 -> 29.46,217.14; KiCadOrientationDeg 180 -> 90
- C1310: FootprintOriginMm 240.89,137.71 -> 14.96,190.64; KiCadOrientationDeg 180 -> 90
- C1311: FootprintOriginMm 244.64,137.71 -> 15.96,209.39; KiCadOrientationDeg 180 -> 90
- C1312: FootprintOriginMm 248.39,137.71 -> 17.21,213.14; KiCadOrientationDeg 180 -> 90
- C1313: BoardSide B.Cu -> F.Cu; FootprintOriginMm 252.14,137.71 -> 29.46,211.89; KiCadOrientationDeg 180 -> 270
- C1314: FootprintOriginMm 99.14,138.21 -> 19.71,198.14; KiCadOrientationDeg 180 -> 90
- C1315: BoardSide B.Cu -> F.Cu; FootprintOriginMm 255.89,138.21 -> 39.71,217.64; KiCadOrientationDeg 180 -> 270
- C1316: FootprintOriginMm 296.39,138.21 -> 23.39,185.46
- C1317: BoardSide B.Cu -> F.Cu; FootprintOriginMm 300.14,138.21 -> 24.21,203.14; KiCadOrientationDeg 180 -> 270
- C1318: FootprintOriginMm 303.89,138.21 -> 35.89,221.21
- C1319: FootprintOriginMm 307.64,138.21 -> 19.71,201.89; KiCadOrientationDeg 180 -> 90
- C1320: FootprintOriginMm 18.64,138.46 -> 20.39,191.21
- C1329: FootprintOriginMm 22.39,138.46 -> 32.23,206.205; KiCadOrientationDeg 180 -> 270
- C1330: FootprintOriginMm 29.89,138.46 -> 22.21,203.665; KiCadOrientationDeg 180 -> 270
- C1331: FootprintOriginMm 33.64,138.46 -> 55.715,205.64000000000001; KiCadOrientationDeg 180 -> 90
- C1332: BoardSide B.Cu -> F.Cu; FootprintOriginMm 102.89,138.46 -> 55.04,202.70999999999998
- C1333: BoardSide B.Cu -> F.Cu; FootprintOriginMm 205.14,138.71 -> 25.46,199.26500000000001; KiCadOrientationDeg 180 -> 90
- C1334: FootprintOriginMm 208.89,138.71 -> 33.93,192.71
- C1335: FootprintOriginMm 212.64,138.71 -> 33.93,203.03
- C1336: BoardSide B.Cu -> F.Cu; FootprintOriginMm 216.39,138.71 -> 42.330000000000005,214.53; KiCadOrientationDeg 180 -> 0
- C1337: BoardSide B.Cu -> F.Cu; FootprintOriginMm 220.14,138.71 -> 42.330000000000005,204.21; KiCadOrientationDeg 180 -> 0
- C1338: FootprintOriginMm 223.89,138.71 -> 28.459999999999997,212.56; KiCadOrientationDeg 180 -> 270
- C1339: FootprintOriginMm 227.64,138.71 -> 38.78,212.56; KiCadOrientationDeg 180 -> 270
- C1342: BoardSide B.Cu -> F.Cu; FootprintOriginMm 235.14,138.71 -> 35.71,198.89999999999998; KiCadOrientationDeg 180 -> 270
- C1343: BoardSide B.Cu -> F.Cu; FootprintOriginMm 259.64,138.71 -> 45.73,198.89999999999998; KiCadOrientationDeg 180 -> 270
- C1344: FootprintOriginMm 263.39,138.71 -> 38.96,208.63; KiCadOrientationDeg 180 -> 270
- C1345: FootprintOriginMm 267.14,138.71 -> 48.98,208.63; KiCadOrientationDeg 180 -> 270
- C1346: FootprintOriginMm 62.39,139.21 -> 48.98,197.5; KiCadOrientationDeg 180 -> 90
- C1347: FootprintOriginMm 69.89,139.21 -> 38.96,197.5; KiCadOrientationDeg 180 -> 90
- C1348: FootprintOriginMm 73.64,139.21 -> 38.73,185.0; KiCadOrientationDeg 180 -> 90
- C1349: FootprintOriginMm 83.89,139.21 -> 28.71,185.0; KiCadOrientationDeg 180 -> 90
- DO1305: BoardSide B.Cu -> F.Cu; FootprintOriginMm 111.43,126.81 -> 22.18,199.31; KiCadOrientationDeg 180 -> 0
- Q1301: FootprintOriginMm 6.1,17.28 -> 23.36,208.6; KiCadOrientationDeg 180 -> 90
- R1317: FootprintOriginMm 36.14,169.66 -> 38.91,201.14; KiCadOrientationDeg 180 -> 90
- R1318: FootprintOriginMm 39.89,169.66 -> 49.89,203.16
- R1319: BoardSide B.Cu -> F.Cu; FootprintOriginMm 43.64,169.66 -> 35.66,195.14; KiCadOrientationDeg 180 -> 270
- R1320: BoardSide B.Cu -> F.Cu; FootprintOriginMm 47.39,169.66 -> 24.41,214.39; KiCadOrientationDeg 180 -> 270
- R1321: FootprintOriginMm 51.14,169.66 -> 30.16,193.64; KiCadOrientationDeg 180 -> 90
- R1322: BoardSide B.Cu -> F.Cu; FootprintOriginMm 58.64,169.66 -> 42.89,219.16; KiCadOrientationDeg 180 -> 0
- R1323: FootprintOriginMm 70.14,169.66 -> 49.16,212.39; KiCadOrientationDeg 180 -> 90
- R1324: FootprintOriginMm 85.14,169.66 -> 44.14,214.16
- R1325: BoardSide B.Cu -> F.Cu; FootprintOriginMm 96.39,169.66 -> 32.64,193.91; KiCadOrientationDeg 180 -> 0
- R1326: FootprintOriginMm 100.14,169.66 -> 14.16,194.39; KiCadOrientationDeg 180 -> 90
- R1327: FootprintOriginMm 103.89,169.66 -> 27.91,193.64; KiCadOrientationDeg 180 -> 90
- R1328: FootprintOriginMm 107.64,169.66 -> 45.89,223.16
- R1329: FootprintOriginMm 118.64,169.66 -> 41.16,214.89; KiCadOrientationDeg 180 -> 90
- R1330: FootprintOriginMm 159.89,169.66 -> 27.14,222.41
- R1331: BoardSide B.Cu -> F.Cu; FootprintOriginMm 163.64,169.66 -> 37.16,209.14; KiCadOrientationDeg 180 -> 270
- R1332: BoardSide B.Cu -> F.Cu; FootprintOriginMm 167.39,169.66 -> 17.41,195.39; KiCadOrientationDeg 180 -> 270
- R1333: BoardSide B.Cu -> F.Cu; FootprintOriginMm 171.14,169.66 -> 46.64,211.16; KiCadOrientationDeg 180 -> 0
- R1334: FootprintOriginMm 178.64,169.66 -> 32.64,225.91
- R1335: FootprintOriginMm 182.39,169.66 -> 28.66,189.89; KiCadOrientationDeg 180 -> 90
- R1336: BoardSide B.Cu -> F.Cu; FootprintOriginMm 186.14,169.66 -> 25.89,217.41; KiCadOrientationDeg 180 -> 0
- R1337: FootprintOriginMm 189.89,169.66 -> 47.89,215.41
- R1338: FootprintOriginMm 227.39,169.66 -> 42.14,228.66
- R1339: FootprintOriginMm 231.14,169.66 -> 45.89,220.91
- R1340: BoardSide B.Cu -> F.Cu; FootprintOriginMm 239.89,169.66 -> 58.16,198.14; KiCadOrientationDeg 180 -> 270
- R1341: BoardSide B.Cu -> F.Cu; FootprintOriginMm 6.14,169.91 -> 26.66,210.64; KiCadOrientationDeg 180 -> 270
- R1342: FootprintOriginMm 306.89,169.91 -> 18.66,194.39; KiCadOrientationDeg 180 -> 90
- R1343: BoardSide B.Cu -> F.Cu; FootprintOriginMm 88.89,170.16 -> 24.16,206.89; KiCadOrientationDeg 180 -> 270
- R1344: FootprintOriginMm 243.64,170.16 -> 32.14,221.16
- R1345: BoardSide B.Cu -> F.Cu; FootprintOriginMm 279.89,170.16 -> 52.91,209.14; KiCadOrientationDeg 180 -> 270
- R1346: FootprintOriginMm 283.64,170.16 -> 44.14,216.41
- R1347: FootprintOriginMm 287.39,170.16 -> 20.66,209.14; KiCadOrientationDeg 180 -> 90
- R1348: FootprintOriginMm 291.14,170.16 -> 42.14,224.16
- R1349: FootprintOriginMm 294.89,170.16 -> 26.39,217.41
- R1350: FootprintOriginMm 298.64,170.16 -> 38.39,223.66
- R1351: FootprintOriginMm 302.39,170.16 -> 13.91,205.64; KiCadOrientationDeg 180 -> 90
- R1352: FootprintOriginMm 13.64,170.41 -> 19.66,188.14; KiCadOrientationDeg 180 -> 90
- R1353: FootprintOriginMm 17.39,170.41 -> 12.91,198.14; KiCadOrientationDeg 180 -> 90
- R1354: FootprintOriginMm 21.14,170.41 -> 21.91,212.89; KiCadOrientationDeg 180 -> 90
- R1355: FootprintOriginMm 24.89,170.41 -> 12.66,201.89; KiCadOrientationDeg 180 -> 90
- R1356: BoardSide B.Cu -> F.Cu; FootprintOriginMm 28.64,170.41 -> 49.66,211.89; KiCadOrientationDeg 180 -> 270
- R1357: FootprintOriginMm 92.64,170.41 -> 28.41,208.64; KiCadOrientationDeg 180 -> 90
- R1358: FootprintOriginMm 193.64,170.66 -> 17.41,198.14; KiCadOrientationDeg 180 -> 90
- R1359: BoardSide B.Cu -> F.Cu; FootprintOriginMm 197.39,170.66 -> 21.91,203.14; KiCadOrientationDeg 180 -> 270
- R1360: FootprintOriginMm 201.14,170.66 -> 23.39,221.16
- R1361: BoardSide B.Cu -> F.Cu; FootprintOriginMm 212.89,170.66 -> 42.89,216.91; KiCadOrientationDeg 180 -> 0
- R1362: FootprintOriginMm 223.64,170.66 -> 38.91,216.39; KiCadOrientationDeg 180 -> 90
- R1363: FootprintOriginMm 247.39,170.66 -> 38.91,220.14; KiCadOrientationDeg 180 -> 90
- R1364: FootprintOriginMm 54.89,171.16 -> 25.66,193.64; KiCadOrientationDeg 180 -> 90
- R1365: FootprintOriginMm 62.39,171.16 -> 17.41,201.89; KiCadOrientationDeg 180 -> 90
- R1366: FootprintOriginMm 66.14,171.16 -> 28.39,220.16
- R1367: FootprintOriginMm 73.89,171.16 -> 34.64,223.66
- R1368: FootprintOriginMm 77.64,171.16 -> 26.41,189.89; KiCadOrientationDeg 180 -> 90
- R1369: BoardSide B.Cu -> F.Cu; FootprintOriginMm 81.39,171.16 -> 42.89,221.41; KiCadOrientationDeg 180 -> 0
- R1370: BoardSide B.Cu -> F.Cu; FootprintOriginMm 122.39,171.16 -> 39.14,220.91; KiCadOrientationDeg 180 -> 0
- R1371: BoardSide B.Cu -> F.Cu; FootprintOriginMm 126.14,171.16 -> 28.89,193.91; KiCadOrientationDeg 180 -> 0
- R1372: FootprintOriginMm 129.89,171.16 -> 28.89,225.66
- R1373: FootprintOriginMm 133.64,171.16 -> 45.89,225.41
- R1374: FootprintOriginMm 137.39,171.16 -> 47.89,217.66
- R1375: FootprintOriginMm 156.14,171.16 -> 38.39,229.66
- R1376: BoardSide B.Cu -> F.Cu; FootprintOriginMm 257.39,171.16 -> 24.41,210.64; KiCadOrientationDeg 180 -> 270
- R1377: BoardSide B.Cu -> F.Cu; FootprintOriginMm 261.14,171.16 -> 36.39,212.16; KiCadOrientationDeg 180 -> 0
- R1378: BoardSide B.Cu -> F.Cu; FootprintOriginMm 264.89,171.16 -> 52.64,212.16; KiCadOrientationDeg 180 -> 0
- R1379: BoardSide B.Cu -> F.Cu; FootprintOriginMm 268.64,171.16 -> 42.89,226.16; KiCadOrientationDeg 180 -> 0
- R1380: FootprintOriginMm 272.39,171.16 -> 19.64,185.16
- R1381: FootprintOriginMm 141.14,171.41 -> 44.14,218.66
- R1382: FootprintOriginMm 144.89,171.41 -> 17.41,190.64; KiCadOrientationDeg 180 -> 90
- R1383: FootprintOriginMm 148.64,171.41 -> 11.91,194.39; KiCadOrientationDeg 180 -> 90
- R1384: FootprintOriginMm 152.39,171.41 -> 41.16,218.64; KiCadOrientationDeg 180 -> 90
- R1385: FootprintOriginMm 9.89,171.66 -> 12.66,190.64; KiCadOrientationDeg 180 -> 90
- R1386: FootprintOriginMm 111.39,171.66 -> 32.64,228.16
- R1387: FootprintOriginMm 174.89,171.66 -> 26.16,208.64; KiCadOrientationDeg 180 -> 90
- R1388: FootprintOriginMm 204.89,171.66 -> 23.41,193.64; KiCadOrientationDeg 180 -> 90
- R1389: BoardSide B.Cu -> F.Cu; FootprintOriginMm 216.64,171.66 -> 32.64,211.16; KiCadOrientationDeg 180 -> 0
- R1390: BoardSide B.Cu -> F.Cu; FootprintOriginMm 234.89,171.66 -> 25.89,219.66; KiCadOrientationDeg 180 -> 0
- R1391: BoardSide B.Cu -> F.Cu; FootprintOriginMm 251.14,171.66 -> 26.66,214.39; KiCadOrientationDeg 180 -> 270
- R1392: FootprintOriginMm 276.14,171.66 -> 13.66,209.39; KiCadOrientationDeg 180 -> 90
- R1393: FootprintOriginMm 32.39,171.91 -> 14.91,213.14; KiCadOrientationDeg 180 -> 90
- R1394: BoardSide B.Cu -> F.Cu; FootprintOriginMm 36.14,171.91 -> 21.39,215.66; KiCadOrientationDeg 180 -> 0
- R1395: BoardSide B.Cu -> F.Cu; FootprintOriginMm 39.89,171.91 -> 21.91,206.89; KiCadOrientationDeg 180 -> 270
- R1396: BoardSide B.Cu -> F.Cu; FootprintOriginMm 43.64,171.91 -> 15.16,195.39; KiCadOrientationDeg 180 -> 270
- R1397: FootprintOriginMm 47.39,171.91 -> 18.41,209.14; KiCadOrientationDeg 180 -> 90
- R1398: FootprintOriginMm 51.14,171.91 -> 16.41,194.39; KiCadOrientationDeg 180 -> 90
- R1399: FootprintOriginMm 58.64,171.91 -> 42.14,226.41
- RB1301: FootprintOriginMm 114.89,216.16 -> 26.41,186.14; KiCadOrientationDeg 180 -> 90
- RB1310: BoardSide B.Cu -> F.Cu; FootprintOriginMm 235.64,216.16 -> 38.39,214.66; KiCadOrientationDeg 180 -> 0
- RB1311: FootprintOriginMm 131.89,216.41 -> 32.64,216.41
- RB1312: FootprintOriginMm 9.89,216.66 -> 22.16,198.14; KiCadOrientationDeg 180 -> 90
- RB1313: BoardSide B.Cu -> F.Cu; FootprintOriginMm 107.14,216.66 -> 26.66,203.14; KiCadOrientationDeg 180 -> 270
- RB1314: FootprintOriginMm 122.39,216.66 -> 30.89,223.41
- RB1315: BoardSide B.Cu -> F.Cu; FootprintOriginMm 165.89,216.66 -> 36.16,221.64; KiCadOrientationDeg 180 -> 270
- RB1316: FootprintOriginMm 190.39,216.66 -> 19.66,212.89; KiCadOrientationDeg 180 -> 90
- RB1317: FootprintOriginMm 220.64,216.66 -> 39.16,226.64; KiCadOrientationDeg 180 -> 90
- RB1318: BoardSide B.Cu -> F.Cu; FootprintOriginMm 252.14,216.66 -> 19.66,195.39; KiCadOrientationDeg 180 -> 270
- RB1319: FootprintOriginMm 22.64,216.91 -> 15.16,198.14; KiCadOrientationDeg 180 -> 90
- RB1320: FootprintOriginMm 26.39,216.91 -> 23.41,218.14; KiCadOrientationDeg 180 -> 90
- RB1321: FootprintOriginMm 39.39,216.91 -> 16.16,205.64; KiCadOrientationDeg 180 -> 90
- RVO1306: FootprintOriginMm 256.2,121.8 -> 25.1,213.2; KiCadOrientationDeg 180 -> 90
- RVO1307: FootprintOriginMm 261.95,121.8 -> 42.35,232.45; KiCadOrientationDeg 180 -> 90
- RVO1308: FootprintOriginMm 267.7,121.8 -> 11.6,185.7; KiCadOrientationDeg 180 -> 90
- RVO1309: BoardSide B.Cu -> F.Cu; FootprintOriginMm 30.2,122.05 -> 17.35,199.55; KiCadOrientationDeg 180 -> 0
- RVO1310: BoardSide B.Cu -> F.Cu; FootprintOriginMm 46.7,122.05 -> 23.85,195.3; KiCadOrientationDeg 180 -> 0
- RVO1311: BoardSide B.Cu -> F.Cu; FootprintOriginMm 52.45,122.05 -> 21.1,211.85; KiCadOrientationDeg 180 -> 270
- U1305: FootprintOriginMm 45.7,14.09 -> 27.22,201.06; KiCadOrientationDeg 180 -> 0
- U1306: FootprintOriginMm 24.7,112.3 -> 53.81,211.33; KiCadOrientationDeg 180 -> 90
- U1307: BoardSide B.Cu -> F.Cu; FootprintOriginMm 293.7,23.45 -> 51.93,197.7; KiCadOrientationDeg 180 -> 270
- U1308: BoardSide B.Cu -> F.Cu; FootprintOriginMm 41.2,112.3 -> 30.47,198.06
- U1309: FootprintOriginMm 137.1,99.38 -> 34.63,197.87; KiCadOrientationDeg 180 -> 270
- U1310: BoardSide B.Cu -> F.Cu; FootprintOriginMm 145.35,99.38 -> 41.63,209.37; KiCadOrientationDeg 180 -> 90
- U1311: FootprintOriginMm 187.1,99.38 -> 33.62,211.86; KiCadOrientationDeg 180 -> 0
- U1312: BoardSide B.Cu -> F.Cu; FootprintOriginMm 301.45,23.45 -> 40.72,198.2; KiCadOrientationDeg 180 -> 0
- U1313: FootprintOriginMm 8.2,24.7 -> 43.97,207.93; KiCadOrientationDeg 180 -> 0
- U1314: FootprintOriginMm 15.95,24.7 -> 43.97,198.2
- U1315: FootprintOriginMm 23.7,24.7 -> 33.72,185.7

Commit message: WIP: spread core module homes and legalize module by module (#43)
The first core negotiation stalled (2501/2727 nets in conflict after 7
iterations). A RUDY map showed placement congestion: header-anchored
homes crowded ~1300 E/A packages into one corner, so modules were
scattered and 751 nets spanned 80 mm or more. Module home discs are now
spread inside the outline and notch, packages are legalized one module
at a time, and the core uses a 0.6 mm courtyard gap with a 0.5 mm IC
channel. Floorplan proxy: HPWL 162 -> 139 m, peak RUDY 1.39 -> 1.09 of
ideal four-signal-layer supply, tiles above 0.7 682 -> 160.

Co-Authored-By: Claude Opus 5.5 <noreply@anthropic.com>
Parts:
- C1301: FootprintOriginMm 20.96,194.39 -> 48.96,252.39
- C1302: BoardSide B.Cu -> F.Cu; FootprintOriginMm 32.64,218.71 -> 34.64,262.71; KiCadOrientationDeg 180 -> 0
- C1303: FootprintOriginMm 26.46,206.89 -> 26.64,233.96; KiCadOrientationDeg 270 -> 0
- C1304: BoardSide B.Cu -> F.Cu; FootprintOriginMm 42.14,221.71 -> 34.64,233.71; KiCadOrientationDeg 180 -> 0
- C1305: FootprintOriginMm 14.96,201.89 -> 52.96,244.39
- C1306: FootprintOriginMm 39.14,223.21 -> 21.64,264.96
- C1307: BoardSide B.Cu -> F.Cu; FootprintOriginMm 16.64,187.46 -> 36.64,230.46; KiCadOrientationDeg 180 -> 0
- C1308: BoardSide F.Cu -> B.Cu; FootprintOriginMm 42.89,223.71 -> 25.89,270.96; KiCadOrientationDeg 0 -> 180
- C1309: FootprintOriginMm 29.46,217.14 -> 11.71,252.39
- C1310: BoardSide B.Cu -> F.Cu; FootprintOriginMm 14.96,190.64 -> 41.96,231.89; KiCadOrientationDeg 90 -> 270
- C1311: BoardSide B.Cu -> F.Cu; FootprintOriginMm 15.96,209.39 -> 44.96,234.39; KiCadOrientationDeg 90 -> 270
- C1312: FootprintOriginMm 17.21,213.14 -> 10.71,235.89
- C1313: BoardSide F.Cu -> B.Cu; FootprintOriginMm 29.46,211.89 -> 47.21,237.89; KiCadOrientationDeg 270 -> 90
- C1314: FootprintOriginMm 19.71,198.14 -> 31.14,228.96; KiCadOrientationDeg 90 -> 180
- C1315: FootprintOriginMm 39.71,217.64 -> 46.46,248.39
- C1316: FootprintOriginMm 23.39,185.46 -> 19.14,232.71
- C1317: BoardSide F.Cu -> B.Cu; FootprintOriginMm 24.21,203.14 -> 14.21,237.89; KiCadOrientationDeg 270 -> 90
- C1318: FootprintOriginMm 35.89,221.21 -> 42.89,263.96
- C1319: BoardSide B.Cu -> F.Cu; FootprintOriginMm 19.71,201.89 -> 42.46,259.14; KiCadOrientationDeg 90 -> 270
- C1320: BoardSide B.Cu -> F.Cu; FootprintOriginMm 20.39,191.21 -> 30.64,232.46; KiCadOrientationDeg 180 -> 0
- C1329: FootprintOriginMm 32.23,206.205 -> 44.705000000000005,229.46; KiCadOrientationDeg 270 -> 0
- C1330: FootprintOriginMm 22.21,203.665 -> 42.165,239.48; KiCadOrientationDeg 270 -> 0
- C1331: FootprintOriginMm 55.715,205.64000000000001 -> 16.89,265.71; KiCadOrientationDeg 90 -> 180
- C1332: BoardSide F.Cu -> B.Cu; FootprintOriginMm 55.04,202.70999999999998 -> 15.139999999999999,253.45999999999998
- C1333: FootprintOriginMm 25.46,199.26500000000001 -> 17.96,261.015
- C1334: FootprintOriginMm 33.93,192.71 -> 24.46,259.31; KiCadOrientationDeg 180 -> 270
- C1335: FootprintOriginMm 33.93,203.03 -> 34.78,259.31; KiCadOrientationDeg 180 -> 270
- C1336: FootprintOriginMm 42.330000000000005,214.53 -> 39.580000000000005,253.53
- C1337: FootprintOriginMm 42.330000000000005,204.21 -> 39.580000000000005,243.21
- C1338: FootprintOriginMm 28.459999999999997,212.56 -> 37.459999999999994,259.31
- C1339: FootprintOriginMm 38.78,212.56 -> 47.78,259.31
- C1342: BoardSide F.Cu -> B.Cu; FootprintOriginMm 35.71,198.89999999999998 -> 42.63,253.48; KiCadOrientationDeg 270 -> 0
- C1343: BoardSide F.Cu -> B.Cu; FootprintOriginMm 45.73,198.89999999999998 -> 42.63,243.46; KiCadOrientationDeg 270 -> 0
- C1344: FootprintOriginMm 38.96,208.63 -> 27.25,232.46; KiCadOrientationDeg 270 -> 180
- C1345: FootprintOriginMm 48.98,208.63 -> 27.25,242.48; KiCadOrientationDeg 270 -> 180
- C1346: FootprintOriginMm 48.98,197.5 -> 31.38,253.48; KiCadOrientationDeg 90 -> 0
- C1347: FootprintOriginMm 38.96,197.5 -> 31.38,243.46; KiCadOrientationDeg 90 -> 0
- C1348: BoardSide B.Cu -> F.Cu; FootprintOriginMm 38.73,185.0 -> 17.89,248.2; KiCadOrientationDeg 90 -> 180
- C1349: BoardSide B.Cu -> F.Cu; FootprintOriginMm 28.71,185.0 -> 29.269999999999996,248.2; KiCadOrientationDeg 90 -> 0
- DO1305: BoardSide F.Cu -> B.Cu; FootprintOriginMm 22.18,199.31 -> 10.31,244.18; KiCadOrientationDeg 0 -> 90
- Q1301: BoardSide B.Cu -> F.Cu; FootprintOriginMm 23.36,208.6 -> 39.1,236.28; KiCadOrientationDeg 90 -> 0
- R1317: BoardSide B.Cu -> F.Cu; FootprintOriginMm 38.91,201.14 -> 32.66,248.39; KiCadOrientationDeg 90 -> 270
- R1318: FootprintOriginMm 49.89,203.16 -> 22.89,254.16
- R1319: BoardSide F.Cu -> B.Cu; FootprintOriginMm 35.66,195.14 -> 38.66,241.89; KiCadOrientationDeg 270 -> 90
- R1320: BoardSide F.Cu -> B.Cu; FootprintOriginMm 24.41,214.39 -> 53.91,248.39; KiCadOrientationDeg 270 -> 90
- R1321: BoardSide B.Cu -> F.Cu; FootprintOriginMm 30.16,193.64 -> 25.64,254.41; KiCadOrientationDeg 90 -> 0
- R1322: BoardSide F.Cu -> B.Cu; FootprintOriginMm 42.89,219.16 -> 49.64,245.16; KiCadOrientationDeg 0 -> 180
- R1323: BoardSide B.Cu -> F.Cu; FootprintOriginMm 49.16,212.39 -> 25.64,241.66; KiCadOrientationDeg 90 -> 0
- R1324: BoardSide B.Cu -> F.Cu; FootprintOriginMm 44.14,214.16 -> 25.64,239.16; KiCadOrientationDeg 180 -> 0
- R1325: FootprintOriginMm 32.64,193.91 -> 36.64,257.41
- R1326: BoardSide B.Cu -> F.Cu; FootprintOriginMm 14.16,194.39 -> 45.91,260.89; KiCadOrientationDeg 90 -> 270
- R1327: FootprintOriginMm 27.91,193.64 -> 20.14,237.91; KiCadOrientationDeg 90 -> 180
- R1328: BoardSide B.Cu -> F.Cu; FootprintOriginMm 45.89,223.16 -> 14.66,248.39; KiCadOrientationDeg 180 -> 270
- R1329: BoardSide B.Cu -> F.Cu; FootprintOriginMm 41.16,214.89 -> 22.41,240.89; KiCadOrientationDeg 90 -> 270
- R1330: FootprintOriginMm 27.14,222.41 -> 23.14,226.66
- R1331: BoardSide F.Cu -> B.Cu; FootprintOriginMm 37.16,209.14 -> 30.64,263.91; KiCadOrientationDeg 270 -> 180
- R1332: FootprintOriginMm 17.41,195.39 -> 25.64,267.41; KiCadOrientationDeg 270 -> 0
- R1333: FootprintOriginMm 46.64,211.16 -> 38.66,239.89; KiCadOrientationDeg 0 -> 270
- R1334: FootprintOriginMm 32.64,225.91 -> 27.14,224.91
- R1335: BoardSide B.Cu -> F.Cu; FootprintOriginMm 28.66,189.89 -> 30.64,260.16; KiCadOrientationDeg 90 -> 0
- R1336: BoardSide F.Cu -> B.Cu; FootprintOriginMm 25.89,217.41 -> 35.89,271.66; KiCadOrientationDeg 0 -> 180
- R1337: FootprintOriginMm 47.89,215.41 -> 35.66,263.39; KiCadOrientationDeg 180 -> 90
- R1338: FootprintOriginMm 42.14,228.66 -> 7.41,248.39; KiCadOrientationDeg 180 -> 90
- R1339: FootprintOriginMm 45.89,220.91 -> 23.14,231.66
- R1340: BoardSide F.Cu -> B.Cu; FootprintOriginMm 58.16,198.14 -> 16.16,241.89; KiCadOrientationDeg 270 -> 90
- R1341: FootprintOriginMm 26.66,210.64 -> 21.64,235.16; KiCadOrientationDeg 270 -> 0
- R1342: FootprintOriginMm 18.66,194.39 -> 49.39,255.66; KiCadOrientationDeg 90 -> 180
- R1343: BoardSide F.Cu -> B.Cu; FootprintOriginMm 24.16,206.89 -> 39.39,266.66; KiCadOrientationDeg 270 -> 180
- R1344: BoardSide B.Cu -> F.Cu; FootprintOriginMm 32.14,221.16 -> 38.64,262.66; KiCadOrientationDeg 180 -> 0
- R1345: BoardSide F.Cu -> B.Cu; FootprintOriginMm 52.91,209.14 -> 26.64,263.91; KiCadOrientationDeg 270 -> 180
- R1346: BoardSide B.Cu -> F.Cu; FootprintOriginMm 44.14,216.41 -> 34.64,260.16; KiCadOrientationDeg 180 -> 0
- R1347: FootprintOriginMm 20.66,209.14 -> 30.64,268.91; KiCadOrientationDeg 90 -> 180
- R1348: FootprintOriginMm 42.14,224.16 -> 23.14,229.16
- R1349: FootprintOriginMm 26.39,217.41 -> 51.41,248.39; KiCadOrientationDeg 180 -> 90
- R1350: FootprintOriginMm 38.39,223.66 -> 9.91,248.39; KiCadOrientationDeg 180 -> 90
- R1351: FootprintOriginMm 13.91,205.64 -> 39.39,226.16; KiCadOrientationDeg 90 -> 180
- R1352: BoardSide B.Cu -> F.Cu; FootprintOriginMm 19.66,188.14 -> 42.41,235.89; KiCadOrientationDeg 90 -> 270
- R1353: FootprintOriginMm 12.91,198.14 -> 31.14,223.91; KiCadOrientationDeg 90 -> 180
- R1354: FootprintOriginMm 21.91,212.89 -> 15.91,233.14
- R1355: FootprintOriginMm 12.66,201.89 -> 49.66,233.89
- R1356: FootprintOriginMm 49.66,211.89 -> 35.91,237.14
- R1357: BoardSide B.Cu -> F.Cu; FootprintOriginMm 28.41,208.64 -> 39.91,256.89; KiCadOrientationDeg 90 -> 270
- R1358: BoardSide B.Cu -> F.Cu; FootprintOriginMm 17.41,198.14 -> 38.64,233.16; KiCadOrientationDeg 90 -> 0
- R1359: FootprintOriginMm 21.91,203.14 -> 25.64,264.91; KiCadOrientationDeg 270 -> 0
- R1360: BoardSide B.Cu -> F.Cu; FootprintOriginMm 23.39,221.16 -> 15.41,260.89; KiCadOrientationDeg 180 -> 270
- R1361: BoardSide F.Cu -> B.Cu; FootprintOriginMm 42.89,216.91 -> 48.41,241.89; KiCadOrientationDeg 0 -> 90
- R1362: FootprintOriginMm 38.91,216.39 -> 45.91,241.89
- R1363: FootprintOriginMm 38.91,220.14 -> 27.14,229.91; KiCadOrientationDeg 90 -> 180
- R1364: FootprintOriginMm 25.66,193.64 -> 20.14,235.41; KiCadOrientationDeg 90 -> 180
- R1365: FootprintOriginMm 17.41,201.89 -> 11.16,239.89
- R1366: FootprintOriginMm 28.39,220.16 -> 27.14,227.41
- R1367: FootprintOriginMm 34.64,223.66 -> 19.14,230.16
- R1368: FootprintOriginMm 26.41,189.89 -> 31.14,231.66; KiCadOrientationDeg 90 -> 180
- R1369: BoardSide F.Cu -> B.Cu; FootprintOriginMm 42.89,221.41 -> 39.39,228.66; KiCadOrientationDeg 0 -> 180
- R1370: FootprintOriginMm 39.14,220.91 -> 22.64,232.66
- R1371: FootprintOriginMm 28.89,193.91 -> 25.64,236.66
- R1372: BoardSide B.Cu -> F.Cu; FootprintOriginMm 28.89,225.66 -> 40.64,265.16; KiCadOrientationDeg 180 -> 0
- R1373: FootprintOriginMm 45.89,225.41 -> 31.14,226.41
- R1374: BoardSide B.Cu -> F.Cu; FootprintOriginMm 47.89,217.66 -> 30.64,235.16; KiCadOrientationDeg 180 -> 0
- R1375: BoardSide B.Cu -> F.Cu; FootprintOriginMm 38.39,229.66 -> 23.14,230.16; KiCadOrientationDeg 180 -> 0
- R1376: BoardSide F.Cu -> B.Cu; FootprintOriginMm 24.41,210.64 -> 9.16,252.39; KiCadOrientationDeg 270 -> 90
- R1377: FootprintOriginMm 36.39,212.16 -> 43.91,248.39; KiCadOrientationDeg 0 -> 270
- R1378: FootprintOriginMm 52.64,212.16 -> 41.16,239.89; KiCadOrientationDeg 0 -> 270
- R1379: BoardSide F.Cu -> B.Cu; FootprintOriginMm 42.89,226.16 -> 13.66,265.39; KiCadOrientationDeg 0 -> 90
- R1380: FootprintOriginMm 19.64,185.16 -> 49.91,237.89; KiCadOrientationDeg 180 -> 90
- R1381: FootprintOriginMm 44.14,218.66 -> 38.89,263.91
- R1382: FootprintOriginMm 17.41,190.64 -> 47.16,233.89
- R1383: FootprintOriginMm 11.91,194.39 -> 15.14,229.91; KiCadOrientationDeg 90 -> 180
- R1384: FootprintOriginMm 41.16,218.64 -> 16.91,237.14
- R1385: FootprintOriginMm 12.66,190.64 -> 6.66,252.39
- R1386: FootprintOriginMm 32.64,228.16 -> 9.66,260.39; KiCadOrientationDeg 180 -> 90
- R1387: BoardSide B.Cu -> F.Cu; FootprintOriginMm 26.16,208.64 -> 42.91,255.14; KiCadOrientationDeg 90 -> 270
- R1388: FootprintOriginMm 23.41,193.64 -> 30.64,266.41; KiCadOrientationDeg 90 -> 180
- R1389: FootprintOriginMm 32.64,211.16 -> 21.64,237.66
- R1390: BoardSide F.Cu -> B.Cu; FootprintOriginMm 25.89,219.66 -> 52.91,258.14; KiCadOrientationDeg 0 -> 90
- R1391: BoardSide F.Cu -> B.Cu; FootprintOriginMm 26.66,214.39 -> 52.39,251.66; KiCadOrientationDeg 270 -> 180
- R1392: FootprintOriginMm 13.66,209.39 -> 43.39,226.91; KiCadOrientationDeg 90 -> 180
- R1393: FootprintOriginMm 14.91,213.14 -> 43.39,269.16; KiCadOrientationDeg 90 -> 180
- R1394: BoardSide F.Cu -> B.Cu; FootprintOriginMm 21.39,215.66 -> 52.41,237.14; KiCadOrientationDeg 0 -> 90
- R1395: FootprintOriginMm 21.91,206.89 -> 36.64,265.41; KiCadOrientationDeg 270 -> 0
- R1396: BoardSide F.Cu -> B.Cu; FootprintOriginMm 15.16,195.39 -> 7.89,239.41; KiCadOrientationDeg 270 -> 180
- R1397: FootprintOriginMm 18.41,209.14 -> 13.39,262.16; KiCadOrientationDeg 90 -> 180
- R1398: BoardSide B.Cu -> F.Cu; FootprintOriginMm 16.41,194.39 -> 26.41,230.64; KiCadOrientationDeg 90 -> 270
- R1399: FootprintOriginMm 42.14,226.41 -> 43.39,266.66
- RB1301: FootprintOriginMm 26.41,186.14 -> 13.66,241.89
- RB1310: FootprintOriginMm 38.39,214.66 -> 38.64,260.16
- RB1311: FootprintOriginMm 32.64,216.41 -> 48.91,248.39; KiCadOrientationDeg 180 -> 90
- RB1312: FootprintOriginMm 22.16,198.14 -> 12.41,248.39
- RB1313: FootprintOriginMm 26.66,203.14 -> 30.64,262.66; KiCadOrientationDeg 270 -> 0
- RB1314: FootprintOriginMm 30.89,223.41 -> 50.41,258.89; KiCadOrientationDeg 180 -> 90
- RB1315: FootprintOriginMm 36.16,221.64 -> 42.64,262.41; KiCadOrientationDeg 270 -> 0
- RB1316: FootprintOriginMm 19.66,212.89 -> 46.89,263.91; KiCadOrientationDeg 90 -> 180
- RB1317: FootprintOriginMm 39.16,226.64 -> 9.66,256.39
- RB1318: FootprintOriginMm 19.66,195.39 -> 49.16,248.39
- RB1319: BoardSide B.Cu -> F.Cu; FootprintOriginMm 15.16,198.14 -> 12.16,248.39; KiCadOrientationDeg 90 -> 270
- RB1320: FootprintOriginMm 23.41,218.14 -> 39.39,269.16; KiCadOrientationDeg 90 -> 180
- RB1321: FootprintOriginMm 16.16,205.64 -> 13.41,233.89
- RVO1306: FootprintOriginMm 25.1,213.2 -> 25.45,267.55; KiCadOrientationDeg 90 -> 180
- RVO1307: BoardSide B.Cu -> F.Cu; FootprintOriginMm 42.35,232.45 -> 8.35,248.35; KiCadOrientationDeg 90 -> 270
- RVO1308: FootprintOriginMm 11.6,185.7 -> 48.85,228.7
- RVO1309: FootprintOriginMm 17.35,199.55 -> 16.85,234.3
- RVO1310: BoardSide F.Cu -> B.Cu; FootprintOriginMm 23.85,195.3 -> 13.1,257.7; KiCadOrientationDeg 0 -> 90
- RVO1311: BoardSide F.Cu -> B.Cu; FootprintOriginMm 21.1,211.85 -> 30.7,272.55; KiCadOrientationDeg 270 -> 180
- U1305: FootprintOriginMm 27.22,201.06 -> 39.56,234.47; KiCadOrientationDeg 0 -> 90
- U1306: FootprintOriginMm 53.81,211.33 -> 19.495,260.7; KiCadOrientationDeg 90 -> 270
- U1307: BoardSide F.Cu -> B.Cu; FootprintOriginMm 51.93,197.7 -> 19.65,248.45
- U1308: FootprintOriginMm 30.47,198.06 -> 22.97,259.81
- U1309: FootprintOriginMm 34.63,197.87 -> 29.62,258.61; KiCadOrientationDeg 270 -> 0
- U1310: FootprintOriginMm 41.63,209.37 -> 38.88,248.37
- U1311: FootprintOriginMm 33.62,211.86 -> 42.62,258.61
- U1312: BoardSide F.Cu -> B.Cu; FootprintOriginMm 40.72,198.2 -> 41.93,248.47; KiCadOrientationDeg 0 -> 90
- U1313: FootprintOriginMm 43.97,207.93 -> 27.95,237.47; KiCadOrientationDeg 0 -> 270
- U1314: FootprintOriginMm 43.97,198.2 -> 30.68,248.47; KiCadOrientationDeg 180 -> 90
- U1315: BoardSide B.Cu -> F.Cu; FootprintOriginMm 33.72,185.7 -> 23.58,248.2; KiCadOrientationDeg 180 -> 0

Commit message: WIP: same-footprint swap pass for the core placement (#43)
Ported span-penalized slot swaps (nets over 60 mm pay a quadratic
penalty), limited to same-footprint slots within 25 mm of each package's
net median. Floorplan proxy: HPWL 139 -> 105 m, median span 28.8 mm,
RUDY p99 0.78 with 68 tiles above 0.7 (JL with swaps: p99 0.81, 42).

Co-Authored-By: Claude Opus 5.5 <noreply@anthropic.com>
Parts:
- C1302: BoardSide F.Cu -> B.Cu; FootprintOriginMm 34.64,262.71 -> 47.21,237.89; KiCadOrientationDeg 0 -> 90
- C1303: FootprintOriginMm 26.64,233.96 -> 44.96,234.39; KiCadOrientationDeg 0 -> 270
- C1304: BoardSide F.Cu -> B.Cu; FootprintOriginMm 34.64,233.71 -> 19.14,232.71; KiCadOrientationDeg 0 -> 180
- C1305: BoardSide B.Cu -> F.Cu; FootprintOriginMm 52.96,244.39 -> 21.64,264.96; KiCadOrientationDeg 90 -> 0
- C1306: BoardSide F.Cu -> B.Cu; FootprintOriginMm 21.64,264.96 -> 11.71,252.39; KiCadOrientationDeg 0 -> 90
- C1307: FootprintOriginMm 36.64,230.46 -> 26.64,233.96
- C1308: FootprintOriginMm 25.89,270.96 -> 14.21,237.89; KiCadOrientationDeg 180 -> 90
- C1309: BoardSide B.Cu -> F.Cu; FootprintOriginMm 11.71,252.39 -> 30.64,232.46; KiCadOrientationDeg 90 -> 0
- C1310: BoardSide F.Cu -> B.Cu; FootprintOriginMm 41.96,231.89 -> 31.14,228.96; KiCadOrientationDeg 270 -> 180
- C1311: FootprintOriginMm 44.96,234.39 -> 34.64,233.71; KiCadOrientationDeg 270 -> 0
- C1313: BoardSide B.Cu -> F.Cu; FootprintOriginMm 47.21,237.89 -> 41.96,231.89; KiCadOrientationDeg 90 -> 270
- C1314: BoardSide B.Cu -> F.Cu; FootprintOriginMm 31.14,228.96 -> 36.64,230.46; KiCadOrientationDeg 180 -> 0
- C1316: FootprintOriginMm 19.14,232.71 -> 52.96,244.39; KiCadOrientationDeg 180 -> 90
- C1317: FootprintOriginMm 14.21,237.89 -> 25.89,270.96; KiCadOrientationDeg 90 -> 180
- C1318: BoardSide B.Cu -> F.Cu; FootprintOriginMm 42.89,263.96 -> 34.64,262.71; KiCadOrientationDeg 180 -> 0
- C1319: BoardSide F.Cu -> B.Cu; FootprintOriginMm 42.46,259.14 -> 42.89,263.96; KiCadOrientationDeg 270 -> 180
- C1320: FootprintOriginMm 30.64,232.46 -> 42.46,259.14; KiCadOrientationDeg 0 -> 270
- R1317: BoardSide F.Cu -> B.Cu; FootprintOriginMm 32.66,248.39 -> 50.41,258.89; KiCadOrientationDeg 270 -> 90
- R1318: FootprintOriginMm 22.89,254.16 -> 49.39,255.66
- R1319: FootprintOriginMm 38.66,241.89 -> 43.39,266.66; KiCadOrientationDeg 90 -> 180
- R1320: FootprintOriginMm 53.91,248.39 -> 39.39,266.66; KiCadOrientationDeg 90 -> 180
- R1321: FootprintOriginMm 25.64,254.41 -> 41.16,239.89; KiCadOrientationDeg 0 -> 270
- R1322: FootprintOriginMm 49.64,245.16 -> 45.91,241.89; KiCadOrientationDeg 180 -> 90
- R1323: BoardSide F.Cu -> B.Cu; FootprintOriginMm 25.64,241.66 -> 49.66,233.89; KiCadOrientationDeg 0 -> 90
- R1324: BoardSide F.Cu -> B.Cu; FootprintOriginMm 25.64,239.16 -> 47.16,233.89; KiCadOrientationDeg 0 -> 90
- R1325: BoardSide F.Cu -> B.Cu; FootprintOriginMm 36.64,257.41 -> 43.39,269.16; KiCadOrientationDeg 0 -> 180
- R1326: FootprintOriginMm 45.91,260.89 -> 40.64,265.16; KiCadOrientationDeg 270 -> 0
- R1327: BoardSide B.Cu -> F.Cu; FootprintOriginMm 20.14,237.91 -> 23.14,230.16; KiCadOrientationDeg 180 -> 0
- R1328: BoardSide F.Cu -> B.Cu; FootprintOriginMm 14.66,248.39 -> 19.14,230.16; KiCadOrientationDeg 270 -> 180
- R1329: BoardSide F.Cu -> B.Cu; FootprintOriginMm 22.41,240.89 -> 39.39,269.16; KiCadOrientationDeg 270 -> 180
- R1330: BoardSide B.Cu -> F.Cu; FootprintOriginMm 23.14,226.66 -> 25.64,267.41; KiCadOrientationDeg 180 -> 0
- R1331: BoardSide B.Cu -> F.Cu; FootprintOriginMm 30.64,263.91 -> 42.91,255.14; KiCadOrientationDeg 180 -> 270
- R1332: BoardSide F.Cu -> B.Cu; FootprintOriginMm 25.64,267.41 -> 9.66,256.39; KiCadOrientationDeg 0 -> 90
- R1333: BoardSide F.Cu -> B.Cu; FootprintOriginMm 38.66,239.89 -> 46.89,263.91; KiCadOrientationDeg 270 -> 180
- R1334: FootprintOriginMm 27.14,224.91 -> 38.89,263.91
- R1335: BoardSide F.Cu -> B.Cu; FootprintOriginMm 30.64,260.16 -> 48.41,241.89; KiCadOrientationDeg 0 -> 90
- R1336: FootprintOriginMm 35.89,271.66 -> 52.91,258.14; KiCadOrientationDeg 180 -> 90
- R1337: FootprintOriginMm 35.66,263.39 -> 27.14,229.91; KiCadOrientationDeg 90 -> 180
- R1338: FootprintOriginMm 7.41,248.39 -> 27.14,227.41; KiCadOrientationDeg 90 -> 180
- R1339: FootprintOriginMm 23.14,231.66 -> 52.41,237.14; KiCadOrientationDeg 180 -> 90
- R1340: FootprintOriginMm 16.16,241.89 -> 26.39,193.91; KiCadOrientationDeg 90 -> 180
- R1341: FootprintOriginMm 21.64,235.16 -> 30.64,260.16
- R1342: FootprintOriginMm 49.39,255.66 -> 26.64,263.91
- R1343: BoardSide B.Cu -> F.Cu; FootprintOriginMm 39.39,266.66 -> 30.64,262.66; KiCadOrientationDeg 180 -> 0
- R1344: FootprintOriginMm 38.64,262.66 -> 49.16,248.39; KiCadOrientationDeg 0 -> 270
- R1345: FootprintOriginMm 26.64,263.91 -> 49.91,237.89; KiCadOrientationDeg 180 -> 90
- R1346: FootprintOriginMm 34.64,260.16 -> 45.91,260.89; KiCadOrientationDeg 0 -> 270
- R1347: FootprintOriginMm 30.64,268.91 -> 30.64,263.91
- R1348: BoardSide B.Cu -> F.Cu; FootprintOriginMm 23.14,229.16 -> 30.64,235.16; KiCadOrientationDeg 180 -> 0
- R1349: FootprintOriginMm 51.41,248.39 -> 31.14,231.66; KiCadOrientationDeg 90 -> 180
- R1350: FootprintOriginMm 9.91,248.39 -> 7.89,239.41; KiCadOrientationDeg 90 -> 180
- R1351: BoardSide B.Cu -> F.Cu; FootprintOriginMm 39.39,226.16 -> 38.64,233.16; KiCadOrientationDeg 180 -> 0
- R1352: BoardSide F.Cu -> B.Cu; FootprintOriginMm 42.41,235.89 -> 39.39,228.66; KiCadOrientationDeg 270 -> 180
- R1353: FootprintOriginMm 31.14,223.91 -> 15.91,233.14; KiCadOrientationDeg 180 -> 90
- R1354: FootprintOriginMm 15.91,233.14 -> 13.41,233.89
- R1355: BoardSide B.Cu -> F.Cu; FootprintOriginMm 49.66,233.89 -> 26.41,230.64; KiCadOrientationDeg 90 -> 270
- R1356: BoardSide F.Cu -> B.Cu; FootprintOriginMm 35.91,237.14 -> 34.64,191.41; KiCadOrientationDeg 270 -> 180
- R1357: FootprintOriginMm 39.91,256.89 -> 34.64,260.16; KiCadOrientationDeg 270 -> 0
- R1358: BoardSide F.Cu -> B.Cu; FootprintOriginMm 38.64,233.16 -> 23.14,226.66; KiCadOrientationDeg 0 -> 180
- R1359: FootprintOriginMm 25.64,264.91 -> 15.41,260.89; KiCadOrientationDeg 0 -> 270
- R1360: BoardSide F.Cu -> B.Cu; FootprintOriginMm 15.41,260.89 -> 9.66,260.39; KiCadOrientationDeg 270 -> 90
- R1361: FootprintOriginMm 48.41,241.89 -> 39.39,226.16; KiCadOrientationDeg 90 -> 180
- R1362: FootprintOriginMm 45.91,241.89 -> 43.39,226.91; KiCadOrientationDeg 90 -> 180
- R1363: FootprintOriginMm 27.14,229.91 -> 43.66,205.89; KiCadOrientationDeg 180 -> 90
- R1364: FootprintOriginMm 20.14,235.41 -> 43.66,213.89; KiCadOrientationDeg 180 -> 90
- R1365: BoardSide B.Cu -> F.Cu; FootprintOriginMm 11.16,239.89 -> 25.64,239.16; KiCadOrientationDeg 90 -> 0
- R1366: BoardSide B.Cu -> F.Cu; FootprintOriginMm 27.14,227.41 -> 21.64,237.66; KiCadOrientationDeg 180 -> 0
- R1367: FootprintOriginMm 19.14,230.16 -> 20.14,237.91
- R1368: FootprintOriginMm 31.14,231.66 -> 11.16,239.89; KiCadOrientationDeg 180 -> 90
- R1369: BoardSide B.Cu -> F.Cu; FootprintOriginMm 39.39,228.66 -> 25.64,236.66; KiCadOrientationDeg 180 -> 0
- R1370: FootprintOriginMm 22.64,232.66 -> 21.64,235.16
- R1371: BoardSide F.Cu -> B.Cu; FootprintOriginMm 25.64,236.66 -> 12.41,248.39; KiCadOrientationDeg 0 -> 90
- R1372: FootprintOriginMm 40.64,265.16 -> 12.16,248.39; KiCadOrientationDeg 0 -> 270
- R1373: FootprintOriginMm 31.14,226.41 -> 20.14,235.41
- R1374: BoardSide F.Cu -> B.Cu; FootprintOriginMm 30.64,235.16 -> 9.16,252.39; KiCadOrientationDeg 0 -> 90
- R1375: BoardSide F.Cu -> B.Cu; FootprintOriginMm 23.14,230.16 -> 6.66,252.39; KiCadOrientationDeg 0 -> 90
- R1376: BoardSide B.Cu -> F.Cu; FootprintOriginMm 9.16,252.39 -> 35.91,237.14; KiCadOrientationDeg 90 -> 270
- R1377: FootprintOriginMm 43.91,248.39 -> 32.66,248.39
- R1378: BoardSide F.Cu -> B.Cu; FootprintOriginMm 41.16,239.89 -> 9.91,248.39; KiCadOrientationDeg 270 -> 90
- R1379: FootprintOriginMm 13.66,265.39 -> 7.41,248.39
- R1380: BoardSide B.Cu -> F.Cu; FootprintOriginMm 49.91,237.89 -> 38.66,239.89; KiCadOrientationDeg 90 -> 270
- R1381: FootprintOriginMm 38.89,263.91 -> 38.66,241.89; KiCadOrientationDeg 180 -> 90
- R1382: FootprintOriginMm 47.16,233.89 -> 23.14,231.66; KiCadOrientationDeg 90 -> 180
- R1383: BoardSide B.Cu -> F.Cu; FootprintOriginMm 15.14,229.91 -> 22.64,232.66; KiCadOrientationDeg 180 -> 0
- R1384: FootprintOriginMm 16.91,237.14 -> 13.39,262.16; KiCadOrientationDeg 90 -> 180
- R1385: FootprintOriginMm 6.66,252.39 -> 13.66,265.39
- R1386: FootprintOriginMm 9.66,260.39 -> 30.64,266.41; KiCadOrientationDeg 90 -> 180
- R1387: FootprintOriginMm 42.91,255.14 -> 22.41,240.89
- R1388: BoardSide B.Cu -> F.Cu; FootprintOriginMm 30.64,266.41 -> 14.66,248.39; KiCadOrientationDeg 180 -> 270
- R1389: BoardSide F.Cu -> B.Cu; FootprintOriginMm 21.64,237.66 -> 31.14,226.41; KiCadOrientationDeg 0 -> 180
- R1390: FootprintOriginMm 52.91,258.14 -> 31.14,223.91; KiCadOrientationDeg 90 -> 180
- R1391: FootprintOriginMm 52.39,251.66 -> 15.14,229.91
- R1392: BoardSide B.Cu -> F.Cu; FootprintOriginMm 43.39,226.91 -> 42.41,235.89; KiCadOrientationDeg 180 -> 270
- R1393: BoardSide B.Cu -> F.Cu; FootprintOriginMm 43.39,269.16 -> 36.64,257.41; KiCadOrientationDeg 180 -> 0
- R1394: FootprintOriginMm 52.41,237.14 -> 16.91,237.14
- R1395: BoardSide F.Cu -> B.Cu; FootprintOriginMm 36.64,265.41 -> 16.16,241.89; KiCadOrientationDeg 0 -> 90
- R1396: FootprintOriginMm 7.89,239.41 -> 13.66,241.89; KiCadOrientationDeg 180 -> 90
- R1397: BoardSide B.Cu -> F.Cu; FootprintOriginMm 13.39,262.16 -> 25.64,254.41; KiCadOrientationDeg 180 -> 0
- R1398: BoardSide F.Cu -> B.Cu; FootprintOriginMm 26.41,230.64 -> 22.89,254.16; KiCadOrientationDeg 270 -> 180
- R1399: BoardSide B.Cu -> F.Cu; FootprintOriginMm 43.39,266.66 -> 25.64,264.91; KiCadOrientationDeg 180 -> 0
- RB1301: BoardSide B.Cu -> F.Cu; FootprintOriginMm 13.66,241.89 -> 25.64,241.66; KiCadOrientationDeg 90 -> 0
- RB1310: FootprintOriginMm 38.64,260.16 -> 43.91,248.39; KiCadOrientationDeg 0 -> 270
- RB1312: FootprintOriginMm 12.41,248.39 -> 49.64,245.16; KiCadOrientationDeg 90 -> 180
- RB1313: BoardSide F.Cu -> B.Cu; FootprintOriginMm 30.64,262.66 -> 51.41,248.39; KiCadOrientationDeg 0 -> 90
- RB1314: FootprintOriginMm 50.41,258.89 -> 30.64,268.91; KiCadOrientationDeg 90 -> 180
- RB1315: BoardSide F.Cu -> B.Cu; FootprintOriginMm 42.64,262.41 -> 35.89,271.66; KiCadOrientationDeg 0 -> 180
- RB1316: BoardSide B.Cu -> F.Cu; FootprintOriginMm 46.89,263.91 -> 36.64,265.41; KiCadOrientationDeg 180 -> 0
- RB1317: FootprintOriginMm 9.66,256.39 -> 35.66,263.39
- RB1318: FootprintOriginMm 49.16,248.39 -> 42.64,262.41; KiCadOrientationDeg 270 -> 0
- RB1319: FootprintOriginMm 12.16,248.39 -> 38.64,262.66; KiCadOrientationDeg 270 -> 0
- RB1320: BoardSide B.Cu -> F.Cu; FootprintOriginMm 39.39,269.16 -> 38.64,260.16; KiCadOrientationDeg 180 -> 0
- RB1321: BoardSide B.Cu -> F.Cu; FootprintOriginMm 13.41,233.89 -> 39.91,256.89; KiCadOrientationDeg 90 -> 270
- RVO1306: FootprintOriginMm 25.45,267.55 -> 30.7,272.55
- RVO1311: FootprintOriginMm 30.7,272.55 -> 25.45,267.55
