File: boards/osc-core/sheets/sample_hold_H1_K.kicad_sch (KiCad schematic)
At the start: 53 parts, among them U101 REF5050AIDR, U103 OPA4197IPWR, U107 LM393BIDR, U111 SN74HC14DR, U112 OPA4196IDR, U113 OPA4196IDR, U114 CD74HC221M96, U115 LF398M/NOPB, U116 OPA4197IPWR, U117 OPA4197IPWR, U118 OPA4197IPWR, U119 OPA4196IDR

Commit message: Split jack partition into two boards with local bypass clusters
Parts:
- C101: FootprintOriginMm 28.89,122.71 -> 164.64,34.96
- C102: FootprintOriginMm 106.89,129.21 -> 178.39,118.21
- C104: FootprintOriginMm 242.71,39.65 -> 242.21,39.65
- C105: FootprintOriginMm 279.96,118.9 -> 129.46,120.9
- C106: FootprintOriginMm 56.21,135.4 -> 75.96,134.15
- C113: FootprintOriginMm 180.64,135.21 -> 195.89,135.21
- C116: FootprintOriginMm 302.64,136.71 -> 222.14,136.21
- C119: FootprintOriginMm 306.39,136.71 -> 225.89,136.21
- C120: FootprintOriginMm 9.89,136.96 -> 229.64,136.21
- C123: FootprintOriginMm 169.39,137.71 -> 288.89,136.71
- C124: FootprintOriginMm 221.89,137.71 -> 43.64,137.71
- C125: FootprintOriginMm 6.14,137.96 -> 112.89,137.71
- C128: FootprintOriginMm 55.64,137.96 -> 116.64,137.71
- C129: FootprintOriginMm 59.39,137.96 -> 120.39,137.71
- C131: FootprintOriginMm 96.89,137.96 -> 201.39,137.71
- C132: FootprintOriginMm 43.64,138.21 -> 311.39,138.21
- C133: FootprintOriginMm 104.39,138.46 -> 26.14,138.46
- C134: FootprintOriginMm 304.39,139.21 -> 231.39,138.71
- C135: FootprintOriginMm 260.39,139.71 -> 87.64,139.21
- C140: FootprintOriginMm 264.14,139.71 -> 91.39,139.21
- C141: FootprintOriginMm 156.89,140.21 -> 282.14,139.21
- C142: FootprintOriginMm 198.14,140.21 -> 37.39,140.21
- C143: FootprintOriginMm 221.89,140.21 -> 48.64,140.21
- C144: FootprintOriginMm 58.64,140.46 -> 171.39,140.21
- C145: FootprintOriginMm 92.39,140.46 -> 238.89,140.21
- C146: FootprintOriginMm 61.21,135.4 -> 87.21,134.15
- C147: FootprintOriginMm 66.21,135.4 -> 92.21,134.15
- C148: FootprintOriginMm 71.21,135.4 -> 153.21,134.4
- DH111: FootprintOriginMm 34.35,135.5 -> 277.1,134.0
- DH112: FootprintOriginMm 39.85,135.5 -> 282.6,134.0
- R101: FootprintOriginMm 32.89,84.91 -> 167.64,77.16
- R102: FootprintOriginMm 50.89,84.91 -> 32.89,84.91
- R103: FootprintOriginMm 68.14,84.91 -> 50.89,84.91
- R104: FootprintOriginMm 84.89,84.91 -> 68.14,84.91
- R109: FootprintOriginMm 310.14,116.91 -> 84.89,84.91
- R110: FootprintOriginMm 301.64,119.16 -> 202.89,84.91
- R111: FootprintOriginMm 218.64,120.66 -> 161.14,96.66
- R112: FootprintOriginMm 208.64,164.66 -> 216.14,120.66
- R113: FootprintOriginMm 133.89,165.16 -> 43.89,165.16
- R122: FootprintOriginMm 286.14,167.41 -> 253.64,167.16
- R123: FootprintOriginMm 81.39,167.66 -> 99.89,167.41
- U101: FootprintOriginMm 111.2,110.3 -> 197.2,92.8
- U103: FootprintOriginMm 162.85,97.38 -> 111.85,97.38
- U107: FootprintOriginMm 128.2,110.3 -> 94.2,110.3
- U116: FootprintOriginMm 247.85,97.38 -> 31.6,99.38
- U117: FootprintOriginMm 264.85,97.38 -> 51.6,99.38
- U118: FootprintOriginMm 8.35,99.38 -> 69.6,99.38
