File: boards/osc-core/sheets/sample_hold_H1_K.kicad_sch (KiCad schematic)
At the start: 53 parts, among them U101 REF5050AIDR, U103 OPA4197IPWR, U107 LM393BIDR, U111 SN74HC14DR, U112 OPA4196IDR, U113 OPA4196IDR, U114 CD74HC221M96, U115 LF398M/NOPB, U116 OPA4197IPWR, U117 OPA4197IPWR, U118 OPA4197IPWR, U119 OPA4196IDR

Commit message: WIP: locality placement source for the core board (#43)
Core packages are placed by the jack locality placer, anchored on the
core GH headers and pulled toward each module's own headers; IC/bypass
clusters stay rigid. Regenerated sources follow. Draft only.

Co-Authored-By: Claude Opus 5.5 <noreply@anthropic.com>
Parts:
- C101: FootprintOriginMm 164.64,34.96 -> 167.39,111.21
- C102: BoardSide B.Cu -> F.Cu; FootprintOriginMm 178.39,118.21 -> 163.64,136.46; KiCadOrientationDeg 180 -> 0
- C104: FootprintOriginMm 242.21,39.65 -> 179.4,126.96; KiCadOrientationDeg 180 -> 90
- C105: FootprintOriginMm 129.46,120.9 -> 171.71,112.4
- C106: FootprintOriginMm 75.96,134.15 -> 157.71,138.15
- C113: FootprintOriginMm 195.89,135.21 -> 153.465,125.71
- C116: BoardSide B.Cu -> F.Cu; FootprintOriginMm 222.14,136.21 -> 182.51500000000001,133.95999999999998
- C119: FootprintOriginMm 225.89,136.21 -> 176.73,126.97999999999999; KiCadOrientationDeg 180 -> 90
- C120: FootprintOriginMm 229.64,136.21 -> 166.71,126.97999999999999; KiCadOrientationDeg 180 -> 90
- C123: BoardSide B.Cu -> F.Cu; FootprintOriginMm 288.89,136.71 -> 177.03,129.57999999999998; KiCadOrientationDeg 180 -> 270
- C124: BoardSide B.Cu -> F.Cu; FootprintOriginMm 43.64,137.71 -> 166.71,129.57999999999998; KiCadOrientationDeg 180 -> 270
- C125: BoardSide B.Cu -> F.Cu; FootprintOriginMm 112.89,137.71 -> 173.715,115.89; KiCadOrientationDeg 180 -> 90
- C128: FootprintOriginMm 116.64,137.71 -> 166.53,122.67999999999999; KiCadOrientationDeg 180 -> 90
- C129: FootprintOriginMm 120.39,137.71 -> 156.21,122.67999999999999; KiCadOrientationDeg 180 -> 90
- C131: BoardSide B.Cu -> F.Cu; FootprintOriginMm 201.39,137.71 -> 163.07999999999998,134.03; KiCadOrientationDeg 180 -> 0
- C132: BoardSide B.Cu -> F.Cu; FootprintOriginMm 311.39,138.21 -> 163.07999999999998,123.71000000000001; KiCadOrientationDeg 180 -> 0
- C133: FootprintOriginMm 26.14,138.46 -> 181.11,122.07000000000001; KiCadOrientationDeg 180 -> 270
- C134: FootprintOriginMm 231.39,138.71 -> 181.11,110.39; KiCadOrientationDeg 180 -> 90
- C135: BoardSide B.Cu -> F.Cu; FootprintOriginMm 87.64,139.21 -> 157.64,112.89; KiCadOrientationDeg 180 -> 90
- C140: FootprintOriginMm 91.39,139.21 -> 162.25,127.71
- C141: FootprintOriginMm 282.14,139.21 -> 162.25,137.73
- C142: FootprintOriginMm 37.39,140.21 -> 176.73,118.25; KiCadOrientationDeg 180 -> 90
- C143: FootprintOriginMm 48.64,140.21 -> 166.71,118.25; KiCadOrientationDeg 180 -> 90
- C144: FootprintOriginMm 171.39,140.21 -> 166.48,114.5; KiCadOrientationDeg 180 -> 90
- C145: FootprintOriginMm 238.89,140.21 -> 156.46,114.5; KiCadOrientationDeg 180 -> 90
- C146: BoardSide B.Cu -> F.Cu; FootprintOriginMm 87.21,134.15 -> 157.4,133.21; KiCadOrientationDeg 180 -> 270
- C147: FootprintOriginMm 92.21,134.15 -> 154.71,119.4
- C148: BoardSide B.Cu -> F.Cu; FootprintOriginMm 153.21,134.4 -> 156.46,125.65; KiCadOrientationDeg 180 -> 0
- DH111: BoardSide B.Cu -> F.Cu; FootprintOriginMm 277.1,134.0 -> 171.86,133.5; KiCadOrientationDeg 180 -> 0
- DH112: FootprintOriginMm 282.6,134.0 -> 171.85,135.25
- R101: FootprintOriginMm 167.64,77.16 -> 176.64,136.91
- R102: BoardSide B.Cu -> F.Cu; FootprintOriginMm 32.89,84.91 -> 176.39,133.16; KiCadOrientationDeg 180 -> 0
- R103: BoardSide B.Cu -> F.Cu; FootprintOriginMm 50.89,84.91 -> 167.91,133.89; KiCadOrientationDeg 180 -> 270
- R104: BoardSide B.Cu -> F.Cu; FootprintOriginMm 68.14,84.91 -> 170.64,116.41; KiCadOrientationDeg 180 -> 0
- R109: FootprintOriginMm 84.89,84.91 -> 176.91,133.89; KiCadOrientationDeg 180 -> 90
- R110: FootprintOriginMm 202.89,84.91 -> 182.64,125.16
- R111: BoardSide B.Cu -> F.Cu; FootprintOriginMm 161.14,96.66 -> 167.39,136.91; KiCadOrientationDeg 180 -> 0
- R112: BoardSide B.Cu -> F.Cu; FootprintOriginMm 216.14,120.66 -> 178.66,123.14; KiCadOrientationDeg 180 -> 270
- R113: BoardSide B.Cu -> F.Cu; FootprintOriginMm 43.89,165.16 -> 159.91,134.89; KiCadOrientationDeg 180 -> 270
- R122: BoardSide B.Cu -> F.Cu; FootprintOriginMm 253.64,167.16 -> 157.91,128.89; KiCadOrientationDeg 180 -> 270
- R123: BoardSide B.Cu -> F.Cu; FootprintOriginMm 99.89,167.41 -> 167.66,115.64; KiCadOrientationDeg 180 -> 270
- U101: FootprintOriginMm 197.2,92.8 -> 154.8,130.72; KiCadOrientationDeg 180 -> 270
- U103: BoardSide B.Cu -> F.Cu; FootprintOriginMm 111.85,97.38 -> 171.87,128.88; KiCadOrientationDeg 180 -> 0
- U107: BoardSide B.Cu -> F.Cu; FootprintOriginMm 94.2,110.3 -> 181.31,128.95; KiCadOrientationDeg 180 -> 270
- U111: BoardSide B.Cu -> F.Cu; FootprintOriginMm 254.95,13.45 -> 161.45,118.58; KiCadOrientationDeg 180 -> 90
- U112: FootprintOriginMm 293.7,13.45 -> 162.95,132.72; KiCadOrientationDeg 180 -> 270
- U113: FootprintOriginMm 301.45,13.45 -> 171.72,118.95
- U114: BoardSide B.Cu -> F.Cu; FootprintOriginMm 30.2,14.09 -> 171.81,121.58; KiCadOrientationDeg 180 -> 270
- U115: FootprintOriginMm 309.2,17.45 -> 171.72,128.95
- U116: FootprintOriginMm 31.6,99.38 -> 161.37,123.38
- U117: BoardSide B.Cu -> F.Cu; FootprintOriginMm 51.6,99.38 -> 162.38,128.87; KiCadOrientationDeg 180 -> 90
- U118: FootprintOriginMm 69.6,99.38 -> 181.11,116.23; KiCadOrientationDeg 180 -> 90
- U119: FootprintOriginMm 247.2,23.45 -> 161.47,115.2

Commit message: Place and rail-route the six-layer core draft (#43)
- Core through-hole packages (NOISE2 U6101) block both faces in the
  locality legalizer; the core POWER-* reserves are the TP load lands
  themselves and no longer emit keepouts over them.
- sync projects the netlist's representative multi-unit fields on the
  core so schematic parity is clean.
- route_jack_grid.py refuses an unclean start board, runs up to 40
  signal batches and skips empty ones.
- Synced, placed and prepared osc-core board; rail plane fanout, rail
  links and rail escapes: 7355 -> 5849 native open edges with 0 DRC
  errors and 0 parity per stage. Routed draft in progress.

Co-Authored-By: Claude Opus 5.5 <noreply@anthropic.com>
Parts:
- C101: BoardSide B.Cu -> F.Cu; FootprintOriginMm 167.39,111.21 -> 157.71,125.14; KiCadOrientationDeg 180 -> 270
- C148: BoardSide F.Cu -> B.Cu; FootprintOriginMm 156.46,125.65 -> 167.15,109.96; KiCadOrientationDeg 0 -> 90
Changed lines of the file:
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@@
     (property "Island" "IO_CORE:${SHEETNAME}" (at 294.64 50.8 0) (effects (font (size 1.27 1.27)) (hide yes)))
     (property "BoardRegion" "core" (at 294.64 50.8 0) (effects (font (size 1.27 1.27)) (hide yes)))
-    (property "BoardSide" "B.Cu" (at 294.64 50.8 0) (effects (font (size 1.27 1.27)) (hide yes)))
+    (property "BoardSide" "F.Cu" (at 294.64 50.8 0) (effects (font (size 1.27 1.27)) (hide yes)))
     (property "BoardAssignment" "K" (at 294.64 50.8 0) (effects (font (size 1.27 1.27)) (hide yes)))
-    (property "KiCadOrientationDeg" "180" (at 294.64 50.8 0) (effects (font (size 1.27 1.27)) (hide yes)))
-    (property "FootprintOriginMm" "167.39,111.21" (at 294.64 50.8 0) (effects (font (size 1.27 1.27)) (hide yes)))
+    (property "KiCadOrientationDeg" "270" (at 294.64 50.8 0) (effects (font (size 1.27 1.27)) (hide yes)))
+    (property "FootprintOriginMm" "157.71,125.14" (at 294.64 50.8 0) (effects (font (size 1.27 1.27)) (hide yes)))
     (property "Sensitive" "" (at 294.64 50.8 0) (effects (font (size 1.27 1.27)) (hide yes)))
     (pin "1")
@@
     (property "Island" "BULK_TBD" (at 416.56 508 0) (effects (font (size 1.27 1.27)) (hide yes)))
     (property "BoardRegion" "core" (at 416.56 508 0) (effects (font (size 1.27 1.27)) (hide yes)))
-    (property "BoardSide" "F.Cu" (at 416.56 508 0) (effects (font (size 1.27 1.27)) (hide yes)))
+    (property "BoardSide" "B.Cu" (at 416.56 508 0) (effects (font (size 1.27 1.27)) (hide yes)))
     (property "BoardAssignment" "K" (at 416.56 508 0) (effects (font (size 1.27 1.27)) (hide yes)))
-    (property "KiCadOrientationDeg" "0" (at 416.56 508 0) (effects (font (size 1.27 1.27)) (hide yes)))
-    (property "FootprintOriginMm" "156.46,125.65" (at 416.56 508 0) (effects (font (size 1.27 1.27)) (hide yes)))
+    (property "KiCadOrientationDeg" "90" (at 416.56 508 0) (effects (font (size 1.27 1.27)) (hide yes)))
+    (property "FootprintOriginMm" "167.15,109.96" (at 416.56 508 0) (effects (font (size 1.27 1.27)) (hide yes)))
     (property "Sensitive" "" (at 416.56 508 0) (effects (font (size 1.27 1.27)) (hide yes)))
     (pin "1")

Commit message: WIP: spread core module homes and legalize module by module (#43)
The first core negotiation stalled (2501/2727 nets in conflict after 7
iterations). A RUDY map showed placement congestion: header-anchored
homes crowded ~1300 E/A packages into one corner, so modules were
scattered and 751 nets spanned 80 mm or more. Module home discs are now
spread inside the outline and notch, packages are legalized one module
at a time, and the core uses a 0.6 mm courtyard gap with a 0.5 mm IC
channel. Floorplan proxy: HPWL 162 -> 139 m, peak RUDY 1.39 -> 1.09 of
ideal four-signal-layer supply, tiles above 0.7 682 -> 160.

Co-Authored-By: Claude Opus 5.5 <noreply@anthropic.com>
Parts:
- C101: BoardSide F.Cu -> B.Cu; FootprintOriginMm 157.71,125.14 -> 158.71,75.39; KiCadOrientationDeg 270 -> 90
- C102: FootprintOriginMm 163.64,136.46 -> 136.89,66.46
- C104: BoardSide B.Cu -> F.Cu; FootprintOriginMm 179.4,126.96 -> 149.9,73.46; KiCadOrientationDeg 90 -> 270
- C105: FootprintOriginMm 171.71,112.4 -> 143.71,60.9
- C106: FootprintOriginMm 157.71,138.15 -> 157.15,70.71; KiCadOrientationDeg 180 -> 90
- C113: FootprintOriginMm 153.465,125.71 -> 153.395,94.21000000000001; KiCadOrientationDeg 180 -> 0
- C116: FootprintOriginMm 182.51500000000001,133.95999999999998 -> 130.46,88.015; KiCadOrientationDeg 180 -> 90
- C119: FootprintOriginMm 176.73,126.97999999999999 -> 146.73,75.48
- C120: FootprintOriginMm 166.71,126.97999999999999 -> 136.71,75.48
- C123: FootprintOriginMm 177.03,129.57999999999998 -> 147.03,73.08
- C124: FootprintOriginMm 166.71,129.57999999999998 -> 136.71,73.08
- C125: BoardSide F.Cu -> B.Cu; FootprintOriginMm 173.715,115.89 -> 139.935,61.39
- C128: FootprintOriginMm 166.53,122.67999999999999 -> 136.71,90.31; KiCadOrientationDeg 90 -> 270
- C129: FootprintOriginMm 156.21,122.67999999999999 -> 147.03,90.31; KiCadOrientationDeg 90 -> 270
- C131: BoardSide F.Cu -> B.Cu; FootprintOriginMm 163.07999999999998,134.03 -> 152.31,72.03
- C132: BoardSide F.Cu -> B.Cu; FootprintOriginMm 163.07999999999998,123.71000000000001 -> 152.31,61.71000000000001
- C133: FootprintOriginMm 181.11,122.07000000000001 -> 130.93,61.71000000000001; KiCadOrientationDeg 270 -> 180
- C134: FootprintOriginMm 181.11,110.39 -> 130.93,72.03; KiCadOrientationDeg 90 -> 180
- C135: BoardSide F.Cu -> B.Cu; FootprintOriginMm 157.64,112.89 -> 135.70999999999998,94.69000000000001; KiCadOrientationDeg 90 -> 270
- C140: FootprintOriginMm 162.25,127.71 -> 147.71,79.63000000000001; KiCadOrientationDeg 180 -> 270
- C141: FootprintOriginMm 162.25,137.73 -> 157.73,79.63000000000001; KiCadOrientationDeg 180 -> 270
- C142: FootprintOriginMm 176.73,118.25 -> 125.71,79.63000000000001; KiCadOrientationDeg 90 -> 270
- C143: FootprintOriginMm 166.71,118.25 -> 135.73,79.63000000000001; KiCadOrientationDeg 90 -> 270
- C144: BoardSide B.Cu -> F.Cu; FootprintOriginMm 166.48,114.5 -> 152.73,87.98
- C145: BoardSide B.Cu -> F.Cu; FootprintOriginMm 156.46,114.5 -> 142.71,87.98
- C146: BoardSide F.Cu -> B.Cu; FootprintOriginMm 157.4,133.21 -> 141.71,95.15; KiCadOrientationDeg 270 -> 180
- C147: BoardSide B.Cu -> F.Cu; FootprintOriginMm 154.71,119.4 -> 130.65,69.46; KiCadOrientationDeg 180 -> 270
- C148: BoardSide B.Cu -> F.Cu; FootprintOriginMm 167.15,109.96 -> 152.9,69.46; KiCadOrientationDeg 90 -> 270
- DH111: FootprintOriginMm 171.86,133.5 -> 141.86,66.75
- DH112: BoardSide B.Cu -> F.Cu; FootprintOriginMm 171.85,135.25 -> 133.75,73.36; KiCadOrientationDeg 180 -> 270
- R101: FootprintOriginMm 176.64,136.91 -> 138.14,84.16
- R102: FootprintOriginMm 176.39,133.16 -> 148.64,69.66
- R103: FootprintOriginMm 167.91,133.89 -> 135.14,69.16; KiCadOrientationDeg 270 -> 0
- R104: BoardSide F.Cu -> B.Cu; FootprintOriginMm 170.64,116.41 -> 136.39,60.91; KiCadOrientationDeg 0 -> 180
- R109: FootprintOriginMm 176.91,133.89 -> 145.14,84.16; KiCadOrientationDeg 90 -> 180
- R110: BoardSide B.Cu -> F.Cu; FootprintOriginMm 182.64,125.16 -> 130.91,74.14; KiCadOrientationDeg 180 -> 270
- R111: FootprintOriginMm 167.39,136.91 -> 152.66,74.14; KiCadOrientationDeg 0 -> 270
- R112: FootprintOriginMm 178.66,123.14 -> 146.64,67.16; KiCadOrientationDeg 270 -> 0
- R113: BoardSide F.Cu -> B.Cu; FootprintOriginMm 159.91,134.89 -> 126.41,71.39; KiCadOrientationDeg 270 -> 90
- R122: FootprintOriginMm 157.91,128.89 -> 141.64,63.91; KiCadOrientationDeg 270 -> 0
- R123: FootprintOriginMm 167.66,115.64 -> 146.64,64.66; KiCadOrientationDeg 270 -> 0
- U101: FootprintOriginMm 154.8,130.72 -> 152.06,89.2; KiCadOrientationDeg 270 -> 90
- U103: FootprintOriginMm 171.87,128.88 -> 141.87,72.38
- U107: FootprintOriginMm 181.31,128.95 -> 135.47,86.81; KiCadOrientationDeg 270 -> 180
- U111: BoardSide F.Cu -> B.Cu; FootprintOriginMm 161.45,118.58 -> 130.7,90.18; KiCadOrientationDeg 90 -> 0
- U112: FootprintOriginMm 162.95,132.72 -> 152.72,78.93; KiCadOrientationDeg 270 -> 0
- U113: FootprintOriginMm 171.72,118.95 -> 130.72,78.93; KiCadOrientationDeg 180 -> 0
- U114: BoardSide F.Cu -> B.Cu; FootprintOriginMm 171.81,121.58 -> 141.84,67.08
- U115: FootprintOriginMm 171.72,128.95 -> 141.72,77.45
- U116: FootprintOriginMm 161.37,123.38 -> 141.87,89.61; KiCadOrientationDeg 180 -> 0
- U117: BoardSide F.Cu -> B.Cu; FootprintOriginMm 162.38,128.87 -> 151.61,66.87
- U118: FootprintOriginMm 181.11,116.23 -> 131.63,66.87; KiCadOrientationDeg 90 -> 270
- U119: BoardSide B.Cu -> F.Cu; FootprintOriginMm 161.47,115.2 -> 147.72,88.68

Commit message: WIP: same-footprint swap pass for the core placement (#43)
Ported span-penalized slot swaps (nets over 60 mm pay a quadratic
penalty), limited to same-footprint slots within 25 mm of each package's
net median. Floorplan proxy: HPWL 139 -> 105 m, median span 28.8 mm,
RUDY p99 0.78 with 68 tiles above 0.7 (JL with swaps: p99 0.81, 42).

Co-Authored-By: Claude Opus 5.5 <noreply@anthropic.com>
Parts:
- C101: BoardSide B.Cu -> F.Cu; FootprintOriginMm 158.71,75.39 -> 136.89,66.46; KiCadOrientationDeg 90 -> 0
- C102: BoardSide F.Cu -> B.Cu; FootprintOriginMm 136.89,66.46 -> 158.71,75.39; KiCadOrientationDeg 0 -> 90
- C104: BoardSide F.Cu -> B.Cu; FootprintOriginMm 149.9,73.46 -> 143.71,60.9; KiCadOrientationDeg 270 -> 180
- C105: BoardSide B.Cu -> F.Cu; FootprintOriginMm 143.71,60.9 -> 149.9,73.46; KiCadOrientationDeg 180 -> 270
- C106: BoardSide B.Cu -> F.Cu; FootprintOriginMm 157.15,70.71 -> 152.9,69.46; KiCadOrientationDeg 90 -> 270
- C148: BoardSide F.Cu -> B.Cu; FootprintOriginMm 152.9,69.46 -> 157.15,70.71; KiCadOrientationDeg 270 -> 90
- DH111: FootprintOriginMm 141.86,66.75 -> 133.75,73.36; KiCadOrientationDeg 0 -> 270
- DH112: BoardSide F.Cu -> B.Cu; FootprintOriginMm 133.75,73.36 -> 167.75,87.1; KiCadOrientationDeg 270 -> 90
- R101: BoardSide B.Cu -> F.Cu; FootprintOriginMm 138.14,84.16 -> 146.64,67.16; KiCadOrientationDeg 180 -> 0
- R103: FootprintOriginMm 135.14,69.16 -> 146.64,64.66
- R104: BoardSide B.Cu -> F.Cu; FootprintOriginMm 136.39,60.91 -> 141.64,63.91; KiCadOrientationDeg 180 -> 0
- R109: FootprintOriginMm 145.14,84.16 -> 126.41,71.39; KiCadOrientationDeg 180 -> 90
- R110: FootprintOriginMm 130.91,74.14 -> 135.14,69.16; KiCadOrientationDeg 270 -> 0
- R111: BoardSide F.Cu -> B.Cu; FootprintOriginMm 152.66,74.14 -> 145.14,84.16; KiCadOrientationDeg 270 -> 180
- R112: BoardSide F.Cu -> B.Cu; FootprintOriginMm 146.64,67.16 -> 138.14,84.16; KiCadOrientationDeg 0 -> 180
- R113: BoardSide B.Cu -> F.Cu; FootprintOriginMm 126.41,71.39 -> 130.91,74.14; KiCadOrientationDeg 90 -> 270
- R122: BoardSide F.Cu -> B.Cu; FootprintOriginMm 141.64,63.91 -> 170.66,94.39; KiCadOrientationDeg 0 -> 90
- R123: BoardSide F.Cu -> B.Cu; FootprintOriginMm 146.64,64.66 -> 136.39,60.91; KiCadOrientationDeg 0 -> 180
