File: boards/osc-core/sheets/sample_hold_H2_K.kicad_sch (KiCad schematic)
At the start: 53 parts, among them U201 REF5050AIDR, U203 OPA4197IPWR, U207 LM393BIDR, U211 SN74HC14DR, U212 OPA4196IDR, U213 OPA4196IDR, U214 CD74HC221M96, U215 LF398M/NOPB, U216 OPA4197IPWR, U217 OPA4197IPWR, U218 OPA4197IPWR, U219 OPA4196IDR

Commit message: Split jack partition into two boards with local bypass clusters
Parts:
- C201: FootprintOriginMm 163.64,142.71 -> 157.89,141.96
- C202: FootprintOriginMm 167.39,142.71 -> 161.64,141.96
- C204: FootprintOriginMm 76.21,135.4 -> 158.21,134.4
- C205: FootprintOriginMm 81.21,135.4 -> 163.21,134.4
- C206: FootprintOriginMm 86.21,135.4 -> 6.71,134.65
- C213: FootprintOriginMm 58.64,142.96 -> 180.39,142.71
- C216: FootprintOriginMm 32.39,143.21 -> 17.39,143.46
- C219: FootprintOriginMm 36.14,143.21 -> 21.14,143.46
- C220: FootprintOriginMm 39.89,143.21 -> 24.89,143.46
- C223: FootprintOriginMm 212.39,144.71 -> 129.14,144.21
- C224: FootprintOriginMm 144.89,145.21 -> 9.89,144.46
- C225: FootprintOriginMm 174.89,145.21 -> 121.39,144.96
- C228: FootprintOriginMm 178.64,145.21 -> 36.14,145.21
- C229: FootprintOriginMm 182.39,145.21 -> 39.89,145.21
- C231: FootprintOriginMm 231.14,145.21 -> 111.14,145.21
- C232: FootprintOriginMm 58.64,145.46 -> 187.89,145.21
- C233: FootprintOriginMm 81.14,145.46 -> 244.14,145.21
- C234: FootprintOriginMm 28.64,145.71 -> 21.14,145.96
- C235: FootprintOriginMm 107.39,145.96 -> 214.14,146.21
- C240: FootprintOriginMm 111.14,145.96 -> 217.89,146.21
- C241: FootprintOriginMm 114.89,145.96 -> 221.64,146.21
- C242: FootprintOriginMm 118.64,145.96 -> 225.39,146.21
- C243: FootprintOriginMm 122.39,145.96 -> 229.14,146.21
- C244: FootprintOriginMm 270.64,146.71 -> 232.89,146.21
- C245: FootprintOriginMm 281.89,146.71 -> 255.39,146.21
- C246: FootprintOriginMm 91.21,135.4 -> 125.71,134.9
- C247: FootprintOriginMm 96.21,135.4 -> 97.21,135.15
- C248: FootprintOriginMm 101.21,135.4 -> 119.71,135.15
- DH211: FootprintOriginMm 45.35,135.5 -> 288.1,134.0
- DH212: FootprintOriginMm 50.85,135.5 -> 12.35,134.25
- R201: FootprintOriginMm 152.39,180.41 -> 13.64,177.16
- R202: FootprintOriginMm 156.14,180.41 -> 17.39,177.16
- R203: FootprintOriginMm 159.89,180.41 -> 21.14,177.16
- R204: FootprintOriginMm 163.64,180.41 -> 24.89,177.16
- R209: FootprintOriginMm 167.39,180.41 -> 28.64,177.16
- R210: FootprintOriginMm 171.14,180.41 -> 92.39,177.16
- R211: FootprintOriginMm 189.89,180.41 -> 219.89,177.41
- R212: FootprintOriginMm 193.64,180.41 -> 246.14,177.41
- R213: FootprintOriginMm 127.64,180.91 -> 130.14,177.91
- R222: FootprintOriginMm 50.39,183.41 -> 253.64,180.16
- R223: FootprintOriginMm 300.64,183.41 -> 201.39,180.66
- U201: FootprintOriginMm 49.45,112.3 -> 143.7,112.3
- U203: FootprintOriginMm 256.1,99.38 -> 297.35,101.13
- U207: FootprintOriginMm 65.95,112.3 -> 186.45,112.3
- U216: FootprintOriginMm 230.35,101.63 -> 281.35,101.63
- U217: FootprintOriginMm 281.35,101.63 -> 305.6,102.13
- U218: FootprintOriginMm 305.6,102.13 -> 170.1,102.63
