File: boards/osc-core/sheets/sample_hold_H2_K.kicad_sch (KiCad schematic)
At the start: 53 parts, among them U201 REF5050AIDR, U203 OPA4197IPWR, U207 LM393BIDR, U211 SN74HC14DR, U212 OPA4196IDR, U213 OPA4196IDR, U214 CD74HC221M96, U215 LF398M/NOPB, U216 OPA4197IPWR, U217 OPA4197IPWR, U218 OPA4197IPWR, U219 OPA4196IDR

Commit message: WIP: locality placement source for the core board (#43)
Core packages are placed by the jack locality placer, anchored on the
core GH headers and pulled toward each module's own headers; IC/bypass
clusters stay rigid. Regenerated sources follow. Draft only.

Co-Authored-By: Claude Opus 5.5 <noreply@anthropic.com>
Parts:
- C201: FootprintOriginMm 157.89,141.96 -> 137.64,94.96
- C202: FootprintOriginMm 161.64,141.96 -> 143.64,97.46
- C204: FootprintOriginMm 158.21,134.4 -> 146.46,101.15
- C205: BoardSide B.Cu -> F.Cu; FootprintOriginMm 163.21,134.4 -> 137.71,100.15; KiCadOrientationDeg 180 -> 0
- C206: FootprintOriginMm 6.71,134.65 -> 153.15,113.71; KiCadOrientationDeg 180 -> 90
- C213: BoardSide B.Cu -> F.Cu; FootprintOriginMm 180.39,142.71 -> 147.245,105.96
- C216: FootprintOriginMm 17.39,143.46 -> 144.64,124.215; KiCadOrientationDeg 180 -> 0
- C219: FootprintOriginMm 21.14,143.46 -> 142.73,109.48; KiCadOrientationDeg 180 -> 90
- C220: FootprintOriginMm 24.89,143.46 -> 132.71,109.48; KiCadOrientationDeg 180 -> 90
- C223: BoardSide B.Cu -> F.Cu; FootprintOriginMm 129.14,144.21 -> 143.03,112.08; KiCadOrientationDeg 180 -> 270
- C224: BoardSide B.Cu -> F.Cu; FootprintOriginMm 9.89,144.46 -> 132.71,112.08; KiCadOrientationDeg 180 -> 270
- C225: FootprintOriginMm 121.39,144.96 -> 122.46,114.165; KiCadOrientationDeg 180 -> 270
- C228: BoardSide B.Cu -> F.Cu; FootprintOriginMm 36.14,145.21 -> 144.28,116.91; KiCadOrientationDeg 180 -> 90
- C229: BoardSide B.Cu -> F.Cu; FootprintOriginMm 39.89,145.21 -> 133.96,116.91; KiCadOrientationDeg 180 -> 90
- C231: BoardSide B.Cu -> F.Cu; FootprintOriginMm 111.14,145.21 -> 132.71,105.58; KiCadOrientationDeg 180 -> 270
- C232: BoardSide B.Cu -> F.Cu; FootprintOriginMm 187.89,145.21 -> 143.03,105.58; KiCadOrientationDeg 180 -> 270
- C233: FootprintOriginMm 244.14,145.21 -> 153.28,105.17999999999999; KiCadOrientationDeg 180 -> 90
- C234: FootprintOriginMm 21.14,145.96 -> 142.96,105.17999999999999; KiCadOrientationDeg 180 -> 90
- C235: FootprintOriginMm 214.14,146.21 -> 122.46,96.64; KiCadOrientationDeg 180 -> 90
- C240: FootprintOriginMm 217.89,146.21 -> 147.38,120.23; KiCadOrientationDeg 180 -> 0
- C241: FootprintOriginMm 221.64,146.21 -> 147.38,110.21; KiCadOrientationDeg 180 -> 0
- C242: FootprintOriginMm 225.39,146.21 -> 142.73,100.75; KiCadOrientationDeg 180 -> 90
- C243: FootprintOriginMm 229.14,146.21 -> 132.71,100.75; KiCadOrientationDeg 180 -> 90
- C244: BoardSide B.Cu -> F.Cu; FootprintOriginMm 232.89,146.21 -> 127.4,116.48; KiCadOrientationDeg 180 -> 0
- C245: BoardSide B.Cu -> F.Cu; FootprintOriginMm 255.39,146.21 -> 127.4,106.46; KiCadOrientationDeg 180 -> 0
- C246: FootprintOriginMm 125.71,134.9 -> 141.96,94.9
- C247: BoardSide B.Cu -> F.Cu; FootprintOriginMm 97.21,135.15 -> 127.9,102.71; KiCadOrientationDeg 180 -> 270
- C248: FootprintOriginMm 119.71,135.15 -> 151.46,101.15
- DH211: BoardSide B.Cu -> F.Cu; FootprintOriginMm 288.1,134.0 -> 147.0,117.86; KiCadOrientationDeg 180 -> 270
- DH212: FootprintOriginMm 12.35,134.25 -> 137.85,117.75
- R201: FootprintOriginMm 13.64,177.16 -> 132.66,105.64; KiCadOrientationDeg 180 -> 90
- R202: FootprintOriginMm 17.39,177.16 -> 143.91,121.14; KiCadOrientationDeg 180 -> 90
- R203: BoardSide B.Cu -> F.Cu; FootprintOriginMm 21.14,177.16 -> 130.41,105.64; KiCadOrientationDeg 180 -> 270
- R204: FootprintOriginMm 24.89,177.16 -> 132.66,96.89; KiCadOrientationDeg 180 -> 90
- R209: FootprintOriginMm 28.64,177.16 -> 132.66,113.14; KiCadOrientationDeg 180 -> 90
- R210: FootprintOriginMm 92.39,177.16 -> 151.14,110.16
- R211: BoardSide B.Cu -> F.Cu; FootprintOriginMm 219.89,177.41 -> 131.89,102.41; KiCadOrientationDeg 180 -> 0
- R212: BoardSide B.Cu -> F.Cu; FootprintOriginMm 246.14,177.41 -> 143.89,102.41; KiCadOrientationDeg 180 -> 0
- R213: BoardSide B.Cu -> F.Cu; FootprintOriginMm 130.14,177.91 -> 133.39,100.16; KiCadOrientationDeg 180 -> 0
- R222: FootprintOriginMm 253.64,180.16 -> 147.39,98.66
- R223: BoardSide B.Cu -> F.Cu; FootprintOriginMm 201.39,180.66 -> 142.14,100.16; KiCadOrientationDeg 180 -> 0
- U201: BoardSide B.Cu -> F.Cu; FootprintOriginMm 143.7,112.3 -> 147.31,110.97; KiCadOrientationDeg 180 -> 270
- U203: BoardSide B.Cu -> F.Cu; FootprintOriginMm 297.35,101.13 -> 137.87,111.38; KiCadOrientationDeg 180 -> 0
- U207: FootprintOriginMm 186.45,112.3 -> 138.95,122.31; KiCadOrientationDeg 180 -> 0
- U211: FootprintOriginMm 108.95,24.7 -> 127.47,101.15
- U212: FootprintOriginMm 170.95,24.7 -> 146.68,115.22; KiCadOrientationDeg 180 -> 90
- U213: FootprintOriginMm 178.7,24.7 -> 137.72,101.45
- U214: FootprintOriginMm 84.45,14.09 -> 127.47,111.56; KiCadOrientationDeg 180 -> 0
- U215: FootprintOriginMm 186.45,24.7 -> 137.72,111.45
- U216: BoardSide B.Cu -> F.Cu; FootprintOriginMm 281.35,101.63 -> 139.12,117.61
- U217: BoardSide B.Cu -> F.Cu; FootprintOriginMm 305.6,102.13 -> 137.87,104.88; KiCadOrientationDeg 180 -> 0
- U218: FootprintOriginMm 170.1,102.63 -> 148.12,105.88
- U219: BoardSide B.Cu -> F.Cu; FootprintOriginMm 194.2,24.7 -> 126.7,111.47; KiCadOrientationDeg 180 -> 90

Commit message: WIP: spread core module homes and legalize module by module (#43)
The first core negotiation stalled (2501/2727 nets in conflict after 7
iterations). A RUDY map showed placement congestion: header-anchored
homes crowded ~1300 E/A packages into one corner, so modules were
scattered and 751 nets spanned 80 mm or more. Module home discs are now
spread inside the outline and notch, packages are legalized one module
at a time, and the core uses a 0.6 mm courtyard gap with a 0.5 mm IC
channel. Floorplan proxy: HPWL 162 -> 139 m, peak RUDY 1.39 -> 1.09 of
ideal four-signal-layer supply, tiles above 0.7 682 -> 160.

Co-Authored-By: Claude Opus 5.5 <noreply@anthropic.com>
Parts:
- C201: BoardSide B.Cu -> F.Cu; FootprintOriginMm 137.64,94.96 -> 139.14,103.21; KiCadOrientationDeg 180 -> 0
- C202: BoardSide B.Cu -> F.Cu; FootprintOriginMm 143.64,97.46 -> 130.14,126.46; KiCadOrientationDeg 180 -> 0
- C204: BoardSide B.Cu -> F.Cu; FootprintOriginMm 146.46,101.15 -> 139.65,122.46; KiCadOrientationDeg 180 -> 270
- C205: BoardSide F.Cu -> B.Cu; FootprintOriginMm 137.71,100.15 -> 120.71,126.9; KiCadOrientationDeg 0 -> 180
- C206: BoardSide B.Cu -> F.Cu; FootprintOriginMm 153.15,113.71 -> 142.65,122.46; KiCadOrientationDeg 90 -> 270
- C213: BoardSide F.Cu -> B.Cu; FootprintOriginMm 147.245,105.96 -> 143.895,131.21; KiCadOrientationDeg 180 -> 0
- C216: BoardSide B.Cu -> F.Cu; FootprintOriginMm 144.64,124.215 -> 120.395,107.89; KiCadOrientationDeg 0 -> 90
- C219: FootprintOriginMm 142.73,109.48 -> 137.23,112.48
- C220: FootprintOriginMm 132.71,109.48 -> 127.21,112.48
- C223: FootprintOriginMm 143.03,112.08 -> 137.53,115.08
- C224: FootprintOriginMm 132.71,112.08 -> 127.21000000000001,115.08
- C225: FootprintOriginMm 122.46,114.165 -> 130.435,98.39; KiCadOrientationDeg 270 -> 90
- C228: FootprintOriginMm 144.28,116.91 -> 127.21000000000001,107.33; KiCadOrientationDeg 90 -> 270
- C229: FootprintOriginMm 133.96,116.91 -> 137.53,107.33; KiCadOrientationDeg 90 -> 270
- C231: BoardSide F.Cu -> B.Cu; FootprintOriginMm 132.71,105.58 -> 127.21000000000001,127.56
- C232: BoardSide F.Cu -> B.Cu; FootprintOriginMm 143.03,105.58 -> 137.53,127.56
- C233: FootprintOriginMm 153.28,105.17999999999999 -> 121.42999999999999,100.96000000000001; KiCadOrientationDeg 90 -> 180
- C234: FootprintOriginMm 142.96,105.17999999999999 -> 121.42999999999999,111.28; KiCadOrientationDeg 90 -> 180
- C235: BoardSide B.Cu -> F.Cu; FootprintOriginMm 122.46,96.64 -> 148.45999999999998,111.34; KiCadOrientationDeg 90 -> 270
- C240: FootprintOriginMm 147.38,120.23 -> 121.5,113.96; KiCadOrientationDeg 0 -> 180
- C241: FootprintOriginMm 147.38,110.21 -> 121.5,123.98; KiCadOrientationDeg 0 -> 180
- C242: FootprintOriginMm 142.73,100.75 -> 138.21,116.63000000000001; KiCadOrientationDeg 90 -> 270
- C243: FootprintOriginMm 132.71,100.75 -> 148.23,116.63000000000001; KiCadOrientationDeg 90 -> 270
- C244: BoardSide F.Cu -> B.Cu; FootprintOriginMm 127.4,116.48 -> 149.73,104.25; KiCadOrientationDeg 0 -> 90
- C245: BoardSide F.Cu -> B.Cu; FootprintOriginMm 127.4,106.46 -> 139.71,104.25; KiCadOrientationDeg 0 -> 90
- C246: BoardSide B.Cu -> F.Cu; FootprintOriginMm 141.96,94.9 -> 132.21,101.15; KiCadOrientationDeg 180 -> 0
- C247: BoardSide F.Cu -> B.Cu; FootprintOriginMm 127.9,102.71 -> 114.9,116.96; KiCadOrientationDeg 270 -> 90
- C248: FootprintOriginMm 151.46,101.15 -> 123.21,129.9
- DH211: FootprintOriginMm 147.0,117.86 -> 124.25,106.11
- DH212: BoardSide B.Cu -> F.Cu; FootprintOriginMm 137.85,117.75 -> 136.5,121.11; KiCadOrientationDeg 180 -> 270
- R201: FootprintOriginMm 132.66,105.64 -> 124.66,125.64
- R202: BoardSide B.Cu -> F.Cu; FootprintOriginMm 143.91,121.14 -> 133.41,125.14; KiCadOrientationDeg 90 -> 270
- R203: FootprintOriginMm 130.41,105.64 -> 140.16,106.64
- R204: FootprintOriginMm 132.66,96.89 -> 133.64,98.16; KiCadOrientationDeg 90 -> 180
- R209: FootprintOriginMm 132.66,113.14 -> 129.89,121.16; KiCadOrientationDeg 90 -> 180
- R210: FootprintOriginMm 151.14,110.16 -> 117.39,113.16
- R211: FootprintOriginMm 131.89,102.41 -> 135.91,125.89; KiCadOrientationDeg 0 -> 270
- R212: BoardSide F.Cu -> B.Cu; FootprintOriginMm 143.89,102.41 -> 116.91,109.89; KiCadOrientationDeg 0 -> 90
- R213: FootprintOriginMm 133.39,100.16 -> 142.66,106.64; KiCadOrientationDeg 0 -> 270
- R222: FootprintOriginMm 147.39,98.66 -> 149.16,112.39; KiCadOrientationDeg 180 -> 90
- R223: BoardSide F.Cu -> B.Cu; FootprintOriginMm 142.14,100.16 -> 124.66,99.39; KiCadOrientationDeg 0 -> 90
- U201: BoardSide F.Cu -> B.Cu; FootprintOriginMm 147.31,110.97 -> 142.56,126.2; KiCadOrientationDeg 270 -> 90
- U203: FootprintOriginMm 137.87,111.38 -> 132.37,114.38
- U207: BoardSide B.Cu -> F.Cu; FootprintOriginMm 138.95,122.31 -> 122.3,113.58; KiCadOrientationDeg 0 -> 90
- U211: BoardSide B.Cu -> F.Cu; FootprintOriginMm 127.47,101.15 -> 143.45,114.45; KiCadOrientationDeg 180 -> 0
- U212: FootprintOriginMm 146.68,115.22 -> 122.2,118.97; KiCadOrientationDeg 90 -> 270
- U213: FootprintOriginMm 137.72,101.45 -> 143.22,115.93; KiCadOrientationDeg 180 -> 0
- U214: FootprintOriginMm 127.47,111.56 -> 132.34,104.08; KiCadOrientationDeg 0 -> 270
- U215: FootprintOriginMm 137.72,111.45 -> 132.22,114.45
- U216: FootprintOriginMm 139.12,117.61 -> 132.37,106.63; KiCadOrientationDeg 180 -> 0
- U217: BoardSide F.Cu -> B.Cu; FootprintOriginMm 137.87,104.88 -> 132.37,126.86
- U218: FootprintOriginMm 148.12,105.88 -> 122.13,106.12; KiCadOrientationDeg 180 -> 270
- U219: BoardSide F.Cu -> B.Cu; FootprintOriginMm 126.7,111.47 -> 144.72,104.95; KiCadOrientationDeg 90 -> 180

Commit message: WIP: same-footprint swap pass for the core placement (#43)
Ported span-penalized slot swaps (nets over 60 mm pay a quadratic
penalty), limited to same-footprint slots within 25 mm of each package's
net median. Floorplan proxy: HPWL 139 -> 105 m, median span 28.8 mm,
RUDY p99 0.78 with 68 tiles above 0.7 (JL with swaps: p99 0.81, 42).

Co-Authored-By: Claude Opus 5.5 <noreply@anthropic.com>
Parts:
- C201: BoardSide F.Cu -> B.Cu; FootprintOriginMm 139.14,103.21 -> 165.64,113.96; KiCadOrientationDeg 0 -> 180
- C204: FootprintOriginMm 139.65,122.46 -> 132.21,101.15; KiCadOrientationDeg 270 -> 0
- C205: BoardSide B.Cu -> F.Cu; FootprintOriginMm 120.71,126.9 -> 139.65,122.46; KiCadOrientationDeg 180 -> 270
- C246: BoardSide F.Cu -> B.Cu; FootprintOriginMm 132.21,101.15 -> 120.71,126.9; KiCadOrientationDeg 0 -> 180
- R201: BoardSide B.Cu -> F.Cu; FootprintOriginMm 124.66,125.64 -> 135.91,125.89; KiCadOrientationDeg 90 -> 270
- R203: BoardSide F.Cu -> B.Cu; FootprintOriginMm 140.16,106.64 -> 129.89,121.16; KiCadOrientationDeg 270 -> 180
- R204: FootprintOriginMm 133.64,98.16 -> 149.16,112.39; KiCadOrientationDeg 180 -> 90
- R209: FootprintOriginMm 129.89,121.16 -> 124.66,99.39; KiCadOrientationDeg 180 -> 90
- R210: FootprintOriginMm 117.39,113.16 -> 124.66,125.64; KiCadOrientationDeg 180 -> 90
- R211: BoardSide F.Cu -> B.Cu; FootprintOriginMm 135.91,125.89 -> 117.39,113.16; KiCadOrientationDeg 270 -> 180
- R222: BoardSide B.Cu -> F.Cu; FootprintOriginMm 149.16,112.39 -> 140.16,106.64; KiCadOrientationDeg 90 -> 270
- R223: FootprintOriginMm 124.66,99.39 -> 133.64,98.16; KiCadOrientationDeg 90 -> 180
