File: boards/osc-core/sheets/board_interfaces_K-p3.kicad_sch (KiCad schematic)
At the start: 24 parts, among them J900098 BM08B-GHS-TBT(LF)(SN), J900100 BM08B-GHS-TBT(LF)(SN), J900102 BM08B-GHS-TBT(LF)(SN), J900104 BM08B-GHS-TBT(LF)(SN), J900113 BM07B-GHS-TBT(LF)(SN), J900115 BM07B-GHS-TBT(LF)(SN), J900117 BM07B-GHS-TBT(LF)(SN), J900119 BM07B-GHS-TBT(LF)(SN), J900121 BM07B-GHS-TBT(LF)(SN), J900123 BM07B-GHS-TBT(LF)(SN), J900125 BM07B-GHS-TBT(LF)(SN), J900127 BM07B-GHS-TBT(LF)(SN), J900129 BM07B-GHS-TBT(LF)(SN), J900131 BM07B-GHS-TBT(LF)(SN), J900133 BM03B-GHS-TBT(LF)(SN), J900135 BM03B-GHS-TBT(LF)(SN), J900137 BM03B-GHS-TBT(LF)(SN), J900139 BM03B-GHS-TBT(LF)(SN), J900141 BM03B-GHS-TBT(LF)(SN), J900143 BM03B-GHS-TBT(LF)(SN), J900145 BM03B-GHS-TBT(LF)(SN), J900147 BM03B-GHS-TBT(LF)(SN), J900149 BM03B-GHS-TBT(LF)(SN), J900151 BM03B-GHS-TBT(LF)(SN)

Commit message: Split jack partition into two boards with local bypass clusters
Parts:
- removed J900098, J900100, J900102, J900104: BM08B-GHS-TBT(LF)(SN), zudo-osc-hole-field:JST_GH8_BM_TopEntry, symbol zudo-osc-hole-field:JST_GH8_BM
- added J900106, J900108, J900110, J900112: BM08B-GHS-TBT(LF)(SN), zudo-osc-hole-field:JST_GH8_BM_TopEntry, symbol zudo-osc-hole-field:JST_GH8_BM
Connections:
- net AGND: now also J900106.2, J900106.4, J900106.6, J900106.8, J900108.2, J900108.4, J900108.6, J900108.8, J900110.2, J900110.4, J900110.6, J900110.8, J900112.2, J900112.4
- net X1D6CB2C11B96B64481EB: now also J900110.5
- net X8B82B2EF48894A1D4808: now also J900112.1
- net XB1B3A0103F218310D268: now also J900110.7
- net XBA4A69FA6E9B2B2B3585: now also J900112.3
- new net X2235AA409133311006A2: J900106.5
- new net X7A887447F4726336445D: J900106.1
- new net X9476738BD551C8789386: J900108.3
- new net XA97921AE972567EF91DF: J900108.7
- new net XB9F7C7FAA057C204FF64: J900106.7
- new net XCE107A8A443162AB8037: J900110.3
- new net XE31A80290D2BC578861C: J900106.3
- new net XE429289AAEFEAA3661F7: J900108.5
- new net XECCA0B06CABC23AB233D: J900110.1
- new net XF12351C36A39088567FF: J900108.1

Commit message: Reassign paired control connectors and rebuild the routing seed
Parts:
- J900133: FootprintOriginMm 97.55,185.0 -> 114.55,255.0
- J900135: FootprintOriginMm 114.55,185.0 -> 216.55,269.0
- J900137: FootprintOriginMm 131.55,185.0 -> 216.55,283.0
- J900139: FootprintOriginMm 148.55,185.0 -> 233.55,269.0
- J900141: FootprintOriginMm 165.55,185.0 -> 233.55,283.0
- J900143: FootprintOriginMm 182.55,185.0 -> 250.55,269.0
- J900145: FootprintOriginMm 199.55,185.0 -> 233.55,255.0
- J900147: FootprintOriginMm 97.55,199.0 -> 199.55,283.0
- J900149: FootprintOriginMm 114.55,199.0 -> 199.55,269.0
- J900151: FootprintOriginMm 131.55,199.0 -> 250.55,283.0
Changed lines of the file:
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@@
     (property "BoardSide" "F.Cu" (at 165 160 0) (effects (font (size 1.27 1.27)) (hide yes)))
     (property "KiCadOrientationDeg" "90" (at 165 160 0) (effects (font (size 1.27 1.27)) (hide yes)))
-    (property "FootprintOriginMm" "97.55,185.0" (at 165 160 0) (effects (font (size 1.27 1.27)) (hide yes)))
+    (property "FootprintOriginMm" "114.55,255.0" (at 165 160 0) (effects (font (size 1.27 1.27)) (hide yes)))
     (property "Sensitive" "" (at 165 160 0) (effects (font (size 1.27 1.27)) (hide yes)))
     (pin "1")
@@
     (property "BoardSide" "F.Cu" (at 35 190 0) (effects (font (size 1.27 1.27)) (hide yes)))
     (property "KiCadOrientationDeg" "90" (at 35 190 0) (effects (font (size 1.27 1.27)) (hide yes)))
-    (property "FootprintOriginMm" "114.55,185.0" (at 35 190 0) (effects (font (size 1.27 1.27)) (hide yes)))
+    (property "FootprintOriginMm" "216.55,269.0" (at 35 190 0) (effects (font (size 1.27 1.27)) (hide yes)))
     (property "Sensitive" "" (at 35 190 0) (effects (font (size 1.27 1.27)) (hide yes)))
     (pin "1")
@@
     (property "BoardSide" "F.Cu" (at 100 190 0) (effects (font (size 1.27 1.27)) (hide yes)))
     (property "KiCadOrientationDeg" "90" (at 100 190 0) (effects (font (size 1.27 1.27)) (hide yes)))
-    (property "FootprintOriginMm" "131.55,185.0" (at 100 190 0) (effects (font (size 1.27 1.27)) (hide yes)))
+    (property "FootprintOriginMm" "216.55,283.0" (at 100 190 0) (effects (font (size 1.27 1.27)) (hide yes)))
     (property "Sensitive" "" (at 100 190 0) (effects (font (size 1.27 1.27)) (hide yes)))
     (pin "1")
@@
     (property "BoardSide" "F.Cu" (at 165 190 0) (effects (font (size 1.27 1.27)) (hide yes)))
     (property "KiCadOrientationDeg" "90" (at 165 190 0) (effects (font (size 1.27 1.27)) (hide yes)))
-    (property "FootprintOriginMm" "148.55,185.0" (at 165 190 0) (effects (font (size 1.27 1.27)) (hide yes)))
+    (property "FootprintOriginMm" "233.55,269.0" (at 165 190 0) (effects (font (size 1.27 1.27)) (hide yes)))
     (property "Sensitive" "" (at 165 190 0) (effects (font (size 1.27 1.27)) (hide yes)))
     (pin "1")
@@
     (property "BoardSide" "F.Cu" (at 35 220 0) (effects (font (size 1.27 1.27)) (hide yes)))
     (property "KiCadOrientationDeg" "90" (at 35 220 0) (effects (font (size 1.27 1.27)) (hide yes)))
-    (property "FootprintOriginMm" "165.55,185.0" (at 35 220 0) (effects (font (size 1.27 1.27)) (hide yes)))
+    (property "FootprintOriginMm" "233.55,283.0" (at 35 220 0) (effects (font (size 1.27 1.27)) (hide yes)))
     (property "Sensitive" "" (at 35 220 0) (effects (font (size 1.27 1.27)) (hide yes)))
     (pin "1")
@@
     (property "BoardSide" "F.Cu" (at 100 220 0) (effects (font (size 1.27 1.27)) (hide yes)))
     (property "KiCadOrientationDeg" "90" (at 100 220 0) (effects (font (size 1.27 1.27)) (hide yes)))
-    (property "FootprintOriginMm" "182.55,185.0" (at 100 220 0) (effects (font (size 1.27 1.27)) (hide yes)))
+    (property "FootprintOriginMm" "250.55,269.0" (at 100 220 0) (effects (font (size 1.27 1.27)) (hide yes)))
     (property "Sensitive" "" (at 100 220 0) (effects (font (size 1.27 1.27)) (hide yes)))
     (pin "1")
@@
     (property "BoardSide" "F.Cu" (at 165 220 0) (effects (font (size 1.27 1.27)) (hide yes)))
     (property "KiCadOrientationDeg" "90" (at 165 220 0) (effects (font (size 1.27 1.27)) (hide yes)))
-    (property "FootprintOriginMm" "199.55,185.0" (at 165 220 0) (effects (font (size 1.27 1.27)) (hide yes)))
+    (property "FootprintOriginMm" "233.55,255.0" (at 165 220 0) (effects (font (size 1.27 1.27)) (hide yes)))
     (property "Sensitive" "" (at 165 220 0) (effects (font (size 1.27 1.27)) (hide yes)))
     (pin "1")
@@
     (property "BoardSide" "F.Cu" (at 35 250 0) (effects (font (size 1.27 1.27)) (hide yes)))
     (property "KiCadOrientationDeg" "90" (at 35 250 0) (effects (font (size 1.27 1.27)) (hide yes)))
-    (property "FootprintOriginMm" "97.55,199.0" (at 35 250 0) (effects (font (size 1.27 1.27)) (hide yes)))
+    (property "FootprintOriginMm" "199.55,283.0" (at 35 250 0) (effects (font (size 1.27 1.27)) (hide yes)))
     (property "Sensitive" "" (at 35 250 0) (effects (font (size 1.27 1.27)) (hide yes)))
     (pin "1")
@@
     (property "BoardSide" "F.Cu" (at 100 250 0) (effects (font (size 1.27 1.27)) (hide yes)))
     (property "KiCadOrientationDeg" "90" (at 100 250 0) (effects (font (size 1.27 1.27)) (hide yes)))
-    (property "FootprintOriginMm" "114.55,199.0" (at 100 250 0) (effects (font (size 1.27 1.27)) (hide yes)))
+    (property "FootprintOriginMm" "199.55,269.0" (at 100 250 0) (effects (font (size 1.27 1.27)) (hide yes)))
     (property "Sensitive" "" (at 100 250 0) (effects (font (size 1.27 1.27)) (hide yes)))
     (pin "1")
@@
     (property "BoardSide" "F.Cu" (at 165 250 0) (effects (font (size 1.27 1.27)) (hide yes)))
     (property "KiCadOrientationDeg" "90" (at 165 250 0) (effects (font (size 1.27 1.27)) (hide yes)))
-    (property "FootprintOriginMm" "131.55,199.0" (at 165 250 0) (effects (font (size 1.27 1.27)) (hide yes)))
+    (property "FootprintOriginMm" "250.55,283.0" (at 165 250 0) (effects (font (size 1.27 1.27)) (hide yes)))
     (property "Sensitive" "" (at 165 250 0) (effects (font (size 1.27 1.27)) (hide yes)))
     (pin "1")
