File: boards/osc-core/sheets/board_interfaces_K-p5.kicad_sch (KiCad schematic)
At the start: 24 parts, among them J900201 BM03B-GHS-TBT(LF)(SN), J900203 BM03B-GHS-TBT(LF)(SN), J900205 BM03B-GHS-TBT(LF)(SN), J900207 BM03B-GHS-TBT(LF)(SN), J900209 BM03B-GHS-TBT(LF)(SN), J900211 BM03B-GHS-TBT(LF)(SN), J900213 BM03B-GHS-TBT(LF)(SN), J900215 BM03B-GHS-TBT(LF)(SN), J900217 BM03B-GHS-TBT(LF)(SN), J900219 BM03B-GHS-TBT(LF)(SN), J900221 BM03B-GHS-TBT(LF)(SN), J900223 BM03B-GHS-TBT(LF)(SN), J900225 BM03B-GHS-TBT(LF)(SN), J900227 BM03B-GHS-TBT(LF)(SN), J900229 BM03B-GHS-TBT(LF)(SN), J900231 BM03B-GHS-TBT(LF)(SN), J900233 BM03B-GHS-TBT(LF)(SN), J900235 BM03B-GHS-TBT(LF)(SN), J900237 BM03B-GHS-TBT(LF)(SN), J900239 BM03B-GHS-TBT(LF)(SN), J900241 BM03B-GHS-TBT(LF)(SN), J900243 BM03B-GHS-TBT(LF)(SN), J900245 BM03B-GHS-TBT(LF)(SN), J900247 BM03B-GHS-TBT(LF)(SN)

Commit message: Reassign paired control connectors and rebuild the routing seed
Parts:
- J900201: FootprintOriginMm 29.55,241.0 -> 250.55,192.0
- J900203: FootprintOriginMm 46.55,241.0 -> 284.55,192.0
- J900205: FootprintOriginMm 63.55,241.0 -> 301.55,241.0
- J900207: FootprintOriginMm 80.55,241.0 -> 301.55,206.0
- J900209: FootprintOriginMm 97.55,241.0 -> 182.55,185.0
- J900211: FootprintOriginMm 114.55,241.0 -> 97.55,199.0
- J900213: FootprintOriginMm 131.55,241.0 -> 114.55,213.0
- J900215: FootprintOriginMm 148.55,241.0 -> 97.55,255.0
- J900217: FootprintOriginMm 165.55,241.0 -> 97.55,227.0
- J900219: FootprintOriginMm 182.55,241.0 -> 114.55,185.0
- J900221: FootprintOriginMm 199.55,241.0 -> 114.55,199.0
- J900223: FootprintOriginMm 216.55,241.0 -> 97.55,213.0
- J900225: FootprintOriginMm 233.55,241.0 -> 114.55,241.0
- J900227: FootprintOriginMm 250.55,241.0 -> 114.55,227.0
- J900229: FootprintOriginMm 267.55,241.0 -> 131.55,185.0
- J900231: FootprintOriginMm 284.55,241.0 -> 131.55,199.0
- J900233: FootprintOriginMm 301.55,241.0 -> 148.55,213.0
- J900235: FootprintOriginMm 12.55,255.0 -> 131.55,241.0
- J900237: FootprintOriginMm 29.55,255.0 -> 97.55,241.0
- J900239: FootprintOriginMm 46.55,255.0 -> 165.55,185.0
- J900241: FootprintOriginMm 63.55,255.0 -> 216.55,219.75
- J900243: FootprintOriginMm 80.55,255.0 -> 148.55,185.0
- J900245: FootprintOriginMm 97.55,255.0 -> 182.55,199.0
- J900247: FootprintOriginMm 114.55,255.0 -> 182.55,227.0
