File: boards/osc-core/sheets/board_interfaces_K-p7.kicad_sch (KiCad schematic)
At the start: 24 parts, among them J900297 BM03B-GHS-TBT(LF)(SN), J900299 BM03B-GHS-TBT(LF)(SN), J900301 BM03B-GHS-TBT(LF)(SN), J900303 BM03B-GHS-TBT(LF)(SN), J900305 BM03B-GHS-TBT(LF)(SN), J900307 BM03B-GHS-TBT(LF)(SN), J900309 BM03B-GHS-TBT(LF)(SN), J900311 BM03B-GHS-TBT(LF)(SN), J900313 BM03B-GHS-TBT(LF)(SN), J900315 BM03B-GHS-TBT(LF)(SN), J900317 BM03B-GHS-TBT(LF)(SN), J900319 BM03B-GHS-TBT(LF)(SN), J900321 BM03B-GHS-TBT(LF)(SN), J900323 BM03B-GHS-TBT(LF)(SN), J900325 BM03B-GHS-TBT(LF)(SN), J900327 BM03B-GHS-TBT(LF)(SN), J900329 BM03B-GHS-TBT(LF)(SN), J900331 BM03B-GHS-TBT(LF)(SN), J900333 BM03B-GHS-TBT(LF)(SN), J900335 BM03B-GHS-TBT(LF)(SN), J900337 BM03B-GHS-TBT(LF)(SN), J900339 BM03B-GHS-TBT(LF)(SN), J900341 BM03B-GHS-TBT(LF)(SN), J900343 BM03B-GHS-TBT(LF)(SN)

Commit message: Reassign paired control connectors and rebuild the routing seed
Parts:
- J900297: FootprintOriginMm 63.55,283.0 -> 12.55,255.0
- J900299: FootprintOriginMm 80.55,283.0 -> 12.55,206.0
- J900301: FootprintOriginMm 131.55,283.0 -> 12.55,241.0
- J900303: FootprintOriginMm 148.55,283.0 -> 29.55,227.0
- J900305: FootprintOriginMm 165.55,283.0 -> 12.55,218.5
- J900307: FootprintOriginMm 182.55,283.0 -> 29.55,283.0
- J900309: FootprintOriginMm 199.55,283.0 -> 29.55,269.0
- J900311: FootprintOriginMm 216.55,283.0 -> 29.55,255.0
- J900313: FootprintOriginMm 233.55,283.0 -> 29.55,206.0
- J900315: FootprintOriginMm 250.55,283.0 -> 29.55,241.0
- J900317: FootprintOriginMm 12.55,206.0 -> 12.55,227.0
- J900319: FootprintOriginMm 12.55,218.5 -> 29.55,218.5
- J900321: FootprintOriginMm 29.55,206.0 -> 46.55,283.0
- J900323: FootprintOriginMm 29.55,218.5 -> 46.55,269.0
- J900325: FootprintOriginMm 46.55,206.0 -> 46.55,255.0
- J900327: FootprintOriginMm 46.55,218.5 -> 46.55,206.0
- J900329: FootprintOriginMm 63.55,206.0 -> 46.55,241.0
- J900331: FootprintOriginMm 63.55,218.5 -> 63.55,227.0
- J900333: FootprintOriginMm 80.55,206.0 -> 46.55,218.5
- J900335: FootprintOriginMm 80.55,218.5 -> 63.55,283.0
- J900337: FootprintOriginMm 216.55,192.0 -> 63.55,269.0
- J900339: FootprintOriginMm 216.55,206.0 -> 63.55,255.0
- J900341: FootprintOriginMm 216.55,219.75 -> 63.55,206.0
- J900343: FootprintOriginMm 233.55,192.0 -> 63.55,241.0
