File: boards/osc-jack-left/sheets/manual_ab_X2_JL.kicad_sch (KiCad schematic)
At the start: 47 parts, among them J1010 WQP518MA, J810 WQP518MA, J910 WQP518MA, U3401 ADG5412FBRUZ, U3402 ADG5412FBRUZ, U3404 OPA4196IDR, U3405 OPA4197IPWR

Commit message: Bind exact precision-feedback resistor and capacitor identities
Parts:
- C3401: symbol zudo-osc-hole-field:C0603C101J5GACTU -> zudo-osc-hole-field:C0603C102J5GACTU; MPN (none) -> C0603C102J5GACTU; Manufacturer (none) -> KEMET
- R3416: symbol zudo-osc-hole-field:RC0603FR-07100KL -> zudo-osc-hole-field:RC0603FR-07100RL; MPN (none) -> RC0603FR-07100RL; Manufacturer (none) -> Yageo
Changed lines of the file:
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@@
   (global_label "X0F7C99D2BDE4560E0201" (shape passive) (at 802.64 104.14 0) (effects (font (size 1.27 1.27)) (justify right)))
   (global_label "X89EBA6E48D6DD31A4A9C" (shape passive) (at 812.8 104.14 180) (effects (font (size 1.27 1.27)) (justify left)))
-  (symbol (lib_id "zudo-osc-hole-field:RC0603FR-07100KL") (at 871.22 104.14 0) (unit 0)
+  (symbol (lib_id "zudo-osc-hole-field:RC0603FR-07100RL") (at 871.22 104.14 0) (unit 0)
     (exclude_from_sim no) (in_bom yes) (on_board yes) (dnp no)
     (property "Reference" "R3416" (at 874.22 101.14 0) (effects (font (size 1.27 1.27))))
@@
     (property "Footprint" "zudo-osc-hole-field:R0603" (at 871.22 104.14 0) (effects (font (size 1.27 1.27)) (hide yes)))
     (property "Datasheet" "" (at 871.22 104.14 0) (effects (font (size 1.27 1.27)) (hide yes)))
-    (property "MPN" "" (at 871.22 104.14 0) (effects (font (size 1.27 1.27)) (hide yes)))
-    (property "Manufacturer" "" (at 871.22 104.14 0) (effects (font (size 1.27 1.27)) (hide yes)))
+    (property "MPN" "RC0603FR-07100RL" (at 871.22 104.14 0) (effects (font (size 1.27 1.27)) (hide yes)))
+    (property "Manufacturer" "Yageo" (at 871.22 104.14 0) (effects (font (size 1.27 1.27)) (hide yes)))
     (property "LCSC" "" (at 871.22 104.14 0) (effects (font (size 1.27 1.27)) (hide yes)))
     (property "Block" "${SHEETNAME}" (at 871.22 104.14 0) (effects (font (size 1.27 1.27)) (hide yes)))
@@
   (global_label "X89EBA6E48D6DD31A4A9C" (shape passive) (at 866.14 104.14 0) (effects (font (size 1.27 1.27)) (justify right)))
   (global_label "X22F3FFA9E72A45A73A4D" (shape passive) (at 876.3 104.14 180) (effects (font (size 1.27 1.27)) (justify left)))
-  (symbol (lib_id "zudo-osc-hole-field:C0603C101J5GACTU") (at 934.72 104.14 0) (unit 0)
+  (symbol (lib_id "zudo-osc-hole-field:C0603C102J5GACTU") (at 934.72 104.14 0) (unit 0)
     (exclude_from_sim no) (in_bom yes) (on_board yes) (dnp no)
     (property "Reference" "C3401" (at 937.72 101.14 0) (effects (font (size 1.27 1.27))))
@@
     (property "Footprint" "zudo-osc-hole-field:C0603" (at 934.72 104.14 0) (effects (font (size 1.27 1.27)) (hide yes)))
     (property "Datasheet" "" (at 934.72 104.14 0) (effects (font (size 1.27 1.27)) (hide yes)))
-    (property "MPN" "" (at 934.72 104.14 0) (effects (font (size 1.27 1.27)) (hide yes)))
-    (property "Manufacturer" "" (at 934.72 104.14 0) (effects (font (size 1.27 1.27)) (hide yes)))
+    (property "MPN" "C0603C102J5GACTU" (at 934.72 104.14 0) (effects (font (size 1.27 1.27)) (hide yes)))
+    (property "Manufacturer" "KEMET" (at 934.72 104.14 0) (effects (font (size 1.27 1.27)) (hide yes)))
     (property "LCSC" "" (at 934.72 104.14 0) (effects (font (size 1.27 1.27)) (hide yes)))
     (property "Block" "${SHEETNAME}" (at 934.72 104.14 0) (effects (font (size 1.27 1.27)) (hide yes)))
