File: boards/osc-jack-left/sheets/manual_ab_X2_JL.kicad_sch (KiCad schematic)
At the start: 47 parts, among them J1010 WQP518MA, J810 WQP518MA, J910 WQP518MA, U3401 ADG5412FBRUZ, U3402 ADG5412FBRUZ, U3404 OPA4196IDR, U3405 OPA4197IPWR

Commit message: Move jack halves to six layers with locality placement and grid routing
Owner decision 2026-10-03 (#38): a cut-line bound showed the four-layer
jack halves could not carry their signal nets with intact planes, so both
halves move to six layers and their free packages are re-placed for
locality.

- Placement: scripts/checks/jack_locality.py replaces the
  connectivity-blind first-fit J placer. Packages are pulled toward the
  fixed jacks, LEDs and headers on their nets and toward their own
  module's hardware, then legalized; IC/bypass clusters stay aligned.
  Panel hardware and headers do not move.
- Stack: F/In2/In3/B signals, In1 AGND plane, -12V fill on In3, +12V
  plane on In4; +5V as tracks.
- Routing: scripts/pcbgen/route_jack_grid.py stages terminal arrays,
  rail fanouts and links, signal batches, rip-up-and-reroute and AGND
  stitching, keeping only natively checked stages (0 DRC errors,
  0 parity). The grid router gains N-layer support, windowed search,
  plane fanout, a plane-fill split guard and rip-up-and-reroute.
- Evidence chain: a bounded jack-locality partition transition is
  chained onto the connector-locality proof; superseded four-layer
  stage reports are removed.

Checkpoint: JL 411 and JR 518 native open edges remain. This is a routed
draft in progress; electrical and physical qualification NOT RUN.

Co-Authored-By: Claude Opus 5.5 <noreply@anthropic.com>
Parts:
- C3401: FootprintOriginMm 10.84,25.26 -> 157.23999999999998,162.36
- C3402: FootprintOriginMm 118.96000000000001,110.955 -> 147.67000000000002,117.90500000000002; KiCadOrientationDeg 90 -> 270
- C3403: FootprintOriginMm 129.87,110.955 -> 136.76000000000002,117.90500000000002; KiCadOrientationDeg 90 -> 270
- C3404: BoardSide B.Cu -> F.Cu; FootprintOriginMm 135.96,110.955 -> 141.605,126.27; KiCadOrientationDeg 90 -> 180
- C3405: BoardSide B.Cu -> F.Cu; FootprintOriginMm 146.87,110.955 -> 141.605,115.36; KiCadOrientationDeg 90 -> 180
- C3408: BoardSide B.Cu -> F.Cu; FootprintOriginMm 27.28,140.63 -> 159.13,155.51999999999998; KiCadOrientationDeg 90 -> 270
- C3409: BoardSide B.Cu -> F.Cu; FootprintOriginMm 16.96,140.63 -> 159.13,143.83999999999997
- C3410: FootprintOriginMm 162.98,55.65 -> 147.67999999999998,124.55
- C3411: FootprintOriginMm 152.96,55.65 -> 137.66,124.55
- D3401: BoardSide B.Cu -> F.Cu; FootprintOriginMm 132.23000000000002,56.910000000000004 -> 109.03,125.41; KiCadOrientationDeg 180 -> 0
- D3402: FootprintOriginMm 149.23000000000002,56.910000000000004 -> 108.81,116.23; KiCadOrientationDeg 180 -> 90
- D3403: BoardSide B.Cu -> F.Cu; FootprintOriginMm 163.35,50.050000000000004 -> 158.21,158.85; KiCadOrientationDeg 90 -> 0
- D3404: BoardSide B.Cu -> F.Cu; FootprintOriginMm 10.45,61.050000000000004 -> 158.21,161.75; KiCadOrientationDeg 90 -> 0
- D3405: BoardSide B.Cu -> F.Cu; FootprintOriginMm 45.25,85.75 -> 143.75,155.01000000000002; KiCadOrientationDeg 90 -> 270
- D3406: BoardSide B.Cu -> F.Cu; FootprintOriginMm 62.25,85.75 -> 143.75,160.41000000000003; KiCadOrientationDeg 90 -> 270
- D3408: BoardSide B.Cu -> F.Cu; FootprintOriginMm 79.25,85.75 -> 140.85,158.51000000000002; KiCadOrientationDeg 90 -> 270
- D3409: FootprintOriginMm 96.25,85.75 -> 130.35,136.65
- D3410: FootprintOriginMm 113.25,85.75 -> 135.85,128.85; KiCadOrientationDeg 90 -> 180
- D3411: FootprintOriginMm 130.25,85.75 -> 130.35,131.25
- D3413: FootprintOriginMm 147.25,85.75 -> 117.95,155.45
- D3414: BoardSide B.Cu -> F.Cu; FootprintOriginMm 164.25,85.75 -> 126.75,137.91000000000003; KiCadOrientationDeg 90 -> 270
- D3415: FootprintOriginMm 10.45,89.05 -> 130.45,127.25; KiCadOrientationDeg 90 -> 180
- D3416: FootprintOriginMm 30.45,99.44999999999999 -> 153.55,116.85
- R3401: FootprintOriginMm 106.24,39.51 -> 153.54,162.51
- R3402: FootprintOriginMm 123.24,39.51 -> 149.83999999999997,162.51
- R3403: FootprintOriginMm 140.23999999999998,39.51 -> 162.64,162.51
- R3404: BoardSide F.Cu -> B.Cu; FootprintOriginMm 157.23999999999998,39.51 -> 149.83999999999997,162.31; KiCadOrientationDeg 0 -> 180
- R3405: BoardSide F.Cu -> B.Cu; FootprintOriginMm 5.9399999999999995,40.809999999999995 -> 168.33999999999997,162.31; KiCadOrientationDeg 0 -> 180
- R3406: FootprintOriginMm 72.24,40.809999999999995 -> 166.33999999999997,162.51
- R3407: FootprintOriginMm 89.24,40.809999999999995 -> 140.44,162.21
- R3408: BoardSide F.Cu -> B.Cu; FootprintOriginMm 21.240000000000002,41.51 -> 160.94,162.31; KiCadOrientationDeg 0 -> 180
- R3414: FootprintOriginMm 69.27,31.900000000000002 -> 122.5,127.67; KiCadOrientationDeg 180 -> 90
- R3415: BoardSide B.Cu -> F.Cu; FootprintOriginMm 74.17,31.900000000000002 -> 123.5,137.27; KiCadOrientationDeg 180 -> 270
- R3416: BoardSide F.Cu -> B.Cu; FootprintOriginMm 38.24,41.51 -> 153.54,162.31; KiCadOrientationDeg 0 -> 180
- R3417: BoardSide F.Cu -> B.Cu; FootprintOriginMm 55.24,41.51 -> 135.04,162.31; KiCadOrientationDeg 0 -> 180
- R3418: FootprintOriginMm 108.74,41.709999999999994 -> 136.73999999999998,162.51
- R3419: FootprintOriginMm 125.74,41.709999999999994 -> 173.51,146.44; KiCadOrientationDeg 0 -> 270
- U3401: FootprintOriginMm 124.12,111.98 -> 142.51000000000002,116.88000000000001; KiCadOrientationDeg 180 -> 0
- U3402: BoardSide B.Cu -> F.Cu; FootprintOriginMm 141.12,111.98 -> 141.98,121.11; KiCadOrientationDeg 180 -> 270
- U3404: FootprintOriginMm 157.97,56.35 -> 142.67,125.25
- U3405: BoardSide B.Cu -> F.Cu; FootprintOriginMm 22.12,141.32999999999998 -> 159.13,149.67999999999998; KiCadOrientationDeg 180 -> 90

Commit message: Place jack halves with span-aware swaps and route jack-left to 173 open edges
Co-Authored-By: Claude Opus 5.5 <noreply@anthropic.com>
Parts:
- D3401: BoardSide F.Cu -> B.Cu; FootprintOriginMm 109.03,125.41 -> 118.71000000000001,128.13; KiCadOrientationDeg 0 -> 90
- D3402: BoardSide B.Cu -> F.Cu; FootprintOriginMm 108.81,116.23 -> 109.03,125.41; KiCadOrientationDeg 90 -> 0
- D3403: FootprintOriginMm 158.21,158.85 -> 142.61,150.15
- D3404: FootprintOriginMm 158.21,161.75 -> 140.85,158.51000000000002; KiCadOrientationDeg 0 -> 270
- D3406: BoardSide F.Cu -> B.Cu; FootprintOriginMm 143.75,160.41000000000003 -> 117.95,155.45; KiCadOrientationDeg 270 -> 90
- D3408: BoardSide F.Cu -> B.Cu; FootprintOriginMm 140.85,158.51000000000002 -> 130.45,127.25; KiCadOrientationDeg 270 -> 180
- D3409: FootprintOriginMm 130.35,136.65 -> 153.55,122.25
- D3411: FootprintOriginMm 130.35,131.25 -> 150.04999999999998,128.85; KiCadOrientationDeg 90 -> 180
- D3413: BoardSide B.Cu -> F.Cu; FootprintOriginMm 117.95,155.45 -> 143.75,160.41000000000003; KiCadOrientationDeg 90 -> 270
- D3414: FootprintOriginMm 126.75,137.91000000000003 -> 158.21,161.75; KiCadOrientationDeg 270 -> 0
- D3415: BoardSide B.Cu -> F.Cu; FootprintOriginMm 130.45,127.25 -> 158.21,158.85; KiCadOrientationDeg 180 -> 0
- D3416: FootprintOriginMm 153.55,116.85 -> 166.95,140.95; KiCadOrientationDeg 90 -> 180
- R3401: BoardSide F.Cu -> B.Cu; FootprintOriginMm 153.54,162.51 -> 149.83999999999997,162.31; KiCadOrientationDeg 0 -> 180
- R3403: FootprintOriginMm 162.64,162.51 -> 153.54,162.51
- R3404: FootprintOriginMm 149.83999999999997,162.31 -> 153.54,162.31
- R3405: BoardSide B.Cu -> F.Cu; FootprintOriginMm 168.33999999999997,162.31 -> 162.64,162.51; KiCadOrientationDeg 180 -> 0
- R3406: BoardSide F.Cu -> B.Cu; FootprintOriginMm 166.33999999999997,162.51 -> 164.64,162.31; KiCadOrientationDeg 0 -> 180
- R3407: BoardSide F.Cu -> B.Cu; FootprintOriginMm 140.44,162.21 -> 142.44,162.31; KiCadOrientationDeg 0 -> 180
- R3408: BoardSide B.Cu -> F.Cu; FootprintOriginMm 160.94,162.31 -> 140.44,162.21; KiCadOrientationDeg 180 -> 0
- R3415: BoardSide F.Cu -> B.Cu; FootprintOriginMm 123.5,137.27 -> 126.1,127.67; KiCadOrientationDeg 270 -> 90
- R3416: FootprintOriginMm 153.54,162.31 -> 160.94,162.31
- R3417: BoardSide B.Cu -> F.Cu; FootprintOriginMm 135.04,162.31 -> 136.73999999999998,162.51; KiCadOrientationDeg 180 -> 0
- R3418: BoardSide F.Cu -> B.Cu; FootprintOriginMm 136.73999999999998,162.51 -> 151.04,126.31; KiCadOrientationDeg 0 -> 180
- R3419: FootprintOriginMm 173.51,146.44 -> 166.33999999999997,162.51; KiCadOrientationDeg 270 -> 0

Commit message: Regenerate and rebuild both jack halves with the hot-quad escape reservation
Evidence rebound (peripheral epoch, foil-collar proposal, control receipt);
jack boards rebuilt from the new placement with source planes and no signal
copper, ready for CI routing.

Co-Authored-By: Claude Opus 5.5 <noreply@anthropic.com>
Parts:
- C3402: BoardSide B.Cu -> F.Cu; FootprintOriginMm 147.67000000000002,117.90500000000002 -> 142.30499999999998,155.51
- C3403: BoardSide B.Cu -> F.Cu; FootprintOriginMm 136.76000000000002,117.90500000000002 -> 142.30499999999998,143.23999999999998; KiCadOrientationDeg 270 -> 90
- C3404: FootprintOriginMm 141.605,126.27 -> 142.30499999999998,139.61; KiCadOrientationDeg 180 -> 270
- C3405: FootprintOriginMm 141.605,115.36 -> 142.30499999999998,127.34; KiCadOrientationDeg 180 -> 90
- C3408: BoardSide F.Cu -> B.Cu; FootprintOriginMm 159.13,155.51999999999998 -> 147.68,124.83; KiCadOrientationDeg 270 -> 90
- C3409: BoardSide F.Cu -> B.Cu; FootprintOriginMm 159.13,143.83999999999997 -> 137.36,124.83
- C3410: FootprintOriginMm 147.67999999999998,124.55 -> 147.67999999999998,115.45
- C3411: FootprintOriginMm 137.66,124.55 -> 137.66,115.45
- D3401: BoardSide B.Cu -> F.Cu; FootprintOriginMm 118.71000000000001,128.13 -> 109.21000000000001,117.33000000000001; KiCadOrientationDeg 90 -> 270
- D3402: FootprintOriginMm 109.03,125.41 -> 109.21000000000001,121.63000000000001; KiCadOrientationDeg 0 -> 270
- D3403: BoardSide F.Cu -> B.Cu; FootprintOriginMm 142.61,150.15 -> 117.95,155.45; KiCadOrientationDeg 0 -> 90
- D3404: FootprintOriginMm 140.85,158.51000000000002 -> 140.85,160.11
- D3405: FootprintOriginMm 143.75,155.01000000000002 -> 143.75,160.11
- D3406: BoardSide B.Cu -> F.Cu; FootprintOriginMm 117.95,155.45 -> 158.21,161.75; KiCadOrientationDeg 90 -> 0
- D3408: FootprintOriginMm 130.45,127.25 -> 128.95,115.25
- D3409: FootprintOriginMm 153.55,122.25 -> 123.55,115.05; KiCadOrientationDeg 90 -> 180
- D3410: BoardSide B.Cu -> F.Cu; FootprintOriginMm 135.85,128.85 -> 140.85,119.01; KiCadOrientationDeg 180 -> 270
- D3411: FootprintOriginMm 150.04999999999998,128.85 -> 136.95,119.85; KiCadOrientationDeg 180 -> 90
- D3413: FootprintOriginMm 143.75,160.41000000000003 -> 158.21,150.55; KiCadOrientationDeg 270 -> 0
- D3414: FootprintOriginMm 158.21,161.75 -> 158.21,158.85
- D3415: FootprintOriginMm 158.21,158.85 -> 158.21,147.65
- D3416: BoardSide B.Cu -> F.Cu; FootprintOriginMm 166.95,140.95 -> 159.35,154.81; KiCadOrientationDeg 180 -> 270
- R3401: FootprintOriginMm 149.83999999999997,162.31 -> 146.14,162.31
- R3402: FootprintOriginMm 149.83999999999997,162.51 -> 148.04,162.51
- R3403: BoardSide F.Cu -> B.Cu; FootprintOriginMm 153.54,162.51 -> 142.44,162.31; KiCadOrientationDeg 0 -> 180
- R3404: FootprintOriginMm 153.54,162.31 -> 138.73999999999998,162.31
- R3405: BoardSide F.Cu -> B.Cu; FootprintOriginMm 162.64,162.51 -> 149.83999999999997,162.31; KiCadOrientationDeg 0 -> 180
- R3406: BoardSide B.Cu -> F.Cu; FootprintOriginMm 164.64,162.31 -> 151.73999999999998,162.51; KiCadOrientationDeg 180 -> 0
- R3407: FootprintOriginMm 142.44,162.31 -> 136.01,136.83999999999997; KiCadOrientationDeg 180 -> 90
- R3408: BoardSide F.Cu -> B.Cu; FootprintOriginMm 140.44,162.21 -> 136.01,133.14; KiCadOrientationDeg 0 -> 90
- R3414: BoardSide B.Cu -> F.Cu; FootprintOriginMm 122.5,127.67 -> 125.77,123.5; KiCadOrientationDeg 90 -> 0
- R3415: BoardSide B.Cu -> F.Cu; FootprintOriginMm 126.1,127.67 -> 126.39999999999999,127.77; KiCadOrientationDeg 90 -> 270
- R3416: FootprintOriginMm 160.94,162.31 -> 153.54,162.31
- R3417: BoardSide F.Cu -> B.Cu; FootprintOriginMm 136.73999999999998,162.51 -> 160.94,162.31; KiCadOrientationDeg 0 -> 180
- R3418: BoardSide B.Cu -> F.Cu; FootprintOriginMm 151.04,126.31 -> 123.50999999999999,119.74; KiCadOrientationDeg 180 -> 270
- R3419: FootprintOriginMm 166.33999999999997,162.51 -> 162.64,162.51
- U3401: BoardSide B.Cu -> F.Cu; FootprintOriginMm 142.51000000000002,116.88000000000001 -> 141.98,149.67; KiCadOrientationDeg 0 -> 270
- U3402: FootprintOriginMm 141.98,121.11 -> 141.98,133.77
- U3404: FootprintOriginMm 142.67,125.25 -> 142.67,116.15
- U3405: BoardSide F.Cu -> B.Cu; FootprintOriginMm 159.13,149.67999999999998 -> 142.52,125.53; KiCadOrientationDeg 90 -> 180
