File: boards/osc-jack-left/sheets/mix5_M5B_JL.kicad_sch (KiCad schematic)
At the start: 106 parts, among them J1001 WQP518MA, J1002 WQP518MA, J1003 WQP518MA, J1004 WQP518MA, J1005 WQP518MA, J1006 WQP518MA, U8202 ADG5412FBRUZ, U8203 ADG5412FBRUZ, U8204 ADG5412FBRUZ, U8205 ADG5412FBRUZ, U8206 ADG5412FBRUZ, U8212 OPA4196IDR, U8213 LM393BIDR, U8214 LM393BIDR, U8215 OPA4196IDR, U8216 OPA4196IDR, U8217 OPA4196IDR

Commit message: Move jack halves to six layers with locality placement and grid routing
Owner decision 2026-10-03 (#38): a cut-line bound showed the four-layer
jack halves could not carry their signal nets with intact planes, so both
halves move to six layers and their free packages are re-placed for
locality.

- Placement: scripts/checks/jack_locality.py replaces the
  connectivity-blind first-fit J placer. Packages are pulled toward the
  fixed jacks, LEDs and headers on their nets and toward their own
  module's hardware, then legalized; IC/bypass clusters stay aligned.
  Panel hardware and headers do not move.
- Stack: F/In2/In3/B signals, In1 AGND plane, -12V fill on In3, +12V
  plane on In4; +5V as tracks.
- Routing: scripts/pcbgen/route_jack_grid.py stages terminal arrays,
  rail fanouts and links, signal batches, rip-up-and-reroute and AGND
  stitching, keeping only natively checked stages (0 DRC errors,
  0 parity). The grid router gains N-layer support, windowed search,
  plane fanout, a plane-fill split guard and rip-up-and-reroute.
- Evidence chain: a bounded jack-locality partition transition is
  chained onto the connector-locality proof; superseded four-layer
  stage reports are removed.

Checkpoint: JL 411 and JR 518 native open edges remain. This is a routed
draft in progress; electrical and physical qualification NOT RUN.

Co-Authored-By: Claude Opus 5.5 <noreply@anthropic.com>
Parts:
- C8215: BoardSide B.Cu -> F.Cu; FootprintOriginMm 65.76,127.35499999999999 -> 142.355,101.96000000000001; KiCadOrientationDeg 90 -> 0
- C8216: BoardSide B.Cu -> F.Cu; FootprintOriginMm 76.67,127.35499999999999 -> 142.355,112.87; KiCadOrientationDeg 90 -> 0
- C8217: FootprintOriginMm 82.76,127.35499999999999 -> 133.61,31.105; KiCadOrientationDeg 90 -> 0
- C8218: FootprintOriginMm 93.67,127.35499999999999 -> 121.34,31.105; KiCadOrientationDeg 90 -> 180
- C8219: FootprintOriginMm 99.76,127.35499999999999 -> 129.605,101.76; KiCadOrientationDeg 90 -> 0
- C8220: FootprintOriginMm 110.67,127.35499999999999 -> 129.605,112.67; KiCadOrientationDeg 90 -> 0
- C8221: FootprintOriginMm 116.76,127.35499999999999 -> 130.67,25.404999999999998; KiCadOrientationDeg 90 -> 270
- C8222: FootprintOriginMm 127.67,127.35499999999999 -> 119.75999999999999,25.404999999999998; KiCadOrientationDeg 90 -> 270
- C8223: FootprintOriginMm 135.96,130.15499999999997 -> 116.61000000000001,45.105; KiCadOrientationDeg 90 -> 0
- C8224: FootprintOriginMm 146.87,130.15499999999997 -> 104.34,45.105; KiCadOrientationDeg 90 -> 180
- C8225: BoardSide B.Cu -> F.Cu; FootprintOriginMm 67.96,139.84 -> 157.245,73.54
- C8226: BoardSide B.Cu -> F.Cu; FootprintOriginMm 77.98,143.65 -> 161.055,84.92; KiCadOrientationDeg 90 -> 270
- C8227: FootprintOriginMm 84.96,139.84 -> 154.66,44.94
- C8228: FootprintOriginMm 94.98,143.65 -> 164.67999999999998,48.74999999999999
- C8239: FootprintOriginMm 128.98,65.64999999999999 -> 166.88,28.85
- C8240: FootprintOriginMm 118.96,65.64999999999999 -> 156.86,28.85
- C8241: FootprintOriginMm 145.98,65.64999999999999 -> 154.66,88.78000000000002; KiCadOrientationDeg 90 -> 270
- C8242: FootprintOriginMm 135.96,65.64999999999999 -> 164.67999999999998,88.78000000000002; KiCadOrientationDeg 90 -> 270
- C8243: FootprintOriginMm 162.98,65.64999999999999 -> 161.38,61.779999999999994; KiCadOrientationDeg 90 -> 0
- C8244: FootprintOriginMm 152.96,65.64999999999999 -> 161.38,51.76; KiCadOrientationDeg 90 -> 0
- C8245: FootprintOriginMm 26.979999999999997,87.65 -> 149.88,28.85
- C8246: FootprintOriginMm 16.96,87.65 -> 139.86,28.85
- D8208: FootprintOriginMm 6.2299999999999995,124.21000000000001 -> 103.91,111.03; KiCadOrientationDeg 180 -> 90
- D8209: FootprintOriginMm 10.53,124.51 -> 95.81,32.230000000000004; KiCadOrientationDeg 180 -> 90
- D8210: FootprintOriginMm 167.13,126.91 -> 104.81,116.23; KiCadOrientationDeg 180 -> 90
- D8211: FootprintOriginMm 130.93,127.21000000000001 -> 95.81,27.93; KiCadOrientationDeg 180 -> 90
- D8212: FootprintOriginMm 6.2299999999999995,128.21 -> 95.81,105.33000000000001; KiCadOrientationDeg 180 -> 90
- D8213: FootprintOriginMm 107.21,21.55 -> 159.61,23.15
- D8214: BoardSide F.Cu -> B.Cu; FootprintOriginMm 124.21,21.55 -> 140.54999999999998,21.75; KiCadOrientationDeg 0 -> 180
- D8215: FootprintOriginMm 141.21,21.55 -> 142.61,25.05
- D8216: FootprintOriginMm 158.21,21.55 -> 142.61,22.15
- D8217: FootprintOriginMm 22.21,24.45 -> 126.75,33.51; KiCadOrientationDeg 0 -> 270
- D8218: BoardSide F.Cu -> B.Cu; FootprintOriginMm 39.21,24.45 -> 134.15,113.44999999999999; KiCadOrientationDeg 0 -> 90
- D8219: BoardSide F.Cu -> B.Cu; FootprintOriginMm 56.21,24.45 -> 123.95,105.35; KiCadOrientationDeg 0 -> 90
- D8220: FootprintOriginMm 73.21,24.45 -> 126.75,102.51; KiCadOrientationDeg 0 -> 270
- D8221: FootprintOriginMm 90.21,24.45 -> 123.85,33.51; KiCadOrientationDeg 0 -> 270
- D8222: BoardSide F.Cu -> B.Cu; FootprintOriginMm 107.21,24.45 -> 117.55,99.44999999999999; KiCadOrientationDeg 0 -> 90
- D8223: FootprintOriginMm 124.21,24.45 -> 126.75,28.11; KiCadOrientationDeg 0 -> 270
- D8224: BoardSide F.Cu -> B.Cu; FootprintOriginMm 141.21,24.45 -> 121.05,105.35; KiCadOrientationDeg 0 -> 90
- D8225: FootprintOriginMm 158.21,24.45 -> 123.85,102.51; KiCadOrientationDeg 0 -> 270
- D8226: BoardSide F.Cu -> B.Cu; FootprintOriginMm 22.21,27.35 -> 128.95,115.25; KiCadOrientationDeg 0 -> 180
- D8227: FootprintOriginMm 39.21,27.35 -> 125.61,106.55
- D8228: BoardSide F.Cu -> B.Cu; FootprintOriginMm 56.21,27.35 -> 123.95,110.75; KiCadOrientationDeg 0 -> 90
- D8229: BoardSide F.Cu -> B.Cu; FootprintOriginMm 73.21,27.35 -> 114.65,99.44999999999999; KiCadOrientationDeg 0 -> 90
- D8230: BoardSide F.Cu -> B.Cu; FootprintOriginMm 90.21,27.35 -> 116.64999999999999,30.85; KiCadOrientationDeg 0 -> 180
- D8231: FootprintOriginMm 22.21,30.25 -> 125.61,109.45
- D8232: FootprintOriginMm 39.21,30.25 -> 125.61,23.85
- D8233: BoardSide F.Cu -> B.Cu; FootprintOriginMm 56.21,30.25 -> 121.05,110.75; KiCadOrientationDeg 0 -> 90
- D8234: BoardSide F.Cu -> B.Cu; FootprintOriginMm 73.21,30.25 -> 111.75,98.05; KiCadOrientationDeg 0 -> 90
- D8235: BoardSide F.Cu -> B.Cu; FootprintOriginMm 90.21,30.25 -> 123.55,115.05; KiCadOrientationDeg 0 -> 180
- D8236: BoardSide F.Cu -> B.Cu; FootprintOriginMm 107.21,31.15 -> 112.65,31.55; KiCadOrientationDeg 0 -> 90
- R8205: FootprintOriginMm 89.24,51.809999999999995 -> 173.51,134.04; KiCadOrientationDeg 0 -> 270
- R8206: FootprintOriginMm 21.240000000000002,52.51 -> 173.51,137.73999999999998; KiCadOrientationDeg 0 -> 270
- R8207: BoardSide F.Cu -> B.Cu; FootprintOriginMm 38.24,52.51 -> 127.04,131.21; KiCadOrientationDeg 0 -> 180
- R8208: FootprintOriginMm 55.24,52.51 -> 173.51,66.84; KiCadOrientationDeg 0 -> 270
- R8215: FootprintOriginMm 106.24,52.709999999999994 -> 123.50999999999999,123.74; KiCadOrientationDeg 0 -> 270
- R8216: FootprintOriginMm 123.24,52.709999999999994 -> 105.81,105.64; KiCadOrientationDeg 0 -> 270
- R8217: BoardSide F.Cu -> B.Cu; FootprintOriginMm 140.23999999999998,52.709999999999994 -> 104.94,21.71; KiCadOrientationDeg 0 -> 180
- R8218: FootprintOriginMm 157.23999999999998,52.709999999999994 -> 173.51,63.14; KiCadOrientationDeg 0 -> 270
- R8225: FootprintOriginMm 5.9399999999999995,54.01 -> 126.34,127.41
- R8226: FootprintOriginMm 72.24,54.01 -> 123.41,127.44; KiCadOrientationDeg 0 -> 270
- R8227: FootprintOriginMm 89.24,54.01 -> 106.11,109.64; KiCadOrientationDeg 0 -> 270
- R8228: BoardSide F.Cu -> B.Cu; FootprintOriginMm 21.240000000000002,54.709999999999994 -> 170.31,76.14; KiCadOrientationDeg 0 -> 90
- R8235: FootprintOriginMm 38.24,54.709999999999994 -> 105.81,25.84; KiCadOrientationDeg 0 -> 270
- R8236: FootprintOriginMm 55.24,54.709999999999994 -> 106.11,22.14; KiCadOrientationDeg 0 -> 270
- R8237: BoardSide F.Cu -> B.Cu; FootprintOriginMm 108.74,54.91 -> 96.71,23.94; KiCadOrientationDeg 0 -> 90
- R8238: BoardSide F.Cu -> B.Cu; FootprintOriginMm 125.74,54.91 -> 170.31,55.74; KiCadOrientationDeg 0 -> 90
- R8245: FootprintOriginMm 142.73999999999998,54.91 -> 106.11,113.34; KiCadOrientationDeg 0 -> 270
- R8246: BoardSide F.Cu -> B.Cu; FootprintOriginMm 159.73999999999998,54.91 -> 92.71,32.54; KiCadOrientationDeg 0 -> 90
- R8247: BoardSide F.Cu -> B.Cu; FootprintOriginMm 5.9399999999999995,56.209999999999994 -> 100.81,112.74; KiCadOrientationDeg 0 -> 90
- R8248: FootprintOriginMm 72.24,56.209999999999994 -> 173.51,73.54; KiCadOrientationDeg 0 -> 270
- R8267: FootprintOriginMm 120.27,31.900000000000002 -> 117.8,113.36999999999999; KiCadOrientationDeg 180 -> 90
- R8268: BoardSide B.Cu -> F.Cu; FootprintOriginMm 125.17,31.900000000000002 -> 125.77,112.69999999999999; KiCadOrientationDeg 180 -> 0
- R8269: BoardSide F.Cu -> B.Cu; FootprintOriginMm 89.24,56.209999999999994 -> 96.71,109.34; KiCadOrientationDeg 0 -> 90
- R8270: FootprintOriginMm 21.240000000000002,56.91 -> 123.50999999999999,131.14; KiCadOrientationDeg 0 -> 270
- R8271: BoardSide F.Cu -> B.Cu; FootprintOriginMm 38.24,56.91 -> 98.61,113.04; KiCadOrientationDeg 0 -> 90
- R8272: FootprintOriginMm 55.24,56.91 -> 106.11,117.04; KiCadOrientationDeg 0 -> 270
- R8273: BoardSide F.Cu -> B.Cu; FootprintOriginMm 108.74,57.11 -> 92.71,28.84; KiCadOrientationDeg 0 -> 90
- R8274: BoardSide F.Cu -> B.Cu; FootprintOriginMm 125.74,57.11 -> 90.50999999999999,32.54; KiCadOrientationDeg 0 -> 90
- R8275: BoardSide F.Cu -> B.Cu; FootprintOriginMm 142.73999999999998,57.11 -> 170.31,79.84; KiCadOrientationDeg 0 -> 90
- R8276: FootprintOriginMm 159.73999999999998,57.11 -> 109.34,122.31
- R8277: BoardSide F.Cu -> B.Cu; FootprintOriginMm 5.9399999999999995,58.41 -> 170.31,83.94; KiCadOrientationDeg 0 -> 90
- U8202: BoardSide B.Cu -> F.Cu; FootprintOriginMm 70.92,128.38 -> 141.98,107.12; KiCadOrientationDeg 180 -> 90
- U8203: FootprintOriginMm 87.92,128.38 -> 127.77000000000001,30.78; KiCadOrientationDeg 180 -> 0
- U8204: FootprintOriginMm 104.92,128.38 -> 128.57999999999998,106.92; KiCadOrientationDeg 180 -> 90
- U8205: FootprintOriginMm 121.92,128.38 -> 125.50999999999999,24.38; KiCadOrientationDeg 180 -> 0
- U8206: FootprintOriginMm 141.12,131.17999999999998 -> 110.77000000000001,44.779999999999994; KiCadOrientationDeg 180 -> 0
- U8212: FootprintOriginMm 123.97,66.35 -> 161.87,29.55
- U8213: BoardSide B.Cu -> F.Cu; FootprintOriginMm 72.97,142.445 -> 159.15,79.23; KiCadOrientationDeg 180 -> 90
- U8214: FootprintOriginMm 89.97,142.445 -> 159.67,47.544999999999995
- U8215: FootprintOriginMm 140.97,66.35 -> 159.67,88.08000000000001; KiCadOrientationDeg 180 -> 0
- U8216: FootprintOriginMm 157.97,66.35 -> 160.68,56.769999999999996; KiCadOrientationDeg 180 -> 90
- U8217: FootprintOriginMm 21.97,88.35000000000001 -> 144.87,29.55

Commit message: Route jack-left with negotiated congestion to 360 open edges
Locality placement with a 0.8 mm IC keep-clear ring on JL (JR keeps none),
a native C grid A*, a PathFinder negotiated-congestion stage on a 0.05 mm
grid, then rip-up-and-reroute and AGND stitching. Native: 360 open edges
(main 411), 0 DRC errors, 0 schematic parity findings. Routed draft;
electrical/physical qualification NOT RUN.

Co-Authored-By: Claude Opus 5.5 <noreply@anthropic.com>
Parts:
- C8215: FootprintOriginMm 142.355,101.96000000000001 -> 125.355,87.66000000000001
- C8216: FootprintOriginMm 142.355,112.87 -> 125.355,98.57000000000001
- C8217: FootprintOriginMm 133.61,31.105 -> 128.805,103.96000000000001
- C8218: FootprintOriginMm 121.34,31.105 -> 128.805,114.87; KiCadOrientationDeg 180 -> 0
- C8219: BoardSide B.Cu -> F.Cu; FootprintOriginMm 129.605,101.76 -> 125.355,100.86000000000001
- C8220: BoardSide B.Cu -> F.Cu; FootprintOriginMm 129.605,112.67 -> 125.355,111.77000000000001
- C8221: FootprintOriginMm 130.67,25.404999999999998 -> 115.81,30.705000000000002; KiCadOrientationDeg 270 -> 0
- C8222: FootprintOriginMm 119.75999999999999,25.404999999999998 -> 103.53999999999999,30.705000000000002; KiCadOrientationDeg 270 -> 180
- C8223: BoardSide B.Cu -> F.Cu; FootprintOriginMm 116.61000000000001,45.105 -> 108.305,55.61; KiCadOrientationDeg 0 -> 270
- C8224: BoardSide B.Cu -> F.Cu; FootprintOriginMm 104.34,45.105 -> 108.305,43.34; KiCadOrientationDeg 180 -> 90
- C8227: FootprintOriginMm 154.66,44.94 -> 152.54000000000002,43.345; KiCadOrientationDeg 90 -> 180
- C8228: FootprintOriginMm 164.67999999999998,48.74999999999999 -> 163.92000000000002,47.155; KiCadOrientationDeg 90 -> 0
- C8239: FootprintOriginMm 166.88,28.85 -> 166.82000000000002,28.75; KiCadOrientationDeg 90 -> 0
- C8240: FootprintOriginMm 156.86,28.85 -> 155.44000000000003,28.75; KiCadOrientationDeg 90 -> 180
- C8241: FootprintOriginMm 154.66,88.78000000000002 -> 154.66,89.58000000000001
- C8242: FootprintOriginMm 164.67999999999998,88.78000000000002 -> 164.67999999999998,89.58000000000001
- C8243: FootprintOriginMm 161.38,61.779999999999994 -> 164.67999999999998,54.349999999999994; KiCadOrientationDeg 0 -> 90
- C8244: FootprintOriginMm 161.38,51.76 -> 154.66,54.349999999999994; KiCadOrientationDeg 0 -> 90
- C8245: FootprintOriginMm 149.88,28.85 -> 137.66,101.18; KiCadOrientationDeg 90 -> 270
- C8246: FootprintOriginMm 139.86,28.85 -> 147.67999999999998,101.18; KiCadOrientationDeg 90 -> 270
- D8208: FootprintOriginMm 103.91,111.03 -> 78.11,27.93
- D8209: FootprintOriginMm 95.81,32.230000000000004 -> 78.81,108.53
- D8210: FootprintOriginMm 104.81,116.23 -> 78.81,23.63
- D8211: FootprintOriginMm 95.81,27.93 -> 74.11,32.230000000000004
- D8212: FootprintOriginMm 95.81,105.33000000000001 -> 80.31,113.03
- D8213: BoardSide F.Cu -> B.Cu; FootprintOriginMm 159.61,23.15 -> 120.94999999999999,112.55; KiCadOrientationDeg 0 -> 180
- D8214: BoardSide B.Cu -> F.Cu; FootprintOriginMm 140.54999999999998,21.75 -> 125.61,114.35; KiCadOrientationDeg 180 -> 0
- D8215: BoardSide F.Cu -> B.Cu; FootprintOriginMm 142.61,25.05 -> 110.25,101.75; KiCadOrientationDeg 0 -> 90
- D8216: FootprintOriginMm 142.61,22.15 -> 109.75,38.91; KiCadOrientationDeg 0 -> 270
- D8217: BoardSide F.Cu -> B.Cu; FootprintOriginMm 126.75,33.51 -> 116.95,113.44999999999999; KiCadOrientationDeg 270 -> 90
- D8218: BoardSide B.Cu -> F.Cu; FootprintOriginMm 134.15,113.44999999999999 -> 125.61,117.25; KiCadOrientationDeg 90 -> 0
- D8219: FootprintOriginMm 123.95,105.35 -> 113.35,23.55
- D8220: BoardSide F.Cu -> B.Cu; FootprintOriginMm 126.75,102.51 -> 107.35,101.75; KiCadOrientationDeg 270 -> 90
- D8221: FootprintOriginMm 123.85,33.51 -> 109.75,98.01
- D8222: BoardSide B.Cu -> F.Cu; FootprintOriginMm 117.55,99.44999999999999 -> 109.75,33.51; KiCadOrientationDeg 90 -> 270
- D8223: FootprintOriginMm 126.75,28.11 -> 106.85,38.91
- D8224: BoardSide B.Cu -> F.Cu; FootprintOriginMm 121.05,105.35 -> 125.61,120.15; KiCadOrientationDeg 90 -> 0
- D8225: BoardSide F.Cu -> B.Cu; FootprintOriginMm 123.85,102.51 -> 110.45,23.55; KiCadOrientationDeg 270 -> 90
- D8226: FootprintOriginMm 128.95,115.25 -> 104.45,101.75; KiCadOrientationDeg 180 -> 90
- D8227: FootprintOriginMm 125.61,106.55 -> 106.85,98.01; KiCadOrientationDeg 0 -> 270
- D8228: BoardSide B.Cu -> F.Cu; FootprintOriginMm 123.95,110.75 -> 109.75,103.41; KiCadOrientationDeg 90 -> 270
- D8229: BoardSide B.Cu -> F.Cu; FootprintOriginMm 114.65,99.44999999999999 -> 125.61,123.05; KiCadOrientationDeg 90 -> 0
- D8230: BoardSide B.Cu -> F.Cu; FootprintOriginMm 116.64999999999999,30.85 -> 106.85,33.51; KiCadOrientationDeg 180 -> 270
- D8231: FootprintOriginMm 125.61,109.45 -> 109.75,28.11; KiCadOrientationDeg 0 -> 270
- D8232: BoardSide F.Cu -> B.Cu; FootprintOriginMm 125.61,23.85 -> 107.55,23.55; KiCadOrientationDeg 0 -> 90
- D8233: FootprintOriginMm 121.05,110.75 -> 121.35,126.65; KiCadOrientationDeg 90 -> 180
- D8234: BoardSide B.Cu -> F.Cu; FootprintOriginMm 111.75,98.05 -> 106.85,103.41; KiCadOrientationDeg 90 -> 270
- D8235: FootprintOriginMm 123.55,115.05 -> 100.14999999999999,99.45
- D8236: BoardSide B.Cu -> F.Cu; FootprintOriginMm 112.65,31.55 -> 109.75,108.81; KiCadOrientationDeg 90 -> 270
- R8205: FootprintOriginMm 173.51,134.04 -> 173.51,147.23999999999998
- R8206: FootprintOriginMm 173.51,137.73999999999998 -> 173.51,150.94
- R8207: BoardSide B.Cu -> F.Cu; FootprintOriginMm 127.04,131.21 -> 109.34,122.50999999999999; KiCadOrientationDeg 180 -> 0
- R8215: FootprintOriginMm 123.50999999999999,123.74 -> 106.41,120.14
- R8216: FootprintOriginMm 105.81,105.64 -> 89.11,110.24
- R8217: BoardSide B.Cu -> F.Cu; FootprintOriginMm 104.94,21.71 -> 173.51,157.54; KiCadOrientationDeg 180 -> 270
- R8218: BoardSide F.Cu -> B.Cu; FootprintOriginMm 173.51,63.14 -> 170.31,74.24; KiCadOrientationDeg 270 -> 90
- R8225: FootprintOriginMm 126.34,127.41 -> 89.50999999999999,32.24; KiCadOrientationDeg 0 -> 270
- R8226: FootprintOriginMm 123.41,127.44 -> 88.81,28.54
- R8227: FootprintOriginMm 106.11,109.64 -> 88.81,24.84
- R8228: BoardSide B.Cu -> F.Cu; FootprintOriginMm 170.31,76.14 -> 173.51,63.14; KiCadOrientationDeg 90 -> 270
- R8235: FootprintOriginMm 105.81,25.84 -> 89.11,113.94
- R8236: FootprintOriginMm 106.11,22.14 -> 76.11,40.14
- R8237: FootprintOriginMm 96.71,23.94 -> 75.00999999999999,28.240000000000002
- R8238: FootprintOriginMm 170.31,55.74 -> 169.54,56.309999999999995; KiCadOrientationDeg 90 -> 180
- R8245: FootprintOriginMm 106.11,113.34 -> 173.51,161.23999999999998
- R8246: BoardSide B.Cu -> F.Cu; FootprintOriginMm 92.71,32.54 -> 89.11,117.64; KiCadOrientationDeg 90 -> 270
- R8247: BoardSide B.Cu -> F.Cu; FootprintOriginMm 100.81,112.74 -> 89.11,121.34; KiCadOrientationDeg 90 -> 270
- R8267: FootprintOriginMm 117.8,113.36999999999999 -> 94.19999999999999,28.37
- R8268: BoardSide F.Cu -> B.Cu; FootprintOriginMm 125.77,112.69999999999999 -> 102.69999999999999,27.07; KiCadOrientationDeg 0 -> 90
- R8269: BoardSide B.Cu -> F.Cu; FootprintOriginMm 96.71,109.34 -> 76.11,36.44; KiCadOrientationDeg 90 -> 270
- R8270: BoardSide F.Cu -> B.Cu; FootprintOriginMm 123.50999999999999,131.14 -> 78.94,116.31; KiCadOrientationDeg 270 -> 180
- R8271: BoardSide B.Cu -> F.Cu; FootprintOriginMm 98.61,113.04 -> 73.91,40.14; KiCadOrientationDeg 90 -> 270
- R8272: BoardSide F.Cu -> B.Cu; FootprintOriginMm 106.11,117.04 -> 75.71,23.94; KiCadOrientationDeg 270 -> 90
- R8273: BoardSide B.Cu -> F.Cu; FootprintOriginMm 92.71,28.84 -> 76.11,32.74; KiCadOrientationDeg 90 -> 270
- R8274: FootprintOriginMm 90.50999999999999,32.54 -> 72.81,28.240000000000002
- R8275: FootprintOriginMm 170.31,79.84 -> 170.31,53.34
- R8276: BoardSide F.Cu -> B.Cu; FootprintOriginMm 109.34,122.31 -> 76.44,114.00999999999999; KiCadOrientationDeg 0 -> 180
- R8277: FootprintOriginMm 170.31,83.94 -> 170.31,81.34
- U8202: FootprintOriginMm 141.98,107.12 -> 124.98,92.82000000000001
- U8203: FootprintOriginMm 127.77000000000001,30.78 -> 127.78,109.12; KiCadOrientationDeg 0 -> 90
- U8204: BoardSide B.Cu -> F.Cu; FootprintOriginMm 128.57999999999998,106.92 -> 124.98,106.02000000000001
- U8205: FootprintOriginMm 125.50999999999999,24.38 -> 109.97,30.380000000000003
- U8206: BoardSide B.Cu -> F.Cu; FootprintOriginMm 110.77000000000001,44.779999999999994 -> 107.98,49.77; KiCadOrientationDeg 0 -> 270
- U8212: FootprintOriginMm 161.87,29.55 -> 161.13000000000002,28.75
- U8214: FootprintOriginMm 159.67,47.544999999999995 -> 158.23000000000002,45.25
- U8215: FootprintOriginMm 159.67,88.08000000000001 -> 159.67,88.88000000000001
- U8216: FootprintOriginMm 160.68,56.769999999999996 -> 159.67,55.05; KiCadOrientationDeg 90 -> 180
- U8217: FootprintOriginMm 144.87,29.55 -> 142.67,100.48; KiCadOrientationDeg 180 -> 0
