File: boards/osc-jack-left/sheets/oscillator_O1_JL.kicad_sch (KiCad schematic)
At the start: 57 parts, among them J101 WQP518MA, J102 WQP518MA, J103 WQP518MA, J104 WQP518MA, J105 WQP518MA, J106 WQP518MA, J107 WQP518MA, J108 WQP518MA, U1101 ADG5412FBRUZ, U1102 ADG5412FBRUZ, U1103 ADG5412FBRUZ, U1104 ADG5412FBRUZ, U1116 OPA4196IDR, U1117 OPA4196IDR, U1118 OPA4197IPWR

Commit message: Move jack halves to six layers with locality placement and grid routing
Owner decision 2026-10-03 (#38): a cut-line bound showed the four-layer
jack halves could not carry their signal nets with intact planes, so both
halves move to six layers and their free packages are re-placed for
locality.

- Placement: scripts/checks/jack_locality.py replaces the
  connectivity-blind first-fit J placer. Packages are pulled toward the
  fixed jacks, LEDs and headers on their nets and toward their own
  module's hardware, then legalized; IC/bypass clusters stay aligned.
  Panel hardware and headers do not move.
- Stack: F/In2/In3/B signals, In1 AGND plane, -12V fill on In3, +12V
  plane on In4; +5V as tracks.
- Routing: scripts/pcbgen/route_jack_grid.py stages terminal arrays,
  rail fanouts and links, signal batches, rip-up-and-reroute and AGND
  stitching, keeping only natively checked stages (0 DRC errors,
  0 parity). The grid router gains N-layer support, windowed search,
  plane fanout, a plane-fill split guard and rip-up-and-reroute.
- Evidence chain: a bounded jack-locality partition transition is
  chained onto the connector-locality proof; superseded four-layer
  stage reports are removed.

Checkpoint: JL 411 and JR 518 native open edges remain. This is a routed
draft in progress; electrical and physical qualification NOT RUN.

Co-Authored-By: Claude Opus 5.5 <noreply@anthropic.com>
Parts:
- C1121: FootprintOriginMm 65.76,85.355 -> 10.605,80.76; KiCadOrientationDeg 90 -> 0
- C1122: FootprintOriginMm 76.67,85.355 -> 10.605,91.67; KiCadOrientationDeg 90 -> 0
- C1123: BoardSide B.Cu -> F.Cu; FootprintOriginMm 82.76,85.355 -> 22.205000000000002,83.16999999999999; KiCadOrientationDeg 90 -> 180
- C1124: BoardSide B.Cu -> F.Cu; FootprintOriginMm 93.67,85.355 -> 22.205000000000002,72.25999999999999; KiCadOrientationDeg 90 -> 180
- C1125: FootprintOriginMm 99.76,85.355 -> 16.96,62.155
- C1126: FootprintOriginMm 110.67,85.355 -> 27.87,62.155
- C1127: BoardSide B.Cu -> F.Cu; FootprintOriginMm 116.76,85.355 -> 22.955000000000002,85.46000000000001; KiCadOrientationDeg 90 -> 0
- C1128: BoardSide B.Cu -> F.Cu; FootprintOriginMm 127.67,85.355 -> 22.955000000000002,96.37; KiCadOrientationDeg 90 -> 0
- C1140: FootprintOriginMm 27.28,134.23000000000002 -> 8.43,66.36000000000001; KiCadOrientationDeg 90 -> 180
- C1141: FootprintOriginMm 16.96,134.23000000000002 -> 8.43,76.68; KiCadOrientationDeg 90 -> 180
- C1150: FootprintOriginMm 60.98,24.55 -> 25.42,71.55; KiCadOrientationDeg 90 -> 0
- C1151: FootprintOriginMm 50.96,24.55 -> 14.040000000000001,71.55; KiCadOrientationDeg 90 -> 180
- C1152: FootprintOriginMm 77.98,24.55 -> 16.96,88.78000000000002; KiCadOrientationDeg 90 -> 270
- C1153: FootprintOriginMm 67.96,24.55 -> 26.979999999999997,88.78000000000002; KiCadOrientationDeg 90 -> 270
- DO1101: BoardSide B.Cu -> F.Cu; FootprintOriginMm 102.93,140.01 -> 7.029999999999999,88.71000000000001; KiCadOrientationDeg 180 -> 0
- DO1102: BoardSide B.Cu -> F.Cu; FootprintOriginMm 107.23,140.01 -> 7.029999999999999,66.01; KiCadOrientationDeg 180 -> 0
- DO1103: FootprintOriginMm 111.53,140.01 -> 10.629999999999999,59.61
- DO1104: FootprintOriginMm 119.93,140.01 -> 22.709999999999997,95.33000000000001; KiCadOrientationDeg 180 -> 90
- R1101: FootprintOriginMm 83.64,28.01 -> 6.84,91.71
- R1102: FootprintOriginMm 100.64,28.01 -> 6.04,93.91
- R1103: FootprintOriginMm 117.64,28.01 -> 6.64,60.51
- R1104: FootprintOriginMm 134.64,28.01 -> 11.71,77.74; KiCadOrientationDeg 180 -> 90
- R1105: FootprintOriginMm 151.64,28.01 -> 14.64,59.209999999999994
- R1106: FootprintOriginMm 27.44,31.61 -> 18.34,58.91
- R1107: BoardSide B.Cu -> F.Cu; FootprintOriginMm 44.44,31.61 -> 7.34,91.81; KiCadOrientationDeg 180 -> 0
- R1108: FootprintOriginMm 61.44,31.61 -> 5.3100000000000005,83.64; KiCadOrientationDeg 180 -> 90
- R1109: FootprintOriginMm 78.44,31.61 -> 10.940000000000001,97.50999999999999
- R1110: FootprintOriginMm 95.44,31.61 -> 6.04,96.11
- R1111: FootprintOriginMm 112.44,31.61 -> 14.64,57.01
- R1112: FootprintOriginMm 129.44,31.61 -> 11.71,65.53999999999999; KiCadOrientationDeg 180 -> 90
- R1113: FootprintOriginMm 146.44,31.61 -> 14.64,98.00999999999999
- R1114: FootprintOriginMm 163.44,31.61 -> 18.34,97.91
- R1115: FootprintOriginMm 10.84,37.01 -> 7.239999999999999,98.31
- R1116: FootprintOriginMm 10.84,39.209999999999994 -> 5.3100000000000005,87.34; KiCadOrientationDeg 180 -> 90
- RB1102: BoardSide B.Cu -> F.Cu; FootprintOriginMm 137.27,31.900000000000002 -> 7.4,70.47; KiCadOrientationDeg 180 -> 270
- RB1103: FootprintOriginMm 142.17000000000002,31.900000000000002 -> 15.27,85.0
- RB1104: FootprintOriginMm 154.27,31.900000000000002 -> 8.17,63.4
- RB1105: BoardSide B.Cu -> F.Cu; FootprintOriginMm 159.17000000000002,31.900000000000002 -> 7.4,75.36999999999999; KiCadOrientationDeg 180 -> 270
- RB1106: FootprintOriginMm 6.57,33.3 -> 18.27,95.0
- RB1107: FootprintOriginMm 6.57,36.9 -> 26.07,74.6
- RB1108: FootprintOriginMm 6.57,40.5 -> 10.37,94.6
- RB1109: BoardSide B.Cu -> F.Cu; FootprintOriginMm 11.469999999999999,42.7 -> 7.4,84.27; KiCadOrientationDeg 180 -> 270
- U1101: FootprintOriginMm 70.92,86.38000000000001 -> 9.58,85.92; KiCadOrientationDeg 180 -> 90
- U1102: BoardSide B.Cu -> F.Cu; FootprintOriginMm 87.92,86.38000000000001 -> 22.580000000000002,78.00999999999999; KiCadOrientationDeg 180 -> 270
- U1103: FootprintOriginMm 104.92,86.38000000000001 -> 22.12,63.18
- U1104: BoardSide B.Cu -> F.Cu; FootprintOriginMm 121.92,86.38000000000001 -> 22.580000000000002,90.62; KiCadOrientationDeg 180 -> 90
- U1116: FootprintOriginMm 55.97,25.25 -> 19.73,71.55
- U1117: FootprintOriginMm 72.97,25.25 -> 21.97,88.08000000000001; KiCadOrientationDeg 180 -> 0
- U1118: FootprintOriginMm 22.12,134.93 -> 9.129999999999999,71.52000000000001; KiCadOrientationDeg 180 -> 270

Commit message: Route jack-left with negotiated congestion to 360 open edges
Locality placement with a 0.8 mm IC keep-clear ring on JL (JR keeps none),
a native C grid A*, a PathFinder negotiated-congestion stage on a 0.05 mm
grid, then rip-up-and-reroute and AGND stitching. Native: 360 open edges
(main 411), 0 DRC errors, 0 schematic parity findings. Routed draft;
electrical/physical qualification NOT RUN.

Co-Authored-By: Claude Opus 5.5 <noreply@anthropic.com>
Parts:
- C1121: FootprintOriginMm 10.605,80.76 -> 9.805000000000001,82.96000000000001
- C1122: FootprintOriginMm 10.605,91.67 -> 9.805000000000001,93.87
- C1125: FootprintOriginMm 16.96,62.155 -> 16.96,59.755
- C1126: FootprintOriginMm 27.87,62.155 -> 27.87,59.755
- C1127: BoardSide F.Cu -> B.Cu; FootprintOriginMm 22.955000000000002,85.46000000000001 -> 7.755000000000001,64.07000000000001; KiCadOrientationDeg 0 -> 180
- C1128: BoardSide F.Cu -> B.Cu; FootprintOriginMm 22.955000000000002,96.37 -> 7.755000000000001,53.160000000000004; KiCadOrientationDeg 0 -> 180
- C1140: FootprintOriginMm 8.43,66.36000000000001 -> 8.23,66.36000000000001
- C1141: FootprintOriginMm 8.43,76.68 -> 8.23,76.68
- C1150: FootprintOriginMm 25.42,71.55 -> 26.22,70.75
- C1151: FootprintOriginMm 14.040000000000001,71.55 -> 14.839999999999998,70.75
- C1152: FootprintOriginMm 16.96,88.78000000000002 -> 16.96,89.58000000000001
- C1153: FootprintOriginMm 26.979999999999997,88.78000000000002 -> 26.979999999999997,89.58000000000001
- DO1101: BoardSide F.Cu -> B.Cu; FootprintOriginMm 7.029999999999999,88.71000000000001 -> 10.629999999999999,97.01; KiCadOrientationDeg 0 -> 180
- DO1102: FootprintOriginMm 7.029999999999999,66.01 -> 7.210000000000001,92.43; KiCadOrientationDeg 0 -> 270
- DO1103: FootprintOriginMm 10.629999999999999,59.61 -> 6.33,97.01
- DO1104: BoardSide B.Cu -> F.Cu; FootprintOriginMm 22.709999999999997,95.33000000000001 -> 7.029999999999999,62.410000000000004; KiCadOrientationDeg 90 -> 0
- R1101: FootprintOriginMm 6.84,91.71 -> 27.04,66.21
- R1102: FootprintOriginMm 6.04,93.91 -> 14.51,58.44; KiCadOrientationDeg 180 -> 90
- R1103: FootprintOriginMm 6.64,60.51 -> 13.91,98.74; KiCadOrientationDeg 180 -> 90
- R1104: FootprintOriginMm 11.71,77.74 -> 11.71,78.24
- R1105: BoardSide B.Cu -> F.Cu; FootprintOriginMm 14.64,59.209999999999994 -> 20.51,62.04; KiCadOrientationDeg 180 -> 270
- R1106: FootprintOriginMm 18.34,58.91 -> 17.54,99.50999999999999
- R1107: BoardSide F.Cu -> B.Cu; FootprintOriginMm 7.34,91.81 -> 10.940000000000001,100.11; KiCadOrientationDeg 0 -> 180
- R1108: FootprintOriginMm 5.3100000000000005,83.64 -> 9.51,79.64
- R1109: FootprintOriginMm 10.940000000000001,97.50999999999999 -> 17.64,55.709999999999994
- R1110: BoardSide B.Cu -> F.Cu; FootprintOriginMm 6.04,96.11 -> 21.240000000000002,58.809999999999995; KiCadOrientationDeg 180 -> 0
- R1111: BoardSide B.Cu -> F.Cu; FootprintOriginMm 14.64,57.01 -> 7.34,95.71; KiCadOrientationDeg 180 -> 0
- R1112: FootprintOriginMm 11.71,65.53999999999999 -> 14.64,84.31; KiCadOrientationDeg 90 -> 180
- R1113: FootprintOriginMm 14.64,98.00999999999999 -> 7.239999999999999,100.11
- R1114: BoardSide B.Cu -> F.Cu; FootprintOriginMm 18.34,97.91 -> 7.34,59.309999999999995; KiCadOrientationDeg 180 -> 0
- R1115: BoardSide B.Cu -> F.Cu; FootprintOriginMm 7.239999999999999,98.31 -> 21.240000000000002,96.21; KiCadOrientationDeg 180 -> 0
- R1116: FootprintOriginMm 5.3100000000000005,87.34 -> 14.64,86.50999999999999; KiCadOrientationDeg 90 -> 180
- RB1102: FootprintOriginMm 7.4,70.47 -> 6.77,66.19999999999999; KiCadOrientationDeg 270 -> 0
- RB1103: BoardSide B.Cu -> F.Cu; FootprintOriginMm 15.27,85.0 -> 7.4,75.36999999999999; KiCadOrientationDeg 180 -> 270
- RB1104: BoardSide B.Cu -> F.Cu; FootprintOriginMm 8.17,63.4 -> 6.77,88.5; KiCadOrientationDeg 180 -> 0
- RB1105: FootprintOriginMm 7.4,75.36999999999999 -> 7.4,84.27
- RB1106: BoardSide B.Cu -> F.Cu; FootprintOriginMm 18.27,95.0 -> 21.87,65.69999999999999; KiCadOrientationDeg 180 -> 0
- RB1107: BoardSide B.Cu -> F.Cu; FootprintOriginMm 26.07,74.6 -> 7.4,70.47; KiCadOrientationDeg 180 -> 270
- RB1108: FootprintOriginMm 10.37,94.6 -> 18.27,96.6
- RB1109: FootprintOriginMm 7.4,84.27 -> 21.87,86.1; KiCadOrientationDeg 270 -> 0
- U1101: FootprintOriginMm 9.58,85.92 -> 8.780000000000001,88.12
- U1103: FootprintOriginMm 22.12,63.18 -> 22.12,60.78
- U1104: BoardSide F.Cu -> B.Cu; FootprintOriginMm 22.580000000000002,90.62 -> 8.780000000000001,58.910000000000004; KiCadOrientationDeg 90 -> 270
- U1116: FootprintOriginMm 19.73,71.55 -> 20.529999999999998,70.75
- U1117: FootprintOriginMm 21.97,88.08000000000001 -> 21.97,88.88000000000001
- U1118: FootprintOriginMm 9.129999999999999,71.52000000000001 -> 8.93,71.52000000000001
