File: boards/osc-jack-left/sheets/wavefolder_W2_JL.kicad_sch (KiCad schematic)
At the start: 54 parts, among them J1007 WQP518MA, J1008 WQP518MA, J907 WQP518MA, J908 WQP518MA, U5102 ADG5412FBRUZ, U5103 ADG5412FBRUZ, U5104 ADG5412FBRUZ, U5112 OPA4196IDR, U5113 OPA4196IDR

Commit message: Move jack halves to six layers with locality placement and grid routing
Owner decision 2026-10-03 (#38): a cut-line bound showed the four-layer
jack halves could not carry their signal nets with intact planes, so both
halves move to six layers and their free packages are re-placed for
locality.

- Placement: scripts/checks/jack_locality.py replaces the
  connectivity-blind first-fit J placer. Packages are pulled toward the
  fixed jacks, LEDs and headers on their nets and toward their own
  module's hardware, then legalized; IC/bypass clusters stay aligned.
  Panel hardware and headers do not move.
- Stack: F/In2/In3/B signals, In1 AGND plane, -12V fill on In3, +12V
  plane on In4; +5V as tracks.
- Routing: scripts/pcbgen/route_jack_grid.py stages terminal arrays,
  rail fanouts and links, signal batches, rip-up-and-reroute and AGND
  stitching, keeping only natively checked stages (0 DRC errors,
  0 parity). The grid router gains N-layer support, windowed search,
  plane fanout, a plane-fill split guard and rip-up-and-reroute.
- Evidence chain: a bounded jack-locality partition transition is
  chained onto the connector-locality proof; superseded four-layer
  stage reports are removed.

Checkpoint: JL 411 and JR 518 native open edges remain. This is a routed
draft in progress; electrical and physical qualification NOT RUN.

Co-Authored-By: Claude Opus 5.5 <noreply@anthropic.com>
Parts:
- C5120: BoardSide B.Cu -> F.Cu; FootprintOriginMm 152.96,110.955 -> 159.30499999999998,124.31; KiCadOrientationDeg 90 -> 270
- C5121: BoardSide B.Cu -> F.Cu; FootprintOriginMm 163.87,110.955 -> 159.30499999999998,112.03999999999999
- C5122: FootprintOriginMm 135.96,117.355 -> 164.67000000000002,110.605; KiCadOrientationDeg 90 -> 270
- C5123: FootprintOriginMm 146.87,117.355 -> 153.76000000000002,110.605; KiCadOrientationDeg 90 -> 270
- C5124: FootprintOriginMm 152.96,117.355 -> 147.67000000000002,111.50500000000001; KiCadOrientationDeg 90 -> 270
- C5125: FootprintOriginMm 163.87,117.355 -> 136.76000000000002,111.50500000000001; KiCadOrientationDeg 90 -> 270
- C5140: FootprintOriginMm 26.979999999999997,65.64999999999999 -> 161.07999999999998,123.98; KiCadOrientationDeg 90 -> 0
- C5141: FootprintOriginMm 16.96,65.64999999999999 -> 161.07999999999998,113.96; KiCadOrientationDeg 90 -> 0
- C5142: FootprintOriginMm 43.98,65.64999999999999 -> 157.35,124.05999999999999; KiCadOrientationDeg 90 -> 180
- C5143: FootprintOriginMm 33.96,65.64999999999999 -> 157.35,134.07999999999998; KiCadOrientationDeg 90 -> 180
- D5101: FootprintOriginMm 168.93,70.91 -> 107.91,111.93; KiCadOrientationDeg 180 -> 90
- D5102: BoardSide B.Cu -> F.Cu; FootprintOriginMm 10.43,76.71000000000001 -> 109.21000000000001,119.03; KiCadOrientationDeg 180 -> 270
- D5103: BoardSide B.Cu -> F.Cu; FootprintOriginMm 17.93,114.41 -> 109.21000000000001,114.73; KiCadOrientationDeg 180 -> 270
- D5114: FootprintOriginMm 47.45,99.44999999999999 -> 168.04999999999998,114.85; KiCadOrientationDeg 90 -> 180
- D5115: FootprintOriginMm 64.45,99.44999999999999 -> 150.65,113.44999999999999
- D5116: FootprintOriginMm 81.45,99.44999999999999 -> 160.45,104.95; KiCadOrientationDeg 90 -> 180
- D5117: BoardSide B.Cu -> F.Cu; FootprintOriginMm 98.45,99.44999999999999 -> 159.61,108.75; KiCadOrientationDeg 90 -> 0
- D5119: FootprintOriginMm 115.45,99.44999999999999 -> 153.35,105.85
- D5120: FootprintOriginMm 132.45,99.44999999999999 -> 162.15,102.05; KiCadOrientationDeg 90 -> 180
- D5121: BoardSide B.Cu -> F.Cu; FootprintOriginMm 149.45,99.44999999999999 -> 159.61,105.85; KiCadOrientationDeg 90 -> 0
- D5122: FootprintOriginMm 10.45,103.05 -> 167.54999999999998,100.85; KiCadOrientationDeg 90 -> 180
- D5124: FootprintOriginMm 149.45,113.44999999999999 -> 145.95,105.85; KiCadOrientationDeg 90 -> 180
- D5125: BoardSide B.Cu -> F.Cu; FootprintOriginMm 28.25,127.75 -> 160.45,101.81; KiCadOrientationDeg 90 -> 270
- D5126: FootprintOriginMm 45.25,127.75 -> 162.15,95.45; KiCadOrientationDeg 90 -> 180
- D5127: FootprintOriginMm 62.25,127.75 -> 140.54999999999998,105.85; KiCadOrientationDeg 90 -> 180
- R5105: BoardSide F.Cu -> B.Cu; FootprintOriginMm 142.73999999999998,41.709999999999994 -> 167.64,112.31; KiCadOrientationDeg 0 -> 180
- R5106: BoardSide F.Cu -> B.Cu; FootprintOriginMm 159.73999999999998,41.709999999999994 -> 164.71,106.84; KiCadOrientationDeg 0 -> 90
- R5107: BoardSide F.Cu -> B.Cu; FootprintOriginMm 5.9399999999999995,43.01 -> 169.91,109.34; KiCadOrientationDeg 0 -> 90
- R5108: BoardSide F.Cu -> B.Cu; FootprintOriginMm 72.24,43.01 -> 157.33999999999997,113.91; KiCadOrientationDeg 0 -> 180
- R5109: BoardSide F.Cu -> B.Cu; FootprintOriginMm 89.24,43.01 -> 169.91,105.64; KiCadOrientationDeg 0 -> 90
- R5110: FootprintOriginMm 21.240000000000002,43.709999999999994 -> 173.51,115.54; KiCadOrientationDeg 0 -> 270
- R5111: FootprintOriginMm 38.24,43.709999999999994 -> 173.51,119.24; KiCadOrientationDeg 0 -> 270
- R5112: BoardSide F.Cu -> B.Cu; FootprintOriginMm 55.24,43.709999999999994 -> 164.01,124.74; KiCadOrientationDeg 0 -> 90
- R5113: FootprintOriginMm 108.74,43.91 -> 173.51,122.94; KiCadOrientationDeg 0 -> 270
- R5114: FootprintOriginMm 125.74,43.91 -> 173.51,126.64; KiCadOrientationDeg 0 -> 270
- R5115: FootprintOriginMm 142.73999999999998,43.91 -> 173.51,109.84; KiCadOrientationDeg 0 -> 270
- R5116: BoardSide F.Cu -> B.Cu; FootprintOriginMm 159.73999999999998,43.91 -> 169.91,119.04; KiCadOrientationDeg 0 -> 90
- R5171: BoardSide B.Cu -> F.Cu; FootprintOriginMm 86.27,31.900000000000002 -> 126.39999999999999,123.86999999999999; KiCadOrientationDeg 180 -> 270
- R5172: BoardSide B.Cu -> F.Cu; FootprintOriginMm 91.17,31.900000000000002 -> 126.39999999999999,118.97; KiCadOrientationDeg 180 -> 270
- R5173: FootprintOriginMm 5.9399999999999995,45.209999999999994 -> 173.51,130.33999999999997; KiCadOrientationDeg 0 -> 270
- R5174: BoardSide F.Cu -> B.Cu; FootprintOriginMm 72.24,45.209999999999994 -> 168.83999999999997,98.31; KiCadOrientationDeg 0 -> 180
- R5175: FootprintOriginMm 89.24,45.209999999999994 -> 173.51,106.14; KiCadOrientationDeg 0 -> 270
- U5102: BoardSide B.Cu -> F.Cu; FootprintOriginMm 158.12,111.98 -> 158.98,118.47; KiCadOrientationDeg 180 -> 270
- U5103: FootprintOriginMm 141.12,118.38000000000001 -> 159.51000000000002,109.58; KiCadOrientationDeg 180 -> 0
- U5104: FootprintOriginMm 158.12,118.38000000000001 -> 142.51000000000002,110.48; KiCadOrientationDeg 180 -> 0
- U5112: FootprintOriginMm 21.97,66.35 -> 160.38,118.97; KiCadOrientationDeg 180 -> 90
- U5113: FootprintOriginMm 38.97,66.35 -> 158.04999999999998,129.07; KiCadOrientationDeg 180 -> 270

Commit message: Route jack-left with negotiated congestion to 360 open edges
Locality placement with a 0.8 mm IC keep-clear ring on JL (JR keeps none),
a native C grid A*, a PathFinder negotiated-congestion stage on a 0.05 mm
grid, then rip-up-and-reroute and AGND stitching. Native: 360 open edges
(main 411), 0 DRC errors, 0 schematic parity findings. Routed draft;
electrical/physical qualification NOT RUN.

Co-Authored-By: Claude Opus 5.5 <noreply@anthropic.com>
Parts:
- C5124: BoardSide B.Cu -> F.Cu; FootprintOriginMm 147.67000000000002,111.50500000000001 -> 141.605,113.07; KiCadOrientationDeg 270 -> 180
- C5125: BoardSide B.Cu -> F.Cu; FootprintOriginMm 136.76000000000002,111.50500000000001 -> 141.605,102.16; KiCadOrientationDeg 270 -> 180
- C5140: FootprintOriginMm 161.07999999999998,123.98 -> 159.45000000000002,113.96; KiCadOrientationDeg 0 -> 180
- C5141: FootprintOriginMm 161.07999999999998,113.96 -> 159.45000000000002,123.98; KiCadOrientationDeg 0 -> 180
- C5142: FootprintOriginMm 157.35,124.05999999999999 -> 154.66,131.48; KiCadOrientationDeg 180 -> 270
- C5143: FootprintOriginMm 157.35,134.07999999999998 -> 164.67999999999998,131.48; KiCadOrientationDeg 180 -> 270
- D5101: FootprintOriginMm 107.91,111.93 -> 88.43,112.11; KiCadOrientationDeg 90 -> 180
- D5102: FootprintOriginMm 109.21000000000001,119.03 -> 92.21000000000001,113.23
- D5103: BoardSide F.Cu -> B.Cu; FootprintOriginMm 109.21000000000001,114.73 -> 84.31,114.13000000000001; KiCadOrientationDeg 270 -> 90
- D5114: FootprintOriginMm 168.04999999999998,114.85 -> 167.25,113.44999999999999; KiCadOrientationDeg 180 -> 90
- D5115: BoardSide B.Cu -> F.Cu; FootprintOriginMm 150.65,113.44999999999999 -> 159.61,108.75; KiCadOrientationDeg 90 -> 0
- D5116: BoardSide B.Cu -> F.Cu; FootprintOriginMm 160.45,104.95 -> 159.61,105.85; KiCadOrientationDeg 180 -> 0
- D5117: BoardSide F.Cu -> B.Cu; FootprintOriginMm 159.61,108.75 -> 145.95,108.75; KiCadOrientationDeg 0 -> 180
- D5119: FootprintOriginMm 153.35,105.85 -> 166.65,100.85; KiCadOrientationDeg 90 -> 180
- D5120: BoardSide B.Cu -> F.Cu; FootprintOriginMm 162.15,102.05 -> 160.45,101.81; KiCadOrientationDeg 180 -> 270
- D5121: BoardSide F.Cu -> B.Cu; FootprintOriginMm 159.61,105.85 -> 140.54999999999998,108.75; KiCadOrientationDeg 0 -> 180
- D5122: FootprintOriginMm 167.54999999999998,100.85 -> 136.45,118.75; KiCadOrientationDeg 180 -> 90
- D5124: BoardSide B.Cu -> F.Cu; FootprintOriginMm 145.95,105.85 -> 160.45,96.41; KiCadOrientationDeg 180 -> 270
- D5125: BoardSide F.Cu -> B.Cu; FootprintOriginMm 160.45,101.81 -> 133.55,113.44999999999999; KiCadOrientationDeg 270 -> 90
- D5126: FootprintOriginMm 162.15,95.45 -> 126.75,126.65
- D5127: FootprintOriginMm 140.54999999999998,105.85 -> 124.05,116.95
- R5105: FootprintOriginMm 167.64,112.31 -> 169.91,119.04; KiCadOrientationDeg 180 -> 90
- R5106: FootprintOriginMm 164.71,106.84 -> 169.91,115.34
- R5107: FootprintOriginMm 169.91,109.34 -> 169.91,111.64
- R5108: FootprintOriginMm 157.33999999999997,113.91 -> 153.10999999999999,119.04; KiCadOrientationDeg 180 -> 90
- R5109: FootprintOriginMm 169.91,105.64 -> 169.91,107.94
- R5110: BoardSide F.Cu -> B.Cu; FootprintOriginMm 173.51,115.54 -> 169.91,104.24; KiCadOrientationDeg 270 -> 90
- R5111: FootprintOriginMm 173.51,119.24 -> 173.51,117.14
- R5112: FootprintOriginMm 164.01,124.74 -> 153.10999999999999,115.34
- R5113: FootprintOriginMm 173.51,122.94 -> 173.51,120.84
- R5114: FootprintOriginMm 173.51,126.64 -> 173.51,124.54
- R5116: FootprintOriginMm 169.91,119.04 -> 153.10999999999999,122.74
- R5171: BoardSide F.Cu -> B.Cu; FootprintOriginMm 126.39999999999999,123.86999999999999 -> 92.39999999999999,115.97; KiCadOrientationDeg 270 -> 90
- R5172: FootprintOriginMm 126.39999999999999,118.97 -> 109.39999999999999,118.97
- R5173: FootprintOriginMm 173.51,130.33999999999997 -> 173.51,128.23999999999998
- R5174: BoardSide B.Cu -> F.Cu; FootprintOriginMm 168.83999999999997,98.31 -> 173.51,106.14; KiCadOrientationDeg 180 -> 270
- R5175: FootprintOriginMm 173.51,106.14 -> 173.51,131.94
- U5104: BoardSide B.Cu -> F.Cu; FootprintOriginMm 142.51000000000002,110.48 -> 141.98,107.91; KiCadOrientationDeg 0 -> 270
- U5112: FootprintOriginMm 160.38,118.97 -> 160.15,118.97; KiCadOrientationDeg 90 -> 270
- U5113: FootprintOriginMm 158.04999999999998,129.07 -> 159.67,130.78; KiCadOrientationDeg 270 -> 0
