File: boards/osc-jack-left/sheets/mix5_M5A_JL.kicad_sch (KiCad schematic)
At the start: 106 parts, among them J901 WQP518MA, J902 WQP518MA, J903 WQP518MA, J904 WQP518MA, J905 WQP518MA, J906 WQP518MA, U8102 ADG5412FBRUZ, U8103 ADG5412FBRUZ, U8104 ADG5412FBRUZ, U8105 ADG5412FBRUZ, U8106 ADG5412FBRUZ, U8112 OPA4196IDR, U8113 LM393BIDR, U8114 LM393BIDR, U8115 OPA4196IDR, U8116 OPA4196IDR, U8117 OPA4196IDR

Commit message: Move jack halves to six layers with locality placement and grid routing
Owner decision 2026-10-03 (#38): a cut-line bound showed the four-layer
jack halves could not carry their signal nets with intact planes, so both
halves move to six layers and their free packages are re-placed for
locality.

- Placement: scripts/checks/jack_locality.py replaces the
  connectivity-blind first-fit J placer. Packages are pulled toward the
  fixed jacks, LEDs and headers on their nets and toward their own
  module's hardware, then legalized; IC/bypass clusters stay aligned.
  Panel hardware and headers do not move.
- Stack: F/In2/In3/B signals, In1 AGND plane, -12V fill on In3, +12V
  plane on In4; +5V as tracks.
- Routing: scripts/pcbgen/route_jack_grid.py stages terminal arrays,
  rail fanouts and links, signal batches, rip-up-and-reroute and AGND
  stitching, keeping only natively checked stages (0 DRC errors,
  0 parity). The grid router gains N-layer support, windowed search,
  plane fanout, a plane-fill split guard and rip-up-and-reroute.
- Evidence chain: a bounded jack-locality partition transition is
  chained onto the connector-locality proof; superseded four-layer
  stage reports are removed.

Checkpoint: JL 411 and JR 518 native open edges remain. This is a routed
draft in progress; electrical and physical qualification NOT RUN.

Co-Authored-By: Claude Opus 5.5 <noreply@anthropic.com>
Parts:
- C8115: BoardSide B.Cu -> F.Cu; FootprintOriginMm 135.96,123.755 -> 159.105,57.510000000000005; KiCadOrientationDeg 90 -> 270
- C8116: BoardSide B.Cu -> F.Cu; FootprintOriginMm 146.87,123.755 -> 159.105,45.24
- C8117: BoardSide B.Cu -> F.Cu; FootprintOriginMm 152.96,123.755 -> 159.105,41.61; KiCadOrientationDeg 90 -> 270
- C8118: BoardSide B.Cu -> F.Cu; FootprintOriginMm 163.87,123.755 -> 159.105,29.339999999999996
- C8119: BoardSide B.Cu -> F.Cu; FootprintOriginMm 14.760000000000002,127.35499999999999 -> 142.30499999999998,40.61; KiCadOrientationDeg 90 -> 270
- C8120: BoardSide B.Cu -> F.Cu; FootprintOriginMm 25.67,127.35499999999999 -> 142.30499999999998,28.339999999999996
- C8121: BoardSide B.Cu -> F.Cu; FootprintOriginMm 31.76,127.35499999999999 -> 125.355,87.66000000000001; KiCadOrientationDeg 90 -> 0
- C8122: BoardSide B.Cu -> F.Cu; FootprintOriginMm 42.67,127.35499999999999 -> 125.355,98.57000000000001; KiCadOrientationDeg 90 -> 0
- C8123: FootprintOriginMm 48.75999999999999,127.35499999999999 -> 123.20500000000001,90.76; KiCadOrientationDeg 90 -> 0
- C8124: FootprintOriginMm 59.669999999999995,127.35499999999999 -> 123.20500000000001,101.67; KiCadOrientationDeg 90 -> 0
- C8125: BoardSide B.Cu -> F.Cu; FootprintOriginMm 33.96,139.84 -> 160.37,71.52; KiCadOrientationDeg 90 -> 270
- C8126: BoardSide B.Cu -> F.Cu; FootprintOriginMm 43.98,143.65 -> 156.56,60.14
- C8127: BoardSide B.Cu -> F.Cu; FootprintOriginMm 50.96,139.84 -> 140.245,60.14
- C8128: BoardSide B.Cu -> F.Cu; FootprintOriginMm 60.98,143.65 -> 144.055,71.52; KiCadOrientationDeg 90 -> 270
- C8139: FootprintOriginMm 60.98,65.64999999999999 -> 150.04000000000002,98.08000000000001; KiCadOrientationDeg 90 -> 180
- C8140: FootprintOriginMm 50.96,65.64999999999999 -> 161.42000000000002,98.08000000000001; KiCadOrientationDeg 90 -> 0
- C8141: FootprintOriginMm 77.98,65.64999999999999 -> 143.95,55.64
- C8142: FootprintOriginMm 67.96,65.64999999999999 -> 143.95,67.02; KiCadOrientationDeg 90 -> 270
- C8143: FootprintOriginMm 94.98,65.64999999999999 -> 157.38,71.88000000000001; KiCadOrientationDeg 90 -> 0
- C8144: FootprintOriginMm 84.96,65.64999999999999 -> 157.38,61.86000000000001; KiCadOrientationDeg 90 -> 0
- C8145: FootprintOriginMm 111.98,65.64999999999999 -> 137.06,98.78000000000002; KiCadOrientationDeg 90 -> 270
- C8146: FootprintOriginMm 101.96,65.64999999999999 -> 147.07999999999998,98.78000000000002; KiCadOrientationDeg 90 -> 270
- D8108: BoardSide B.Cu -> F.Cu; FootprintOriginMm 22.23,114.41 -> 109.03,26.41; KiCadOrientationDeg 180 -> 0
- D8109: FootprintOriginMm 6.2299999999999995,116.21000000000001 -> 100.53,30.31
- D8110: FootprintOriginMm 10.53,116.51 -> 104.03,24.81
- D8111: BoardSide B.Cu -> F.Cu; FootprintOriginMm 6.2299999999999995,120.21000000000001 -> 109.21000000000001,109.93; KiCadOrientationDeg 180 -> 270
- D8112: BoardSide B.Cu -> F.Cu; FootprintOriginMm 10.53,120.51 -> 109.21000000000001,22.23; KiCadOrientationDeg 180 -> 270
- D8113: FootprintOriginMm 79.25,127.75 -> 165.54999999999998,72.25; KiCadOrientationDeg 90 -> 180
- D8114: FootprintOriginMm 96.25,127.75 -> 167.25,57.45
- D8115: FootprintOriginMm 113.25,127.75 -> 169.85,71.44999999999999
- D8116: FootprintOriginMm 14.15,141.45 -> 166.15,84.65; KiCadOrientationDeg 90 -> 180
- D8117: FootprintOriginMm 115.15,141.45 -> 158.35,42.75; KiCadOrientationDeg 90 -> 180
- D8118: FootprintOriginMm 113.05,148.54999999999998 -> 166.15,44.85; KiCadOrientationDeg 90 -> 180
- D8119: BoardSide B.Cu -> F.Cu; FootprintOriginMm 10.95,149.04999999999998 -> 158.21,88.25; KiCadOrientationDeg 90 -> 0
- D8120: BoardSide B.Cu -> F.Cu; FootprintOriginMm 102.25,157.25 -> 158.21,91.15; KiCadOrientationDeg 90 -> 0
- D8121: BoardSide B.Cu -> F.Cu; FootprintOriginMm 10.95,158.35 -> 158.21,94.05; KiCadOrientationDeg 90 -> 0
- D8122: FootprintOriginMm 28.05,158.35 -> 154.35,32.95; KiCadOrientationDeg 90 -> 180
- D8123: FootprintOriginMm 44.65,158.35 -> 138.04999999999998,32.95; KiCadOrientationDeg 90 -> 180
- D8124: FootprintOriginMm 61.65,158.35 -> 134.45,99.44999999999999
- D8125: FootprintOriginMm 78.65,158.35 -> 153.85,28.650000000000002
- D8126: FootprintOriginMm 95.65,158.35 -> 169.45,29.450000000000003
- D8127: FootprintOriginMm 112.65,158.35 -> 137.25,28.650000000000002
- D8128: FootprintOriginMm 34.25,158.65 -> 136.35,104.85
- D8129: FootprintOriginMm 51.25,158.65 -> 154.35,24.65; KiCadOrientationDeg 90 -> 180
- D8130: BoardSide B.Cu -> F.Cu; FootprintOriginMm 68.25,158.65 -> 126.75,38.91; KiCadOrientationDeg 90 -> 270
- D8131: FootprintOriginMm 85.25,158.65 -> 159.75,22.95; KiCadOrientationDeg 90 -> 180
- D8132: BoardSide F.Cu -> B.Cu; FootprintOriginMm 22.21,21.55 -> 145.95,22.95; KiCadOrientationDeg 0 -> 180
- D8133: FootprintOriginMm 39.21,21.55 -> 123.85,38.91; KiCadOrientationDeg 0 -> 270
- D8134: FootprintOriginMm 56.21,21.55 -> 158.21,26.05
- D8135: BoardSide F.Cu -> B.Cu; FootprintOriginMm 73.21,21.55 -> 138.04999999999998,24.65; KiCadOrientationDeg 0 -> 180
- D8136: BoardSide F.Cu -> B.Cu; FootprintOriginMm 90.21,21.55 -> 154.25,21.75; KiCadOrientationDeg 0 -> 180
- R8105: FootprintOriginMm 21.240000000000002,45.91 -> 173.51,53.84; KiCadOrientationDeg 0 -> 270
- R8106: BoardSide F.Cu -> B.Cu; FootprintOriginMm 38.24,45.91 -> 169.91,40.94; KiCadOrientationDeg 0 -> 90
- R8107: FootprintOriginMm 55.24,45.91 -> 173.51,50.14; KiCadOrientationDeg 0 -> 270
- R8108: BoardSide F.Cu -> B.Cu; FootprintOriginMm 106.24,46.11 -> 163.64,64.31; KiCadOrientationDeg 0 -> 180
- R8115: FootprintOriginMm 123.24,46.11 -> 173.51,80.94; KiCadOrientationDeg 0 -> 270
- R8116: FootprintOriginMm 140.23999999999998,46.11 -> 173.51,46.44; KiCadOrientationDeg 0 -> 270
- R8117: BoardSide F.Cu -> B.Cu; FootprintOriginMm 157.23999999999998,46.11 -> 169.91,37.24; KiCadOrientationDeg 0 -> 90
- R8118: FootprintOriginMm 5.9399999999999995,47.41 -> 159.54,60.809999999999995
- R8125: FootprintOriginMm 72.24,47.41 -> 173.51,87.54; KiCadOrientationDeg 0 -> 270
- R8126: FootprintOriginMm 89.24,47.41 -> 173.51,91.24; KiCadOrientationDeg 0 -> 270
- R8127: FootprintOriginMm 21.240000000000002,48.11 -> 173.51,39.84; KiCadOrientationDeg 0 -> 270
- R8128: BoardSide F.Cu -> B.Cu; FootprintOriginMm 38.24,48.11 -> 157.44,51.709999999999994; KiCadOrientationDeg 0 -> 180
- R8135: FootprintOriginMm 55.24,48.11 -> 173.51,94.94; KiCadOrientationDeg 0 -> 270
- R8136: FootprintOriginMm 106.24,48.309999999999995 -> 123.50999999999999,116.34; KiCadOrientationDeg 0 -> 270
- R8137: FootprintOriginMm 123.24,48.309999999999995 -> 173.51,36.14; KiCadOrientationDeg 0 -> 270
- R8138: BoardSide F.Cu -> B.Cu; FootprintOriginMm 140.23999999999998,48.309999999999995 -> 169.91,66.84; KiCadOrientationDeg 0 -> 90
- R8145: FootprintOriginMm 157.23999999999998,48.309999999999995 -> 173.51,32.44; KiCadOrientationDeg 0 -> 270
- R8146: BoardSide F.Cu -> B.Cu; FootprintOriginMm 5.9399999999999995,49.61 -> 169.91,25.04; KiCadOrientationDeg 0 -> 90
- R8147: BoardSide F.Cu -> B.Cu; FootprintOriginMm 72.24,49.61 -> 163.71,22.54; KiCadOrientationDeg 0 -> 90
- R8148: BoardSide F.Cu -> B.Cu; FootprintOriginMm 89.24,49.61 -> 169.91,63.14; KiCadOrientationDeg 0 -> 90
- R8167: FootprintOriginMm 103.27,31.900000000000002 -> 109.39999999999999,31.97; KiCadOrientationDeg 180 -> 90
- R8168: FootprintOriginMm 108.17,31.900000000000002 -> 153.79999999999998,49.67; KiCadOrientationDeg 180 -> 90
- R8169: FootprintOriginMm 21.240000000000002,50.309999999999995 -> 173.51,25.84; KiCadOrientationDeg 0 -> 270
- R8170: FootprintOriginMm 38.24,50.309999999999995 -> 173.51,22.14; KiCadOrientationDeg 0 -> 270
- R8171: FootprintOriginMm 55.24,50.309999999999995 -> 123.44,26.61
- R8172: FootprintOriginMm 106.24,50.51 -> 126.34,21.31
- R8173: BoardSide F.Cu -> B.Cu; FootprintOriginMm 123.24,50.51 -> 114.14,112.81; KiCadOrientationDeg 0 -> 180
- R8174: BoardSide F.Cu -> B.Cu; FootprintOriginMm 140.23999999999998,50.51 -> 108.64,21.71; KiCadOrientationDeg 0 -> 180
- R8175: BoardSide F.Cu -> B.Cu; FootprintOriginMm 157.23999999999998,50.51 -> 169.91,59.44; KiCadOrientationDeg 0 -> 90
- R8176: FootprintOriginMm 5.9399999999999995,51.809999999999995 -> 123.50999999999999,120.04; KiCadOrientationDeg 0 -> 270
- R8177: BoardSide F.Cu -> B.Cu; FootprintOriginMm 72.24,51.809999999999995 -> 151.64,87.21; KiCadOrientationDeg 0 -> 180
- U8102: BoardSide B.Cu -> F.Cu; FootprintOriginMm 141.12,124.78 -> 158.78,51.67; KiCadOrientationDeg 180 -> 270
- U8103: BoardSide B.Cu -> F.Cu; FootprintOriginMm 158.12,124.78 -> 158.78,35.769999999999996; KiCadOrientationDeg 180 -> 270
- U8104: BoardSide B.Cu -> F.Cu; FootprintOriginMm 19.92,128.38 -> 141.98,34.769999999999996; KiCadOrientationDeg 180 -> 270
- U8105: BoardSide B.Cu -> F.Cu; FootprintOriginMm 36.92,128.38 -> 124.98,92.82000000000001; KiCadOrientationDeg 180 -> 90
- U8106: FootprintOriginMm 53.919999999999995,128.38 -> 122.18,95.92; KiCadOrientationDeg 180 -> 90
- U8112: FootprintOriginMm 55.97,66.35 -> 155.73000000000002,98.08000000000001; KiCadOrientationDeg 180 -> 0
- U8113: BoardSide B.Cu -> F.Cu; FootprintOriginMm 38.97,142.445 -> 158.465,65.83; KiCadOrientationDeg 180 -> 270
- U8114: BoardSide B.Cu -> F.Cu; FootprintOriginMm 55.97,142.445 -> 142.15,65.83; KiCadOrientationDeg 180 -> 90
- U8115: FootprintOriginMm 72.97,66.35 -> 143.95,61.33; KiCadOrientationDeg 180 -> 270
- U8116: FootprintOriginMm 89.97,66.35 -> 156.68,66.87; KiCadOrientationDeg 180 -> 90
- U8117: FootprintOriginMm 106.97,66.35 -> 142.07,98.08000000000001; KiCadOrientationDeg 180 -> 0

Commit message: Place jack halves with span-aware swaps and route jack-left to 173 open edges
Co-Authored-By: Claude Opus 5.5 <noreply@anthropic.com>
Parts:
- D8108: FootprintOriginMm 109.03,26.41 -> 109.21000000000001,109.93; KiCadOrientationDeg 0 -> 270
- D8109: FootprintOriginMm 100.53,30.31 -> 103.01,106.73; KiCadOrientationDeg 180 -> 90
- D8110: FootprintOriginMm 104.03,24.81 -> 107.91,111.93; KiCadOrientationDeg 180 -> 90
- D8111: BoardSide F.Cu -> B.Cu; FootprintOriginMm 109.21000000000001,109.93 -> 103.91,111.03; KiCadOrientationDeg 270 -> 90
- D8112: FootprintOriginMm 109.21000000000001,22.23 -> 109.03,34.410000000000004; KiCadOrientationDeg 270 -> 0
- D8113: FootprintOriginMm 165.54999999999998,72.25 -> 138.04999999999998,24.65
- D8114: FootprintOriginMm 167.25,57.45 -> 137.25,28.650000000000002
- D8115: BoardSide B.Cu -> F.Cu; FootprintOriginMm 169.85,71.44999999999999 -> 142.61,25.05; KiCadOrientationDeg 90 -> 0
- D8116: FootprintOriginMm 166.15,84.65 -> 138.04999999999998,32.95
- D8117: FootprintOriginMm 158.35,42.75 -> 135.54999999999998,44.45
- D8118: FootprintOriginMm 166.15,44.85 -> 144.75,44.45
- D8119: BoardSide F.Cu -> B.Cu; FootprintOriginMm 158.21,88.25 -> 150.15,44.85; KiCadOrientationDeg 0 -> 180
- D8120: BoardSide F.Cu -> B.Cu; FootprintOriginMm 158.21,91.15 -> 158.35,42.75; KiCadOrientationDeg 0 -> 180
- D8121: BoardSide F.Cu -> B.Cu; FootprintOriginMm 158.21,94.05 -> 145.95,22.95; KiCadOrientationDeg 0 -> 180
- D8122: FootprintOriginMm 154.35,32.95 -> 154.25,21.75
- D8123: BoardSide B.Cu -> F.Cu; FootprintOriginMm 138.04999999999998,32.95 -> 142.61,22.15; KiCadOrientationDeg 180 -> 0
- D8124: FootprintOriginMm 134.45,99.44999999999999 -> 140.54999999999998,21.75; KiCadOrientationDeg 90 -> 180
- D8125: FootprintOriginMm 153.85,28.650000000000002 -> 153.25,60.050000000000004
- D8126: FootprintOriginMm 169.45,29.450000000000003 -> 150.25,57.45
- D8127: FootprintOriginMm 137.25,28.650000000000002 -> 146.55,68.64999999999999
- D8128: FootprintOriginMm 136.35,104.85 -> 149.55,71.44999999999999
- D8129: BoardSide B.Cu -> F.Cu; FootprintOriginMm 154.35,24.65 -> 158.21,88.25; KiCadOrientationDeg 180 -> 0
- D8130: FootprintOriginMm 126.75,38.91 -> 158.21,91.15; KiCadOrientationDeg 270 -> 0
- D8131: FootprintOriginMm 159.75,22.95 -> 152.85,84.65
- D8132: FootprintOriginMm 145.95,22.95 -> 147.45,84.65
- D8133: BoardSide F.Cu -> B.Cu; FootprintOriginMm 123.85,38.91 -> 157.25,74.45; KiCadOrientationDeg 270 -> 180
- D8134: BoardSide F.Cu -> B.Cu; FootprintOriginMm 158.21,26.05 -> 161.55,73.35; KiCadOrientationDeg 0 -> 90
- D8135: FootprintOriginMm 138.04999999999998,24.65 -> 145.25,74.05
- D8136: FootprintOriginMm 154.25,21.75 -> 153.25,73.35; KiCadOrientationDeg 180 -> 90
- R8105: FootprintOriginMm 173.51,53.84 -> 173.51,50.14
- R8106: BoardSide B.Cu -> F.Cu; FootprintOriginMm 169.91,40.94 -> 173.51,46.44; KiCadOrientationDeg 90 -> 270
- R8107: FootprintOriginMm 173.51,50.14 -> 173.51,53.84
- R8108: FootprintOriginMm 163.64,64.31 -> 165.14,98.00999999999999
- R8115: FootprintOriginMm 173.51,80.94 -> 173.51,36.14
- R8116: FootprintOriginMm 173.51,46.44 -> 173.51,32.44
- R8117: FootprintOriginMm 169.91,37.24 -> 163.04,42.309999999999995; KiCadOrientationDeg 90 -> 180
- R8118: FootprintOriginMm 159.54,60.809999999999995 -> 157.23999999999998,96.61
- R8125: FootprintOriginMm 173.51,87.54 -> 173.51,25.84
- R8126: FootprintOriginMm 173.51,91.24 -> 173.51,22.14
- R8127: BoardSide F.Cu -> B.Cu; FootprintOriginMm 173.51,39.84 -> 157.44,51.709999999999994; KiCadOrientationDeg 270 -> 180
- R8128: FootprintOriginMm 157.44,51.709999999999994 -> 153.64,91.71
- R8135: FootprintOriginMm 173.51,94.94 -> 123.50999999999999,120.04
- R8136: FootprintOriginMm 123.50999999999999,116.34 -> 123.50999999999999,123.74
- R8137: FootprintOriginMm 173.51,36.14 -> 106.11,117.04
- R8138: BoardSide B.Cu -> F.Cu; FootprintOriginMm 169.91,66.84 -> 106.11,109.64; KiCadOrientationDeg 90 -> 270
- R8145: BoardSide F.Cu -> B.Cu; FootprintOriginMm 173.51,32.44 -> 147.10999999999999,102.44; KiCadOrientationDeg 270 -> 90
- R8146: FootprintOriginMm 169.91,25.04 -> 147.10999999999999,94.64
- R8147: FootprintOriginMm 163.71,22.54 -> 114.14,112.81; KiCadOrientationDeg 90 -> 180
- R8148: FootprintOriginMm 169.91,63.14 -> 112.00999999999999,70.74
- R8167: FootprintOriginMm 109.39999999999999,31.97 -> 100.07,44.5; KiCadOrientationDeg 90 -> 180
- R8169: BoardSide F.Cu -> B.Cu; FootprintOriginMm 173.51,25.84 -> 133.64,28.81; KiCadOrientationDeg 270 -> 180
- R8170: BoardSide F.Cu -> B.Cu; FootprintOriginMm 173.51,22.14 -> 166.73999999999998,42.309999999999995; KiCadOrientationDeg 270 -> 180
- R8171: BoardSide F.Cu -> B.Cu; FootprintOriginMm 123.44,26.61 -> 163.71,22.54; KiCadOrientationDeg 0 -> 90
- R8172: BoardSide F.Cu -> B.Cu; FootprintOriginMm 126.34,21.31 -> 169.91,63.14; KiCadOrientationDeg 0 -> 90
- R8173: FootprintOriginMm 114.14,112.81 -> 167.64,87.21
- R8174: BoardSide B.Cu -> F.Cu; FootprintOriginMm 108.64,21.71 -> 173.51,66.84; KiCadOrientationDeg 180 -> 270
- R8175: FootprintOriginMm 169.91,59.44 -> 151.64,87.21; KiCadOrientationDeg 90 -> 180
- R8176: BoardSide F.Cu -> B.Cu; FootprintOriginMm 123.50999999999999,120.04 -> 169.91,66.84; KiCadOrientationDeg 270 -> 90
- R8177: FootprintOriginMm 151.64,87.21 -> 168.83999999999997,98.31

Commit message: Regenerate and rebuild both jack halves with the hot-quad escape reservation
Evidence rebound (peripheral epoch, foil-collar proposal, control receipt);
jack boards rebuilt from the new placement with source planes and no signal
copper, ready for CI routing.

Co-Authored-By: Claude Opus 5.5 <noreply@anthropic.com>
Parts:
- C8115: BoardSide F.Cu -> B.Cu; FootprintOriginMm 159.105,57.510000000000005 -> 152.96,45.155; KiCadOrientationDeg 270 -> 90
- C8116: BoardSide F.Cu -> B.Cu; FootprintOriginMm 159.105,45.24 -> 163.87,45.155
- C8117: FootprintOriginMm 159.105,41.61 -> 159.105,42.510000000000005
- C8118: FootprintOriginMm 159.105,29.339999999999996 -> 159.105,30.240000000000002
- C8139: FootprintOriginMm 150.04000000000002,98.08000000000001 -> 151.24,98.08000000000001
- C8140: FootprintOriginMm 161.42000000000002,98.08000000000001 -> 162.62,98.08000000000001
- C8141: FootprintOriginMm 143.95,55.64 -> 143.95,54.44
- C8142: FootprintOriginMm 143.95,67.02 -> 143.95,65.82
- C8145: FootprintOriginMm 137.06,98.78000000000002 -> 138.26000000000002,98.78000000000002
- C8146: FootprintOriginMm 147.07999999999998,98.78000000000002 -> 148.28,98.78000000000002
- D8108: FootprintOriginMm 109.21000000000001,109.93 -> 109.03,108.01; KiCadOrientationDeg 270 -> 0
- D8109: BoardSide B.Cu -> F.Cu; FootprintOriginMm 103.01,106.73 -> 109.03,104.01; KiCadOrientationDeg 90 -> 0
- D8110: FootprintOriginMm 107.91,111.93 -> 105.43,108.91; KiCadOrientationDeg 90 -> 180
- D8111: FootprintOriginMm 103.91,111.03 -> 95.81,109.83000000000001
- D8112: FootprintOriginMm 109.03,34.410000000000004 -> 92.21000000000001,39.33; KiCadOrientationDeg 0 -> 270
- D8113: FootprintOriginMm 138.04999999999998,24.65 -> 145.95,22.95
- D8114: BoardSide B.Cu -> F.Cu; FootprintOriginMm 137.25,28.650000000000002 -> 142.61,22.15; KiCadOrientationDeg 90 -> 0
- D8115: BoardSide F.Cu -> B.Cu; FootprintOriginMm 142.61,25.05 -> 153.05,29.450000000000003; KiCadOrientationDeg 0 -> 90
- D8116: BoardSide B.Cu -> F.Cu; FootprintOriginMm 138.04999999999998,32.95 -> 142.61,25.05; KiCadOrientationDeg 180 -> 0
- D8117: FootprintOriginMm 135.54999999999998,44.45 -> 138.04999999999998,32.95
- D8118: FootprintOriginMm 144.75,44.45 -> 144.75,42.75
- D8119: FootprintOriginMm 150.15,44.85 -> 135.54999999999998,43.25
- D8120: FootprintOriginMm 158.35,42.75 -> 146.25,46.75; KiCadOrientationDeg 180 -> 90
- D8121: BoardSide B.Cu -> F.Cu; FootprintOriginMm 145.95,22.95 -> 158.21,23.35; KiCadOrientationDeg 180 -> 0
- D8122: BoardSide B.Cu -> F.Cu; FootprintOriginMm 154.25,21.75 -> 158.21,26.25; KiCadOrientationDeg 180 -> 0
- D8123: BoardSide F.Cu -> B.Cu; FootprintOriginMm 142.61,22.15 -> 157.85,22.95; KiCadOrientationDeg 0 -> 180
- D8124: FootprintOriginMm 140.54999999999998,21.75 -> 153.85,24.05; KiCadOrientationDeg 180 -> 90
- D8125: BoardSide B.Cu -> F.Cu; FootprintOriginMm 153.25,60.050000000000004 -> 158.21,91.15; KiCadOrientationDeg 90 -> 0
- D8126: FootprintOriginMm 150.25,57.45 -> 167.35,84.65; KiCadOrientationDeg 90 -> 180
- D8127: BoardSide B.Cu -> F.Cu; FootprintOriginMm 146.55,68.64999999999999 -> 158.21,88.25; KiCadOrientationDeg 90 -> 0
- D8128: FootprintOriginMm 149.55,71.44999999999999 -> 157.25,74.45; KiCadOrientationDeg 90 -> 180
- D8129: BoardSide F.Cu -> B.Cu; FootprintOriginMm 158.21,88.25 -> 136.25,62.35; KiCadOrientationDeg 0 -> 90
- D8130: BoardSide F.Cu -> B.Cu; FootprintOriginMm 158.21,91.15 -> 146.55,52.15; KiCadOrientationDeg 0 -> 90
- D8131: FootprintOriginMm 152.85,84.65 -> 145.25,74.05
- D8132: FootprintOriginMm 147.45,84.65 -> 146.55,68.64999999999999; KiCadOrientationDeg 180 -> 90
- D8133: BoardSide B.Cu -> F.Cu; FootprintOriginMm 157.25,74.45 -> 158.21,94.05; KiCadOrientationDeg 180 -> 0
- D8134: BoardSide B.Cu -> F.Cu; FootprintOriginMm 161.55,73.35 -> 159.35,98.31; KiCadOrientationDeg 90 -> 270
- D8135: FootprintOriginMm 145.25,74.05 -> 164.54999999999998,100.85
- D8136: FootprintOriginMm 153.25,73.35 -> 168.85,99.44999999999999
- R8105: FootprintOriginMm 173.51,50.14 -> 173.51,39.84
- R8106: BoardSide F.Cu -> B.Cu; FootprintOriginMm 173.51,46.44 -> 169.91,41.54; KiCadOrientationDeg 270 -> 90
- R8107: BoardSide F.Cu -> B.Cu; FootprintOriginMm 173.51,53.84 -> 169.91,52.04; KiCadOrientationDeg 270 -> 90
- R8108: FootprintOriginMm 165.14,98.00999999999999 -> 167.64,87.21
- R8115: FootprintOriginMm 173.51,36.14 -> 173.51,22.14
- R8116: FootprintOriginMm 173.51,32.44 -> 173.51,25.84
- R8117: FootprintOriginMm 163.04,42.309999999999995 -> 169.91,37.84; KiCadOrientationDeg 180 -> 90
- R8118: FootprintOriginMm 157.23999999999998,96.61 -> 159.54,60.809999999999995
- R8125: FootprintOriginMm 173.51,25.84 -> 173.51,32.44
- R8126: FootprintOriginMm 173.51,22.14 -> 173.51,36.14
- R8127: FootprintOriginMm 157.44,51.709999999999994 -> 136.64,55.809999999999995
- R8128: FootprintOriginMm 153.64,91.71 -> 136.64,94.31
- R8135: FootprintOriginMm 123.50999999999999,120.04 -> 123.50999999999999,127.14
- R8136: FootprintOriginMm 123.50999999999999,123.74 -> 123.50999999999999,130.83999999999997
- R8137: BoardSide F.Cu -> B.Cu; FootprintOriginMm 106.11,117.04 -> 104.34,112.00999999999999; KiCadOrientationDeg 270 -> 180
- R8138: FootprintOriginMm 106.11,109.64 -> 105.81,111.24
- R8145: FootprintOriginMm 147.10999999999999,102.44 -> 169.91,90.14
- R8146: FootprintOriginMm 147.10999999999999,94.64 -> 170.31,81.34
- R8147: FootprintOriginMm 114.14,112.81 -> 169.91,66.84; KiCadOrientationDeg 180 -> 90
- R8148: BoardSide B.Cu -> F.Cu; FootprintOriginMm 112.00999999999999,70.74 -> 143.23999999999998,60.809999999999995; KiCadOrientationDeg 90 -> 0
- R8167: BoardSide B.Cu -> F.Cu; FootprintOriginMm 100.07,44.5 -> 108.77,100.19999999999999; KiCadOrientationDeg 180 -> 0
- R8168: FootprintOriginMm 153.79999999999998,49.67 -> 108.5,100.36999999999999
- R8169: FootprintOriginMm 133.64,28.81 -> 109.34,22.51
- R8170: FootprintOriginMm 166.73999999999998,42.309999999999995 -> 166.83999999999997,42.309999999999995
- R8171: FootprintOriginMm 163.71,22.54 -> 169.91,25.04
- R8172: FootprintOriginMm 169.91,63.14 -> 170.31,76.14
- R8173: BoardSide B.Cu -> F.Cu; FootprintOriginMm 167.64,87.21 -> 173.51,53.84; KiCadOrientationDeg 180 -> 270
- R8174: FootprintOriginMm 173.51,66.84 -> 173.51,73.54
- R8175: FootprintOriginMm 151.64,87.21 -> 148.94,87.21
- R8176: BoardSide B.Cu -> F.Cu; FootprintOriginMm 169.91,66.84 -> 173.51,66.84; KiCadOrientationDeg 90 -> 270
- R8177: FootprintOriginMm 168.83999999999997,98.31 -> 169.91,105.64; KiCadOrientationDeg 180 -> 90
- U8102: BoardSide F.Cu -> B.Cu; FootprintOriginMm 158.78,51.67 -> 158.12,46.18; KiCadOrientationDeg 270 -> 180
- U8103: FootprintOriginMm 158.78,35.769999999999996 -> 158.78,36.67
- U8112: FootprintOriginMm 155.73000000000002,98.08000000000001 -> 156.93,98.08000000000001
- U8115: FootprintOriginMm 143.95,61.33 -> 143.95,60.129999999999995
- U8117: FootprintOriginMm 142.07,98.08000000000001 -> 143.27,98.08000000000001
