File: boards/osc-jack-left/sheets/oscillator_O2_JL.kicad_sch (KiCad schematic)
At the start: 57 parts, among them J201 WQP518MA, J202 WQP518MA, J203 WQP518MA, J204 WQP518MA, J205 WQP518MA, J206 WQP518MA, J207 WQP518MA, J208 WQP518MA, U1201 ADG5412FBRUZ, U1202 ADG5412FBRUZ, U1203 ADG5412FBRUZ, U1204 ADG5412FBRUZ, U1216 OPA4196IDR, U1217 OPA4196IDR, U1218 OPA4197IPWR

Commit message: Move jack halves to six layers with locality placement and grid routing
Owner decision 2026-10-03 (#38): a cut-line bound showed the four-layer
jack halves could not carry their signal nets with intact planes, so both
halves move to six layers and their free packages are re-placed for
locality.

- Placement: scripts/checks/jack_locality.py replaces the
  connectivity-blind first-fit J placer. Packages are pulled toward the
  fixed jacks, LEDs and headers on their nets and toward their own
  module's hardware, then legalized; IC/bypass clusters stay aligned.
  Panel hardware and headers do not move.
- Stack: F/In2/In3/B signals, In1 AGND plane, -12V fill on In3, +12V
  plane on In4; +5V as tracks.
- Routing: scripts/pcbgen/route_jack_grid.py stages terminal arrays,
  rail fanouts and links, signal batches, rip-up-and-reroute and AGND
  stitching, keeping only natively checked stages (0 DRC errors,
  0 parity). The grid router gains N-layer support, windowed search,
  plane fanout, a plane-fill split guard and rip-up-and-reroute.
- Evidence chain: a bounded jack-locality partition transition is
  chained onto the connector-locality proof; superseded four-layer
  stage reports are removed.

Checkpoint: JL 411 and JR 518 native open edges remain. This is a routed
draft in progress; electrical and physical qualification NOT RUN.

Co-Authored-By: Claude Opus 5.5 <noreply@anthropic.com>
Parts:
- C1221: FootprintOriginMm 133.76000000000002,85.355 -> 33.959999999999994,62.155
- C1222: FootprintOriginMm 144.67000000000002,85.355 -> 44.87,62.155
- C1223: BoardSide B.Cu -> F.Cu; FootprintOriginMm 150.76000000000002,85.355 -> 39.205,70.57; KiCadOrientationDeg 90 -> 180
- C1224: BoardSide B.Cu -> F.Cu; FootprintOriginMm 161.67000000000002,85.355 -> 39.205,59.66; KiCadOrientationDeg 90 -> 180
- C1225: BoardSide B.Cu -> F.Cu; FootprintOriginMm 33.959999999999994,91.755 -> 39.955,85.46000000000001; KiCadOrientationDeg 90 -> 0
- C1226: BoardSide B.Cu -> F.Cu; FootprintOriginMm 44.87,91.755 -> 39.955,96.37; KiCadOrientationDeg 90 -> 0
- C1227: BoardSide B.Cu -> F.Cu; FootprintOriginMm 50.959999999999994,91.755 -> 22.605,69.97; KiCadOrientationDeg 90 -> 180
- C1228: BoardSide B.Cu -> F.Cu; FootprintOriginMm 61.87,91.755 -> 22.605,59.06; KiCadOrientationDeg 90 -> 180
- C1240: BoardSide B.Cu -> F.Cu; FootprintOriginMm 44.28,134.23000000000002 -> 38.76,72.86000000000001; KiCadOrientationDeg 90 -> 180
- C1241: BoardSide B.Cu -> F.Cu; FootprintOriginMm 33.959999999999994,134.23000000000002 -> 38.76,83.18; KiCadOrientationDeg 90 -> 180
- C1250: FootprintOriginMm 94.98,24.55 -> 42.419999999999995,71.55; KiCadOrientationDeg 90 -> 0
- C1251: FootprintOriginMm 84.96,24.55 -> 31.04,71.55; KiCadOrientationDeg 90 -> 180
- C1252: FootprintOriginMm 111.98,24.55 -> 33.96,88.78000000000002; KiCadOrientationDeg 90 -> 270
- C1253: FootprintOriginMm 101.96,24.55 -> 43.98,88.78000000000002; KiCadOrientationDeg 90 -> 270
- DO1201: FootprintOriginMm 124.23,140.01 -> 27.93,58.010000000000005
- DO1202: FootprintOriginMm 128.53,140.01 -> 31.53,98.91
- DO1203: FootprintOriginMm 10.43,140.51 -> 42.03,58.010000000000005
- DO1204: FootprintOriginMm 30.53,140.91 -> 27.23,98.81
- R1201: FootprintOriginMm 163.73999999999998,59.61 -> 23.94,58.91
- R1202: FootprintOriginMm 27.740000000000002,60.01 -> 34.64,55.309999999999995
- R1203: FootprintOriginMm 44.74,60.01 -> 39.709999999999994,97.24; KiCadOrientationDeg 180 -> 90
- R1204: FootprintOriginMm 61.74,60.01 -> 27.91,85.04; KiCadOrientationDeg 180 -> 90
- R1205: FootprintOriginMm 78.74,60.01 -> 35.54,99.21
- R1206: FootprintOriginMm 95.74,60.01 -> 39.24,100.21
- R1207: FootprintOriginMm 112.74,60.01 -> 23.240000000000002,98.61
- R1208: FootprintOriginMm 129.73999999999998,60.01 -> 27.94,91.71
- R1209: FootprintOriginMm 146.73999999999998,60.01 -> 23.94,56.709999999999994
- R1210: FootprintOriginMm 27.740000000000002,62.209999999999994 -> 27.94,54.91
- R1211: FootprintOriginMm 44.74,62.209999999999994 -> 35.54,101.41
- R1212: FootprintOriginMm 61.74,62.209999999999994 -> 44.01,85.04; KiCadOrientationDeg 180 -> 90
- R1213: FootprintOriginMm 78.74,62.209999999999994 -> 38.34,54.91
- R1214: FootprintOriginMm 95.74,62.209999999999994 -> 24.240000000000002,54.51
- R1215: FootprintOriginMm 112.74,62.209999999999994 -> 20.240000000000002,56.709999999999994
- R1216: FootprintOriginMm 129.73999999999998,62.209999999999994 -> 33.91,92.44; KiCadOrientationDeg 180 -> 90
- RB1202: FootprintOriginMm 168.67000000000002,42.7 -> 27.37,95.0
- RB1203: FootprintOriginMm 6.57,44.1 -> 31.47,85.0
- RB1204: FootprintOriginMm 6.57,47.7 -> 36.800000000000004,95.67; KiCadOrientationDeg 180 -> 90
- RB1205: FootprintOriginMm 6.57,51.300000000000004 -> 27.37,68.5
- RB1206: FootprintOriginMm 6.57,54.9 -> 32.57,58.5
- RB1207: FootprintOriginMm 11.469999999999999,56.7 -> 43.07,74.6
- RB1208: FootprintOriginMm 166.57000000000002,56.7 -> 37.470000000000006,58.2
- RB1209: FootprintOriginMm 6.57,58.5 -> 43.07,68.5
- U1201: FootprintOriginMm 138.92000000000002,86.38000000000001 -> 39.12,63.18
- U1202: BoardSide B.Cu -> F.Cu; FootprintOriginMm 155.92000000000002,86.38000000000001 -> 39.58,65.41; KiCadOrientationDeg 180 -> 270
- U1203: BoardSide B.Cu -> F.Cu; FootprintOriginMm 39.12,92.78 -> 39.58,90.62; KiCadOrientationDeg 180 -> 90
- U1204: BoardSide B.Cu -> F.Cu; FootprintOriginMm 56.12,92.78 -> 22.98,64.81; KiCadOrientationDeg 180 -> 270
- U1216: FootprintOriginMm 89.97,25.25 -> 36.73,71.55
- U1217: FootprintOriginMm 106.97,25.25 -> 38.97,88.08000000000001; KiCadOrientationDeg 180 -> 0
- U1218: BoardSide B.Cu -> F.Cu; FootprintOriginMm 39.12,134.93 -> 39.46,78.02000000000001; KiCadOrientationDeg 180 -> 270

Commit message: Place jack halves with span-aware swaps and route jack-left to 173 open edges
Co-Authored-By: Claude Opus 5.5 <noreply@anthropic.com>
Parts:
- DO1201: FootprintOriginMm 27.93,58.010000000000005 -> 27.23,98.81
- DO1203: FootprintOriginMm 42.03,58.010000000000005 -> 44.63,101.11
- DO1204: FootprintOriginMm 27.23,98.81 -> 27.93,58.010000000000005
- R1201: FootprintOriginMm 23.94,58.91 -> 27.94,54.91
- R1203: FootprintOriginMm 39.709999999999994,97.24 -> 27.94,91.71; KiCadOrientationDeg 90 -> 180
- R1205: BoardSide B.Cu -> F.Cu; FootprintOriginMm 35.54,99.21 -> 42.11,58.84; KiCadOrientationDeg 180 -> 270
- R1206: FootprintOriginMm 39.24,100.21 -> 38.34,54.91
- R1207: FootprintOriginMm 23.240000000000002,98.61 -> 35.54,101.41
- R1208: FootprintOriginMm 27.94,91.71 -> 35.54,99.21
- R1209: FootprintOriginMm 23.94,56.709999999999994 -> 23.240000000000002,98.61
- R1210: FootprintOriginMm 27.94,54.91 -> 33.91,92.44; KiCadOrientationDeg 180 -> 90
- R1211: FootprintOriginMm 35.54,101.41 -> 39.24,100.21
- R1212: FootprintOriginMm 44.01,85.04 -> 39.709999999999994,97.24
- R1213: FootprintOriginMm 38.34,54.91 -> 23.94,56.709999999999994
- R1214: FootprintOriginMm 24.240000000000002,54.51 -> 20.240000000000002,56.709999999999994
- R1215: FootprintOriginMm 20.240000000000002,56.709999999999994 -> 24.240000000000002,54.51
- R1216: FootprintOriginMm 33.91,92.44 -> 23.94,58.91; KiCadOrientationDeg 90 -> 180
- RB1202: FootprintOriginMm 27.37,95.0 -> 26.07,74.6
- RB1204: FootprintOriginMm 36.800000000000004,95.67 -> 43.07,74.6; KiCadOrientationDeg 90 -> 180
- RB1205: FootprintOriginMm 27.37,68.5 -> 36.800000000000004,95.67; KiCadOrientationDeg 180 -> 90
- RB1206: FootprintOriginMm 32.57,58.5 -> 43.07,68.5
- RB1207: FootprintOriginMm 43.07,74.6 -> 27.37,68.5
- RB1209: FootprintOriginMm 43.07,68.5 -> 32.57,58.5

Commit message: Regenerate and rebuild both jack halves with the hot-quad escape reservation
Evidence rebound (peripheral epoch, foil-collar proposal, control receipt);
jack boards rebuilt from the new placement with source planes and no signal
copper, ready for CI routing.

Co-Authored-By: Claude Opus 5.5 <noreply@anthropic.com>
Parts:
- C1227: FootprintOriginMm 22.605,69.97 -> 23.355,85.46000000000001; KiCadOrientationDeg 180 -> 0
- C1228: FootprintOriginMm 22.605,59.06 -> 23.355,96.37; KiCadOrientationDeg 180 -> 0
- C1250: FootprintOriginMm 42.419999999999995,71.55 -> 43.62,71.55
- C1251: FootprintOriginMm 31.04,71.55 -> 32.24,71.55
- DO1201: FootprintOriginMm 27.23,98.81 -> 31.53,58.31
- DO1202: FootprintOriginMm 31.53,98.91 -> 40.13,58.010000000000005
- DO1203: FootprintOriginMm 44.63,101.11 -> 35.83,58.010000000000005
- DO1204: FootprintOriginMm 27.93,58.010000000000005 -> 27.23,58.010000000000005
- R1201: FootprintOriginMm 27.94,54.91 -> 31.64,100.21
- R1202: FootprintOriginMm 34.64,55.309999999999995 -> 31.64,98.00999999999999
- R1203: BoardSide B.Cu -> F.Cu; FootprintOriginMm 27.94,91.71 -> 25.11,62.04; KiCadOrientationDeg 180 -> 270
- R1204: FootprintOriginMm 27.91,85.04 -> 28.71,66.24
- R1205: BoardSide F.Cu -> B.Cu; FootprintOriginMm 42.11,58.84 -> 27.94,69.21; KiCadOrientationDeg 270 -> 180
- R1206: FootprintOriginMm 38.34,54.91 -> 27.11,74.54; KiCadOrientationDeg 180 -> 90
- R1207: BoardSide B.Cu -> F.Cu; FootprintOriginMm 35.54,101.41 -> 42.11,72.04; KiCadOrientationDeg 180 -> 270
- R1208: BoardSide B.Cu -> F.Cu; FootprintOriginMm 35.54,99.21 -> 42.11,58.84; KiCadOrientationDeg 180 -> 270
- R1209: FootprintOriginMm 23.240000000000002,98.61 -> 39.04,97.91
- R1210: FootprintOriginMm 33.91,92.44 -> 39.04,100.11; KiCadOrientationDeg 90 -> 180
- R1211: FootprintOriginMm 39.24,100.21 -> 35.34,100.11
- R1212: FootprintOriginMm 39.709999999999994,97.24 -> 35.34,97.91; KiCadOrientationDeg 90 -> 180
- R1213: FootprintOriginMm 23.94,56.709999999999994 -> 24.240000000000002,100.11
- R1214: FootprintOriginMm 20.240000000000002,56.709999999999994 -> 27.94,100.31
- R1215: FootprintOriginMm 24.240000000000002,54.51 -> 28.71,97.34; KiCadOrientationDeg 180 -> 90
- R1216: FootprintOriginMm 23.94,58.91 -> 27.91,85.04; KiCadOrientationDeg 180 -> 90
- RB1202: FootprintOriginMm 26.07,74.6 -> 45.370000000000005,85.0
- RB1204: FootprintOriginMm 43.07,74.6 -> 28.0,93.07; KiCadOrientationDeg 180 -> 90
- RB1205: FootprintOriginMm 36.800000000000004,95.67 -> 23.77,95.0; KiCadOrientationDeg 90 -> 180
- RB1206: FootprintOriginMm 43.07,68.5 -> 40.17,95.0
- RB1207: FootprintOriginMm 27.37,68.5 -> 35.27,95.0
- RB1208: BoardSide B.Cu -> F.Cu; FootprintOriginMm 37.470000000000006,58.2 -> 23.77,65.69999999999999; KiCadOrientationDeg 180 -> 0
- RB1209: BoardSide B.Cu -> F.Cu; FootprintOriginMm 32.57,58.5 -> 23.77,69.3; KiCadOrientationDeg 180 -> 0
- U1204: FootprintOriginMm 22.98,64.81 -> 22.98,90.62; KiCadOrientationDeg 270 -> 90
- U1216: FootprintOriginMm 36.73,71.55 -> 37.93,71.55
