File: boards/osc-jack-right/sheets/offset_A03_JR.kicad_sch (KiCad schematic)
At the start: 59 parts, among them J1508 WQP518MA, J1509 WQP518MA, J1510 WQP518MA, U7302 ADG5412FBRUZ, U7303 ADG5412FBRUZ, U7306 OPA4197IPWR, U7307 LM393BIDR, U7308 LM393BIDR, U7309 OPA4196IDR

Commit message: Bind exact precision-feedback resistor and capacitor identities
Parts:
- C7306: symbol zudo-osc-hole-field:C0603C101J5GACTU -> zudo-osc-hole-field:C0603C102J5GACTU; MPN (none) -> C0603C102J5GACTU; Manufacturer (none) -> KEMET
- R7329: symbol zudo-osc-hole-field:RC0603FR-07100KL -> zudo-osc-hole-field:RC0603FR-07100RL; MPN (none) -> RC0603FR-07100RL; Manufacturer (none) -> Yageo
Changed lines of the file:
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@@
   (global_label "X84E51647AEFBA0482D1F" (shape passive) (at 993.14 142.24 0) (effects (font (size 1.27 1.27)) (justify right)))
   (global_label "XAAFC7EABDDD9A637A91C" (shape passive) (at 1003.3 142.24 180) (effects (font (size 1.27 1.27)) (justify left)))
-  (symbol (lib_id "zudo-osc-hole-field:RC0603FR-07100KL") (at 1061.72 142.24 0) (unit 0)
+  (symbol (lib_id "zudo-osc-hole-field:RC0603FR-07100RL") (at 1061.72 142.24 0) (unit 0)
     (exclude_from_sim no) (in_bom yes) (on_board yes) (dnp no)
     (property "Reference" "R7329" (at 1064.72 139.24 0) (effects (font (size 1.27 1.27))))
@@
     (property "Footprint" "zudo-osc-hole-field:R0603" (at 1061.72 142.24 0) (effects (font (size 1.27 1.27)) (hide yes)))
     (property "Datasheet" "" (at 1061.72 142.24 0) (effects (font (size 1.27 1.27)) (hide yes)))
-    (property "MPN" "" (at 1061.72 142.24 0) (effects (font (size 1.27 1.27)) (hide yes)))
-    (property "Manufacturer" "" (at 1061.72 142.24 0) (effects (font (size 1.27 1.27)) (hide yes)))
+    (property "MPN" "RC0603FR-07100RL" (at 1061.72 142.24 0) (effects (font (size 1.27 1.27)) (hide yes)))
+    (property "Manufacturer" "Yageo" (at 1061.72 142.24 0) (effects (font (size 1.27 1.27)) (hide yes)))
     (property "LCSC" "" (at 1061.72 142.24 0) (effects (font (size 1.27 1.27)) (hide yes)))
     (property "Block" "${SHEETNAME}" (at 1061.72 142.24 0) (effects (font (size 1.27 1.27)) (hide yes)))
@@
   (global_label "XAAFC7EABDDD9A637A91C" (shape passive) (at 1056.64 142.24 0) (effects (font (size 1.27 1.27)) (justify right)))
   (global_label "XEFF08C1287643021E67D" (shape passive) (at 1066.8 142.24 180) (effects (font (size 1.27 1.27)) (justify left)))
-  (symbol (lib_id "zudo-osc-hole-field:C0603C101J5GACTU") (at 45.72 180.34 0) (unit 0)
+  (symbol (lib_id "zudo-osc-hole-field:C0603C102J5GACTU") (at 45.72 180.34 0) (unit 0)
     (exclude_from_sim no) (in_bom yes) (on_board yes) (dnp no)
     (property "Reference" "C7306" (at 48.72 177.34 0) (effects (font (size 1.27 1.27))))
@@
     (property "Footprint" "zudo-osc-hole-field:C0603" (at 45.72 180.34 0) (effects (font (size 1.27 1.27)) (hide yes)))
     (property "Datasheet" "" (at 45.72 180.34 0) (effects (font (size 1.27 1.27)) (hide yes)))
-    (property "MPN" "" (at 45.72 180.34 0) (effects (font (size 1.27 1.27)) (hide yes)))
-    (property "Manufacturer" "" (at 45.72 180.34 0) (effects (font (size 1.27 1.27)) (hide yes)))
+    (property "MPN" "C0603C102J5GACTU" (at 45.72 180.34 0) (effects (font (size 1.27 1.27)) (hide yes)))
+    (property "Manufacturer" "KEMET" (at 45.72 180.34 0) (effects (font (size 1.27 1.27)) (hide yes)))
     (property "LCSC" "" (at 45.72 180.34 0) (effects (font (size 1.27 1.27)) (hide yes)))
     (property "Block" "${SHEETNAME}" (at 45.72 180.34 0) (effects (font (size 1.27 1.27)) (hide yes)))
