File: boards/osc-jack-right/sheets/offset_A03_JR.kicad_sch (KiCad schematic)
At the start: 59 parts, among them J1508 WQP518MA, J1509 WQP518MA, J1510 WQP518MA, U7302 ADG5412FBRUZ, U7303 ADG5412FBRUZ, U7306 OPA4197IPWR, U7307 LM393BIDR, U7308 LM393BIDR, U7309 OPA4196IDR

Commit message: Move jack halves to six layers with locality placement and grid routing
Owner decision 2026-10-03 (#38): a cut-line bound showed the four-layer
jack halves could not carry their signal nets with intact planes, so both
halves move to six layers and their free packages are re-placed for
locality.

- Placement: scripts/checks/jack_locality.py replaces the
  connectivity-blind first-fit J placer. Packages are pulled toward the
  fixed jacks, LEDs and headers on their nets and toward their own
  module's hardware, then legalized; IC/bypass clusters stay aligned.
  Panel hardware and headers do not move.
- Stack: F/In2/In3/B signals, In1 AGND plane, -12V fill on In3, +12V
  plane on In4; +5V as tracks.
- Routing: scripts/pcbgen/route_jack_grid.py stages terminal arrays,
  rail fanouts and links, signal batches, rip-up-and-reroute and AGND
  stitching, keeping only natively checked stages (0 DRC errors,
  0 parity). The grid router gains N-layer support, windowed search,
  plane fanout, a plane-fill split guard and rip-up-and-reroute.
- Evidence chain: a bounded jack-locality partition transition is
  chained onto the connector-locality proof; superseded four-layer
  stage reports are removed.

Checkpoint: JL 411 and JR 518 native open edges remain. This is a routed
draft in progress; electrical and physical qualification NOT RUN.

Co-Authored-By: Claude Opus 5.5 <noreply@anthropic.com>
Parts:
- C7306: BoardSide B.Cu -> F.Cu; FootprintOriginMm 231.73999999999998,21.26 -> 261.74,153.26000000000002; KiCadOrientationDeg 180 -> 0
- C7308: FootprintOriginMm 252.76000000000002,127.35499999999999 -> 252.76000000000002,114.155
- C7309: FootprintOriginMm 263.67,127.35499999999999 -> 263.67,114.155
- C7310: FootprintOriginMm 269.76,127.35499999999999 -> 254.96,107.755
- C7311: FootprintOriginMm 280.67,127.35499999999999 -> 265.87,107.755
- C7312: BoardSide F.Cu -> B.Cu; FootprintOriginMm 262.37,42.919999999999995 -> 269.03999999999996,127.445; KiCadOrientationDeg 270 -> 180
- C7313: BoardSide F.Cu -> B.Cu; FootprintOriginMm 258.56000000000006,31.54 -> 280.41999999999996,131.255; KiCadOrientationDeg 90 -> 0
- C7314: FootprintOriginMm 279.37,42.919999999999995 -> 262.37,127.52
- C7315: FootprintOriginMm 275.56000000000006,31.54 -> 258.56000000000006,116.14
- C7320: FootprintOriginMm 259.76000000000005,58.86 -> 261.83,150.98; KiCadOrientationDeg 180 -> 0
- C7321: FootprintOriginMm 259.76000000000005,69.17999999999999 -> 261.83,140.66; KiCadOrientationDeg 180 -> 0
- C7322: FootprintOriginMm 230.98,65.64999999999999 -> 264.98,136.85
- C7323: FootprintOriginMm 220.96,65.64999999999999 -> 254.96000000000004,136.85
- D7301: BoardSide B.Cu -> F.Cu; FootprintOriginMm 197.13,140.01 -> 259.53000000000003,106.91; KiCadOrientationDeg 180 -> 0
- D7302: FootprintOriginMm 204.93,140.01 -> 248.63,103.51
- D7303: BoardSide F.Cu -> B.Cu; FootprintOriginMm 192.21,103.15 -> 264.15000000000003,128.55; KiCadOrientationDeg 0 -> 180
- D7304: FootprintOriginMm 209.21,103.15 -> 275.85,136.91000000000003; KiCadOrientationDeg 0 -> 270
- D7305: FootprintOriginMm 243.21,103.65 -> 275.85,131.51000000000002; KiCadOrientationDeg 0 -> 270
- D7306: BoardSide F.Cu -> B.Cu; FootprintOriginMm 260.21000000000004,103.65 -> 283.45000000000005,140.95; KiCadOrientationDeg 0 -> 180
- D7308: FootprintOriginMm 277.21000000000004,103.65 -> 278.75,136.91000000000003; KiCadOrientationDeg 0 -> 270
- D7309: BoardSide F.Cu -> B.Cu; FootprintOriginMm 294.21000000000004,103.65 -> 249.35,115.55; KiCadOrientationDeg 0 -> 90
- D7310: BoardSide F.Cu -> B.Cu; FootprintOriginMm 226.21,104.65 -> 281.15000000000003,128.55; KiCadOrientationDeg 0 -> 180
- D7311: BoardSide F.Cu -> B.Cu; FootprintOriginMm 192.21,106.05 -> 266.25,115.55; KiCadOrientationDeg 0 -> 90
- D7313: FootprintOriginMm 209.21,106.05 -> 261.15,115.31; KiCadOrientationDeg 0 -> 270
- D7314: BoardSide F.Cu -> B.Cu; FootprintOriginMm 243.21,106.55 -> 269.15,113.44999999999999; KiCadOrientationDeg 0 -> 90
- D7315: BoardSide F.Cu -> B.Cu; FootprintOriginMm 260.21000000000004,106.55 -> 247.95,110.55; KiCadOrientationDeg 0 -> 180
- D7316: BoardSide F.Cu -> B.Cu; FootprintOriginMm 277.21000000000004,106.55 -> 242.54999999999998,110.55; KiCadOrientationDeg 0 -> 180
- R7305: BoardSide B.Cu -> F.Cu; FootprintOriginMm 220.91,91.34 -> 269.74,162.51; KiCadOrientationDeg 90 -> 0
- R7306: FootprintOriginMm 237.91,91.34 -> 272.64,117.31; KiCadOrientationDeg 90 -> 180
- R7307: FootprintOriginMm 254.91,91.34 -> 255.64,104.50999999999999; KiCadOrientationDeg 90 -> 180
- R7308: BoardSide B.Cu -> F.Cu; FootprintOriginMm 271.91,91.34 -> 262.14,133.01; KiCadOrientationDeg 90 -> 0
- R7309: BoardSide B.Cu -> F.Cu; FootprintOriginMm 288.91,91.34 -> 283.03999999999996,162.51; KiCadOrientationDeg 90 -> 0
- R7310: BoardSide B.Cu -> F.Cu; FootprintOriginMm 305.91,94.64 -> 286.74,162.51; KiCadOrientationDeg 90 -> 0
- R7311: BoardSide B.Cu -> F.Cu; FootprintOriginMm 311.91,94.74 -> 262.81,107.04; KiCadOrientationDeg 90 -> 270
- R7312: BoardSide B.Cu -> F.Cu; FootprintOriginMm 312.31,98.44 -> 262.14,130.81; KiCadOrientationDeg 90 -> 0
- R7325: FootprintOriginMm 312.31,102.14 -> 254.14,141.31; KiCadOrientationDeg 90 -> 180
- R7326: FootprintOriginMm 312.31,105.84 -> 266.03999999999996,162.31; KiCadOrientationDeg 90 -> 180
- R7327: BoardSide B.Cu -> F.Cu; FootprintOriginMm 244.17000000000002,31.900000000000002 -> 244.77,111.6; KiCadOrientationDeg 180 -> 0
- R7328: FootprintOriginMm 256.27,31.900000000000002 -> 248.37,107.3
- R7329: FootprintOriginMm 305.91,107.84 -> 248.94,133.91; KiCadOrientationDeg 90 -> 180
- R7330: BoardSide B.Cu -> F.Cu; FootprintOriginMm 312.31,109.54 -> 246.10999999999999,107.94; KiCadOrientationDeg 90 -> 270
- R7331: FootprintOriginMm 312.31,113.24 -> 245.41,103.54
- R7332: BoardSide B.Cu -> F.Cu; FootprintOriginMm 198.01,116.34 -> 243.14,106.50999999999999; KiCadOrientationDeg 90 -> 0
- R7333: BoardSide B.Cu -> F.Cu; FootprintOriginMm 312.31,116.94 -> 255.54,162.51; KiCadOrientationDeg 90 -> 0
- R7334: FootprintOriginMm 312.31,120.64 -> 272.64,103.41; KiCadOrientationDeg 90 -> 180
- R7335: BoardSide B.Cu -> F.Cu; FootprintOriginMm 305.91,121.04 -> 258.51000000000005,151.73999999999998; KiCadOrientationDeg 90 -> 270
- U7302: FootprintOriginMm 257.92,128.38 -> 257.92,115.18
- U7303: FootprintOriginMm 274.92,128.38 -> 260.12,108.78
- U7306: FootprintOriginMm 260.46000000000004,64.02 -> 261.13,145.82; KiCadOrientationDeg 270 -> 90
- U7307: BoardSide F.Cu -> B.Cu; FootprintOriginMm 260.46500000000003,37.23 -> 274.72999999999996,129.35; KiCadOrientationDeg 270 -> 180
- U7308: FootprintOriginMm 277.46500000000003,37.23 -> 260.46500000000003,121.83
- U7309: FootprintOriginMm 225.97,66.35 -> 259.97,137.54999999999998

Commit message: Place jack-right with span-aware swaps and route it to 190 open edges
Rebuilt from the swap-pass placement; rails, negotiated routing (1236 -> 283),
re-offered rip-up, signal batches, AGND stitching and escapes. Reports come
from the adopted stage's native DRC (0 errors, 0 parity) and native ratsnest.

Co-Authored-By: Claude Opus 5.5 <noreply@anthropic.com>
Parts:
- D7301: BoardSide F.Cu -> B.Cu; FootprintOriginMm 259.53000000000003,106.91 -> 248.91,99.33000000000001; KiCadOrientationDeg 0 -> 90
- D7303: FootprintOriginMm 264.15000000000003,128.55 -> 264.95000000000005,104.15
- D7304: BoardSide F.Cu -> B.Cu; FootprintOriginMm 275.85,136.91000000000003 -> 269.65000000000003,100.85; KiCadOrientationDeg 270 -> 180
- D7305: BoardSide F.Cu -> B.Cu; FootprintOriginMm 275.85,131.51000000000002 -> 266.25,115.55; KiCadOrientationDeg 270 -> 90
- D7306: FootprintOriginMm 283.45000000000005,140.95 -> 269.15,113.44999999999999; KiCadOrientationDeg 180 -> 90
- D7309: FootprintOriginMm 249.35,115.55 -> 283.45000000000005,140.95; KiCadOrientationDeg 90 -> 180
- D7310: BoardSide B.Cu -> F.Cu; FootprintOriginMm 281.15000000000003,128.55 -> 275.85,136.91000000000003; KiCadOrientationDeg 180 -> 270
- D7311: FootprintOriginMm 266.25,115.55 -> 266.45000000000005,140.95; KiCadOrientationDeg 90 -> 180
- D7314: FootprintOriginMm 269.15,113.44999999999999 -> 264.15000000000003,128.55; KiCadOrientationDeg 90 -> 180
- D7315: BoardSide B.Cu -> F.Cu; FootprintOriginMm 247.95,110.55 -> 258.85,131.51000000000002; KiCadOrientationDeg 180 -> 270
- D7316: BoardSide B.Cu -> F.Cu; FootprintOriginMm 242.54999999999998,110.55 -> 261.75,136.91000000000003; KiCadOrientationDeg 180 -> 270
- R7305: FootprintOriginMm 269.74,162.51 -> 283.03999999999996,162.51
- R7306: FootprintOriginMm 272.64,117.31 -> 283.03999999999996,162.31
- R7307: FootprintOriginMm 255.64,104.50999999999999 -> 244.81,99.04; KiCadOrientationDeg 180 -> 90
- R7308: BoardSide F.Cu -> B.Cu; FootprintOriginMm 262.14,133.01 -> 245.41,103.54; KiCadOrientationDeg 0 -> 90
- R7309: FootprintOriginMm 283.03999999999996,162.51 -> 262.81,107.04; KiCadOrientationDeg 0 -> 270
- R7310: BoardSide F.Cu -> B.Cu; FootprintOriginMm 286.74,162.51 -> 272.64,117.31; KiCadOrientationDeg 0 -> 180
- R7311: BoardSide F.Cu -> B.Cu; FootprintOriginMm 262.81,107.04 -> 244.81,107.24; KiCadOrientationDeg 270 -> 90
- R7312: FootprintOriginMm 262.14,130.81 -> 246.10999999999999,107.94; KiCadOrientationDeg 0 -> 270
- R7325: BoardSide B.Cu -> F.Cu; FootprintOriginMm 254.14,141.31 -> 244.44,98.21; KiCadOrientationDeg 180 -> 0
- R7326: BoardSide B.Cu -> F.Cu; FootprintOriginMm 266.03999999999996,162.31 -> 258.51000000000005,151.73999999999998; KiCadOrientationDeg 180 -> 270
- R7329: BoardSide B.Cu -> F.Cu; FootprintOriginMm 248.94,133.91 -> 255.54,162.51; KiCadOrientationDeg 180 -> 0
- R7330: BoardSide F.Cu -> B.Cu; FootprintOriginMm 246.10999999999999,107.94 -> 265.94,133.91; KiCadOrientationDeg 270 -> 180
- R7331: FootprintOriginMm 245.41,103.54 -> 288.14,141.31; KiCadOrientationDeg 90 -> 180
- R7332: FootprintOriginMm 243.14,106.50999999999999 -> 262.14,130.81
- R7333: BoardSide F.Cu -> B.Cu; FootprintOriginMm 255.54,162.51 -> 266.03999999999996,162.31; KiCadOrientationDeg 0 -> 180
- R7334: BoardSide B.Cu -> F.Cu; FootprintOriginMm 272.64,103.41 -> 269.74,162.51; KiCadOrientationDeg 180 -> 0
- R7335: FootprintOriginMm 258.51000000000005,151.73999999999998 -> 266.03999999999996,162.51; KiCadOrientationDeg 270 -> 0

Commit message: Regenerate and rebuild both jack halves with the hot-quad escape reservation
Evidence rebound (peripheral epoch, foil-collar proposal, control receipt);
jack boards rebuilt from the new placement with source planes and no signal
copper, ready for CI routing.

Co-Authored-By: Claude Opus 5.5 <noreply@anthropic.com>
Parts:
- C7308: BoardSide B.Cu -> F.Cu; FootprintOriginMm 252.76000000000002,114.155 -> 261.105,127.50999999999999; KiCadOrientationDeg 90 -> 270
- C7309: BoardSide B.Cu -> F.Cu; FootprintOriginMm 263.67,114.155 -> 261.105,115.23999999999998
- C7310: FootprintOriginMm 254.96,107.755 -> 252.76000000000002,114.155
- C7311: FootprintOriginMm 265.87,107.755 -> 263.67,114.155
- C7312: FootprintOriginMm 269.03999999999996,127.445 -> 252.04000000000002,127.445
- C7313: FootprintOriginMm 280.41999999999996,131.255 -> 263.42,131.255
- C7314: BoardSide F.Cu -> B.Cu; FootprintOriginMm 262.37,127.52 -> 269.03999999999996,127.445; KiCadOrientationDeg 270 -> 180
- C7315: BoardSide F.Cu -> B.Cu; FootprintOriginMm 258.56000000000006,116.14 -> 280.41999999999996,131.255; KiCadOrientationDeg 90 -> 0
- D7301: FootprintOriginMm 248.91,99.33000000000001 -> 244.33,103.51; KiCadOrientationDeg 90 -> 180
- D7302: FootprintOriginMm 248.63,103.51 -> 248.63,104.21000000000001
- D7303: FootprintOriginMm 264.95000000000005,104.15 -> 264.15000000000003,128.55
- D7304: FootprintOriginMm 269.65000000000003,100.85 -> 281.55,116.95
- D7305: BoardSide B.Cu -> F.Cu; FootprintOriginMm 266.25,115.55 -> 261.75,136.91000000000003; KiCadOrientationDeg 90 -> 270
- D7306: FootprintOriginMm 269.15,113.44999999999999 -> 283.75,114.05; KiCadOrientationDeg 90 -> 180
- D7308: BoardSide F.Cu -> B.Cu; FootprintOriginMm 278.75,136.91000000000003 -> 264.95000000000005,104.15; KiCadOrientationDeg 270 -> 180
- D7309: FootprintOriginMm 283.45000000000005,140.95 -> 269.65000000000003,100.85
- D7310: FootprintOriginMm 275.85,136.91000000000003 -> 260.21000000000004,111.95; KiCadOrientationDeg 270 -> 0
- D7311: FootprintOriginMm 266.45000000000005,140.95 -> 266.25,115.55; KiCadOrientationDeg 180 -> 90
- D7313: FootprintOriginMm 261.15,115.31 -> 275.85,144.51000000000002
- D7314: BoardSide B.Cu -> F.Cu; FootprintOriginMm 264.15000000000003,128.55 -> 278.75,146.21; KiCadOrientationDeg 180 -> 270
- D7315: BoardSide F.Cu -> B.Cu; FootprintOriginMm 258.85,131.51000000000002 -> 266.45000000000005,140.95; KiCadOrientationDeg 270 -> 180
- D7316: FootprintOriginMm 261.75,136.91000000000003 -> 275.85,149.91000000000003
- R7307: BoardSide B.Cu -> F.Cu; FootprintOriginMm 244.81,99.04 -> 245.81,107.94; KiCadOrientationDeg 90 -> 270
- R7308: BoardSide B.Cu -> F.Cu; FootprintOriginMm 245.41,103.54 -> 245.33999999999997,104.71; KiCadOrientationDeg 90 -> 0
- R7309: BoardSide F.Cu -> B.Cu; FootprintOriginMm 262.81,107.04 -> 249.04,101.11; KiCadOrientationDeg 270 -> 180
- R7310: FootprintOriginMm 272.64,117.31 -> 249.04,98.91
- R7311: BoardSide B.Cu -> F.Cu; FootprintOriginMm 244.81,107.24 -> 249.04,162.51; KiCadOrientationDeg 90 -> 0
- R7312: FootprintOriginMm 246.10999999999999,107.94 -> 255.54,162.51; KiCadOrientationDeg 270 -> 0
- R7325: FootprintOriginMm 244.44,98.21 -> 246.10999999999999,98.04; KiCadOrientationDeg 0 -> 270
- R7326: BoardSide F.Cu -> B.Cu; FootprintOriginMm 258.51000000000005,151.73999999999998 -> 254.14,141.31; KiCadOrientationDeg 270 -> 180
- R7327: BoardSide F.Cu -> B.Cu; FootprintOriginMm 244.77,111.6 -> 242.97,107.3; KiCadOrientationDeg 0 -> 180
- R7328: BoardSide B.Cu -> F.Cu; FootprintOriginMm 248.37,107.3 -> 244.77,111.6; KiCadOrientationDeg 180 -> 0
- R7329: FootprintOriginMm 255.54,162.51 -> 258.51000000000005,151.73999999999998; KiCadOrientationDeg 0 -> 270
- R7330: FootprintOriginMm 265.94,133.91 -> 282.94,133.91
- R7331: FootprintOriginMm 288.14,141.31 -> 265.94,133.91
- R7332: FootprintOriginMm 262.14,130.81 -> 268.84,162.51
- R7334: BoardSide F.Cu -> B.Cu; FootprintOriginMm 269.74,162.51 -> 269.74,162.31; KiCadOrientationDeg 0 -> 180
- R7335: BoardSide F.Cu -> B.Cu; FootprintOriginMm 266.03999999999996,162.51 -> 255.54,162.31; KiCadOrientationDeg 0 -> 180
- U7302: BoardSide B.Cu -> F.Cu; FootprintOriginMm 257.92,115.18 -> 260.78000000000003,121.66999999999999; KiCadOrientationDeg 180 -> 270
- U7303: FootprintOriginMm 260.12,108.78 -> 257.92,115.18
- U7307: FootprintOriginMm 274.72999999999996,129.35 -> 257.73,129.35
- U7308: BoardSide F.Cu -> B.Cu; FootprintOriginMm 260.46500000000003,121.83 -> 274.72999999999996,129.35; KiCadOrientationDeg 270 -> 180
