File: boards/osc-jack-right/sheets/envelope_E1_JR.kicad_sch (KiCad schematic)
At the start: 66 parts, among them J1301 WQP518MA, J1302 WQP518MA, J1303 WQP518MA, J1304 WQP518MA, J1305 WQP518MA, J1306 WQP518MA, J1307 WQP518MA, U4102 ADG5412FBRUZ, U4103 ADG5412FBRUZ, U4104 ADG5412FBRUZ, U4146 OPA4196IDR, U4147 OPA4196IDR, U4148 OPA4196IDR

Commit message: Move jack halves to six layers with locality placement and grid routing
Owner decision 2026-10-03 (#38): a cut-line bound showed the four-layer
jack halves could not carry their signal nets with intact planes, so both
halves move to six layers and their free packages are re-placed for
locality.

- Placement: scripts/checks/jack_locality.py replaces the
  connectivity-blind first-fit J placer. Packages are pulled toward the
  fixed jacks, LEDs and headers on their nets and toward their own
  module's hardware, then legalized; IC/bypass clusters stay aligned.
  Panel hardware and headers do not move.
- Stack: F/In2/In3/B signals, In1 AGND plane, -12V fill on In3, +12V
  plane on In4; +5V as tracks.
- Routing: scripts/pcbgen/route_jack_grid.py stages terminal arrays,
  rail fanouts and links, signal batches, rip-up-and-reroute and AGND
  stitching, keeping only natively checked stages (0 DRC errors,
  0 parity). The grid router gains N-layer support, windowed search,
  plane fanout, a plane-fill split guard and rip-up-and-reroute.
- Evidence chain: a bounded jack-locality partition transition is
  chained onto the connector-locality proof; superseded four-layer
  stage reports are removed.

Checkpoint: JL 411 and JR 518 native open edges remain. This is a routed
draft in progress; electrical and physical qualification NOT RUN.

Co-Authored-By: Claude Opus 5.5 <noreply@anthropic.com>
Parts:
- C4115: FootprintOriginMm 186.96,95.355 -> 218.04,71.555; KiCadOrientationDeg 90 -> 180
- C4116: FootprintOriginMm 197.87,95.355 -> 230.31,71.555; KiCadOrientationDeg 90 -> 0
- C4117: BoardSide B.Cu -> F.Cu; FootprintOriginMm 203.96,95.355 -> 226.95499999999998,58.86; KiCadOrientationDeg 90 -> 0
- C4118: BoardSide B.Cu -> F.Cu; FootprintOriginMm 214.87,95.355 -> 226.95499999999998,69.77; KiCadOrientationDeg 90 -> 0
- C4119: FootprintOriginMm 220.96,95.355 -> 215.67000000000002,48.504999999999995; KiCadOrientationDeg 90 -> 270
- C4120: FootprintOriginMm 231.87,95.355 -> 204.76000000000002,48.504999999999995; KiCadOrientationDeg 90 -> 270
- C4172: FootprintOriginMm 196.98,24.55 -> 230.98,50.85
- C4173: FootprintOriginMm 186.96,24.55 -> 220.96,50.85
- C4174: FootprintOriginMm 213.98,24.55 -> 225.38,67.58; KiCadOrientationDeg 90 -> 0
- C4175: FootprintOriginMm 203.96,24.55 -> 225.38,57.56; KiCadOrientationDeg 90 -> 0
- C4176: FootprintOriginMm 230.98,24.55 -> 220.96,88.78000000000002; KiCadOrientationDeg 90 -> 270
- C4177: FootprintOriginMm 220.96,24.55 -> 230.98,88.78000000000002; KiCadOrientationDeg 90 -> 270
- D4101: FootprintOriginMm 306.93,22.11 -> 221.93,25.91
- D4102: FootprintOriginMm 200.23000000000002,43.21 -> 226.23000000000002,25.91
- D4103: BoardSide B.Cu -> F.Cu; FootprintOriginMm 217.23000000000002,43.21 -> 228.03,30.31; KiCadOrientationDeg 180 -> 0
- D4107: FootprintOriginMm 298.95000000000005,139.45 -> 215.35,62.550000000000004; KiCadOrientationDeg 180 -> 90
- D4108: FootprintOriginMm 304.35,140.35 -> 216.95,58.55
- D4109: FootprintOriginMm 183.65,43.45 -> 214.75,67.94999999999999
- D4110: FootprintOriginMm 197.35,50.050000000000004 -> 231.25,62.550000000000004
- D4112: FootprintOriginMm 214.35,50.050000000000004 -> 213.35,72.25; KiCadOrientationDeg 90 -> 180
- D4113: FootprintOriginMm 231.35,50.050000000000004 -> 231.35,57.15
- D4114: FootprintOriginMm 248.35,50.050000000000004 -> 234.25,57.45
- D4115: FootprintOriginMm 265.35,50.050000000000004 -> 207.95,74.45; KiCadOrientationDeg 90 -> 180
- D4117: FootprintOriginMm 282.35,50.050000000000004 -> 220.35,44.85; KiCadOrientationDeg 90 -> 180
- D4118: FootprintOriginMm 299.35,50.050000000000004 -> 225.75,44.95; KiCadOrientationDeg 90 -> 180
- D4119: FootprintOriginMm 183.65,57.45 -> 202.15,58.85; KiCadOrientationDeg 90 -> 180
- D4120: FootprintOriginMm 183.65,85.44999999999999 -> 231.35,46.15
- R4105: FootprintOriginMm 299.74,21.21 -> 216.71,44.44; KiCadOrientationDeg 180 -> 90
- R4106: FootprintOriginMm 202.64,28.01 -> 220.33999999999997,42.309999999999995
- R4107: FootprintOriginMm 219.64,28.01 -> 220.14,84.31
- R4108: FootprintOriginMm 236.64,28.01 -> 221.64,67.61
- R4109: FootprintOriginMm 253.64,28.01 -> 224.04,42.309999999999995
- R4110: FootprintOriginMm 270.64,28.01 -> 227.73999999999998,42.41
- R4111: FootprintOriginMm 287.64,28.01 -> 231.44,42.51
- R4112: FootprintOriginMm 214.44,31.61 -> 221.64,57.51
- R4113: FootprintOriginMm 231.44,31.61 -> 231.73999999999998,84.31
- R4114: FootprintOriginMm 248.44,31.61 -> 217.94,87.21
- R4115: FootprintOriginMm 265.44,31.61 -> 235.14,42.309999999999995
- R4116: FootprintOriginMm 282.44,31.61 -> 217.94,56.01
- RB4105: FootprintOriginMm 249.37,70.69999999999999 -> 229.47,29.700000000000003
- RB4106: FootprintOriginMm 266.37,70.69999999999999 -> 230.97,74.5
- RB4107: FootprintOriginMm 283.37,70.69999999999999 -> 234.37,30.5
- RB4108: FootprintOriginMm 300.37,70.69999999999999 -> 247.97,68.3
- RB4109: FootprintOriginMm 189.57000000000002,73.0 -> 239.27,32.6
- RB4110: FootprintOriginMm 205.27,73.0 -> 247.97,74.5
- RB4111: FootprintOriginMm 210.17000000000002,73.0 -> 239.27,95.0
- RB4112: BoardSide B.Cu -> F.Cu; FootprintOriginMm 222.27,73.0 -> 225.87,34.1; KiCadOrientationDeg 180 -> 0
- RB4113: FootprintOriginMm 242.23999999999998,150.81 -> 242.23999999999998,33.41
- RB4114: FootprintOriginMm 259.24,150.81 -> 242.23999999999998,31.21
- RB4115: FootprintOriginMm 276.24,150.81 -> 245.21,32.64; KiCadOrientationDeg 0 -> 270
- U4102: FootprintOriginMm 192.12,96.38000000000001 -> 223.88,71.88000000000001
- U4103: BoardSide B.Cu -> F.Cu; FootprintOriginMm 209.12,96.38000000000001 -> 226.57999999999998,64.02; KiCadOrientationDeg 180 -> 90
- U4104: FootprintOriginMm 226.12,96.38000000000001 -> 210.51000000000002,47.48; KiCadOrientationDeg 180 -> 0
- U4146: FootprintOriginMm 191.97,25.25 -> 225.97,51.550000000000004
- U4147: FootprintOriginMm 208.97,25.25 -> 224.68,62.57; KiCadOrientationDeg 180 -> 90
- U4148: FootprintOriginMm 225.97,25.25 -> 225.97,88.08000000000001; KiCadOrientationDeg 180 -> 0

Commit message: Place jack-right with span-aware swaps and route it to 190 open edges
Rebuilt from the swap-pass placement; rails, negotiated routing (1236 -> 283),
re-offered rip-up, signal batches, AGND stitching and escapes. Reports come
from the adopted stage's native DRC (0 errors, 0 parity) and native ratsnest.

Co-Authored-By: Claude Opus 5.5 <noreply@anthropic.com>
Parts:
- D4107: BoardSide B.Cu -> F.Cu; FootprintOriginMm 215.35,62.550000000000004 -> 226.21,37.35; KiCadOrientationDeg 90 -> 0
- D4108: FootprintOriginMm 216.95,58.55 -> 227.75,32.95
- D4109: BoardSide B.Cu -> F.Cu; FootprintOriginMm 214.75,67.94999999999999 -> 226.21,40.25; KiCadOrientationDeg 90 -> 0
- D4110: FootprintOriginMm 231.25,62.550000000000004 -> 222.35,32.95; KiCadOrientationDeg 90 -> 180
- D4112: FootprintOriginMm 213.35,72.25 -> 227.75,94.65
- D4113: FootprintOriginMm 231.35,57.15 -> 232.05,93.14999999999999
- D4114: FootprintOriginMm 234.25,57.45 -> 227.75,97.55; KiCadOrientationDeg 90 -> 180
- D4115: FootprintOriginMm 207.95,74.45 -> 227.65,100.45
- D4117: FootprintOriginMm 220.35,44.85 -> 231.35,57.15; KiCadOrientationDeg 180 -> 90
- D4118: FootprintOriginMm 225.75,44.95 -> 234.25,57.45; KiCadOrientationDeg 180 -> 90
- D4119: FootprintOriginMm 202.15,58.85 -> 231.25,62.550000000000004; KiCadOrientationDeg 180 -> 90
- D4120: FootprintOriginMm 231.35,46.15 -> 216.95,58.55; KiCadOrientationDeg 90 -> 180
- R4105: FootprintOriginMm 216.71,44.44 -> 237.91,54.54
- R4106: FootprintOriginMm 220.33999999999997,42.309999999999995 -> 235.14,42.309999999999995
- R4107: FootprintOriginMm 220.14,84.31 -> 238.64,67.61
- R4109: FootprintOriginMm 224.04,42.309999999999995 -> 231.44,42.51
- R4111: BoardSide B.Cu -> F.Cu; FootprintOriginMm 231.44,42.51 -> 225.23999999999998,24.41; KiCadOrientationDeg 180 -> 0
- R4112: BoardSide B.Cu -> F.Cu; FootprintOriginMm 221.64,57.51 -> 225.23999999999998,26.61; KiCadOrientationDeg 180 -> 0
- R4113: FootprintOriginMm 231.73999999999998,84.31 -> 216.71,44.44; KiCadOrientationDeg 180 -> 90
- R4114: FootprintOriginMm 217.94,87.21 -> 220.33999999999997,42.309999999999995
- R4115: FootprintOriginMm 235.14,42.309999999999995 -> 229.51,26.04; KiCadOrientationDeg 180 -> 90
- R4116: BoardSide B.Cu -> F.Cu; FootprintOriginMm 217.94,56.01 -> 228.21,26.44; KiCadOrientationDeg 180 -> 270
- RB4106: FootprintOriginMm 230.97,74.5 -> 234.37,30.5
- RB4107: FootprintOriginMm 234.37,30.5 -> 264.96999999999997,68.3
- RB4109: FootprintOriginMm 239.27,32.6 -> 224.57000000000002,29.700000000000003
- RB4110: BoardSide B.Cu -> F.Cu; FootprintOriginMm 247.97,74.5 -> 225.87,34.1; KiCadOrientationDeg 180 -> 0
- RB4111: BoardSide B.Cu -> F.Cu; FootprintOriginMm 239.27,95.0 -> 242.87,39.9; KiCadOrientationDeg 180 -> 0
- RB4112: FootprintOriginMm 225.87,34.1 -> 242.87,84.3
- RB4113: BoardSide F.Cu -> B.Cu; FootprintOriginMm 242.23999999999998,33.41 -> 224.04,42.309999999999995; KiCadOrientationDeg 0 -> 180
- RB4114: BoardSide F.Cu -> B.Cu; FootprintOriginMm 242.23999999999998,31.21 -> 236.01,98.74; KiCadOrientationDeg 0 -> 90
- RB4115: BoardSide F.Cu -> B.Cu; FootprintOriginMm 245.21,32.64 -> 237.54,57.51; KiCadOrientationDeg 270 -> 180

Commit message: Regenerate and rebuild both jack halves with the hot-quad escape reservation
Evidence rebound (peripheral epoch, foil-collar proposal, control receipt);
jack boards rebuilt from the new placement with source planes and no signal
copper, ready for CI routing.

Co-Authored-By: Claude Opus 5.5 <noreply@anthropic.com>
Parts:
- D4102: BoardSide B.Cu -> F.Cu; FootprintOriginMm 226.23000000000002,25.91 -> 228.03,30.31; KiCadOrientationDeg 180 -> 0
- D4103: BoardSide F.Cu -> B.Cu; FootprintOriginMm 228.03,30.31 -> 226.23000000000002,25.91; KiCadOrientationDeg 0 -> 180
- D4107: BoardSide F.Cu -> B.Cu; FootprintOriginMm 226.21,37.35 -> 231.35,57.15; KiCadOrientationDeg 0 -> 90
- D4108: FootprintOriginMm 227.75,32.95 -> 234.25,57.45; KiCadOrientationDeg 180 -> 90
- D4109: BoardSide F.Cu -> B.Cu; FootprintOriginMm 226.21,40.25 -> 227.75,32.95; KiCadOrientationDeg 0 -> 180
- D4112: FootprintOriginMm 227.75,94.65 -> 225.75,44.95
- D4113: FootprintOriginMm 232.05,93.14999999999999 -> 231.35,46.15
- D4114: BoardSide B.Cu -> F.Cu; FootprintOriginMm 227.75,97.55 -> 226.21,40.25; KiCadOrientationDeg 180 -> 0
- D4115: BoardSide B.Cu -> F.Cu; FootprintOriginMm 227.65,100.45 -> 226.21,37.35; KiCadOrientationDeg 180 -> 0
- D4117: FootprintOriginMm 231.35,57.15 -> 227.75,97.55; KiCadOrientationDeg 90 -> 180
- D4118: FootprintOriginMm 234.25,57.45 -> 231.25,62.550000000000004
- D4119: FootprintOriginMm 231.25,62.550000000000004 -> 227.75,94.65; KiCadOrientationDeg 90 -> 180
- D4120: FootprintOriginMm 216.95,58.55 -> 232.05,93.14999999999999; KiCadOrientationDeg 180 -> 90
- R4105: FootprintOriginMm 237.91,54.54 -> 227.73999999999998,42.41; KiCadOrientationDeg 90 -> 180
- R4106: FootprintOriginMm 235.14,42.309999999999995 -> 224.04,42.309999999999995
- R4107: FootprintOriginMm 238.64,67.61 -> 227.44,22.81
- R4108: BoardSide B.Cu -> F.Cu; FootprintOriginMm 221.64,67.61 -> 225.23999999999998,24.41; KiCadOrientationDeg 180 -> 0
- R4109: BoardSide B.Cu -> F.Cu; FootprintOriginMm 231.44,42.51 -> 242.23999999999998,26.61; KiCadOrientationDeg 180 -> 0
- R4110: BoardSide B.Cu -> F.Cu; FootprintOriginMm 227.73999999999998,42.41 -> 245.21,26.04; KiCadOrientationDeg 180 -> 270
- R4111: BoardSide F.Cu -> B.Cu; FootprintOriginMm 225.23999999999998,24.41 -> 238.83999999999997,42.309999999999995; KiCadOrientationDeg 0 -> 180
- R4112: BoardSide F.Cu -> B.Cu; FootprintOriginMm 225.23999999999998,26.61 -> 231.44,42.51; KiCadOrientationDeg 0 -> 180
- R4113: FootprintOriginMm 216.71,44.44 -> 240.83999999999997,21.31; KiCadOrientationDeg 90 -> 180
- R4114: FootprintOriginMm 220.33999999999997,42.309999999999995 -> 240.83999999999997,23.51
- R4115: BoardSide B.Cu -> F.Cu; FootprintOriginMm 229.51,26.04 -> 228.21,22.740000000000002; KiCadOrientationDeg 90 -> 270
- RB4105: FootprintOriginMm 229.47,29.700000000000003 -> 239.27,32.6
- RB4111: BoardSide F.Cu -> B.Cu; FootprintOriginMm 242.87,39.9 -> 231.6,67.86999999999999; KiCadOrientationDeg 0 -> 90
- RB4113: BoardSide B.Cu -> F.Cu; FootprintOriginMm 224.04,42.309999999999995 -> 245.21,32.64; KiCadOrientationDeg 180 -> 270
- RB4114: FootprintOriginMm 236.01,98.74 -> 235.14,42.309999999999995; KiCadOrientationDeg 90 -> 180
- RB4115: FootprintOriginMm 237.54,57.51 -> 238.64,67.61
