File: boards/osc-jack-right/sheets/envelope_E2_JR.kicad_sch (KiCad schematic)
At the start: 66 parts, among them J1401 WQP518MA, J1402 WQP518MA, J1403 WQP518MA, J1404 WQP518MA, J1405 WQP518MA, J1406 WQP518MA, J1407 WQP518MA, U4202 ADG5412FBRUZ, U4203 ADG5412FBRUZ, U4204 ADG5412FBRUZ, U4246 OPA4196IDR, U4247 OPA4196IDR, U4248 OPA4196IDR

Commit message: Move jack halves to six layers with locality placement and grid routing
Owner decision 2026-10-03 (#38): a cut-line bound showed the four-layer
jack halves could not carry their signal nets with intact planes, so both
halves move to six layers and their free packages are re-placed for
locality.

- Placement: scripts/checks/jack_locality.py replaces the
  connectivity-blind first-fit J placer. Packages are pulled toward the
  fixed jacks, LEDs and headers on their nets and toward their own
  module's hardware, then legalized; IC/bypass clusters stay aligned.
  Panel hardware and headers do not move.
- Stack: F/In2/In3/B signals, In1 AGND plane, -12V fill on In3, +12V
  plane on In4; +5V as tracks.
- Routing: scripts/pcbgen/route_jack_grid.py stages terminal arrays,
  rail fanouts and links, signal batches, rip-up-and-reroute and AGND
  stitching, keeping only natively checked stages (0 DRC errors,
  0 parity). The grid router gains N-layer support, windowed search,
  plane fanout, a plane-fill split guard and rip-up-and-reroute.
- Evidence chain: a bounded jack-locality partition transition is
  chained onto the connector-locality proof; superseded four-layer
  stage reports are removed.

Checkpoint: JL 411 and JR 518 native open edges remain. This is a routed
draft in progress; electrical and physical qualification NOT RUN.

Co-Authored-By: Claude Opus 5.5 <noreply@anthropic.com>
Parts:
- C4215: FootprintOriginMm 237.96,95.355 -> 235.04,71.555; KiCadOrientationDeg 90 -> 180
- C4216: FootprintOriginMm 248.87,95.355 -> 247.31,71.555; KiCadOrientationDeg 90 -> 0
- C4217: BoardSide B.Cu -> F.Cu; FootprintOriginMm 254.96,95.355 -> 243.95499999999998,58.86; KiCadOrientationDeg 90 -> 0
- C4218: BoardSide B.Cu -> F.Cu; FootprintOriginMm 265.87,95.355 -> 243.95499999999998,69.77; KiCadOrientationDeg 90 -> 0
- C4219: BoardSide B.Cu -> F.Cu; FootprintOriginMm 271.96,95.355 -> 244.105,55.91; KiCadOrientationDeg 90 -> 270
- C4220: BoardSide B.Cu -> F.Cu; FootprintOriginMm 282.87,95.355 -> 244.105,43.64
- C4272: FootprintOriginMm 247.98,24.55 -> 247.98,50.85
- C4273: FootprintOriginMm 237.96,24.55 -> 237.96,50.85
- C4274: FootprintOriginMm 264.98,24.55 -> 242.38,67.58; KiCadOrientationDeg 90 -> 0
- C4275: FootprintOriginMm 254.96000000000004,24.55 -> 242.38,57.56; KiCadOrientationDeg 90 -> 0
- C4276: FootprintOriginMm 281.98,24.55 -> 237.96,88.78000000000002; KiCadOrientationDeg 90 -> 270
- C4277: FootprintOriginMm 271.96000000000004,24.55 -> 247.98,88.78000000000002; KiCadOrientationDeg 90 -> 270
- D4201: FootprintOriginMm 234.23000000000002,43.21 -> 238.93,28.81
- D4202: FootprintOriginMm 251.23000000000002,43.21 -> 243.83,95.21000000000001
- D4203: FootprintOriginMm 268.23,43.21 -> 243.23000000000002,28.81
- D4207: FootprintOriginMm 183.65,99.44999999999999 -> 248.25,62.550000000000004
- D4208: FootprintOriginMm 200.45,99.44999999999999 -> 248.35,57.15
- D4209: FootprintOriginMm 217.45,99.44999999999999 -> 251.25,57.45
- D4210: BoardSide B.Cu -> F.Cu; FootprintOriginMm 234.45,99.44999999999999 -> 243.21,72.35; KiCadOrientationDeg 90 -> 0
- D4212: FootprintOriginMm 251.45,99.44999999999999 -> 237.35,44.85; KiCadOrientationDeg 90 -> 180
- D4213: BoardSide B.Cu -> F.Cu; FootprintOriginMm 268.45,99.44999999999999 -> 243.21,75.25; KiCadOrientationDeg 90 -> 0
- D4214: FootprintOriginMm 285.45,99.44999999999999 -> 242.75,44.95; KiCadOrientationDeg 90 -> 180
- D4215: FootprintOriginMm 302.45,99.44999999999999 -> 248.35,46.15
- D4217: BoardSide B.Cu -> F.Cu; FootprintOriginMm 198.25,127.75 -> 243.21,78.15; KiCadOrientationDeg 90 -> 0
- D4218: FootprintOriginMm 215.25,127.75 -> 236.15,84.65; KiCadOrientationDeg 90 -> 180
- D4219: FootprintOriginMm 232.25,127.75 -> 252.35,44.85; KiCadOrientationDeg 90 -> 180
- D4220: BoardSide B.Cu -> F.Cu; FootprintOriginMm 249.25,127.75 -> 243.21,81.05; KiCadOrientationDeg 90 -> 0
- R4205: FootprintOriginMm 299.44,31.61 -> 238.83999999999997,42.309999999999995
- R4206: FootprintOriginMm 197.73999999999998,60.01 -> 242.54,42.41
- R4207: FootprintOriginMm 214.73999999999998,60.01 -> 246.23999999999998,42.41
- R4208: FootprintOriginMm 231.73999999999998,60.01 -> 237.54,57.51
- R4209: FootprintOriginMm 248.73999999999998,60.01 -> 249.94,42.309999999999995
- R4210: FootprintOriginMm 265.74,60.01 -> 248.73999999999998,84.31
- R4211: FootprintOriginMm 282.74,60.01 -> 234.94,87.21
- R4212: FootprintOriginMm 299.74,60.01 -> 238.64,67.61
- R4213: FootprintOriginMm 197.73999999999998,62.209999999999994 -> 253.64,42.309999999999995
- R4214: FootprintOriginMm 214.73999999999998,62.209999999999994 -> 257.34,42.41
- R4215: FootprintOriginMm 231.73999999999998,62.209999999999994 -> 261.71000000000004,44.54; KiCadOrientationDeg 180 -> 90
- R4216: FootprintOriginMm 248.73999999999998,62.209999999999994 -> 237.91,54.54; KiCadOrientationDeg 180 -> 90
- RB4205: FootprintOriginMm 227.17000000000002,73.0 -> 244.17000000000002,32.6
- RB4206: BoardSide B.Cu -> F.Cu; FootprintOriginMm 239.27,73.0 -> 242.87,84.3; KiCadOrientationDeg 180 -> 0
- RB4207: BoardSide B.Cu -> F.Cu; FootprintOriginMm 244.17000000000002,73.0 -> 242.87,36.300000000000004; KiCadOrientationDeg 180 -> 0
- RB4208: BoardSide B.Cu -> F.Cu; FootprintOriginMm 256.27,73.0 -> 242.87,39.9; KiCadOrientationDeg 180 -> 0
- RB4209: FootprintOriginMm 261.16999999999996,73.0 -> 248.7,93.07; KiCadOrientationDeg 180 -> 90
- RB4210: FootprintOriginMm 273.27,73.0 -> 264.96999999999997,68.3
- RB4211: FootprintOriginMm 278.16999999999996,73.0 -> 248.4,31.97; KiCadOrientationDeg 180 -> 90
- RB4212: BoardSide B.Cu -> F.Cu; FootprintOriginMm 290.27,73.0 -> 242.87,87.89999999999999; KiCadOrientationDeg 180 -> 0
- RB4213: BoardSide F.Cu -> B.Cu; FootprintOriginMm 293.24,150.81 -> 247.23999999999998,28.41; KiCadOrientationDeg 0 -> 180
- RB4214: BoardSide F.Cu -> B.Cu; FootprintOriginMm 208.23999999999998,151.10999999999999 -> 242.33999999999997,25.71; KiCadOrientationDeg 0 -> 180
- RB4215: FootprintOriginMm 310.24,151.60999999999999 -> 244.44,98.21
- U4202: FootprintOriginMm 243.12,96.38000000000001 -> 240.88,71.88000000000001
- U4203: BoardSide B.Cu -> F.Cu; FootprintOriginMm 260.12,96.38000000000001 -> 243.57999999999998,64.02; KiCadOrientationDeg 180 -> 90
- U4204: BoardSide B.Cu -> F.Cu; FootprintOriginMm 277.12,96.38000000000001 -> 243.78,50.07; KiCadOrientationDeg 180 -> 270
- U4246: FootprintOriginMm 242.97,25.25 -> 242.97,51.550000000000004
- U4247: FootprintOriginMm 259.97,25.25 -> 241.68,62.57; KiCadOrientationDeg 180 -> 90
- U4248: FootprintOriginMm 276.97,25.25 -> 242.97,88.08000000000001; KiCadOrientationDeg 180 -> 0

Commit message: Place jack-right with span-aware swaps and route it to 190 open edges
Rebuilt from the swap-pass placement; rails, negotiated routing (1236 -> 283),
re-offered rip-up, signal batches, AGND stitching and escapes. Reports come
from the adopted stage's native DRC (0 errors, 0 parity) and native ratsnest.

Co-Authored-By: Claude Opus 5.5 <noreply@anthropic.com>
Parts:
- D4210: BoardSide F.Cu -> B.Cu; FootprintOriginMm 243.21,72.35 -> 252.35,44.85; KiCadOrientationDeg 0 -> 180
- D4212: BoardSide B.Cu -> F.Cu; FootprintOriginMm 237.35,44.85 -> 243.21,72.35; KiCadOrientationDeg 180 -> 0
- D4213: BoardSide F.Cu -> B.Cu; FootprintOriginMm 243.21,75.25 -> 248.35,46.15; KiCadOrientationDeg 0 -> 90
- D4215: FootprintOriginMm 248.35,46.15 -> 237.35,44.85; KiCadOrientationDeg 90 -> 180
- D4218: BoardSide B.Cu -> F.Cu; FootprintOriginMm 236.15,84.65 -> 243.21,75.25; KiCadOrientationDeg 180 -> 0
- D4219: BoardSide B.Cu -> F.Cu; FootprintOriginMm 252.35,44.85 -> 243.21,81.05; KiCadOrientationDeg 180 -> 0
- D4220: BoardSide F.Cu -> B.Cu; FootprintOriginMm 243.21,81.05 -> 236.15,84.65; KiCadOrientationDeg 0 -> 180
- R4207: BoardSide B.Cu -> F.Cu; FootprintOriginMm 246.23999999999998,42.41 -> 242.23999999999998,31.21; KiCadOrientationDeg 180 -> 0
- R4208: BoardSide B.Cu -> F.Cu; FootprintOriginMm 237.54,57.51 -> 242.23999999999998,33.41; KiCadOrientationDeg 180 -> 0
- R4209: FootprintOriginMm 249.94,42.309999999999995 -> 247.23999999999998,28.41
- R4210: BoardSide B.Cu -> F.Cu; FootprintOriginMm 248.73999999999998,84.31 -> 245.21,32.64; KiCadOrientationDeg 180 -> 270
- R4211: BoardSide B.Cu -> F.Cu; FootprintOriginMm 234.94,87.21 -> 245.91,91.54; KiCadOrientationDeg 180 -> 270
- R4212: BoardSide B.Cu -> F.Cu; FootprintOriginMm 238.64,67.61 -> 243.71,91.54; KiCadOrientationDeg 180 -> 270
- R4215: FootprintOriginMm 261.71000000000004,44.54 -> 249.94,42.309999999999995; KiCadOrientationDeg 90 -> 180
- R4216: FootprintOriginMm 237.91,54.54 -> 246.23999999999998,42.41; KiCadOrientationDeg 90 -> 180
- RB4206: BoardSide F.Cu -> B.Cu; FootprintOriginMm 242.87,84.3 -> 248.4,31.97; KiCadOrientationDeg 0 -> 90
- RB4208: BoardSide F.Cu -> B.Cu; FootprintOriginMm 242.87,39.9 -> 239.27,32.6; KiCadOrientationDeg 0 -> 180
- RB4209: BoardSide B.Cu -> F.Cu; FootprintOriginMm 248.7,93.07 -> 242.87,87.89999999999999; KiCadOrientationDeg 90 -> 0
- RB4210: FootprintOriginMm 264.96999999999997,68.3 -> 239.27,95.0
- RB4211: FootprintOriginMm 248.4,31.97 -> 247.97,74.5; KiCadOrientationDeg 90 -> 180
- RB4212: BoardSide F.Cu -> B.Cu; FootprintOriginMm 242.87,87.89999999999999 -> 248.7,93.07; KiCadOrientationDeg 0 -> 90
- RB4213: FootprintOriginMm 247.23999999999998,28.41 -> 252.71,30.44; KiCadOrientationDeg 180 -> 90
- RB4214: FootprintOriginMm 242.33999999999997,25.71 -> 248.73999999999998,84.31
- RB4215: FootprintOriginMm 244.44,98.21 -> 241.51,91.54; KiCadOrientationDeg 0 -> 270

Commit message: Regenerate and rebuild both jack halves with the hot-quad escape reservation
Evidence rebound (peripheral epoch, foil-collar proposal, control receipt);
jack boards rebuilt from the new placement with source planes and no signal
copper, ready for CI routing.

Co-Authored-By: Claude Opus 5.5 <noreply@anthropic.com>
Parts:
- D4207: BoardSide B.Cu -> F.Cu; FootprintOriginMm 248.25,62.550000000000004 -> 243.21,72.35; KiCadOrientationDeg 90 -> 0
- D4208: FootprintOriginMm 248.35,57.15 -> 251.25,57.45
- D4209: FootprintOriginMm 251.25,57.45 -> 248.25,62.550000000000004
- D4210: FootprintOriginMm 252.35,44.85 -> 248.35,57.15; KiCadOrientationDeg 180 -> 90
- D4212: BoardSide F.Cu -> B.Cu; FootprintOriginMm 243.21,72.35 -> 248.35,46.15; KiCadOrientationDeg 0 -> 90
- D4213: FootprintOriginMm 248.35,46.15 -> 252.35,44.85; KiCadOrientationDeg 90 -> 180
- D4219: BoardSide F.Cu -> B.Cu; FootprintOriginMm 243.21,81.05 -> 236.15,84.65; KiCadOrientationDeg 0 -> 180
- D4220: BoardSide B.Cu -> F.Cu; FootprintOriginMm 236.15,84.65 -> 243.21,81.05; KiCadOrientationDeg 180 -> 0
- R4205: FootprintOriginMm 238.83999999999997,42.309999999999995 -> 253.64,42.309999999999995
- R4206: FootprintOriginMm 242.54,42.41 -> 257.34,42.41
- R4209: FootprintOriginMm 247.23999999999998,28.41 -> 246.04,25.71
- R4210: BoardSide F.Cu -> B.Cu; FootprintOriginMm 245.21,32.64 -> 249.01,25.44; KiCadOrientationDeg 270 -> 90
- R4211: FootprintOriginMm 245.91,91.54 -> 243.91,100.24
- R4212: FootprintOriginMm 243.71,91.54 -> 243.71,95.24
- R4213: FootprintOriginMm 253.64,42.309999999999995 -> 255.64,25.71
- R4214: FootprintOriginMm 257.34,42.41 -> 252.71,30.44; KiCadOrientationDeg 180 -> 90
- R4215: FootprintOriginMm 249.94,42.309999999999995 -> 247.23999999999998,28.41
- R4216: BoardSide B.Cu -> F.Cu; FootprintOriginMm 246.23999999999998,42.41 -> 244.73999999999998,29.01; KiCadOrientationDeg 180 -> 0
- RB4208: BoardSide B.Cu -> F.Cu; FootprintOriginMm 239.27,32.6 -> 242.87,39.9; KiCadOrientationDeg 180 -> 0
- RB4213: FootprintOriginMm 252.71,30.44 -> 254.54,57.51; KiCadOrientationDeg 90 -> 180
- RB4214: FootprintOriginMm 248.73999999999998,84.31 -> 249.94,42.309999999999995
- RB4215: BoardSide F.Cu -> B.Cu; FootprintOriginMm 241.51,91.54 -> 248.73999999999998,84.31; KiCadOrientationDeg 270 -> 180
