File: boards/osc-jack-right/sheets/envelope_E3_JR.kicad_sch (KiCad schematic)
At the start: 66 parts, among them J1501 WQP518MA, J1502 WQP518MA, J1503 WQP518MA, J1504 WQP518MA, J1505 WQP518MA, J1506 WQP518MA, J1507 WQP518MA, U4302 ADG5412FBRUZ, U4303 ADG5412FBRUZ, U4304 ADG5412FBRUZ, U4346 OPA4196IDR, U4347 OPA4196IDR, U4348 OPA4196IDR

Commit message: Move jack halves to six layers with locality placement and grid routing
Owner decision 2026-10-03 (#38): a cut-line bound showed the four-layer
jack halves could not carry their signal nets with intact planes, so both
halves move to six layers and their free packages are re-placed for
locality.

- Placement: scripts/checks/jack_locality.py replaces the
  connectivity-blind first-fit J placer. Packages are pulled toward the
  fixed jacks, LEDs and headers on their nets and toward their own
  module's hardware, then legalized; IC/bypass clusters stay aligned.
  Panel hardware and headers do not move.
- Stack: F/In2/In3/B signals, In1 AGND plane, -12V fill on In3, +12V
  plane on In4; +5V as tracks.
- Routing: scripts/pcbgen/route_jack_grid.py stages terminal arrays,
  rail fanouts and links, signal batches, rip-up-and-reroute and AGND
  stitching, keeping only natively checked stages (0 DRC errors,
  0 parity). The grid router gains N-layer support, windowed search,
  plane fanout, a plane-fill split guard and rip-up-and-reroute.
- Evidence chain: a bounded jack-locality partition transition is
  chained onto the connector-locality proof; superseded four-layer
  stage reports are removed.

Checkpoint: JL 411 and JR 518 native open edges remain. This is a routed
draft in progress; electrical and physical qualification NOT RUN.

Co-Authored-By: Claude Opus 5.5 <noreply@anthropic.com>
Parts:
- C4315: FootprintOriginMm 288.96,95.355 -> 252.04,71.555; KiCadOrientationDeg 90 -> 180
- C4316: FootprintOriginMm 299.87,95.355 -> 264.31,71.555; KiCadOrientationDeg 90 -> 0
- C4317: BoardSide B.Cu -> F.Cu; FootprintOriginMm 186.96,101.755 -> 260.95500000000004,58.86; KiCadOrientationDeg 90 -> 0
- C4318: BoardSide B.Cu -> F.Cu; FootprintOriginMm 197.87,101.755 -> 260.95500000000004,69.77; KiCadOrientationDeg 90 -> 0
- C4319: BoardSide B.Cu -> F.Cu; FootprintOriginMm 203.96,101.755 -> 261.105,55.91; KiCadOrientationDeg 90 -> 270
- C4320: BoardSide B.Cu -> F.Cu; FootprintOriginMm 214.87,101.755 -> 261.105,43.64
- C4372: FootprintOriginMm 298.98,24.55 -> 264.98,50.85
- C4373: FootprintOriginMm 288.96000000000004,24.55 -> 254.96000000000004,50.85
- C4374: FootprintOriginMm 196.98,45.65 -> 259.38,67.58; KiCadOrientationDeg 90 -> 0
- C4375: FootprintOriginMm 186.96,45.65 -> 259.38,57.56; KiCadOrientationDeg 90 -> 0
- C4376: FootprintOriginMm 213.98,45.65 -> 254.96000000000004,88.78000000000002; KiCadOrientationDeg 90 -> 270
- C4377: FootprintOriginMm 203.96,45.65 -> 264.98,88.78000000000002; KiCadOrientationDeg 90 -> 270
- D4301: FootprintOriginMm 285.23,43.21 -> 255.93,28.81
- D4302: FootprintOriginMm 302.23,43.21 -> 255.93,95.21000000000001
- D4303: FootprintOriginMm 200.23000000000002,56.910000000000004 -> 260.23,28.81
- D4307: FootprintOriginMm 266.25,127.75 -> 265.25,62.550000000000004
- D4308: FootprintOriginMm 283.25,127.75 -> 265.35,57.15
- D4309: FootprintOriginMm 311.65,142.35 -> 268.25,57.45
- D4310: BoardSide B.Cu -> F.Cu; FootprintOriginMm 311.65,147.75 -> 260.21000000000004,72.35; KiCadOrientationDeg 90 -> 0
- D4312: BoardSide B.Cu -> F.Cu; FootprintOriginMm 311.65,153.15 -> 260.21000000000004,75.25; KiCadOrientationDeg 90 -> 0
- D4313: BoardSide F.Cu -> B.Cu; FootprintOriginMm 192.21,21.55 -> 257.75,44.95; KiCadOrientationDeg 0 -> 180
- D4314: BoardSide F.Cu -> B.Cu; FootprintOriginMm 209.21,21.55 -> 265.35,46.15; KiCadOrientationDeg 0 -> 90
- D4315: FootprintOriginMm 226.21,21.55 -> 260.21000000000004,78.15
- D4317: BoardSide F.Cu -> B.Cu; FootprintOriginMm 243.21,21.55 -> 253.15,84.65; KiCadOrientationDeg 0 -> 180
- D4318: BoardSide F.Cu -> B.Cu; FootprintOriginMm 260.21000000000004,21.55 -> 269.35,44.85; KiCadOrientationDeg 0 -> 180
- D4319: FootprintOriginMm 277.21000000000004,21.55 -> 260.21000000000004,81.05
- D4320: BoardSide F.Cu -> B.Cu; FootprintOriginMm 294.21000000000004,21.55 -> 266.45000000000005,84.65; KiCadOrientationDeg 0 -> 180
- R4305: FootprintOriginMm 265.74,62.209999999999994 -> 264.64,42.51
- R4306: FootprintOriginMm 282.74,62.209999999999994 -> 268.34,42.309999999999995
- R4307: FootprintOriginMm 299.74,62.209999999999994 -> 251.94,87.21
- R4308: FootprintOriginMm 202.64,70.00999999999999 -> 254.54,57.51
- R4309: FootprintOriginMm 219.64,70.00999999999999 -> 272.03999999999996,42.309999999999995
- R4310: FootprintOriginMm 236.64,70.00999999999999 -> 271.14,84.31
- R4311: FootprintOriginMm 253.64,70.00999999999999 -> 267.94,87.21
- R4312: FootprintOriginMm 270.64,70.00999999999999 -> 255.64,67.61
- R4313: FootprintOriginMm 287.64,70.00999999999999 -> 275.74,42.41
- R4314: FootprintOriginMm 214.44,73.61 -> 278.71000000000004,44.54; KiCadOrientationDeg 180 -> 90
- R4315: FootprintOriginMm 231.44,73.61 -> 252.71,30.44; KiCadOrientationDeg 180 -> 90
- R4316: FootprintOriginMm 248.44,73.61 -> 254.91,54.54; KiCadOrientationDeg 180 -> 90
- RB4305: BoardSide B.Cu -> F.Cu; FootprintOriginMm 295.16999999999996,73.0 -> 259.87,87.89999999999999; KiCadOrientationDeg 180 -> 0
- RB4306: FootprintOriginMm 194.47,74.3 -> 264.96999999999997,74.5
- RB4307: FootprintOriginMm 184.67000000000002,112.69999999999999 -> 256.46999999999997,32.6
- RB4308: BoardSide B.Cu -> F.Cu; FootprintOriginMm 199.27,112.69999999999999 -> 259.87,84.3; KiCadOrientationDeg 180 -> 0
- RB4309: FootprintOriginMm 216.27,112.69999999999999 -> 261.37,32.6
- RB4310: BoardSide B.Cu -> F.Cu; FootprintOriginMm 233.27,112.69999999999999 -> 259.87,39.9; KiCadOrientationDeg 180 -> 0
- RB4311: BoardSide B.Cu -> F.Cu; FootprintOriginMm 250.27,112.69999999999999 -> 259.87,36.300000000000004; KiCadOrientationDeg 180 -> 0
- RB4312: FootprintOriginMm 267.27,112.69999999999999 -> 281.96999999999997,68.3
- RB4313: FootprintOriginMm 191.23999999999998,152.81 -> 258.51000000000005,91.54; KiCadOrientationDeg 0 -> 270
- RB4314: FootprintOriginMm 227.73999999999998,153.01 -> 258.51000000000005,32.64; KiCadOrientationDeg 0 -> 270
- RB4315: FootprintOriginMm 244.73999999999998,153.01 -> 259.24,95.11
- U4302: FootprintOriginMm 294.12,96.38000000000001 -> 257.88,71.88000000000001
- U4303: BoardSide B.Cu -> F.Cu; FootprintOriginMm 192.12,102.78 -> 260.58000000000004,64.02; KiCadOrientationDeg 180 -> 90
- U4304: BoardSide B.Cu -> F.Cu; FootprintOriginMm 209.12,102.78 -> 260.78000000000003,50.07; KiCadOrientationDeg 180 -> 270
- U4346: FootprintOriginMm 293.97,25.25 -> 259.97,51.550000000000004
- U4347: FootprintOriginMm 191.97,46.35 -> 258.68,62.57; KiCadOrientationDeg 180 -> 90
- U4348: FootprintOriginMm 208.97,46.35 -> 259.97,88.08000000000001; KiCadOrientationDeg 180 -> 0

Commit message: Place jack-right with span-aware swaps and route it to 190 open edges
Rebuilt from the swap-pass placement; rails, negotiated routing (1236 -> 283),
re-offered rip-up, signal batches, AGND stitching and escapes. Reports come
from the adopted stage's native DRC (0 errors, 0 parity) and native ratsnest.

Co-Authored-By: Claude Opus 5.5 <noreply@anthropic.com>
Parts:
- D4307: FootprintOriginMm 265.25,62.550000000000004 -> 268.25,57.45
- D4309: FootprintOriginMm 268.25,57.45 -> 265.35,46.15
- D4310: BoardSide F.Cu -> B.Cu; FootprintOriginMm 260.21000000000004,72.35 -> 257.75,44.95; KiCadOrientationDeg 0 -> 180
- D4313: BoardSide B.Cu -> F.Cu; FootprintOriginMm 257.75,44.95 -> 260.21000000000004,78.15; KiCadOrientationDeg 180 -> 0
- D4314: BoardSide B.Cu -> F.Cu; FootprintOriginMm 265.35,46.15 -> 260.21000000000004,72.35; KiCadOrientationDeg 90 -> 0
- D4315: BoardSide F.Cu -> B.Cu; FootprintOriginMm 260.21000000000004,78.15 -> 265.25,62.550000000000004; KiCadOrientationDeg 0 -> 90
- D4317: FootprintOriginMm 253.15,84.65 -> 266.45000000000005,84.65
- D4318: FootprintOriginMm 269.35,44.85 -> 276.55,96.65
- D4320: FootprintOriginMm 266.45000000000005,84.65 -> 253.15,84.65
- R4307: FootprintOriginMm 251.94,87.21 -> 255.64,67.61
- R4308: FootprintOriginMm 254.54,57.51 -> 254.91,54.54; KiCadOrientationDeg 180 -> 90
- R4309: FootprintOriginMm 272.03999999999996,42.309999999999995 -> 271.91,54.54; KiCadOrientationDeg 180 -> 90
- R4310: FootprintOriginMm 271.14,84.31 -> 271.53999999999996,57.51
- R4311: BoardSide B.Cu -> F.Cu; FootprintOriginMm 267.94,87.21 -> 258.51000000000005,91.54; KiCadOrientationDeg 180 -> 270
- R4312: BoardSide B.Cu -> F.Cu; FootprintOriginMm 255.64,67.61 -> 259.24,95.11; KiCadOrientationDeg 180 -> 0
- R4313: FootprintOriginMm 275.74,42.41 -> 272.03999999999996,42.309999999999995
- R4314: FootprintOriginMm 278.71000000000004,44.54 -> 275.74,42.41; KiCadOrientationDeg 90 -> 180
- R4315: FootprintOriginMm 252.71,30.44 -> 261.71000000000004,44.54
- R4316: BoardSide B.Cu -> F.Cu; FootprintOriginMm 254.91,54.54 -> 258.51000000000005,32.64; KiCadOrientationDeg 90 -> 270
- RB4305: FootprintOriginMm 259.87,87.89999999999999 -> 259.87,39.9
- RB4306: BoardSide B.Cu -> F.Cu; FootprintOriginMm 264.96999999999997,74.5 -> 259.87,36.300000000000004; KiCadOrientationDeg 180 -> 0
- RB4307: BoardSide B.Cu -> F.Cu; FootprintOriginMm 256.46999999999997,32.6 -> 259.87,84.3; KiCadOrientationDeg 180 -> 0
- RB4308: FootprintOriginMm 259.87,84.3 -> 259.87,87.89999999999999
- RB4310: BoardSide F.Cu -> B.Cu; FootprintOriginMm 259.87,39.9 -> 256.46999999999997,32.6; KiCadOrientationDeg 0 -> 180
- RB4311: BoardSide F.Cu -> B.Cu; FootprintOriginMm 259.87,36.300000000000004 -> 264.96999999999997,74.5; KiCadOrientationDeg 0 -> 180
- RB4312: FootprintOriginMm 281.96999999999997,68.3 -> 266.0,93.07; KiCadOrientationDeg 180 -> 90
- RB4313: BoardSide F.Cu -> B.Cu; FootprintOriginMm 258.51000000000005,91.54 -> 254.54,57.51; KiCadOrientationDeg 270 -> 180
- RB4314: BoardSide F.Cu -> B.Cu; FootprintOriginMm 258.51000000000005,32.64 -> 267.94,87.21; KiCadOrientationDeg 270 -> 180
- RB4315: BoardSide F.Cu -> B.Cu; FootprintOriginMm 259.24,95.11 -> 251.94,87.21; KiCadOrientationDeg 0 -> 180

Commit message: Regenerate and rebuild both jack halves with the hot-quad escape reservation
Evidence rebound (peripheral epoch, foil-collar proposal, control receipt);
jack boards rebuilt from the new placement with source planes and no signal
copper, ready for CI routing.

Co-Authored-By: Claude Opus 5.5 <noreply@anthropic.com>
Parts:
- D4307: FootprintOriginMm 268.25,57.45 -> 265.25,62.550000000000004
- D4309: FootprintOriginMm 265.35,46.15 -> 268.25,57.45
- D4310: FootprintOriginMm 257.75,44.95 -> 269.35,44.85
- D4313: BoardSide F.Cu -> B.Cu; FootprintOriginMm 260.21000000000004,78.15 -> 265.35,46.15; KiCadOrientationDeg 0 -> 90
- D4315: FootprintOriginMm 265.25,62.550000000000004 -> 257.75,44.95; KiCadOrientationDeg 90 -> 180
- D4317: BoardSide B.Cu -> F.Cu; FootprintOriginMm 266.45000000000005,84.65 -> 260.21000000000004,78.15; KiCadOrientationDeg 180 -> 0
- D4318: FootprintOriginMm 276.55,96.65 -> 266.45000000000005,84.65
- R4305: FootprintOriginMm 264.64,42.51 -> 272.03999999999996,42.309999999999995
- R4306: FootprintOriginMm 268.34,42.309999999999995 -> 269.84,31.21
- R4307: FootprintOriginMm 255.64,67.61 -> 259.34,25.71
- R4308: BoardSide B.Cu -> F.Cu; FootprintOriginMm 254.91,54.54 -> 259.24,31.21; KiCadOrientationDeg 90 -> 0
- R4309: FootprintOriginMm 271.91,54.54 -> 255.64,67.61; KiCadOrientationDeg 90 -> 180
- R4310: FootprintOriginMm 271.53999999999996,57.51 -> 254.91,54.54; KiCadOrientationDeg 180 -> 90
- R4311: BoardSide F.Cu -> B.Cu; FootprintOriginMm 258.51000000000005,91.54 -> 264.64,42.51; KiCadOrientationDeg 270 -> 180
- R4312: BoardSide F.Cu -> B.Cu; FootprintOriginMm 259.24,95.11 -> 261.71000000000004,44.54; KiCadOrientationDeg 0 -> 90
- R4313: FootprintOriginMm 272.03999999999996,42.309999999999995 -> 262.31,24.94; KiCadOrientationDeg 180 -> 90
- R4314: BoardSide B.Cu -> F.Cu; FootprintOriginMm 275.74,42.41 -> 261.74,29.01; KiCadOrientationDeg 180 -> 0
- R4315: BoardSide B.Cu -> F.Cu; FootprintOriginMm 261.71000000000004,44.54 -> 262.21000000000004,32.64; KiCadOrientationDeg 90 -> 270
- R4316: FootprintOriginMm 258.51000000000005,32.64 -> 259.24,33.41; KiCadOrientationDeg 270 -> 0
- RB4312: FootprintOriginMm 266.0,93.07 -> 265.3,100.27
- RB4313: FootprintOriginMm 254.54,57.51 -> 271.91,54.54; KiCadOrientationDeg 180 -> 90
- RB4314: FootprintOriginMm 267.94,87.21 -> 268.34,42.309999999999995
- RB4315: FootprintOriginMm 251.94,87.21 -> 250.94,87.21
