File: boards/osc-jack-right/sheets/wavefolder_W1_JR.kicad_sch (KiCad schematic)
At the start: 54 parts, among them J1107 WQP518MA, J1108 WQP518MA, J1207 WQP518MA, J1208 WQP518MA, U5202 ADG5412FBRUZ, U5203 ADG5412FBRUZ, U5204 ADG5412FBRUZ, U5212 OPA4196IDR, U5213 OPA4196IDR

Commit message: Move jack halves to six layers with locality placement and grid routing
Owner decision 2026-10-03 (#38): a cut-line bound showed the four-layer
jack halves could not carry their signal nets with intact planes, so both
halves move to six layers and their free packages are re-placed for
locality.

- Placement: scripts/checks/jack_locality.py replaces the
  connectivity-blind first-fit J placer. Packages are pulled toward the
  fixed jacks, LEDs and headers on their nets and toward their own
  module's hardware, then legalized; IC/bypass clusters stay aligned.
  Panel hardware and headers do not move.
- Stack: F/In2/In3/B signals, In1 AGND plane, -12V fill on In3, +12V
  plane on In4; +5V as tracks.
- Routing: scripts/pcbgen/route_jack_grid.py stages terminal arrays,
  rail fanouts and links, signal batches, rip-up-and-reroute and AGND
  stitching, keeping only natively checked stages (0 DRC errors,
  0 parity). The grid router gains N-layer support, windowed search,
  plane fanout, a plane-fill split guard and rip-up-and-reroute.
- Evidence chain: a bounded jack-locality partition transition is
  chained onto the connector-locality proof; superseded four-layer
  stage reports are removed.

Checkpoint: JL 411 and JR 518 native open edges remain. This is a routed
draft in progress; electrical and physical qualification NOT RUN.

Co-Authored-By: Claude Opus 5.5 <noreply@anthropic.com>
Parts:
- C5220: BoardSide B.Cu -> F.Cu; FootprintOriginMm 254.96,108.155 -> 193.30499999999998,124.81; KiCadOrientationDeg 90 -> 270
- C5221: BoardSide B.Cu -> F.Cu; FootprintOriginMm 265.87,108.155 -> 193.30499999999998,112.53999999999999
- C5222: FootprintOriginMm 271.96,108.155 -> 189.26000000000002,127.35499999999999
- C5223: FootprintOriginMm 282.87,108.155 -> 200.17000000000002,127.35499999999999
- C5224: FootprintOriginMm 288.96,108.155 -> 202.46,127.35499999999999
- C5225: FootprintOriginMm 299.87,108.155 -> 213.37,127.35499999999999
- C5240: FootprintOriginMm 264.98,55.65 -> 199.48,112.85
- C5241: FootprintOriginMm 254.96000000000004,55.65 -> 189.46,112.85
- C5242: FootprintOriginMm 281.98,55.65 -> 211.78,112.85
- C5243: FootprintOriginMm 271.96000000000004,55.65 -> 201.76000000000002,112.85
- D5201: BoardSide B.Cu -> F.Cu; FootprintOriginMm 234.23000000000002,85.21000000000001 -> 194.03,102.91; KiCadOrientationDeg 180 -> 0
- D5202: BoardSide B.Cu -> F.Cu; FootprintOriginMm 251.23000000000002,85.21000000000001 -> 208.53,109.61; KiCadOrientationDeg 180 -> 0
- D5203: FootprintOriginMm 268.23,85.21000000000001 -> 221.81,112.63000000000001; KiCadOrientationDeg 180 -> 90
- D5214: BoardSide F.Cu -> B.Cu; FootprintOriginMm 277.21000000000004,86.25 -> 186.85,113.44999999999999; KiCadOrientationDeg 0 -> 90
- D5215: BoardSide F.Cu -> B.Cu; FootprintOriginMm 294.21000000000004,86.25 -> 183.95,113.44999999999999; KiCadOrientationDeg 0 -> 90
- D5216: BoardSide F.Cu -> B.Cu; FootprintOriginMm 192.21,87.15 -> 185.25,126.65; KiCadOrientationDeg 0 -> 180
- D5217: BoardSide F.Cu -> B.Cu; FootprintOriginMm 209.21,87.15 -> 194.45,106.95; KiCadOrientationDeg 0 -> 180
- D5219: BoardSide F.Cu -> B.Cu; FootprintOriginMm 226.21,87.25 -> 189.05,108.05; KiCadOrientationDeg 0 -> 90
- D5220: FootprintOriginMm 243.21,89.15 -> 193.61,109.25
- D5221: FootprintOriginMm 260.21000000000004,89.15 -> 193.61,129.15
- D5222: BoardSide F.Cu -> B.Cu; FootprintOriginMm 277.21000000000004,89.15 -> 187.55,131.75; KiCadOrientationDeg 0 -> 90
- D5224: BoardSide F.Cu -> B.Cu; FootprintOriginMm 294.21000000000004,89.15 -> 196.15,104.05; KiCadOrientationDeg 0 -> 180
- D5225: BoardSide F.Cu -> B.Cu; FootprintOriginMm 192.21,90.05 -> 205.35,106.95; KiCadOrientationDeg 0 -> 180
- D5226: FootprintOriginMm 209.21,90.05 -> 193.61,106.35
- D5227: FootprintOriginMm 226.21,90.15 -> 193.61,132.05
- R5205: FootprintOriginMm 249.04,162.31 -> 188.04,104.41
- R5206: FootprintOriginMm 252.73999999999998,162.31 -> 204.64,104.41
- R5207: FootprintOriginMm 266.03999999999996,162.31 -> 200.83999999999997,101.21
- R5208: FootprintOriginMm 269.74,162.31 -> 189.41,116.54; KiCadOrientationDeg 180 -> 90
- R5209: FootprintOriginMm 283.03999999999996,162.31 -> 209.31,106.54; KiCadOrientationDeg 180 -> 90
- R5210: BoardSide B.Cu -> F.Cu; FootprintOriginMm 286.74,162.31 -> 211.10999999999999,119.04; KiCadOrientationDeg 180 -> 270
- R5211: FootprintOriginMm 290.44,162.31 -> 187.14,140.01
- R5212: FootprintOriginMm 294.14,162.31 -> 184.23999999999998,129.21
- R5213: BoardSide B.Cu -> F.Cu; FootprintOriginMm 297.84,162.31 -> 208.23999999999998,106.50999999999999; KiCadOrientationDeg 180 -> 0
- R5214: BoardSide B.Cu -> F.Cu; FootprintOriginMm 301.53999999999996,162.31 -> 211.81,109.74; KiCadOrientationDeg 180 -> 270
- R5215: FootprintOriginMm 305.24,162.31 -> 194.71,95.04; KiCadOrientationDeg 180 -> 90
- R5216: FootprintOriginMm 312.31,26.14 -> 191.73999999999998,104.41; KiCadOrientationDeg 90 -> 180
- R5271: FootprintOriginMm 184.67000000000002,28.700000000000003 -> 213.17000000000002,116.6
- R5272: BoardSide B.Cu -> F.Cu; FootprintOriginMm 198.37,28.700000000000003 -> 208.2,118.97; KiCadOrientationDeg 180 -> 270
- R5273: FootprintOriginMm 312.31,29.84 -> 211.71,95.04
- R5274: FootprintOriginMm 198.01,32.339999999999996 -> 217.83999999999997,101.21; KiCadOrientationDeg 90 -> 180
- R5275: FootprintOriginMm 312.31,33.54 -> 199.94,87.21; KiCadOrientationDeg 90 -> 180
- U5202: BoardSide B.Cu -> F.Cu; FootprintOriginMm 260.12,109.18 -> 192.98,118.97; KiCadOrientationDeg 180 -> 270
- U5203: FootprintOriginMm 277.12,109.18 -> 194.42000000000002,128.38
- U5204: FootprintOriginMm 294.12,109.18 -> 207.62,128.38
- U5212: FootprintOriginMm 259.97,56.35 -> 194.47,113.55
- U5213: FootprintOriginMm 276.97,56.35 -> 206.77,113.55

Commit message: Place jack-right with span-aware swaps and route it to 190 open edges
Rebuilt from the swap-pass placement; rails, negotiated routing (1236 -> 283),
re-offered rip-up, signal batches, AGND stitching and escapes. Reports come
from the adopted stage's native DRC (0 errors, 0 parity) and native ratsnest.

Co-Authored-By: Claude Opus 5.5 <noreply@anthropic.com>
Parts:
- D5201: BoardSide F.Cu -> B.Cu; FootprintOriginMm 194.03,102.91 -> 221.81,112.63000000000001; KiCadOrientationDeg 0 -> 90
- D5203: FootprintOriginMm 221.81,112.63000000000001 -> 221.93,106.81; KiCadOrientationDeg 90 -> 180
- D5214: BoardSide B.Cu -> F.Cu; FootprintOriginMm 186.85,113.44999999999999 -> 193.61,109.25; KiCadOrientationDeg 90 -> 0
- D5215: FootprintOriginMm 183.95,113.44999999999999 -> 189.05,108.05
- D5216: FootprintOriginMm 185.25,126.65 -> 183.95,113.44999999999999; KiCadOrientationDeg 180 -> 90
- D5217: FootprintOriginMm 194.45,106.95 -> 186.85,113.44999999999999; KiCadOrientationDeg 180 -> 90
- D5219: BoardSide B.Cu -> F.Cu; FootprintOriginMm 189.05,108.05 -> 193.61,106.35; KiCadOrientationDeg 90 -> 0
- D5220: BoardSide F.Cu -> B.Cu; FootprintOriginMm 193.61,109.25 -> 213.15,104.15; KiCadOrientationDeg 0 -> 180
- D5221: BoardSide F.Cu -> B.Cu; FootprintOriginMm 193.61,129.15 -> 194.45,106.95; KiCadOrientationDeg 0 -> 180
- D5222: FootprintOriginMm 187.55,131.75 -> 205.35,106.95; KiCadOrientationDeg 90 -> 180
- D5224: BoardSide B.Cu -> F.Cu; FootprintOriginMm 196.15,104.05 -> 193.61,129.15; KiCadOrientationDeg 180 -> 0
- D5225: BoardSide B.Cu -> F.Cu; FootprintOriginMm 205.35,106.95 -> 193.61,132.05; KiCadOrientationDeg 180 -> 0
- D5226: BoardSide F.Cu -> B.Cu; FootprintOriginMm 193.61,106.35 -> 185.25,126.65; KiCadOrientationDeg 0 -> 180
- D5227: BoardSide F.Cu -> B.Cu; FootprintOriginMm 193.61,132.05 -> 187.55,131.75; KiCadOrientationDeg 0 -> 90
- R5205: BoardSide B.Cu -> F.Cu; FootprintOriginMm 188.04,104.41 -> 228.33999999999997,111.61; KiCadOrientationDeg 180 -> 0
- R5206: BoardSide B.Cu -> F.Cu; FootprintOriginMm 204.64,104.41 -> 228.21,106.84; KiCadOrientationDeg 180 -> 270
- R5207: FootprintOriginMm 200.83999999999997,101.21 -> 188.04,104.41
- R5209: BoardSide B.Cu -> F.Cu; FootprintOriginMm 209.31,106.54 -> 225.23999999999998,108.31; KiCadOrientationDeg 90 -> 0
- R5210: BoardSide F.Cu -> B.Cu; FootprintOriginMm 211.10999999999999,119.04 -> 225.94,108.41; KiCadOrientationDeg 270 -> 180
- R5213: FootprintOriginMm 208.23999999999998,106.50999999999999 -> 211.10999999999999,119.04; KiCadOrientationDeg 0 -> 270
- R5215: BoardSide B.Cu -> F.Cu; FootprintOriginMm 194.71,95.04 -> 208.23999999999998,106.50999999999999; KiCadOrientationDeg 90 -> 0
- R5216: FootprintOriginMm 191.73999999999998,104.41 -> 209.31,106.54; KiCadOrientationDeg 180 -> 90
- R5271: FootprintOriginMm 213.17000000000002,116.6 -> 213.17000000000002,109.19999999999999
- R5272: BoardSide F.Cu -> B.Cu; FootprintOriginMm 208.2,118.97 -> 215.37,113.0; KiCadOrientationDeg 270 -> 180
- R5273: FootprintOriginMm 211.71,95.04 -> 204.64,104.41; KiCadOrientationDeg 90 -> 180
- R5274: BoardSide B.Cu -> F.Cu; FootprintOriginMm 217.83999999999997,101.21 -> 225.23999999999998,106.11; KiCadOrientationDeg 180 -> 0
- R5275: BoardSide B.Cu -> F.Cu; FootprintOriginMm 199.94,87.21 -> 194.33999999999997,154.51; KiCadOrientationDeg 180 -> 0

Commit message: Regenerate and rebuild both jack halves with the hot-quad escape reservation
Evidence rebound (peripheral epoch, foil-collar proposal, control receipt);
jack boards rebuilt from the new placement with source planes and no signal
copper, ready for CI routing.

Co-Authored-By: Claude Opus 5.5 <noreply@anthropic.com>
Parts:
- C5224: BoardSide B.Cu -> F.Cu; FootprintOriginMm 202.46,127.35499999999999 -> 193.355,128.86; KiCadOrientationDeg 90 -> 0
- C5225: BoardSide B.Cu -> F.Cu; FootprintOriginMm 213.37,127.35499999999999 -> 193.355,139.77; KiCadOrientationDeg 90 -> 0
- D5201: BoardSide B.Cu -> F.Cu; FootprintOriginMm 221.81,112.63000000000001 -> 208.41,106.73; KiCadOrientationDeg 90 -> 270
- D5202: BoardSide F.Cu -> B.Cu; FootprintOriginMm 208.53,109.61 -> 221.81,109.73; KiCadOrientationDeg 0 -> 90
- D5203: FootprintOriginMm 221.93,106.81 -> 225.81,109.73; KiCadOrientationDeg 180 -> 90
- D5214: BoardSide F.Cu -> B.Cu; FootprintOriginMm 193.61,109.25 -> 183.95,113.44999999999999; KiCadOrientationDeg 0 -> 90
- D5215: BoardSide B.Cu -> F.Cu; FootprintOriginMm 189.05,108.05 -> 193.61,109.25; KiCadOrientationDeg 90 -> 0
- D5216: FootprintOriginMm 183.95,113.44999999999999 -> 186.85,113.44999999999999
- D5217: FootprintOriginMm 186.85,113.44999999999999 -> 187.85,108.05
- D5219: BoardSide F.Cu -> B.Cu; FootprintOriginMm 193.61,106.35 -> 209.25,126.65; KiCadOrientationDeg 0 -> 180
- D5221: FootprintOriginMm 194.45,106.95 -> 205.35,106.95
- D5222: BoardSide B.Cu -> F.Cu; FootprintOriginMm 205.35,106.95 -> 209.21,103.15; KiCadOrientationDeg 180 -> 0
- D5224: BoardSide F.Cu -> B.Cu; FootprintOriginMm 193.61,129.15 -> 205.35,129.55; KiCadOrientationDeg 0 -> 180
- D5225: BoardSide F.Cu -> B.Cu; FootprintOriginMm 193.61,132.05 -> 187.55,131.75; KiCadOrientationDeg 0 -> 90
- D5226: FootprintOriginMm 185.25,126.65 -> 203.85,126.65
- D5227: FootprintOriginMm 187.55,131.75 -> 185.25,126.65; KiCadOrientationDeg 90 -> 180
- R5205: BoardSide F.Cu -> B.Cu; FootprintOriginMm 228.33999999999997,111.61 -> 187.14,140.01; KiCadOrientationDeg 0 -> 180
- R5206: FootprintOriginMm 228.21,106.84 -> 194.33999999999997,154.51; KiCadOrientationDeg 270 -> 0
- R5207: FootprintOriginMm 188.04,104.41 -> 187.83999999999997,104.41
- R5208: FootprintOriginMm 189.41,116.54 -> 190.81,106.54
- R5209: BoardSide F.Cu -> B.Cu; FootprintOriginMm 225.23999999999998,108.31 -> 200.83999999999997,101.21; KiCadOrientationDeg 0 -> 180
- R5210: BoardSide B.Cu -> F.Cu; FootprintOriginMm 225.94,108.41 -> 194.33999999999997,103.11; KiCadOrientationDeg 180 -> 0
- R5211: FootprintOriginMm 187.14,140.01 -> 203.91,132.83999999999997; KiCadOrientationDeg 180 -> 90
- R5212: BoardSide B.Cu -> F.Cu; FootprintOriginMm 184.23999999999998,129.21 -> 211.10999999999999,117.14; KiCadOrientationDeg 180 -> 270
- R5213: FootprintOriginMm 211.10999999999999,119.04 -> 200.83999999999997,162.51; KiCadOrientationDeg 270 -> 0
- R5214: BoardSide F.Cu -> B.Cu; FootprintOriginMm 211.81,109.74 -> 200.83999999999997,162.31; KiCadOrientationDeg 270 -> 180
- R5215: BoardSide F.Cu -> B.Cu; FootprintOriginMm 208.23999999999998,106.50999999999999 -> 209.31,106.54; KiCadOrientationDeg 0 -> 90
- R5216: BoardSide B.Cu -> F.Cu; FootprintOriginMm 209.31,106.54 -> 211.51,107.04; KiCadOrientationDeg 90 -> 270
- R5272: BoardSide B.Cu -> F.Cu; FootprintOriginMm 215.37,113.0 -> 210.7,111.36999999999999; KiCadOrientationDeg 180 -> 270
- R5274: BoardSide F.Cu -> B.Cu; FootprintOriginMm 225.23999999999998,106.11 -> 221.54,106.50999999999999; KiCadOrientationDeg 0 -> 180
- R5275: BoardSide F.Cu -> B.Cu; FootprintOriginMm 194.33999999999997,154.51 -> 184.23999999999998,129.21; KiCadOrientationDeg 0 -> 180
- U5204: BoardSide B.Cu -> F.Cu; FootprintOriginMm 207.62,128.38 -> 192.98,134.02; KiCadOrientationDeg 180 -> 90
