File: boards/osc-control/sheets/manual_ab_X1_P.kicad_sch (KiCad schematic)
At the start: 9 parts, among them SW608 2MS1T1B1M2QES-5, U3303 OPA4197IPWR

Commit message: Keep control-board bypass groups local and connect their supply loops
Parts:
- C3306: FootprintOriginMm 240.64,187.46 -> 94.46000000000001,287.81; KiCadOrientationDeg 180 -> 270
- C3307: FootprintOriginMm 244.39,187.46 -> 104.78,287.81; KiCadOrientationDeg 180 -> 270
- U3303: FootprintOriginMm 217.35,179.63 -> 99.62,287.11; KiCadOrientationDeg 180 -> 0
Changed lines of the file:
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@@
     (property "BoardSide" "B.Cu" (at 1061.72 104.14 0) (effects (font (size 1.27 1.27)) (hide yes)))
     (property "BoardAssignment" "P" (at 1061.72 104.14 0) (effects (font (size 1.27 1.27)) (hide yes)))
-    (property "KiCadOrientationDeg" "180" (at 1061.72 104.14 0) (effects (font (size 1.27 1.27)) (hide yes)))
-    (property "FootprintOriginMm" "217.35,179.63" (at 1061.72 104.14 0) (effects (font (size 1.27 1.27)) (hide yes)))
+    (property "KiCadOrientationDeg" "0" (at 1061.72 104.14 0) (effects (font (size 1.27 1.27)) (hide yes)))
+    (property "FootprintOriginMm" "99.62,287.11" (at 1061.72 104.14 0) (effects (font (size 1.27 1.27)) (hide yes)))
     (property "Sensitive" "" (at 1061.72 104.14 0) (effects (font (size 1.27 1.27)) (hide yes)))
     (pin "1")
@@
     (property "BoardSide" "B.Cu" (at 45.72 142.24 0) (effects (font (size 1.27 1.27)) (hide yes)))
     (property "BoardAssignment" "P" (at 45.72 142.24 0) (effects (font (size 1.27 1.27)) (hide yes)))
-    (property "KiCadOrientationDeg" "180" (at 45.72 142.24 0) (effects (font (size 1.27 1.27)) (hide yes)))
-    (property "FootprintOriginMm" "217.35,179.63" (at 45.72 142.24 0) (effects (font (size 1.27 1.27)) (hide yes)))
+    (property "KiCadOrientationDeg" "0" (at 45.72 142.24 0) (effects (font (size 1.27 1.27)) (hide yes)))
+    (property "FootprintOriginMm" "99.62,287.11" (at 45.72 142.24 0) (effects (font (size 1.27 1.27)) (hide yes)))
     (property "Sensitive" "" (at 45.72 142.24 0) (effects (font (size 1.27 1.27)) (hide yes)))
     (pin "5")
@@
     (property "BoardSide" "B.Cu" (at 109.22 142.24 0) (effects (font (size 1.27 1.27)) (hide yes)))
     (property "BoardAssignment" "P" (at 109.22 142.24 0) (effects (font (size 1.27 1.27)) (hide yes)))
-    (property "KiCadOrientationDeg" "180" (at 109.22 142.24 0) (effects (font (size 1.27 1.27)) (hide yes)))
-    (property "FootprintOriginMm" "217.35,179.63" (at 109.22 142.24 0) (effects (font (size 1.27 1.27)) (hide yes)))
+    (property "KiCadOrientationDeg" "0" (at 109.22 142.24 0) (effects (font (size 1.27 1.27)) (hide yes)))
+    (property "FootprintOriginMm" "99.62,287.11" (at 109.22 142.24 0) (effects (font (size 1.27 1.27)) (hide yes)))
     (property "Sensitive" "" (at 109.22 142.24 0) (effects (font (size 1.27 1.27)) (hide yes)))
     (pin "8")
@@
     (property "BoardSide" "B.Cu" (at 172.72 142.24 0) (effects (font (size 1.27 1.27)) (hide yes)))
     (property "BoardAssignment" "P" (at 172.72 142.24 0) (effects (font (size 1.27 1.27)) (hide yes)))
-    (property "KiCadOrientationDeg" "180" (at 172.72 142.24 0) (effects (font (size 1.27 1.27)) (hide yes)))
-    (property "FootprintOriginMm" "217.35,179.63" (at 172.72 142.24 0) (effects (font (size 1.27 1.27)) (hide yes)))
+    (property "KiCadOrientationDeg" "0" (at 172.72 142.24 0) (effects (font (size 1.27 1.27)) (hide yes)))
+    (property "FootprintOriginMm" "99.62,287.11" (at 172.72 142.24 0) (effects (font (size 1.27 1.27)) (hide yes)))
     (property "Sensitive" "" (at 172.72 142.24 0) (effects (font (size 1.27 1.27)) (hide yes)))
     (pin "12")
@@
     (property "BoardSide" "B.Cu" (at 236.22 142.24 0) (effects (font (size 1.27 1.27)) (hide yes)))
     (property "BoardAssignment" "P" (at 236.22 142.24 0) (effects (font (size 1.27 1.27)) (hide yes)))
-    (property "KiCadOrientationDeg" "180" (at 236.22 142.24 0) (effects (font (size 1.27 1.27)) (hide yes)))
-    (property "FootprintOriginMm" "217.35,179.63" (at 236.22 142.24 0) (effects (font (size 1.27 1.27)) (hide yes)))
+    (property "KiCadOrientationDeg" "0" (at 236.22 142.24 0) (effects (font (size 1.27 1.27)) (hide yes)))
+    (property "FootprintOriginMm" "99.62,287.11" (at 236.22 142.24 0) (effects (font (size 1.27 1.27)) (hide yes)))
     (property "Sensitive" "" (at 236.22 142.24 0) (effects (font (size 1.27 1.27)) (hide yes)))
     (pin "4")
@@
     (property "BoardSide" "B.Cu" (at 553.72 142.24 0) (effects (font (size 1.27 1.27)) (hide yes)))
     (property "BoardAssignment" "P" (at 553.72 142.24 0) (effects (font (size 1.27 1.27)) (hide yes)))
-    (property "KiCadOrientationDeg" "180" (at 553.72 142.24 0) (effects (font (size 1.27 1.27)) (hide yes)))
-    (property "FootprintOriginMm" "240.64,187.46" (at 553.72 142.24 0) (effects (font (size 1.27 1.27)) (hide yes)))
+    (property "KiCadOrientationDeg" "270" (at 553.72 142.24 0) (effects (font (size 1.27 1.27)) (hide yes)))
+    (property "FootprintOriginMm" "94.46000000000001,287.81" (at 553.72 142.24 0) (effects (font (size 1.27 1.27)) (hide yes)))
     (property "Sensitive" "" (at 553.72 142.24 0) (effects (font (size 1.27 1.27)) (hide yes)))
     (pin "1")
@@
     (property "BoardSide" "B.Cu" (at 617.22 142.24 0) (effects (font (size 1.27 1.27)) (hide yes)))
     (property "BoardAssignment" "P" (at 617.22 142.24 0) (effects (font (size 1.27 1.27)) (hide yes)))
-    (property "KiCadOrientationDeg" "180" (at 617.22 142.24 0) (effects (font (size 1.27 1.27)) (hide yes)))
-    (property "FootprintOriginMm" "244.39,187.46" (at 617.22 142.24 0) (effects (font (size 1.27 1.27)) (hide yes)))
+    (property "KiCadOrientationDeg" "270" (at 617.22 142.24 0) (effects (font (size 1.27 1.27)) (hide yes)))
+    (property "FootprintOriginMm" "104.78,287.81" (at 617.22 142.24 0) (effects (font (size 1.27 1.27)) (hide yes)))
     (property "Sensitive" "" (at 617.22 142.24 0) (effects (font (size 1.27 1.27)) (hide yes)))
     (pin "1")
