File: boards/osc-control/sheets/sample_hold_H2_P.kicad_sch (KiCad schematic)
At the start: 16 parts, among them SW707 B3F-1020, U202 OPA4197IPWR, U208 SN74HC14DR

Commit message: fix(pcb): place complete slew circuits near fixed controls
Parts:
- C207: FootprintOriginMm 267.06,177.84 -> 128.0,288.0; KiCadOrientationDeg 180 -> 90
- C208: FootprintOriginMm 284.06,177.84 -> 139.0,288.0; KiCadOrientationDeg 180 -> 90
- C209: FootprintOriginMm 301.06,177.84 -> 140.25,279.5
- C210: FootprintOriginMm 250.06,181.09 -> 124.75,281.25; KiCadOrientationDeg 180 -> 90
- C211: FootprintOriginMm 267.06,181.09 -> 142.5,288.0; KiCadOrientationDeg 180 -> 90
- C221: FootprintOriginMm 229.14,186.46 -> 112.46000000000001,286.68; KiCadOrientationDeg 180 -> 90
- C222: FootprintOriginMm 210.14,187.21 -> 122.78,286.68; KiCadOrientationDeg 180 -> 90
- R224: FootprintOriginMm 189.64,195.16 -> 128.5,279.25; KiCadOrientationDeg 180 -> 90
- U202: FootprintOriginMm 123.85,179.63 -> 117.62,287.38
Changed lines of the file:
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@@
     (property "BoardAssignment" "P" (at 416.56 50.8 0) (effects (font (size 1.27 1.27)) (hide yes)))
     (property "KiCadOrientationDeg" "180" (at 416.56 50.8 0) (effects (font (size 1.27 1.27)) (hide yes)))
-    (property "FootprintOriginMm" "123.85,179.63" (at 416.56 50.8 0) (effects (font (size 1.27 1.27)) (hide yes)))
+    (property "FootprintOriginMm" "117.62,287.38" (at 416.56 50.8 0) (effects (font (size 1.27 1.27)) (hide yes)))
     (property "Sensitive" "" (at 416.56 50.8 0) (effects (font (size 1.27 1.27)) (hide yes)))
     (pin "1")
@@
     (property "BoardAssignment" "P" (at 477.52 50.8 0) (effects (font (size 1.27 1.27)) (hide yes)))
     (property "KiCadOrientationDeg" "180" (at 477.52 50.8 0) (effects (font (size 1.27 1.27)) (hide yes)))
-    (property "FootprintOriginMm" "123.85,179.63" (at 477.52 50.8 0) (effects (font (size 1.27 1.27)) (hide yes)))
+    (property "FootprintOriginMm" "117.62,287.38" (at 477.52 50.8 0) (effects (font (size 1.27 1.27)) (hide yes)))
     (property "Sensitive" "" (at 477.52 50.8 0) (effects (font (size 1.27 1.27)) (hide yes)))
     (pin "5")
@@
     (property "BoardAssignment" "P" (at 538.48 50.8 0) (effects (font (size 1.27 1.27)) (hide yes)))
     (property "KiCadOrientationDeg" "180" (at 538.48 50.8 0) (effects (font (size 1.27 1.27)) (hide yes)))
-    (property "FootprintOriginMm" "123.85,179.63" (at 538.48 50.8 0) (effects (font (size 1.27 1.27)) (hide yes)))
+    (property "FootprintOriginMm" "117.62,287.38" (at 538.48 50.8 0) (effects (font (size 1.27 1.27)) (hide yes)))
     (property "Sensitive" "" (at 538.48 50.8 0) (effects (font (size 1.27 1.27)) (hide yes)))
     (pin "8")
@@
     (property "BoardAssignment" "P" (at 599.44 50.8 0) (effects (font (size 1.27 1.27)) (hide yes)))
     (property "KiCadOrientationDeg" "180" (at 599.44 50.8 0) (effects (font (size 1.27 1.27)) (hide yes)))
-    (property "FootprintOriginMm" "123.85,179.63" (at 599.44 50.8 0) (effects (font (size 1.27 1.27)) (hide yes)))
+    (property "FootprintOriginMm" "117.62,287.38" (at 599.44 50.8 0) (effects (font (size 1.27 1.27)) (hide yes)))
     (property "Sensitive" "" (at 599.44 50.8 0) (effects (font (size 1.27 1.27)) (hide yes)))
     (pin "12")
@@
     (property "BoardAssignment" "P" (at 660.4 50.8 0) (effects (font (size 1.27 1.27)) (hide yes)))
     (property "KiCadOrientationDeg" "180" (at 660.4 50.8 0) (effects (font (size 1.27 1.27)) (hide yes)))
-    (property "FootprintOriginMm" "123.85,179.63" (at 660.4 50.8 0) (effects (font (size 1.27 1.27)) (hide yes)))
+    (property "FootprintOriginMm" "117.62,287.38" (at 660.4 50.8 0) (effects (font (size 1.27 1.27)) (hide yes)))
     (property "Sensitive" "" (at 660.4 50.8 0) (effects (font (size 1.27 1.27)) (hide yes)))
     (pin "4")
@@
     (property "BoardSide" "B.Cu" (at 660.4 325.12 0) (effects (font (size 1.27 1.27)) (hide yes)))
     (property "BoardAssignment" "P" (at 660.4 325.12 0) (effects (font (size 1.27 1.27)) (hide yes)))
-    (property "KiCadOrientationDeg" "180" (at 660.4 325.12 0) (effects (font (size 1.27 1.27)) (hide yes)))
-    (property "FootprintOriginMm" "189.64,195.16" (at 660.4 325.12 0) (effects (font (size 1.27 1.27)) (hide yes)))
+    (property "KiCadOrientationDeg" "90" (at 660.4 325.12 0) (effects (font (size 1.27 1.27)) (hide yes)))
+    (property "FootprintOriginMm" "128.5,279.25" (at 660.4 325.12 0) (effects (font (size 1.27 1.27)) (hide yes)))
     (property "Sensitive" "" (at 660.4 325.12 0) (effects (font (size 1.27 1.27)) (hide yes)))
     (pin "1")
@@
     (property "BoardSide" "B.Cu" (at 50.8 355.6 0) (effects (font (size 1.27 1.27)) (hide yes)))
     (property "BoardAssignment" "P" (at 50.8 355.6 0) (effects (font (size 1.27 1.27)) (hide yes)))
-    (property "KiCadOrientationDeg" "180" (at 50.8 355.6 0) (effects (font (size 1.27 1.27)) (hide yes)))
-    (property "FootprintOriginMm" "267.06,177.84" (at 50.8 355.6 0) (effects (font (size 1.27 1.27)) (hide yes)))
+    (property "KiCadOrientationDeg" "90" (at 50.8 355.6 0) (effects (font (size 1.27 1.27)) (hide yes)))
+    (property "FootprintOriginMm" "128.0,288.0" (at 50.8 355.6 0) (effects (font (size 1.27 1.27)) (hide yes)))
     (property "Sensitive" "" (at 50.8 355.6 0) (effects (font (size 1.27 1.27)) (hide yes)))
     (pin "1")
@@
     (property "BoardSide" "B.Cu" (at 111.76 355.6 0) (effects (font (size 1.27 1.27)) (hide yes)))
     (property "BoardAssignment" "P" (at 111.76 355.6 0) (effects (font (size 1.27 1.27)) (hide yes)))
-    (property "KiCadOrientationDeg" "180" (at 111.76 355.6 0) (effects (font (size 1.27 1.27)) (hide yes)))
-    (property "FootprintOriginMm" "284.06,177.84" (at 111.76 355.6 0) (effects (font (size 1.27 1.27)) (hide yes)))
+    (property "KiCadOrientationDeg" "90" (at 111.76 355.6 0) (effects (font (size 1.27 1.27)) (hide yes)))
+    (property "FootprintOriginMm" "139.0,288.0" (at 111.76 355.6 0) (effects (font (size 1.27 1.27)) (hide yes)))
     (property "Sensitive" "" (at 111.76 355.6 0) (effects (font (size 1.27 1.27)) (hide yes)))
     (pin "1")
@@
     (property "BoardAssignment" "P" (at 172.72 355.6 0) (effects (font (size 1.27 1.27)) (hide yes)))
     (property "KiCadOrientationDeg" "180" (at 172.72 355.6 0) (effects (font (size 1.27 1.27)) (hide yes)))
-    (property "FootprintOriginMm" "301.06,177.84" (at 172.72 355.6 0) (effects (font (size 1.27 1.27)) (hide yes)))
+    (property "FootprintOriginMm" "140.25,279.5" (at 172.72 355.6 0) (effects (font (size 1.27 1.27)) (hide yes)))
     (property "Sensitive" "" (at 172.72 355.6 0) (effects (font (size 1.27 1.27)) (hide yes)))
     (pin "1")
@@
     (property "BoardSide" "B.Cu" (at 233.68 355.6 0) (effects (font (size 1.27 1.27)) (hide yes)))
     (property "BoardAssignment" "P" (at 233.68 355.6 0) (effects (font (size 1.27 1.27)) (hide yes)))
-    (property "KiCadOrientationDeg" "180" (at 233.68 355.6 0) (effects (font (size 1.27 1.27)) (hide yes)))
-    (property "FootprintOriginMm" "250.06,181.09" (at 233.68 355.6 0) (effects (font (size 1.27 1.27)) (hide yes)))
+    (property "KiCadOrientationDeg" "90" (at 233.68 355.6 0) (effects (font (size 1.27 1.27)) (hide yes)))
+    (property "FootprintOriginMm" "124.75,281.25" (at 233.68 355.6 0) (effects (font (size 1.27 1.27)) (hide yes)))
     (property "Sensitive" "" (at 233.68 355.6 0) (effects (font (size 1.27 1.27)) (hide yes)))
     (pin "1")
@@
     (property "BoardSide" "B.Cu" (at 294.64 355.6 0) (effects (font (size 1.27 1.27)) (hide yes)))
     (property "BoardAssignment" "P" (at 294.64 355.6 0) (effects (font (size 1.27 1.27)) (hide yes)))
-    (property "KiCadOrientationDeg" "180" (at 294.64 355.6 0) (effects (font (size 1.27 1.27)) (hide yes)))
-    (property "FootprintOriginMm" "267.06,181.09" (at 294.64 355.6 0) (effects (font (size 1.27 1.27)) (hide yes)))
+    (property "KiCadOrientationDeg" "90" (at 294.64 355.6 0) (effects (font (size 1.27 1.27)) (hide yes)))
+    (property "FootprintOriginMm" "142.5,288.0" (at 294.64 355.6 0) (effects (font (size 1.27 1.27)) (hide yes)))
     (property "Sensitive" "" (at 294.64 355.6 0) (effects (font (size 1.27 1.27)) (hide yes)))
     (pin "1")
@@
     (property "BoardSide" "B.Cu" (at 233.68 447.04 0) (effects (font (size 1.27 1.27)) (hide yes)))
     (property "BoardAssignment" "P" (at 233.68 447.04 0) (effects (font (size 1.27 1.27)) (hide yes)))
-    (property "KiCadOrientationDeg" "180" (at 233.68 447.04 0) (effects (font (size 1.27 1.27)) (hide yes)))
-    (property "FootprintOriginMm" "229.14,186.46" (at 233.68 447.04 0) (effects (font (size 1.27 1.27)) (hide yes)))
+    (property "KiCadOrientationDeg" "90" (at 233.68 447.04 0) (effects (font (size 1.27 1.27)) (hide yes)))
+    (property "FootprintOriginMm" "112.46000000000001,286.68" (at 233.68 447.04 0) (effects (font (size 1.27 1.27)) (hide yes)))
     (property "Sensitive" "" (at 233.68 447.04 0) (effects (font (size 1.27 1.27)) (hide yes)))
     (pin "1")
@@
     (property "BoardSide" "B.Cu" (at 294.64 447.04 0) (effects (font (size 1.27 1.27)) (hide yes)))
     (property "BoardAssignment" "P" (at 294.64 447.04 0) (effects (font (size 1.27 1.27)) (hide yes)))
-    (property "KiCadOrientationDeg" "180" (at 294.64 447.04 0) (effects (font (size 1.27 1.27)) (hide yes)))
-    (property "FootprintOriginMm" "210.14,187.21" (at 294.64 447.04 0) (effects (font (size 1.27 1.27)) (hide yes)))
+    (property "KiCadOrientationDeg" "90" (at 294.64 447.04 0) (effects (font (size 1.27 1.27)) (hide yes)))
+    (property "FootprintOriginMm" "122.78,286.68" (at 294.64 447.04 0) (effects (font (size 1.27 1.27)) (hide yes)))
     (property "Sensitive" "" (at 294.64 447.04 0) (effects (font (size 1.27 1.27)) (hide yes)))
     (pin "1")

Commit message: Keep control-board bypass groups local and connect their supply loops
Parts:
- C230: FootprintOriginMm 223.64,187.21 -> 248.70999999999998,232.19; KiCadOrientationDeg 180 -> 270
- U208: FootprintOriginMm 260.2,181.45 -> 243.7,227.68; KiCadOrientationDeg 180 -> 0
Changed lines of the file:
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@@
     (property "BoardSide" "B.Cu" (at 50.8 172.72 0) (effects (font (size 1.27 1.27)) (hide yes)))
     (property "BoardAssignment" "P" (at 50.8 172.72 0) (effects (font (size 1.27 1.27)) (hide yes)))
-    (property "KiCadOrientationDeg" "180" (at 50.8 172.72 0) (effects (font (size 1.27 1.27)) (hide yes)))
-    (property "FootprintOriginMm" "260.2,181.45" (at 50.8 172.72 0) (effects (font (size 1.27 1.27)) (hide yes)))
+    (property "KiCadOrientationDeg" "0" (at 50.8 172.72 0) (effects (font (size 1.27 1.27)) (hide yes)))
+    (property "FootprintOriginMm" "243.7,227.68" (at 50.8 172.72 0) (effects (font (size 1.27 1.27)) (hide yes)))
     (property "Sensitive" "" (at 50.8 172.72 0) (effects (font (size 1.27 1.27)) (hide yes)))
     (pin "1")
@@
     (property "BoardSide" "B.Cu" (at 111.76 172.72 0) (effects (font (size 1.27 1.27)) (hide yes)))
     (property "BoardAssignment" "P" (at 111.76 172.72 0) (effects (font (size 1.27 1.27)) (hide yes)))
-    (property "KiCadOrientationDeg" "180" (at 111.76 172.72 0) (effects (font (size 1.27 1.27)) (hide yes)))
-    (property "FootprintOriginMm" "260.2,181.45" (at 111.76 172.72 0) (effects (font (size 1.27 1.27)) (hide yes)))
+    (property "KiCadOrientationDeg" "0" (at 111.76 172.72 0) (effects (font (size 1.27 1.27)) (hide yes)))
+    (property "FootprintOriginMm" "243.7,227.68" (at 111.76 172.72 0) (effects (font (size 1.27 1.27)) (hide yes)))
     (property "Sensitive" "" (at 111.76 172.72 0) (effects (font (size 1.27 1.27)) (hide yes)))
     (pin "3")
@@
     (property "BoardSide" "B.Cu" (at 172.72 172.72 0) (effects (font (size 1.27 1.27)) (hide yes)))
     (property "BoardAssignment" "P" (at 172.72 172.72 0) (effects (font (size 1.27 1.27)) (hide yes)))
-    (property "KiCadOrientationDeg" "180" (at 172.72 172.72 0) (effects (font (size 1.27 1.27)) (hide yes)))
-    (property "FootprintOriginMm" "260.2,181.45" (at 172.72 172.72 0) (effects (font (size 1.27 1.27)) (hide yes)))
+    (property "KiCadOrientationDeg" "0" (at 172.72 172.72 0) (effects (font (size 1.27 1.27)) (hide yes)))
+    (property "FootprintOriginMm" "243.7,227.68" (at 172.72 172.72 0) (effects (font (size 1.27 1.27)) (hide yes)))
     (property "Sensitive" "" (at 172.72 172.72 0) (effects (font (size 1.27 1.27)) (hide yes)))
     (pin "5")
@@
     (property "BoardSide" "B.Cu" (at 233.68 172.72 0) (effects (font (size 1.27 1.27)) (hide yes)))
     (property "BoardAssignment" "P" (at 233.68 172.72 0) (effects (font (size 1.27 1.27)) (hide yes)))
-    (property "KiCadOrientationDeg" "180" (at 233.68 172.72 0) (effects (font (size 1.27 1.27)) (hide yes)))
-    (property "FootprintOriginMm" "260.2,181.45" (at 233.68 172.72 0) (effects (font (size 1.27 1.27)) (hide yes)))
+    (property "KiCadOrientationDeg" "0" (at 233.68 172.72 0) (effects (font (size 1.27 1.27)) (hide yes)))
+    (property "FootprintOriginMm" "243.7,227.68" (at 233.68 172.72 0) (effects (font (size 1.27 1.27)) (hide yes)))
     (property "Sensitive" "" (at 233.68 172.72 0) (effects (font (size 1.27 1.27)) (hide yes)))
     (pin "8")
@@
     (property "BoardSide" "B.Cu" (at 294.64 172.72 0) (effects (font (size 1.27 1.27)) (hide yes)))
     (property "BoardAssignment" "P" (at 294.64 172.72 0) (effects (font (size 1.27 1.27)) (hide yes)))
-    (property "KiCadOrientationDeg" "180" (at 294.64 172.72 0) (effects (font (size 1.27 1.27)) (hide yes)))
-    (property "FootprintOriginMm" "260.2,181.45" (at 294.64 172.72 0) (effects (font (size 1.27 1.27)) (hide yes)))
+    (property "KiCadOrientationDeg" "0" (at 294.64 172.72 0) (effects (font (size 1.27 1.27)) (hide yes)))
+    (property "FootprintOriginMm" "243.7,227.68" (at 294.64 172.72 0) (effects (font (size 1.27 1.27)) (hide yes)))
     (property "Sensitive" "" (at 294.64 172.72 0) (effects (font (size 1.27 1.27)) (hide yes)))
     (pin "10")
@@
     (property "BoardSide" "B.Cu" (at 355.6 172.72 0) (effects (font (size 1.27 1.27)) (hide yes)))
     (property "BoardAssignment" "P" (at 355.6 172.72 0) (effects (font (size 1.27 1.27)) (hide yes)))
-    (property "KiCadOrientationDeg" "180" (at 355.6 172.72 0) (effects (font (size 1.27 1.27)) (hide yes)))
-    (property "FootprintOriginMm" "260.2,181.45" (at 355.6 172.72 0) (effects (font (size 1.27 1.27)) (hide yes)))
+    (property "KiCadOrientationDeg" "0" (at 355.6 172.72 0) (effects (font (size 1.27 1.27)) (hide yes)))
+    (property "FootprintOriginMm" "243.7,227.68" (at 355.6 172.72 0) (effects (font (size 1.27 1.27)) (hide yes)))
     (property "Sensitive" "" (at 355.6 172.72 0) (effects (font (size 1.27 1.27)) (hide yes)))
     (pin "12")
@@
     (property "BoardSide" "B.Cu" (at 416.56 172.72 0) (effects (font (size 1.27 1.27)) (hide yes)))
     (property "BoardAssignment" "P" (at 416.56 172.72 0) (effects (font (size 1.27 1.27)) (hide yes)))
-    (property "KiCadOrientationDeg" "180" (at 416.56 172.72 0) (effects (font (size 1.27 1.27)) (hide yes)))
-    (property "FootprintOriginMm" "260.2,181.45" (at 416.56 172.72 0) (effects (font (size 1.27 1.27)) (hide yes)))
+    (property "KiCadOrientationDeg" "0" (at 416.56 172.72 0) (effects (font (size 1.27 1.27)) (hide yes)))
+    (property "FootprintOriginMm" "243.7,227.68" (at 416.56 172.72 0) (effects (font (size 1.27 1.27)) (hide yes)))
     (property "Sensitive" "" (at 416.56 172.72 0) (effects (font (size 1.27 1.27)) (hide yes)))
     (pin "7")
@@
     (property "BoardSide" "B.Cu" (at 50.8 477.52 0) (effects (font (size 1.27 1.27)) (hide yes)))
     (property "BoardAssignment" "P" (at 50.8 477.52 0) (effects (font (size 1.27 1.27)) (hide yes)))
-    (property "KiCadOrientationDeg" "180" (at 50.8 477.52 0) (effects (font (size 1.27 1.27)) (hide yes)))
-    (property "FootprintOriginMm" "223.64,187.21" (at 50.8 477.52 0) (effects (font (size 1.27 1.27)) (hide yes)))
+    (property "KiCadOrientationDeg" "270" (at 50.8 477.52 0) (effects (font (size 1.27 1.27)) (hide yes)))
+    (property "FootprintOriginMm" "248.70999999999998,232.19" (at 50.8 477.52 0) (effects (font (size 1.27 1.27)) (hide yes)))
     (property "Sensitive" "" (at 50.8 477.52 0) (effects (font (size 1.27 1.27)) (hide yes)))
     (pin "1")
