File: boards/osc-control/sheets/board_interfaces_P-p4.kicad_sch (KiCad schematic)
At the start: 24 parts, among them J900270 BM03B-GHS-TBT(LF)(SN), J900272 BM03B-GHS-TBT(LF)(SN), J900274 BM03B-GHS-TBT(LF)(SN), J900276 BM03B-GHS-TBT(LF)(SN), J900278 BM03B-GHS-TBT(LF)(SN), J900280 BM03B-GHS-TBT(LF)(SN), J900282 BM03B-GHS-TBT(LF)(SN), J900284 BM03B-GHS-TBT(LF)(SN), J900286 BM03B-GHS-TBT(LF)(SN), J900288 BM03B-GHS-TBT(LF)(SN), J900290 BM03B-GHS-TBT(LF)(SN), J900292 BM03B-GHS-TBT(LF)(SN), J900294 BM03B-GHS-TBT(LF)(SN), J900296 BM03B-GHS-TBT(LF)(SN), J900298 BM03B-GHS-TBT(LF)(SN), J900300 BM03B-GHS-TBT(LF)(SN), J900302 BM03B-GHS-TBT(LF)(SN), J900304 BM03B-GHS-TBT(LF)(SN), J900306 BM03B-GHS-TBT(LF)(SN), J900308 BM03B-GHS-TBT(LF)(SN), J900310 BM03B-GHS-TBT(LF)(SN), J900312 BM03B-GHS-TBT(LF)(SN), J900314 BM03B-GHS-TBT(LF)(SN), J900316 BM03B-GHS-TBT(LF)(SN)

Commit message: Reassign paired control connectors and rebuild the routing seed
Parts:
- J900270: FootprintOriginMm 50.45,269.0 -> 152.45,199.0
- J900272: FootprintOriginMm 67.45,269.0 -> 152.45,227.0
- J900274: FootprintOriginMm 84.45,269.0 -> 152.45,255.0
- J900276: FootprintOriginMm 135.45,269.0 -> 50.45,227.0
- J900278: FootprintOriginMm 152.45,269.0 -> 143.95,234.0
- J900280: FootprintOriginMm 169.45,269.0 -> 152.45,241.0
- J900282: FootprintOriginMm 186.45,269.0 -> 169.45,199.0
- J900284: FootprintOriginMm 203.45,269.0 -> 169.45,227.0
- J900286: FootprintOriginMm 220.45,269.0 -> 169.45,255.0
- J900288: FootprintOriginMm 237.45,269.0 -> 169.45,213.0
- J900290: FootprintOriginMm 254.45,269.0 -> 203.45,213.0
- J900292: FootprintOriginMm 16.45,283.0 -> 169.45,241.0
- J900294: FootprintOriginMm 33.45,283.0 -> 16.45,283.0
- J900296: FootprintOriginMm 50.45,283.0 -> 16.45,269.0
- J900298: FootprintOriginMm 67.45,283.0 -> 16.45,255.0
- J900300: FootprintOriginMm 84.45,283.0 -> 16.45,206.0
- J900302: FootprintOriginMm 135.45,283.0 -> 16.45,241.0
- J900304: FootprintOriginMm 152.45,283.0 -> 33.45,227.0
- J900306: FootprintOriginMm 169.45,283.0 -> 16.45,218.5
- J900308: FootprintOriginMm 186.45,283.0 -> 33.45,283.0
- J900310: FootprintOriginMm 203.45,283.0 -> 33.45,269.0
- J900312: FootprintOriginMm 220.45,283.0 -> 33.45,255.0
- J900314: FootprintOriginMm 237.45,283.0 -> 33.45,206.0
- J900316: FootprintOriginMm 254.45,283.0 -> 33.45,241.0
