File: boards/osc-control/sheets/board_interfaces_P-p5.kicad_sch (KiCad schematic)
At the start: 24 parts, among them J900318 BM03B-GHS-TBT(LF)(SN), J900320 BM03B-GHS-TBT(LF)(SN), J900322 BM03B-GHS-TBT(LF)(SN), J900324 BM03B-GHS-TBT(LF)(SN), J900326 BM03B-GHS-TBT(LF)(SN), J900328 BM03B-GHS-TBT(LF)(SN), J900330 BM03B-GHS-TBT(LF)(SN), J900332 BM03B-GHS-TBT(LF)(SN), J900334 BM03B-GHS-TBT(LF)(SN), J900336 BM03B-GHS-TBT(LF)(SN), J900338 BM03B-GHS-TBT(LF)(SN), J900340 BM03B-GHS-TBT(LF)(SN), J900342 BM03B-GHS-TBT(LF)(SN), J900344 BM03B-GHS-TBT(LF)(SN), J900346 BM03B-GHS-TBT(LF)(SN), J900348 BM03B-GHS-TBT(LF)(SN), J900350 BM03B-GHS-TBT(LF)(SN), J900352 BM03B-GHS-TBT(LF)(SN), J900354 BM03B-GHS-TBT(LF)(SN), J900356 BM03B-GHS-TBT(LF)(SN), J900358 BM03B-GHS-TBT(LF)(SN), J900360 BM03B-GHS-TBT(LF)(SN), J900362 BM03B-GHS-TBT(LF)(SN), J900364 BM03B-GHS-TBT(LF)(SN)

Commit message: Reassign paired control connectors and rebuild the routing seed
Parts:
- J900318: FootprintOriginMm 16.45,206.0 -> 16.45,227.0
- J900320: FootprintOriginMm 16.45,218.5 -> 33.45,218.5
- J900322: FootprintOriginMm 33.45,206.0 -> 50.45,283.0
- J900324: FootprintOriginMm 33.45,218.5 -> 50.45,269.0
- J900326: FootprintOriginMm 50.45,206.0 -> 50.45,255.0
- J900328: FootprintOriginMm 50.45,218.5 -> 50.45,206.0
- J900330: FootprintOriginMm 67.45,206.0 -> 50.45,241.0
- J900332: FootprintOriginMm 67.45,218.5 -> 67.45,227.0
- J900334: FootprintOriginMm 84.45,206.0 -> 50.45,218.5
- J900336: FootprintOriginMm 84.45,218.5 -> 67.45,283.0
- J900338: FootprintOriginMm 220.45,192.0 -> 67.45,269.0
- J900340: FootprintOriginMm 220.45,206.0 -> 67.45,255.0
- J900342: FootprintOriginMm 220.45,219.75 -> 67.45,206.0
- J900344: FootprintOriginMm 237.45,192.0 -> 67.45,241.0
- J900346: FootprintOriginMm 237.45,206.0 -> 84.45,269.0
- J900348: FootprintOriginMm 237.45,219.75 -> 67.45,218.5
- J900350: FootprintOriginMm 254.45,192.0 -> 84.45,283.0
- J900352: FootprintOriginMm 254.45,206.0 -> 84.45,241.0
- J900354: FootprintOriginMm 254.45,219.75 -> 84.45,255.0
- J900356: FootprintOriginMm 271.45,192.0 -> 101.45,185.0
- J900358: FootprintOriginMm 271.45,206.0 -> 84.45,227.0
- J900360: FootprintOriginMm 271.45,219.75 -> 84.45,218.5
- J900362: FootprintOriginMm 288.45,192.0 -> 84.45,206.0
- J900364: FootprintOriginMm 288.45,206.0 -> 152.45,269.0
