File: boards/osc-control/sheets/board_interfaces_P-p6.kicad_sch (KiCad schematic)
At the start: 7 parts, among them J900366 BM03B-GHS-TBT(LF)(SN), J900368 BM03B-GHS-TBT(LF)(SN), J900370 BM03B-GHS-TBT(LF)(SN), J900372 BM03B-GHS-TBT(LF)(SN), J900374 BM03B-GHS-TBT(LF)(SN), J900376 BM03B-GHS-TBT(LF)(SN), J900378 BM03B-GHS-TBT(LF)(SN)

Commit message: Reassign paired control connectors and rebuild the routing seed
Parts:
- J900366: FootprintOriginMm 288.45,219.75 -> 186.45,269.0
- J900368: FootprintOriginMm 305.45,192.0 -> 169.45,269.0
- J900370: FootprintOriginMm 305.45,206.0 -> 186.45,283.0
- J900372: FootprintOriginMm 305.45,219.75 -> 135.45,283.0
- J900374: FootprintOriginMm 143.95,234.0 -> 135.45,269.0
- J900376: FootprintOriginMm 160.95,234.0 -> 169.45,283.0
- J900378: FootprintOriginMm 177.95,234.0 -> 152.45,283.0
Changed lines of the file:
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@@
     (property "BoardSide" "B.Cu" (at 35 40 0) (effects (font (size 1.27 1.27)) (hide yes)))
     (property "KiCadOrientationDeg" "90" (at 35 40 0) (effects (font (size 1.27 1.27)) (hide yes)))
-    (property "FootprintOriginMm" "288.45,219.75" (at 35 40 0) (effects (font (size 1.27 1.27)) (hide yes)))
+    (property "FootprintOriginMm" "186.45,269.0" (at 35 40 0) (effects (font (size 1.27 1.27)) (hide yes)))
     (property "Sensitive" "" (at 35 40 0) (effects (font (size 1.27 1.27)) (hide yes)))
     (pin "1")
@@
     (property "BoardSide" "B.Cu" (at 100 40 0) (effects (font (size 1.27 1.27)) (hide yes)))
     (property "KiCadOrientationDeg" "90" (at 100 40 0) (effects (font (size 1.27 1.27)) (hide yes)))
-    (property "FootprintOriginMm" "305.45,192.0" (at 100 40 0) (effects (font (size 1.27 1.27)) (hide yes)))
+    (property "FootprintOriginMm" "169.45,269.0" (at 100 40 0) (effects (font (size 1.27 1.27)) (hide yes)))
     (property "Sensitive" "" (at 100 40 0) (effects (font (size 1.27 1.27)) (hide yes)))
     (pin "1")
@@
     (property "BoardSide" "B.Cu" (at 165 40 0) (effects (font (size 1.27 1.27)) (hide yes)))
     (property "KiCadOrientationDeg" "90" (at 165 40 0) (effects (font (size 1.27 1.27)) (hide yes)))
-    (property "FootprintOriginMm" "305.45,206.0" (at 165 40 0) (effects (font (size 1.27 1.27)) (hide yes)))
+    (property "FootprintOriginMm" "186.45,283.0" (at 165 40 0) (effects (font (size 1.27 1.27)) (hide yes)))
     (property "Sensitive" "" (at 165 40 0) (effects (font (size 1.27 1.27)) (hide yes)))
     (pin "1")
@@
     (property "BoardSide" "B.Cu" (at 35 70 0) (effects (font (size 1.27 1.27)) (hide yes)))
     (property "KiCadOrientationDeg" "90" (at 35 70 0) (effects (font (size 1.27 1.27)) (hide yes)))
-    (property "FootprintOriginMm" "305.45,219.75" (at 35 70 0) (effects (font (size 1.27 1.27)) (hide yes)))
+    (property "FootprintOriginMm" "135.45,283.0" (at 35 70 0) (effects (font (size 1.27 1.27)) (hide yes)))
     (property "Sensitive" "" (at 35 70 0) (effects (font (size 1.27 1.27)) (hide yes)))
     (pin "1")
@@
     (property "BoardSide" "B.Cu" (at 100 70 0) (effects (font (size 1.27 1.27)) (hide yes)))
     (property "KiCadOrientationDeg" "90" (at 100 70 0) (effects (font (size 1.27 1.27)) (hide yes)))
-    (property "FootprintOriginMm" "143.95,234.0" (at 100 70 0) (effects (font (size 1.27 1.27)) (hide yes)))
+    (property "FootprintOriginMm" "135.45,269.0" (at 100 70 0) (effects (font (size 1.27 1.27)) (hide yes)))
     (property "Sensitive" "" (at 100 70 0) (effects (font (size 1.27 1.27)) (hide yes)))
     (pin "1")
@@
     (property "BoardSide" "B.Cu" (at 165 70 0) (effects (font (size 1.27 1.27)) (hide yes)))
     (property "KiCadOrientationDeg" "90" (at 165 70 0) (effects (font (size 1.27 1.27)) (hide yes)))
-    (property "FootprintOriginMm" "160.95,234.0" (at 165 70 0) (effects (font (size 1.27 1.27)) (hide yes)))
+    (property "FootprintOriginMm" "169.45,283.0" (at 165 70 0) (effects (font (size 1.27 1.27)) (hide yes)))
     (property "Sensitive" "" (at 165 70 0) (effects (font (size 1.27 1.27)) (hide yes)))
     (pin "1")
@@
     (property "BoardSide" "B.Cu" (at 35 100 0) (effects (font (size 1.27 1.27)) (hide yes)))
     (property "KiCadOrientationDeg" "90" (at 35 100 0) (effects (font (size 1.27 1.27)) (hide yes)))
-    (property "FootprintOriginMm" "177.95,234.0" (at 35 100 0) (effects (font (size 1.27 1.27)) (hide yes)))
+    (property "FootprintOriginMm" "152.45,283.0" (at 35 100 0) (effects (font (size 1.27 1.27)) (hide yes)))
     (property "Sensitive" "" (at 35 100 0) (effects (font (size 1.27 1.27)) (hide yes)))
     (pin "1")
