File: boards/osc-control/sheets/envelope_E1_P.kicad_sch (KiCad schematic)
At the start: 23 parts, among them SW1301 2MS3T1B1M2QES, SW1302 2MS1T1B1M2QES-5, SW1303 2MS1T1B1M2QES-5, SW1304 B3F-1020, U4111 SN74HC14DR

Commit message: Keep control-board bypass groups local and connect their supply loops
Parts:
- C4156: FootprintOriginMm 312.39,187.46 -> 238.21,181.39000000000001; KiCadOrientationDeg 180 -> 90
- U4111: FootprintOriginMm 277.2,181.45 -> 243.22,185.9
Changed lines of the file:
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@@
     (property "BoardAssignment" "P" (at 1107.44 304.8 0) (effects (font (size 1.27 1.27)) (hide yes)))
     (property "KiCadOrientationDeg" "180" (at 1107.44 304.8 0) (effects (font (size 1.27 1.27)) (hide yes)))
-    (property "FootprintOriginMm" "277.2,181.45" (at 1107.44 304.8 0) (effects (font (size 1.27 1.27)) (hide yes)))
+    (property "FootprintOriginMm" "243.22,185.9" (at 1107.44 304.8 0) (effects (font (size 1.27 1.27)) (hide yes)))
     (property "Sensitive" "" (at 1107.44 304.8 0) (effects (font (size 1.27 1.27)) (hide yes)))
     (pin "1")
@@
     (property "BoardAssignment" "P" (at 40.64 336.55 0) (effects (font (size 1.27 1.27)) (hide yes)))
     (property "KiCadOrientationDeg" "180" (at 40.64 336.55 0) (effects (font (size 1.27 1.27)) (hide yes)))
-    (property "FootprintOriginMm" "277.2,181.45" (at 40.64 336.55 0) (effects (font (size 1.27 1.27)) (hide yes)))
+    (property "FootprintOriginMm" "243.22,185.9" (at 40.64 336.55 0) (effects (font (size 1.27 1.27)) (hide yes)))
     (property "Sensitive" "" (at 40.64 336.55 0) (effects (font (size 1.27 1.27)) (hide yes)))
     (pin "3")
@@
     (property "BoardAssignment" "P" (at 91.44 336.55 0) (effects (font (size 1.27 1.27)) (hide yes)))
     (property "KiCadOrientationDeg" "180" (at 91.44 336.55 0) (effects (font (size 1.27 1.27)) (hide yes)))
-    (property "FootprintOriginMm" "277.2,181.45" (at 91.44 336.55 0) (effects (font (size 1.27 1.27)) (hide yes)))
+    (property "FootprintOriginMm" "243.22,185.9" (at 91.44 336.55 0) (effects (font (size 1.27 1.27)) (hide yes)))
     (property "Sensitive" "" (at 91.44 336.55 0) (effects (font (size 1.27 1.27)) (hide yes)))
     (pin "5")
@@
     (property "BoardAssignment" "P" (at 142.24 336.55 0) (effects (font (size 1.27 1.27)) (hide yes)))
     (property "KiCadOrientationDeg" "180" (at 142.24 336.55 0) (effects (font (size 1.27 1.27)) (hide yes)))
-    (property "FootprintOriginMm" "277.2,181.45" (at 142.24 336.55 0) (effects (font (size 1.27 1.27)) (hide yes)))
+    (property "FootprintOriginMm" "243.22,185.9" (at 142.24 336.55 0) (effects (font (size 1.27 1.27)) (hide yes)))
     (property "Sensitive" "" (at 142.24 336.55 0) (effects (font (size 1.27 1.27)) (hide yes)))
     (pin "8")
@@
     (property "BoardAssignment" "P" (at 193.04 336.55 0) (effects (font (size 1.27 1.27)) (hide yes)))
     (property "KiCadOrientationDeg" "180" (at 193.04 336.55 0) (effects (font (size 1.27 1.27)) (hide yes)))
-    (property "FootprintOriginMm" "277.2,181.45" (at 193.04 336.55 0) (effects (font (size 1.27 1.27)) (hide yes)))
+    (property "FootprintOriginMm" "243.22,185.9" (at 193.04 336.55 0) (effects (font (size 1.27 1.27)) (hide yes)))
     (property "Sensitive" "" (at 193.04 336.55 0) (effects (font (size 1.27 1.27)) (hide yes)))
     (pin "10")
@@
     (property "BoardAssignment" "P" (at 243.84 336.55 0) (effects (font (size 1.27 1.27)) (hide yes)))
     (property "KiCadOrientationDeg" "180" (at 243.84 336.55 0) (effects (font (size 1.27 1.27)) (hide yes)))
-    (property "FootprintOriginMm" "277.2,181.45" (at 243.84 336.55 0) (effects (font (size 1.27 1.27)) (hide yes)))
+    (property "FootprintOriginMm" "243.22,185.9" (at 243.84 336.55 0) (effects (font (size 1.27 1.27)) (hide yes)))
     (property "Sensitive" "" (at 243.84 336.55 0) (effects (font (size 1.27 1.27)) (hide yes)))
     (pin "12")
@@
     (property "BoardAssignment" "P" (at 294.64 336.55 0) (effects (font (size 1.27 1.27)) (hide yes)))
     (property "KiCadOrientationDeg" "180" (at 294.64 336.55 0) (effects (font (size 1.27 1.27)) (hide yes)))
-    (property "FootprintOriginMm" "277.2,181.45" (at 294.64 336.55 0) (effects (font (size 1.27 1.27)) (hide yes)))
+    (property "FootprintOriginMm" "243.22,185.9" (at 294.64 336.55 0) (effects (font (size 1.27 1.27)) (hide yes)))
     (property "Sensitive" "" (at 294.64 336.55 0) (effects (font (size 1.27 1.27)) (hide yes)))
     (pin "7")
@@
     (property "BoardSide" "B.Cu" (at 701.04 685.8 0) (effects (font (size 1.27 1.27)) (hide yes)))
     (property "BoardAssignment" "P" (at 701.04 685.8 0) (effects (font (size 1.27 1.27)) (hide yes)))
-    (property "KiCadOrientationDeg" "180" (at 701.04 685.8 0) (effects (font (size 1.27 1.27)) (hide yes)))
-    (property "FootprintOriginMm" "312.39,187.46" (at 701.04 685.8 0) (effects (font (size 1.27 1.27)) (hide yes)))
+    (property "KiCadOrientationDeg" "90" (at 701.04 685.8 0) (effects (font (size 1.27 1.27)) (hide yes)))
+    (property "FootprintOriginMm" "238.21,181.39000000000001" (at 701.04 685.8 0) (effects (font (size 1.27 1.27)) (hide yes)))
     (property "Sensitive" "" (at 701.04 685.8 0) (effects (font (size 1.27 1.27)) (hide yes)))
     (pin "1")

Commit message: Localize envelope debounce networks and continue control routing
Parts:
- C4103: FootprintOriginMm 274.64,187.46 -> 245.0,179.25
- C4104: FootprintOriginMm 278.39,187.46 -> 242.0,178.5; KiCadOrientationDeg 180 -> 90
- C4105: FootprintOriginMm 291.64,187.46 -> 247.0,193.0; KiCadOrientationDeg 180 -> 270
- C4106: FootprintOriginMm 295.39,187.46 -> 240.5,193.0; KiCadOrientationDeg 180 -> 270
- C4107: FootprintOriginMm 308.64,187.46 -> 235.0,182.5
- R4122: FootprintOriginMm 25.89,195.41 -> 253.0,177.5
- R4123: FootprintOriginMm 29.64,195.41 -> 249.0,177.5
- R4124: FootprintOriginMm 33.39,195.41 -> 234.5,177.5; KiCadOrientationDeg 180 -> 0
- R4125: FootprintOriginMm 37.14,195.41 -> 238.5,177.5; KiCadOrientationDeg 180 -> 0
- R4126: FootprintOriginMm 40.89,195.41 -> 243.0,197.0; KiCadOrientationDeg 180 -> 90
- R4127: FootprintOriginMm 44.64,195.41 -> 246.0,196.0; KiCadOrientationDeg 180 -> 0
- R4128: FootprintOriginMm 48.39,195.41 -> 241.5,200.0
- R4129: FootprintOriginMm 52.14,195.41 -> 240.5,197.0; KiCadOrientationDeg 180 -> 90
- R4130: FootprintOriginMm 55.89,195.41 -> 232.0,180.5; KiCadOrientationDeg 180 -> 90
- R4131: FootprintOriginMm 59.64,195.41 -> 235.0,180.0; KiCadOrientationDeg 180 -> 0
