File: boards/osc-control/sheets/envelope_E3_P.kicad_sch (KiCad schematic)
At the start: 23 parts, among them SW1501 2MS3T1B1M2QES, SW1502 2MS1T1B1M2QES-5, SW1503 2MS1T1B1M2QES-5, SW1504 B3F-1020, U4311 SN74HC14DR

Commit message: Keep control-board bypass groups local and connect their supply loops
Parts:
- C4356: FootprintOriginMm 155.89,190.21 -> 282.71,232.19; KiCadOrientationDeg 180 -> 270
- U4311: FootprintOriginMm 311.2,181.45 -> 277.7,227.68; KiCadOrientationDeg 180 -> 0
Changed lines of the file:
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@@
     (property "BoardSide" "B.Cu" (at 1107.44 304.8 0) (effects (font (size 1.27 1.27)) (hide yes)))
     (property "BoardAssignment" "P" (at 1107.44 304.8 0) (effects (font (size 1.27 1.27)) (hide yes)))
-    (property "KiCadOrientationDeg" "180" (at 1107.44 304.8 0) (effects (font (size 1.27 1.27)) (hide yes)))
-    (property "FootprintOriginMm" "311.2,181.45" (at 1107.44 304.8 0) (effects (font (size 1.27 1.27)) (hide yes)))
+    (property "KiCadOrientationDeg" "0" (at 1107.44 304.8 0) (effects (font (size 1.27 1.27)) (hide yes)))
+    (property "FootprintOriginMm" "277.7,227.68" (at 1107.44 304.8 0) (effects (font (size 1.27 1.27)) (hide yes)))
     (property "Sensitive" "" (at 1107.44 304.8 0) (effects (font (size 1.27 1.27)) (hide yes)))
     (pin "1")
@@
     (property "BoardSide" "B.Cu" (at 40.64 336.55 0) (effects (font (size 1.27 1.27)) (hide yes)))
     (property "BoardAssignment" "P" (at 40.64 336.55 0) (effects (font (size 1.27 1.27)) (hide yes)))
-    (property "KiCadOrientationDeg" "180" (at 40.64 336.55 0) (effects (font (size 1.27 1.27)) (hide yes)))
-    (property "FootprintOriginMm" "311.2,181.45" (at 40.64 336.55 0) (effects (font (size 1.27 1.27)) (hide yes)))
+    (property "KiCadOrientationDeg" "0" (at 40.64 336.55 0) (effects (font (size 1.27 1.27)) (hide yes)))
+    (property "FootprintOriginMm" "277.7,227.68" (at 40.64 336.55 0) (effects (font (size 1.27 1.27)) (hide yes)))
     (property "Sensitive" "" (at 40.64 336.55 0) (effects (font (size 1.27 1.27)) (hide yes)))
     (pin "3")
@@
     (property "BoardSide" "B.Cu" (at 91.44 336.55 0) (effects (font (size 1.27 1.27)) (hide yes)))
     (property "BoardAssignment" "P" (at 91.44 336.55 0) (effects (font (size 1.27 1.27)) (hide yes)))
-    (property "KiCadOrientationDeg" "180" (at 91.44 336.55 0) (effects (font (size 1.27 1.27)) (hide yes)))
-    (property "FootprintOriginMm" "311.2,181.45" (at 91.44 336.55 0) (effects (font (size 1.27 1.27)) (hide yes)))
+    (property "KiCadOrientationDeg" "0" (at 91.44 336.55 0) (effects (font (size 1.27 1.27)) (hide yes)))
+    (property "FootprintOriginMm" "277.7,227.68" (at 91.44 336.55 0) (effects (font (size 1.27 1.27)) (hide yes)))
     (property "Sensitive" "" (at 91.44 336.55 0) (effects (font (size 1.27 1.27)) (hide yes)))
     (pin "5")
@@
     (property "BoardSide" "B.Cu" (at 142.24 336.55 0) (effects (font (size 1.27 1.27)) (hide yes)))
     (property "BoardAssignment" "P" (at 142.24 336.55 0) (effects (font (size 1.27 1.27)) (hide yes)))
-    (property "KiCadOrientationDeg" "180" (at 142.24 336.55 0) (effects (font (size 1.27 1.27)) (hide yes)))
-    (property "FootprintOriginMm" "311.2,181.45" (at 142.24 336.55 0) (effects (font (size 1.27 1.27)) (hide yes)))
+    (property "KiCadOrientationDeg" "0" (at 142.24 336.55 0) (effects (font (size 1.27 1.27)) (hide yes)))
+    (property "FootprintOriginMm" "277.7,227.68" (at 142.24 336.55 0) (effects (font (size 1.27 1.27)) (hide yes)))
     (property "Sensitive" "" (at 142.24 336.55 0) (effects (font (size 1.27 1.27)) (hide yes)))
     (pin "8")
@@
     (property "BoardSide" "B.Cu" (at 193.04 336.55 0) (effects (font (size 1.27 1.27)) (hide yes)))
     (property "BoardAssignment" "P" (at 193.04 336.55 0) (effects (font (size 1.27 1.27)) (hide yes)))
-    (property "KiCadOrientationDeg" "180" (at 193.04 336.55 0) (effects (font (size 1.27 1.27)) (hide yes)))
-    (property "FootprintOriginMm" "311.2,181.45" (at 193.04 336.55 0) (effects (font (size 1.27 1.27)) (hide yes)))
+    (property "KiCadOrientationDeg" "0" (at 193.04 336.55 0) (effects (font (size 1.27 1.27)) (hide yes)))
+    (property "FootprintOriginMm" "277.7,227.68" (at 193.04 336.55 0) (effects (font (size 1.27 1.27)) (hide yes)))
     (property "Sensitive" "" (at 193.04 336.55 0) (effects (font (size 1.27 1.27)) (hide yes)))
     (pin "10")
@@
     (property "BoardSide" "B.Cu" (at 243.84 336.55 0) (effects (font (size 1.27 1.27)) (hide yes)))
     (property "BoardAssignment" "P" (at 243.84 336.55 0) (effects (font (size 1.27 1.27)) (hide yes)))
-    (property "KiCadOrientationDeg" "180" (at 243.84 336.55 0) (effects (font (size 1.27 1.27)) (hide yes)))
-    (property "FootprintOriginMm" "311.2,181.45" (at 243.84 336.55 0) (effects (font (size 1.27 1.27)) (hide yes)))
+    (property "KiCadOrientationDeg" "0" (at 243.84 336.55 0) (effects (font (size 1.27 1.27)) (hide yes)))
+    (property "FootprintOriginMm" "277.7,227.68" (at 243.84 336.55 0) (effects (font (size 1.27 1.27)) (hide yes)))
     (property "Sensitive" "" (at 243.84 336.55 0) (effects (font (size 1.27 1.27)) (hide yes)))
     (pin "12")
@@
     (property "BoardSide" "B.Cu" (at 294.64 336.55 0) (effects (font (size 1.27 1.27)) (hide yes)))
     (property "BoardAssignment" "P" (at 294.64 336.55 0) (effects (font (size 1.27 1.27)) (hide yes)))
-    (property "KiCadOrientationDeg" "180" (at 294.64 336.55 0) (effects (font (size 1.27 1.27)) (hide yes)))
-    (property "FootprintOriginMm" "311.2,181.45" (at 294.64 336.55 0) (effects (font (size 1.27 1.27)) (hide yes)))
+    (property "KiCadOrientationDeg" "0" (at 294.64 336.55 0) (effects (font (size 1.27 1.27)) (hide yes)))
+    (property "FootprintOriginMm" "277.7,227.68" (at 294.64 336.55 0) (effects (font (size 1.27 1.27)) (hide yes)))
     (property "Sensitive" "" (at 294.64 336.55 0) (effects (font (size 1.27 1.27)) (hide yes)))
     (pin "7")
@@
     (property "BoardSide" "B.Cu" (at 701.04 685.8 0) (effects (font (size 1.27 1.27)) (hide yes)))
     (property "BoardAssignment" "P" (at 701.04 685.8 0) (effects (font (size 1.27 1.27)) (hide yes)))
-    (property "KiCadOrientationDeg" "180" (at 701.04 685.8 0) (effects (font (size 1.27 1.27)) (hide yes)))
-    (property "FootprintOriginMm" "155.89,190.21" (at 701.04 685.8 0) (effects (font (size 1.27 1.27)) (hide yes)))
+    (property "KiCadOrientationDeg" "270" (at 701.04 685.8 0) (effects (font (size 1.27 1.27)) (hide yes)))
+    (property "FootprintOriginMm" "282.71,232.19" (at 701.04 685.8 0) (effects (font (size 1.27 1.27)) (hide yes)))
     (property "Sensitive" "" (at 701.04 685.8 0) (effects (font (size 1.27 1.27)) (hide yes)))
     (pin "1")

Commit message: Localize envelope debounce networks and continue control routing
Parts:
- C4303: FootprintOriginMm 227.39,188.96 -> 274.0,234.25
- C4304: FootprintOriginMm 206.89,189.71 -> 271.5,227.0
- C4305: FootprintOriginMm 210.64,189.71 -> 275.0,220.5; KiCadOrientationDeg 180 -> 90
- C4306: FootprintOriginMm 308.64,189.96 -> 281.0,220.5; KiCadOrientationDeg 180 -> 90
- C4307: FootprintOriginMm 312.39,189.96 -> 281.0,236.0; KiCadOrientationDeg 180 -> 270
- R4322: FootprintOriginMm 227.39,195.91 -> 266.0,235.5; KiCadOrientationDeg 180 -> 0
- R4323: FootprintOriginMm 240.64,195.91 -> 270.0,234.5; KiCadOrientationDeg 180 -> 0
- R4324: FootprintOriginMm 244.39,195.91 -> 269.5,232.0
- R4325: FootprintOriginMm 257.64,195.91 -> 269.5,229.5; KiCadOrientationDeg 180 -> 0
- R4326: FootprintOriginMm 261.39,195.91 -> 278.5,216.5; KiCadOrientationDeg 180 -> 270
- R4327: FootprintOriginMm 274.64,195.91 -> 275.5,217.5
- R4328: FootprintOriginMm 278.39,195.91 -> 280.0,213.5; KiCadOrientationDeg 180 -> 0
- R4329: FootprintOriginMm 291.64,195.91 -> 281.0,216.5; KiCadOrientationDeg 180 -> 270
- R4330: FootprintOriginMm 295.39,195.91 -> 274.5,237.25; KiCadOrientationDeg 180 -> 270
- R4331: FootprintOriginMm 210.14,197.16 -> 277.5,238.0; KiCadOrientationDeg 180 -> 0
