File: boards/osc-control/sheets/envelope_E5_P.kicad_sch (KiCad schematic)
At the start: 23 parts, among them SW1701 2MS3T1B1M2QES, SW1702 2MS1T1B1M2QES-5, SW1703 2MS1T1B1M2QES-5, SW1704 B3F-1020, U4511 SN74HC14DR

Commit message: Keep control-board bypass groups local and connect their supply loops
Parts:
- C4556: FootprintOriginMm 172.89,192.71 -> 256.21000000000004,181.39000000000001; KiCadOrientationDeg 180 -> 90
- U4511: FootprintOriginMm 123.95,191.7 -> 261.22,185.9
Changed lines of the file:
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@@
     (property "BoardAssignment" "P" (at 1107.44 304.8 0) (effects (font (size 1.27 1.27)) (hide yes)))
     (property "KiCadOrientationDeg" "180" (at 1107.44 304.8 0) (effects (font (size 1.27 1.27)) (hide yes)))
-    (property "FootprintOriginMm" "123.95,191.7" (at 1107.44 304.8 0) (effects (font (size 1.27 1.27)) (hide yes)))
+    (property "FootprintOriginMm" "261.22,185.9" (at 1107.44 304.8 0) (effects (font (size 1.27 1.27)) (hide yes)))
     (property "Sensitive" "" (at 1107.44 304.8 0) (effects (font (size 1.27 1.27)) (hide yes)))
     (pin "1")
@@
     (property "BoardAssignment" "P" (at 40.64 336.55 0) (effects (font (size 1.27 1.27)) (hide yes)))
     (property "KiCadOrientationDeg" "180" (at 40.64 336.55 0) (effects (font (size 1.27 1.27)) (hide yes)))
-    (property "FootprintOriginMm" "123.95,191.7" (at 40.64 336.55 0) (effects (font (size 1.27 1.27)) (hide yes)))
+    (property "FootprintOriginMm" "261.22,185.9" (at 40.64 336.55 0) (effects (font (size 1.27 1.27)) (hide yes)))
     (property "Sensitive" "" (at 40.64 336.55 0) (effects (font (size 1.27 1.27)) (hide yes)))
     (pin "3")
@@
     (property "BoardAssignment" "P" (at 91.44 336.55 0) (effects (font (size 1.27 1.27)) (hide yes)))
     (property "KiCadOrientationDeg" "180" (at 91.44 336.55 0) (effects (font (size 1.27 1.27)) (hide yes)))
-    (property "FootprintOriginMm" "123.95,191.7" (at 91.44 336.55 0) (effects (font (size 1.27 1.27)) (hide yes)))
+    (property "FootprintOriginMm" "261.22,185.9" (at 91.44 336.55 0) (effects (font (size 1.27 1.27)) (hide yes)))
     (property "Sensitive" "" (at 91.44 336.55 0) (effects (font (size 1.27 1.27)) (hide yes)))
     (pin "5")
@@
     (property "BoardAssignment" "P" (at 142.24 336.55 0) (effects (font (size 1.27 1.27)) (hide yes)))
     (property "KiCadOrientationDeg" "180" (at 142.24 336.55 0) (effects (font (size 1.27 1.27)) (hide yes)))
-    (property "FootprintOriginMm" "123.95,191.7" (at 142.24 336.55 0) (effects (font (size 1.27 1.27)) (hide yes)))
+    (property "FootprintOriginMm" "261.22,185.9" (at 142.24 336.55 0) (effects (font (size 1.27 1.27)) (hide yes)))
     (property "Sensitive" "" (at 142.24 336.55 0) (effects (font (size 1.27 1.27)) (hide yes)))
     (pin "8")
@@
     (property "BoardAssignment" "P" (at 193.04 336.55 0) (effects (font (size 1.27 1.27)) (hide yes)))
     (property "KiCadOrientationDeg" "180" (at 193.04 336.55 0) (effects (font (size 1.27 1.27)) (hide yes)))
-    (property "FootprintOriginMm" "123.95,191.7" (at 193.04 336.55 0) (effects (font (size 1.27 1.27)) (hide yes)))
+    (property "FootprintOriginMm" "261.22,185.9" (at 193.04 336.55 0) (effects (font (size 1.27 1.27)) (hide yes)))
     (property "Sensitive" "" (at 193.04 336.55 0) (effects (font (size 1.27 1.27)) (hide yes)))
     (pin "10")
@@
     (property "BoardAssignment" "P" (at 243.84 336.55 0) (effects (font (size 1.27 1.27)) (hide yes)))
     (property "KiCadOrientationDeg" "180" (at 243.84 336.55 0) (effects (font (size 1.27 1.27)) (hide yes)))
-    (property "FootprintOriginMm" "123.95,191.7" (at 243.84 336.55 0) (effects (font (size 1.27 1.27)) (hide yes)))
+    (property "FootprintOriginMm" "261.22,185.9" (at 243.84 336.55 0) (effects (font (size 1.27 1.27)) (hide yes)))
     (property "Sensitive" "" (at 243.84 336.55 0) (effects (font (size 1.27 1.27)) (hide yes)))
     (pin "12")
@@
     (property "BoardAssignment" "P" (at 294.64 336.55 0) (effects (font (size 1.27 1.27)) (hide yes)))
     (property "KiCadOrientationDeg" "180" (at 294.64 336.55 0) (effects (font (size 1.27 1.27)) (hide yes)))
-    (property "FootprintOriginMm" "123.95,191.7" (at 294.64 336.55 0) (effects (font (size 1.27 1.27)) (hide yes)))
+    (property "FootprintOriginMm" "261.22,185.9" (at 294.64 336.55 0) (effects (font (size 1.27 1.27)) (hide yes)))
     (property "Sensitive" "" (at 294.64 336.55 0) (effects (font (size 1.27 1.27)) (hide yes)))
     (pin "7")
@@
     (property "BoardSide" "B.Cu" (at 701.04 685.8 0) (effects (font (size 1.27 1.27)) (hide yes)))
     (property "BoardAssignment" "P" (at 701.04 685.8 0) (effects (font (size 1.27 1.27)) (hide yes)))
-    (property "KiCadOrientationDeg" "180" (at 701.04 685.8 0) (effects (font (size 1.27 1.27)) (hide yes)))
-    (property "FootprintOriginMm" "172.89,192.71" (at 701.04 685.8 0) (effects (font (size 1.27 1.27)) (hide yes)))
+    (property "KiCadOrientationDeg" "90" (at 701.04 685.8 0) (effects (font (size 1.27 1.27)) (hide yes)))
+    (property "FootprintOriginMm" "256.21000000000004,181.39000000000001" (at 701.04 685.8 0) (effects (font (size 1.27 1.27)) (hide yes)))
     (property "Sensitive" "" (at 701.04 685.8 0) (effects (font (size 1.27 1.27)) (hide yes)))
     (pin "1")

Commit message: Localize envelope debounce networks and continue control routing
Parts:
- C4503: FootprintOriginMm 210.64,192.21 -> 263.0,179.25
- C4504: FootprintOriginMm 308.64,192.46 -> 267.5,182.5; KiCadOrientationDeg 180 -> 0
- C4505: FootprintOriginMm 312.39,192.46 -> 264.0,193.0; KiCadOrientationDeg 180 -> 270
- C4506: FootprintOriginMm 155.89,192.71 -> 258.0,193.0; KiCadOrientationDeg 180 -> 270
- C4507: FootprintOriginMm 159.64,192.71 -> 253.0,182.5
- R4522: FootprintOriginMm 88.14,197.66 -> 268.5,178.5; KiCadOrientationDeg 180 -> 90
- R4523: FootprintOriginMm 224.14,198.16 -> 266.0,178.5; KiCadOrientationDeg 180 -> 270
- R4524: FootprintOriginMm 227.89,198.16 -> 274.5,183.0; KiCadOrientationDeg 180 -> 90
- R4525: FootprintOriginMm 241.14,198.16 -> 271.5,182.5
- R4526: FootprintOriginMm 244.89,198.16 -> 260.0,197.0; KiCadOrientationDeg 180 -> 90
- R4527: FootprintOriginMm 258.14,198.16 -> 263.0,196.0; KiCadOrientationDeg 180 -> 0
- R4528: FootprintOriginMm 261.89,198.16 -> 258.5,200.0
- R4529: FootprintOriginMm 275.14,198.16 -> 257.5,197.0; KiCadOrientationDeg 180 -> 90
- R4530: FootprintOriginMm 278.89,198.16 -> 250.0,180.5; KiCadOrientationDeg 180 -> 90
- R4531: FootprintOriginMm 292.14,198.16 -> 253.0,180.0; KiCadOrientationDeg 180 -> 0
