File: boards/osc-control/sheets/envelope_E6_P.kicad_sch (KiCad schematic)
At the start: 23 parts, among them SW1801 2MS3T1B1M2QES, SW1802 2MS1T1B1M2QES-5, SW1803 2MS1T1B1M2QES-5, SW1804 B3F-1020, U4611 SN74HC14DR

Commit message: Keep control-board bypass groups local and connect their supply loops
Parts:
- C4656: FootprintOriginMm 308.64,194.96 -> 300.71,279.94; KiCadOrientationDeg 180 -> 270
- U4611: FootprintOriginMm 140.95,191.7 -> 295.7,275.43; KiCadOrientationDeg 180 -> 0
Changed lines of the file:
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@@
     (property "BoardSide" "B.Cu" (at 1107.44 304.8 0) (effects (font (size 1.27 1.27)) (hide yes)))
     (property "BoardAssignment" "P" (at 1107.44 304.8 0) (effects (font (size 1.27 1.27)) (hide yes)))
-    (property "KiCadOrientationDeg" "180" (at 1107.44 304.8 0) (effects (font (size 1.27 1.27)) (hide yes)))
-    (property "FootprintOriginMm" "140.95,191.7" (at 1107.44 304.8 0) (effects (font (size 1.27 1.27)) (hide yes)))
+    (property "KiCadOrientationDeg" "0" (at 1107.44 304.8 0) (effects (font (size 1.27 1.27)) (hide yes)))
+    (property "FootprintOriginMm" "295.7,275.43" (at 1107.44 304.8 0) (effects (font (size 1.27 1.27)) (hide yes)))
     (property "Sensitive" "" (at 1107.44 304.8 0) (effects (font (size 1.27 1.27)) (hide yes)))
     (pin "1")
@@
     (property "BoardSide" "B.Cu" (at 40.64 336.55 0) (effects (font (size 1.27 1.27)) (hide yes)))
     (property "BoardAssignment" "P" (at 40.64 336.55 0) (effects (font (size 1.27 1.27)) (hide yes)))
-    (property "KiCadOrientationDeg" "180" (at 40.64 336.55 0) (effects (font (size 1.27 1.27)) (hide yes)))
-    (property "FootprintOriginMm" "140.95,191.7" (at 40.64 336.55 0) (effects (font (size 1.27 1.27)) (hide yes)))
+    (property "KiCadOrientationDeg" "0" (at 40.64 336.55 0) (effects (font (size 1.27 1.27)) (hide yes)))
+    (property "FootprintOriginMm" "295.7,275.43" (at 40.64 336.55 0) (effects (font (size 1.27 1.27)) (hide yes)))
     (property "Sensitive" "" (at 40.64 336.55 0) (effects (font (size 1.27 1.27)) (hide yes)))
     (pin "3")
@@
     (property "BoardSide" "B.Cu" (at 91.44 336.55 0) (effects (font (size 1.27 1.27)) (hide yes)))
     (property "BoardAssignment" "P" (at 91.44 336.55 0) (effects (font (size 1.27 1.27)) (hide yes)))
-    (property "KiCadOrientationDeg" "180" (at 91.44 336.55 0) (effects (font (size 1.27 1.27)) (hide yes)))
-    (property "FootprintOriginMm" "140.95,191.7" (at 91.44 336.55 0) (effects (font (size 1.27 1.27)) (hide yes)))
+    (property "KiCadOrientationDeg" "0" (at 91.44 336.55 0) (effects (font (size 1.27 1.27)) (hide yes)))
+    (property "FootprintOriginMm" "295.7,275.43" (at 91.44 336.55 0) (effects (font (size 1.27 1.27)) (hide yes)))
     (property "Sensitive" "" (at 91.44 336.55 0) (effects (font (size 1.27 1.27)) (hide yes)))
     (pin "5")
@@
     (property "BoardSide" "B.Cu" (at 142.24 336.55 0) (effects (font (size 1.27 1.27)) (hide yes)))
     (property "BoardAssignment" "P" (at 142.24 336.55 0) (effects (font (size 1.27 1.27)) (hide yes)))
-    (property "KiCadOrientationDeg" "180" (at 142.24 336.55 0) (effects (font (size 1.27 1.27)) (hide yes)))
-    (property "FootprintOriginMm" "140.95,191.7" (at 142.24 336.55 0) (effects (font (size 1.27 1.27)) (hide yes)))
+    (property "KiCadOrientationDeg" "0" (at 142.24 336.55 0) (effects (font (size 1.27 1.27)) (hide yes)))
+    (property "FootprintOriginMm" "295.7,275.43" (at 142.24 336.55 0) (effects (font (size 1.27 1.27)) (hide yes)))
     (property "Sensitive" "" (at 142.24 336.55 0) (effects (font (size 1.27 1.27)) (hide yes)))
     (pin "8")
@@
     (property "BoardSide" "B.Cu" (at 193.04 336.55 0) (effects (font (size 1.27 1.27)) (hide yes)))
     (property "BoardAssignment" "P" (at 193.04 336.55 0) (effects (font (size 1.27 1.27)) (hide yes)))
-    (property "KiCadOrientationDeg" "180" (at 193.04 336.55 0) (effects (font (size 1.27 1.27)) (hide yes)))
-    (property "FootprintOriginMm" "140.95,191.7" (at 193.04 336.55 0) (effects (font (size 1.27 1.27)) (hide yes)))
+    (property "KiCadOrientationDeg" "0" (at 193.04 336.55 0) (effects (font (size 1.27 1.27)) (hide yes)))
+    (property "FootprintOriginMm" "295.7,275.43" (at 193.04 336.55 0) (effects (font (size 1.27 1.27)) (hide yes)))
     (property "Sensitive" "" (at 193.04 336.55 0) (effects (font (size 1.27 1.27)) (hide yes)))
     (pin "10")
@@
     (property "BoardSide" "B.Cu" (at 243.84 336.55 0) (effects (font (size 1.27 1.27)) (hide yes)))
     (property "BoardAssignment" "P" (at 243.84 336.55 0) (effects (font (size 1.27 1.27)) (hide yes)))
-    (property "KiCadOrientationDeg" "180" (at 243.84 336.55 0) (effects (font (size 1.27 1.27)) (hide yes)))
-    (property "FootprintOriginMm" "140.95,191.7" (at 243.84 336.55 0) (effects (font (size 1.27 1.27)) (hide yes)))
+    (property "KiCadOrientationDeg" "0" (at 243.84 336.55 0) (effects (font (size 1.27 1.27)) (hide yes)))
+    (property "FootprintOriginMm" "295.7,275.43" (at 243.84 336.55 0) (effects (font (size 1.27 1.27)) (hide yes)))
     (property "Sensitive" "" (at 243.84 336.55 0) (effects (font (size 1.27 1.27)) (hide yes)))
     (pin "12")
@@
     (property "BoardSide" "B.Cu" (at 294.64 336.55 0) (effects (font (size 1.27 1.27)) (hide yes)))
     (property "BoardAssignment" "P" (at 294.64 336.55 0) (effects (font (size 1.27 1.27)) (hide yes)))
-    (property "KiCadOrientationDeg" "180" (at 294.64 336.55 0) (effects (font (size 1.27 1.27)) (hide yes)))
-    (property "FootprintOriginMm" "140.95,191.7" (at 294.64 336.55 0) (effects (font (size 1.27 1.27)) (hide yes)))
+    (property "KiCadOrientationDeg" "0" (at 294.64 336.55 0) (effects (font (size 1.27 1.27)) (hide yes)))
+    (property "FootprintOriginMm" "295.7,275.43" (at 294.64 336.55 0) (effects (font (size 1.27 1.27)) (hide yes)))
     (property "Sensitive" "" (at 294.64 336.55 0) (effects (font (size 1.27 1.27)) (hide yes)))
     (pin "7")
@@
     (property "BoardSide" "B.Cu" (at 701.04 685.8 0) (effects (font (size 1.27 1.27)) (hide yes)))
     (property "BoardAssignment" "P" (at 701.04 685.8 0) (effects (font (size 1.27 1.27)) (hide yes)))
-    (property "KiCadOrientationDeg" "180" (at 701.04 685.8 0) (effects (font (size 1.27 1.27)) (hide yes)))
-    (property "FootprintOriginMm" "308.64,194.96" (at 701.04 685.8 0) (effects (font (size 1.27 1.27)) (hide yes)))
+    (property "KiCadOrientationDeg" "270" (at 701.04 685.8 0) (effects (font (size 1.27 1.27)) (hide yes)))
+    (property "FootprintOriginMm" "300.71,279.94" (at 701.04 685.8 0) (effects (font (size 1.27 1.27)) (hide yes)))
     (property "Sensitive" "" (at 701.04 685.8 0) (effects (font (size 1.27 1.27)) (hide yes)))
     (pin "1")

Commit message: Localize envelope debounce networks and continue control routing
Parts:
- C4603: FootprintOriginMm 176.64,192.71 -> 290.5,279.5; KiCadOrientationDeg 180 -> 270
- C4604: FootprintOriginMm 189.89,192.71 -> 290.5,273.0; KiCadOrientationDeg 180 -> 90
- C4605: FootprintOriginMm 193.64,192.71 -> 294.5,268.5; KiCadOrientationDeg 180 -> 90
- C4606: FootprintOriginMm 206.64,194.71 -> 301.5,273.0; KiCadOrientationDeg 180 -> 0
- C4607: FootprintOriginMm 210.39,194.71 -> 304.0,278.5; KiCadOrientationDeg 180 -> 0
- R4622: FootprintOriginMm 295.89,198.16 -> 288.5,282.5
- R4623: FootprintOriginMm 3.1399999999999997,199.41 -> 288.0,279.5; KiCadOrientationDeg 180 -> 90
- R4624: FootprintOriginMm 210.14,199.41 -> 288.5,270.0
- R4625: FootprintOriginMm 312.89,199.41 -> 288.0,273.0; KiCadOrientationDeg 180 -> 270
- R4626: FootprintOriginMm 309.14,199.66 -> 289.5,265.5; KiCadOrientationDeg 180 -> 90
- R4627: FootprintOriginMm 6.89,199.91 -> 292.0,265.5; KiCadOrientationDeg 180 -> 270
- R4628: FootprintOriginMm 20.14,199.91 -> 304.5,271.0; KiCadOrientationDeg 180 -> 90
- R4629: FootprintOriginMm 23.89,199.91 -> 301.5,270.5
- R4630: FootprintOriginMm 37.14,199.91 -> 307.0,279.5; KiCadOrientationDeg 180 -> 270
- R4631: FootprintOriginMm 40.89,199.91 -> 304.0,281.0
