File: boards/osc-control/osc-control-routed-draft.kicad_pcb (KiCad board)
At the start: 4 copper layers, 316 x 116 mm, 454 parts, among them J900052 BM03B-GHS-TBT(LF)(SN), J900054 BM03B-GHS-TBT(LF)(SN), J900056 BM03B-GHS-TBT(LF)(SN), J900058 BM03B-GHS-TBT(LF)(SN), J900134 BM03B-GHS-TBT(LF)(SN), J900136 BM03B-GHS-TBT(LF)(SN), J900138 BM03B-GHS-TBT(LF)(SN), J900140 BM03B-GHS-TBT(LF)(SN), J900142 BM03B-GHS-TBT(LF)(SN), J900144 BM03B-GHS-TBT(LF)(SN), J900146 BM03B-GHS-TBT(LF)(SN), J900148 BM03B-GHS-TBT(LF)(SN), J900150 BM03B-GHS-TBT(LF)(SN), J900152 BM03B-GHS-TBT(LF)(SN), J900154 BM03B-GHS-TBT(LF)(SN), J900156 BM03B-GHS-TBT(LF)(SN), J900158 BM03B-GHS-TBT(LF)(SN), J900160 BM03B-GHS-TBT(LF)(SN), J900162 BM03B-GHS-TBT(LF)(SN), J900164 BM03B-GHS-TBT(LF)(SN), J900166 BM03B-GHS-TBT(LF)(SN), J900168 BM03B-GHS-TBT(LF)(SN), J900170 BM03B-GHS-TBT(LF)(SN), J900172 BM03B-GHS-TBT(LF)(SN), J900174 BM03B-GHS-TBT(LF)(SN), J900176 BM03B-GHS-TBT(LF)(SN), J900178 BM03B-GHS-TBT(LF)(SN), J900180 BM03B-GHS-TBT(LF)(SN), J900182 BM03B-GHS-TBT(LF)(SN), J900184 BM03B-GHS-TBT(LF)(SN), J900186 BM03B-GHS-TBT(LF)(SN), J900188 BM03B-GHS-TBT(LF)(SN), J900190 BM03B-GHS-TBT(LF)(SN), J900192 BM03B-GHS-TBT(LF)(SN), J900194 BM03B-GHS-TBT(LF)(SN), J900196 BM03B-GHS-TBT(LF)(SN), J900198 BM03B-GHS-TBT(LF)(SN), J900200 BM03B-GHS-TBT(LF)(SN), J900202 BM03B-GHS-TBT(LF)(SN), J900204 BM03B-GHS-TBT(LF)(SN), J900206 BM03B-GHS-TBT(LF)(SN), J900208 BM03B-GHS-TBT(LF)(SN), J900210 BM03B-GHS-TBT(LF)(SN), J900212 BM03B-GHS-TBT(LF)(SN), J900214 BM03B-GHS-TBT(LF)(SN), J900216 BM03B-GHS-TBT(LF)(SN), J900218 BM03B-GHS-TBT(LF)(SN), J900220 BM03B-GHS-TBT(LF)(SN), J900222 BM03B-GHS-TBT(LF)(SN), J900224 BM03B-GHS-TBT(LF)(SN), J900226 BM03B-GHS-TBT(LF)(SN), J900228 BM03B-GHS-TBT(LF)(SN), J900230 BM03B-GHS-TBT(LF)(SN), J900232 BM03B-GHS-TBT(LF)(SN), J900234 BM03B-GHS-TBT(LF)(SN), J900236 BM03B-GHS-TBT(LF)(SN), J900238 BM03B-GHS-TBT(LF)(SN), J900240 BM03B-GHS-TBT(LF)(SN), J900242 BM03B-GHS-TBT(LF)(SN), J900244 BM03B-GHS-TBT(LF)(SN), J900246 BM03B-GHS-TBT(LF)(SN), J900248 BM03B-GHS-TBT(LF)(SN), J900250 BM03B-GHS-TBT(LF)(SN), J900252 BM03B-GHS-TBT(LF)(SN), J900254 BM03B-GHS-TBT(LF)(SN), J900256 BM03B-GHS-TBT(LF)(SN), J900258 BM03B-GHS-TBT(LF)(SN), J900260 BM03B-GHS-TBT(LF)(SN), J900262 BM03B-GHS-TBT(LF)(SN), J900264 BM03B-GHS-TBT(LF)(SN), J900266 BM03B-GHS-TBT(LF)(SN), J900268 BM03B-GHS-TBT(LF)(SN), J900270 BM03B-GHS-TBT(LF)(SN), J900272 BM03B-GHS-TBT(LF)(SN), J900274 BM03B-GHS-TBT(LF)(SN), J900276 BM03B-GHS-TBT(LF)(SN), J900278 BM03B-GHS-TBT(LF)(SN), J900280 BM03B-GHS-TBT(LF)(SN), J900282 BM03B-GHS-TBT(LF)(SN), J900284 BM03B-GHS-TBT(LF)(SN)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

Commit message: Connect 23 local control paths and verify per-net refill stability
Routing:
- net X1897FA4CC6D2320FE9FC: track 0.00 -> 35.9 mm, vias 0 -> 3
- net XB6FA1BCBBFA3EEA95431: track 0.00 -> 19.3 mm, vias 0 -> 1
- net X98302BA4179BABC520A9: track 0.00 -> 16.6 mm, vias 0 -> 1
- net XA1D49D92DDF2AA0DEFCB: track 0.00 -> 14.3 mm, vias 0 -> 1
- net XF2827D8A0A013B839CAA: track 0.00 -> 14.0 mm
- net XED165ED96D75C15A85C4: track 0.00 -> 14.0 mm
- net XEA71DBF9A3F5D1DD1ED4: track 0.00 -> 14.0 mm
- net XC22E458B0CC1481C514F: track 0.00 -> 14.0 mm
- net XBB7C344851AF8D0601AC: track 0.00 -> 14.0 mm
- net XB26BE8615EDC7481E388: track 55.9 -> 69.9 mm
- net XAC9F56A148C41BDAFC02: track 0.00 -> 14.0 mm
- net XA82AFE6CDE755FEB4702: track 131.0 -> 145.0 mm
- net X9F47443B516E90FF872D: track 0.00 -> 14.0 mm
- net X89D5E3CA45DE92E8F54F: track 148.7 -> 162.7 mm
- net X69F956D2CD0D8F7D7812: track 0.00 -> 14.0 mm
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