File: boards/osc-stage-optical/sheets/envelope_E1_EL.kicad_sch (KiCad schematic)
At the start: 23 parts, among them Q4107 MMBT3904,215, Q4108 2N7002,215, Q4109 MMBT3904,215, Q4110 2N7002,215, U4142 OPA4196IDR

Commit message: Add placed and fully routed stage-optical PCB draft (#42)
- Add draft routing classes (signals 0.25 mm, rails/AGND 0.4 mm, 0.25 mm
  clearance) and F.Cu/B.Cu AGND pours for osc-stage-optical.
- Move free stage parts below the 11 mm passages: bottom-up packing,
  0.7 mm spacing, 1.5 mm around fixed LEDs, bypass capacitors nearest
  their amplifier. Fixed LEDs, passages and connectivity are unchanged.
- Extend the peripheral source epoch with an exact stage-optical layout
  transition proof (free-part origins/angles, regions, routing only).
- Sync representative multi-unit fields so schematic parity is clean.
- Strip the SES placement block before import, add --max-passes, and add
  a grid maze finishing pass (finish_routes.py) with bounded rip-up.
- Add a disposable native CI check and the verification page.

Native KiCad 10: 0 open edges, 0 DRC errors, 0 parity issues.
Unvalidated routed draft; no fabrication files.

Co-Authored-By: Claude Opus 5.5 <noreply@anthropic.com>
Parts:
- C4164: FootprintOriginMm 221.64,176.96 -> 223.71,263.89; KiCadOrientationDeg 0 -> 270
- C4165: FootprintOriginMm 221.64,191.96 -> 230.46,263.89; KiCadOrientationDeg 0 -> 270
- D4123: FootprintOriginMm 227.11,189.25 -> 225.11,245.25
- D4125: FootprintOriginMm 227.11,200.25 -> 226.61,231.25
- Q4107: FootprintOriginMm 226.43,177.81 -> 224.43,258.81
- Q4108: FootprintOriginMm 226.43,181.81 -> 229.18,258.81
- Q4109: FootprintOriginMm 226.43,185.81 -> 228.93,254.31
- Q4110: FootprintOriginMm 226.43,196.81 -> 221.93,249.31
- RB4116: FootprintOriginMm 226.14,202.91 -> 229.89,245.66
- RB4117: FootprintOriginMm 221.64,205.91 -> 229.89,242.91
- RB4118: FootprintOriginMm 226.14,209.91 -> 228.64,240.16
- RB4119: FootprintOriginMm 226.14,212.16 -> 221.64,236.16
- RB4120: FootprintOriginMm 226.14,214.41 -> 221.64,233.41
- RB4121: FootprintOriginMm 226.14,216.66 -> 225.64,228.16
- RB4122: FootprintOriginMm 221.64,219.91 -> 225.64,225.41
- RB4123: FootprintOriginMm 225.39,223.91 -> 221.64,220.41
- RB4124: FootprintOriginMm 225.39,226.16 -> 226.39,217.66
- RB4125: FootprintOriginMm 225.39,228.41 -> 220.91,263.39; KiCadOrientationDeg 0 -> 270
- RB4126: FootprintOriginMm 225.39,230.66 -> 230.41,250.14; KiCadOrientationDeg 0 -> 270
- RB4127: FootprintOriginMm 221.64,233.16 -> 230.41,236.89; KiCadOrientationDeg 0 -> 270
- U4142: FootprintOriginMm 225.7,269.95 -> 226.2,271.2
