File: boards/osc-stage-optical/sheets/envelope_E2_EL.kicad_sch (KiCad schematic)
At the start: 23 parts, among them Q4207 MMBT3904,215, Q4208 2N7002,215, Q4209 MMBT3904,215, Q4210 2N7002,215, U4242 OPA4196IDR

Commit message: Add placed and fully routed stage-optical PCB draft (#42)
- Add draft routing classes (signals 0.25 mm, rails/AGND 0.4 mm, 0.25 mm
  clearance) and F.Cu/B.Cu AGND pours for osc-stage-optical.
- Move free stage parts below the 11 mm passages: bottom-up packing,
  0.7 mm spacing, 1.5 mm around fixed LEDs, bypass capacitors nearest
  their amplifier. Fixed LEDs, passages and connectivity are unchanged.
- Extend the peripheral source epoch with an exact stage-optical layout
  transition proof (free-part origins/angles, regions, routing only).
- Sync representative multi-unit fields so schematic parity is clean.
- Strip the SES placement block before import, add --max-passes, and add
  a grid maze finishing pass (finish_routes.py) with bounded rip-up.
- Add a disposable native CI check and the verification page.

Native KiCad 10: 0 open edges, 0 DRC errors, 0 parity issues.
Unvalidated routed draft; no fabrication files.

Co-Authored-By: Claude Opus 5.5 <noreply@anthropic.com>
Parts:
- C4264: FootprintOriginMm 238.64,176.96 -> 240.71,263.89; KiCadOrientationDeg 0 -> 270
- C4265: FootprintOriginMm 238.64,191.96 -> 247.46,263.89; KiCadOrientationDeg 0 -> 270
- D4223: FootprintOriginMm 244.11,189.25 -> 242.11,245.25
- D4225: FootprintOriginMm 244.11,200.25 -> 243.61,231.25
- Q4207: FootprintOriginMm 243.43,177.81 -> 241.43,258.81
- Q4208: FootprintOriginMm 243.43,181.81 -> 246.18,258.81
- Q4209: FootprintOriginMm 243.43,185.81 -> 245.93,254.31
- Q4210: FootprintOriginMm 243.43,196.81 -> 238.93,249.31
- RB4216: FootprintOriginMm 243.14,202.91 -> 246.89,245.66
- RB4217: FootprintOriginMm 238.64,205.91 -> 246.89,242.91
- RB4218: FootprintOriginMm 243.14,209.91 -> 245.64,240.16
- RB4219: FootprintOriginMm 243.14,212.16 -> 238.64,236.16
- RB4220: FootprintOriginMm 243.14,214.41 -> 238.64,233.41
- RB4221: FootprintOriginMm 243.14,216.66 -> 242.64,228.16
- RB4222: FootprintOriginMm 238.64,219.91 -> 242.64,225.41
- RB4223: FootprintOriginMm 242.39,223.91 -> 238.64,220.41
- RB4224: FootprintOriginMm 242.39,226.16 -> 243.39,217.66
- RB4225: FootprintOriginMm 242.39,228.41 -> 237.91,263.39; KiCadOrientationDeg 0 -> 270
- RB4226: FootprintOriginMm 242.39,230.66 -> 247.41,250.14; KiCadOrientationDeg 0 -> 270
- RB4227: FootprintOriginMm 238.64,233.16 -> 247.41,236.89; KiCadOrientationDeg 0 -> 270
- U4242: FootprintOriginMm 242.7,269.95 -> 243.2,271.2
