File: boards/osc-stage-optical/sheets/envelope_E4_EL.kicad_sch (KiCad schematic)
At the start: 23 parts, among them Q4407 MMBT3904,215, Q4408 2N7002,215, Q4409 MMBT3904,215, Q4410 2N7002,215, U4442 OPA4196IDR

Commit message: Add placed and fully routed stage-optical PCB draft (#42)
- Add draft routing classes (signals 0.25 mm, rails/AGND 0.4 mm, 0.25 mm
  clearance) and F.Cu/B.Cu AGND pours for osc-stage-optical.
- Move free stage parts below the 11 mm passages: bottom-up packing,
  0.7 mm spacing, 1.5 mm around fixed LEDs, bypass capacitors nearest
  their amplifier. Fixed LEDs, passages and connectivity are unchanged.
- Extend the peripheral source epoch with an exact stage-optical layout
  transition proof (free-part origins/angles, regions, routing only).
- Sync representative multi-unit fields so schematic parity is clean.
- Strip the SES placement block before import, add --max-passes, and add
  a grid maze finishing pass (finish_routes.py) with bounded rip-up.
- Add a disposable native CI check and the verification page.

Native KiCad 10: 0 open edges, 0 DRC errors, 0 parity issues.
Unvalidated routed draft; no fabrication files.

Co-Authored-By: Claude Opus 5.5 <noreply@anthropic.com>
Parts:
- C4464: FootprintOriginMm 272.64,176.96 -> 274.71,263.89; KiCadOrientationDeg 0 -> 270
- C4465: FootprintOriginMm 272.64,191.96 -> 281.46,263.89; KiCadOrientationDeg 0 -> 270
- D4423: FootprintOriginMm 278.11,189.25 -> 276.11,245.25
- D4425: FootprintOriginMm 278.11,200.25 -> 277.61,231.25
- Q4407: FootprintOriginMm 277.43,177.81 -> 275.43,258.81
- Q4408: FootprintOriginMm 277.43,181.81 -> 280.18,258.81
- Q4409: FootprintOriginMm 277.43,185.81 -> 279.93,254.31
- Q4410: FootprintOriginMm 277.43,196.81 -> 272.93,249.31
- RB4416: FootprintOriginMm 277.14,202.91 -> 280.89,245.66
- RB4417: FootprintOriginMm 272.64,205.91 -> 280.89,242.91
- RB4418: FootprintOriginMm 277.14,209.91 -> 279.64,240.16
- RB4419: FootprintOriginMm 277.14,212.16 -> 272.64,236.16
- RB4420: FootprintOriginMm 277.14,214.41 -> 272.64,233.41
- RB4421: FootprintOriginMm 277.14,216.66 -> 276.64,228.16
- RB4422: FootprintOriginMm 272.64,219.91 -> 276.64,225.41
- RB4423: FootprintOriginMm 276.39,223.91 -> 272.64,220.41
- RB4424: FootprintOriginMm 276.39,226.16 -> 277.39,217.66
- RB4425: FootprintOriginMm 276.39,228.41 -> 271.91,263.39; KiCadOrientationDeg 0 -> 270
- RB4426: FootprintOriginMm 276.39,230.66 -> 281.41,250.14; KiCadOrientationDeg 0 -> 270
- RB4427: FootprintOriginMm 272.64,233.16 -> 281.41,236.89; KiCadOrientationDeg 0 -> 270
- U4442: FootprintOriginMm 276.7,269.95 -> 277.2,271.2
