File: boards/osc-stage-optical/sheets/envelope_E6_EL.kicad_sch (KiCad schematic)
At the start: 23 parts, among them Q4607 MMBT3904,215, Q4608 2N7002,215, Q4609 MMBT3904,215, Q4610 2N7002,215, U4642 OPA4196IDR

Commit message: Add placed and fully routed stage-optical PCB draft (#42)
- Add draft routing classes (signals 0.25 mm, rails/AGND 0.4 mm, 0.25 mm
  clearance) and F.Cu/B.Cu AGND pours for osc-stage-optical.
- Move free stage parts below the 11 mm passages: bottom-up packing,
  0.7 mm spacing, 1.5 mm around fixed LEDs, bypass capacitors nearest
  their amplifier. Fixed LEDs, passages and connectivity are unchanged.
- Extend the peripheral source epoch with an exact stage-optical layout
  transition proof (free-part origins/angles, regions, routing only).
- Sync representative multi-unit fields so schematic parity is clean.
- Strip the SES placement block before import, add --max-passes, and add
  a grid maze finishing pass (finish_routes.py) with bounded rip-up.
- Add a disposable native CI check and the verification page.

Native KiCad 10: 0 open edges, 0 DRC errors, 0 parity issues.
Unvalidated routed draft; no fabrication files.

Co-Authored-By: Claude Opus 5.5 <noreply@anthropic.com>
Parts:
- C4664: FootprintOriginMm 306.64,176.96 -> 311.14,264.46
- C4665: FootprintOriginMm 306.64,191.96 -> 314.46,263.89; KiCadOrientationDeg 0 -> 270
- D4623: FootprintOriginMm 312.11,193.25 -> 307.61,246.75
- D4625: FootprintOriginMm 312.11,196.25 -> 313.36,246.75
- Q4607: FootprintOriginMm 311.43,177.81 -> 306.93,260.81
- Q4608: FootprintOriginMm 311.43,181.81 -> 311.68,259.56
- Q4609: FootprintOriginMm 311.43,185.81 -> 313.93,255.06
- Q4610: FootprintOriginMm 311.43,189.81 -> 309.43,250.56
- RB4616: FootprintOriginMm 311.14,198.91 -> 313.89,251.41
- RB4617: FootprintOriginMm 314.89,198.91 -> 313.64,243.66
- RB4618: FootprintOriginMm 311.14,201.16 -> 313.64,240.91
- RB4619: FootprintOriginMm 314.89,201.16 -> 313.64,238.16
- RB4620: FootprintOriginMm 311.14,203.41 -> 309.14,237.66
- RB4621: FootprintOriginMm 314.89,203.41 -> 313.14,235.41
- RB4622: FootprintOriginMm 311.14,205.66 -> 306.64,234.91
- RB4623: FootprintOriginMm 314.89,205.66 -> 310.64,232.66
- RB4624: FootprintOriginMm 306.64,205.91 -> 314.64,232.66
- RB4625: FootprintOriginMm 311.14,207.91 -> 310.64,229.91
- RB4626: FootprintOriginMm 314.89,207.91 -> 314.64,229.91
- RB4627: FootprintOriginMm 311.14,210.16 -> 310.64,227.16
- U4642: FootprintOriginMm 312.45,223.95 -> 311.2,271.2
